Commit message: add changingtek gripper

File: gripper/changingtek_description/xacro/ros2_control/2f.ros2_control.xacro (robot description, xacro)
@@ -1,14 +1,14 @@
 <?xml version="1.0"?>
 <robot xmlns:xacro="http://www.ros.org/wiki/xacro">
-  <xacro:macro name="robotiq85_system" params="name ros2_control_hardware_type">
+  <xacro:macro name="changingtek_2f_system" params="name hardware">
     <ros2_control name="${name}" type="system">
       <hardware>
-        <xacro:if value="${ros2_control_hardware_type == 'gz'}">
+        <xacro:if value="${hardware == 'gz'}">
           <plugin>gz_ros2_control/GazeboSimSystem</plugin>
         </xacro:if>
-        <xacro:if value="${ros2_control_hardware_type == 'mock_components'}">
+        <xacro:if value="${hardware == 'mock_components'}">
           <plugin>mock_components/GenericSystem</plugin>
         </xacro:if>
-        <xacro:if value="${ros2_control_hardware_type == 'isaac'}">
+        <xacro:if value="${hardware == 'isaac'}">
           <plugin>topic_based_ros2_control/TopicBasedSystem</plugin>
           <param name="joint_commands_topic">/isaac/joint_command</param>
@@ -16,6 +16,5 @@
         </xacro:if>
       </hardware>
-      <!-- 关节接口定义 -->
-      <joint name="finger_joint">
+      <joint name="gripper_joint">
         <command_interface name="position"/>
         <state_interface name="position">

File: gripper/robotiq_description/xacro/2F85.xacro (robot description, xacro)
@@ -3,5 +3,5 @@
   <xacro:macro name="Robotiq85" params="name">
     <xacro:property name="prefix" value="${name + '_' if name else ''}"/>
-    <link name="${prefix}base_link">
+    <link name="${prefix}gripper_base">
       <inertial>
         <origin xyz="8.625E-08 -4.6583E-06 0.03145"/>
@@ -24,5 +24,5 @@
       </collision>
     </link>
-    <link name="left_outer_knuckle">
+    <link name="${prefix}left_outer_knuckle">
       <inertial>
         <origin xyz="-0.000200000000003065 0.0199435877845359 0.0292245259211331"/>
@@ -42,5 +42,5 @@
       </collision>
     </link>
-    <link name="left_outer_finger">
+    <link name="${prefix}left_outer_finger">
       <inertial>
         <origin xyz="0.00030115855001899 0.0373907951953854 -0.0208027427000385"/>
@@ -60,5 +60,5 @@
       </collision>
     </link>
-    <link name="left_inner_finger">
+    <link name="${prefix}left_inner_finger">
       <inertial>
         <origin xyz="0.000299999999999317 0.0160078233491243 -0.0136945669206257"/>
@@ -78,5 +78,5 @@
       </collision>
     </link>
-    <link name="left_inner_finger_pad">
+    <link name="${prefix}left_inner_finger_pad">
       <visual>
         <geometry>
@@ -93,5 +93,5 @@
       </collision>
     </link>
-    <link name="left_inner_knuckle">
+    <link name="${prefix}left_inner_knuckle">
       <inertial>
         <origin xyz="0.000123011831763771 0.0507850843201817 0.00103968640075166"/>
@@ -111,5 +111,5 @@
       </collision>
     </link>
-    <link name="right_outer_knuckle">
+    <link name="${prefix}right_outer_knuckle">
       <inertial>
         <origin xyz="-0.000200000000003065 0.0199435877845359 0.0292245259211331"/>
@@ -129,5 +129,5 @@
       </collision>
     </link>
-    <link name="right_outer_finger">
+    <link name="${prefix}right_outer_finger">
       <inertial>
         <origin xyz="0.00030115855001899 0.0373907951953854 -0.0208027427000385"/>
@@ -147,5 +147,5 @@
       </collision>
     </link>
-    <link name="right_inner_finger">
+    <link name="${prefix}right_inner_finger">
       <inertial>
         <origin xyz="0.000299999999999317 0.0160078233491243 -0.0136945669206257"/>
@@ -165,5 +165,5 @@
       </collision>
     </link>
-    <link name="right_inner_finger_pad">
+    <link name="${prefix}right_inner_finger_pad">
       <visual>
         <geometry>
@@ -180,5 +180,5 @@
       </collision>
     </link>
-    <link name="right_inner_knuckle">
+    <link name="${prefix}right_inner_knuckle">
       <inertial>
         <origin xyz="0.000123011831763771 0.0507850843201817 0.00103968640075166"/>
@@ -199,77 +199,75 @@
     </link>
     <!-- Main actuated joint - left outer knuckle -->
-    <joint name="finger_joint" type="revolute">
+    <joint name="${prefix}gripper_joint" type="revolute">
       <origin rpy="0 0 3.14159265359" xyz="0 -0.0306011 0.054904"/>
-      <parent link="${prefix}base_link"/>
-      <child link="left_outer_knuckle"/>
+      <parent link="${prefix}gripper_base"/>
+      <child link="${prefix}left_outer_knuckle"/>
       <axis xyz="1 0 0"/>
       <limit effort="1000" lower="0" upper="0.81" velocity="2.0"/>
     </joint>
-    <joint name="left_outer_finger_joint" type="fixed">
+    <joint name="${prefix}left_outer_finger_joint" type="fixed">
       <origin xyz="0 0.0315 -0.0041"/>
-      <parent link="left_outer_knuckle"/>
-      <child link="left_outer_finger"/>
+      <parent link="${prefix}left_outer_knuckle"/>
+      <child link="${prefix}left_outer_finger"/>
       <axis xyz="1 0 0"/>
     </joint>
     <!-- Left inner knuckle mimics the outer knuckle with a mechanical coupling -->
-    <joint name="left_inner_knuckle_joint" type="revolute">
+    <joint name="${prefix}left_inner_knuckle_joint" type="revolute">
       <origin rpy="0 0 3.14159265359" xyz="0 -0.0127 0.06142"/>
-      <parent link="${prefix}base_link"/>
-      <child link="left_inner_knuckle"/>
+      <parent link="${prefix}gripper_base"/>
+      <child link="${prefix}left_inner_knuckle"/>
       <axis xyz="1 0 0"/>
       <limit effort="1000" lower="0" upper="0.8757" velocity="2.0"/>
-      <mimic joint="finger_joint" multiplier="1" offset="0"/>
+      <mimic joint="${prefix}gripper_joint" multiplier="1" offset="0"/>
     </joint>
     <!-- Left inner finger has opposite motion to simulate the mechanical linkage -->
-    <joint name="left_inner_finger_joint" type="revolute">
+    <joint name="${prefix}left_inner_finger_joint" type="revolute">
       <origin xyz="0 0.0061 0.0471"/>
-      <parent link="left_outer_finger"/>
-      <child link="left_inner_finger"/>
+      <parent link="${prefix}left_outer_finger"/>
+      <child link="${prefix}left_inner_finger"/>
       <axis xyz="1 0 0"/>
       <limit effort="1000" lower="-0.8757" upper="0" velocity="2.0"/>
-      <mimic joint="finger_joint" multiplier="-1" offset="0"/>
-    </joint>
-    <joint name="left_inner_finger_pad_joint" type="fixed">
+      <mimic joint="${prefix}gripper_joint" multiplier="-1" offset="0"/>
+    </joint>
+    <joint name="${prefix}left_inner_finger_pad_joint" type="fixed">
       <origin xyz="0 -0.0220203446692936 0.03242"/>
-      <parent link="left_inner_finger"/>
-      <child link="left_inner_finger_pad"/>
+      <parent link="${prefix}left_inner_finger"/>
+      <child link="${prefix}left_inner_finger_pad"/>
       <axis xyz="0 0 1"/>
     </joint>
     <!-- Right side joints mimic the left side with opposite motion -->
-    <joint name="right_outer_knuckle_joint" type="revolute">
+    <joint name="${prefix}right_outer_knuckle_joint" type="revolute">
       <origin xyz="0 0.0306011 0.054904"/>
-      <parent link="${prefix}base_link"/>
-      <child link="right_outer_knuckle"/>
+      <parent link="${prefix}gripper_base"/>
+      <child link="${prefix}right_outer_knuckle"/>
       <axis xyz="1 0 0"/>
       <limit effort="1000" lower="0" upper="0.81" velocity="2.0"/>
-      <mimic joint="finger_joint" multiplier="1" offset="0"/>
-    </joint>
-    <joint name="right_outer_finger_joint" type="fixed">
+      <mimic joint="${prefix}gripper_joint" multiplier="1" offset="0"/>
+    </joint>
+    <joint name="${prefix}right_outer_finger_joint" type="fixed">
       <origin xyz="0 0.0315 -0.0041"/>
-      <parent link="right_outer_knuckle"/>
-      <child link="right_outer_finger"/>
-      <axis xyz="1 0 0"/>
-    </joint>
-    <joint name="right_inner_knuckle_joint" type="revolute">
+      <parent link="${prefix}right_outer_knuckle"/>
+      <child link="${prefix}right_outer_finger"/>
+    </joint>
+    <joint name="${prefix}right_inner_knuckle_joint" type="revolute">
       <origin rpy="0 0 0.0" xyz="0 0.0127 0.06142"/>
-      <parent link="${prefix}base_link"/>
-      <child link="right_inner_knuckle"/>
+      <parent link="${prefix}gripper_base"/>
+      <child link="${prefix}right_inner_knuckle"/>
       <axis xyz="1 0 0"/>
       <limit effort="1000" lower="0" upper="0.8757" velocity="2.0"/>
-      <mimic joint="finger_joint" multiplier="1" offset="0"/>
-    </joint>
-    <joint name="right_inner_finger_joint" type="revolute">
+      <mimic joint="${prefix}gripper_joint" multiplier="1" offset="0"/>
+    </joint>
+    <joint name="${prefix}right_inner_finger_joint" type="revolute">
       <origin xyz="0 0.0061 0.0471"/>
-      <parent link="right_outer_finger"/>
-      <child link="right_inner_finger"/>
+      <parent link="${prefix}right_outer_finger"/>
+      <child link="${prefix}right_inner_finger"/>
       <axis xyz="1 0 0"/>
       <limit effort="1000" lower="-0.8757" upper="0" velocity="2.0"/>
-      <mimic joint="finger_joint" multiplier="-1" offset="0"/>
-    </joint>
-    <joint name="right_inner_finger_pad_joint" type="fixed">
+      <mimic joint="${prefix}gripper_joint" multiplier="-1" offset="0"/>
+    </joint>
+    <joint name="${prefix}right_inner_finger_pad_joint" type="fixed">
       <origin xyz="0 -0.0220203446692936 0.03242"/>
-      <parent link="right_inner_finger"/>
-      <child link="right_inner_finger_pad"/>
-      <axis xyz="0 0 1"/>
+      <parent link="${prefix}right_inner_finger"/>
+      <child link="${prefix}right_inner_finger_pad"/>
     </joint>
   </xacro:macro>

File: gripper/robotiq_description/xacro/gripper.xacro (robot description, xacro)
@@ -1,8 +1,8 @@
 <?xml version="1.0"?>
-<robot name="Robotiq85" xmlns:xacro="http://www.ros.org/wiki/xacro">
+<robot name="Robotiq_$(arg type)" xmlns:xacro="http://www.ros.org/wiki/xacro">
   <xacro:arg name="type" default="85"/>
   <!-- 根据type参数决定使用哪种夹爪 -->
   <xacro:if value="${'$(arg type)' == '85'}">
-    <xacro:include filename="$(find robotiq_description)/xacro/robotiq85.xacro"/>
+    <xacro:include filename="$(find robotiq_description)/xacro/2F85.xacro"/>
     <xacro:Robotiq85 name=""/>
   </xacro:if>

File: manipulator/Dobot/cr5_description/xacro/robot.xacro (robot description, xacro)
@@ -5,12 +5,18 @@
   <xacro:include filename="$(find cr5_description)/xacro/arm.xacro"/>
   <xacro:CR5 name="" collider="$(arg collider)"/>
+  <xacro:if value="${'$(arg type)' != 'empty'}">
+    <joint name="gripper_fix" type="fixed">
+      <parent link="Link6"/>
+      <child link="gripper_base"/>
+    </joint>
+  </xacro:if>
   <!-- 根据type参数决定使用哪种夹爪 -->
   <xacro:if value="${'$(arg type)' == 'robotiq85'}">
-    <joint name="gripper_fix" type="fixed">
-      <parent link="Link6"/>
-      <child link="eef_base_link"/>
-    </joint>
     <xacro:include filename="$(find robotiq_description)/xacro/robotiq85.xacro"/>
-    <xacro:Robotiq85 name="eef"/>
+    <xacro:Robotiq85 name=""/>
+  </xacro:if>
+  <xacro:if value="${'$(arg type)' == 'AG2F90-C'}">
+    <xacro:include filename="$(find changingtek_description)/xacro/AG2F90-C.xacro"/>
+    <xacro:AG2F90-C name=""/>
   </xacro:if>
 </robot>

Commit message: cr5 ocs2 ros2 control

File: gripper/changingtek_description/xacro/ros2_control/2f.ros2_control.xacro (robot description, xacro)
@@ -14,4 +14,5 @@
           <param name="joint_commands_topic">/isaac/joint_command</param>
           <param name="joint_states_topic">/isaac/joint_states</param>
+          <param name="sum_wrapped_joint_states">true</param>
         </xacro:if>
       </hardware>

File: gripper/changingtek_description/xacro/ros2_control/gripper.xacro (robot description, xacro)
@@ -7,5 +7,5 @@
       <xacro:AG2F90-C name=""/>
       <xacro:include filename="$(find changingtek_description)/xacro/ros2_control/2f.ros2_control.xacro"/>
-      <xacro:changingtek_2f_system name="AG2F90-C_System" hardware="${hardware}"/>
+      <xacro:changingtek_2f_system name="AG2F90_C_System" hardware="${hardware}"/>
     </xacro:if>
     <xacro:if value="${type == 'AG2F120S'}">

File: manipulator/ARX/arx5_description/xacro/ros2_control/arx5.ros2_control.xacro (robot description, xacro)
@@ -59,12 +59,8 @@
         <state_interface name="effort"/>
       </joint>
-      <joint name="joint7">
+      <joint name="gripper_joint">
         <command_interface name="position"/>
-        <state_interface name="position">
-          <param name="initial_value">0.0</param>
-        </state_interface>
-        <state_interface name="velocity">
-          <param name="initial_value">0.0</param>
-        </state_interface>
+        <state_interface name="position"/>
+        <state_interface name="velocity"/>
       </joint>
     </ros2_control>

File: manipulator/Dobot/cr5_description/xacro/ros2_control/cr5.ros2_control.xacro (robot description, xacro)
@@ -14,4 +14,5 @@
           <param name="joint_commands_topic">/isaac/joint_command</param>
           <param name="joint_states_topic">/isaac/joint_states</param>
+          <param name="sum_wrapped_joint_states">true</param>
         </xacro:if>
       </hardware>

File: manipulator/Dobot/cr5_description/xacro/ros2_control/robot.xacro (robot description, xacro)
@@ -6,5 +6,5 @@
     <parent link="world"/>
     <child link="base_link"/>
-    <origin xyz="0.0 0.0 0.0" rpy="0 0 0"/>
+    <origin/>
   </joint>
   <xacro:include filename="$(find cr5_description)/xacro/arm.xacro"/>
