Commit message: agilex split aloha

File: manipulator/AgileX/agilex_aloha_description/xacro/aloha_split.xacro (robot description, xacro)
@@ -5,6 +5,6 @@
   <link name="box_link">
     <inertial>
-      <origin xyz="0.10921 -0.0087718 0.52779"  />
-      <mass value="27.261" />
+      <origin xyz="0.10921 -0.0087718 0.52779"/>
+      <mass value="27.261"/>
       <inertia
           ixx="1.8122"
@@ -13,5 +13,5 @@
           iyy="1.7779"
           iyz="-4.0693E-05"
-          izz="0.28053" />
+          izz="0.28053"/>
     </inertial>
     <visual>
@@ -27,11 +27,11 @@
   </link>
   <joint name="box_joint" type="fixed">
-    <parent link="base_link" />
-    <child link="box_link" />
+    <parent link="base_link"/>
+    <child link="box_link"/>
   </joint>
   <link name="front_camera_link">
     <inertial>
       <origin xyz="-0.011443 0.0003607 -0.0012124"/>
-      <mass value="0.020053" />
+      <mass value="0.020053"/>
       <inertia
           ixx="1.1182E-05"
@@ -40,9 +40,9 @@
           iyy="2.2729E-06"
           iyz="-6.7447E-07"
-          izz="1.0081E-05" />
+          izz="1.0081E-05"/>
     </inertial>
     <visual>
       <geometry>
-        <mesh filename="file://$(find agilex_aloha_description)/meshes/aloha_split/camera.obj" />
+        <mesh filename="file://$(find agilex_aloha_description)/meshes/aloha_split/camera.obj"/>
       </geometry>
     </visual>
@@ -54,12 +54,12 @@
   </link>
   <joint name="front_camera_joint" type="fixed">
-    <origin xyz="0.35679 0 0.15819" rpy="0 0.6606 -0.0051043" />
-    <parent link="box_link" />
-    <child link="front_camera_link" />
+    <origin xyz="0.35679 0 0.15819" rpy="0 0.6606 -0.0051043"/>
+    <parent link="box_link"/>
+    <child link="front_camera_link"/>
   </joint>
   <link name="lidar_link">
     <inertial>
       <origin xyz="-0.0022133 -0.00090659 0.025996"/>
-      <mass value="0.048617" />
+      <mass value="0.048617"/>
       <inertia
           ixx="1.0358E-05"
@@ -68,5 +68,5 @@
           iyy="1.0387E-05"
           iyz="-2.6377E-07"
-          izz="1.7919E-05" />
+          izz="1.7919E-05"/>
     </inertial>
     <visual>
@@ -82,12 +82,12 @@
   </link>
   <joint name="lidar_joint" type="fixed">
-    <origin xyz="0.31755 0 0.036188" rpy="-0.035132 0.20001 -0.001242" />
-    <parent link="box_link" />
-    <child link="lidar_link" />
+    <origin xyz="0.31755 0 0.036188" rpy="-0.035132 0.20001 -0.001242"/>
+    <parent link="box_link"/>
+    <child link="lidar_link"/>
   </joint>
   <link name="lifting_link">
     <inertial>
       <origin xyz="0.071327 0.00032985 0.10599"/>
-      <mass value="0.47066" />
+      <mass value="0.47066"/>
       <inertia
           ixx="0.010952"
@@ -96,5 +96,5 @@
           iyy="0.0018329"
           iyz="-4.6428E-06"
-          izz="0.010201" />
+          izz="0.010201"/>
     </inertial>
     <visual>
@@ -111,13 +111,13 @@
   <joint name="lifting_joint" type="prismatic">
     <origin xyz="0.22448 0 1.1147"/>
-    <parent link="box_link" />
-    <child link="lifting_link" />
-    <axis xyz="0 0 1" />
-    <limit lower="-0.6" upper="0.0" effort="100" velocity="10.0"/>
+    <parent link="box_link"/>
+    <child link="lifting_link"/>
+    <axis xyz="0 0 1"/>
+    <limit lower="-0.6" upper="0.0" effort="1000" velocity="10.0"/>
   </joint>
   <link name="top_camera_link">
     <inertial>
       <origin xyz="-0.011443 2.4833E-05 -0.0012615"/>
-      <mass value="0.020053" />
+      <mass value="0.020053"/>
       <inertia
           ixx="1.1181E-05"
@@ -126,5 +126,5 @@
           iyy="2.2587E-06"
           iyz="5.7637E-07"
-          izz="1.0097E-05" />
+          izz="1.0097E-05"/>
     </inertial>
     <visual>
@@ -140,7 +140,7 @@
   </link>
   <joint name="top_camera_joint" type="fixed">
-    <origin xyz="0.16194 0 0.29838" rpy="0 0.00080758 -0.01623" />
-    <parent link="lifting_link" />
-    <child link="top_camera_link" />
+    <origin xyz="0.16194 0 0.29838" rpy="0 0.00080758 -0.01623"/>
+    <parent link="lifting_link"/>
+    <child link="top_camera_link"/>
   </joint>
   <link name="top_camera_support">
@@ -152,11 +152,11 @@
   </link>
   <joint name="top_camera_support_joint" type="fixed">
-    <origin xyz="0.16194 0 0.29838" rpy="0 0.00080758 -0.01623" />
-    <parent link="lifting_link" />
-    <child link="top_camera_support" />
+    <origin xyz="0.16194 0 0.29838" rpy="0 0.00080758 -0.01623"/>
+    <parent link="lifting_link"/>
+    <child link="top_camera_support"/>
   </joint>
   <xacro:Piper name="left"/>
   <joint name="arm_and_lifting_left" type="fixed">
-    <origin xyz="0.144 0.306 0.138" rpy="0.0 0.0 0.0"/>
+    <origin xyz="0.144 0.306 0.138"/>
     <parent link="lifting_link"/>
     <child link="left_base_link"/>
@@ -166,5 +166,5 @@
   <xacro:Piper name="right"/>
   <joint name="arm_and_lifting_right" type="fixed">
-    <origin xyz="0.144 -0.306 0.138" rpy="0.0 0.0 0.0"/>
+    <origin xyz="0.144 -0.306 0.138"/>
     <parent link="lifting_link"/>
     <child link="right_base_link"/>
