Commit message: fix cobot magic planning urdf

File: manipulator/AgileX/agilex_aloha_description/xacro/component.xacro (robot description, xacro)
@@ -15,10 +15,4 @@
 		<xacro:include filename="$(find agilex_aloha_description)/xacro/base/tracer_v2.xacro"/>
 	</xacro:if>
-	<xacro:if value="${'$(arg type)' == 'body_v1'}">
-		<link name="base_footprint"/>
-		<link name="left_base_link"/>
-		<link name="right_base_link"/>
-		<xacro:include filename="$(find agilex_aloha_description)/xacro/body/v1.xacro"/>
-	</xacro:if>
 	<xacro:if value="${'$(arg type)' == 'body_v2'}">
 		<link name="base_footprint"/>

File: manipulator/AgileX/agilex_aloha_description/xacro/robot.xacro (robot description, xacro)
@@ -5,12 +5,4 @@
   <xacro:if value="${'$(arg type)' == 'split'}">
     <xacro:include filename="$(find agilex_aloha_description)/xacro/aloha_split.xacro"/>
-  </xacro:if>
-  <xacro:if value="${'$(arg type)' == 'v1'}">
-    <xacro:include filename="$(find agilex_aloha_description)/xacro/aloha_v1.xacro"/>
-    <xacro:aloha_v1/>
-  </xacro:if>
-  <xacro:if value="${'$(arg type)' == 'v1_x5'}">
-    <xacro:include filename="$(find agilex_aloha_description)/xacro/aloha_v1.xacro"/>
-    <xacro:aloha_v1 arm="x5"/>
   </xacro:if>
   <xacro:if value="${'$(arg type)' == 'v2'}">
