Commit message: add agilex split aloha

File: manipulator/AgileX/agilex_aloha_description/xacro/aloha_v2.xacro (robot description, xacro)
@@ -3,4 +3,5 @@
 	<xacro:macro name="aloha_v2" params="chassis:=tracer enable_master:=false">
 		<xacro:include filename="$(find piper_description)/xacro/Piper.xacro"/>
+		<xacro:include filename="$(find piper_description)/xacro/eefs.xacro"/>
 		<xacro:include filename="$(find agilex_aloha_description)/xacro/body/v2.xacro"/>
 		<xacro:if value="${chassis == 'tracer'}">
@@ -11,8 +12,11 @@
 		</xacro:if>
 		<xacro:Piper name="left"/>
+		<xacro:PiperEndEffectors name="left" type="gripper" camera_type="true" arms="piper"/>
 		<xacro:Piper name="right"/>
+		<xacro:PiperEndEffectors name="right" type="gripper" camera_type="true" arms="piper"/>
 		<!--***************************** back-left ****************************** -->
 		<xacro:if value="${enable_master}">
-			<xacro:Piper name="bl" is_master="true"/>
+			<xacro:Piper name="bl"/>
+			<xacro:PiperEndEffectors name="bl" type="gripper" camera_type="false" arms="piper"/>
 			<joint name="bl_base_joint" type="fixed">
 				<origin xyz="-0.379 0.3075 0.733"/>
@@ -24,5 +28,6 @@
 		<!--***************************** back-right ****************************** -->
 		<xacro:if value="${enable_master}">
-			<xacro:Piper name="br" is_master="true"/>
+			<xacro:Piper name="br"/>
+			<xacro:PiperEndEffectors name="br" type="gripper" camera_type="false" arms="piper"/>
 			<joint name="br_base_joint" type="fixed">
 				<origin xyz="-0.379 -0.3075 0.733"/>

File: manipulator/AgileX/agilex_aloha_description/xacro/component.xacro (robot description, xacro)
@@ -4,9 +4,6 @@
 <!-- |    This file includes the base robot structure and both arms                    | -->
 <!-- =================================================================================== -->
-<robot name="Agilex_Aloha_Spilt" xmlns:xacro="http://www.ros.org/wiki/xacro">
-	<xacro:arg name="type" default="ranger_mini"/>
-	<xacro:if value="${'$(arg type)' == 'ranger_mini'}">
-		<xacro:include filename="$(find agilex_aloha_description)/xacro/base/ranger_mini.xacro"/>
-	</xacro:if>
+<robot name="Agilex_Aloha" xmlns:xacro="http://www.ros.org/wiki/xacro">
+	<xacro:arg name="type" default="tracer"/>
 	<xacro:if value="${'$(arg type)' == 'tracer'}">
 		<xacro:include filename="$(find agilex_aloha_description)/xacro/base/tracer.xacro"/>
@@ -21,9 +18,3 @@
 		<xacro:include filename="$(find agilex_aloha_description)/xacro/body/v2.xacro"/>
 	</xacro:if>
-	<xacro:if value="${'$(arg type)' == 'body_split'}">
-		<link name="base"/>
-		<link name="left_base_link"/>
-		<link name="right_base_link"/>
-		<xacro:include filename="$(find agilex_aloha_description)/xacro/body/split.xacro"/>
-	</xacro:if>
 </robot>

File: manipulator/AgileX/agilex_aloha_description/xacro/robot.xacro (robot description, xacro)
@@ -1,9 +1,6 @@
 <?xml version="1.0"?>
 <robot name="AgileX Aloha" xmlns:xacro="http://www.ros.org/wiki/xacro">
-  <xacro:arg name="type" default="split"/>
+  <xacro:arg name="type" default="v2"/>
   <!-- 根据type参数决定机器人类型 -->
-  <xacro:if value="${'$(arg type)' == 'split'}">
-    <xacro:include filename="$(find agilex_aloha_description)/xacro/aloha_split.xacro"/>
-  </xacro:if>
   <xacro:if value="${'$(arg type)' == 'v2'}">
     <xacro:include filename="$(find agilex_aloha_description)/xacro/aloha_v2.xacro"/>

File: manipulator/AgileX/agilex_aloha_description/xacro/ros2_control/robot.xacro (robot description, xacro)
@@ -2,16 +2,16 @@
 <robot xmlns:xacro="http://www.ros.org/wiki/xacro" name="AgileX Aloha">
   <xacro:arg name="ros2_control_hardware_type" default="mock_components" />
-  <!-- Import Piper ros2_control description -->
-  <xacro:include filename="$(find piper_description)/xacro/ros2_control/piper.ros2_control.xacro" />
-  <xacro:arg name="type" default="split"/>
-  <xacro:if value="${'$(arg type)' == 'split'}">
-    <xacro:include filename="$(find agilex_aloha_description)/xacro/aloha_split.xacro"/>
-    <xacro:include filename="$(find agilex_aloha_description)/xacro/ros2_control/aloha_split.ros2_control.xacro" />
-    <xacro:aloha_split_system ros2_control_hardware_type="$(arg ros2_control_hardware_type)"/>
-    <xacro:piper_system name="left" ros2_control_hardware_type="$(arg ros2_control_hardware_type)"/>
-    <xacro:piper_system name="right" ros2_control_hardware_type="$(arg ros2_control_hardware_type)"/>
-  </xacro:if>
+  <xacro:arg name="type" default="v2"/>
   <xacro:if value="${'$(arg type)' == 'v2'}">
     <xacro:include filename="$(find agilex_aloha_description)/xacro/aloha_v2.xacro"/>
+    <xacro:aloha_v2/>
+  </xacro:if>
+  <xacro:if value="${'$(arg type)' == 'v2-1'}">
+    <xacro:include filename="$(find agilex_aloha_description)/xacro/aloha_v2.xacro"/>
+    <xacro:aloha_v2 chassis="tracer_v2"/>
+  </xacro:if>
+  <xacro:if value="${'$(arg type)' == 'v2-master'}">
+    <xacro:include filename="$(find agilex_aloha_description)/xacro/aloha_v2.xacro"/>
+    <xacro:aloha_v2 chassis="tracer_v2" enable_master="true"/>
   </xacro:if>
   <xacro:arg name="gazebo" default="false" />

File: manipulator/AgileX/piper_description/xacro/Piper.xacro (robot description, xacro)
@@ -1,12 +1,6 @@
 <?xml version="1.0" encoding="utf-8"?>
 <robot xmlns:xacro="http://www.ros.org/wiki/xacro">
-  <xacro:macro name="Piper" params="name is_master:=false">
+  <xacro:macro name="Piper" params="name">
     <xacro:property name="prefix" value="${name + '_' if name else ''}"/>
-    <xacro:if value="${is_master}">
-      <xacro:include filename="$(find piper_description)/xacro/master.xacro"/>
-    </xacro:if>
-    <xacro:unless value="${is_master}">
-      <xacro:include filename="$(find piper_description)/xacro/slave.xacro"/>
-    </xacro:unless>
     <link name="${prefix}base_link">
       <inertial>
@@ -23,5 +17,5 @@
       <collision>
         <geometry>
-          <mesh filename="file://$(find piper_description)/meshes/collision/base_link.obj"/>
+          <mesh filename="file://$(find piper_description)/meshes/visual/base_link.glb"/>
         </geometry>
       </collision>
@@ -41,5 +35,5 @@
       <collision>
         <geometry>
-          <mesh filename="file://$(find piper_description)/meshes/collision/link1.obj"/>
+          <mesh filename="file://$(find piper_description)/meshes/visual/link1.glb"/>
         </geometry>
       </collision>
@@ -66,5 +60,5 @@
       <collision>
         <geometry>
-          <mesh filename="file://$(find piper_description)/meshes/collision/link2.obj"/>
+          <mesh filename="file://$(find piper_description)/meshes/visual/link2.glb"/>
         </geometry>
       </collision>
@@ -86,10 +80,10 @@
       <visual>
         <geometry>
-          <mesh filename="file://$(find piper_description)/meshes/visual/link3.obj"/>
+          <mesh filename="file://$(find piper_description)/meshes/visual/link3.glb"/>
         </geometry>
       </visual>
       <collision>
         <geometry>
-          <mesh filename="file://$(find piper_description)/meshes/collision/link3.obj"/>
+          <mesh filename="file://$(find piper_description)/meshes/visual/link3.glb"/>
         </geometry>
       </collision>
@@ -111,10 +105,10 @@
       <visual>
         <geometry>
-          <mesh filename="file://$(find piper_description)/meshes/visual/link4.obj"/>
+          <mesh filename="file://$(find piper_description)/meshes/visual/link4.glb"/>
         </geometry>
       </visual>
       <collision>
         <geometry>
-          <mesh filename="file://$(find piper_description)/meshes/collision/link4.obj"/>
+          <mesh filename="file://$(find piper_description)/meshes/visual/link4.glb"/>
         </geometry>
       </collision>
@@ -136,10 +130,10 @@
       <visual>
         <geometry>
-          <mesh filename="file://$(find piper_description)/meshes/visual/link5.obj"/>
+          <mesh filename="file://$(find piper_description)/meshes/visual/link5.glb"/>
         </geometry>
       </visual>
       <collision>
         <geometry>
-          <mesh filename="file://$(find piper_description)/meshes/collision/link5.obj"/>
+          <mesh filename="file://$(find piper_description)/meshes/visual/link5.glb"/>
         </geometry>
       </collision>
@@ -152,4 +146,22 @@
       <limit lower="-1.22" upper="1.22" effort="100" velocity="5"/>
     </joint>
+    <link name="${prefix}link6">
+      <inertial>
+        <origin xyz="-0.000183807162235591 8.05033155577911E-05 0.0321436689908876"/>
+        <mass value="0.657"/>
+        <inertia ixx="0.00092934" ixy="0.00000034" ixz="-0.00000738" iyy="0.00071447" iyz="0.00000005"
+                 izz="0.00039442"/>
+      </inertial>
+      <visual>
+        <geometry>
+          <mesh filename="file://$(find piper_description)/meshes/visual/link6.glb"/>
+        </geometry>
+      </visual>
+      <collision>
+        <geometry>
+          <mesh filename="file://$(find piper_description)/meshes/visual/link6.glb"/>
+        </geometry>
+      </collision>
+    </link>
     <joint name="${prefix}joint6" type="revolute">
       <origin xyz="0 -0.091 0" rpy="1.5708 0 0"/>
@@ -159,5 +171,9 @@
       <limit lower="-2.0944" upper="2.0944" effort="100" velocity="3"/>
     </joint>
-    <xacro:Gripper name="${prefix}"/>
+    <link name="${prefix}tcp"/>
+    <joint name="${prefix}tcp_joint" type="fixed">
+      <parent link="${prefix}link6"/>
+      <child link="${prefix}tcp"/>
+    </joint>
   </xacro:macro>
 </robot>

File: manipulator/AgileX/piper_description/xacro/robot.xacro (robot description, xacro)
@@ -1,12 +1,43 @@
 <?xml version="1.0"?>
 <robot name="Piper" xmlns:xacro="http://www.ros.org/wiki/xacro">
-  <xacro:arg name="type" default="slave"/>
-  <xacro:include filename="$(find piper_description)/xacro/Piper.xacro"/>
-  <!-- 根据type参数决定is_master的值 -->
-  <xacro:if value="${'$(arg type)' == 'master'}">
-    <xacro:Piper name="" is_master="true"/>
+  <xacro:arg name="arms" default="piper"/>
+  <xacro:arg name="type" default=""/>
+  <xacro:arg name="camera" default=""/>
+  <xacro:arg name="name" default=""/>
+  <xacro:arg name="eef_fixed_joints" default="false"/>
+  <xacro:property name="arms_arg" value="$(arg arms)"/>
+  <xacro:property name="type_arg" value="$(arg type)"/>
+  <xacro:property name="camera_arg" value="$(arg camera)"/>
+  <xacro:property name="name_arg" value="$(arg name)"/>
+  <xacro:property name="ee_type" value="${type_arg if type_arg else 'gripper'}"/>
+  <xacro:property name="camera_key" value="${camera_arg if camera_arg != '' else ('true' if (arms_arg == 'piper' and ee_type == 'gripper') else 'none')}"/>
+  <xacro:if value="${arms_arg == 'piper'}">
+    <xacro:include filename="$(find piper_description)/xacro/Piper.xacro"/>
+    <xacro:Piper name="${name_arg}"/>
   </xacro:if>
-  <xacro:unless value="${'$(arg type)' == 'master'}">
-    <xacro:Piper name="" is_master="false"/>
-  </xacro:unless>
+  <xacro:if value="${arms_arg == 'h'}">
+    <xacro:include filename="$(find piper_description)/xacro/PiperH.xacro"/>
+    <xacro:PiperH name="${name_arg}"/>
+  </xacro:if>
+  <xacro:if value="${arms_arg == 'l'}">
+    <xacro:include filename="$(find piper_description)/xacro/PiperL.xacro"/>
+    <xacro:PiperL name="${name_arg}"/>
+  </xacro:if>
+  <xacro:if value="${arms_arg == 'x'}">
+    <xacro:include filename="$(find piper_description)/xacro/PiperX.xacro"/>
+    <xacro:PiperX name="${name_arg}"/>
+  </xacro:if>
+  <xacro:include filename="$(find piper_description)/xacro/eefs.xacro"/>
+  <xacro:if value="${ee_type == 'revo1'}">
+    <xacro:include filename="$(find brainco_description)/xacro/revo1.xacro"/>
+  </xacro:if>
+  <xacro:if value="${ee_type == 'revo2'}">
+    <xacro:include filename="$(find brainco_description)/xacro/revo2.xacro"/>
+  </xacro:if>
+  <xacro:PiperEndEffectors
+      name="${name_arg}"
+      type="${ee_type}"
+      camera_type="${camera_key}"
+      arms="${arms_arg}"
+      fixed_joints="$(arg eef_fixed_joints)"/>
 </robot>

File: manipulator/AgileX/piper_description/xacro/ros2_control/piper.ros2_control.xacro (robot description, xacro)
@@ -1,4 +1,7 @@
 <?xml version="1.0"?>
 <robot xmlns:xacro="http://www.ros.org/wiki/xacro">
+  <!-- Compatibility wrapper exposing piper_system (dual-arm hardware macros). -->
+  <xacro:include filename="$(find piper_description)/xacro/ros2_control/interfaces.xacro"/>
+  <xacro:include filename="$(find piper_description)/xacro/ros2_control/end_effector_interfaces.xacro"/>
   <xacro:macro name="piper_system" params="name ros2_control_hardware_type">
     <xacro:property name="prefix" value="${name + '_' if name else ''}"/>
@@ -17,51 +20,6 @@
         </xacro:if>
       </hardware>
-      <!-- 关节接口定义 -->
-      <joint name="${prefix}joint1">
-        <command_interface name="position"/>
-        <state_interface name="position"/>
-        <state_interface name="velocity"/>
-        <state_interface name="effort"/>
-      </joint>
-      <joint name="${prefix}joint2">
-        <command_interface name="position"/>
-        <state_interface name="position">
-          <param name="initial_value">0.255</param>
-        </state_interface>
-        <state_interface name="velocity"/>
-        <state_interface name="effort"/>
-      </joint>
-      <joint name="${prefix}joint3">
-        <command_interface name="position"/>
-        <state_interface name="position">
-          <param name="initial_value">-0.2</param>
-        </state_interface>
-        <state_interface name="velocity"/>
-        <state_interface name="effort"/>
-      </joint>
-      <joint name="${prefix}joint4">
-        <command_interface name="position"/>
-        <state_interface name="position"/>
-        <state_interface name="velocity"/>
-        <state_interface name="effort"/>
-      </joint>
-      <joint name="${prefix}joint5">
-        <command_interface name="position"/>
-        <state_interface name="position"/>
-        <state_interface name="velocity"/>
-        <state_interface name="effort"/>
-      </joint>
-      <joint name="${prefix}joint6">
-        <command_interface name="position"/>
-        <state_interface name="position"/>
-        <state_interface name="velocity"/>
-        <state_interface name="effort"/>
-      </joint>
-      <joint name="${prefix}gripper_joint">
-        <command_interface name="position"/>
-        <state_interface name="position"/>
-        <state_interface name="velocity"/>
-        <state_interface name="effort"/>
-      </joint>
+      <xacro:piper_interfaces name="${name}"/>
+      <xacro:piper_gripper_interfaces name="${name}"/>
     </ros2_control>
   </xacro:macro>

File: manipulator/AgileX/piper_description/xacro/ros2_control/robot.xacro (robot description, xacro)
@@ -1,5 +1,6 @@
 <?xml version="1.0"?>
-<robot xmlns:xacro="http://www.ros.org/wiki/xacro" name="R5a">
-  <xacro:arg name="ros2_control_hardware_type" default="mock_components" />
+<robot xmlns:xacro="http://www.ros.org/wiki/xacro" name="Piper">
+  <xacro:arg name="ros2_control_hardware_type" default="mock_components"/>
+  <xacro:arg name="gazebo" default="false"/>
   <link name="world"/>
   <joint name="world_fixed" type="fixed">
@@ -7,12 +8,34 @@
     <child link="base_link"/>
   </joint>
-  <xacro:arg name="type" default="slave"/>
-  <xacro:include filename="$(find piper_description)/xacro/Piper.xacro"/>
-  <!-- 根据type参数决定is_master的值 -->
-  <xacro:Piper name="" is_master="false"/>
-  <!-- Import Piper ros2_control description -->
-  <xacro:include filename="$(find piper_description)/xacro/ros2_control/piper.ros2_control.xacro" />
-  <xacro:piper_system name="" ros2_control_hardware_type="$(arg ros2_control_hardware_type)"/>
-  <xacro:arg name="gazebo" default="false" />
+  <xacro:include filename="$(find piper_description)/xacro/robot.xacro"/>
+  <xacro:include filename="$(find piper_description)/xacro/ros2_control/interfaces.xacro"/>
+  <xacro:include filename="$(find piper_description)/xacro/ros2_control/end_effector_interfaces.xacro"/>
+  <ros2_control name="piper_system" type="system">
+    <hardware>
+      <xacro:if value="${'$(arg ros2_control_hardware_type)' == 'gz'}">
+        <plugin>gz_ros2_control/GazeboSimSystem</plugin>
+      </xacro:if>
+      <xacro:if value="${'$(arg ros2_control_hardware_type)' == 'mock_components'}">
+        <plugin>mock_components/GenericSystem</plugin>
+      </xacro:if>
+      <xacro:if value="${'$(arg ros2_control_hardware_type)' == 'isaac'}">
+        <plugin>topic_based_ros2_control/TopicBasedSystem</plugin>
+        <param name="joint_commands_topic">/isaac/joint_command</param>
+        <param name="joint_states_topic">/isaac/joint_states</param>
+      </xacro:if>
+    </hardware>
+    <xacro:piper_interfaces name="$(arg name)"/>
+    <xacro:unless value="${'$(arg type)' == 'none' or '$(arg type)' == 'revo1' or '$(arg type)' == 'revo2'}">
+      <xacro:piper_gripper_interfaces name="$(arg name)"/>
+    </xacro:unless>
+    <xacro:if value="${'$(arg type)' == 'revo1'}">
+      <xacro:include filename="$(find brainco_description)/xacro/ros2_control/revo1.xacro"/>
+      <xacro:revo1_interfaces name="${'$(arg name)' + '_hand' if '$(arg name)' else 'hand'}"/>
+    </xacro:if>
+    <xacro:if value="${'$(arg type)' == 'revo2'}">
+      <xacro:include filename="$(find brainco_description)/xacro/ros2_control/revo2.xacro"/>
+      <xacro:revo2_interfaces name="${'$(arg name)' + '_hand' if '$(arg name)' else 'hand'}"/>
+    </xacro:if>
+  </ros2_control>
   <xacro:if value="$(arg gazebo)">
     <gazebo>
