Commit message: reorganize inspire gripper

File: gripper/inspire_description/xacro/EG2-4C2.xacro (robot description, xacro)
@@ -3,5 +3,5 @@
   <xacro:macro name="Gripper" params="name">
     <xacro:property name="prefix" value="${name + '_' if name else ''}"/>
-    <link name="${prefix}base_link">
+    <link name="${prefix}gripper_base">
       <inertial>
         <origin xyz="1.5645E-05 -4.1838E-06 0.038"/>
@@ -17,10 +17,10 @@
       <visual>
         <geometry>
-          <mesh filename="file://$(find inspire_eg2_description)/meshes/baselink.obj"/>
-        </geometry>
-      </visual>
-      <collision>
-        <geometry>
-          <mesh filename="file://$(find inspire_eg2_description)/meshes/baselink.obj"/>
+          <mesh filename="file://$(find inspire_description)/meshes/EG2-4C2/baselink.obj"/>
+        </geometry>
+      </visual>
+      <collision>
+        <geometry>
+          <mesh filename="file://$(find inspire_description)/meshes/EG2-4C2/baselink.obj"/>
         </geometry>
       </collision>
@@ -40,16 +40,16 @@
       <visual>
         <geometry>
-          <mesh filename="file://$(find inspire_eg2_description)/meshes/Link1.obj"/>
-        </geometry>
-      </visual>
-      <collision>
-        <geometry>
-          <mesh filename="file://$(find inspire_eg2_description)/meshes/Link1.obj"/>
-        </geometry>
-      </collision>
-    </link>
-    <joint name="${prefix}Joint1" type="revolute">
+          <mesh filename="file://$(find inspire_description)/meshes/EG2-4C2/Link1.obj"/>
+        </geometry>
+      </visual>
+      <collision>
+        <geometry>
+          <mesh filename="file://$(find inspire_description)/meshes/EG2-4C2/Link1.obj"/>
+        </geometry>
+      </collision>
+    </link>
+    <joint name="${prefix}gripper_joint" type="revolute">
       <origin xyz="-0.04 -0.009 0.079"/>
-      <parent link="${prefix}base_link"/>
+      <parent link="${prefix}gripper_base"/>
       <child link="${prefix}Link1"/>
       <axis xyz="0 -1 0"/>
@@ -70,20 +70,20 @@
       <visual>
         <geometry>
-          <mesh filename="file://$(find inspire_eg2_description)/meshes/Link2.obj"/>
-        </geometry>
-      </visual>
-      <collision>
-        <geometry>
-          <mesh filename="file://$(find inspire_eg2_description)/meshes/Link2.obj"/>
-        </geometry>
-      </collision>
-    </link>
-    <joint name="${prefix}Joint2" type="revolute">
+          <mesh filename="file://$(find inspire_description)/meshes/EG2-4C2/Link2.obj"/>
+        </geometry>
+      </visual>
+      <collision>
+        <geometry>
+          <mesh filename="file://$(find inspire_description)/meshes/EG2-4C2/Link2.obj"/>
+        </geometry>
+      </collision>
+    </link>
+    <joint name="${prefix}gripper_joint2" type="revolute">
       <origin xyz="-0.03 -0.009 0.081" rpy="0 0 0"/>
-      <parent link="${prefix}base_link"/>
+      <parent link="${prefix}gripper_base"/>
       <child link="${prefix}Link2"/>
       <axis xyz="0 -1 0"/>
       <limit lower="0" upper="0.82" effort="1" velocity="1"/>
-      <mimic joint="${prefix}Joint1"/>
+      <mimic joint="${prefix}gripper_joint"/>
     </joint>
     <link name="${prefix}Link3">
@@ -101,20 +101,20 @@
       <visual>
         <geometry>
-          <mesh filename="file://$(find inspire_eg2_description)/meshes/Link3.obj"/>
-        </geometry>
-      </visual>
-      <collision>
-        <geometry>
-          <mesh filename="file://$(find inspire_eg2_description)/meshes/Link3.obj"/>
-        </geometry>
-      </collision>
-    </link>
-    <joint name="${prefix}Joint3" type="revolute">
+          <mesh filename="file://$(find inspire_description)/meshes/EG2-4C2/Link3.obj"/>
+        </geometry>
+      </visual>
+      <collision>
+        <geometry>
+          <mesh filename="file://$(find inspire_description)/meshes/EG2-4C2/Link3.obj"/>
+        </geometry>
+      </collision>
+    </link>
+    <joint name="${prefix}gripper_joint3" type="revolute">
       <origin xyz="0.03 -0.009 0.081" rpy="0 0 0"/>
-      <parent link="${prefix}base_link"/>
+      <parent link="${prefix}gripper_base"/>
       <child link="${prefix}Link3"/>
       <axis xyz="0 -1 0"/>
       <limit lower="-0.82" upper="0" effort="1" velocity="1"/>
-      <mimic joint="${prefix}Joint1" multiplier="-1" offset="0"/>
+      <mimic joint="${prefix}gripper_joint" multiplier="-1" offset="0"/>
     </joint>
     <link name="${prefix}Link4">
@@ -132,20 +132,20 @@
       <visual>
         <geometry>
-          <mesh filename="file://$(find inspire_eg2_description)/meshes/Link4.obj"/>
-        </geometry>
-      </visual>
-      <collision>
-        <geometry>
-          <mesh filename="file://$(find inspire_eg2_description)/meshes/Link4.obj"/>
-        </geometry>
-      </collision>
-    </link>
-    <joint name="${prefix}Joint4" type="revolute">
+          <mesh filename="file://$(find inspire_description)/meshes/EG2-4C2/Link4.obj"/>
+        </geometry>
+      </visual>
+      <collision>
+        <geometry>
+          <mesh filename="file://$(find inspire_description)/meshes/EG2-4C2/Link4.obj"/>
+        </geometry>
+      </collision>
+    </link>
+    <joint name="${prefix}gripper_joint4" type="revolute">
       <origin xyz="0.04 -0.009 0.079" rpy="0 0 0"/>
-      <parent link="${prefix}base_link"/>
+      <parent link="${prefix}gripper_base"/>
       <child link="${prefix}Link4"/>
       <axis xyz="0 -1 0"/>
       <limit lower="-0.82" upper="0" effort="1" velocity="1"/>
-      <mimic joint="${prefix}Joint1" multiplier="-1" offset="0"/>
+      <mimic joint="${prefix}gripper_joint" multiplier="-1" offset="0"/>
     </joint>
     <link name="${prefix}Link5">
@@ -163,14 +163,14 @@
       <visual>
         <geometry>
-          <mesh filename="file://$(find inspire_eg2_description)/meshes/Link5.obj"/>
-        </geometry>
-      </visual>
-      <collision>
-        <geometry>
-          <mesh filename="file://$(find inspire_eg2_description)/meshes/Link5.obj"/>
-        </geometry>
-      </collision>
-    </link>
-    <joint name="${prefix}Joint5" type="revolute">
+          <mesh filename="file://$(find inspire_description)/meshes/EG2-4C2/Link5.obj"/>
+        </geometry>
+      </visual>
+      <collision>
+        <geometry>
+          <mesh filename="file://$(find inspire_description)/meshes/EG2-4C2/Link5.obj"/>
+        </geometry>
+      </collision>
+    </link>
+    <joint name="${prefix}gripper_joint5" type="revolute">
       <origin xyz="0.0223 0.003 0.035591" rpy="0 0 0"/>
       <parent link="${prefix}Link1"/>
@@ -178,5 +178,5 @@
       <axis xyz="0 1 0"/>
       <limit lower="0" upper="0.82" effort="1" velocity="1"/>
-      <mimic joint="${prefix}Joint1"/>
+      <mimic joint="${prefix}gripper_joint"/>
     </joint>
     <link name="${prefix}Link6">
@@ -194,14 +194,14 @@
       <visual>
         <geometry>
-          <mesh filename="file://$(find inspire_eg2_description)/meshes/Link6.obj"/>
-        </geometry>
-      </visual>
-      <collision>
-        <geometry>
-          <mesh filename="file://$(find inspire_eg2_description)/meshes/Link6.obj"/>
-        </geometry>
-      </collision>
-    </link>
-    <joint name="${prefix}Joint6" type="revolute">
+          <mesh filename="file://$(find inspire_description)/meshes/EG2-4C2/Link6.obj"/>
+        </geometry>
+      </visual>
+      <collision>
+        <geometry>
+          <mesh filename="file://$(find inspire_description)/meshes/EG2-4C2/Link6.obj"/>
+        </geometry>
+      </collision>
+    </link>
+    <joint name="${prefix}gripper_joint6" type="revolute">
       <origin xyz="-0.0223 0.003 0.035591"/>
       <parent link="${prefix}Link4"/>
@@ -209,5 +209,5 @@
       <axis xyz="0 -1 0"/>
       <limit lower="0" upper="0.82" effort="1" velocity="1"/>
-      <mimic joint="${prefix}Joint1"/>
+      <mimic joint="${prefix}gripper_joint"/>
     </joint>
   </xacro:macro>

File: manipulator/Realman/rm65_description/xacro/arm.xacro (robot description, xacro)
@@ -220,10 +220,10 @@
       <child link="${prefix}gripper_plate"/>
     </joint>
-    <xacro:include filename="$(find inspire_eg2_description)/xacro/eg2_4c2.xacro"/>
-    <xacro:Gripper name="${prefix}gripper"/>
-    <joint name="${prefix}gripper_joint" type="fixed">
-      <origin xyz="0 0 0.0043" rpy="0 0 0"/>
+    <xacro:include filename="$(find inspire_description)/xacro/EG2-4C2.xacro"/>
+    <xacro:Gripper name="${name}"/>
+    <joint name="${prefix}gripper_base_joint" type="fixed">
+      <origin xyz="0 0 0.0043"/>
       <parent link="${prefix}gripper_plate" />
-      <child link="${prefix}gripper_base_link" />
+      <child link="${prefix}gripper_base" />
     </joint>
   </xacro:macro>

Commit message: better rm65 visualize

File: gripper/inspire_description/xacro/EG2-4C2.xacro (robot description, xacro)
@@ -26,7 +26,7 @@
       </collision>
     </link>
-    <link name="${prefix}Link1">
-      <inertial>
-        <origin xyz="0.0087669 0.009 0.013992" rpy="0 0 0"/>
+    <link name="${prefix}left_outer_link">
+      <inertial>
+        <origin xyz="0.0087669 0.009 0.013992" />
         <mass value="0.0024292"/>
         <inertia
@@ -40,10 +40,10 @@
       <visual>
         <geometry>
-          <mesh filename="file://$(find inspire_description)/meshes/EG2-4C2/Link1.obj"/>
-        </geometry>
-      </visual>
-      <collision>
-        <geometry>
-          <mesh filename="file://$(find inspire_description)/meshes/EG2-4C2/Link1.obj"/>
+          <mesh filename="file://$(find inspire_description)/meshes/EG2-4C2/outer_link.obj"/>
+        </geometry>
+      </visual>
+      <collision>
+        <geometry>
+          <mesh filename="file://$(find inspire_description)/meshes/EG2-4C2/outer_link.obj"/>
         </geometry>
       </collision>
@@ -52,11 +52,11 @@
       <origin xyz="-0.04 -0.009 0.079"/>
       <parent link="${prefix}gripper_base"/>
-      <child link="${prefix}Link1"/>
+      <child link="${prefix}left_outer_link"/>
       <axis xyz="0 -1 0"/>
       <limit lower="0" upper="0.82" effort="1" velocity="1"/>
     </joint>
-    <link name="${prefix}Link2">
-      <inertial>
-        <origin xyz="0.0087435 0.009 0.013955" rpy="0 0 0"/>
+    <link name="${prefix}left_inner_link">
+      <inertial>
+        <origin xyz="0.0087435 0.009 0.013955" />
         <mass value="0.0038971"/>
         <inertia
@@ -70,24 +70,24 @@
       <visual>
         <geometry>
-          <mesh filename="file://$(find inspire_description)/meshes/EG2-4C2/Link2.obj"/>
-        </geometry>
-      </visual>
-      <collision>
-        <geometry>
-          <mesh filename="file://$(find inspire_description)/meshes/EG2-4C2/Link2.obj"/>
-        </geometry>
-      </collision>
-    </link>
-    <joint name="${prefix}gripper_joint2" type="revolute">
-      <origin xyz="-0.03 -0.009 0.081" rpy="0 0 0"/>
-      <parent link="${prefix}gripper_base"/>
-      <child link="${prefix}Link2"/>
+          <mesh filename="file://$(find inspire_description)/meshes/EG2-4C2/inner_link.obj"/>
+        </geometry>
+      </visual>
+      <collision>
+        <geometry>
+          <mesh filename="file://$(find inspire_description)/meshes/EG2-4C2/inner_link.obj"/>
+        </geometry>
+      </collision>
+    </link>
+    <joint name="${prefix}left_inner_joint" type="revolute">
+      <origin xyz="-0.03 -0.009 0.081" />
+      <parent link="${prefix}gripper_base"/>
+      <child link="${prefix}left_inner_link"/>
       <axis xyz="0 -1 0"/>
       <limit lower="0" upper="0.82" effort="1" velocity="1"/>
       <mimic joint="${prefix}gripper_joint"/>
     </joint>
-    <link name="${prefix}Link3">
-      <inertial>
-        <origin xyz="-0.0087435 0.009 0.013955" rpy="0 0 0"/>
+    <link name="${prefix}right_inner_link">
+      <inertial>
+        <origin xyz="-0.0087435 0.009 0.013955" />
         <mass value="0.0038971"/>
         <inertia
@@ -101,24 +101,24 @@
       <visual>
         <geometry>
-          <mesh filename="file://$(find inspire_description)/meshes/EG2-4C2/Link3.obj"/>
-        </geometry>
-      </visual>
-      <collision>
-        <geometry>
-          <mesh filename="file://$(find inspire_description)/meshes/EG2-4C2/Link3.obj"/>
-        </geometry>
-      </collision>
-    </link>
-    <joint name="${prefix}gripper_joint3" type="revolute">
-      <origin xyz="0.03 -0.009 0.081" rpy="0 0 0"/>
-      <parent link="${prefix}gripper_base"/>
-      <child link="${prefix}Link3"/>
-      <axis xyz="0 -1 0"/>
-      <limit lower="-0.82" upper="0" effort="1" velocity="1"/>
-      <mimic joint="${prefix}gripper_joint" multiplier="-1" offset="0"/>
-    </joint>
-    <link name="${prefix}Link4">
-      <inertial>
-        <origin xyz="-0.0087669 0.009 0.013992" rpy="0 0 0"/>
+          <mesh filename="file://$(find inspire_description)/meshes/EG2-4C2/inner_link.obj" scale="-1 1 1"/>
+        </geometry>
+      </visual>
+      <collision>
+        <geometry>
+          <mesh filename="file://$(find inspire_description)/meshes/EG2-4C2/inner_link.obj" scale="-1 1 1"/>
+        </geometry>
+      </collision>
+    </link>
+    <joint name="${prefix}right_inner_joint" type="revolute">
+      <origin xyz="0.03 -0.009 0.081" />
+      <parent link="${prefix}gripper_base"/>
+      <child link="${prefix}right_inner_link"/>
+      <axis xyz="0 1 0"/>
+      <limit lower="0.82" upper="0" effort="1" velocity="1"/>
+      <mimic joint="${prefix}gripper_joint" multiplier="1" offset="0"/>
+    </joint>
+    <link name="${prefix}right_outer_link">
+      <inertial>
+        <origin xyz="-0.0087669 0.009 0.013992" />
         <mass value="0.0024292"/>
         <inertia
@@ -132,24 +132,24 @@
       <visual>
         <geometry>
-          <mesh filename="file://$(find inspire_description)/meshes/EG2-4C2/Link4.obj"/>
-        </geometry>
-      </visual>
-      <collision>
-        <geometry>
-          <mesh filename="file://$(find inspire_description)/meshes/EG2-4C2/Link4.obj"/>
-        </geometry>
-      </collision>
-    </link>
-    <joint name="${prefix}gripper_joint4" type="revolute">
-      <origin xyz="0.04 -0.009 0.079" rpy="0 0 0"/>
-      <parent link="${prefix}gripper_base"/>
-      <child link="${prefix}Link4"/>
-      <axis xyz="0 -1 0"/>
-      <limit lower="-0.82" upper="0" effort="1" velocity="1"/>
-      <mimic joint="${prefix}gripper_joint" multiplier="-1" offset="0"/>
-    </joint>
-    <link name="${prefix}Link5">
-      <inertial>
-        <origin xyz="0.011864 0.006 0.011367" rpy="0 0 0"/>
+          <mesh filename="file://$(find inspire_description)/meshes/EG2-4C2/outer_link.obj" scale="-1 1 1"/>
+        </geometry>
+      </visual>
+      <collision>
+        <geometry>
+          <mesh filename="file://$(find inspire_description)/meshes/EG2-4C2/outer_link.obj" scale="-1 1 1"/>
+        </geometry>
+      </collision>
+    </link>
+    <joint name="${prefix}right_outer_joint" type="revolute">
+      <origin xyz="0.04 -0.009 0.079" />
+      <parent link="${prefix}gripper_base"/>
+      <child link="${prefix}right_outer_link"/>
+      <axis xyz="0 1 0"/>
+      <limit lower="0" upper="0.82" effort="1" velocity="1"/>
+      <mimic joint="${prefix}gripper_joint" multiplier="1" offset="0"/>
+    </joint>
+    <link name="${prefix}left_pad">
+      <inertial>
+        <origin xyz="0.011864 0.006 0.011367" />
         <mass value="0.0045068"/>
         <inertia
@@ -163,24 +163,24 @@
       <visual>
         <geometry>
-          <mesh filename="file://$(find inspire_description)/meshes/EG2-4C2/Link5.obj"/>
-        </geometry>
-      </visual>
-      <collision>
-        <geometry>
-          <mesh filename="file://$(find inspire_description)/meshes/EG2-4C2/Link5.obj"/>
-        </geometry>
-      </collision>
-    </link>
-    <joint name="${prefix}gripper_joint5" type="revolute">
-      <origin xyz="0.0223 0.003 0.035591" rpy="0 0 0"/>
-      <parent link="${prefix}Link1"/>
-      <child link="${prefix}Link5"/>
+          <mesh filename="file://$(find inspire_description)/meshes/EG2-4C2/pad.obj"/>
+        </geometry>
+      </visual>
+      <collision>
+        <geometry>
+          <mesh filename="file://$(find inspire_description)/meshes/EG2-4C2/pad.obj"/>
+        </geometry>
+      </collision>
+    </link>
+    <joint name="${prefix}left_pad_joint" type="revolute">
+      <origin xyz="0.0223 0.003 0.035591" />
+      <parent link="${prefix}left_outer_link"/>
+      <child link="${prefix}left_pad"/>
       <axis xyz="0 1 0"/>
       <limit lower="0" upper="0.82" effort="1" velocity="1"/>
-      <mimic joint="${prefix}gripper_joint"/>
-    </joint>
-    <link name="${prefix}Link6">
-      <inertial>
-        <origin xyz="-0.011864 0.006 0.011367" rpy="0 0 0"/>
+      <mimic joint="${prefix}gripper_joint" multiplier="1" offset="0"/>
+    </joint>
+    <link name="${prefix}right_pad">
+      <inertial>
+        <origin xyz="-0.011864 0.006 0.011367" />
         <mass value="0.0045068"/>
         <inertia
@@ -194,20 +194,20 @@
       <visual>
         <geometry>
-          <mesh filename="file://$(find inspire_description)/meshes/EG2-4C2/Link6.obj"/>
-        </geometry>
-      </visual>
-      <collision>
-        <geometry>
-          <mesh filename="file://$(find inspire_description)/meshes/EG2-4C2/Link6.obj"/>
-        </geometry>
-      </collision>
-    </link>
-    <joint name="${prefix}gripper_joint6" type="revolute">
+          <mesh filename="file://$(find inspire_description)/meshes/EG2-4C2/pad.obj" scale="-1 1 1"/>
+        </geometry>
+      </visual>
+      <collision>
+        <geometry>
+          <mesh filename="file://$(find inspire_description)/meshes/EG2-4C2/pad.obj"  scale="-1 1 1"/>
+        </geometry>
+      </collision>
+    </link>
+    <joint name="${prefix}right_pad_joint" type="revolute">
       <origin xyz="-0.0223 0.003 0.035591"/>
-      <parent link="${prefix}Link4"/>
-      <child link="${prefix}Link6"/>
+      <parent link="${prefix}right_outer_link"/>
+      <child link="${prefix}right_pad"/>
       <axis xyz="0 -1 0"/>
       <limit lower="0" upper="0.82" effort="1" velocity="1"/>
-      <mimic joint="${prefix}gripper_joint"/>
+      <mimic joint="${prefix}gripper_joint" multiplier="1" offset="0"/>
     </joint>
   </xacro:macro>

File: manipulator/Realman/rm65_description/xacro/arm.xacro (robot description, xacro)
@@ -11,7 +11,4 @@
           <mesh filename="${mesh_path}${mesh}"/>
         </geometry>
-        <material name="">
-          <color rgba="0.79216 0.81961 0.93333 1"/>
-        </material>
       </visual>
       <collision>
