Commit message: ros2 control for galaxea a1 robot

File: manipulator/ARX/arx5_description/xacro/ros2_control/robot.xacro (robot description, xacro)
@@ -23,5 +23,10 @@
     <gazebo>
       <plugin filename="gz_ros2_control-system" name="gz_ros2_control::GazeboSimROS2ControlPlugin">
-        <parameters>$(find arx5_description)/config/ros2_control/ros2_controllers.yaml</parameters>
+        <xacro:if value="${'$(arg type)' == 'r5'}">
+          <parameters>$(find arx5_description)/config/ros2_control/arx_r5.yaml</parameters>
+        </xacro:if>
+        <xacro:if value="${'$(arg type)' == 'x5'}">
+          <parameters>$(find arx5_description)/config/ros2_control/ros2_controllers.yaml</parameters>
+        </xacro:if>
       </plugin>
     </gazebo>

File: manipulator/Galaxea/galaxea_a1_description/xacro/a1.xacro (robot description, xacro)
@@ -3,8 +3,9 @@
   <xacro:macro name="Arm" params="name direction:=normal">
     <xacro:property name="prefix" value="${name + '_' if name else ''}"/>
+    <!-- Base Link -->
     <link name="${prefix}base_link">
       <inertial>
         <origin xyz="-0.0005634 0.038934 3.1874E-06"/>
-        <mass value="1.658" />
+        <mass value="1.658"/>
         <inertia
             ixx="0.0010597"
@@ -13,22 +14,22 @@
             iyy="0.0011787"
             iyz="-1.9146E-07"
-            izz="0.0010647" />
-      </inertial>
-      <visual>
-        <geometry>
-          <mesh filename="file://$(find galaxea_a1_description)/meshes/a1/base_link.obj" />
-        </geometry>
-      </visual>
-      <collision>
-        <geometry>
-          <mesh
-              filename="file://$(find galaxea_a1_description)/meshes/a1/base_link.obj" />
-        </geometry>
-      </collision>
-    </link>
+            izz="0.0010647"/>
+      </inertial>
+      <visual>
+        <geometry>
+          <mesh filename="file://$(find galaxea_a1_description)/meshes/a1/base_link.obj"/>
+        </geometry>
+      </visual>
+      <collision>
+        <geometry>
+          <mesh filename="file://$(find galaxea_a1_description)/meshes/a1/base_link.obj"/>
+        </geometry>
+      </collision>
+    </link>
+    <!-- Link 1 -->
     <link name="${prefix}link1">
       <inertial>
         <origin xyz="0.000015 0.105259 -0.001954"/>
-        <mass value="1.164" />
+        <mass value="1.164"/>
         <inertia
             ixx="0.001125"
@@ -37,32 +38,30 @@
             iyy="0.001084"
             iyz="-0.000023"
-            izz="0.001158" />
-      </inertial>
-      <visual>
-        <geometry>
-          <mesh filename="file://$(find galaxea_a1_description)/meshes/a1/link1.obj" />
-        </geometry>
-      </visual>
-      <collision>
-        <geometry>
-          <mesh filename="file://$(find galaxea_a1_description)/meshes/a1/link1.obj" />
-        </geometry>
-      </collision>
-    </link>
+            izz="0.001158"/>
+      </inertial>
+      <visual>
+        <geometry>
+          <mesh filename="file://$(find galaxea_a1_description)/meshes/a1/link1.obj"/>
+        </geometry>
+      </visual>
+      <collision>
+        <geometry>
+          <mesh filename="file://$(find galaxea_a1_description)/meshes/a1/link1.obj"/>
+        </geometry>
+      </collision>
+    </link>
+    <!-- Joint 1: Base to Link1 -->
     <joint name="${prefix}joint1" type="revolute">
-      <origin xyz="-0.0011147 0 0.0446" />
-      <parent link="${prefix}base_link" />
-      <child link="${prefix}link1" />
-      <axis xyz="0 0 1" />
-      <limit lower="-2.8798" upper="2.8798" effort="40" velocity="20.944" />
-    </joint>
-    <link
-        name="${prefix}link2">
-      <inertial>
-        <origin
-            xyz="-0.23622 0.016352 -0.00013275"
-            rpy="0 0 0" />
-        <mass
-            value="1.3" />
+      <origin xyz="-0.0011147 0 0.0446"/>
+      <parent link="${prefix}base_link"/>
+      <child link="${prefix}link1"/>
+      <axis xyz="0 0 1"/>
+      <limit lower="-2.8798" upper="2.8798" effort="40" velocity="20.944"/>
+    </joint>
+    <!-- Link 2 -->
+    <link name="${prefix}link2">
+      <inertial>
+        <origin xyz="-0.23622 0.016352 -0.00013275"/>
+        <mass value="1.3"/>
         <inertia
             ixx="0.00060638"
@@ -71,44 +70,30 @@
             iyy="0.0075936"
             iyz="-8.0916E-06"
-            izz="0.0075712" />
-      </inertial>
-      <visual>
-        <geometry>
-          <mesh filename="file://$(find galaxea_a1_description)/meshes/a1/link2.obj" />
-        </geometry>
-      </visual>
-      <collision>
-        <geometry>
-          <mesh
-              filename="file://$(find galaxea_a1_description)/meshes/a1/link2.obj" />
-        </geometry>
-      </collision>
-    </link>
-    <joint
-        name="${prefix}joint2"
-        type="revolute">
-      <origin
-          xyz="0 0 0.1061"
-          rpy="1.5708 0 0" />
-      <parent
-          link="${prefix}link1" />
-      <child
-          link="${prefix}link2" />
-      <axis
-          xyz="0 0 -1" />
-      <limit
-          lower="0"
-          upper="3.2289"
-          effort="40"
-          velocity="20.944" />
-    </joint>
-    <link
-        name="${prefix}link3">
-      <inertial>
-        <origin
-            xyz="0.045114 0.054616 -0.00045593"
-            rpy="0 0 0" />
-        <mass
-            value="0.818" />
+            izz="0.0075712"/>
+      </inertial>
+      <visual>
+        <geometry>
+          <mesh filename="file://$(find galaxea_a1_description)/meshes/a1/link2.obj"/>
+        </geometry>
+      </visual>
+      <collision>
+        <geometry>
+          <mesh filename="file://$(find galaxea_a1_description)/meshes/a1/link2.obj"/>
+        </geometry>
+      </collision>
+    </link>
+    <!-- Joint 2: Link1 to Link2 -->
+    <joint name="${prefix}joint2" type="revolute">
+      <origin xyz="0 0 0.1061" rpy="1.5708 0 0"/>
+      <parent link="${prefix}link1"/>
+      <child link="${prefix}link2"/>
+      <axis xyz="0 0 -1"/>
+      <limit lower="0" upper="3.2289" effort="40" velocity="20.944"/>
+    </joint>
+    <!-- Link 3 -->
+    <link name="${prefix}link3">
+      <inertial>
+        <origin xyz="0.045114 0.054616 -0.00045593"/>
+        <mass value="0.818"/>
         <inertia
             ixx="0.00060107"
@@ -117,56 +102,30 @@
             iyy="0.0013959"
             iyz="-9.7503E-06"
-            izz="0.0015027" />
-      </inertial>
-      <visual>
-        <origin
-            xyz="0 0 0"
-            rpy="0 0 0" />
-        <geometry>
-          <mesh
-              filename="file://$(find galaxea_a1_description)/meshes/a1/link3.obj" />
-        </geometry>
-        <material
-            name="">
-          <color
-              rgba="0.79216 0.81961 0.93333 1" />
-        </material>
-      </visual>
-      <collision>
-        <origin
-            xyz="0 0 0"
-            rpy="0 0 0" />
-        <geometry>
-          <mesh
-              filename="file://$(find galaxea_a1_description)/meshes/a1/link3.obj" />
-        </geometry>
-      </collision>
-    </link>
-    <joint
-        name="${prefix}joint3"
-        type="revolute">
-      <origin
-          xyz="-0.34928 0.019998 0"
-          rpy="0 0 0" />
-      <parent
-          link="${prefix}link2" />
-      <child
-          link="${prefix}link3" />
-      <axis
-          xyz="0 0 -1" />
-      <limit
-          lower="-3.3161"
-          upper="0"
-          effort="27"
-          velocity="7.5398" />
-    </joint>
-    <link
-        name="${prefix}link4">
-      <inertial>
-        <origin
-            xyz="0.24285 0.0023784 1.279E-06"
-            rpy="0 0 0" />
-        <mass
-            value="0.698" />
+            izz="0.0015027"/>
+      </inertial>
+      <visual>
+        <geometry>
+          <mesh filename="file://$(find galaxea_a1_description)/meshes/a1/link3.obj"/>
+        </geometry>
+      </visual>
+      <collision>
+        <geometry>
+          <mesh filename="file://$(find galaxea_a1_description)/meshes/a1/link3.obj"/>
+        </geometry>
+      </collision>
+    </link>
+    <!-- Joint 3: Link2 to Link3 -->
+    <joint name="${prefix}joint3" type="revolute">
+      <origin xyz="-0.34928 0.019998 0"/>
+      <parent link="${prefix}link2"/>
+      <child link="${prefix}link3"/>
+      <axis xyz="0 0 -1"/>
+      <limit lower="-3.3161" upper="0" effort="27" velocity="7.5398"/>
+    </joint>
+    <!-- Link 4 -->
+    <link name="${prefix}link4">
+      <inertial>
+        <origin xyz="0.24285 0.0023784 1.279E-06"/>
+        <mass value="0.698"/>
         <inertia
             ixx="8.45E-05"
@@ -175,56 +134,30 @@
             iyy="0.00010174"
             iyz="5.3612E-09"
-            izz="9.7044E-05" />
-      </inertial>
-      <visual>
-        <origin
-            xyz="0 0 0"
-            rpy="0 0 0" />
-        <geometry>
-          <mesh
-              filename="file://$(find galaxea_a1_description)/meshes/a1/link4.obj" />
-        </geometry>
-        <material
-            name="">
-          <color
-              rgba="1 1 1 1" />
-        </material>
-      </visual>
-      <collision>
-        <origin
-            xyz="0 0 0"
-            rpy="0 0 0" />
-        <geometry>
-          <mesh
-              filename="file://$(find galaxea_a1_description)/meshes/a1/link4.obj" />
-        </geometry>
-      </collision>
-    </link>
-    <joint
-        name="${prefix}joint4"
-        type="revolute">
-      <origin
-          xyz="0.02735 0.069767 0"
-          rpy="0 0 0" />
-      <parent
-          link="${prefix}link3" />
-      <child
-          link="${prefix}link4" />
-      <axis
-          xyz="1 0 0" />
-      <limit
-          lower="-2.8798"
-          upper="2.8798"
-          effort="7"
-          velocity="25.133" />
-    </joint>
-    <link
-        name="${prefix}link5">
-      <inertial>
-        <origin
-            xyz="0.054309 0.0041811 4.0699E-06"
-            rpy="0 0 0" />
-        <mass
-            value="0.417" />
+            izz="9.7044E-05"/>
+      </inertial>
+      <visual>
+        <geometry>
+          <mesh filename="file://$(find galaxea_a1_description)/meshes/a1/link4.obj"/>
+        </geometry>
+      </visual>
+      <collision>
+        <geometry>
+          <mesh filename="file://$(find galaxea_a1_description)/meshes/a1/link4.obj"/>
+        </geometry>
+      </collision>
+    </link>
+    <!-- Joint 4: Link3 to Link4 -->
+    <joint name="${prefix}joint4" type="revolute">
+      <origin xyz="0.02735 0.069767 0"/>
+      <parent link="${prefix}link3"/>
+      <child link="${prefix}link4"/>
+      <axis xyz="1 0 0"/>
+      <limit lower="-2.8798" upper="2.8798" effort="7" velocity="25.133"/>
+    </joint>
+    <!-- Link 5 -->
+    <link name="${prefix}link5">
+      <inertial>
+        <origin xyz="0.054309 0.0041811 4.0699E-06"/>
+        <mass value="0.417"/>
         <inertia
             ixx="8.3999E-05"
@@ -233,56 +166,30 @@
             iyy="9.8498E-05"
             iyz="-1.3811E-08"
-            izz="0.00011333" />
-      </inertial>
-      <visual>
-        <origin
-            xyz="0 0 0"
-            rpy="0 0 0" />
-        <geometry>
-          <mesh
-              filename="file://$(find galaxea_a1_description)/meshes/a1/link5.obj" />
-        </geometry>
-        <material
-            name="">
-          <color
-              rgba="1 1 1 1" />
-        </material>
-      </visual>
-      <collision>
-        <origin
-            xyz="0 0 0"
-            rpy="0 0 0" />
-        <geometry>
-          <mesh
-              filename="file://$(find galaxea_a1_description)/meshes/a1/link5.obj" />
-        </geometry>
-      </collision>
-    </link>
-    <joint
-        name="${prefix}joint5"
-        type="revolute">
-      <origin
-          xyz="0.2463 -0.00049894 0"
-          rpy="0 0 0" />
-      <parent
-          link="${prefix}link4" />
-      <child
-          link="${prefix}link5" />
-      <axis
-          xyz="0 1 0" />
-      <limit
-          lower="-1.6581"
-          upper="1.6581"
-          effort="7"
-          velocity="25.133" />
-    </joint>
-    <link
-        name="${prefix}link6">
-      <inertial>
-        <origin
-            xyz="0.028138 1.2134E-07 5.4049E-08"
-            rpy="0 0 0" />
-        <mass
-            value="0.037" />
+            izz="0.00011333"/>
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
File: manipulator/Galaxea/galaxea_a1_description/xacro/gripper.xacro (robot description, xacro)
@@ -3,5 +3,5 @@
   <xacro:macro name="Gripper" params="name">
     <xacro:property name="prefix" value="${name + '_' if name else ''}"/>
-    <link name="${prefix}base_link">
+    <link name="${prefix}gripper_base">
       <inertial>
         <origin xyz="-0.0311072323899603 1.17979991887118E-08 7.93394685505433E-08"/>
@@ -17,14 +17,14 @@
       <visual>
         <geometry>
-          <mesh filename="file://$(find galaxea_g1_description)/meshes/gripper_link.obj"/>
+          <mesh filename="file://$(find galaxea_a1_description)/meshes/gripper/gripper_link.obj"/>
         </geometry>
       </visual>
       <collision>
         <geometry>
-          <mesh filename="file://$(find galaxea_g1_description)/meshes/gripper_link.obj"/>
+          <mesh filename="file://$(find galaxea_a1_description)/meshes/gripper/gripper_link.obj"/>
         </geometry>
       </collision>
     </link>
-    <link name="${prefix}link1">
+    <link name="${prefix}finger1">
       <inertial>
         <origin xyz="-0.0195895895552112 -0.0151136845490034 0.00542254359093075"/>
@@ -40,21 +40,21 @@
       <visual>
         <geometry>
-          <mesh filename="file://$(find galaxea_g1_description)/meshes/gripper_finger1.obj"/>
+          <mesh filename="file://$(find galaxea_a1_description)/meshes/gripper/finger.obj"/>
         </geometry>
       </visual>
       <collision>
         <geometry>
-          <mesh filename="file://$(find galaxea_g1_description)/meshes/gripper_finger1.obj"/>
+          <mesh filename="file://$(find galaxea_a1_description)/meshes/gripper/finger.obj"/>
         </geometry>
       </collision>
     </link>
-    <joint name="${prefix}joint1" type="prismatic">
+    <joint name="${prefix}gripper_joint" type="prismatic">
       <origin xyz="0.03689 0.013453 0.00012059"/>
-      <parent link="${prefix}base_link"/>
-      <child link="${prefix}link1"/>
+      <parent link="${prefix}gripper_base"/>
+      <child link="${prefix}finger1"/>
       <axis xyz="0 1 0"/>
       <limit lower="0" upper="0.05" effort="100" velocity="0.25"/>
     </joint>
-    <link name="${prefix}link2">
+    <link name="${prefix}finger2">
       <inertial>
         <origin xyz="-0.0195895857999098 0.0151136893508115 -0.00542254357246619"/>
@@ -70,20 +70,26 @@
       <visual>
         <geometry>
-          <mesh filename="file://$(find galaxea_g1_description)/meshes/gripper_finger2.obj"/>
+          <mesh filename="file://$(find galaxea_a1_description)/meshes/gripper/finger.obj" scale="1 -1 -1"/>
         </geometry>
       </visual>
       <collision>
         <geometry>
-          <mesh filename="file://$(find galaxea_g1_description)/meshes/gripper_finger2.obj"/>
+          <mesh filename="file://$(find galaxea_a1_description)/meshes/gripper/finger.obj" scale="1 -1 -1"/>
         </geometry>
       </collision>
     </link>
-    <joint name="${prefix}joint2" type="prismatic">
+    <joint name="${prefix}gripper_joint2" type="prismatic">
       <origin xyz="0.03689 -0.013453 -0.00012059"/>
-      <parent link="${prefix}base_link"/>
-      <child link="${prefix}link2"/>
+      <parent link="${prefix}gripper_base"/>
+      <child link="${prefix}finger2"/>
       <axis xyz="0 -1 0"/>
       <limit lower="0" upper="0.05" effort="100" velocity="0.25"/>
-      <mimic joint="${prefix}joint1" multiplier="1" offset="0"/>
+      <mimic joint="${prefix}gripper_joint" multiplier="1" offset="0"/>
+    </joint>
+    <link name="${prefix}gripper_center"/>
+    <joint name="${prefix}gripper_center_joint" type="fixed">
+      <origin xyz="0.03689 0 -0.00012059"/>
+      <parent link="${prefix}gripper_base"/>
+      <child link="${prefix}gripper_center"/>
     </joint>
   </xacro:macro>

File: manipulator/Galaxea/galaxea_a1_description/xacro/ros2_control/galaxea_a1.ros2_control.xacro (robot description, xacro)
@@ -1,5 +1,5 @@
 <?xml version="1.0"?>
 <robot xmlns:xacro="http://www.ros.org/wiki/xacro">
-  <xacro:macro name="airbot_play_system" params="name ros2_control_hardware_type">
+  <xacro:macro name="galaxea_a1_system" params="name ros2_control_hardware_type">
     <xacro:property name="prefix" value="${name + '_' if name else ''}"/>
     <ros2_control name="${prefix}piper_system" type="system">
