Commit message: arx lift ocs2 gazebo

File: manipulator/ARX/arx5_description/xacro/ros2_control/arx5.ros2_control.xacro (robot description, xacro)
@@ -2,5 +2,6 @@
 <robot xmlns:xacro="http://www.ros.org/wiki/xacro">
   <xacro:macro name="arx5_system" params="name ros2_control_hardware_type">
-    <ros2_control name="${name}" type="system">
+    <xacro:property name="prefix" value="${name + '_' if name else ''}"/>
+    <ros2_control name="${prefix}ARX5System" type="system">
       <hardware>
         <xacro:if value="${ros2_control_hardware_type == 'gz'}">
@@ -17,5 +18,5 @@
       </hardware>
       <!-- 关节接口定义 -->
-      <joint name="joint1">
+      <joint name="${prefix}joint1">
         <command_interface name="position"/>
         <state_interface name="position"/>
@@ -23,5 +24,5 @@
         <state_interface name="effort"/>
       </joint>
-      <joint name="joint2">
+      <joint name="${prefix}joint2">
         <command_interface name="position"/>
         <state_interface name="position">
@@ -31,5 +32,5 @@
         <state_interface name="effort"/>
       </joint>
-      <joint name="joint3">
+      <joint name="${prefix}joint3">
         <command_interface name="position"/>
         <state_interface name="position">
@@ -39,5 +40,5 @@
         <state_interface name="effort"/>
       </joint>
-      <joint name="joint4">
+      <joint name="${prefix}joint4">
         <command_interface name="position"/>
         <state_interface name="position">
@@ -47,5 +48,5 @@
         <state_interface name="effort"/>
       </joint>
-      <joint name="joint5">
+      <joint name="${prefix}joint5">
         <command_interface name="position"/>
         <state_interface name="position"/>
@@ -53,5 +54,5 @@
         <state_interface name="effort"/>
       </joint>
-      <joint name="joint6">
+      <joint name="${prefix}joint6">
         <command_interface name="position"/>
         <state_interface name="position"/>
@@ -59,5 +60,5 @@
         <state_interface name="effort"/>
       </joint>
-      <joint name="gripper_joint">
+      <joint name="${prefix}gripper_joint">
         <command_interface name="position"/>
         <state_interface name="position"/>

File: manipulator/ARX/arx5_description/xacro/ros2_control/robot.xacro (robot description, xacro)
@@ -18,5 +18,5 @@
   <!-- Import R5 ros2_control description -->
   <xacro:include filename="$(find arx5_description)/xacro/ros2_control/arx5.ros2_control.xacro" />
-  <xacro:arx5_system name="ARX5System" ros2_control_hardware_type="$(arg ros2_control_hardware_type)"/>
+  <xacro:arx5_system name="" ros2_control_hardware_type="$(arg ros2_control_hardware_type)"/>
   <xacro:arg name="gazebo" default="false" />
   <xacro:if value="$(arg gazebo)">

Commit message: fix: isaac sim topic bug

File: manipulator/ARX/arx5_description/xacro/ros2_control/arx5.ros2_control.xacro (robot description, xacro)
@@ -13,5 +13,5 @@
         <xacro:if value="${ros2_control_hardware_type == 'isaac'}">
           <plugin>topic_based_ros2_control/TopicBasedSystem</plugin>
-          <param name="joint_commands_topic">/isaac/joint_commands</param>
+          <param name="joint_commands_topic">/isaac/joint_command</param>
           <param name="joint_states_topic">/isaac/joint_states</param>
         </xacro:if>

File: manipulator/AgileX/piper_description/xacro/ros2_control/piper.ros2_control.xacro (robot description, xacro)
@@ -13,5 +13,5 @@
         <xacro:if value="${ros2_control_hardware_type == 'isaac'}">
           <plugin>topic_based_ros2_control/TopicBasedSystem</plugin>
-          <param name="joint_commands_topic">/isaac/joint_commands</param>
+          <param name="joint_commands_topic">/isaac/joint_command</param>
           <param name="joint_states_topic">/isaac/joint_states</param>
         </xacro:if>

File: manipulator/Galaxea/galaxea_a1_description/xacro/ros2_control/galaxea_a1.ros2_control.xacro (robot description, xacro)
@@ -13,5 +13,5 @@
         <xacro:if value="${ros2_control_hardware_type == 'isaac'}">
           <plugin>topic_based_ros2_control/TopicBasedSystem</plugin>
-          <param name="joint_commands_topic">/isaac/joint_commands</param>
+          <param name="joint_commands_topic">/isaac/joint_command</param>
           <param name="joint_states_topic">/isaac/joint_states</param>
         </xacro:if>

File: manipulator/OpenArm/openarm_v10_description/urdf/openarm_v10_bimanual.urdf (robot description, URDF)
Before this commit: robot OpenArm, 26 links, 25 joints
Links:
- removed link body_link0
- link base_link: mass None -> 13.89; geometry collision mesh filename=package://openarm_v10_description/meshes/body/v10/collision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 scale=0.001 0.001 0.001; visual mesh filename=package://openarm_v10_description/meshes/body/v10/visual/bo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 scale=0.001 0.001 0.001
Joints:
- removed joint base_link_joint
- joint left_body_link0_joint: parent body_link0 -> base_link
- joint right_body_link0_joint: parent body_link0 -> base_link

File: manipulator/OpenArm/openarm_v10_description/urdf/openarm_v10_single.urdf (robot description, URDF)
Before this commit: robot OpenArm, 13 links, 12 joints
Links:
- removed link link0
- link base_link: mass None -> 1.1432284943239561; geometry collision mesh filename=package://openarm_v10_description/meshes/arm/v10/collision/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 scale=0.001 -0.001 0.001; visual mesh filename=package://openarm_v10_description/meshes/arm/v10/visual/lin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 scale=0.001 -0.001 0.001
Joints:
- removed joint base_link_joint
- joint joint1: parent link0 -> base_link

File: manipulator/OpenArm/openarm_v10_description/xacro/openarm_bimanual.xacro (robot description, xacro)
@@ -1,15 +1,15 @@
 <?xml version="1.0" encoding="utf-8"?>
 <robot xmlns:xacro="http://www.ros.org/wiki/xacro">
-  <xacro:macro name="OpenArm" params="name direction:=normal">
+  <xacro:macro name="openarm_bimanual" params="name direction:=normal">
     <xacro:property name="prefix" value="${name + '_' if name else ''}"/>
     <!-- Is the robot being simulated in gazebo? -->
     <!-- <xacro:arg name="gazebo" default="false" /> -->
-    <link name="${prefix}base_link"/>
+    <!-- <link name="${prefix}base_link"/>
     <joint name="${prefix}base_link_joint" type="fixed">
       <parent link="${prefix}base_link"/>
       <child link="${prefix}body_link0"/>
       <origin rpy="0 0 0" xyz="0 0 0"/>
-    </joint>
-    <link name="${prefix}body_link0">
+    </joint> -->
+    <link name="${prefix}base_link">
       <visual name="${prefix}body_link0_visual">
         <origin rpy="0.0 0.0 0.0" xyz="0.0 0.0 0.0"/>
@@ -32,5 +32,5 @@
     </link>
     <joint name="${prefix}left_opnarm_body_link0_joint" type="fixed">
-      <parent link="${prefix}body_link0"/>
+      <parent link="${prefix}base_link"/>
       <child link="${prefix}left_link0"/>
       <origin rpy="-1.5708 0 0" xyz="0.0 0.031 0.698"/>
@@ -252,5 +252,5 @@
       </joint> -->
     <joint name="${prefix}right_body_link0_joint" type="fixed">
-      <parent link="${prefix}body_link0"/>
+      <parent link="${prefix}base_link"/>
       <child link="${prefix}right_link0"/>
       <origin rpy="1.5708 0 0" xyz="0.0 -0.031 0.698"/>

File: manipulator/OpenArm/openarm_v10_description/xacro/openarm_single.xacro (robot description, xacro)
@@ -1,15 +1,15 @@
 <?xml version="1.0" encoding="utf-8"?>
 <robot xmlns:xacro="http://www.ros.org/wiki/xacro">
-  <xacro:macro name="OpenArm" params="name direction:=normal">
+  <xacro:macro name="openarm_single" params="name direction:=normal">
     <xacro:property name="prefix" value="${name + '_' if name else ''}"/>
     <!-- Is the robot being simulated in gazebo? -->
     <!-- <xacro:arg name="gazebo" default="false" /> -->
-    <link name="${prefix}base_link"/>
+    <!-- <link name="${prefix}base_link"/>
     <joint name="${prefix}base_link_joint" type="fixed">
       <parent link="${prefix}base_link"/>
       <child link="${prefix}link0"/>
       <origin rpy="0 0 0" xyz="0 0 0"/>
-    </joint>
-    <link name="${prefix}link0">
+    </joint> -->
+    <link name="${prefix}base_link">
       <visual name="${prefix}link0_visual">
         <origin rpy="0.0 0.0 0.0" xyz="0.0 0.0 0.0"/>
@@ -53,5 +53,5 @@
     <joint name="${prefix}joint1" type="revolute">
       <origin rpy="0 0 0" xyz="0.0 0.0 0.0625"/>
-      <parent link="${prefix}link0"/>
+      <parent link="${prefix}base_link"/>
       <child link="${prefix}link1"/>
       <axis xyz="0 0 1"/>

File: manipulator/OpenArm/openarm_v10_description/xacro/robot.xacro (robot description, xacro)
@@ -1,13 +1,13 @@
 <?xml version="1.0"?>
-<robot name="OpenArm" xmlns:xacro="http://www.ros.org/wiki/xacro">
+<robot name="openarm_single" xmlns:xacro="http://www.ros.org/wiki/xacro">
   <xacro:arg name="type" default="bimanual"/>
   <!-- 根据type参数决定机器人类型 -->
   <xacro:if value="${'$(arg type)' == 'bimanual'}">
     <xacro:include filename="$(find openarm_v10_description)/xacro/openarm_bimanual.xacro"/>
-    <xacro:OpenArm name=""/>
+    <xacro:openarm_bimanual name=""/>
   </xacro:if>
   <xacro:if value="${'$(arg type)' == 'single'}">
     <xacro:include filename="$(find openarm_v10_description)/xacro/openarm_single.xacro"/>
-    <xacro:OpenArm name=""/>
+    <xacro:openarm_single name=""/>
   </xacro:if>
 </robot>

File: manipulator/OpenArm/openarm_v10_description/xacro/ros2_control/openarm_bimanual.ros2_control.xacro (robot description, xacro)
@@ -14,6 +14,15 @@
         <xacro:if value="${ros2_control_hardware_type == 'isaac'}">
           <plugin>topic_based_ros2_control/TopicBasedSystem</plugin>
-          <param name="joint_commands_topic">/isaac/joint_commands</param>
+          <param name="joint_commands_topic">/isaac/joint_command</param>
           <param name="joint_states_topic">/isaac/joint_states</param>
+          <param name="sum_wrapped_joint_states">false</param>
+          <param name="initialize_commands_from_state">true</param>
+        </xacro:if>
+        <xacro:if value="${ros2_control_hardware_type == 'real'}">
+          <plugin>topic_based_ros2_control/TopicBasedSystem</plugin>
+          <param name="joint_commands_topic">/joint_command_robot</param>
+          <param name="joint_states_topic">/joint_states_robot</param>
+          <param name="sum_wrapped_joint_states">false</param>
+          <param name="initialize_commands_from_state">true</param>
         </xacro:if>
       </hardware>
@@ -79,5 +88,5 @@
         <xacro:if value="${ros2_control_hardware_type == 'isaac'}">
           <plugin>topic_based_ros2_control/TopicBasedSystem</plugin>
-          <param name="joint_commands_topic">/isaac/joint_commands</param>
+          <param name="joint_commands_topic">/isaac/joint_command</param>
           <param name="joint_states_topic">/isaac/joint_states</param>
         </xacro:if>

File: manipulator/OpenArm/openarm_v10_description/xacro/ros2_control/openarm_single.ros2_control.xacro (robot description, xacro)
@@ -13,6 +13,15 @@
         <xacro:if value="${ros2_control_hardware_type == 'isaac'}">
           <plugin>topic_based_ros2_control/TopicBasedSystem</plugin>
-          <param name="joint_commands_topic">/isaac/joint_commands</param>
+          <param name="joint_commands_topic">/isaac/joint_command</param>
           <param name="joint_states_topic">/isaac/joint_states</param>
+          <param name="sum_wrapped_joint_states">false</param>
+          <param name="initialize_commands_from_state">true</param>
+        </xacro:if>
+        <xacro:if value="${ros2_control_hardware_type == 'real'}">
+          <plugin>topic_based_ros2_control/TopicBasedSystem</plugin>
+          <param name="joint_commands_topic">/joint_command_robot</param>
+          <param name="joint_states_topic">/joint_states_robot</param>
+          <param name="sum_wrapped_joint_states">false</param>
+          <param name="initialize_commands_from_state">true</param>
         </xacro:if>
       </hardware>

File: manipulator/OpenArm/openarm_v10_description/xacro/ros2_control/robot.xacro (robot description, xacro)
@@ -11,9 +11,9 @@
   <xacro:if value="${'$(arg type)' == 'bimanual'}">
     <xacro:include filename="$(find openarm_v10_description)/xacro/openarm_bimanual.xacro"/>
-    <xacro:OpenArm name=""/>
+    <xacro:openarm_bimanual name=""/>
   </xacro:if>
   <xacro:if value="${'$(arg type)' == 'single'}">
     <xacro:include filename="$(find openarm_v10_description)/xacro/openarm_single.xacro"/>
-    <xacro:OpenArm name=""/>
+    <xacro:openarm_single name=""/>
   </xacro:if>
   <!-- 根据type参数决定ros2_control类型 -->
