Commit message: add galaxea r1 description

File: humanoid/Galaxea/galaxea_r1_description/xacro/ros2_control/galaxea_r1.ros2_control.xacro (robot description, xacro)
@@ -1,7 +1,6 @@
 <?xml version="1.0"?>
 <robot xmlns:xacro="http://www.ros.org/wiki/xacro">
-  <xacro:macro name="galaxea_a1_system" params="name ros2_control_hardware_type">
-    <xacro:property name="prefix" value="${name + '_' if name else ''}"/>
-    <ros2_control name="${prefix}galaxea_a1_system" type="system">
+  <xacro:macro name="galaxea_r1_system" params="ros2_control_hardware_type">
+    <ros2_control name="galaxea_r1_system" type="system">
       <hardware>
         <xacro:if value="${ros2_control_hardware_type == 'gz'}">
@@ -17,6 +16,5 @@
         </xacro:if>
       </hardware>
-      <!-- 关节接口定义 -->
-      <joint name="${prefix}joint1">
+      <joint name="torso_joint1">
         <command_interface name="position"/>
         <state_interface name="position"/>
@@ -24,5 +22,5 @@
         <state_interface name="effort"/>
       </joint>
-      <joint name="${prefix}joint2">
+      <joint name="torso_joint2">
         <command_interface name="position"/>
         <state_interface name="position"/>
@@ -30,5 +28,5 @@
         <state_interface name="effort"/>
       </joint>
-      <joint name="${prefix}joint3">
+      <joint name="torso_joint3">
         <command_interface name="position"/>
         <state_interface name="position"/>
@@ -36,5 +34,5 @@
         <state_interface name="effort"/>
       </joint>
-      <joint name="${prefix}joint4">
+      <joint name="torso_joint4">
         <command_interface name="position"/>
         <state_interface name="position"/>
@@ -42,21 +40,4 @@
         <state_interface name="effort"/>
       </joint>
-      <joint name="${prefix}joint5">
-        <command_interface name="position"/>
-        <state_interface name="position"/>
-        <state_interface name="velocity"/>
-        <state_interface name="effort"/>
-      </joint>
-      <joint name="${prefix}joint6">
-        <command_interface name="position"/>
-        <state_interface name="position"/>
-        <state_interface name="velocity"/>
-        <state_interface name="effort"/>
-      </joint>
-      <joint name="${prefix}gripper_joint">
-        <command_interface name="position"/>
-        <state_interface name="position"/>
-        <state_interface name="velocity"/>
-      </joint>
     </ros2_control>
   </xacro:macro>

File: humanoid/Galaxea/galaxea_r1_description/xacro/ros2_control/robot.xacro (robot description, xacro)
@@ -29,3 +29,22 @@
   <!-- Include Right RealSense Camera -->
   <xacro:RealSense side="right"/>
+  <link name="world"/>
+  <joint name="world_fixed" type="fixed">
+    <parent link="world"/>
+    <child link="base_link"/>
+  </joint>
+  <!-- Import Piper ros2_control description -->
+  <xacro:include filename="$(find galaxea_a1_description)/xacro/ros2_control/galaxea_a1.ros2_control.xacro" />
+  <xacro:galaxea_a1_system name="left" ros2_control_hardware_type="$(arg ros2_control_hardware_type)"/>
+  <xacro:galaxea_a1_system name="right" ros2_control_hardware_type="$(arg ros2_control_hardware_type)"/>
+  <xacro:include filename="$(find galaxea_r1_description)/xacro/ros2_control/galaxea_r1.ros2_control.xacro" />
+  <xacro:galaxea_r1_system ros2_control_hardware_type="$(arg ros2_control_hardware_type)"/>
+  <xacro:arg name="gazebo" default="false" />
+  <xacro:if value="$(arg gazebo)">
+    <gazebo>
+      <plugin filename="gz_ros2_control-system" name="gz_ros2_control::GazeboSimROS2ControlPlugin">
+        <parameters>$(find galaxea_r1_description)/config/ros2_control/ros2_controllers.yaml</parameters>
+      </plugin>
+    </gazebo>
+  </xacro:if>
 </robot>

Commit message: add wheel for galaxea r1 and agilex aloha

File: humanoid/Galaxea/galaxea_r1_description/xacro/ros2_control/galaxea_r1.ros2_control.xacro (robot description, xacro)
@@ -40,4 +40,46 @@
         <state_interface name="effort"/>
       </joint>
+      <joint name="steer_motor_joint1">
+        <command_interface name="position"/>
+        <state_interface name="position"/>
+        <state_interface name="velocity"/>
+        <state_interface name="effort"/>
+      </joint>
+      <joint name="steer_motor_joint2">
+        <command_interface name="position"/>
+        <state_interface name="position"/>
+        <state_interface name="velocity"/>
+        <state_interface name="effort"/>
+      </joint>
+      <joint name="steer_motor_joint3">
+        <command_interface name="position"/>
+        <state_interface name="position"/>
+        <state_interface name="velocity"/>
+        <state_interface name="effort"/>
+      </joint>
+      <joint name="wheel_motor_joint1">
+        <command_interface name="velocity">
+          <param name="min">-1</param>
+          <param name="max">1</param>
+        </command_interface>
+        <state_interface name="position"/>
+        <state_interface name="velocity"/>
+      </joint>
+      <joint name="wheel_motor_joint2">
+        <command_interface name="velocity">
+          <param name="min">-1</param>
+          <param name="max">1</param>
+        </command_interface>
+        <state_interface name="position"/>
+        <state_interface name="velocity"/>
+      </joint>
+      <joint name="wheel_motor_joint3">
+        <command_interface name="velocity">
+          <param name="min">-1</param>
+          <param name="max">1</param>
+        </command_interface>
+        <state_interface name="position"/>
+        <state_interface name="velocity"/>
+      </joint>
     </ros2_control>
   </xacro:macro>

File: humanoid/Galaxea/galaxea_r1_description/xacro/ros2_control/robot.xacro (robot description, xacro)
@@ -29,9 +29,4 @@
   <!-- Include Right RealSense Camera -->
   <xacro:RealSense side="right"/>
-  <link name="world"/>
-  <joint name="world_fixed" type="fixed">
-    <parent link="world"/>
-    <child link="base_link"/>
-  </joint>
   <!-- Import Piper ros2_control description -->
   <xacro:include filename="$(find galaxea_a1_description)/xacro/ros2_control/galaxea_a1.ros2_control.xacro" />

File: manipulator/AgileX/agilex_aloha_description/xacro/aloha_split.xacro (robot description, xacro)
@@ -27,5 +27,5 @@
   </link>
   <joint name="box_joint" type="fixed">
-    <parent link="base_link"/>
+    <parent link="base"/>
     <child link="box_link"/>
   </joint>

File: manipulator/AgileX/agilex_aloha_description/xacro/ros2_control/aloha_split.ros2_control.xacro (robot description, xacro)
@@ -17,6 +17,24 @@
       </hardware>
       <!-- 移动平台轮子关节 -->
-      <joint name="left_wheel">
-        <command_interface name="velocity"/>
+      <joint name="fl_steering_joint">
+        <command_interface name="position"/>
+        <state_interface name="position"/>
+        <state_interface name="velocity"/>
+        <state_interface name="effort"/>
+      </joint>
+      <joint name="fr_steering_joint">
+        <command_interface name="position"/>
+        <state_interface name="position"/>
+        <state_interface name="velocity"/>
+        <state_interface name="effort"/>
+      </joint>
+      <joint name="rl_steering_joint">
+        <command_interface name="position"/>
+        <state_interface name="position"/>
+        <state_interface name="velocity"/>
+        <state_interface name="effort"/>
+      </joint>
+      <joint name="rr_steering_joint">
+        <command_interface name="position"/>
         <state_interface name="position"/>
         <state_interface name="velocity"/>
@@ -30,26 +48,34 @@
       </joint>
       <joint name="fl_wheel">
-        <command_interface name="velocity"/>
+        <command_interface name="velocity">
+          <param name="min">-1</param>
+          <param name="max">1</param>
+        </command_interface>
         <state_interface name="position"/>
         <state_interface name="velocity"/>
-        <state_interface name="effort"/>
       </joint>
       <joint name="fr_wheel">
-        <command_interface name="velocity"/>
+        <command_interface name="velocity">
+          <param name="min">-1</param>
+          <param name="max">1</param>
+        </command_interface>
         <state_interface name="position"/>
         <state_interface name="velocity"/>
-        <state_interface name="effort"/>
       </joint>
       <joint name="rl_wheel">
-        <command_interface name="velocity"/>
+        <command_interface name="velocity">
+          <param name="min">-1</param>
+          <param name="max">1</param>
+        </command_interface>
         <state_interface name="position"/>
         <state_interface name="velocity"/>
-        <state_interface name="effort"/>
       </joint>
       <joint name="rr_wheel">
-        <command_interface name="velocity"/>
+        <command_interface name="velocity">
+          <param name="min">-1</param>
+          <param name="max">1</param>
+        </command_interface>
         <state_interface name="position"/>
         <state_interface name="velocity"/>
-        <state_interface name="effort"/>
       </joint>
       <!-- 升降机构关节 -->

File: manipulator/AgileX/agilex_aloha_description/xacro/ros2_control/robot.xacro (robot description, xacro)
@@ -2,9 +2,4 @@
 <robot xmlns:xacro="http://www.ros.org/wiki/xacro" name="AgileX Aloha">
   <xacro:arg name="ros2_control_hardware_type" default="mock_components" />
-  <link name="world"/>
-  <joint name="world_fixed" type="fixed">
-    <parent link="world"/>
-    <child link="base_footprint"/>
-  </joint>
   <!-- Import Piper ros2_control description -->
   <xacro:include filename="$(find piper_description)/xacro/ros2_control/piper.ros2_control.xacro" />

File: manipulator/Galaxea/galaxea_a1_description/xacro/a1.xacro (robot description, xacro)
@@ -57,5 +57,5 @@
       <child link="${prefix}link1"/>
       <axis xyz="0 0 1"/>
-      <limit lower="-2.8798" upper="2.8798" effort="40" velocity="20.944"/>
+      <limit lower="-2.8798" upper="2.8798" effort="100" velocity="20.944"/>
     </joint>
     <!-- Link 2 -->
@@ -89,5 +89,5 @@
       <child link="${prefix}link2"/>
       <axis xyz="0 0 -1"/>
-      <limit lower="0" upper="3.2289" effort="40" velocity="20.944"/>
+      <limit lower="0" upper="3.2289" effort="100" velocity="20.944"/>
     </joint>
     <!-- Link 3 -->
@@ -121,5 +121,5 @@
       <child link="${prefix}link3"/>
       <axis xyz="0 0 -1"/>
-      <limit lower="-3.3161" upper="0" effort="27" velocity="7.5398"/>
+      <limit lower="-3.3161" upper="0" effort="100" velocity="7.5398"/>
     </joint>
     <!-- Link 4 -->
@@ -153,5 +153,5 @@
       <child link="${prefix}link4"/>
       <axis xyz="1 0 0"/>
-      <limit lower="-2.8798" upper="2.8798" effort="7" velocity="25.133"/>
+      <limit lower="-2.8798" upper="2.8798" effort="100" velocity="25.133"/>
     </joint>
     <!-- Link 5 -->
@@ -185,5 +185,5 @@
       <child link="${prefix}link5"/>
       <axis xyz="0 1 0"/>
-      <limit lower="-1.6581" upper="1.6581" effort="7" velocity="25.133"/>
+      <limit lower="-1.6581" upper="1.6581" effort="100" velocity="25.133"/>
     </joint>
     <!-- Link 6 -->
@@ -217,5 +217,5 @@
       <child link="${prefix}link6"/>
       <axis xyz="1 0 0"/>
-      <limit lower="-2.8798" upper="2.8798" effort="7" velocity="25.133"/>
+      <limit lower="-2.8798" upper="2.8798" effort="100" velocity="25.133"/>
     </joint>
     <!-- Include Gripper -->
