Commit message: piper model simplified

File: manipulator/AgileX/piper_description/xacro/slave.xacro (robot description, xacro)
@@ -11,10 +11,20 @@
       <visual>
         <geometry>
-          <mesh filename="file://$(find piper_description)/meshes/link6.obj"/>
+          <mesh filename="file://$(find piper_description)/meshes/visual/link6.obj"/>
         </geometry>
       </visual>
       <collision>
         <geometry>
-          <mesh filename="file://$(find piper_description)/meshes/link6.obj"/>
+          <mesh filename="file://$(find piper_description)/meshes/collision/link6_collision_0.obj"/>
+        </geometry>
+      </collision>
+      <collision>
+        <geometry>
+          <mesh filename="file://$(find piper_description)/meshes/collision/link6_collision_1.obj"/>
+        </geometry>
+      </collision>
+      <collision>
+        <geometry>
+          <mesh filename="file://$(find piper_description)/meshes/collision/link6_collision_2.obj"/>
         </geometry>
       </collision>
@@ -22,5 +32,5 @@
     <link name="${prefix}link7">
       <inertial>
-        <origin xyz="0.00065123185041968 -0.0491929869131989 0.00972258769184025" rpy="0 0 0"/>
+        <origin xyz="0.00065123185041968 -0.0491929869131989 0.00972258769184025"/>
         <mass value="0.025"/>
         <inertia ixx="0.00007371" ixy="-0.00000113" ixz="0.00000021" iyy="0.00000781" iyz="-0.00001372"
@@ -29,10 +39,10 @@
       <visual>
         <geometry>
-          <mesh filename="file://$(find piper_description)/meshes/link7.obj"/>
+          <mesh filename="file://$(find piper_description)/meshes/visual/gripper.obj"/>
         </geometry>
       </visual>
       <collision>
         <geometry>
-          <mesh filename="file://$(find piper_description)/meshes/link7.obj"/>
+          <mesh filename="file://$(find piper_description)/meshes/collision/gripper.obj"/>
         </geometry>
       </collision>
@@ -54,10 +64,10 @@
       <visual>
         <geometry>
-          <mesh filename="file://$(find piper_description)/meshes/link8.obj"/>
+          <mesh filename="file://$(find piper_description)/meshes/visual/gripper.obj" scale="1 -1 1"/>
         </geometry>
       </visual>
       <collision>
         <geometry>
-          <mesh filename="file://$(find piper_description)/meshes/link8.obj"/>
+          <mesh filename="file://$(find piper_description)/meshes/collision/gripper.obj" scale="1 -1 1"/>
         </geometry>
       </collision>

Commit message: agilex modified

File: manipulator/AgileX/piper_description/xacro/slave.xacro (robot description, xacro)
@@ -89,5 +89,5 @@
     <link name="${prefix}camera"/>
     <joint name="${prefix}camera_fixed" type="fixed">
-      <origin xyz="-0.073 0 0.041" rpy="0 -1.22 0"/>
+      <origin xyz="-0.073 0 0.041" rpy="-0.3463 0 -1.5708"/>
       <parent link="${prefix}link6"/>
       <child link="${prefix}camera"/>
