Commit message: 初步拆分复用三种松灵机械臂piper,piper_x,piper_l

File: manipulator/AgileX/piper_description/xacro/Piper.xacro (robot description, xacro)
@@ -18,10 +18,10 @@
       <visual>
         <geometry>
-          <mesh filename="file://$(find piper_description)/meshes/visual/base_link.obj"/>
+          <mesh filename="file://$(find piper_description)/meshes/piper/base_link.obj"/>
         </geometry>
       </visual>
       <collision>
         <geometry>
-          <mesh filename="file://$(find piper_description)/meshes/collision/base_link.obj"/>
+          <mesh filename="file://$(find piper_description)/meshes/piper/base_link.obj"/>
         </geometry>
       </collision>
@@ -36,10 +36,10 @@
       <visual>
         <geometry>
-          <mesh filename="file://$(find piper_description)/meshes/visual/link1.obj"/>
+          <mesh filename="file://$(find piper_description)/meshes/piper/link1.obj"/>
         </geometry>
       </visual>
       <collision>
         <geometry>
-          <mesh filename="file://$(find piper_description)/meshes/collision/link1.obj"/>
+          <mesh filename="file://$(find piper_description)/meshes/piper/link1.obj"/>
         </geometry>
       </collision>
@@ -61,10 +61,10 @@
       <visual>
         <geometry>
-          <mesh filename="file://$(find piper_description)/meshes/visual/link2.obj"/>
+          <mesh filename="file://$(find piper_description)/meshes/piper/link2.obj"/>
         </geometry>
       </visual>
       <collision>
         <geometry>
-          <mesh filename="file://$(find piper_description)/meshes/collision/link2.obj"/>
+          <mesh filename="file://$(find piper_description)/meshes/piper/link2.obj"/>
         </geometry>
       </collision>
@@ -86,10 +86,10 @@
       <visual>
         <geometry>
-          <mesh filename="file://$(find piper_description)/meshes/visual/link3.obj"/>
+          <mesh filename="file://$(find piper_description)/meshes/piper/link3.obj"/>
         </geometry>
       </visual>
       <collision>
         <geometry>
-          <mesh filename="file://$(find piper_description)/meshes/collision/link3.obj"/>
+          <mesh filename="file://$(find piper_description)/meshes/piper/link3.obj"/>
         </geometry>
       </collision>
@@ -111,10 +111,10 @@
       <visual>
         <geometry>
-          <mesh filename="file://$(find piper_description)/meshes/visual/link4.obj"/>
+          <mesh filename="file://$(find piper_description)/meshes/piper/link4.obj"/>
         </geometry>
       </visual>
       <collision>
         <geometry>
-          <mesh filename="file://$(find piper_description)/meshes/collision/link4.obj"/>
+          <mesh filename="file://$(find piper_description)/meshes/piper/link4.obj"/>
         </geometry>
       </collision>
@@ -136,10 +136,10 @@
       <visual>
         <geometry>
-          <mesh filename="file://$(find piper_description)/meshes/visual/link5.obj"/>
+          <mesh filename="file://$(find piper_description)/meshes/piper/link5.obj"/>
         </geometry>
       </visual>
       <collision>
         <geometry>
-          <mesh filename="file://$(find piper_description)/meshes/collision/link5.obj"/>
+          <mesh filename="file://$(find piper_description)/meshes/piper/link5.obj"/>
         </geometry>
       </collision>

File: manipulator/AgileX/piper_description/xacro/robot.xacro (robot description, xacro)
@@ -1,12 +1,23 @@
 <?xml version="1.0"?>
-<robot name="Piper" xmlns:xacro="http://www.ros.org/wiki/xacro">
-  <xacro:arg name="type" default="slave"/>
-  <xacro:include filename="$(find piper_description)/xacro/Piper.xacro"/>
-  <!-- 根据type参数决定is_master的值 -->
-  <xacro:if value="${'$(arg type)' == 'master'}">
-    <xacro:Piper name="" is_master="true"/>
-  </xacro:if>
-  <xacro:unless value="${'$(arg type)' == 'master'}">
-    <xacro:Piper name="" is_master="false"/>
-  </xacro:unless>
+<robot name="piper" xmlns:xacro="http://www.ros.org/wiki/xacro">
+    <xacro:arg name="collider" default="convex"/>
+    <xacro:arg name="type" default="piper"/>
+    <xacro:arg name="style" default="slave"/>
+    <xacro:if value="${'$(arg type)' == 'piper'}">
+        <xacro:include filename="$(find piper_description)/xacro/piper_arm.xacro"/>
+        <xacro:if value="${'$(arg style)' == 'master'}">
+            <xacro:piper_arm name="" collider="$(arg collider)" is_master="true"/>
+        </xacro:if>
+        <xacro:if value="${'$(arg style)' == 'slave'}">
+            <xacro:piper_arm name="" collider="$(arg collider)" is_master="false"/>
+        </xacro:if>
+    </xacro:if>
+    <xacro:if value="${'$(arg type)' == 'piper_x'}">
+        <xacro:include filename="$(find piper_description)/xacro/piper_x_arm.xacro"/>
+        <xacro:piper_x_arm name="" collider="$(arg collider)"/>
+    </xacro:if>
+    <xacro:if value="${'$(arg type)' == 'piper_l'}">
+        <xacro:include filename="$(find piper_description)/xacro/piper_l_arm.xacro"/>
+        <xacro:piper_l_arm name="" collider="$(arg collider)"/>
+    </xacro:if>
 </robot>
