Commit message: gripper modified

File: gripper/changingtek_description/xacro/AG2F120S.xacro (robot description, xacro)
@@ -17,10 +17,10 @@
       <visual>
         <geometry>
-          <mesh filename="file://$(find changingtek_description)/meshes/AG2F120S/gripper_base.obj"/>
-        </geometry>
-      </visual>
-      <collision>
-        <geometry>
-          <mesh filename="file://$(find changingtek_description)/meshes/AG2F120S/gripper_base.obj"/>
+          <mesh filename="file://$(find changingtek_description)/meshes/AG2F120S/visual/gripper_base.obj"/>
+        </geometry>
+      </visual>
+      <collision>
+        <geometry>
+          <mesh filename="file://$(find changingtek_description)/meshes/AG2F120S/collision/gripper_base.obj"/>
         </geometry>
       </collision>
@@ -40,10 +40,10 @@
       <visual>
         <geometry>
-          <mesh filename="file://$(find changingtek_description)/meshes/AG2F120S/link_1.obj"/>
-        </geometry>
-      </visual>
-      <collision>
-        <geometry>
-          <mesh filename="file://$(find changingtek_description)/meshes/AG2F120S/link_1.obj"/>
+          <mesh filename="file://$(find changingtek_description)/meshes/AG2F120S/visual/link_1.obj"/>
+        </geometry>
+      </visual>
+      <collision>
+        <geometry>
+          <mesh filename="file://$(find changingtek_description)/meshes/AG2F120S/collision/link_1.obj"/>
         </geometry>
       </collision>
@@ -54,5 +54,5 @@
       <child link="${prefix}left_1_link"/>
       <axis xyz="0 0 -1"/>
-      <limit lower="0" upper="1" effort="2" velocity="1000"/>
+      <limit lower="0" upper="1" effort="40" velocity="4.1887902047863905"/>
     </joint>
     <link name="${prefix}left_support_link">
@@ -70,10 +70,10 @@
       <visual>
         <geometry>
-          <mesh filename="file://$(find changingtek_description)/meshes/AG2F120S/support_link.obj"/>
-        </geometry>
-      </visual>
-      <collision>
-        <geometry>
-          <mesh filename="file://$(find changingtek_description)/meshes/AG2F120S/support_link.obj"/>
+          <mesh filename="file://$(find changingtek_description)/meshes/AG2F120S/visual/support_link.obj"/>
+        </geometry>
+      </visual>
+      <collision>
+        <geometry>
+          <mesh filename="file://$(find changingtek_description)/meshes/AG2F120S/collision/support_link.obj"/>
         </geometry>
       </collision>
@@ -84,5 +84,5 @@
       <child link="${prefix}left_support_link"/>
       <axis xyz="0 0 1"/>
-      <limit lower="0" upper="0" effort="0" velocity="0"/>
+      <limit lower="0" upper="1" effort="40"  velocity="4.1887902047863905"/>
       <mimic joint="${prefix}gripper_joint" multiplier="1" offset="0"/>
     </joint>
@@ -101,10 +101,10 @@
       <visual>
         <geometry>
-          <mesh filename="file://$(find changingtek_description)/meshes/AG2F120S/pad_link.obj"/>
-        </geometry>
-      </visual>
-      <collision>
-        <geometry>
-          <mesh filename="file://$(find changingtek_description)/meshes/AG2F120S/pad_link.obj"/>
+          <mesh filename="file://$(find changingtek_description)/meshes/AG2F120S/visual/pad_link.obj"/>
+        </geometry>
+      </visual>
+      <collision>
+        <geometry>
+          <mesh filename="file://$(find changingtek_description)/meshes/AG2F120S/collision/pad_link.obj"/>
         </geometry>
       </collision>
@@ -129,10 +129,10 @@
       <visual>
         <geometry>
-          <mesh filename="file://$(find changingtek_description)/meshes/AG2F120S/link_2.obj"/>
-        </geometry>
-      </visual>
-      <collision>
-        <geometry>
-          <mesh filename="file://$(find changingtek_description)/meshes/AG2F120S/link_2.obj"/>
+          <mesh filename="file://$(find changingtek_description)/meshes/AG2F120S/visual/link_2.obj"/>
+        </geometry>
+      </visual>
+      <collision>
+        <geometry>
+          <mesh filename="file://$(find changingtek_description)/meshes/AG2F120S/collision/link_2.obj"/>
         </geometry>
       </collision>
@@ -143,5 +143,5 @@
       <child link="${prefix}left_2_link"/>
       <axis xyz="0 0 -1"/>
-      <limit lower="0" upper="0" effort="0" velocity="0"/>
+      <limit lower="0" upper="1" effort="40"  velocity="4.1887902047863905"/>
       <mimic joint="${prefix}gripper_joint" multiplier="1" offset="0"/>
     </joint>
@@ -160,10 +160,10 @@
       <visual>
         <geometry>
-          <mesh filename="file://$(find changingtek_description)/meshes/AG2F120S/link_2.obj"/>
-        </geometry>
-      </visual>
-      <collision>
-        <geometry>
-          <mesh filename="file://$(find changingtek_description)/meshes/AG2F120S/link_2.obj"/>
+          <mesh filename="file://$(find changingtek_description)/meshes/AG2F120S/visual/link_2.obj"/>
+        </geometry>
+      </visual>
+      <collision>
+        <geometry>
+          <mesh filename="file://$(find changingtek_description)/meshes/AG2F120S/collision/link_2.obj"/>
         </geometry>
       </collision>
@@ -174,5 +174,5 @@
       <child link="${prefix}right_2_link"/>
       <axis xyz="0 0 1"/>
-      <limit lower="0" upper="0" effort="0" velocity="0"/>
+      <limit lower="0" upper="1" effort="40"  velocity="4.1887902047863905"/>
       <mimic joint="${prefix}left_2_joint" multiplier="-1" offset="0"/>
     </joint>
@@ -191,10 +191,10 @@
       <visual>
         <geometry>
-          <mesh filename="file://$(find changingtek_description)/meshes/AG2F120S/link_1.obj"/>
-        </geometry>
-      </visual>
-      <collision>
-        <geometry>
-          <mesh filename="file://$(find changingtek_description)/meshes/AG2F120S/link_1.obj"/>
+          <mesh filename="file://$(find changingtek_description)/meshes/AG2F120S/visual/link_1.obj"/>
+        </geometry>
+      </visual>
+      <collision>
+        <geometry>
+          <mesh filename="file://$(find changingtek_description)/meshes/AG2F120S/collision/link_1.obj"/>
         </geometry>
       </collision>
@@ -205,5 +205,5 @@
       <child link="${prefix}right_1_link"/>
       <axis xyz="0 0 1"/>
-      <limit lower="0" upper="0" effort="0" velocity="0"/>
+      <limit lower="0" upper="1" effort="40"  velocity="4.1887902047863905"/>
       <mimic joint="${prefix}gripper_joint" multiplier="-1" offset="0"/>
     </joint>
@@ -222,10 +222,10 @@
       <visual>
         <geometry>
-          <mesh filename="file://$(find changingtek_description)/meshes/AG2F120S/support_link.obj"/>
-        </geometry>
-      </visual>
-      <collision>
-        <geometry>
-          <mesh filename="file://$(find changingtek_description)/meshes/AG2F120S/support_link.obj"/>
+          <mesh filename="file://$(find changingtek_description)/meshes/AG2F120S/visual/support_link.obj"/>
+        </geometry>
+      </visual>
+      <collision>
+        <geometry>
+          <mesh filename="file://$(find changingtek_description)/meshes/AG2F120S/collision/support_link.obj"/>
         </geometry>
       </collision>
@@ -236,5 +236,5 @@
       <child link="${prefix}right_support_link"/>
       <axis xyz="0 0 1"/>
-      <limit lower="0" upper="0" effort="0" velocity="0"/>
+      <limit lower="0" upper="1" effort="40"  velocity="4.1887902047863905"/>
       <mimic joint="${prefix}right_1_joint" multiplier="-1" offset="0"/>
     </joint>
@@ -253,10 +253,10 @@
       <visual>
         <geometry>
-          <mesh filename="file://$(find changingtek_description)/meshes/AG2F120S/pad_link.obj"/>
-        </geometry>
-      </visual>
-      <collision>
-        <geometry>
-          <mesh filename="file://$(find changingtek_description)/meshes/AG2F120S/pad_link.obj"/>
+          <mesh filename="file://$(find changingtek_description)/meshes/AG2F120S/visual/pad_link.obj"/>
+        </geometry>
+      </visual>
+      <collision>
+        <geometry>
+          <mesh filename="file://$(find changingtek_description)/meshes/AG2F120S/collision/pad_link.obj"/>
         </geometry>
       </collision>

File: gripper/changingtek_description/xacro/AG2F90-C.xacro (robot description, xacro)
@@ -17,10 +17,10 @@
       <visual>
         <geometry>
-          <mesh filename="file://$(find changingtek_description)/meshes/AG2F90-C/gripper_base.obj"/>
-        </geometry>
-      </visual>
-      <collision>
-        <geometry>
-          <mesh filename="file://$(find changingtek_description)/meshes/AG2F90-C/gripper_base.obj"/>
+          <mesh filename="file://$(find changingtek_description)/meshes/AG2F90-C/visual/gripper_base.obj"/>
+        </geometry>
+      </visual>
+      <collision>
+        <geometry>
+          <mesh filename="file://$(find changingtek_description)/meshes/AG2F90-C/collision/gripper_base.obj"/>
         </geometry>
       </collision>
@@ -40,10 +40,10 @@
       <visual>
         <geometry>
-          <mesh filename="file://$(find changingtek_description)/meshes/AG2F90-C/link_1.obj"/>
-        </geometry>
-      </visual>
-      <collision>
-        <geometry>
-          <mesh filename="file://$(find changingtek_description)/meshes/AG2F90-C/link_1.obj"/>
+          <mesh filename="file://$(find changingtek_description)/meshes/AG2F90-C/visual/link_1.obj"/>
+        </geometry>
+      </visual>
+      <collision>
+        <geometry>
+          <mesh filename="file://$(find changingtek_description)/meshes/AG2F90-C/collision/link_1.obj"/>
         </geometry>
       </collision>
@@ -54,5 +54,5 @@
       <child link="${prefix}left_1_link"/>
       <axis xyz="1 0 0"/>
-      <limit lower="0" upper="1" effort="10"  velocity="4.1887902047863905"/>
+      <limit lower="0" upper="1" effort="25"  velocity="4.1887902047863905"/>
     </joint>
     <link name="${prefix}left_in_link">
@@ -70,10 +70,10 @@
       <visual>
         <geometry>
-          <mesh filename="file://$(find changingtek_description)/meshes/AG2F90-C/in_link.obj"/>
-        </geometry>
-      </visual>
-      <collision>
-        <geometry>
-          <mesh filename="file://$(find changingtek_description)/meshes/AG2F90-C/in_link.obj"/>
+          <mesh filename="file://$(find changingtek_description)/meshes/AG2F90-C/visual/in_link.obj"/>
+        </geometry>
+      </visual>
+      <collision>
+        <geometry>
+          <mesh filename="file://$(find changingtek_description)/meshes/AG2F90-C/collision/in_link.obj"/>
         </geometry>
       </collision>
@@ -101,10 +101,10 @@
       <visual>
         <geometry>
-          <mesh filename="file://$(find changingtek_description)/meshes/AG2F90-C/up_link.obj"/>
-        </geometry>
-      </visual>
-      <collision>
-        <geometry>
-          <mesh filename="file://$(find changingtek_description)/meshes/AG2F90-C/up_link.obj"/>
+          <mesh filename="file://$(find changingtek_description)/meshes/AG2F90-C/visual/up_link.obj"/>
+        </geometry>
+      </visual>
+      <collision>
+        <geometry>
+          <mesh filename="file://$(find changingtek_description)/meshes/AG2F90-C/collision/up_link.obj"/>
         </geometry>
       </collision>
@@ -132,10 +132,10 @@
       <visual>
         <geometry>
-          <mesh filename="file://$(find changingtek_description)/meshes/AG2F90-C/pad_link.obj"/>
-        </geometry>
-      </visual>
-      <collision>
-        <geometry>
-          <mesh filename="file://$(find changingtek_description)/meshes/AG2F90-C/pad_link.obj"/>
+          <mesh filename="file://$(find changingtek_description)/meshes/AG2F90-C/visual/pad_link.obj"/>
+        </geometry>
+      </visual>
+      <collision>
+        <geometry>
+          <mesh filename="file://$(find changingtek_description)/meshes/AG2F90-C/collision/pad_link.obj"/>
         </geometry>
       </collision>
@@ -160,10 +160,10 @@
       <visual>
         <geometry>
-          <mesh filename="file://$(find changingtek_description)/meshes/AG2F90-C/link_2.obj"/>
-        </geometry>
-      </visual>
-      <collision>
-        <geometry>
-          <mesh filename="file://$(find changingtek_description)/meshes/AG2F90-C/link_2.obj"/>
+          <mesh filename="file://$(find changingtek_description)/meshes/AG2F90-C/visual/link_2.obj"/>
+        </geometry>
+      </visual>
+      <collision>
+        <geometry>
+          <mesh filename="file://$(find changingtek_description)/meshes/AG2F90-C/collision/link_2.obj"/>
         </geometry>
       </collision>
@@ -191,10 +191,10 @@
       <visual>
         <geometry>
-          <mesh filename="file://$(find changingtek_description)/meshes/AG2F90-C/link_2.obj"/>
-        </geometry>
-      </visual>
-      <collision>
-        <geometry>
-          <mesh filename="file://$(find changingtek_description)/meshes/AG2F90-C/link_2.obj"/>
+          <mesh filename="file://$(find changingtek_description)/meshes/AG2F90-C/visual/link_2.obj"/>
+        </geometry>
+      </visual>
+      <collision>
+        <geometry>
+          <mesh filename="file://$(find changingtek_description)/meshes/AG2F90-C/collision/link_2.obj"/>
         </geometry>
       </collision>
@@ -222,10 +222,10 @@
       <visual>
         <geometry>
-          <mesh filename="file://$(find changingtek_description)/meshes/AG2F90-C/link_1.obj"/>
-        </geometry>
-      </visual>
-      <collision>
-        <geometry>
-          <mesh filename="file://$(find changingtek_description)/meshes/AG2F90-C/link_1.obj"/>
+          <mesh filename="file://$(find changingtek_description)/meshes/AG2F90-C/visual/link_1.obj"/>
+        </geometry>
+      </visual>
+      <collision>
+        <geometry>
+          <mesh filename="file://$(find changingtek_description)/meshes/AG2F90-C/collision/link_1.obj"/>
         </geometry>
       </collision>
@@ -253,10 +253,10 @@
       <visual>
         <geometry>
-          <mesh filename="file://$(find changingtek_description)/meshes/AG2F90-C/in_link.obj"/>
-        </geometry>
-      </visual>
-      <collision>
-        <geometry>
-          <mesh filename="file://$(find changingtek_description)/meshes/AG2F90-C/in_link.obj"/>
+          <mesh filename="file://$(find changingtek_description)/meshes/AG2F90-C/visual/in_link.obj"/>
+        </geometry>
+      </visual>
+      <collision>
+        <geometry>
+          <mesh filename="file://$(find changingtek_description)/meshes/AG2F90-C/collision/in_link.obj"/>
         </geometry>
       </collision>
@@ -284,10 +284,10 @@
       <visual>
         <geometry>
-          <mesh filename="file://$(find changingtek_description)/meshes/AG2F90-C/up_link.obj"/>
-        </geometry>
-      </visual>
-      <collision>
-        <geometry>
-          <mesh filename="file://$(find changingtek_description)/meshes/AG2F90-C/up_link.obj"/>
+          <mesh filename="file://$(find changingtek_description)/meshes/AG2F90-C/visual/up_link.obj"/>
+        </geometry>
+      </visual>
+      <collision>
+        <geometry>
+          <mesh filename="file://$(find changingtek_description)/meshes/AG2F90-C/collision/up_link.obj"/>
         </geometry>
       </collision>
@@ -315,10 +315,10 @@
       <visual>
         <geometry>
-          <mesh filename="file://$(find changingtek_description)/meshes/AG2F90-C/pad_link.obj"/>
-        </geometry>
-      </visual>
-      <collision>
-        <geometry>
-          <mesh filename="file://$(find changingtek_description)/meshes/AG2F90-C/pad_link.obj"/>
+          <mesh filename="file://$(find changingtek_description)/meshes/AG2F90-C/visual/pad_link.obj"/>
+        </geometry>
+      </visual>
+      <collision>
+        <geometry>
+          <mesh filename="file://$(find changingtek_description)/meshes/AG2F90-C/collision/pad_link.obj"/>
         </geometry>
       </collision>

File: gripper/changingtek_description/xacro/ros2_control/2f.ros2_control.xacro (robot description, xacro)
@@ -23,4 +23,5 @@
         </state_interface>
         <state_interface name="velocity"/>
+        <state_interface name="effort"/>
       </joint>
     </ros2_control>

File: manipulator/Galaxea/galaxea_a1_description/xacro/a1.xacro (robot description, xacro)
@@ -220,5 +220,5 @@
     </joint>
     <!-- Include Gripper -->
-    <xacro:include filename="$(find galaxea_a1_description)/xacro/gripper.xacro"/>
+    <xacro:include filename="$(find galaxea_a1_description)/xacro/gripper_g1.xacro"/>
     <xacro:Gripper name="${name}"/>
     <!-- Gripper Properties -->
