Commit message: add unitree g1 with brainco revo2

File: dexhands/brainco_description/xacro/hand.xacro (robot description, xacro)
@@ -5,4 +5,4 @@
 	<xacro:include filename="$(find brainco_description)/xacro/revo2.xacro"/>
 	<!-- 创建左手 (direction=1) -->
-	<xacro:BraincoGripper name="" direction="$(arg direction)"/>
+	<xacro:BrainCoHand name="" direction="$(arg direction)"/>
 </robot>

File: dexhands/brainco_description/xacro/revo2.xacro (robot description, xacro)
@@ -1,5 +1,5 @@
 <?xml version="1.0" encoding="utf-8"?>
 <robot xmlns:xacro="http://www.ros.org/wiki/xacro">
-	<xacro:macro name="BraincoGripper" params="name direction:=1">
+	<xacro:macro name="BrainCoHand" params="name direction:=1">
 		<xacro:property name="prefix" value="${name + '_' if name else ''}"/>
 		<link name="${prefix}hand_base">
