Commit message: fix: openarm_single.xacro error

File: manipulator/OpenArm/openarm_v10_description/xacro/openarm_single.xacro (robot description, xacro)
@@ -9,5 +9,5 @@
         <origin rpy="0.0 0.0 0.0" xyz="0.0 0.0 0.0"/>
         <geometry>
-          <mesh filename="file://$(find openarm_v10_description/meshes/arm/v10/visual/link0.dae" scale="0.001 -0.001 0.001"/>
+          <mesh filename="file://$(find openarm_v10_description)/meshes/arm/v10/visual/link0.stl" scale="0.001 -0.001 0.001"/>
         </geometry>
       </visual>
@@ -15,6 +15,6 @@
         <origin rpy="0.0 0.0 0.0" xyz="0.0 0.0 0.0"/>
         <geometry>
-          <mesh filename="file://$(find openarm_v10_description/meshes/arm/v10/collision/link0_symp.stl" scale="0.001 -0.001 0.001"/>
-          <!-- <mesh filename="file://$(find openarm_v10_description/meshes/arm/${arm_type}/collision/${name}.stl" scale="0.001 0.001 0.001" /> -->
+          <mesh filename="file://$(find openarm_v10_description)/meshes/arm/v10/collision/link0_symp.stl" scale="0.001 -0.001 0.001"/>
+          <!-- <mesh filename="file://$(find openarm_v10_description)/meshes/arm/${arm_type}/collision/${name}.stl" scale="0.001 0.001 0.001" /> -->
         </geometry>
       </collision>
@@ -29,5 +29,5 @@
         <origin rpy="0.0 0.0 0.0" xyz="-0.0 0.0 -0.0625"/>
         <geometry>
-          <mesh filename="file://$(find openarm_v10_description/meshes/arm/v10/visual/link1.dae" scale="0.001 -0.001 0.001"/>
+          <mesh filename="file://$(find openarm_v10_description)/meshes/arm/v10/visual/link1.dae" scale="0.001 -0.001 0.001"/>
         </geometry>
       </visual>
@@ -35,6 +35,6 @@
         <origin rpy="0.0 0.0 0.0" xyz="-0.0 0.0 -0.0625"/>
         <geometry>
-          <mesh filename="file://$(find openarm_v10_description/meshes/arm/v10/collision/link1_symp.stl" scale="0.001 -0.001 0.001"/>
-          <!-- <mesh filename="file://$(find openarm_v10_description/meshes/arm/${arm_type}/collision/${name}.stl" scale="0.001 0.001 0.001" /> -->
+          <mesh filename="file://$(find openarm_v10_description)/meshes/arm/v10/collision/link1_symp.stl" scale="0.001 -0.001 0.001"/>
+          <!-- <mesh filename="file://$(find openarm_v10_description)/meshes/arm/${arm_type}/collision/${name}.stl" scale="0.001 0.001 0.001" /> -->
         </geometry>
       </collision>
@@ -56,5 +56,5 @@
         <origin rpy="0.0 0.0 0.0" xyz="0.0301 0.0 -0.1225"/>
         <geometry>
-          <mesh filename="file://$(find openarm_v10_description/meshes/arm/v10/visual/link2.dae" scale="0.001 -0.001 0.001"/>
+          <mesh filename="file://$(find openarm_v10_description)/meshes/arm/v10/visual/link2.dae" scale="0.001 -0.001 0.001"/>
         </geometry>
       </visual>
@@ -62,6 +62,6 @@
         <origin rpy="0.0 0.0 0.0" xyz="0.0301 0.0 -0.1225"/>
         <geometry>
-          <mesh filename="file://$(find openarm_v10_description/meshes/arm/v10/collision/link2_symp.stl" scale="0.001 -0.001 0.001"/>
-          <!-- <mesh filename="file://$(find openarm_v10_description/meshes/arm/${arm_type}/collision/${name}.stl" scale="0.001 0.001 0.001" /> -->
+          <mesh filename="file://$(find openarm_v10_description)/meshes/arm/v10/collision/link2_symp.stl" scale="0.001 -0.001 0.001"/>
+          <!-- <mesh filename="file://$(find openarm_v10_description)/meshes/arm/${arm_type}/collision/${name}.stl" scale="0.001 0.001 0.001" /> -->
         </geometry>
       </collision>
@@ -83,5 +83,5 @@
         <origin rpy="0.0 0.0 0.0" xyz="-0.0 -0.0 -0.18875"/>
         <geometry>
-          <mesh filename="file://$(find openarm_v10_description/meshes/arm/v10/visual/link3.dae" scale="0.001 -0.001 0.001"/>
+          <mesh filename="file://$(find openarm_v10_description)/meshes/arm/v10/visual/link3.dae" scale="0.001 -0.001 0.001"/>
         </geometry>
       </visual>
@@ -89,6 +89,6 @@
         <origin rpy="0.0 0.0 0.0" xyz="-0.0 -0.0 -0.18875"/>
         <geometry>
-          <mesh filename="file://$(find openarm_v10_description/meshes/arm/v10/collision/link3_symp.stl" scale="0.001 -0.001 0.001"/>
-          <!-- <mesh filename="file://$(find openarm_v10_description/meshes/arm/${arm_type}/collision/${name}.stl" scale="0.001 0.001 0.001" /> -->
+          <mesh filename="file://$(find openarm_v10_description)/meshes/arm/v10/collision/link3_symp.stl" scale="0.001 -0.001 0.001"/>
+          <!-- <mesh filename="file://$(find openarm_v10_description)/meshes/arm/${arm_type}/collision/${name}.stl" scale="0.001 0.001 0.001" /> -->
         </geometry>
       </collision>
@@ -110,5 +110,5 @@
         <origin rpy="0.0 0.0 0.0" xyz="0.0 -0.0315 -0.3425"/>
         <geometry>
-          <mesh filename="file://$(find openarm_v10_description/meshes/arm/v10/visual/link4.dae" scale="0.001 0.001 0.001"/>
+          <mesh filename="file://$(find openarm_v10_description)/meshes/arm/v10/visual/link4.dae" scale="0.001 0.001 0.001"/>
         </geometry>
       </visual>
@@ -116,6 +116,6 @@
         <origin rpy="0.0 0.0 0.0" xyz="0.0 -0.0315 -0.3425"/>
         <geometry>
-          <mesh filename="file://$(find openarm_v10_description/meshes/arm/v10/collision/link4_symp.stl" scale="0.001 0.001 0.001"/>
-          <!-- <mesh filename="file://$(find openarm_v10_description/meshes/arm/${arm_type}/collision/${name}.stl" scale="0.001 0.001 0.001" /> -->
+          <mesh filename="file://$(find openarm_v10_description)/meshes/arm/v10/collision/link4_symp.stl" scale="0.001 0.001 0.001"/>
+          <!-- <mesh filename="file://$(find openarm_v10_description)/meshes/arm/${arm_type}/collision/${name}.stl" scale="0.001 0.001 0.001" /> -->
         </geometry>
       </collision>
@@ -137,5 +137,5 @@
         <origin rpy="0.0 0.0 0.0" xyz="-0.0 -0.0 -0.438"/>
         <geometry>
-          <mesh filename="file://$(find openarm_v10_description/meshes/arm/v10/visual/link5.dae" scale="0.001 -0.001 0.001"/>
+          <mesh filename="file://$(find openarm_v10_description)/meshes/arm/v10/visual/link5.dae" scale="0.001 -0.001 0.001"/>
         </geometry>
       </visual>
@@ -143,6 +143,6 @@
         <origin rpy="0.0 0.0 0.0" xyz="-0.0 -0.0 -0.438"/>
         <geometry>
-          <mesh filename="file://$(find openarm_v10_description/meshes/arm/v10/collision/link5_symp.stl" scale="0.001 -0.001 0.001"/>
-          <!-- <mesh filename="file://$(find openarm_v10_description/meshes/arm/${arm_type}/collision/${name}.stl" scale="0.001 0.001 0.001" /> -->
+          <mesh filename="file://$(find openarm_v10_description)/meshes/arm/v10/collision/link5_symp.stl" scale="0.001 -0.001 0.001"/>
+          <!-- <mesh filename="file://$(find openarm_v10_description)/meshes/arm/${arm_type}/collision/${name}.stl" scale="0.001 0.001 0.001" /> -->
         </geometry>
       </collision>
@@ -164,5 +164,5 @@
         <origin rpy="0.0 0.0 0.0" xyz="-0.0375 -0.0 -0.5585"/>
         <geometry>
-          <mesh filename="file://$(find openarm_v10_description/meshes/arm/v10/visual/link6.dae" scale="0.001 -0.001 0.001"/>
+          <mesh filename="file://$(find openarm_v10_description)/meshes/arm/v10/visual/link6.dae" scale="0.001 -0.001 0.001"/>
         </geometry>
       </visual>
@@ -170,6 +170,6 @@
         <origin rpy="0.0 0.0 0.0" xyz="-0.0375 -0.0 -0.5585"/>
         <geometry>
-          <mesh filename="file://$(find openarm_v10_description/meshes/arm/v10/collision/link6_symp.stl" scale="0.001 -0.001 0.001"/>
-          <!-- <mesh filename="file://$(find openarm_v10_description/meshes/arm/${arm_type}/collision/${name}.stl" scale="0.001 0.001 0.001" /> -->
+          <mesh filename="file://$(find openarm_v10_description)/meshes/arm/v10/collision/link6_symp.stl" scale="0.001 -0.001 0.001"/>
+          <!-- <mesh filename="file://$(find openarm_v10_description)/meshes/arm/${arm_type}/collision/${name}.stl" scale="0.001 0.001 0.001" /> -->
         </geometry>
       </collision>
@@ -191,5 +191,5 @@
         <origin rpy="0.0 0.0 0.0" xyz="0.0 -0.0 -0.5585"/>
         <geometry>
-          <mesh filename="file://$(find openarm_v10_description/meshes/arm/v10/visual/link7.dae" scale="0.001 -0.001 0.001"/>
+          <mesh filename="file://$(find openarm_v10_description)/meshes/arm/v10/visual/link7.dae" scale="0.001 -0.001 0.001"/>
         </geometry>
       </visual>
@@ -197,6 +197,6 @@
         <origin rpy="0.0 0.0 0.0" xyz="0.0 -0.0 -0.5585"/>
         <geometry>
-          <mesh filename="file://$(find openarm_v10_description/meshes/arm/v10/collision/link7_symp.stl" scale="0.001 -0.001 0.001"/>
-          <!-- <mesh filename="file://$(find openarm_v10_description/meshes/arm/${arm_type}/collision/${name}.stl" scale="0.001 0.001 0.001" /> -->
+          <mesh filename="file://$(find openarm_v10_description)/meshes/arm/v10/collision/link7_symp.stl" scale="0.001 -0.001 0.001"/>
+          <!-- <mesh filename="file://$(find openarm_v10_description)/meshes/arm/${arm_type}/collision/${name}.stl" scale="0.001 0.001 0.001" /> -->
         </geometry>
       </collision>
@@ -224,5 +224,5 @@
         <origin rpy="0.0 0.0 0.0" xyz="0.0 0.0 -0.6585"/>
         <geometry>
-          <mesh filename="file://$(find openarm_v10_description/meshes/ee/openarm_hand/visual/hand.dae" scale="0.001 0.001 0.001"/>
+          <mesh filename="file://$(find openarm_v10_description)/meshes/ee/openarm_hand/visual/hand.dae" scale="0.001 0.001 0.001"/>
         </geometry>
       </visual>
@@ -230,5 +230,5 @@
         <origin rpy="0.0 0.0 0.0" xyz="0.0 0.0 -0.6585"/>
         <geometry>
-          <mesh filename="file://$(find openarm_v10_description/meshes/ee/openarm_hand/collision/hand.stl" scale="0.001 0.001 0.001"/>
+          <mesh filename="file://$(find openarm_v10_description)/meshes/ee/openarm_hand/collision/hand.stl" scale="0.001 0.001 0.001"/>
         </geometry>
       </collision>
@@ -257,5 +257,5 @@
         <origin rpy="0.0 0.0 0.0" xyz="0.0 -0.05 -0.673001"/>
         <geometry>
-          <mesh filename="file://$(find openarm_v10_description/meshes/ee/openarm_hand/visual/finger.dae" scale="0.001 0.001 0.001"/>
+          <mesh filename="file://$(find openarm_v10_description)/meshes/ee/openarm_hand/visual/finger.dae" scale="0.001 0.001 0.001"/>
         </geometry>
       </visual>
@@ -263,5 +263,5 @@
         <origin rpy="0.0 0.0 0.0" xyz="0.0 -0.05 -0.673001"/>
         <geometry>
-          <mesh filename="file://$(find openarm_v10_description/meshes/ee/openarm_hand/collision/finger.stl" scale="0.001 0.001 0.001"/>
+          <mesh filename="file://$(find openarm_v10_description)/meshes/ee/openarm_hand/collision/finger.stl" scale="0.001 0.001 0.001"/>
         </geometry>
       </collision>
@@ -276,5 +276,5 @@
         <origin rpy="0.0 0.0 0.0" xyz="0.0 0.05 -0.673001"/>
         <geometry>
-          <mesh filename="file://$(find openarm_v10_description/meshes/ee/openarm_hand/visual/finger.dae" scale="0.001 -0.001 0.001"/>
+          <mesh filename="file://$(find openarm_v10_description)/meshes/ee/openarm_hand/visual/finger.dae" scale="0.001 -0.001 0.001"/>
         </geometry>
       </visual>
@@ -282,5 +282,5 @@
         <origin rpy="0.0 0.0 0.0" xyz="0.0 0.05 -0.673001"/>
         <geometry>
-          <mesh filename="file://$(find openarm_v10_description/meshes/ee/openarm_hand/collision/finger.stl" scale="0.001 -0.001 0.001"/>
+          <mesh filename="file://$(find openarm_v10_description)/meshes/ee/openarm_hand/collision/finger.stl" scale="0.001 -0.001 0.001"/>
         </geometry>
       </collision>
