Commit message: add: test on rviz2 have error on finger inertia value

File: manipulator/OpenArm/openarm_v10_description/xacro/openarm_bimanual.xacro (robot description, xacro)
@@ -15,5 +15,5 @@
         <origin rpy="0.0 0.0 0.0" xyz="0.0 0.0 0.0"/>
         <geometry>
-          <mesh filename="file://$(find openarm_v10_description/meshes/body/v10/visual/body_link0.dae" scale="0.001 0.001 0.001"/>
+          <mesh filename="file://$(find openarm_v10_description)/meshes/body/v10/visual/body_link0.stl" scale="0.001 0.001 0.001"/>
         </geometry>
       </visual>
@@ -21,6 +21,6 @@
         <origin rpy="0.0 0.0 0.0" xyz="0.0 0.0 0.0"/>
         <geometry>
-          <mesh filename="file://$(find openarm_v10_description/meshes/body/v10/collision/body_link0_symp.stl" scale="0.001 0.001 0.001"/>
-          <!-- <mesh filename="file://$(find openarm_v10_description/meshes/arm/${arm_type}/collision/${name}.stl" scale="0.001 0.001 0.001" /> -->
+          <mesh filename="file://$(find openarm_v10_description)/meshes/body/v10/collision/body_link0_symp.stl" scale="0.001 0.001 0.001"/>
+          <!-- <mesh filename="file://$(find openarm_v10_description)/meshes/arm/${arm_type}/collision/${name}.stl" scale="0.001 0.001 0.001" /> -->
         </geometry>
       </collision>
@@ -40,5 +40,5 @@
         <origin rpy="0.0 0.0 0.0" xyz="0.0 0.0 0.0"/>
         <geometry>
-          <mesh filename="file://$(find openarm_v10_description/meshes/arm/v10/visual/link0.dae" scale="0.001 -0.001 0.001"/>
+          <mesh filename="file://$(find openarm_v10_description)/meshes/arm/v10/visual/link0.stl" scale="0.001 -0.001 0.001"/>
         </geometry>
       </visual>
@@ -46,6 +46,6 @@
         <origin rpy="0.0 0.0 0.0" xyz="0.0 0.0 0.0"/>
         <geometry>
-          <mesh filename="file://$(find openarm_v10_description/meshes/arm/v10/collision/link0_symp.stl" scale="0.001 -0.001 0.001"/>
-          <!-- <mesh filename="file://$(find openarm_v10_description/meshes/arm/${arm_type}/collision/${name}.stl" scale="0.001 0.001 0.001" /> -->
+          <mesh filename="file://$(find openarm_v10_description)/meshes/arm/v10/collision/link0_symp.stl" scale="0.001 -0.001 0.001"/>
+          <!-- <mesh filename="file://$(find openarm_v10_description)/meshes/arm/${arm_type}/collision/${name}.stl" scale="0.001 0.001 0.001" /> -->
         </geometry>
       </collision>
@@ -60,5 +60,5 @@
         <origin rpy="0.0 0.0 0.0" xyz="-0.0 0.0 -0.0625"/>
         <geometry>
-          <mesh filename="file://$(find openarm_v10_description/meshes/arm/v10/visual/link1.dae" scale="0.001 -0.001 0.001"/>
+          <mesh filename="file://$(find openarm_v10_description)/meshes/arm/v10/visual/link1.dae" scale="0.001 -0.001 0.001"/>
         </geometry>
       </visual>
@@ -66,6 +66,6 @@
         <origin rpy="0.0 0.0 0.0" xyz="-0.0 0.0 -0.0625"/>
         <geometry>
-          <mesh filename="file://$(find openarm_v10_description/meshes/arm/v10/collision/link1_symp.stl" scale="0.001 -0.001 0.001"/>
-          <!-- <mesh filename="file://$(find openarm_v10_description/meshes/arm/${arm_type}/collision/${name}.stl" scale="0.001 0.001 0.001" /> -->
+          <mesh filename="file://$(find openarm_v10_description)/meshes/arm/v10/collision/link1_symp.stl" scale="0.001 -0.001 0.001"/>
+          <!-- <mesh filename="file://$(find openarm_v10_description)/meshes/arm/${arm_type}/collision/${name}.stl" scale="0.001 0.001 0.001" /> -->
         </geometry>
       </collision>
@@ -87,5 +87,5 @@
         <origin rpy="0.0 0.0 0.0" xyz="0.0301 0.0 -0.1225"/>
         <geometry>
-          <mesh filename="file://$(find openarm_v10_description/meshes/arm/v10/visual/link2.dae" scale="0.001 -0.001 0.001"/>
+          <mesh filename="file://$(find openarm_v10_description)/meshes/arm/v10/visual/link2.dae" scale="0.001 -0.001 0.001"/>
         </geometry>
       </visual>
@@ -93,6 +93,6 @@
         <origin rpy="0.0 0.0 0.0" xyz="0.0301 0.0 -0.1225"/>
         <geometry>
-          <mesh filename="file://$(find openarm_v10_description/meshes/arm/v10/collision/link2_symp.stl" scale="0.001 -0.001 0.001"/>
-          <!-- <mesh filename="file://$(find openarm_v10_description/meshes/arm/${arm_type}/collision/${name}.stl" scale="0.001 0.001 0.001" /> -->
+          <mesh filename="file://$(find openarm_v10_description)/meshes/arm/v10/collision/link2_symp.stl" scale="0.001 -0.001 0.001"/>
+          <!-- <mesh filename="file://$(find openarm_v10_description)/meshes/arm/${arm_type}/collision/${name}.stl" scale="0.001 0.001 0.001" /> -->
         </geometry>
       </collision>
@@ -114,5 +114,5 @@
         <origin rpy="0.0 0.0 0.0" xyz="-0.0 -0.0 -0.18875"/>
         <geometry>
-          <mesh filename="file://$(find openarm_v10_description/meshes/arm/v10/visual/link3.dae" scale="0.001 -0.001 0.001"/>
+          <mesh filename="file://$(find openarm_v10_description)/meshes/arm/v10/visual/link3.dae" scale="0.001 -0.001 0.001"/>
         </geometry>
       </visual>
@@ -120,6 +120,6 @@
         <origin rpy="0.0 0.0 0.0" xyz="-0.0 -0.0 -0.18875"/>
         <geometry>
-          <mesh filename="file://$(find openarm_v10_description/meshes/arm/v10/collision/link3_symp.stl" scale="0.001 -0.001 0.001"/>
-          <!-- <mesh filename="file://$(find openarm_v10_description/meshes/arm/${arm_type}/collision/${name}.stl" scale="0.001 0.001 0.001" /> -->
+          <mesh filename="file://$(find openarm_v10_description)/meshes/arm/v10/collision/link3_symp.stl" scale="0.001 -0.001 0.001"/>
+          <!-- <mesh filename="file://$(find openarm_v10_description)/meshes/arm/${arm_type}/collision/${name}.stl" scale="0.001 0.001 0.001" /> -->
         </geometry>
       </collision>
@@ -141,5 +141,5 @@
         <origin rpy="0.0 0.0 0.0" xyz="0.0 -0.0315 -0.3425"/>
         <geometry>
-          <mesh filename="file://$(find openarm_v10_description/meshes/arm/v10/visual/link4.dae" scale="0.001 0.001 0.001"/>
+          <mesh filename="file://$(find openarm_v10_description)/meshes/arm/v10/visual/link4.dae" scale="0.001 0.001 0.001"/>
         </geometry>
       </visual>
@@ -147,6 +147,6 @@
         <origin rpy="0.0 0.0 0.0" xyz="0.0 -0.0315 -0.3425"/>
         <geometry>
-          <mesh filename="file://$(find openarm_v10_description/meshes/arm/v10/collision/link4_symp.stl" scale="0.001 0.001 0.001"/>
-          <!-- <mesh filename="file://$(find openarm_v10_description/meshes/arm/${arm_type}/collision/${name}.stl" scale="0.001 0.001 0.001" /> -->
+          <mesh filename="file://$(find openarm_v10_description)/meshes/arm/v10/collision/link4_symp.stl" scale="0.001 0.001 0.001"/>
+          <!-- <mesh filename="file://$(find openarm_v10_description)/meshes/arm/${arm_type}/collision/${name}.stl" scale="0.001 0.001 0.001" /> -->
         </geometry>
       </collision>
@@ -168,5 +168,5 @@
         <origin rpy="0.0 0.0 0.0" xyz="-0.0 -0.0 -0.438"/>
         <geometry>
-          <mesh filename="file://$(find openarm_v10_description/meshes/arm/v10/visual/link5.dae" scale="0.001 -0.001 0.001"/>
+          <mesh filename="file://$(find openarm_v10_description)/meshes/arm/v10/visual/link5.dae" scale="0.001 -0.001 0.001"/>
         </geometry>
       </visual>
@@ -174,6 +174,6 @@
         <origin rpy="0.0 0.0 0.0" xyz="-0.0 -0.0 -0.438"/>
         <geometry>
-          <mesh filename="file://$(find openarm_v10_description/meshes/arm/v10/collision/link5_symp.stl" scale="0.001 -0.001 0.001"/>
-          <!-- <mesh filename="file://$(find openarm_v10_description/meshes/arm/${arm_type}/collision/${name}.stl" scale="0.001 0.001 0.001" /> -->
+          <mesh filename="file://$(find openarm_v10_description)/meshes/arm/v10/collision/link5_symp.stl" scale="0.001 -0.001 0.001"/>
+          <!-- <mesh filename="file://$(find openarm_v10_description)/meshes/arm/${arm_type}/collision/${name}.stl" scale="0.001 0.001 0.001" /> -->
         </geometry>
       </collision>
@@ -195,5 +195,5 @@
         <origin rpy="0.0 0.0 0.0" xyz="-0.0375 -0.0 -0.5585"/>
         <geometry>
-          <mesh filename="file://$(find openarm_v10_description/meshes/arm/v10/visual/link6.dae" scale="0.001 -0.001 0.001"/>
+          <mesh filename="file://$(find openarm_v10_description)/meshes/arm/v10/visual/link6.dae" scale="0.001 -0.001 0.001"/>
         </geometry>
       </visual>
@@ -201,6 +201,6 @@
         <origin rpy="0.0 0.0 0.0" xyz="-0.0375 -0.0 -0.5585"/>
         <geometry>
-          <mesh filename="file://$(find openarm_v10_description/meshes/arm/v10/collision/link6_symp.stl" scale="0.001 -0.001 0.001"/>
-          <!-- <mesh filename="file://$(find openarm_v10_description/meshes/arm/${arm_type}/collision/${name}.stl" scale="0.001 0.001 0.001" /> -->
+          <mesh filename="file://$(find openarm_v10_description)/meshes/arm/v10/collision/link6_symp.stl" scale="0.001 -0.001 0.001"/>
+          <!-- <mesh filename="file://$(find openarm_v10_description)/meshes/arm/${arm_type}/collision/${name}.stl" scale="0.001 0.001 0.001" /> -->
         </geometry>
       </collision>
@@ -222,5 +222,5 @@
         <origin rpy="0.0 0.0 0.0" xyz="0.0 -0.0 -0.5585"/>
         <geometry>
-          <mesh filename="file://$(find openarm_v10_description/meshes/arm/v10/visual/link7.dae" scale="0.001 -0.001 0.001"/>
+          <mesh filename="file://$(find openarm_v10_description)/meshes/arm/v10/visual/link7.dae" scale="0.001 -0.001 0.001"/>
         </geometry>
       </visual>
@@ -228,6 +228,6 @@
         <origin rpy="0.0 0.0 0.0" xyz="0.0 -0.0 -0.5585"/>
         <geometry>
-          <mesh filename="file://$(find openarm_v10_description/meshes/arm/v10/collision/link7_symp.stl" scale="0.001 -0.001 0.001"/>
-          <!-- <mesh filename="file://$(find openarm_v10_description/meshes/arm/${arm_type}/collision/${name}.stl" scale="0.001 0.001 0.001" /> -->
+          <mesh filename="file://$(find openarm_v10_description)/meshes/arm/v10/collision/link7_symp.stl" scale="0.001 -0.001 0.001"/>
+          <!-- <mesh filename="file://$(find openarm_v10_description)/meshes/arm/${arm_type}/collision/${name}.stl" scale="0.001 0.001 0.001" /> -->
         </geometry>
       </collision>
@@ -260,5 +260,5 @@
         <origin rpy="0.0 0.0 0.0" xyz="0.0 0.0 0.0"/>
         <geometry>
-          <mesh filename="file://$(find openarm_v10_description/meshes/arm/v10/visual/link0.dae" scale="0.001 0.001 0.001"/>
+          <mesh filename="file://$(find openarm_v10_description)/meshes/arm/v10/visual/link0.stl" scale="0.001 0.001 0.001"/>
         </geometry>
       </visual>
@@ -266,6 +266,6 @@
         <origin rpy="0.0 0.0 0.0" xyz="0.0 0.0 0.0"/>
         <geometry>
-          <mesh filename="file://$(find openarm_v10_description/meshes/arm/v10/collision/link0_symp.stl" scale="0.001 0.001 0.001"/>
-          <!-- <mesh filename="file://$(find openarm_v10_description/meshes/arm/${arm_type}/collision/${name}.stl" scale="0.001 0.001 0.001" /> -->
+          <mesh filename="file://$(find openarm_v10_description)/meshes/arm/v10/collision/link0_symp.stl" scale="0.001 0.001 0.001"/>
+          <!-- <mesh filename="file://$(find openarm_v10_description)/meshes/arm/${arm_type}/collision/${name}.stl" scale="0.001 0.001 0.001" /> -->
         </geometry>
       </collision>
@@ -280,5 +280,5 @@
         <origin rpy="0.0 0.0 0.0" xyz="-0.0 0.0 -0.0625"/>
         <geometry>
-          <mesh filename="file://$(find openarm_v10_description/meshes/arm/v10/visual/link1.dae" scale="0.001 0.001 0.001"/>
+          <mesh filename="file://$(find openarm_v10_description)/meshes/arm/v10/visual/link1.dae" scale="0.001 0.001 0.001"/>
         </geometry>
       </visual>
@@ -286,6 +286,6 @@
         <origin rpy="0.0 0.0 0.0" xyz="-0.0 0.0 -0.0625"/>
         <geometry>
-          <mesh filename="file://$(find openarm_v10_description/meshes/arm/v10/collision/link1_symp.stl" scale="0.001 0.001 0.001"/>
-          <!-- <mesh filename="file://$(find openarm_v10_description/meshes/arm/${arm_type}/collision/${name}.stl" scale="0.001 0.001 0.001" /> -->
+          <mesh filename="file://$(find openarm_v10_description)/meshes/arm/v10/collision/link1_symp.stl" scale="0.001 0.001 0.001"/>
+          <!-- <mesh filename="file://$(find openarm_v10_description)/meshes/arm/${arm_type}/collision/${name}.stl" scale="0.001 0.001 0.001" /> -->
         </geometry>
       </collision>
@@ -307,5 +307,5 @@
         <origin rpy="0.0 0.0 0.0" xyz="0.0301 0.0 -0.1225"/>
         <geometry>
-          <mesh filename="file://$(find openarm_v10_description/meshes/arm/v10/visual/link2.dae" scale="0.001 0.001 0.001"/>
+          <mesh filename="file://$(find openarm_v10_description)/meshes/arm/v10/visual/link2.dae" scale="0.001 0.001 0.001"/>
         </geometry>
       </visual>
@@ -313,6 +313,6 @@
         <origin rpy="0.0 0.0 0.0" xyz="0.0301 0.0 -0.1225"/>
         <geometry>
-          <mesh filename="file://$(find openarm_v10_description/meshes/arm/v10/collision/link2_symp.stl" scale="0.001 0.001 0.001"/>
-          <!-- <mesh filename="file://$(find openarm_v10_description/meshes/arm/${arm_type}/collision/${name}.stl" scale="0.001 0.001 0.001" /> -->
+          <mesh filename="file://$(find openarm_v10_description)/meshes/arm/v10/collision/link2_symp.stl" scale="0.001 0.001 0.001"/>
+          <!-- <mesh filename="file://$(find openarm_v10_description)/meshes/arm/${arm_type}/collision/${name}.stl" scale="0.001 0.001 0.001" /> -->
         </geometry>
       </collision>
@@ -334,5 +334,5 @@
         <origin rpy="0.0 0.0 0.0" xyz="-0.0 -0.0 -0.18875"/>
         <geometry>
-          <mesh filename="file://$(find openarm_v10_description/meshes/arm/v10/visual/link3.dae" scale="0.001 0.001 0.001"/>
+          <mesh filename="file://$(find openarm_v10_description)/meshes/arm/v10/visual/link3.dae" scale="0.001 0.001 0.001"/>
         </geometry>
       </visual>
@@ -340,6 +340,6 @@
         <origin rpy="0.0 0.0 0.0" xyz="-0.0 -0.0 -0.18875"/>
         <geometry>
-          <mesh filename="file://$(find openarm_v10_description/meshes/arm/v10/collision/link3_symp.stl" scale="0.001 0.001 0.001"/>
-          <!-- <mesh filename="file://$(find openarm_v10_description/meshes/arm/${arm_type}/collision/${name}.stl" scale="0.001 0.001 0.001" /> -->
+          <mesh filename="file://$(find openarm_v10_description)/meshes/arm/v10/collision/link3_symp.stl" scale="0.001 0.001 0.001"/>
+          <!-- <mesh filename="file://$(find openarm_v10_description)/meshes/arm/${arm_type}/collision/${name}.stl" scale="0.001 0.001 0.001" /> -->
         </geometry>
       </collision>
@@ -361,5 +361,5 @@
         <origin rpy="0.0 0.0 0.0" xyz="0.0 -0.0315 -0.3425"/>
         <geometry>
-          <mesh filename="file://$(find openarm_v10_description/meshes/arm/v10/visual/link4.dae" scale="0.001 0.001 0.001"/>
+          <mesh filename="file://$(find openarm_v10_description)/meshes/arm/v10/visual/link4.dae" scale="0.001 0.001 0.001"/>
         </geometry>
       </visual>
@@ -367,6 +367,6 @@
         <origin rpy="0.0 0.0 0.0" xyz="0.0 -0.0315 -0.3425"/>
         <geometry>
-          <mesh filename="file://$(find openarm_v10_description/meshes/arm/v10/collision/link4_symp.stl" scale="0.001 0.001 0.001"/>
-          <!-- <mesh filename="file://$(find openarm_v10_description/meshes/arm/${arm_type}/collision/${name}.stl" scale="0.001 0.001 0.001" /> -->
+          <mesh filename="file://$(find openarm_v10_description)/meshes/arm/v10/collision/link4_symp.stl" scale="0.001 0.001 0.001"/>
+          <!-- <mesh filename="file://$(find openarm_v10_description)/meshes/arm/${arm_type}/collision/${name}.stl" scale="0.001 0.001 0.001" /> -->
         </geometry>
       </collision>
@@ -388,5 +388,5 @@
         <origin rpy="0.0 0.0 0.0" xyz="-0.0 -0.0 -0.438"/>
         <geometry>
-          <mesh filename="file://$(find openarm_v10_description/meshes/arm/v10/visual/link5.dae" scale="0.001 0.001 0.001"/>
+          <mesh filename="file://$(find openarm_v10_description)/meshes/arm/v10/visual/link5.dae" scale="0.001 0.001 0.001"/>
         </geometry>
       </visual>
@@ -394,6 +394,6 @@
         <origin rpy="0.0 0.0 0.0" xyz="-0.0 -0.0 -0.438"/>
         <geometry>
-          <mesh filename="file://$(find openarm_v10_description/meshes/arm/v10/collision/link5_symp.stl" scale="0.001 0.001 0.001"/>
-          <!-- <mesh filename="file://$(find openarm_v10_description/meshes/arm/${arm_type}/collision/${name}.stl" scale="0.001 0.001 0.001" /> -->
+          <mesh filename="file://$(find openarm_v10_description)/meshes/arm/v10/collision/link5_symp.stl" scale="0.001 0.001 0.001"/>
+          <!-- <mesh filename="file://$(find openarm_v10_description)/meshes/arm/${arm_type}/collision/${name}.stl" scale="0.001 0.001 0.001" /> -->
         </geometry>
       </collision>
@@ -415,5 +415,5 @@
         <origin rpy="0.0 0.0 0.0" xyz="-0.0375 -0.0 -0.5585"/>
         <geometry>
-          <mesh filename="file://$(find openarm_v10_description/meshes/arm/v10/visual/link6.dae" scale="0.001 0.001 0.001"/>
+          <mesh filename="file://$(find openarm_v10_description)/meshes/arm/v10/visual/link6.dae" scale="0.001 0.001 0.001"/>
         </geometry>
       </visual>
@@ -421,6 +421,6 @@
         <origin rpy="0.0 0.0 0.0" xyz="-0.0375 -0.0 -0.5585"/>
         <geometry>
-          <mesh filename="file://$(find openarm_v10_description/meshes/arm/v10/collision/link6_symp.stl" scale="0.001 0.001 0.001"/>
-          <!-- <mesh filename="file://$(find openarm_v10_description/meshes/arm/${arm_type}/collision/${name}.stl" scale="0.001 0.001 0.001" /> -->
+          <mesh filename="file://$(find openarm_v10_description)/meshes/arm/v10/collision/link6_symp.stl" scale="0.001 0.001 0.001"/>
+          <!-- <mesh filename="file://$(find openarm_v10_description)/meshes/arm/${arm_type}/collision/${name}.stl" scale="0.001 0.001 0.001" /> -->
         </geometry>
       </collision>
@@ -442,5 +442,5 @@
         <origin rpy="0.0 0.0 0.0" xyz="0.0 -0.0 -0.5585"/>
         <geometry>
-          <mesh filename="file://$(find openarm_v10_description/meshes/arm/v10/visual/link7.dae" scale="0.001 0.001 0.001"/>
+          <mesh filename="file://$(find openarm_v10_description)/meshes/arm/v10/visual/link7.dae" scale="0.001 0.001 0.001"/>
         </geometry>
       </visual>
@@ -448,6 +448,6 @@
         <origin rpy="0.0 0.0 0.0" xyz="0.0 -0.0 -0.5585"/>
         <geometry>
-          <mesh filename="file://$(find openarm_v10_description/meshes/arm/v10/collision/link7_symp.stl" scale="0.001 0.001 0.001"/>
-          <!-- <mesh filename="file://$(find openarm_v10_description/meshes/arm/${arm_type}/collision/${name}.stl" scale="0.001 0.001 0.001" /> -->
+          <mesh filename="file://$(find openarm_v10_description)/meshes/arm/v10/collision/link7_symp.stl" scale="0.001 0.001 0.001"/>
+          <!-- <mesh filename="file://$(find openarm_v10_description)/meshes/arm/${arm_type}/collision/${name}.stl" scale="0.001 0.001 0.001" /> -->
         </geometry>
       </collision>
@@ -475,5 +475,5 @@
         <origin rpy="0.0 0.0 0.0" xyz="0.0 0.0 -0.6585"/>
         <geometry>
-          <mesh filename="file://$(find openarm_v10_description/meshes/ee/openarm_hand/visual/hand.dae" scale="0.001 0.001 0.001"/>
+          <mesh filename="file://$(find openarm_v10_description)/meshes/ee/openarm_hand/visual/hand.dae" scale="0.001 0.001 0.001"/>
         </geometry>
       </visual>
@@ -481,5 +481,5 @@
         <origin rpy="0.0 0.0 0.0" xyz="0.0 0.0 -0.6585"/>
         <geometry>
-          <mesh filename="file://$(find openarm_v10_description/meshes/ee/openarm_hand/collision/hand.stl" scale="0.001 0.001 0.001"/>
+          <mesh filename="file://$(find openarm_v10_description)/meshes/ee/openarm_hand/collision/hand.stl" scale="0.001 0.001 0.001"/>
         </geometry>
       </collision>
@@ -508,5 +508,5 @@
         <origin rpy="0.0 0.0 0.0" xyz="0.0 -0.05 -0.673001"/>
         <geometry>
-          <mesh filename="file://$(find openarm_v10_description/meshes/ee/openarm_hand/visual/finger.dae" scale="0.001 0.001 0.001"/>
+          <mesh filename="file://$(find openarm_v10_description)/meshes/ee/openarm_hand/visual/finger.dae" scale="0.001 0.001 0.001"/>
         </geometry>
       </visual>
@@ -514,5 +514,5 @@
         <origin rpy="0.0 0.0 0.0" xyz="0.0 -0.05 -0.673001"/>
         <geometry>
-          <mesh filename="file://$(find openarm_v10_description/meshes/ee/openarm_hand/collision/finger.stl" scale="0.001 0.001 0.001"/>
+          <mesh filename="file://$(find openarm_v10_description)/meshes/ee/openarm_hand/collision/finger.stl" scale="0.001 0.001 0.001"/>
         </geometry>
       </collision>
@@ -527,5 +527,5 @@
         <origin rpy="0.0 0.0 0.0" xyz="0.0 0.05 -0.673001"/>
         <geometry>
-          <mesh filename="file://$(find openarm_v10_description/meshes/ee/openarm_hand/visual/finger.dae" scale="0.001 -0.001 0.001"/>
+          <mesh filename="file://$(find openarm_v10_description)/meshes/ee/openarm_hand/visual/finger.dae" scale="0.001 -0.001 0.001"/>
         </geometry>
       </visual>
@@ -533,5 +533,5 @@
         <origin rpy="0.0 0.0 0.0" xyz="0.0 0.05 -0.673001"/>
         <geometry>
-          <mesh filename="file://$(find openarm_v10_description/meshes/ee/openarm_hand/collision/finger.stl" scale="0.001 -0.001 0.001"/>
+          <mesh filename="file://$(find openarm_v10_description)/meshes/ee/openarm_hand/collision/finger.stl" scale="0.001 -0.001 0.001"/>
         </geometry>
       </collision>
@@ -561,5 +561,5 @@
         <origin rpy="0.0 0.0 0.0" xyz="0.0 0.0 -0.6585"/>
         <geometry>
-          <mesh filename="file://$(find openarm_v10_description/meshes/ee/openarm_hand/visual/hand.dae" scale="0.001 0.001 0.001"/>
+          <mesh filename="file://$(find openarm_v10_description)/meshes/ee/openarm_hand/visual/hand.dae" scale="0.001 0.001 0.001"/>
         </geometry>
       </visual>
@@ -567,5 +567,5 @@
         <origin rpy="0.0 0.0 0.0" xyz="0.0 0.0 -0.6585"/>
         <geometry>
-          <mesh filename="file://$(find openarm_v10_description/meshes/ee/openarm_hand/collision/hand.stl" scale="0.001 0.001 0.001"/>
+          <mesh filename="file://$(find openarm_v10_description)/meshes/ee/openarm_hand/collision/hand.stl" scale="0.001 0.001 0.001"/>
         </geometry>
       </collision>
@@ -594,5 +594,5 @@
         <origin rpy="0.0 0.0 0.0" xyz="0.0 -0.05 -0.673001"/>
         <geometry>
-          <mesh filename="file://$(find openarm_v10_description/meshes/ee/openarm_hand/visual/finger.dae" scale="0.001 0.001 0.001"/>
+          <mesh filename="file://$(find openarm_v10_description)/meshes/ee/openarm_hand/visual/finger.dae" scale="0.001 0.001 0.001"/>
         </geometry>
       </visual>
@@ -600,5 +600,5 @@
         <origin rpy="0.0 0.0 0.0" xyz="0.0 -0.05 -0.673001"/>
         <geometry>
-          <mesh filename="file://$(find openarm_v10_description/meshes/ee/openarm_hand/collision/finger.stl" scale="0.001 0.001 0.001"/>
+          <mesh filename="file://$(find openarm_v10_description)/meshes/ee/openarm_hand/collision/finger.stl" scale="0.001 0.001 0.001"/>
         </geometry>
       </collision>
@@ -613,5 +613,5 @@
         <origin rpy="0.0 0.0 0.0" xyz="0.0 0.05 -0.673001"/>
         <geometry>
-          <mesh filename="file://$(find openarm_v10_description/meshes/ee/openarm_hand/visual/finger.dae" scale="0.001 -0.001 0.001"/>
+          <mesh filename="file://$(find openarm_v10_description)/meshes/ee/openarm_hand/visual/finger.dae" scale="0.001 -0.001 0.001"/>
         </geometry>
       </visual>
@@ -619,5 +619,5 @@
         <origin rpy="0.0 0.0 0.0" xyz="0.0 0.05 -0.673001"/>
         <geometry>
-          <mesh filename="file://$(find openarm_v10_description/meshes/ee/openarm_hand/collision/finger.stl" scale="0.001 -0.001 0.001"/>
+          <mesh filename="file://$(find openarm_v10_description)/meshes/ee/openarm_hand/collision/finger.stl" scale="0.001 -0.001 0.001"/>
         </geometry>
       </collision>
