Commit message: add: test on rviz2 have error on finger inertia value

File: manipulator/OpenArm/openarm_v10_description/xacro/robot.xacro (robot description, xacro)
@@ -3,9 +3,9 @@
   <xacro:arg name="type" default="bimanual"/>
   <!-- 根据type参数决定机器人类型 -->
-  <xacro:if value="${'$(arg type)' == 'single'}">
+  <xacro:if value="${'$(arg type)' == 'bimanual'}">
     <xacro:include filename="$(find openarm_v10_description)/xacro/openarm_bimanual.xacro"/>
     <xacro:OpenArm name=""/>
   </xacro:if>
-  <xacro:if value="${'$(arg type)' == 'bimanual'}">
+  <xacro:if value="${'$(arg type)' == 'single'}">
     <xacro:include filename="$(find openarm_v10_description)/xacro/openarm_single.xacro"/>
     <xacro:OpenArm name=""/>

Commit message: bug: robot in rviz is white and can't be manipulate

File: manipulator/OpenArm/openarm_v10_description/xacro/openarm_bimanual.xacro (robot description, xacro)
@@ -520,5 +520,5 @@
         <origin rpy="0 0 0" xyz="0.0064528 0.01702 0.0219685"/>
         <mass value="0.03602545343277134"/>
-        <inertia ixx="2.3749999999999997e-06" ixy="1e-06" ixz="1e-06" iyy="2.3749999999999997e-06" iyz="1e-06" izz="7.5e-07"/>
+        <inertia ixx="0.0001" ixy="0" ixz="0" iyy="0.0001" iyz="0" izz="0.0001"/> <!-- Adjust inertial for finger -->
       </inertial>
     </link>
@@ -539,5 +539,5 @@
         <origin rpy="0 0 0" xyz="0.0064528 -0.01702 0.0219685"/>
         <mass value="0.03602545343277134"/>
-        <inertia ixx="2.3749999999999997e-06" ixy="1e-06" ixz="1e-06" iyy="2.3749999999999997e-06" iyz="1e-06" izz="7.5e-07"/>
+        <inertia ixx="0.0001" ixy="0" ixz="0" iyy="0.0001" iyz="0" izz="0.0001"/> <!-- Adjust inertial for finger -->
       </inertial>
     </link>
@@ -606,5 +606,5 @@
         <origin rpy="0 0 0" xyz="0.0064528 0.01702 0.0219685"/>
         <mass value="0.03602545343277134"/>
-        <inertia ixx="2.3749999999999997e-06" ixy="1e-06" ixz="1e-06" iyy="2.3749999999999997e-06" iyz="1e-06" izz="7.5e-07"/>
+        <inertia ixx="0.0001" ixy="0" ixz="0" iyy="0.0001" iyz="0" izz="0.0001"/> <!-- Adjust inertial for finger -->
       </inertial>
     </link>
@@ -625,5 +625,5 @@
         <origin rpy="0 0 0" xyz="0.0064528 -0.01702 0.0219685"/>
         <mass value="0.03602545343277134"/>
-        <inertia ixx="2.3749999999999997e-06" ixy="1e-06" ixz="1e-06" iyy="2.3749999999999997e-06" iyz="1e-06" izz="7.5e-07"/>
+        <inertia ixx="0.0001" ixy="0" ixz="0" iyy="0.0001" iyz="0" izz="0.0001"/> <!-- Adjust inertial for finger -->
       </inertial>
     </link>

File: manipulator/OpenArm/openarm_v10_description/xacro/openarm_single.xacro (robot description, xacro)
@@ -269,5 +269,5 @@
         <origin rpy="0 0 0" xyz="0.0064528 0.01702 0.0219685"/>
         <mass value="0.03602545343277134"/>
-        <inertia ixx="2.3749999999999997e-06" ixy="1e-06" ixz="1e-06" iyy="2.3749999999999997e-06" iyz="1e-06" izz="7.5e-07"/>
+        <inertia ixx="0.0001" ixy="0" ixz="0" iyy="0.0001" iyz="0" izz="0.0001"/> <!-- Adjust inertial for finger -->
       </inertial>
     </link>
@@ -288,5 +288,5 @@
         <origin rpy="0 0 0" xyz="0.0064528 -0.01702 0.0219685"/>
         <mass value="0.03602545343277134"/>
-        <inertia ixx="2.3749999999999997e-06" ixy="1e-06" ixz="1e-06" iyy="2.3749999999999997e-06" iyz="1e-06" izz="7.5e-07"/>
+        <inertia ixx="0.0001" ixy="0" ixz="0" iyy="0.0001" iyz="0" izz="0.0001"/> # Adjust inertial for finger
       </inertial>
     </link>

Commit message: bug: arm/v10/visual/link0.dae cause not enough data accessor problem in RTX 4060ti

File: manipulator/OpenArm/openarm_v10_description/xacro/openarm_bimanual.xacro (robot description, xacro)
@@ -15,5 +15,5 @@
         <origin rpy="0.0 0.0 0.0" xyz="0.0 0.0 0.0"/>
         <geometry>
-          <mesh filename="file://$(find openarm_v10_description)/meshes/body/v10/visual/body_link0.stl" scale="0.001 0.001 0.001"/>
+          <mesh filename="file://$(find openarm_v10_description)/meshes/body/v10/visual/body_link0.dae" scale="0.001 0.001 0.001"/>
         </geometry>
       </visual>

Commit message: add: repaint arm/visual/link0 with blender

File: manipulator/OpenArm/openarm_v10_description/xacro/openarm_bimanual.xacro (robot description, xacro)
@@ -40,5 +40,5 @@
         <origin rpy="0.0 0.0 0.0" xyz="0.0 0.0 0.0"/>
         <geometry>
-          <mesh filename="file://$(find openarm_v10_description)/meshes/arm/v10/visual/link0.stl" scale="0.001 -0.001 0.001"/>
+          <mesh filename="file://$(find openarm_v10_description)/meshes/arm/v10/visual/link0.obj" scale="0.001 -0.001 0.001"/>
         </geometry>
       </visual>

File: manipulator/OpenArm/openarm_v10_description/xacro/openarm_single.xacro (robot description, xacro)
@@ -15,5 +15,5 @@
         <origin rpy="0.0 0.0 0.0" xyz="0.0 0.0 0.0"/>
         <geometry>
-          <mesh filename="file://$(find openarm_v10_description)/meshes/arm/v10/visual/link0.stl" scale="0.001 -0.001 0.001"/>
+          <mesh filename="file://$(find openarm_v10_description)/meshes/arm/v10/visual/link0.obj" scale="0.001 -0.001 0.001"/>
         </geometry>
       </visual>

Commit message: fix: bimanual right_link0 to obj

File: manipulator/OpenArm/openarm_v10_description/xacro/openarm_bimanual.xacro (robot description, xacro)
@@ -260,5 +260,5 @@
         <origin rpy="0.0 0.0 0.0" xyz="0.0 0.0 0.0"/>
         <geometry>
-          <mesh filename="file://$(find openarm_v10_description)/meshes/arm/v10/visual/link0.stl" scale="0.001 0.001 0.001"/>
+          <mesh filename="file://$(find openarm_v10_description)/meshes/arm/v10/visual/link0.obj" scale="0.001 0.001 0.001"/>
         </geometry>
       </visual>
