Commit message: add: ocs2 task.info for bimanual openarm

File: manipulator/OpenArm/openarm_v10_description/urdf/openarm_bimanual.urdf (robot description, URDF)
Before this commit: robot openarm, 26 links, 25 joints
Links:
- removed link openarm_body_link0
- removed link openarm_left_hand
- removed link openarm_left_hand_tcp
- removed link openarm_left_left_finger
- removed link openarm_left_link0
- removed link openarm_left_link1
- removed link openarm_left_link2
- removed link openarm_left_link3
- removed link openarm_left_link4
- removed link openarm_left_link5
- removed link openarm_left_link6
- removed link openarm_left_link7
- removed link openarm_left_right_finger
- removed link openarm_right_hand
- removed link openarm_right_hand_tcp
- removed link openarm_right_left_finger
- removed link openarm_right_link0
- removed link openarm_right_link1
- removed link openarm_right_link2
- removed link openarm_right_link3
- removed link openarm_right_link4
- removed link openarm_right_link5
- removed link openarm_right_link6
- removed link openarm_right_link7
- removed link openarm_right_right_finger
- added link body_link0, mass 13.89; collision mesh filename=package://openarm_v10_description/meshes/body/v10/collision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 scale=0.001 0.001 0.001; visual mesh filename=package://openarm_v10_description/meshes/body/v10/visual/bo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 scale=0.001 0.001 0.001
- added link left_hand, mass 0.35; collision mesh filename=package://openarm_v10_description/meshes/ee/openarm_hand/co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 scale=0.001 0.001 0.001; visual mesh filename=package://openarm_v10_description/meshes/ee/openarm_hand/vi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 scale=0.001 0.001 0.001
- added link left_hand_tcp
- added link left_left_finger, mass 0.03602545343277134; collision mesh filename=package://openarm_v10_description/meshes/ee/openarm_hand/co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 scale=0.001 0.001 0.001; visual mesh filename=package://openarm_v10_description/meshes/ee/openarm_hand/vi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 scale=0.001 0.001 0.001
- added link left_link0, mass 1.1432284943239561; collision mesh filename=package://openarm_v10_description/meshes/arm/v10/collision/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 scale=0.001 -0.001 0.001; visual mesh filename=package://openarm_v10_description/meshes/arm/v10/visual/lin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 scale=0.001 -0.001 0.001
- added link left_link1, mass 1.1416684646202298; collision mesh filename=package://openarm_v10_description/meshes/arm/v10/collision/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 scale=0.001 -0.001 0.001; visual mesh filename=package://openarm_v10_description/meshes/arm/v10/visual/lin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 scale=0.001 -0.001 0.001
- added link left_link2, mass 0.2775092746011571; collision mesh filename=package://openarm_v10_description/meshes/arm/v10/collision/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 scale=0.001 -0.001 0.001; visual mesh filename=package://openarm_v10_description/meshes/arm/v10/visual/lin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 scale=0.001 -0.001 0.001
- added link left_link3, mass 1.073863338202347; collision mesh filename=package://openarm_v10_description/meshes/arm/v10/collision/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 scale=0.001 -0.001 0.001; visual mesh filename=package://openarm_v10_description/meshes/arm/v10/visual/lin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 scale=0.001 -0.001 0.001
- added link left_link4, mass 0.6348534566833373; collision mesh filename=package://openarm_v10_description/meshes/arm/v10/collision/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 scale=0.001 0.001 0.001; visual mesh filename=package://openarm_v10_description/meshes/arm/v10/visual/lin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 scale=0.001 0.001 0.001
- added link left_link5, mass 0.6156588026168502; collision mesh filename=package://openarm_v10_description/meshes/arm/v10/collision/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 scale=0.001 -0.001 0.001; visual mesh filename=package://openarm_v10_description/meshes/arm/v10/visual/lin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 scale=0.001 -0.001 0.001
- added link left_link6, mass 0.475202773187987; collision mesh filename=package://openarm_v10_description/meshes/arm/v10/collision/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 scale=0.001 -0.001 0.001; visual mesh filename=package://openarm_v10_description/meshes/arm/v10/visual/lin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 scale=0.001 -0.001 0.001
- added link left_link7, mass 0.4659771327380578; collision mesh filename=package://openarm_v10_description/meshes/arm/v10/collision/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 scale=0.001 -0.001 0.001; visual mesh filename=package://openarm_v10_description/meshes/arm/v10/visual/lin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 scale=0.001 -0.001 0.001
- added link left_right_finger, mass 0.03602545343277134; collision mesh filename=package://openarm_v10_description/meshes/ee/openarm_hand/co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 scale=0.001 -0.001 0.001; visual mesh filename=package://openarm_v10_description/meshes/ee/openarm_hand/vi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 scale=0.001 -0.001 0.001
- added link right_hand, mass 0.35; collision mesh filename=package://openarm_v10_description/meshes/ee/openarm_hand/co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 scale=0.001 0.001 0.001; visual mesh filename=package://openarm_v10_description/meshes/ee/openarm_hand/vi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 scale=0.001 0.001 0.001
- added link right_hand_tcp
- added link right_left_finger, mass 0.03602545343277134; collision mesh filename=package://openarm_v10_description/meshes/ee/openarm_hand/co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 scale=0.001 0.001 0.001; visual mesh filename=package://openarm_v10_description/meshes/ee/openarm_hand/vi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 scale=0.001 0.001 0.001
- added link right_link0, mass 1.1432284943239561; collision mesh filename=package://openarm_v10_description/meshes/arm/v10/collision/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 scale=0.001 0.001 0.001; visual mesh filename=package://openarm_v10_description/meshes/arm/v10/visual/lin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 scale=0.001 0.001 0.001
- added link right_link1, mass 1.1416684646202298; collision mesh filename=package://openarm_v10_description/meshes/arm/v10/collision/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 scale=0.001 0.001 0.001; visual mesh filename=package://openarm_v10_description/meshes/arm/v10/visual/lin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 scale=0.001 0.001 0.001
- added link right_link2, mass 0.2775092746011571; collision mesh filename=package://openarm_v10_description/meshes/arm/v10/collision/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 scale=0.001 0.001 0.001; visual mesh filename=package://openarm_v10_description/meshes/arm/v10/visual/lin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 scale=0.001 0.001 0.001
- added link right_link3, mass 1.073863338202347; collision mesh filename=package://openarm_v10_description/meshes/arm/v10/collision/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 scale=0.001 0.001 0.001; visual mesh filename=package://openarm_v10_description/meshes/arm/v10/visual/lin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 scale=0.001 0.001 0.001
- added link right_link4, mass 0.6348534566833373; collision mesh filename=package://openarm_v10_description/meshes/arm/v10/collision/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 scale=0.001 0.001 0.001; visual mesh filename=package://openarm_v10_description/meshes/arm/v10/visual/lin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 scale=0.001 0.001 0.001
- added link right_link5, mass 0.6156588026168502; collision mesh filename=package://openarm_v10_description/meshes/arm/v10/collision/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 scale=0.001 0.001 0.001; visual mesh filename=package://openarm_v10_description/meshes/arm/v10/visual/lin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 scale=0.001 0.001 0.001
- added link right_link6, mass 0.475202773187987; collision mesh filename=package://openarm_v10_description/meshes/arm/v10/collision/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 scale=0.001 0.001 0.001; visual mesh filename=package://openarm_v10_description/meshes/arm/v10/visual/lin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 scale=0.001 0.001 0.001
- added link right_link7, mass 0.4659771327380578; collision mesh filename=package://openarm_v10_description/meshes/arm/v10/collision/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 scale=0.001 0.001 0.001; visual mesh filename=package://openarm_v10_description/meshes/arm/v10/visual/lin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 scale=0.001 0.001 0.001
- added link right_right_finger, mass 0.03602545343277134; collision mesh filename=package://openarm_v10_description/meshes/ee/openarm_hand/co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 scale=0.001 -0.001 0.001; visual mesh filename=package://openarm_v10_description/meshes/ee/openarm_hand/vi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 scale=0.001 -0.001 0.001
Joints:
- removed joint left_openarm_hand_joint
- removed joint openarm_body_world_joint
- removed joint openarm_left_finger_joint1
- removed joint openarm_left_finger_joint2
- removed joint openarm_left_hand_tcp_joint
- removed joint openarm_left_joint1
- removed joint openarm_left_joint2
- removed joint openarm_left_joint3
- removed joint openarm_left_joint4
- removed joint openarm_left_joint5
- removed joint openarm_left_joint6
- removed joint openarm_left_joint7
- removed joint openarm_left_openarm_body_link0_joint
- removed joint openarm_right_finger_joint1
- removed joint openarm_right_finger_joint2
- removed joint openarm_right_hand_tcp_joint
- removed joint openarm_right_joint1
- removed joint openarm_right_joint2
- removed joint openarm_right_joint3
- removed joint openarm_right_joint4
- removed joint openarm_right_joint5
- removed joint openarm_right_joint6
- removed joint openarm_right_joint7
- removed joint openarm_right_openarm_body_link0_joint
- removed joint right_openarm_hand_joint
- added joint body_world_joint: type fixed, parent world, child body_link0, origin xyz=0 0 0 rpy=0 0 0
- added joint left_body_link0_joint: type fixed, parent body_link0, child left_link0, origin xyz=0.0 0.031 0.698 rpy=-1.5708 0 0
- added joint left_finger_joint1: type prismatic, parent left_hand, child left_right_finger, origin xyz=0 -0.006 0.015 rpy=0 0 0, axis 0 -1 0, limit lower=0.0 upper=0.044 effort=333 velocity=10.0
- added joint left_finger_joint2: type prismatic, parent left_hand, child left_left_finger, origin xyz=0 0.006 0.015 rpy=0 0 0, axis 0 1 0, limit lower=0.0 upper=0.044 effort=333 velocity=10.0, mimic joint=left_finger_joint1
- added joint left_hand_joint: type fixed, parent left_link7, child left_hand, origin xyz=0 -0.0 0.1001 rpy=0 0 0
- added joint left_hand_tcp_joint: type fixed, parent left_hand, child left_hand_tcp, origin xyz=0 -0.0 0.08 rpy=0 0 0
- added joint left_joint1: type revolute, parent left_link0, child left_link1, origin xyz=0.0 0.0 0.0625 rpy=0 0 0, axis 0 0 1, limit lower=-3.490659 upper=1.3962629999999998 effort=40 velocity=16.754666
- added joint left_joint2: type revolute, parent left_link1, child left_link2, origin xyz=-0.0301 0.0 0.06 rpy=-1.57079632679 0 0, axis -1 0 0, limit lower=-3.3161253267948965 upper=0.17453267320510335 effort=40 velocity=16.754666
- added joint left_joint3: type revolute, parent left_link2, child left_link3, origin xyz=0.0301 0.0 0.06625 rpy=0 0 0, axis 0 0 1, limit lower=-1.570796 upper=1.570796 effort=27 velocity=5.445426
- added joint left_joint4: type revolute, parent left_link3, child left_link4, origin xyz=-0.0 0.0315 0.15375 rpy=0 0 0, axis 0 1 0, limit lower=0.0 upper=2.443461 effort=27 velocity=5.445426
- added joint left_joint5: type revolute, parent left_link4, child left_link5, origin xyz=0.0 -0.0315 0.0955 rpy=0 0 0, axis 0 0 1, limit lower=-1.570796 upper=1.570796 effort=7 velocity=20.943946
- added joint left_joint6: type revolute, parent left_link5, child left_link6, origin xyz=0.0375 0.0 0.1205 rpy=0 0 0, axis 1 0 0, limit lower=-0.785398 upper=0.785398 effort=7 velocity=20.943946
- added joint left_joint7: type revolute, parent left_link6, child left_link7, origin xyz=-0.0375 0.0 0.0 rpy=0 0 0, axis 0 -1 0, limit lower=-1.570796 upper=1.570796 effort=7 velocity=20.943946
- added joint right_body_link0_joint: type fixed, parent body_link0, child right_link0, origin xyz=0.0 -0.031 0.698 rpy=1.5708 0 0
- added joint right_finger_joint1: type prismatic, parent right_hand, child right_right_finger, origin xyz=0 -0.006 0.015 rpy=0 0 0, axis 0 -1 0, limit lower=0.0 upper=0.044 effort=333 velocity=10.0
- added joint right_finger_joint2: type prismatic, parent right_hand, child right_left_finger, origin xyz=0 0.006 0.015 rpy=0 0 0, axis 0 1 0, limit lower=0.0 upper=0.044 effort=333 velocity=10.0, mimic joint=right_finger_joint1
- added joint right_hand_joint: type fixed, parent right_link7, child right_hand, origin xyz=0 -0.0 0.1001 rpy=0 0 0
- added joint right_hand_tcp_joint: type fixed, parent right_hand, child right_hand_tcp, origin xyz=0 -0.0 0.08 rpy=0 0 0
- added joint right_joint1: type revolute, parent right_link0, child right_link1, origin xyz=0.0 0.0 0.0625 rpy=0 0 0, axis 0 0 1, limit lower=-1.396263 upper=3.490659 effort=40 velocity=16.754666
- added joint right_joint2: type revolute, parent right_link1, child right_link2, origin xyz=-0.0301 0.0 0.06 rpy=1.57079632679 0 0, axis -1 0 0, limit lower=-0.17453267320510335 upper=3.3161253267948965 effort=40 velocity=16.754666
- added joint right_joint3: type revolute, parent right_link2, child right_link3, origin xyz=0.0301 0.0 0.06625 rpy=0 0 0, axis 0 0 1, limit lower=-1.570796 upper=1.570796 effort=27 velocity=5.445426
- added joint right_joint4: type revolute, parent right_link3, child right_link4, origin xyz=-0.0 0.0315 0.15375 rpy=0 0 0, axis 0 1 0, limit lower=0.0 upper=2.443461 effort=27 velocity=5.445426
- added joint right_joint5: type revolute, parent right_link4, child right_link5, origin xyz=0.0 -0.0315 0.0955 rpy=0 0 0, axis 0 0 1, limit lower=-1.570796 upper=1.570796 effort=7 velocity=20.943946
- added joint right_joint6: type revolute, parent right_link5, child right_link6, origin xyz=0.0375 0.0 0.1205 rpy=0 0 0, axis 1 0 0, limit lower=-0.785398 upper=0.785398 effort=7 velocity=20.943946
- added joint right_joint7: type revolute, parent right_link6, child right_link7, origin xyz=-0.0375 0.0 0.0 rpy=0 0 0, axis 0 1 0, limit lower=-1.570796 upper=1.570796 effort=7 velocity=20.943946

File: manipulator/OpenArm/openarm_v10_description/urdf/openarm_single.urdf (robot description, URDF)
Before this commit: robot openarm, 12 links, 11 joints
Links:
- removed link openarm_hand
- removed link openarm_hand_tcp
- removed link openarm_left_finger
- removed link openarm_link0
- removed link openarm_link1
- removed link openarm_link2
- removed link openarm_link3
- removed link openarm_link4
- removed link openarm_link5
- removed link openarm_link6
- removed link openarm_link7
- removed link openarm_right_finger
- added link hand, mass 0.35; collision mesh filename=package://openarm_v10_description/meshes/ee/openarm_hand/co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 scale=0.001 0.001 0.001; visual mesh filename=package://openarm_v10_description/meshes/ee/openarm_hand/vi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 scale=0.001 0.001 0.001
- added link hand_tcp
- added link left_finger, mass 0.03602545343277134; collision mesh filename=package://openarm_v10_description/meshes/ee/openarm_hand/co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 scale=0.001 0.001 0.001; visual mesh filename=package://openarm_v10_description/meshes/ee/openarm_hand/vi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 scale=0.001 0.001 0.001
- added link link0, mass 1.1432284943239561; collision mesh filename=package://openarm_v10_description/meshes/arm/v10/collision/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 scale=0.001 -0.001 0.001; visual mesh filename=package://openarm_v10_description/meshes/arm/v10/visual/lin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 scale=0.001 -0.001 0.001
- added link link1, mass 1.1416684646202298; collision mesh filename=package://openarm_v10_description/meshes/arm/v10/collision/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 scale=0.001 -0.001 0.001; visual mesh filename=package://openarm_v10_description/meshes/arm/v10/visual/lin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 scale=0.001 -0.001 0.001
- added link link2, mass 0.2775092746011571; collision mesh filename=package://openarm_v10_description/meshes/arm/v10/collision/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 scale=0.001 -0.001 0.001; visual mesh filename=package://openarm_v10_description/meshes/arm/v10/visual/lin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 scale=0.001 -0.001 0.001
- added link link3, mass 1.073863338202347; collision mesh filename=package://openarm_v10_description/meshes/arm/v10/collision/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 scale=0.001 -0.001 0.001; visual mesh filename=package://openarm_v10_description/meshes/arm/v10/visual/lin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 scale=0.001 -0.001 0.001
- added link link4, mass 0.6348534566833373; collision mesh filename=package://openarm_v10_description/meshes/arm/v10/collision/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 scale=0.001 0.001 0.001; visual mesh filename=package://openarm_v10_description/meshes/arm/v10/visual/lin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 scale=0.001 0.001 0.001
- added link link5, mass 0.6156588026168502; collision mesh filename=package://openarm_v10_description/meshes/arm/v10/collision/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 scale=0.001 -0.001 0.001; visual mesh filename=package://openarm_v10_description/meshes/arm/v10/visual/lin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 scale=0.001 -0.001 0.001
- added link link6, mass 0.475202773187987; collision mesh filename=package://openarm_v10_description/meshes/arm/v10/collision/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 scale=0.001 -0.001 0.001; visual mesh filename=package://openarm_v10_description/meshes/arm/v10/visual/lin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 scale=0.001 -0.001 0.001
- added link link7, mass 0.4659771327380578; collision mesh filename=package://openarm_v10_description/meshes/arm/v10/collision/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 scale=0.001 -0.001 0.001; visual mesh filename=package://openarm_v10_description/meshes/arm/v10/visual/lin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 scale=0.001 -0.001 0.001
- added link right_finger, mass 0.03602545343277134; collision mesh filename=package://openarm_v10_description/meshes/ee/openarm_hand/co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 scale=0.001 -0.001 0.001; visual mesh filename=package://openarm_v10_description/meshes/ee/openarm_hand/vi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 scale=0.001 -0.001 0.001
Joints:
- removed joint openarm_finger_joint1
- removed joint openarm_finger_joint2
- removed joint openarm_hand_joint
- removed joint openarm_hand_tcp_joint
- removed joint openarm_joint1
- removed joint openarm_joint2
- removed joint openarm_joint3
- removed joint openarm_joint4
- removed joint openarm_joint5
- removed joint openarm_joint6
- removed joint openarm_joint7
- added joint finger_joint1: type prismatic, parent hand, child right_finger, origin xyz=0 -0.006 0.015 rpy=0 0 0, axis 0 -1 0, limit lower=0.0 upper=0.044 effort=333 velocity=10.0
- added joint finger_joint2: type prismatic, parent hand, child left_finger, origin xyz=0 0.006 0.015 rpy=0 0 0, axis 0 1 0, limit lower=0.0 upper=0.044 effort=333 velocity=10.0, mimic joint=finger_joint1
- added joint hand_joint: type fixed, parent link7, child hand, origin xyz=0 -0.0 0.1001 rpy=0 0 0
- added joint hand_tcp_joint: type fixed, parent hand, child hand_tcp, origin xyz=0 -0.0 0.08 rpy=0 0 0
- added joint joint1: type revolute, parent link0, child link1, origin xyz=0.0 0.0 0.0625 rpy=0 0 0, axis 0 0 1, limit lower=-1.396263 upper=3.490659 effort=40 velocity=16.754666
- added joint joint2: type revolute, parent link1, child link2, origin xyz=-0.0301 0.0 0.06 rpy=0 0 0, axis -1 0 0, limit lower=-1.745329 upper=1.745329 effort=40 velocity=16.754666
- added joint joint3: type revolute, parent link2, child link3, origin xyz=0.0301 0.0 0.06625 rpy=0 0 0, axis 0 0 1, limit lower=-1.570796 upper=1.570796 effort=27 velocity=5.445426
- added joint joint4: type revolute, parent link3, child link4, origin xyz=-0.0 0.0315 0.15375 rpy=0 0 0, axis 0 1 0, limit lower=0.0 upper=2.443461 effort=27 velocity=5.445426
- added joint joint5: type revolute, parent link4, child link5, origin xyz=0.0 -0.0315 0.0955 rpy=0 0 0, axis 0 0 1, limit lower=-1.570796 upper=1.570796 effort=7 velocity=20.943946
- added joint joint6: type revolute, parent link5, child link6, origin xyz=0.0375 0.0 0.1205 rpy=0 0 0, axis 1 0 0, limit lower=-0.785398 upper=0.785398 effort=7 velocity=20.943946
- added joint joint7: type revolute, parent link6, child link7, origin xyz=-0.0375 0.0 0.0 rpy=0 0 0, axis 0 -1 0, limit lower=-1.570796 upper=1.570796 effort=7 velocity=20.943946

File: manipulator/OpenArm/openarm_v10_description/xacro/openarm_bimanual.xacro (robot description, xacro)
@@ -251,5 +251,5 @@
         <child link="${prefix}link8" />
       </joint> -->
-    <joint name="${prefix}right_openarm_body_link0_joint" type="fixed">
+    <joint name="${prefix}right_body_link0_joint" type="fixed">
       <parent link="${prefix}body_link0"/>
       <child link="${prefix}right_link0"/>
@@ -492,5 +492,5 @@
     <!-- <link name="${ee_prefix}hand"/> -->
     <!-- <joint name="${ee_prefix}hand_joint" type="fixed"> -->
-    <joint name="${prefix}left_openarm_hand_joint" type="fixed">
+    <joint name="${prefix}left_hand_joint" type="fixed">
       <parent link="${prefix}left_link7"/>
       <child link="${prefix}left_hand"/>
@@ -578,5 +578,5 @@
     <!-- <link name="${ee_prefix}hand"/> -->
     <!-- <joint name="${ee_prefix}hand_joint" type="fixed"> -->
-    <joint name="${prefix}right_openarm_hand_joint" type="fixed">
+    <joint name="${prefix}right_hand_joint" type="fixed">
       <parent link="${prefix}right_link7"/>
       <child link="${prefix}right_hand"/>

Commit message: fix: rename the 'world' link to 'base_link' solve the error. But rviz show the base support to black color instead of silver

File: manipulator/OpenArm/openarm_v10_description/urdf/openarm_bimanual.urdf (robot description, URDF)
Before this commit: robot openarm, 26 links, 25 joints
Links:
- removed link world
- added link base_link
Joints:
- removed joint body_world_joint
- added joint base_link_joint: type fixed, parent base_link, child body_link0, origin xyz=0 0 0 rpy=0 0 0

File: manipulator/OpenArm/openarm_v10_description/urdf/openarm_single.urdf (robot description, URDF)
Before this commit: robot openarm, 12 links, 11 joints
Links:
- added link base_link
Joints:
- added joint base_link_joint: type fixed, parent base_link, child link0, origin xyz=0 0 0 rpy=0 0 0

File: manipulator/OpenArm/openarm_v10_description/xacro/openarm_bimanual.xacro (robot description, xacro)
@@ -5,7 +5,7 @@
     <!-- Is the robot being simulated in gazebo? -->
     <!-- <xacro:arg name="gazebo" default="false" /> -->
-    <link name="${prefix}world"/>
-    <joint name="${prefix}body_world_joint" type="fixed">
-      <parent link="${prefix}world"/>
+    <link name="${prefix}base_link"/>
+    <joint name="${prefix}base_link_joint" type="fixed">
+      <parent link="${prefix}base_link"/>
       <child link="${prefix}body_link0"/>
       <origin rpy="0 0 0" xyz="0 0 0"/>

File: manipulator/OpenArm/openarm_v10_description/xacro/openarm_single.xacro (robot description, xacro)
@@ -5,4 +5,10 @@
     <!-- Is the robot being simulated in gazebo? -->
     <!-- <xacro:arg name="gazebo" default="false" /> -->
+    <link name="${prefix}base_link"/>
+    <joint name="${prefix}base_link_joint" type="fixed">
+      <parent link="${prefix}base_link"/>
+      <child link="${prefix}link0"/>
+      <origin rpy="0 0 0" xyz="0 0 0"/>
+    </joint>
     <link name="${prefix}link0">
       <visual name="${prefix}link0_visual">
