Commit message: add: support arm ocs2 control. Not test gazebo

File: manipulator/OpenArm/openarm_v10_description/xacro/ros2_control/openarm_bimanual.ros2_control.xacro (robot description, xacro)
@@ -1,8 +1,8 @@
 <?xml version="1.0"?>
 <robot xmlns:xacro="http://www.ros.org/wiki/xacro">
-  <xacro:macro name="openarm_system" params="name ros2_control_hardware_type">
+  <xacro:macro name="openarm_v10_system" params="name ros2_control_hardware_type">
     <xacro:property name="prefix" value="${name + '_' if name else ''}"/>
     <!-- Left Arm Hardware Interface -->
-    <ros2_control name="${prefix}openarm_left_system" type="system">
+    <ros2_control name="${prefix}openarm_v10_system" type="system">
       <hardware>
         <xacro:if value="${ros2_control_hardware_type == 'gz'}">
@@ -67,7 +67,7 @@
         <state_interface name="effort"/>
       </joint>
-    </ros2_control>
+    <!-- </ros2_control> -->
     <!-- Right Arm Hardware Interface -->
-    <ros2_control name="${prefix}openarm_right_system" type="system">
+    <!-- <ros2_control name="${prefix}openarm_right_system" type="system">
       <hardware>
         <xacro:if value="${ros2_control_hardware_type == 'gz'}">
@@ -82,5 +82,5 @@
           <param name="joint_states_topic">/isaac/joint_states</param>
         </xacro:if>
-      </hardware>
+      </hardware> -->
       <!-- Right Arm Joints -->
       <joint name="${prefix}right_joint1">

File: manipulator/OpenArm/openarm_v10_description/xacro/ros2_control/openarm_single.ros2_control.xacro (robot description, xacro)
@@ -1,7 +1,7 @@
 <?xml version="1.0"?>
 <robot xmlns:xacro="http://www.ros.org/wiki/xacro">
-  <xacro:macro name="openarm_system" params="name ros2_control_hardware_type">
+  <xacro:macro name="openarm_v10_system" params="name ros2_control_hardware_type">
     <xacro:property name="prefix" value="${name + '_' if name else ''}"/>
-    <ros2_control name="${prefix}openarm_system" type="system">
+    <ros2_control name="${prefix}openarm_v10_system" type="system">
       <hardware>
         <xacro:if value="${ros2_control_hardware_type == 'gz'}">

File: manipulator/OpenArm/openarm_v10_description/xacro/ros2_control/robot.xacro (robot description, xacro)
@@ -1,4 +1,4 @@
 <?xml version="1.0"?>
-<robot name="openarm" xmlns:xacro="http://www.ros.org/wiki/xacro">
+<robot name="openarm_v10" xmlns:xacro="http://www.ros.org/wiki/xacro">
   <xacro:arg name="ros2_control_hardware_type" default="mock_components"/>
   <link name="world"/>
@@ -9,29 +9,39 @@
   <xacro:arg name="type" default="bimanual"/>
   <!-- 根据type参数决定机器人类型 -->
-  <xacro:if value="${'$(arg type)' == 'single'}">
+  <xacro:if value="${'$(arg type)' == 'bimanual'}">
     <xacro:include filename="$(find openarm_v10_description)/xacro/openarm_bimanual.xacro"/>
     <xacro:OpenArm name=""/>
   </xacro:if>
-  <xacro:if value="${'$(arg type)' == 'bimanual'}">
+  <xacro:if value="${'$(arg type)' == 'single'}">
     <xacro:include filename="$(find openarm_v10_description)/xacro/openarm_single.xacro"/>
     <xacro:OpenArm name=""/>
   </xacro:if>
   <!-- 根据type参数决定ros2_control类型 -->
+  <xacro:if value="${'$(arg type)' == 'bimanual'}">
+    <xacro:include filename="$(find openarm_v10_description)/xacro/ros2_control/openarm_bimanual.ros2_control.xacro"/>
+    <xacro:openarm_v10_system name="" ros2_control_hardware_type="$(arg ros2_control_hardware_type)"/>
+  </xacro:if>
   <xacro:if value="${'$(arg type)' == 'single'}">
     <xacro:include filename="$(find openarm_v10_description)/xacro/ros2_control/openarm_single.ros2_control.xacro"/>
-    <xacro:openarm_system name="" ros2_control_hardware_type="$(arg ros2_control_hardware_type)"/>
+    <xacro:openarm_v10_system name="" ros2_control_hardware_type="$(arg ros2_control_hardware_type)"/>
   </xacro:if>
-  <xacro:if value="${'$(arg type)' == 'bimanual'}">
-    <xacro:include filename="$(find openarm_v10_description)/xacro/ros2_control/openarm_bimanual.ros2_control.xacro"/>
-    <xacro:openarm_system name="" ros2_control_hardware_type="$(arg ros2_control_hardware_type)"/>
-  </xacro:if>
+  <!-- Dynamically choose the correct YAML file -->
+  <!-- <ros2_control>
+    <xacro:if value="${'$(arg type)' == 'bimanual'}">
+      <parameters>$(find openarm_v10_description)/config/ros2_control/ros2_controllers.yaml</parameters>
+    </xacro:if>
+    <xacro:if value="${'$(arg type)' == 'single'}">
+      <parameters>$(find openarm_v10_description)/config/ros2_control/openarm_single.yaml</parameters>
+    </xacro:if>
+  </ros2_control> -->
+  <!-- Gazebo plugin configuration -->
   <xacro:arg name="gazebo" default="false" />
   <xacro:if value="$(arg gazebo)">
     <gazebo>
       <plugin filename="gz_ros2_control-system" name="gz_ros2_control::GazeboSimROS2ControlPlugin">
-        <xacro:if value="${'$(arg type)' == 'single'}">
+        <xacro:if value="${'$(arg type)' == 'bimanual'}">
           <parameters>$(find openarm_v10_description)/config/ros2_control/ros2_controllers.yaml</parameters>
         </xacro:if>
-        <xacro:if value="${'$(arg type)' == 'bimanual'}">
+        <xacro:if value="${'$(arg type)' == 'single'}">
           <parameters>$(find openarm_v10_description)/config/ros2_control/openarm_single.yaml</parameters>
         </xacro:if>
@@ -40,3 +50,2 @@
   </xacro:if>
 </robot>
-</robot>
