Commit message: fix gazebo error for agibot g1

File: common/gripper/changingtek_description/xacro/AG2F120S.xacro (robot description, xacro)
@@ -173,7 +173,7 @@
       <parent link="${prefix}gripper_base"/>
       <child link="${prefix}right_2_link"/>
-      <axis xyz="0 0 1"/>
-      <limit lower="0" upper="1" effort="40"  velocity="4.1887902047863905"/>
-      <mimic joint="${prefix}left_2_joint" multiplier="-1" offset="0"/>
+      <axis xyz="0 0 -1"/>
+      <limit lower="0" upper="1" effort="40"  velocity="4.1887902047863905"/>
+      <mimic joint="${prefix}left_2_joint" multiplier="1" offset="0"/>
     </joint>
     <link name="${prefix}right_1_link">
@@ -204,7 +204,7 @@
       <parent link="${prefix}gripper_base"/>
       <child link="${prefix}right_1_link"/>
-      <axis xyz="0 0 1"/>
-      <limit lower="0" upper="1" effort="40"  velocity="4.1887902047863905"/>
-      <mimic joint="${prefix}gripper_joint" multiplier="-1" offset="0"/>
+      <axis xyz="0 0 -1"/>
+      <limit lower="0" upper="1" effort="40"  velocity="4.1887902047863905"/>
+      <mimic joint="${prefix}gripper_joint" multiplier="1" offset="0"/>
     </joint>
     <link name="${prefix}right_support_link">
@@ -237,5 +237,5 @@
       <axis xyz="0 0 1"/>
       <limit lower="0" upper="1" effort="40"  velocity="4.1887902047863905"/>
-      <mimic joint="${prefix}right_1_joint" multiplier="-1" offset="0"/>
+      <mimic joint="${prefix}right_1_joint" multiplier="1" offset="0"/>
     </joint>
     <link name="${prefix}right_pad_link">

File: humanoid/Agibot/agibot_g1_description/xacro/120s_camera_stand.xacro (robot description, xacro)
@@ -3,5 +3,5 @@
 	<xacro:macro name="Camera" params="name">
 		<xacro:property name="prefix" value="${name + '_' if name else ''}"/>
-		<joint name="${prefix}camera_stand" type="fixed">
+		<joint name="${prefix}camera_stand_joint" type="fixed">
 			<parent link="${prefix}end_link"/>
 			<child link="${prefix}camera_stand"/>
@@ -14,5 +14,5 @@
 			</visual>
 		</link>
-		<joint name="${prefix}camera" type="fixed">
+		<joint name="${prefix}camera_joint" type="fixed">
 			<origin xyz="0 -0.079320 0.108617" rpy="0 -1.117 1.5708"/>
 			<parent link="${prefix}camera_stand"/>
