Commit message: grippers for cr5 robot

File: common/gripper/changingtek_description/xacro/AG2F90-C.xacro (robot description, xacro)
@@ -1,332 +1,346 @@
 <?xml version="1.0" ?>
 <robot xmlns:xacro="http://ros.org/wiki/xacro">
-  <xacro:macro name="AG2F90-C" params="name">
-    <xacro:property name="prefix" value="${name + '_' if name else ''}"/>
-    <link name="${prefix}gripper_base">
-      <inertial>
-        <origin xyz="3.45207417426861E-05 -0.000141443719270944 0.0415526970475172"/>
-        <mass value="0.310447980489903"/>
-        <inertia
-            ixx="0.000404388005636034"
-            ixy="-6.8589621466727E-08"
-            ixz="5.84928727366459E-08"
-            iyy="0.000296494720930083"
-            iyz="-1.79342738400452E-07"
-            izz="0.000212447969282029"/>
-      </inertial>
-      <visual>
-        <geometry>
-          <mesh filename="file://$(find changingtek_description)/meshes/AG2F90-C/visual/gripper_base.obj"/>
-        </geometry>
-      </visual>
-      <collision>
-        <geometry>
-          <mesh filename="file://$(find changingtek_description)/meshes/AG2F90-C/collision/gripper_base.obj"/>
-        </geometry>
-      </collision>
-    </link>
-    <link name="${prefix}left_1_link">
-      <inertial>
-        <origin xyz="-1.28088127539536E-18 0.0252734640095115 -0.00214040614650292"/>
-        <mass value="0.0129014357535444"/>
-        <inertia
-            ixx="3.35976482443235E-06"
-            ixy="-3.3181849198807E-25"
-            ixz="-3.35726667613063E-23"
-            iyy="1.65185846940368E-07"
-            iyz="2.63476012977044E-07"
-            izz="3.25394125032869E-06"/>
-      </inertial>
-      <visual>
-        <geometry>
-          <mesh filename="file://$(find changingtek_description)/meshes/AG2F90-C/visual/link_1.obj"/>
-        </geometry>
-      </visual>
-      <collision>
-        <geometry>
-          <mesh filename="file://$(find changingtek_description)/meshes/AG2F90-C/collision/link_1.obj"/>
-        </geometry>
-      </collision>
-    </link>
-    <joint name="${prefix}gripper_joint" type="revolute">
-      <origin xyz="0 -0.030141 0.090147" rpy="1.5708 0 0"/>
-      <parent link="${prefix}gripper_base"/>
-      <child link="${prefix}left_1_link"/>
-      <axis xyz="1 0 0"/>
-      <limit lower="0" upper="1" effort="25"  velocity="4.1887902047863905"/>
-    </joint>
-    <link name="${prefix}left_in_link">
-      <inertial>
-        <origin xyz="-1.75682286192042E-11 -0.0108820145632286 -0.00405362317350415"/>
-        <mass value="0.0134557296415635"/>
-        <inertia
-            ixx="1.43307384392376E-06"
-            ixy="-1.06834632214133E-14"
-            ixz="-4.88547951587875E-15"
-            iyy="3.88838933230828E-07"
-            iyz="-4.1814613493025E-07"
-            izz="1.33747540965672E-06"/>
-      </inertial>
-      <visual>
-        <geometry>
-          <mesh filename="file://$(find changingtek_description)/meshes/AG2F90-C/visual/in_link.obj"/>
-        </geometry>
-      </visual>
-      <collision>
-        <geometry>
-          <mesh filename="file://$(find changingtek_description)/meshes/AG2F90-C/collision/in_link.obj"/>
-        </geometry>
-      </collision>
-    </link>
-    <joint name="${prefix}left_in_Joint" type="revolute">
-      <origin xyz="0 0.023914 -0.0020253"/>
-      <parent link="${prefix}left_1_link"/>
-      <child link="${prefix}left_in_link"/>
-      <axis xyz="-1 0 0"/>
-      <limit lower="0" upper="1" effort="0" velocity="0"/>
-      <mimic joint="${prefix}gripper_joint" multiplier="0.1" offset="0"/>
-    </joint>
-    <link name="${prefix}left_up_link">
-      <inertial>
-        <origin xyz="8.69802213948566E-11 0.0124078988097444 -0.0072525614743534"/>
-        <mass value="0.014692561982481"/>
-        <inertia
-            ixx="2.35283034039115E-06"
-            ixy="3.49796352982052E-14"
-            ixz="-4.72158842036621E-15"
-            iyy="5.8942945477579E-07"
-            iyz="7.05860796345956E-07"
-            izz="2.07228020361883E-06"/>
-      </inertial>
-      <visual>
-        <geometry>
-          <mesh filename="file://$(find changingtek_description)/meshes/AG2F90-C/visual/up_link.obj"/>
-        </geometry>
-      </visual>
-      <collision>
-        <geometry>
-          <mesh filename="file://$(find changingtek_description)/meshes/AG2F90-C/collision/up_link.obj"/>
-        </geometry>
-      </collision>
-    </link>
-    <joint name="${prefix}left_up_Joint" type="revolute">
-      <origin xyz="0 0.054804 -0.0046413"/>
-      <parent link="${prefix}left_1_link"/>
-      <child link="${prefix}left_up_link"/>
-      <axis xyz="-1 0 0"/>
-      <limit lower="0" upper="1" effort="10"  velocity="4.1887902047863905"/>
-      <mimic joint="${prefix}gripper_joint" multiplier="1" offset="0"/>
-    </joint>
-    <link name="${prefix}left_Pad_link">
-      <inertial>
-        <origin xyz="-3.83777509579761E-08 0.00303135276101582 0.0028336970357949"/>
-        <mass value="0.0183171479595721"/>
-        <inertia
-            ixx="2.35683098270332E-06"
-            ixy="-4.7353365844279E-12"
-            ixz="-9.31433971475514E-13"
-            iyy="9.08136064346118E-07"
-            iyz="-1.55873132053129E-08"
-            izz="3.18448591439082E-06"/>
-      </inertial>
-      <visual>
-        <geometry>
-          <mesh filename="file://$(find changingtek_description)/meshes/AG2F90-C/visual/pad_link.obj"/>
-        </geometry>
-      </visual>
-      <collision>
-        <geometry>
-          <mesh filename="file://$(find changingtek_description)/meshes/AG2F90-C/collision/pad_link.obj"/>
-        </geometry>
-      </collision>
-    </link>
-    <joint name="${prefix}left_Pad_Joint" type="fixed">
-      <origin xyz="0 0.04125 -0.02425"/>
-      <parent link="${prefix}left_up_link"/>
-      <child link="${prefix}left_Pad_link"/>
-    </joint>
-    <link name="${prefix}left_2_link">
-      <inertial>
-        <origin xyz="5.08224485200288E-06 0.0327050710040551 -0.00276963392800038"/>
-        <mass value="0.0188752657753052"/>
-        <inertia
-            ixx="3.4145090175335E-06"
-            ixy="-3.3317063785682E-22"
-            ixz="-8.3582474326843E-22"
-            iyy="2.86837057727488E-07"
-            iyz="2.64809197911117E-07"
-            izz="3.39111483394506E-06"/>
-      </inertial>
-      <visual>
-        <geometry>
-          <mesh filename="file://$(find changingtek_description)/meshes/AG2F90-C/visual/link_2.obj"/>
-        </geometry>
-      </visual>
-      <collision>
-        <geometry>
-          <mesh filename="file://$(find changingtek_description)/meshes/AG2F90-C/collision/link_2.obj"/>
-        </geometry>
-      </collision>
-    </link>
-    <joint name="${prefix}left_2_Joint" type="revolute">
-      <origin xyz="0 -0.016 0.107" rpy="1.5708 0 0"/>
-      <parent link="${prefix}gripper_base"/>
-      <child link="${prefix}left_2_link"/>
-      <axis xyz="1 0 0"/>
-      <limit lower="0" upper="1" effort="10"  velocity="4.1887902047863905"/>
-      <mimic joint="${prefix}gripper_joint" multiplier="1" offset="0"/>
-    </joint>
-    <link name="${prefix}right_2_link">
-      <inertial>
-        <origin xyz="1.94651792710713E-17 0.0327174794493866 -0.00277053098700989"/>
-        <mass value="0.0188856364479881"/>
-        <inertia
-            ixx="3.41458781978465E-06"
-            ixy="2.85152078238725E-22"
-            ixz="9.8903086622122E-22"
-            iyy="2.86883124998043E-07"
-            iyz="2.64817198026894E-07"
-            izz="3.39114800103702E-06"/>
-      </inertial>
-      <visual>
-        <geometry>
-          <mesh filename="file://$(find changingtek_description)/meshes/AG2F90-C/visual/link_2.obj"/>
-        </geometry>
-      </visual>
-      <collision>
-        <geometry>
-          <mesh filename="file://$(find changingtek_description)/meshes/AG2F90-C/collision/link_2.obj"/>
-        </geometry>
-      </collision>
-    </link>
-    <joint name="${prefix}right_2_Joint" type="revolute">
-      <origin xyz="0 0.016 0.107" rpy="1.5708 0 3.1416"/>
-      <parent link="${prefix}gripper_base"/>
-      <child link="${prefix}right_2_link"/>
-      <axis xyz="1 0 0"/>
-      <limit lower="0" upper="1" effort="10"  velocity="4.1887902047863905"/>
-      <mimic joint="${prefix}gripper_joint" multiplier="1" offset="0"/>
-    </joint>
-    <link name="${prefix}right_1_link">
-      <inertial>
-        <origin xyz="-5.25233292439781E-19 0.0252734640095115 -0.00214040614650291"/>
-        <mass value="0.0129014357535444"/>
-        <inertia
-            ixx="3.35976482443235E-06"
-            ixy="-3.94978742494071E-23"
-            ixz="-2.72484926002331E-23"
-            iyy="1.65185846940368E-07"
-            iyz="2.63476012977044E-07"
-            izz="3.25394125032869E-06"/>
-      </inertial>
-      <visual>
-        <geometry>
-          <mesh filename="file://$(find changingtek_description)/meshes/AG2F90-C/visual/link_1.obj"/>
-        </geometry>
-      </visual>
-      <collision>
-        <geometry>
-          <mesh filename="file://$(find changingtek_description)/meshes/AG2F90-C/collision/link_1.obj"/>
-        </geometry>
-      </collision>
-    </link>
-    <joint name="${prefix}right_1_Joint" type="revolute">
-      <origin xyz="0 0.030141 0.090147" rpy="1.5708 0 3.1416"/>
-      <parent link="${prefix}gripper_base"/>
-      <child link="${prefix}right_1_link"/>
-      <axis xyz="1 0 0"/>
-      <limit lower="0" upper="1" effort="10"  velocity="4.1887902047863905"/>
-      <mimic joint="${prefix}gripper_joint" multiplier="1" offset="0"/>
-    </joint>
-    <link name="${prefix}right_in_link">
-      <inertial>
-        <origin xyz="-1.7568261982498E-11 -0.0108820145632292 -0.00405362317350229"/>
-        <mass value="0.0134557296415635"/>
-        <inertia
-            ixx="1.43307384392376E-06"
-            ixy="-1.06834687803419E-14"
-            ixz="-4.88548199727378E-15"
-            iyy="3.88838933230828E-07"
-            iyz="-4.1814613493025E-07"
-            izz="1.33747540965672E-06"/>
-      </inertial>
-      <visual>
-        <geometry>
-          <mesh filename="file://$(find changingtek_description)/meshes/AG2F90-C/visual/in_link.obj"/>
-        </geometry>
-      </visual>
-      <collision>
-        <geometry>
-          <mesh filename="file://$(find changingtek_description)/meshes/AG2F90-C/collision/in_link.obj"/>
-        </geometry>
-      </collision>
-    </link>
-    <joint name="${prefix}right_in_Joint" type="revolute">
-      <origin xyz="0 0.023914 -0.0020253"/>
-      <parent link="${prefix}right_1_link"/>
-      <child link="${prefix}right_in_link"/>
-      <axis xyz="-1 0 0"/>
-      <limit lower="0" upper="1" effort="0" velocity="0"/>
-      <mimic joint="${prefix}gripper_joint" multiplier="0.1" offset="0"/>
-    </joint>
-    <link name="${prefix}right_up_link">
-      <inertial>
-        <origin xyz="8.69814518862609E-11 0.0124078988097266 -0.00725256147435587"/>
-        <mass value="0.014692561982481"/>
-        <inertia
-            ixx="2.35283034039115E-06"
-            ixy="3.49796366331572E-14"
-            ixz="-4.72158801523363E-15"
-            iyy="5.89429454773258E-07"
-            iyz="7.05860796343296E-07"
-            izz="2.07228020362137E-06"/>
-      </inertial>
-      <visual>
-        <geometry>
-          <mesh filename="file://$(find changingtek_description)/meshes/AG2F90-C/visual/up_link.obj"/>
-        </geometry>
-      </visual>
-      <collision>
-        <geometry>
-          <mesh filename="file://$(find changingtek_description)/meshes/AG2F90-C/collision/up_link.obj"/>
-        </geometry>
-      </collision>
-    </link>
-    <joint name="${prefix}right_up_Joint" type="revolute">
-      <origin xyz="0 0.054804 -0.0046413"/>
-      <parent link="${prefix}right_1_link"/>
-      <child link="${prefix}right_up_link"/>
-      <axis xyz="-1 0 0"/>
-      <limit lower="0" upper="1" effort="10"  velocity="4.1887902047863905"/>
-      <mimic joint="${prefix}gripper_joint" multiplier="1" offset="0"/>
-    </joint>
-    <link name="${prefix}right_Pad_link">
-      <inertial>
-        <origin xyz="-3.83777500494227E-08 0.0030313527610159 0.00283369703564792"/>
-        <mass value="0.0366342959191441"/>
-        <inertia
-            ixx="4.71366196540664E-06"
-            ixy="-9.47067316877366E-12"
-            ixz="-1.8628679404863E-12"
-            iyy="1.81627212869223E-06"
-            iyz="-3.11746264105278E-08"
-            izz="6.36897182878164E-06"/>
-      </inertial>
-      <visual>
-        <geometry>
-          <mesh filename="file://$(find changingtek_description)/meshes/AG2F90-C/visual/pad_link.obj"/>
-        </geometry>
-      </visual>
-      <collision>
-        <geometry>
-          <mesh filename="file://$(find changingtek_description)/meshes/AG2F90-C/collision/pad_link.obj"/>
-        </geometry>
-      </collision>
-    </link>
-    <joint name="${prefix}right_Pad_Joint" type="fixed">
-      <origin xyz="0 0.04125 -0.02425"/>
-      <parent link="${prefix}right_up_link"/>
-      <child link="${prefix}right_Pad_link"/>
-    </joint>
-  </xacro:macro>
+	<xacro:macro name="AG2F90-C" params="name use_flange:=false">
+		<xacro:property name="prefix" value="${name + '_' if name else ''}"/>
+		<xacro:if value="${use_flange}">
+			<link name="${prefix}flange">
+				<visual>
+					<geometry>
+						<mesh filename="file://$(find changingtek_description)/meshes/AG2F90-C/visual/flange.obj"/>
+					</geometry>
+				</visual>
+			</link>
+			<joint name="${prefix}flange_joint" type="fixed">
+				<origin xyz="0 0 0.0195"/>
+				<parent link="${prefix}flange"/>
+				<child link="${prefix}gripper_base"/>
+			</joint>
+		</xacro:if>
+		<link name="${prefix}gripper_base">
+			<inertial>
+				<origin xyz="3.45207417426861E-05 -0.000141443719270944 0.0415526970475172"/>
+				<mass value="0.310447980489903"/>
+				<inertia
+						ixx="0.000404388005636034"
+						ixy="-6.8589621466727E-08"
+						ixz="5.84928727366459E-08"
+						iyy="0.000296494720930083"
+						iyz="-1.79342738400452E-07"
+						izz="0.000212447969282029"/>
+			</inertial>
+			<visual>
+				<geometry>
+					<mesh filename="file://$(find changingtek_description)/meshes/AG2F90-C/visual/gripper_base.obj"/>
+				</geometry>
+			</visual>
+			<collision>
+				<geometry>
+					<mesh filename="file://$(find changingtek_description)/meshes/AG2F90-C/collision/gripper_base.obj"/>
+				</geometry>
+			</collision>
+		</link>
+		<link name="${prefix}left_1_link">
+			<inertial>
+				<origin xyz="-1.28088127539536E-18 0.0252734640095115 -0.00214040614650292"/>
+				<mass value="0.0129014357535444"/>
+				<inertia
+						ixx="3.35976482443235E-06"
+						ixy="-3.3181849198807E-25"
+						ixz="-3.35726667613063E-23"
+						iyy="1.65185846940368E-07"
+						iyz="2.63476012977044E-07"
+						izz="3.25394125032869E-06"/>
+			</inertial>
+			<visual>
+				<geometry>
+					<mesh filename="file://$(find changingtek_description)/meshes/AG2F90-C/visual/link_1.obj"/>
+				</geometry>
+			</visual>
+			<collision>
+				<geometry>
+					<mesh filename="file://$(find changingtek_description)/meshes/AG2F90-C/collision/link_1.obj"/>
+				</geometry>
+			</collision>
+		</link>
+		<joint name="${prefix}gripper_joint" type="revolute">
+			<origin xyz="0 -0.030141 0.090147" rpy="1.5708 0 0"/>
+			<parent link="${prefix}gripper_base"/>
+			<child link="${prefix}left_1_link"/>
+			<axis xyz="1 0 0"/>
+			<limit lower="0" upper="1" effort="25" velocity="4.1887902047863905"/>
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
File: manipulator/Dobot/cr5_description/urdf/cr5.urdf (robot description, URDF)
Before this commit: robot DobotCR5, 7 links, 6 joints
Links:
- link Link6: geometry collision cylinder length=0.28 radius=0.04; visual mesh filename=package://cr5_description/meshes/visual/Link6.obj

File: manipulator/Dobot/cr5_description/xacro/arm.xacro (robot description, xacro)
@@ -1,7 +1,7 @@
 <?xml version="1.0"?>
 <robot name="cr5_robot" xmlns:xacro="http://ros.org/wiki/xacro">
+	<xacro:property name="PI" value="3.1415926535897931"/>
 	<xacro:macro name="CR5" params="name collider:=convex">
 		<xacro:property name="prefix" value="${name + '_' if name else ''}"/>
-		<xacro:property name="PI" value="3.1415926535897931"/>
 		<link name="base_link">
 			<inertial>

Commit message: grippers for cr5 robot

File: common/gripper/changingtek_description/xacro/AG2F90-C.xacro (robot description, xacro)
@@ -5,4 +5,15 @@
 		<xacro:if value="${use_flange}">
 			<link name="${prefix}flange">
+				<inertial>
+					<origin xyz="-0.000388 0.002345 0.0"/>
+					<mass value="0.114"/>
+					<inertia
+						ixx="0.000040105"
+						ixy="0.000000214"
+						ixz="0.0"
+						iyy="0.000085776"
+						iyz="0.0"
+						izz="0.000054044"/>
+				</inertial>
 				<visual>
 					<geometry>
@@ -10,4 +21,9 @@
 					</geometry>
 				</visual>
+				<collision>
+					<geometry>
+						<mesh filename="file://$(find changingtek_description)/meshes/AG2F90-C/collision/flange.obj"/>
+					</geometry>
+				</collision>
 			</link>
 			<joint name="${prefix}flange_joint" type="fixed">

Commit message: galaxea r1x gripper fix

File: common/gripper/changingtek_description/xacro/AG2F90-C.xacro (robot description, xacro)
@@ -21,9 +21,4 @@
 					</geometry>
 				</visual>
-				<collision>
-					<geometry>
-						<mesh filename="file://$(find changingtek_description)/meshes/AG2F90-C/collision/flange.obj"/>
-					</geometry>
-				</collision>
 			</link>
 			<joint name="${prefix}flange_joint" type="fixed">
