Commit message: gazebo sim by dart engine

File: common/gripper/changingtek_description/xacro/AG2F90-C.xacro (robot description, xacro)
@@ -3,4 +3,5 @@
 	<xacro:macro name="AG2F90-C" params="name use_flange:=false">
 		<xacro:property name="prefix" value="${name + '_' if name else ''}"/>
+		<xacro:property name="PI" value="3.1415926535897931"/>
 		<xacro:if value="${use_flange}">
 			<link name="${prefix}flange">
@@ -47,5 +48,5 @@
 			<collision>
 				<geometry>
-					<mesh filename="file://$(find changingtek_description)/meshes/AG2F90-C/collision/gripper_base.obj"/>
+					<mesh filename="file://$(find changingtek_description)/meshes/AG2F90-C/collision/base.stl"/>
 				</geometry>
 			</collision>
@@ -70,14 +71,14 @@
 			<collision>
 				<geometry>
-					<mesh filename="file://$(find changingtek_description)/meshes/AG2F90-C/collision/link_1.obj"/>
+					<mesh filename="file://$(find changingtek_description)/meshes/AG2F90-C/collision/link_1.stl"/>
 				</geometry>
 			</collision>
 		</link>
 		<joint name="${prefix}gripper_joint" type="revolute">
-			<origin xyz="0 -0.030141 0.090147" rpy="1.5708 0 0"/>
+			<origin xyz="0 -0.030141 0.090147" rpy="${PI/2} 0 0"/>
 			<parent link="${prefix}gripper_base"/>
 			<child link="${prefix}left_1_link"/>
 			<axis xyz="1 0 0"/>
-			<limit lower="0" upper="1" effort="25" velocity="4.1887902047863905"/>
+			<limit lower="0" upper="1" effort="50" velocity="${PI}"/>
 		</joint>
 		<link name="${prefix}left_in_link">
@@ -100,5 +101,5 @@
 			<collision>
 				<geometry>
-					<mesh filename="file://$(find changingtek_description)/meshes/AG2F90-C/collision/in_link.obj"/>
+					<mesh filename="file://$(find changingtek_description)/meshes/AG2F90-C/collision/in_link.stl"/>
 				</geometry>
 			</collision>
@@ -109,5 +110,5 @@
 			<child link="${prefix}left_in_link"/>
 			<axis xyz="-1 0 0"/>
-			<limit lower="0" upper="1" effort="0" velocity="0"/>
+			<limit lower="0" upper="1" effort="50" velocity="${PI}"/>
 			<mimic joint="${prefix}gripper_joint" multiplier="0.1" offset="0"/>
 		</joint>
@@ -131,5 +132,5 @@
 			<collision>
 				<geometry>
-					<mesh filename="file://$(find changingtek_description)/meshes/AG2F90-C/collision/up_link.obj"/>
+					<mesh filename="file://$(find changingtek_description)/meshes/AG2F90-C/collision/up_link.stl"/>
 				</geometry>
 			</collision>
@@ -140,6 +141,6 @@
 			<child link="${prefix}left_up_link"/>
 			<axis xyz="-1 0 0"/>
-			<limit lower="0" upper="1" effort="10" velocity="4.1887902047863905"/>
-			<mimic joint="${prefix}gripper_joint" multiplier="1" offset="0"/>
+			<limit lower="0" upper="1" effort="50" velocity="${PI}"/>
+			<mimic joint="${prefix}gripper_joint"/>
 		</joint>
 		<link name="${prefix}left_Pad_link">
@@ -162,5 +163,5 @@
 			<collision>
 				<geometry>
-					<mesh filename="file://$(find changingtek_description)/meshes/AG2F90-C/collision/pad_link.obj"/>
+					<mesh filename="file://$(find changingtek_description)/meshes/AG2F90-C/collision/pad_link.stl"/>
 				</geometry>
 			</collision>
@@ -190,15 +191,15 @@
 			<collision>
 				<geometry>
-					<mesh filename="file://$(find changingtek_description)/meshes/AG2F90-C/collision/link_2.obj"/>
+					<mesh filename="file://$(find changingtek_description)/meshes/AG2F90-C/collision/link_2.stl"/>
 				</geometry>
 			</collision>
 		</link>
 		<joint name="${prefix}left_2_Joint" type="revolute">
-			<origin xyz="0 -0.016 0.107" rpy="1.5708 0 0"/>
+			<origin xyz="0 -0.016 0.107" rpy="${PI/2} 0 0"/>
 			<parent link="${prefix}gripper_base"/>
 			<child link="${prefix}left_2_link"/>
 			<axis xyz="1 0 0"/>
-			<limit lower="0" upper="1" effort="10" velocity="4.1887902047863905"/>
-			<mimic joint="${prefix}gripper_joint" multiplier="1" offset="0"/>
+			<limit lower="0" upper="1" effort="50" velocity="${PI}"/>
+			<mimic joint="${prefix}gripper_joint"/>
 		</joint>
 		<link name="${prefix}right_2_link">
@@ -221,15 +222,15 @@
 			<collision>
 				<geometry>
-					<mesh filename="file://$(find changingtek_description)/meshes/AG2F90-C/collision/link_2.obj"/>
+					<mesh filename="file://$(find changingtek_description)/meshes/AG2F90-C/collision/link_2.stl"/>
 				</geometry>
 			</collision>
 		</link>
 		<joint name="${prefix}right_2_Joint" type="revolute">
-			<origin xyz="0 0.016 0.107" rpy="1.5708 0 3.1416"/>
+			<origin xyz="0 0.016 0.107" rpy="${PI/2} 0 ${PI}"/>
 			<parent link="${prefix}gripper_base"/>
 			<child link="${prefix}right_2_link"/>
 			<axis xyz="1 0 0"/>
-			<limit lower="0" upper="1" effort="10" velocity="4.1887902047863905"/>
-			<mimic joint="${prefix}gripper_joint" multiplier="1" offset="0"/>
+			<limit lower="0" upper="1" effort="50" velocity="${PI}"/>
+			<mimic joint="${prefix}left_2_Joint"/>
 		</joint>
 		<link name="${prefix}right_1_link">
@@ -252,15 +253,15 @@
 			<collision>
 				<geometry>
-					<mesh filename="file://$(find changingtek_description)/meshes/AG2F90-C/collision/link_1.obj"/>
+					<mesh filename="file://$(find changingtek_description)/meshes/AG2F90-C/collision/link_1.stl"/>
 				</geometry>
 			</collision>
 		</link>
 		<joint name="${prefix}right_1_Joint" type="revolute">
-			<origin xyz="0 0.030141 0.090147" rpy="1.5708 0 3.1416"/>
+			<origin xyz="0 0.030141 0.090147" rpy="${PI/2} 0 ${PI}"/>
 			<parent link="${prefix}gripper_base"/>
 			<child link="${prefix}right_1_link"/>
 			<axis xyz="1 0 0"/>
-			<limit lower="0" upper="1" effort="10" velocity="4.1887902047863905"/>
-			<mimic joint="${prefix}gripper_joint" multiplier="1" offset="0"/>
+			<limit lower="0" upper="1" effort="50" velocity="${PI}"/>
+			<mimic joint="${prefix}gripper_joint"/>
 		</joint>
 		<link name="${prefix}right_in_link">
@@ -283,5 +284,5 @@
 			<collision>
 				<geometry>
-					<mesh filename="file://$(find changingtek_description)/meshes/AG2F90-C/collision/in_link.obj"/>
+					<mesh filename="file://$(find changingtek_description)/meshes/AG2F90-C/collision/in_link.stl"/>
 				</geometry>
 			</collision>
@@ -292,6 +293,6 @@
 			<child link="${prefix}right_in_link"/>
 			<axis xyz="-1 0 0"/>
-			<limit lower="0" upper="1" effort="0" velocity="0"/>
-			<mimic joint="${prefix}gripper_joint" multiplier="0.1" offset="0"/>
+			<limit lower="0" upper="1" effort="50" velocity="${PI}"/>
+			<mimic joint="${prefix}right_1_Joint" multiplier="0.1" offset="0"/>
 		</joint>
 		<link name="${prefix}right_up_link">
@@ -314,5 +315,5 @@
 			<collision>
 				<geometry>
-					<mesh filename="file://$(find changingtek_description)/meshes/AG2F90-C/collision/up_link.obj"/>
+					<mesh filename="file://$(find changingtek_description)/meshes/AG2F90-C/collision/up_link.stl"/>
 				</geometry>
 			</collision>
@@ -323,6 +324,6 @@
 			<child link="${prefix}right_up_link"/>
 			<axis xyz="-1 0 0"/>
-			<limit lower="0" upper="1" effort="10" velocity="4.1887902047863905"/>
-			<mimic joint="${prefix}gripper_joint" multiplier="1" offset="0"/>
+			<limit lower="0" upper="1" effort="50" velocity="${PI}"/>
+			<mimic joint="${prefix}right_1_Joint"/>
 		</joint>
 		<link name="${prefix}right_Pad_link">
@@ -345,5 +346,5 @@
 			<collision>
 				<geometry>
-					<mesh filename="file://$(find changingtek_description)/meshes/AG2F90-C/collision/pad_link.obj"/>
+					<mesh filename="file://$(find changingtek_description)/meshes/AG2F90-C/collision/pad_link.stl"/>
 				</geometry>
 			</collision>

File: manipulator/Dobot/cr5_description/xacro/arm.xacro (robot description, xacro)
@@ -18,5 +18,5 @@
 				<collision>
 					<geometry>
-						<mesh filename="file://$(find cr5_description)/meshes/collision/base_link.obj"/>
+						<mesh filename="file://$(find cr5_description)/meshes/collision/base_link.stl"/>
 					</geometry>
 				</collision>
@@ -51,10 +51,10 @@
 				<collision>
 					<geometry>
-						<mesh filename="file://$(find cr5_description)/meshes/collision/Link1_0.obj"/>
-					</geometry>
-				</collision>
-				<collision>
-					<geometry>
-						<mesh filename="file://$(find cr5_description)/meshes/collision/Link1_1.obj"/>
+						<mesh filename="file://$(find cr5_description)/meshes/collision/Link1_0.stl"/>
+					</geometry>
+				</collision>
+				<collision>
+					<geometry>
+						<mesh filename="file://$(find cr5_description)/meshes/collision/Link1_1.stl"/>
 					</geometry>
 				</collision>
@@ -89,15 +89,15 @@
 				<collision>
 					<geometry>
-						<mesh filename="file://$(find cr5_description)/meshes/collision/Link2_0.obj"/>
-					</geometry>
-				</collision>
-				<collision>
-					<geometry>
-						<mesh filename="file://$(find cr5_description)/meshes/collision/Link2_1.obj"/>
-					</geometry>
-				</collision>
-				<collision>
-					<geometry>
-						<mesh filename="file://$(find cr5_description)/meshes/collision/Link2_2.obj"/>
+						<mesh filename="file://$(find cr5_description)/meshes/collision/Link2_0.stl"/>
+					</geometry>
+				</collision>
+				<collision>
+					<geometry>
+						<mesh filename="file://$(find cr5_description)/meshes/collision/Link2_1.stl"/>
+					</geometry>
+				</collision>
+				<collision>
+					<geometry>
+						<mesh filename="file://$(find cr5_description)/meshes/collision/Link2_2.stl"/>
 					</geometry>
 				</collision>
@@ -145,15 +145,15 @@
 				<collision>
 					<geometry>
-						<mesh filename="file://$(find cr5_description)/meshes/collision/Link3_0.obj"/>
-					</geometry>
-				</collision>
-				<collision>
-					<geometry>
-						<mesh filename="file://$(find cr5_description)/meshes/collision/Link3_1.obj"/>
-					</geometry>
-				</collision>
-				<collision>
-					<geometry>
-						<mesh filename="file://$(find cr5_description)/meshes/collision/Link3_2.obj"/>
+						<mesh filename="file://$(find cr5_description)/meshes/collision/Link3_0.stl"/>
+					</geometry>
+				</collision>
+				<collision>
+					<geometry>
+						<mesh filename="file://$(find cr5_description)/meshes/collision/Link3_1.stl"/>
+					</geometry>
+				</collision>
+				<collision>
+					<geometry>
+						<mesh filename="file://$(find cr5_description)/meshes/collision/Link3_2.stl"/>
 					</geometry>
 				</collision>
@@ -201,10 +201,5 @@
 				<collision>
 					<geometry>
-						<mesh filename="file://$(find cr5_description)/meshes/collision/Link4_0.obj"/>
-					</geometry>
-				</collision>
-				<collision>
-					<geometry>
-						<mesh filename="file://$(find cr5_description)/meshes/collision/Link4_1.obj"/>
+						<mesh filename="file://$(find cr5_description)/meshes/collision/Link4.stl"/>
 					</geometry>
 				</collision>
@@ -240,5 +235,5 @@
 				<collision>
 					<geometry>
-						<mesh filename="file://$(find cr5_description)/meshes/collision/Link5.obj"/>
+						<mesh filename="file://$(find cr5_description)/meshes/collision/Link5.stl"/>
 					</geometry>
 				</collision>
@@ -274,5 +269,5 @@
 				<collision>
 					<geometry>
-						<mesh filename="file://$(find cr5_description)/meshes/collision/Link6.obj"/>
+						<mesh filename="file://$(find cr5_description)/meshes/collision/Link6.stl"/>
 					</geometry>
 				</collision>

File: manipulator/Dobot/cr5_description/xacro/ros2_control/cr5.ros2_control.xacro (robot description, xacro)
@@ -74,13 +74,16 @@
         <state_interface name="effort"/>
       </joint>
-      <xacro:if value="${'$(arg type)' != 'empty'}">
-        <joint name="${prefix}gripper_joint">
-          <command_interface name="position"/>
-          <state_interface name="position">
-            <param name="initial_value">0.0</param>
-          </state_interface>
-          <state_interface name="velocity"/>
-          <state_interface name="effort"/>
-        </joint>
+      <!-- 夹爪接口定义 -->
+      <xacro:if value="${'$(arg type)' == 'AG2F90-C'}">
+        <xacro:include filename="$(find changingtek_description)/xacro/ros2_control/AG2F90-C.xacro"/>
+        <xacro:ag2f90c_interfaces name=""/>
+      </xacro:if>
+      <xacro:if value="${'$(arg type)' == 'AG2F120S'}">
+        <xacro:include filename="$(find changingtek_description)/xacro/ros2_control/AG2F120S.xacro"/>
+        <xacro:ag2f120s_interfaces name="" />
+      </xacro:if>
+      <xacro:if value="${'$(arg type)' == 'robotiq85'}">
+        <xacro:include filename="$(find robotiq_description)/xacro/ros2_control/2F85.xacro"/>
+        <xacro:robotiq_2f85_interfaces name=""/>
       </xacro:if>
     </ros2_control>

Commit message: add soft pad for ag2f90c

File: common/gripper/changingtek_description/xacro/AG2F90-C.xacro (robot description, xacro)
@@ -1,5 +1,5 @@
 <?xml version="1.0" ?>
 <robot xmlns:xacro="http://ros.org/wiki/xacro">
-	<xacro:macro name="AG2F90-C" params="name use_flange:=false">
+	<xacro:macro name="AG2F90-C" params="name use_flange:=false pad:=default">
 		<xacro:property name="prefix" value="${name + '_' if name else ''}"/>
 		<xacro:property name="PI" value="3.1415926535897931"/>
@@ -80,5 +80,10 @@
 			<child link="${prefix}left_1_link"/>
 			<axis xyz="1 0 0"/>
-			<limit lower="0" upper="1" effort="50" velocity="${PI}"/>
+			<xacro:if value="${pad == 'soft'}">
+				<limit lower="0.189" upper="1" effort="50" velocity="${PI}"/>
+			</xacro:if>
+			<xacro:if value="${pad == 'default' or pad == ''}">
+				<limit lower="0" upper="1" effort="50" velocity="${PI}"/>
+			</xacro:if>
 		</joint>
 		<link name="${prefix}left_in_link">
@@ -158,10 +163,20 @@
 			<visual>
 				<geometry>
-					<mesh filename="file://$(find changingtek_description)/meshes/AG2F90-C/visual/pad_link.obj"/>
-				</geometry>
-			</visual>
-			<collision>
-				<geometry>
-					<mesh filename="file://$(find changingtek_description)/meshes/AG2F90-C/collision/pad_link.stl"/>
+					<xacro:if value="${pad == 'soft'}">
+						<mesh filename="file://$(find changingtek_description)/meshes/AG2F90-C/visual/pad_link_soft.obj"/>
+					</xacro:if>
+					<xacro:if value="${pad == 'default' or pad == ''}">
+						<mesh filename="file://$(find changingtek_description)/meshes/AG2F90-C/visual/pad_link.obj"/>
+					</xacro:if>
+				</geometry>
+			</visual>
+			<collision>
+				<geometry>
+					<xacro:if value="${pad == 'soft'}">
+						<mesh filename="file://$(find changingtek_description)/meshes/AG2F90-C/visual/pad_link_soft.obj"/>
+					</xacro:if>
+					<xacro:if value="${pad == 'default' or pad == ''}">
+						<mesh filename="file://$(find changingtek_description)/meshes/AG2F90-C/collision/pad_link.stl"/>
+					</xacro:if>
 				</geometry>
 			</collision>
@@ -341,10 +356,20 @@
 			<visual>
 				<geometry>
-					<mesh filename="file://$(find changingtek_description)/meshes/AG2F90-C/visual/pad_link.obj"/>
-				</geometry>
-			</visual>
-			<collision>
-				<geometry>
-					<mesh filename="file://$(find changingtek_description)/meshes/AG2F90-C/collision/pad_link.stl"/>
+					<xacro:if value="${pad == 'soft'}">
+						<mesh filename="file://$(find changingtek_description)/meshes/AG2F90-C/visual/pad_link_soft.obj"/>
+					</xacro:if>
+					<xacro:if value="${pad == 'default' or pad == ''}">
+						<mesh filename="file://$(find changingtek_description)/meshes/AG2F90-C/visual/pad_link.obj"/>
+					</xacro:if>
+				</geometry>
+			</visual>
+			<collision>
+				<geometry>
+					<xacro:if value="${pad == 'soft'}">
+						<mesh filename="file://$(find changingtek_description)/meshes/AG2F90-C/visual/pad_link_soft.obj"/>
+					</xacro:if>
+					<xacro:if value="${pad == 'default' or pad == ''}">
+						<mesh filename="file://$(find changingtek_description)/meshes/AG2F90-C/collision/pad_link.stl"/>
+					</xacro:if>
 				</geometry>
 			</collision>

File: common/gripper/changingtek_description/xacro/ros2_control/AG2F90-C.xacro (robot description, xacro)
@@ -9,5 +9,5 @@
       <command_interface name="position"/>
       <state_interface name="position">
-        <param name="initial_value">0.0</param>
+        <param name="initial_value">1.0</param>
       </state_interface>
       <state_interface name="velocity"/>

File: manipulator/Dobot/cr5_description/xacro/grippers.xacro (robot description, xacro)
@@ -20,4 +20,13 @@
 		</joint>
 	</xacro:if>
+	<xacro:if value="${'$(arg type)' == 'AG2F90-C-Soft'}">
+		<xacro:include filename="$(find changingtek_description)/xacro/AG2F90-C.xacro"/>
+		<xacro:AG2F90-C name="" use_flange="true" pad="soft"/>
+		<joint name="gripper_fix" type="fixed">
+			<parent link="Link6"/>
+			<child link="flange"/>
+			<origin rpy="0 0 ${PI/2}"/>
+		</joint>
+	</xacro:if>
 	<xacro:if value="${'$(arg type)' == 'AG2F120S'}">
 		<xacro:include filename="$(find changingtek_description)/xacro/AG2F120S.xacro"/>

File: manipulator/Dobot/cr5_description/xacro/ros2_control/cr5.ros2_control.xacro (robot description, xacro)
@@ -75,5 +75,5 @@
       </joint>
       <!-- 夹爪接口定义 -->
-      <xacro:if value="${'$(arg type)' == 'AG2F90-C'}">
+      <xacro:if value="${'$(arg type)' == 'AG2F90-C' or '$(arg type)' == 'AG2F90-C-Soft'}">
         <xacro:include filename="$(find changingtek_description)/xacro/ros2_control/AG2F90-C.xacro"/>
         <xacro:ag2f90c_interfaces name=""/>
