Commit message: open arm collision

File: manipulator/OpenArm/openarm_description/xacro/arm.xacro (robot description, xacro)
@@ -13,6 +13,5 @@
 			<collision>
 				<geometry>
-					<mesh filename="file://$(find openarm_description)/meshes/arm/v10/collision/link0_symp.stl"
-								scale="0.001 ${direction*0.001} 0.001"/>
+					<mesh filename="file://$(find openarm_description)/meshes/arm/collision/base.stl"/>
 				</geometry>
 			</collision>
@@ -32,8 +31,7 @@
 			</visual>
 			<collision>
-				<origin xyz="-0.0 0.0 -0.0625"/>
-				<geometry>
-					<mesh filename="file://$(find openarm_description)/meshes/arm/v10/collision/link1_symp.stl"
-								scale="0.001 ${direction*0.001} 0.001"/>
+				<geometry>
+					<mesh filename="file://$(find openarm_description)/meshes/arm/collision/link1.stl"
+								scale="1 ${direction*1} 1"/>
 				</geometry>
 			</collision>
@@ -66,6 +64,6 @@
 				<origin xyz="0.0301 0.0 -0.1225"/>
 				<geometry>
-					<mesh filename="file://$(find openarm_description)/meshes/arm/v10/collision/link2_symp.stl"
-								scale="0.001 ${direction*0.001} 0.001"/>
+					<mesh filename="file://$(find openarm_description)/meshes/arm/collision/link2.stl"
+								scale="1 ${direction} 1"/>
 				</geometry>
 			</collision>
@@ -77,10 +75,10 @@
 		</link>
 		<joint name="${prefix}joint2" type="revolute">
-			<xacro:if value="${direction == -1}">
-				<origin rpy="-1.57079632679 0 0" xyz="-0.0301 0.0 0.06"/>
-			</xacro:if>
-			<xacro:if value="${direction == 1}">
-				<origin rpy="1.57079632679 0 0" xyz="-0.0301 0.0 0.06"/>
-			</xacro:if>
+			<xacro:if value="${prefix == ''}">
+				<origin xyz="-0.0301 0.0 0.06"/>
+			</xacro:if>
+			<xacro:unless value="${prefix == ''}">
+				<origin rpy="${direction*1.57079632679} 0 0" xyz="-0.0301 0.0 0.06"/>
+			</xacro:unless>
 			<parent link="${prefix}link1"/>
 			<child link="${prefix}link2"/>
@@ -101,8 +99,7 @@
 			</visual>
 			<collision>
-				<origin xyz="-0.0 -0.0 -0.18875"/>
-				<geometry>
-					<mesh filename="file://$(find openarm_description)/meshes/arm/v10/collision/link3_symp.stl"
-								scale="0.001 ${direction*0.001} 0.001"/>
+				<geometry>
+					<mesh filename="file://$(find openarm_description)/meshes/arm/collision/link3.stl"
+								scale="1 ${direction} 1"/>
 				</geometry>
 			</collision>
@@ -128,8 +125,6 @@
 			</visual>
 			<collision>
-				<origin xyz="0.0 -0.0315 -0.3425"/>
-				<geometry>
-					<mesh filename="file://$(find openarm_description)/meshes/arm/v10/collision/link4_symp.stl"
-								scale="0.001 0.001 0.001"/>
+				<geometry>
+					<mesh filename="file://$(find openarm_description)/meshes/arm/collision/link4.stl"/>
 				</geometry>
 			</collision>
@@ -155,8 +150,7 @@
 			</visual>
 			<collision>
-				<origin xyz="-0.0 -0.0 -0.438"/>
-				<geometry>
-					<mesh filename="file://$(find openarm_description)/meshes/arm/v10/collision/link5_symp.stl"
-								scale="0.001 ${direction*0.001} 0.001"/>
+				<geometry>
+					<mesh filename="file://$(find openarm_description)/meshes/arm/collision/link5.stl"
+								scale="1 ${direction} 1"/>
 				</geometry>
 			</collision>
@@ -183,8 +177,7 @@
 			</visual>
 			<collision>
-				<origin xyz="-0.0375 -0.0 -0.5585"/>
-				<geometry>
-					<mesh filename="file://$(find openarm_description)/meshes/arm/v10/collision/link6_symp.stl"
-								scale="0.001 ${direction*0.001} 0.001"/>
+				<geometry>
+					<mesh filename="file://$(find openarm_description)/meshes/arm/collision/link6.stl"
+								scale="1 ${direction*1} 1"/>
 				</geometry>
 			</collision>
@@ -211,8 +204,7 @@
 			</visual>
 			<collision>
-				<origin xyz="0.0 -0.0 -0.5585"/>
-				<geometry>
-					<mesh filename="file://$(find openarm_description)/meshes/arm/v10/collision/link7_symp.stl"
-								scale="0.001 ${direction*0.001} 0.001"/>
+				<geometry>
+					<mesh filename="file://$(find openarm_description)/meshes/arm/collision/link7.stl"
+								scale="1 ${direction*1} 1"/>
 				</geometry>
 			</collision>

File: manipulator/OpenArm/openarm_description/xacro/robot.xacro (robot description, xacro)
@@ -1,13 +1,72 @@
 <?xml version="1.0"?>
 <robot name="OpenArm" xmlns:xacro="http://www.ros.org/wiki/xacro">
-  <xacro:arg name="type" default="single"/>
-  <!-- 根据type参数决定机器人类型 -->
-  <xacro:if value="${'$(arg type)' == 'bimanual'}">
-    <xacro:include filename="$(find openarm_description)/xacro/openarm_bimanual.xacro"/>
-    <xacro:openarm_bimanual name=""/>
-  </xacro:if>
-  <xacro:if value="${'$(arg type)' == 'single'}">
-    <xacro:include filename="$(find openarm_description)/xacro/openarm_single.xacro"/>
-    <xacro:openarm_single name=""/>
-  </xacro:if>
+	<xacro:include filename="$(find openarm_description)/xacro/arm.xacro"/>
+	<xacro:include filename="$(find openarm_description)/xacro/gripper.xacro"/>
+	<xacro:arg name="type" default="bimanual"/>
+	<!-- 根据type参数决定机器人类型 -->
+	<xacro:if value="${'$(arg type)' == 'bimanual'}">
+		<!-- Base link -->
+		<link name="base_link">
+			<inertial>
+				<mass value="13.89"/>
+				<inertia ixx="1.653" ixy="0.0" ixz="0.0" iyy="1.653" iyz="0.0" izz="0.051"/>
+			</inertial>
+			<visual>
+				<geometry>
+					<mesh filename="file://$(find openarm_description)/meshes/body/body.obj"/>
+				</geometry>
+			</visual>
+			<collision>
+				<geometry>
+					<mesh filename="file://$(find openarm_description)/meshes/body/body.stl"/>
+				</geometry>
+			</collision>
+		</link>
+		<!-- Left Arm -->
+		<joint name="left_arm_base_joint" type="fixed">
+			<parent link="base_link"/>
+			<child link="left_base_link"/>
+			<origin rpy="-1.5708 0 0" xyz="0.0 0.031 0.698"/>
+		</joint>
+		<xacro:OpenArm name="left" direction="-1"/>
+		<!-- Right Arm -->
+		<joint name="right_arm_base_joint" type="fixed">
+			<parent link="base_link"/>
+			<child link="right_base_link"/>
+			<origin rpy="1.5708 0 0" xyz="0.0 -0.031 0.698"/>
+		</joint>
+		<xacro:OpenArm name="right" direction="1"/>
+		<!-- Left Gripper -->
+		<joint name="left_hand_joint" type="fixed">
+			<parent link="left_link7"/>
+			<child link="left_hand"/>
+			<origin xyz="0 -0.0 0.1001"/>
+		</joint>
+		<xacro:OpenArmGripper name="left"/>
+		<!-- Right Gripper -->
+		<joint name="right_hand_joint" type="fixed">
+			<parent link="right_link7"/>
+			<child link="right_hand"/>
+			<origin xyz="0 -0.0 0.1001"/>
+		</joint>
+		<xacro:OpenArmGripper name="right"/>
+	</xacro:if>
+	<xacro:if value="${'$(arg type)' == 'right'}">
+		<xacro:OpenArm name=""/>
+		<joint name="hand_joint" type="fixed">
+			<parent link="link7"/>
+			<child link="hand"/>
+			<origin xyz="0 -0.0 0.1001"/>
+		</joint>
+		<xacro:OpenArmGripper name=""/>
+	</xacro:if>
+	<xacro:if value="${'$(arg type)' == 'left'}">
+		<xacro:OpenArm name="" direction="-1"/>
+		<joint name="hand_joint" type="fixed">
+			<parent link="link7"/>
+			<child link="hand"/>
+			<origin xyz="0 -0.0 0.1001"/>
+		</joint>
+		<xacro:OpenArmGripper name=""/>
+	</xacro:if>
 </robot>
