Commit message: fix: ocs2 demo for bimanual gz, isaac,none hardware. But left/right arm only support none hardware

File: manipulator/OpenArm/openarm_description/xacro/ros2_control/openarm_bimanual.ros2_control.xacro (robot description, xacro)
@@ -70,5 +70,5 @@
         <state_interface name="effort"/>
       </joint>
-      <joint name="${prefix}left_finger_joint1">
+      <joint name="${prefix}left_gripper_joint">
         <command_interface name="position"/>
         <state_interface name="position"/>
@@ -119,5 +119,5 @@
         <state_interface name="effort"/>
       </joint>
-      <joint name="${prefix}right_finger_joint1">
+      <joint name="${prefix}right_gripper_joint">
         <command_interface name="position"/>
         <state_interface name="position"/>

File: manipulator/OpenArm/openarm_description/xacro/ros2_control/openarm_single.ros2_control.xacro (robot description, xacro)
@@ -69,5 +69,5 @@
         <state_interface name="effort"/>
       </joint>
-      <joint name="${prefix}finger_joint1">
+      <joint name="${prefix}gripper_joint">
         <command_interface name="position"/>
         <state_interface name="position"/>

File: manipulator/OpenArm/openarm_description/xacro/ros2_control/robot.xacro (robot description, xacro)
@@ -8,13 +8,6 @@
 	</joint>
   <xacro:arg name="type" default="bimanual"/>
-  <!-- 根据type参数决定机器人类型 -->
-  <xacro:if value="${'$(arg type)' == 'bimanual'}">
-    <xacro:include filename="$(find openarm_description)/xacro/openarm_bimanual.xacro"/>
-    <xacro:openarm_bimanual name=""/>
-  </xacro:if>
-  <xacro:if value="${'$(arg type)' == 'single'}">
-    <xacro:include filename="$(find openarm_description)/xacro/openarm_single.xacro"/>
-    <xacro:openarm_single name=""/>
-  </xacro:if>
+  <!-- 直接include robot.xacro并根据type参数传递 -->
+  <xacro:include filename="$(find openarm_description)/xacro/robot.xacro" type="$(arg type)"/>
   <!-- 根据type参数决定ros2_control类型 -->
   <xacro:if value="${'$(arg type)' == 'bimanual'}">
@@ -22,5 +15,9 @@
     <xacro:openarm_v10_system name="" ros2_control_hardware_type="$(arg ros2_control_hardware_type)"/>
   </xacro:if>
-  <xacro:if value="${'$(arg type)' == 'single'}">
+  <xacro:if value="${'$(arg type)' == 'left'}">
+    <xacro:include filename="$(find openarm_description)/xacro/ros2_control/openarm_single.ros2_control.xacro"/>
+    <xacro:openarm_v10_system name="" ros2_control_hardware_type="$(arg ros2_control_hardware_type)"/>
+  </xacro:if>
+  <xacro:if value="${'$(arg type)' == 'right'}">
     <xacro:include filename="$(find openarm_description)/xacro/ros2_control/openarm_single.ros2_control.xacro"/>
     <xacro:openarm_v10_system name="" ros2_control_hardware_type="$(arg ros2_control_hardware_type)"/>
@@ -34,5 +31,8 @@
           <parameters>$(find openarm_description)/config/ros2_control/openarm_bimanual.yaml</parameters>
         </xacro:if>
-        <xacro:if value="${'$(arg type)' == 'single'}">
+        <xacro:if value="${'$(arg type)' == 'left'}">
+          <parameters>$(find openarm_description)/config/ros2_control/openarm_single.yaml</parameters>
+        </xacro:if>
+        <xacro:if value="${'$(arg type)' == 'right'}">
           <parameters>$(find openarm_description)/config/ros2_control/openarm_single.yaml</parameters>
         </xacro:if>

Commit message: add: modulize the ros2 control xacro files

File: manipulator/OpenArm/openarm_description/xacro/ros2_control/openarm_bimanual.ros2_control.xacro (robot description, xacro)
@@ -2,127 +2,13 @@
 <robot xmlns:xacro="http://www.ros.org/wiki/xacro">
   <xacro:macro name="openarm_v10_system" params="name ros2_control_hardware_type">
-    <xacro:property name="prefix" value="${name + '_' if name else ''}"/>
-    <!-- Left Arm Hardware Interface -->
-    <ros2_control name="${prefix}openarm_v10_system" type="system">
-      <hardware>
-        <xacro:if value="${ros2_control_hardware_type == 'gz'}">
-          <plugin>gz_ros2_control/GazeboSimSystem</plugin>
-        </xacro:if>
-        <xacro:if value="${ros2_control_hardware_type == 'mock_components'}">
-          <plugin>mock_components/GenericSystem</plugin>
-        </xacro:if>
-        <xacro:if value="${ros2_control_hardware_type == 'isaac'}">
-          <plugin>topic_based_ros2_control/TopicBasedSystem</plugin>
-          <param name="joint_commands_topic">/isaac/joint_command</param>
-          <param name="joint_states_topic">/isaac/joint_states</param>
-          <param name="sum_wrapped_joint_states">false</param>
-          <param name="initialize_commands_from_state">true</param>
-        </xacro:if>
-        <xacro:if value="${ros2_control_hardware_type == 'real'}">
-          <plugin>topic_based_ros2_control/TopicBasedSystem</plugin>
-          <param name="joint_commands_topic">/joint_command_robot</param>
-          <param name="joint_states_topic">/joint_states_robot</param>
-          <param name="sum_wrapped_joint_states">false</param>
-          <param name="initialize_commands_from_state">true</param>
-        </xacro:if>
-      </hardware>
+    <xacro:include filename="$(find openarm_description)/xacro/ros2_control/openarm_arm_gripper_system.xacro"/>
+    <xacro:include filename="$(find openarm_description)/xacro/ros2_control/hardware_system.xacro"/>
+    <!-- Hardware Interface -->
+    <ros2_control name="$openarm_v10_system" type="system">
+      <xacro:hardware_system ros2_control_hardware_type="${ros2_control_hardware_type}"/>
       <!-- Left Arm Joints -->
-      <joint name="${prefix}left_joint1">
-        <command_interface name="position"/>
-        <state_interface name="position"/>
-        <state_interface name="velocity"/>
-        <state_interface name="effort"/>
-      </joint>
-      <joint name="${prefix}left_joint2">
-        <command_interface name="position"/>
-        <state_interface name="position"/>
-        <state_interface name="velocity"/>
-        <state_interface name="effort"/>
-      </joint>
-      <joint name="${prefix}left_joint3">
-        <command_interface name="position"/>
-        <state_interface name="position"/>
-        <state_interface name="velocity"/>
-        <state_interface name="effort"/>
-      </joint>
-      <joint name="${prefix}left_joint4">
-        <command_interface name="position"/>
-        <state_interface name="position"/>
-        <state_interface name="velocity"/>
-        <state_interface name="effort"/>
-      </joint>
-      <joint name="${prefix}left_joint5">
-        <command_interface name="position"/>
-        <state_interface name="position"/>
-        <state_interface name="velocity"/>
-        <state_interface name="effort"/>
-      </joint>
-      <joint name="${prefix}left_joint6">
-        <command_interface name="position"/>
-        <state_interface name="position"/>
-        <state_interface name="velocity"/>
-        <state_interface name="effort"/>
-      </joint>
-      <joint name="${prefix}left_joint7">
-        <command_interface name="position"/>
-        <state_interface name="position"/>
-        <state_interface name="velocity"/>
-        <state_interface name="effort"/>
-      </joint>
-      <joint name="${prefix}left_gripper_joint">
-        <command_interface name="position"/>
-        <state_interface name="position"/>
-        <state_interface name="velocity"/>
-        <state_interface name="effort"/>
-      </joint>
+      <xacro:openarm_arm_gripper_system name="left" />
       <!-- Right Arm Joints -->
-      <joint name="${prefix}right_joint1">
-        <command_interface name="position"/>
-        <state_interface name="position"/>
-        <state_interface name="velocity"/>
-        <state_interface name="effort"/>
-      </joint>
-      <joint name="${prefix}right_joint2">
-        <command_interface name="position"/>
-        <state_interface name="position"/>
-        <state_interface name="velocity"/>
-        <state_interface name="effort"/>
-      </joint>
-      <joint name="${prefix}right_joint3">
-        <command_interface name="position"/>
-        <state_interface name="position"/>
-        <state_interface name="velocity"/>
-        <state_interface name="effort"/>
-      </joint>
-      <joint name="${prefix}right_joint4">
-        <command_interface name="position"/>
-        <state_interface name="position"/>
-        <state_interface name="velocity"/>
-        <state_interface name="effort"/>
-      </joint>
-      <joint name="${prefix}right_joint5">
-        <command_interface name="position"/>
-        <state_interface name="position"/>
-        <state_interface name="velocity"/>
-        <state_interface name="effort"/>
-      </joint>
-      <joint name="${prefix}right_joint6">
-        <command_interface name="position"/>
-        <state_interface name="position"/>
-        <state_interface name="velocity"/>
-        <state_interface name="effort"/>
-      </joint>
-      <joint name="${prefix}right_joint7">
-        <command_interface name="position"/>
-        <state_interface name="position"/>
-        <state_interface name="velocity"/>
-        <state_interface name="effort"/>
-      </joint>
-      <joint name="${prefix}right_gripper_joint">
-        <command_interface name="position"/>
-        <state_interface name="position"/>
-        <state_interface name="velocity"/>
-        <state_interface name="effort"/>
-      </joint>
+      <xacro:openarm_arm_gripper_system name="right" />
     </ros2_control>
   </xacro:macro>

File: manipulator/OpenArm/openarm_description/xacro/ros2_control/openarm_single.ros2_control.xacro (robot description, xacro)
@@ -2,77 +2,11 @@
 <robot xmlns:xacro="http://www.ros.org/wiki/xacro">
   <xacro:macro name="openarm_v10_system" params="name ros2_control_hardware_type">
+    <xacro:include filename="$(find openarm_description)/xacro/ros2_control/openarm_arm_gripper_system.xacro"/>
+    <xacro:include filename="$(find openarm_description)/xacro/ros2_control/hardware_system.xacro"/>
     <xacro:property name="prefix" value="${name + '_' if name else ''}"/>
-    <ros2_control name="${prefix}openarm_v10_system" type="system">
-      <hardware>
-        <xacro:if value="${ros2_control_hardware_type == 'gz'}">
-          <plugin>gz_ros2_control/GazeboSimSystem</plugin>
-        </xacro:if>
-        <xacro:if value="${ros2_control_hardware_type == 'mock_components'}">
-          <plugin>mock_components/GenericSystem</plugin>
-        </xacro:if>
-        <xacro:if value="${ros2_control_hardware_type == 'isaac'}">
-          <plugin>topic_based_ros2_control/TopicBasedSystem</plugin>
-          <param name="joint_commands_topic">/isaac/joint_command</param>
-          <param name="joint_states_topic">/isaac/joint_states</param>
-          <param name="sum_wrapped_joint_states">false</param>
-          <param name="initialize_commands_from_state">true</param>
-        </xacro:if>
-        <xacro:if value="${ros2_control_hardware_type == 'real'}">
-          <plugin>topic_based_ros2_control/TopicBasedSystem</plugin>
-          <param name="joint_commands_topic">/joint_command_robot</param>
-          <param name="joint_states_topic">/joint_states_robot</param>
-          <param name="sum_wrapped_joint_states">false</param>
-          <param name="initialize_commands_from_state">true</param>
-        </xacro:if>
-      </hardware>
+    <ros2_control name="$openarm_v10_system" type="system">
+      <xacro:hardware_system ros2_control_hardware_type="${ros2_control_hardware_type}"/>
       <!-- 关节接口定义 -->
-      <joint name="${prefix}joint1">
-        <command_interface name="position"/>
-        <state_interface name="position"/>
-        <state_interface name="velocity"/>
-        <state_interface name="effort"/>
-      </joint>
-      <joint name="${prefix}joint2">
-        <command_interface name="position"/>
-        <state_interface name="position"/>
-        <state_interface name="velocity"/>
-        <state_interface name="effort"/>
-      </joint>
-      <joint name="${prefix}joint3">
-        <command_interface name="position"/>
-        <state_interface name="position"/>
-        <state_interface name="velocity"/>
-        <state_interface name="effort"/>
-      </joint>
-      <joint name="${prefix}joint4">
-        <command_interface name="position"/>
-        <state_interface name="position"/>
-        <state_interface name="velocity"/>
-        <state_interface name="effort"/>
-      </joint>
-      <joint name="${prefix}joint5">
-        <command_interface name="position"/>
-        <state_interface name="position"/>
-        <state_interface name="velocity"/>
-        <state_interface name="effort"/>
-      </joint>
-      <joint name="${prefix}joint6">
-        <command_interface name="position"/>
-        <state_interface name="position"/>
-        <state_interface name="velocity"/>
-        <state_interface name="effort"/>
-      </joint>
-      <joint name="${prefix}joint7">
-        <command_interface name="position"/>
-        <state_interface name="position"/>
-        <state_interface name="velocity"/>
-        <state_interface name="effort"/>
-      </joint>
-      <joint name="${prefix}gripper_joint">
-        <command_interface name="position"/>
-        <state_interface name="position"/>
-        <state_interface name="velocity"/>
-        <state_interface name="effort"/>
-      </joint>
+      <xacro:openarm_arm_gripper_system name="" />
     </ros2_control>
   </xacro:macro>
