Commit message: fix openarm xacro

File: manipulator/OpenArm/openarm_description/xacro/ros2_control/interfaces.xacro (robot description, xacro)
@@ -1,5 +1,5 @@
 <?xml version="1.0"?>
 <robot xmlns:xacro="http://www.ros.org/wiki/xacro">
-  <xacro:macro name="openarm_arm_gripper_system" params="name">
+  <xacro:macro name="openarm_interfaces" params="name">
     <xacro:property name="prefix" value="${name + '_' if name else ''}"/>
     <!-- 关节接口定义 -->

File: manipulator/OpenArm/openarm_description/xacro/ros2_control/robot.xacro (robot description, xacro)
@@ -1,42 +1,63 @@
 <?xml version="1.0"?>
 <robot name="openarm_v10" xmlns:xacro="http://www.ros.org/wiki/xacro">
-  <xacro:arg name="ros2_control_hardware_type" default="mock_components"/>
-  <link name="world"/>
+	<xacro:arg name="ros2_control_hardware_type" default="mock_components"/>
+	<link name="world"/>
 	<joint name="world_fixed" type="fixed">
 		<parent link="world"/>
 		<child link="base_link"/>
 	</joint>
-  <xacro:arg name="type" default="bimanual"/>
-  <!-- 直接include robot.xacro并根据type参数传递 -->
-  <xacro:include filename="$(find openarm_description)/xacro/robot.xacro" type="$(arg type)"/>
-  <!-- 根据type参数决定ros2_control类型 -->
-  <xacro:if value="${'$(arg type)' == 'bimanual'}">
-    <xacro:include filename="$(find openarm_description)/xacro/ros2_control/openarm_bimanual.ros2_control.xacro"/>
-    <xacro:openarm_v10_system name="" ros2_control_hardware_type="$(arg ros2_control_hardware_type)"/>
-  </xacro:if>
-  <xacro:if value="${'$(arg type)' == 'left'}">
-    <xacro:include filename="$(find openarm_description)/xacro/ros2_control/openarm_single.ros2_control.xacro"/>
-    <xacro:openarm_v10_system name="" ros2_control_hardware_type="$(arg ros2_control_hardware_type)"/>
-  </xacro:if>
-  <xacro:if value="${'$(arg type)' == 'right'}">
-    <xacro:include filename="$(find openarm_description)/xacro/ros2_control/openarm_single.ros2_control.xacro"/>
-    <xacro:openarm_v10_system name="" ros2_control_hardware_type="$(arg ros2_control_hardware_type)"/>
-  </xacro:if>
-  <!-- Gazebo plugin configuration -->
-  <xacro:arg name="gazebo" default="false" />
-  <xacro:if value="$(arg gazebo)">
-    <gazebo>
-      <plugin filename="gz_ros2_control-system" name="gz_ros2_control::GazeboSimROS2ControlPlugin">
-        <xacro:if value="${'$(arg type)' == 'bimanual'}">
-          <parameters>$(find openarm_description)/config/ros2_control/ros2_controllers.yaml</parameters>
-        </xacro:if>
-        <xacro:if value="${'$(arg type)' == 'left'}">
-          <parameters>$(find openarm_description)/config/ros2_control/left.yaml</parameters>
-        </xacro:if>
-        <xacro:if value="${'$(arg type)' == 'right'}">
-          <parameters>$(find openarm_description)/config/ros2_control/right.yaml</parameters>
-        </xacro:if>
-      </plugin>
-    </gazebo>
-  </xacro:if>
+	<xacro:arg name="type" default="bimanual"/>
+	<!-- 直接include robot.xacro并根据type参数传递 -->
+	<xacro:include filename="$(find openarm_description)/xacro/robot.xacro"/>
+	<xacro:include filename="$(find openarm_description)/xacro/ros2_control/interfaces.xacro"/>
+	<ros2_control name="openarm_$(arg type)_system" type="system">
+		<hardware>
+			<xacro:if value="${'$(arg ros2_control_hardware_type)' == 'gz'}">
+				<plugin>gz_ros2_control/GazeboSimSystem</plugin>
+			</xacro:if>
+			<xacro:if value="${'$(arg ros2_control_hardware_type)' == 'mock_components'}">
+				<plugin>mock_components/GenericSystem</plugin>
+			</xacro:if>
+			<xacro:if value="${'$(arg ros2_control_hardware_type)' == 'isaac'}">
+				<plugin>topic_based_ros2_control/TopicBasedSystem</plugin>
+				<param name="joint_commands_topic">/isaac/joint_command</param>
+				<param name="joint_states_topic">/isaac/joint_states</param>
+				<param name="sum_wrapped_joint_states">false</param>
+				<param name="initialize_commands_from_state">true</param>
+			</xacro:if>
+			<xacro:if value="${'$(arg ros2_control_hardware_type)' == 'real'}">
+				<plugin>topic_based_ros2_control/TopicBasedSystem</plugin>
+				<param name="joint_commands_topic">/joint_command_robot</param>
+				<param name="joint_states_topic">/joint_states_robot</param>
+				<param name="sum_wrapped_joint_states">false</param>
+				<param name="initialize_commands_from_state">true</param>
+			</xacro:if>
+		</hardware>
+		<xacro:if value="${'$(arg type)' == 'bimanual'}">
+			<!-- Left Arm Joints -->
+			<xacro:openarm_interfaces name="left"/>
+			<!-- Right Arm Joints -->
+			<xacro:openarm_interfaces name="right"/>
+		</xacro:if>
+		<xacro:if value="${'$(arg type)' == 'left' or '$(arg type)' == 'right'}">
+			<xacro:openarm_interfaces name=""/>
+		</xacro:if>
+	</ros2_control>
+	<!-- Gazebo plugin configuration -->
+	<xacro:arg name="gazebo" default="false"/>
+	<xacro:if value="$(arg gazebo)">
+		<gazebo>
+			<plugin filename="gz_ros2_control-system" name="gz_ros2_control::GazeboSimROS2ControlPlugin">
+				<xacro:if value="${'$(arg type)' == 'bimanual'}">
+					<parameters>$(find openarm_description)/config/ros2_control/ros2_controllers.yaml</parameters>
+				</xacro:if>
+				<xacro:if value="${'$(arg type)' == 'left'}">
+					<parameters>$(find openarm_description)/config/ros2_control/left.yaml</parameters>
+				</xacro:if>
+				<xacro:if value="${'$(arg type)' == 'right'}">
+					<parameters>$(find openarm_description)/config/ros2_control/right.yaml</parameters>
+				</xacro:if>
+			</plugin>
+		</gazebo>
+	</xacro:if>
 </robot>
