Commit message: add pi

File: humanoid/Unitree/unitree_g1_description/xacro/arm.xacro (robot description, xacro)
@@ -1,4 +1,5 @@
 <?xml version="1.0" ?>
 <robot xmlns:xacro="http://www.ros.org/wiki/xacro">
+	<xacro:property name="PI" value="3.1415926535897931"/>
 	<xacro:macro name="UnitreeG1Arm" params="name direction:=1">
 		<!--
@@ -24,5 +25,5 @@
 			</visual>
 			<collision>
-				<origin xyz="0 ${direction*0.04} -0.01" rpy="0 1.5707963267948966 0"/>
+				<origin xyz="0 ${direction*0.04} -0.01" rpy="0 ${PI/2} 0"/>
 				<geometry>
 					<cylinder radius="0.03" length="0.05"/>

File: humanoid/Unitree/unitree_g1_description/xacro/robot.xacro (robot description, xacro)
@@ -1,3 +1,4 @@
 <robot name="g1_29dof" xmlns:xacro="http://www.ros.org/wiki/xacro">
+	<xacro:property name="PI" value="3.1415926535897931"/>
 	<xacro:arg name="end_effector" default="rubber_hand"/>
 	<!-- Include the modular macros -->
@@ -36,10 +37,10 @@
 		<xacro:BrainCoHand name="right" direction="-1"/>
 		<joint name="left_hand_palm_joint" type="fixed" dont_collapse="true">
-			<origin xyz="0.0415 0.003 0" rpy="-1.5708 0 -1.5708"/>
+			<origin xyz="0.0415 0.003 0" rpy="${-PI/2} 0 ${-PI/2}"/>
 			<parent link="left_wrist_yaw_link"/>
 			<child link="left_hand_base"/>
 		</joint>
 		<joint name="right_hand_palm_joint" type="fixed" dont_collapse="true">
-			<origin xyz="0.0415 -0.003 0" rpy="1.5708 0 1.5708"/>
+			<origin xyz="0.0415 -0.003 0" rpy="${PI/2} 0 ${PI/2}"/>
 			<parent link="right_wrist_yaw_link"/>
 			<child link="right_hand_base"/>

File: manipulator/Dobot/cr5_description/urdf/cr5.urdf (robot description, URDF)
Before this commit: robot DobotCR5, 7 links, 6 joints
Joints:
- joint joint1: limit lower=-6.28318 upper=6.28318 effort=300 velocity=3.14159 -> lower=-6.283185307179586 upper=6.283185307179586 effort=300 velocity=3.141592653589793
- joint joint2: limit lower=-6.28318 upper=6.28318 effort=300 velocity=3.14159 -> lower=-6.283185307179586 upper=6.283185307179586 effort=300 velocity=3.141592653589793; origin rpy=1.5708 1.5708 0 -> rpy=1.5707963267948966 1.5707963267948966 0
- joint joint4: limit lower=-6.28318 upper=6.28318 effort=300 velocity=3.14159 -> lower=-6.283185307179586 upper=6.283185307179586 effort=300 velocity=3.141592653589793; origin xyz=-0.357 0 0.141 rpy=0 0 -1.5708 -> xyz=-0.357 0 0.141 rpy=0 0 -1.5707963267948966
- joint joint5: limit lower=-6.28318 upper=6.28318 effort=300 velocity=3.14159 -> lower=-6.283185307179586 upper=6.283185307179586 effort=300 velocity=3.141592653589793; origin xyz=0 -0.116 0 rpy=1.5708 0 0 -> xyz=0 -0.116 0 rpy=1.5707963267948966 0 0
- joint joint6: limit lower=-6.28318 upper=6.28318 effort=300 velocity=3.14159 -> lower=-6.283185307179586 upper=6.283185307179586 effort=300 velocity=3.141592653589793; origin xyz=0 0.105 0 rpy=-1.5708 0 0 -> xyz=0 0.105 0 rpy=-1.5707963267948966 0 0

File: manipulator/Dobot/cr5_description/xacro/arm.xacro (robot description, xacro)
@@ -3,15 +3,10 @@
 	<xacro:macro name="CR5" params="name collider:=convex">
 		<xacro:property name="prefix" value="${name + '_' if name else ''}"/>
+		<xacro:property name="PI" value="3.1415926535897931"/>
 		<link name="base_link">
 			<inertial>
 				<origin xyz="-8.0961E-06 0.0019103 0.028995"/>
 				<mass value="0.90882"/>
-				<inertia
-						ixx="0.0014545"
-						ixy="4.2968E-08"
-						ixz="-1.8199E-07"
-						iyy="0.001345"
-						iyz="-6.243E-06"
-						izz="0.002155"/>
+			<inertia ixx="0.0014545" ixy="4.2968E-08" ixz="-1.8199E-07" iyy="0.001345" iyz="-6.243E-06" izz="0.002155"/>
 			</inertial>
 			<visual>
@@ -46,11 +41,5 @@
 				<origin xyz="-8.7268E-07 -0.0032576 -0.0076748"/>
 				<mass value="1.6123"/>
-				<inertia
-						ixx="0.0029122"
-						ixy="5.7387E-09"
-						ixz="1.9945E-08"
-						iyy="0.0028191"
-						iyz="0.00044094"
-						izz="0.0032836"/>
+			<inertia ixx="0.0029122" ixy="5.7387E-09" ixz="1.9945E-08" iyy="0.0028191" iyz="0.00044094" izz="0.0032836"/>
 			</inertial>
 			<visual>
@@ -84,5 +73,5 @@
 			<child link="Link1"/>
 			<axis xyz="0 0 1"/>
-			<limit lower="-6.28318" upper="6.28318" effort="300" velocity="3.14159"/>
+			<limit lower="${-2*PI}" upper="${2*PI}" effort="300" velocity="${PI}"/>
 		</joint>
 		<link name="Link2">
@@ -90,11 +79,5 @@
 				<origin xyz="-0.21351 -1.3842E-06 0.14252"/>
 				<mass value="5.5186"/>
-				<inertia
-						ixx="0.0085919"
-						ixy="7.5552E-07"
-						ixz="-7.8922E-07"
-						iyy="0.027553"
-						iyz="1.4629E-07"
-						izz="0.028294"/>
+			<inertia ixx="0.0085919" ixy="7.5552E-07" ixz="-7.8922E-07" iyy="0.027553" iyz="1.4629E-07" izz="0.028294"/>
 			</inertial>
 			<visual>
@@ -128,5 +111,5 @@
 				</collision>
 				<collision>
-					<origin rpy="0 1.5708 0" xyz="-0.2 0 0.15"/>
+					<origin rpy="0 ${PI/2} 0" xyz="-0.2 0 0.15"/>
 					<geometry>
 						<cylinder length="0.43" radius="0.065"/>
@@ -142,9 +125,9 @@
 		</link>
 		<joint name="joint2" type="revolute">
-			<origin rpy="1.5708 1.5708 0"/>
+			<origin rpy="${PI/2} ${PI/2} 0"/>
 			<parent link="Link1"/>
 			<child link="Link2"/>
 			<axis xyz="0 0 1"/>
-			<limit lower="-6.28318" upper="6.28318" effort="300" velocity="3.14159"/>
+			<limit lower="${-2*PI}" upper="${2*PI}" effort="300" velocity="${PI}"/>
 		</joint>
 		<link name="Link3">
@@ -152,11 +135,5 @@
 				<origin xyz="-0.15231 -1.4079E-07 0.022693"/>
 				<mass value="2.8536"/>
-				<inertia
-						ixx="0.0032608"
-						ixy="-3.2147E-10"
-						ixz="0.00012363"
-						iyy="0.0092967"
-						iyz="2.9478E-10"
-						izz="0.0095552"/>
+			<inertia ixx="0.0032608" ixy="-3.2147E-10" ixz="0.00012363" iyy="0.0092967" iyz="2.9478E-10" izz="0.0095552"/>
 			</inertial>
 			<visual>
@@ -190,5 +167,5 @@
 				</collision>
 				<collision>
-					<origin rpy="0 1.5708 0" xyz="-0.2 0 0.03"/>
+					<origin rpy="0 ${PI/2} 0" xyz="-0.2 0 0.03"/>
 					<geometry>
 						<cylinder length="0.26" radius="0.05"/>
@@ -214,11 +191,5 @@
 				<origin xyz="-3.2386E-07 -0.002077 -0.0015548"/>
 				<mass value="0.67058"/>
-				<inertia
-						ixx="0.00066939"
-						ixy="4.1975E-10"
-						ixz="-1.0734E-08"
-						iyy="0.00065424"
-						iyz="0.00011081"
-						izz="0.00065365"/>
+			<inertia ixx="0.00066939" ixy="4.1975E-10" ixz="-1.0734E-08" iyy="0.00065424" iyz="0.00011081" izz="0.00065365"/>
 			</inertial>
 			<visual>
@@ -241,5 +212,5 @@
 			<xacro:if value="${collider == 'simple'}">
 				<collision>
-					<origin rpy="1.5708 0 0"/>
+					<origin rpy="${PI/2} 0 0"/>
 					<geometry>
 						<cylinder length="0.155" radius="0.055"/>
@@ -249,9 +220,9 @@
 		</link>
 		<joint name="joint4" type="revolute">
-			<origin xyz="-0.357 0 0.141" rpy="0 0 -1.5708"/>
+			<origin xyz="-0.357 0 0.141" rpy="0 0 ${-PI/2}"/>
 			<parent link="Link3"/>
 			<child link="Link4"/>
 			<axis xyz="0 0 1"/>
-			<limit lower="-6.28318" upper="6.28318" effort="300" velocity="3.14159"/>
+			<limit lower="${-2*PI}" upper="${2*PI}" effort="300" velocity="${PI}"/>
 		</joint>
 		<link name="Link5">
@@ -259,11 +230,5 @@
 				<origin xyz="-3.7738E-07 -0.0045777 -0.0012971"/>
 				<mass value="0.7269"/>
-				<inertia
-						ixx="0.00073069"
-						ixy="-5.7806E-09"
-						ixz="6.7132E-09"
-						iyy="0.00071195"
-						iyz="-0.00011926"
-						izz="0.00071391"/>
+			<inertia ixx="0.00073069" ixy="-5.7806E-09" ixz="6.7132E-09" iyy="0.00071195" iyz="-0.00011926" izz="0.00071391"/>
 			</inertial>
 			<visual>
@@ -281,5 +246,5 @@
 			<xacro:if value="${collider == 'simple'}">
 				<collision>
-					<origin rpy="1.5708 0 0"/>
+					<origin rpy="${PI/2} 0 0"/>
 					<geometry>
 						<cylinder length="0.18" radius="0.055"/>
@@ -289,9 +254,9 @@
 		</link>
 		<joint name="joint5" type="revolute">
-			<origin xyz="0 -0.116 0" rpy="1.5708 0 0"/>
+			<origin xyz="0 -0.116 0" rpy="${PI/2} 0 0"/>
 			<parent link="Link4"/>
 			<child link="Link5"/>
 			<axis xyz="0 0 1"/>
-			<limit lower="-6.28318" upper="6.28318" effort="300" velocity="3.14159"/>
+			<limit lower="${-2*PI}" upper="${2*PI}" effort="300" velocity="${PI}"/>
 		</joint>
 		<link name="Link6">
@@ -299,11 +264,5 @@
 				<origin xyz="5.0777E-11 9.3774E-05 -0.019285"/>
 				<mass value="0.15789"/>
-				<inertia
-						ixx="7.8045E-05"
-						ixy="6.1582E-15"
-						ixz="6.2471E-14"
-						iyy="7.9168E-05"
-						iyz="-1.3822E-07"
-						izz="0.00012951"/>
+			<inertia ixx="7.8045E-05" ixy="6.1582E-15" ixz="6.2471E-14" iyy="7.9168E-05" iyz="-1.3822E-07" izz="0.00012951"/>
 			</inertial>
 			<visual>
@@ -329,9 +288,9 @@
 		</link>
 		<joint name="joint6" type="revolute">
-			<origin xyz="0 0.105 0" rpy="-1.5708 0 0"/>
+			<origin xyz="0 0.105 0" rpy="${-PI/2} 0 0"/>
 			<parent link="Link5"/>
 			<child link="Link6"/>
 			<axis xyz="0 0 1"/>
-			<limit lower="-6.28318" upper="6.28318" effort="300" velocity="3.14159"/>
+			<limit lower="${-2*PI}" upper="${2*PI}" effort="300" velocity="${PI}"/>
 		</joint>
 	</xacro:macro>
