Commit message: modified d405 direction

File: humanoid/Agibot/agibot_g1_description/xacro/120s_camera_stand.xacro (robot description, xacro)
@@ -15,5 +15,5 @@
 		</link>
 		<joint name="${prefix}camera_joint" type="fixed">
-			<origin xyz="0 -0.079320 0.108617" rpy="0 -1.117 1.5708"/>
+			<origin xyz="0 -0.079320 0.108617" rpy="-0.4538 0 0"/>
 			<parent link="${prefix}camera_stand"/>
 			<child link="${prefix}camera"/>
@@ -22,5 +22,5 @@
 			<visual>
 				<geometry>
-					<mesh filename="file://$(find sensor_models)/meshes/d405/d405.obj"/>
+					<mesh filename="file://$(find sensor_models)/meshes/realsense/d405.glb"/>
 				</geometry>
 			</visual>

File: humanoid/Agibot/agibot_g1_description/xacro/omnipicker_camera_stand.xacro (robot description, xacro)
@@ -16,5 +16,5 @@
 		</link>
 		<joint name="${prefix}camera_joint" type="fixed">
-			<origin xyz="0 -0.07754 0.028618" rpy="0 -1.117 1.5708"/>
+			<origin xyz="0 -0.07754 0.028618" rpy="-0.4538 0 0"/>
 			<parent link="${prefix}camera_stand"/>
 			<child link="${prefix}camera"/>
@@ -23,5 +23,5 @@
 			<visual>
 				<geometry>
-					<mesh filename="file://$(find sensor_models)/meshes/d405/d405.obj"/>
+					<mesh filename="file://$(find sensor_models)/meshes/realsense/d405.glb"/>
 				</geometry>
 			</visual>

File: humanoid/Zerith/zerith_h1_description/xacro/components/arm.xacro (robot description, xacro)
@@ -277,11 +277,10 @@
 			<visual>
 				<geometry>
-					<mesh filename="file://$(find sensor_models)/meshes/d405/d405.obj"/>
-				</geometry>
-				<origin xyz="0.009 0 0.00377" rpy="1.5708 -1.5708 0"/>
+					<mesh filename="file://$(find sensor_models)/meshes/realsense/d405.glb"/>
+				</geometry>
 			</visual>
 		</link>
 		<joint name="${prefix}jaw_camera_joint" type="fixed">
-			<origin xyz="0.11933 0.009 0.060373" rpy="-2.0071 0 -1.5708"/>
+			<origin xyz="0.12275 0.000 0.05878" rpy="-2.0071 0 -1.5708"/>
 			<parent link="${prefix}wrist_pitch_link"/>
 			<child link="${prefix}jaw_camera_link"/>

File: manipulator/Galaxea/galaxea_r1lite_description/xacro/camera.xacro (robot description, xacro)
@@ -28,10 +28,10 @@
 			<visual>
 				<geometry>
-					<mesh filename="file://$(find sensor_models)/meshes/d405/d405.obj"/>
+					<mesh filename="file://$(find sensor_models)/meshes/realsense/d405.glb"/>
 				</geometry>
 			</visual>
 		</link>
 		<joint name="${prefix}camera_joint" type="fixed">
-			<origin rpy="0 ${-PI/2} ${PI/2}" xyz="0.008996 0 0"/>
+			<origin xyz="0.008996 0 0"/>
 			<parent link="${prefix}camera_stand"/>
 			<child link="${prefix}camera"/>

File: manipulator/Ragtime-Lab/panthera_description/xacro/d405.xacro (robot description, xacro)
@@ -6,5 +6,5 @@
       <visual>
         <geometry>
-          <mesh filename="file://$(find arx5_description)/meshes/camera_support.obj"/>
+          <mesh filename="file://$(find arx5_description)/meshes/camera_stand/stand_d405.glb"/>
         </geometry>
       </visual>
@@ -18,10 +18,10 @@
       <visual>
         <geometry>
-          <mesh filename="file://$(find arx5_description)/meshes/d405.obj"/>
+          <mesh filename="file://$(find sensor_models)/meshes/realsense/d405.glb"/>
         </geometry>
       </visual>
     </link>
     <joint name="${prefix}camera_fixed" type="fixed">
-      <origin xyz="0.0385 0 0.0475" rpy="0 0.523 0"/>
+      <origin xyz="0.0385 0 0.0475" rpy="-2.093 0 -1.5708"/>
       <parent link="${prefix}camera_support"/>
       <child link="${prefix}camera"/>

File: manipulator/Realman/rm75_description/xacro/components/fb75_camera.xacro (robot description, xacro)
@@ -5,4 +5,10 @@
 		<xacro:property name="mount_link" value="${prefix + 'fb75_ee' if with_fb75_ee_bool else parent_link}"/>
 		<xacro:if value="${with_fb75_ee_bool}">
+			<inertial>
+				<origin xyz="0.0 0.0 -0.0171573759779855"/>
+				<mass value="0.165822774021484"/>
+				<inertia ixx="4.88486899397696E-05" ixy="-9.4591722796062E-08" ixz="3.0611887075293E-07"
+								 iyy="4.94603620572993E-05" iyz="8.02154219939052E-09" izz="7.6901626133018E-05"/>
+			</inertial>
 			<link name="${prefix}fb75_ee">
 				<visual>
@@ -42,5 +48,5 @@
 		</link>
 		<joint name="${prefix}camera_joint" type="fixed">
-			<origin xyz="-0.10022 0.008 0.029031" rpy="0 -1.5708 -1.5708"/>
+			<origin xyz="-0.10022 0.008 0.029031" rpy="0 0 3.1415926535"/>
 			<parent link="${prefix}camera_stand"/>
 			<child link="${prefix}camera"/>
