Commit message: modified agibot g1 models

File: humanoid/Agibot/agibot_g1_description/xacro/robot.xacro (robot description, xacro)
@@ -36,10 +36,15 @@
 	<!-- Gripper joints -->
 	<joint name="ee_left_joint" type="fixed">
+		<origin xyz="0 0 0.027727"/>
 		<parent link="left_end_link"/>
 		<child link="left_gripper_base"/>
 	</joint>
 	<joint name="ee_right_joint" type="fixed">
+		<origin xyz="0 0 0.027727"/>
 		<parent link="right_end_link"/>
 		<child link="right_gripper_base"/>
 	</joint>
+	<xacro:include filename="$(find agibot_g1_description)/xacro/120s_camera_stand.xacro"/>
+	<xacro:Camera name="left"/>
+	<xacro:Camera name="right"/>
 </robot>

Commit message: fixed agibot g1 ocs2

File: humanoid/Agibot/agibot_g1_description/xacro/robot.xacro (robot description, xacro)
@@ -36,10 +36,10 @@
 	<!-- Gripper joints -->
 	<joint name="ee_left_joint" type="fixed">
-		<origin xyz="0 0 0.027727"/>
+		<origin xyz="0 0 0.027727" rpy="0 0 3.1415"/>
 		<parent link="left_end_link"/>
 		<child link="left_gripper_base"/>
 	</joint>
 	<joint name="ee_right_joint" type="fixed">
-		<origin xyz="0 0 0.027727"/>
+		<origin xyz="0 0 0.027727" rpy="0 0 3.1415"/>
 		<parent link="right_end_link"/>
 		<child link="right_gripper_base"/>

Commit message: adapt more robots

File: humanoid/Agibot/agibot_g1_description/xacro/robot.xacro (robot description, xacro)
@@ -6,4 +6,7 @@
 <robot name="Agibot G1" xmlns:xacro="http://www.ros.org/wiki/xacro">
 	<xacro:arg name="type" default="AG2F120S"/>
+	<!-- false: ros2_control / 可视化默认可驱动夹爪；OCS2 planning 由 robot_common_launch 注入 eef_fixed_joints:=true -->
+	<xacro:arg name="eef_fixed_joints" default="false"/>
+	<xacro:property name="eef_fixed" value="$(arg eef_fixed_joints)"/>
 	<!-- Include the base robot structure -->
 	<xacro:include filename="$(find agibot_g1_description)/xacro/g1_base.xacro"/>
@@ -34,6 +37,6 @@
 		<!-- Include gripper -->
 		<xacro:include filename="$(find changingtek_description)/xacro/AG2F120S.xacro"/>
-		<xacro:AG2F120S name="left"/>
-		<xacro:AG2F120S name="right"/>
+		<xacro:AG2F120S name="left" kinematic_only="${eef_fixed}"/>
+		<xacro:AG2F120S name="right" kinematic_only="${eef_fixed}"/>
 		<!-- Gripper joints -->
 		<joint name="ee_left_joint" type="fixed">
@@ -53,6 +56,6 @@
 	<xacro:if value="${'$(arg type)' == 'omni-picker'}">
 		<xacro:include filename="$(find agibot_omni_description)/xacro/omni_picker.xacro"/>
-		<xacro:omni-picker name="left"/>
-		<xacro:omni-picker name="right"/>
+		<xacro:omni-picker name="left" kinematic_only="${eef_fixed}"/>
+		<xacro:omni-picker name="right" kinematic_only="${eef_fixed}"/>
 		<!-- Gripper joints -->
 		<joint name="ee_left_joint" type="fixed">

File: humanoid/Agibot/agibot_g1_description/xacro/ros2_control/robot.xacro (robot description, xacro)
@@ -5,5 +5,6 @@
 <!-- =================================================================================== -->
 <robot name="genie" xmlns:xacro="http://www.ros.org/wiki/xacro">
-	<!-- Include the base robot structure -->
+	<!-- 夹爪由 adaptive_gripper_controller 控制，与 OCS2 分离；勿对 ros2_control 使用 eef_fixed_joints -->
+	<xacro:arg name="eef_fixed_joints" default="false"/>
 	<xacro:include filename="$(find agibot_g1_description)/xacro/robot.xacro"/>
 	<!-- Import modular interface components -->
@@ -34,5 +35,5 @@
 		<!-- 右臂接口 -->
 		<xacro:g1_arm_interfaces name="right"/>
-		<!-- 夹爪接口 - 参考CR5的模块化设计 -->
+		<!-- 夹爪接口 → adaptive_gripper_controller（不归 ocs2_wbc_controller） -->
 		<xacro:if value="${'$(arg type)' == 'AG2F120S'}">
 			<xacro:include filename="$(find changingtek_description)/xacro/ros2_control/AG2F120S.xacro"/>

File: humanoid/Agibot/agibot_omni_description/xacro/omni_picker.xacro (robot description, xacro)
@@ -1,8 +1,9 @@
 <?xml version="1.0"?>
 <robot xmlns:xacro="http://ros.org/wiki/xacro">
-	<xacro:macro name="omni-picker" params="name">
+	<xacro:macro name="omni-picker" params="name kinematic_only:=false">
 		<xacro:property name="mesh_path" value="file://$(find agibot_omni_description)/meshes/omni_picker"/>
 		<xacro:property name="prefix" value="${name + '_' if name else ''}"/>
 		<xacro:property name="PI" value="3.1415926535897931"/>
+		<xacro:property name="joint_type" value="${kinematic_only and 'fixed' or 'revolute'}"/>
 		<link name="${prefix}gripper_base">
 			<inertial>
@@ -40,10 +41,12 @@
 			</collision>
 		</link>
-		<joint name="${prefix}gripper_joint" type="revolute">
+		<joint name="${prefix}gripper_joint" type="${joint_type}">
 			<origin xyz="0 -0.0195 0.0565" rpy="-2.9951 -${PI/2} -0.15964"/>
 			<parent link="${prefix}gripper_base"/>
 			<child link="${prefix}narrow1_Link"/>
-			<axis xyz="0 0 1"/>
-			<limit lower="0" upper="1" effort="50" velocity="${PI}"/>
+			<xacro:unless value="${kinematic_only}">
+				<axis xyz="0 0 1"/>
+				<limit lower="0" upper="1" effort="50" velocity="${PI}"/>
+			</xacro:unless>
 		</joint>
 		<link name="${prefix}narrow2_Link">
@@ -70,11 +73,13 @@
 			</collision>
 		</link>
-		<joint name="${prefix}narrow2_joint" type="revolute">
+		<joint name="${prefix}narrow2_joint" type="${joint_type}">
 			<origin xyz="0.030852 0.018551 0"/>
 			<parent link="${prefix}narrow1_Link"/>
 			<child link="${prefix}narrow2_Link"/>
-			<axis xyz="0 0 -1"/>
-			<limit lower="-${PI}" upper="${PI}" effort="50" velocity="${PI}"/>
-			<mimic joint="${prefix}gripper_joint" multiplier="0.02" offset="0"/>
+			<xacro:unless value="${kinematic_only}">
+				<axis xyz="0 0 -1"/>
+				<limit lower="-${PI}" upper="${PI}" effort="50" velocity="${PI}"/>
+				<mimic joint="${prefix}gripper_joint" multiplier="0.02" offset="0"/>
+			</xacro:unless>
 		</joint>
 		<link name="${prefix}narrow3_Link">
@@ -101,11 +106,13 @@
 			</collision>
 		</link>
-		<joint name="${prefix}narrow3_joint" type="revolute">
+		<joint name="${prefix}narrow3_joint" type="${joint_type}">
 			<origin xyz="0.018118 -0.01574 0"/>
 			<parent link="${prefix}narrow2_Link"/>
 			<child link="${prefix}narrow3_Link"/>
-			<axis xyz="0 0 -1"/>
-			<limit lower="-${PI}" upper="${PI}" effort="50" velocity="${PI}"/>
-			<mimic joint="${prefix}gripper_joint" multiplier="0.4" offset="0"/>
+			<xacro:unless value="${kinematic_only}">
+				<axis xyz="0 0 -1"/>
+				<limit lower="-${PI}" upper="${PI}" effort="50" velocity="${PI}"/>
+				<mimic joint="${prefix}gripper_joint" multiplier="0.4" offset="0"/>
+			</xacro:unless>
 		</joint>
 		<link name="${prefix}narrow4_Link"/>
@@ -140,11 +147,13 @@
 			</collision>
 		</link>
-		<joint name="${prefix}narrow_loop_joint" type="revolute">
+		<joint name="${prefix}narrow_loop_joint" type="${joint_type}">
 			<origin xyz="0 -0.021633 0.07387" rpy="-2.9951 -${PI/2} -0.15964"/>
 			<parent link="${prefix}gripper_base"/>
 			<child link="${prefix}narrow_loop_Link"/>
-			<axis xyz="0 0 1"/>
-			<limit lower="-${PI}" upper="${PI}" effort="50" velocity="${PI}"/>
-			<mimic joint="${prefix}gripper_joint" multiplier="1.5" offset="0"/>
+			<xacro:unless value="${kinematic_only}">
+				<axis xyz="0 0 1"/>
+				<limit lower="-${PI}" upper="${PI}" effort="50" velocity="${PI}"/>
+				<mimic joint="${prefix}gripper_joint" multiplier="1.5" offset="0"/>
+			</xacro:unless>
 		</joint>
 		<link name="${prefix}wide1_Link">
@@ -171,11 +180,13 @@
 			</collision>
 		</link>
-		<joint name="${prefix}wide1_joint" type="revolute">
+		<joint name="${prefix}wide1_joint" type="${joint_type}">
 			<origin xyz="0 0.0195 0.0565" rpy="-2.9951 -${PI/2} -0.15964"/>
 			<parent link="${prefix}gripper_base"/>
 			<child link="${prefix}wide1_Link"/>
-			<axis xyz="0 0 -1"/>
-			<limit lower="-${PI}" upper="${PI}" effort="50" velocity="${PI}"/>
-			<mimic joint="${prefix}gripper_joint" multiplier="1" offset="0"/>
+			<xacro:unless value="${kinematic_only}">
+				<axis xyz="0 0 -1"/>
+				<limit lower="-${PI}" upper="${PI}" effort="50" velocity="${PI}"/>
+				<mimic joint="${prefix}gripper_joint" multiplier="1" offset="0"/>
+			</xacro:unless>
 		</joint>
 		<link name="${prefix}wide2_Link">
@@ -202,11 +213,13 @@
 			</collision>
 		</link>
-		<joint name="${prefix}wide2_joint" type="revolute">
+		<joint name="${prefix}wide2_joint" type="${joint_type}">
 			<origin xyz="0.030852 -0.018551 0"/>
 			<parent link="${prefix}wide1_Link"/>
 			<child link="${prefix}wide2_Link"/>
-			<axis xyz="0 0 1"/>
-			<limit lower="-${PI}" upper="${PI}" effort="50" velocity="${PI}"/>
-			<mimic joint="${prefix}gripper_joint" multiplier="0.02" offset="0"/>
+			<xacro:unless value="${kinematic_only}">
+				<axis xyz="0 0 1"/>
+				<limit lower="-${PI}" upper="${PI}" effort="50" velocity="${PI}"/>
+				<mimic joint="${prefix}gripper_joint" multiplier="0.02" offset="0"/>
+			</xacro:unless>
 		</joint>
 		<link name="${prefix}wide3_Link">
@@ -233,11 +246,13 @@
 			</collision>
 		</link>
-		<joint name="${prefix}wide3_joint" type="revolute">
+		<joint name="${prefix}wide3_joint" type="${joint_type}">
 			<origin xyz="0.018118 0.01574 0"/>
 			<parent link="${prefix}wide2_Link"/>
 			<child link="${prefix}wide3_Link"/>
-			<axis xyz="0 0 1"/>
-			<limit lower="-${PI}" upper="${PI}" effort="50" velocity="${PI}"/>
-			<mimic joint="${prefix}gripper_joint" multiplier="0.4" offset="0"/>
+			<xacro:unless value="${kinematic_only}">
+				<axis xyz="0 0 1"/>
+				<limit lower="-${PI}" upper="${PI}" effort="50" velocity="${PI}"/>
+				<mimic joint="${prefix}gripper_joint" multiplier="0.4" offset="0"/>
+			</xacro:unless>
 		</joint>
 		<link name="${prefix}wide4_Link"/>
@@ -270,11 +285,26 @@
 			</collision>
 		</link>
-		<joint name="${prefix}wide_loop_joint" type="revolute">
+		<joint name="${prefix}wide_loop_joint" type="${joint_type}">
 			<origin xyz="0 0.021633 0.07387" rpy="-2.9951 -${PI/2} -0.15964"/>
 			<parent link="${prefix}gripper_base"/>
 			<child link="${prefix}wide_loop_Link"/>
-			<axis xyz="0 0 -1"/>
-			<limit lower="-${PI}" upper="${PI}" effort="50" velocity="${PI}"/>
-			<mimic joint="${prefix}gripper_joint" multiplier="1.5" offset="0"/>
+			<xacro:unless value="${kinematic_only}">
+				<axis xyz="0 0 -1"/>
+				<limit lower="-${PI}" upper="${PI}" effort="50" velocity="${PI}"/>
+				<mimic joint="${prefix}gripper_joint" multiplier="1.5" offset="0"/>
+			</xacro:unless>
+		</joint>
+		<!-- OCS2 eeFrame (fixed_base.info); TCP offset aligned with MOZ1 omni mount -->
+		<link name="${prefix}gripper_center"/>
+		<joint name="${prefix}gripper_center_joint" type="fixed">
+			<origin xyz="0 0 0.14" rpy="0 0 0"/>
+			<parent link="${prefix}gripper_base"/>
+			<child link="${prefix}gripper_center"/>
+		</joint>
+		<link name="${prefix}eef"/>
+		<joint name="${prefix}eef_joint" type="fixed">
+			<origin xyz="0 0 0" rpy="0 0 0"/>
+			<parent link="${prefix}gripper_center"/>
+			<child link="${prefix}eef"/>
 		</joint>
 	</xacro:macro>

File: humanoid/SpiritAI/moz1_description/xacro/components/arm.xacro (robot description, xacro)
@@ -4,5 +4,5 @@
 	<xacro:include filename="$(find moz1_description)/xacro/components/omni_gripper.xacro"/>
 	<!-- direction:=1 left arm, direction:=-1 right arm (mirror mount & asymmetric limits). -->
-	<xacro:macro name="Moz1Arm" params="parent_link:=waist03 direction:=1">
+	<xacro:macro name="Moz1Arm" params="parent_link:=waist03 direction:=1 kinematic_only:=false">
 		<xacro:if value="${direction == 1}">
 			<xacro:property name="prefix" value="left"/>
@@ -277,5 +277,5 @@
 			</xacro:unless>
 		</joint>
-		<xacro:Moz1OmniGripper direction="${direction}"/>
+		<xacro:Moz1OmniGripper direction="${direction}" kinematic_only="${kinematic_only}"/>
 	</xacro:macro>
 </robot>

File: humanoid/SpiritAI/moz1_description/xacro/components/omni_gripper.xacro (robot description, xacro)
@@ -2,6 +2,6 @@
 <robot xmlns:xacro="http://www.ros.org/wiki/xacro">
   <xacro:include filename="$(find agibot_omni_description)/xacro/omni_picker.xacro"/>
-  <!-- Agibot omni-picker on MOZ1 flange; tool frame (eef) on gripper_base. -->
-  <xacro:macro name="Moz1OmniGripper" params="direction:=1 side:=''">
+  <!-- Omni-picker + OCS2 eeFrame (left/right_eef) from agibot_omni_description; TCP z=0.14 on gripper_base. -->
+  <xacro:macro name="Moz1OmniGripper" params="direction:=1 side:='' kinematic_only:=false">
     <xacro:if value="${side != ''}">
       <xacro:property name="gripper_side" value="${side}"/>
@@ -23,5 +23,5 @@
       <xacro:property name="gripper_rpy_z" value="0"/>
     </xacro:unless>
-    <xacro:omni-picker name="${gripper_side}"/>
+    <xacro:omni-picker name="${gripper_side}" kinematic_only="${kinematic_only}"/>
     <joint name="${ee_mount_joint}" type="fixed">
       <origin xyz="-0.01 0.001 -0.05" rpy="0 -3.14 ${gripper_rpy_z}"/>
@@ -29,10 +29,4 @@
       <child link="${gripper_side}_gripper_base"/>
     </joint>
-    <link name="${gripper_side}_eef"/>
-    <joint name="${gripper_side}_eef_joint" type="fixed">
-      <origin xyz="0.0 0 0.14"/>
-      <parent link="${gripper_side}_gripper_base"/>
-      <child link="${gripper_side}_eef"/>
-    </joint>
   </xacro:macro>
 </robot>

File: humanoid/SpiritAI/moz1_description/xacro/robot.xacro (robot description, xacro)
@@ -4,4 +4,7 @@
   <xacro:arg name="enable_wheel_joints" default="false"/>
   <xacro:arg name="type" default="omni_gripper"/>
+  <!-- false: ros2_control; OCS2 planning injects eef_fixed_joints:=true via robot_common_launch -->
+  <xacro:arg name="eef_fixed_joints" default="false"/>
+  <xacro:property name="eef_fixed" value="$(arg eef_fixed_joints)"/>
   <material name="black_color">
     <color rgba="0.1 0.1 0.1 1.0"/>
@@ -19,6 +22,6 @@
   <xacro:Moz1Chassis enable_wheel_joints="$(arg enable_wheel_joints)"/>
   <xacro:Moz1Body parent_link="base_link"/>
-  <xacro:Moz1Arm parent_link="waist03" direction="1"/>
-  <xacro:Moz1Arm parent_link="waist03" direction="-1"/>
+  <xacro:Moz1Arm parent_link="waist03" direction="1" kinematic_only="${eef_fixed}"/>
+  <xacro:Moz1Arm parent_link="waist03" direction="-1" kinematic_only="${eef_fixed}"/>
   <xacro:Moz1Head parent_link="waist03"/>
 </robot>

File: humanoid/SpiritAI/moz1_description/xacro/ros2_control/robot.xacro (robot description, xacro)
@@ -3,4 +3,5 @@
   <xacro:arg name="ros2_control_hardware_type" default="mock_components"/>
   <xacro:arg name="enable_wheel_joints" default="false"/>
+  <xacro:arg name="eef_fixed_joints" default="false"/>
   <xacro:arg name="gazebo" default="false"/>
   <xacro:include filename="$(find moz1_description)/xacro/robot.xacro"/>

File: manipulator/Realman/rm75_description/xacro/ros2_control/arm.xacro (robot description, xacro)
@@ -1,5 +1,5 @@
 <?xml version="1.0"?>
 <robot xmlns:xacro="http://www.ros.org/wiki/xacro">
-  <!-- RM65机械臂接口定义宏 -->
+  <!-- RM75 7-DOF: enable_joint3:=true adds joint7; RM65 6-DOF (type:=65) leaves it false -->
   <xacro:macro name="rm65_interfaces" params="name enable_joint3:=false">
     <xacro:property name="prefix" value="${name + '_' if name else ''}"/>

File: manipulator/Realman/rm75_description/xacro/ros2_control/robot.xacro (robot description, xacro)
@@ -34,6 +34,6 @@
 			</xacro:if>
 		</hardware>
-		<!-- 机械臂接口 -->
-		<xacro:rm65_interfaces name=""/>
+		<!-- 7-DOF (joint7) when enable_joint3:=true; 6-DOF (type:=65) omits joint7 -->
+		<xacro:rm65_interfaces name="" enable_joint3="${enable_joint3}"/>
 		<!-- 夹爪接口定义 -->
 		<xacro:if value="${selected_gripper_type == 'eg2-4c2'}">
