Commit message: gripper direction based on inital value

File: common/gripper/changingtek_description/xacro/ros2_control/AG2F120S.xacro (robot description, xacro)
@@ -13,7 +13,4 @@
 			<state_interface name="velocity"/>
 			<state_interface name="effort"/>
-			<state_interface name="reverse_flag">
-				<param name="initial_value">1.0</param>
-			</state_interface>
 		</joint>
 		<xacro:if value="$(arg gazebo)">

File: common/gripper/changingtek_description/xacro/ros2_control/AG2F90-C.xacro (robot description, xacro)
@@ -9,11 +9,8 @@
       <command_interface name="position"/>
       <state_interface name="position">
-        <param name="initial_value">1.0</param>
+        <param name="initial_value">0.0</param>
       </state_interface>
       <state_interface name="velocity"/>
       <state_interface name="effort"/>
-      <state_interface name="reverse_flag">
-        <param name="initial_value">1.0</param>
-      </state_interface>
     </joint>
     <xacro:if value="$(arg gazebo)">

File: common/gripper/robotiq_description/xacro/ros2_control/2F85.xacro (robot description, xacro)
@@ -8,11 +8,8 @@
       <command_interface name="position"/>
       <state_interface name="position">
-        <param name="initial_value">0.0</param>
+        <param name="initial_value">0.810000</param>
       </state_interface>
       <state_interface name="velocity"/>
       <state_interface name="effort"/>
-      <state_interface name="reverse_flag">
-        <param name="initial_value">-1.0</param>
-      </state_interface>
     </joint>
     <!-- Robotiq 2F85夹爪的mimic关节接口 -->

File: humanoid/Astribot/astribot_s1_description/xacro/ros2_control/astribot_s1_gripper_interfaces.xacro (robot description, xacro)
@@ -1,48 +1,45 @@
 <?xml version="1.0"?>
 <robot xmlns:xacro="http://www.ros.org/wiki/xacro">
-    <!-- Astribot S1夹爪完整接口定义宏 - 参考AG2F120S的设计模式 -->
-    <xacro:macro name="astribot_s1_gripper_interfaces" params="name">
-        <xacro:arg name="gazebo" default="false"/>
-        <xacro:property name="prefix" value="${name + '_' if name else ''}"/>
-        <!-- 夹爪主关节接口定义 -->
-        <joint name="${prefix}gripper_joint">
-            <command_interface name="position"/>
-            <state_interface name="position">
-                <param name="initial_value">0.0</param>
-            </state_interface>
-            <state_interface name="velocity"/>
-            <state_interface name="effort"/>
-            <state_interface name="reverse_flag">
-                <param name="initial_value">-1.0</param>
-            </state_interface>
-        </joint>
-        <xacro:if value="$(arg gazebo)">
-            <!-- Astribot S1夹爪的mimic关节接口 -->
-            <joint name="${prefix}gripper_joint_L2">
-                <state_interface name="position"/>
-                <state_interface name="velocity"/>
-                <state_interface name="effort"/>
-            </joint>
-            <joint name="${prefix}gripper_joint_L11">
-                <state_interface name="position"/>
-                <state_interface name="velocity"/>
-                <state_interface name="effort"/>
-            </joint>
-            <joint name="${prefix}gripper_joint_R1">
-                <state_interface name="position"/>
-                <state_interface name="velocity"/>
-                <state_interface name="effort"/>
-            </joint>
-            <joint name="${prefix}gripper_joint_R2">
-                <state_interface name="position"/>
-                <state_interface name="velocity"/>
-                <state_interface name="effort"/>
-            </joint>
-            <joint name="${prefix}gripper_joint_R11">
-                <state_interface name="position"/>
-                <state_interface name="velocity"/>
-                <state_interface name="effort"/>
-            </joint>
-        </xacro:if>
-    </xacro:macro>
+	<!-- Astribot S1夹爪完整接口定义宏 - 参考AG2F120S的设计模式 -->
+	<xacro:macro name="astribot_s1_gripper_interfaces" params="name">
+		<xacro:arg name="gazebo" default="false"/>
+		<xacro:property name="prefix" value="${name + '_' if name else ''}"/>
+		<!-- 夹爪主关节接口定义 -->
+		<joint name="${prefix}gripper_joint">
+			<command_interface name="position"/>
+			<state_interface name="position">
+				<param name="initial_value">1.0</param>
+			</state_interface>
+			<state_interface name="velocity"/>
+			<state_interface name="effort"/>
+		</joint>
+		<xacro:if value="$(arg gazebo)">
+			<!-- Astribot S1夹爪的mimic关节接口 -->
+			<joint name="${prefix}gripper_joint_L2">
+				<state_interface name="position"/>
+				<state_interface name="velocity"/>
+				<state_interface name="effort"/>
+			</joint>
+			<joint name="${prefix}gripper_joint_L11">
+				<state_interface name="position"/>
+				<state_interface name="velocity"/>
+				<state_interface name="effort"/>
+			</joint>
+			<joint name="${prefix}gripper_joint_R1">
+				<state_interface name="position"/>
+				<state_interface name="velocity"/>
+				<state_interface name="effort"/>
+			</joint>
+			<joint name="${prefix}gripper_joint_R2">
+				<state_interface name="position"/>
+				<state_interface name="velocity"/>
+				<state_interface name="effort"/>
+			</joint>
+			<joint name="${prefix}gripper_joint_R11">
+				<state_interface name="position"/>
+				<state_interface name="velocity"/>
+				<state_interface name="effort"/>
+			</joint>
+		</xacro:if>
+	</xacro:macro>
 </robot>

File: humanoid/Galaxea/galaxea_r1pro_description/xacro/ros2_control/pro_arm.ros2_control.xacro (robot description, xacro)
@@ -66,7 +66,4 @@
         <state_interface name="velocity"/>
         <state_interface name="effort"/>
-        <state_interface name="reverse_flag">
-          <param name="initial_value">1.0</param>
-        </state_interface>
       </joint>
     </ros2_control>

File: manipulator/ARX/arx5_description/xacro/ros2_control/interfaces.xacro (robot description, xacro)
@@ -51,7 +51,4 @@
 			<state_interface name="velocity"/>
 			<state_interface name="effort"/>
-			<state_interface name="reverse_flag">
-				<param name="initial_value">1.0</param>
-			</state_interface>
 		</joint>
 		<joint name="${prefix}joint8">

File: manipulator/Galaxea/galaxea_a1_description/xacro/a1_x.xacro (robot description, xacro)
@@ -1,3 +1,3 @@
- <?xml version="1.0" encoding="utf-8"?>
+<?xml version="1.0" encoding="utf-8"?>
 <robot xmlns:xacro="http://www.ros.org/wiki/xacro">
   <xacro:macro name="Arm" params="name">

File: manipulator/Galaxea/galaxea_a1_description/xacro/ros2_control/interfaces.xacro (robot description, xacro)
@@ -1,5 +1,5 @@
 <?xml version="1.0"?>
 <robot xmlns:xacro="http://www.ros.org/wiki/xacro">
-  <xacro:macro name="airbot_play_interfaces" params="name">
+  <xacro:macro name="galaxea_a1_interfaces" params="name">
     <xacro:property name="prefix" value="${name + '_' if name else ''}"/>
     <!-- 关节接口定义 -->
@@ -48,5 +48,5 @@
       <state_interface name="effort"/>
     </joint>
-    <joint name="${prefix}gripper_joint1">
+    <joint name="${prefix}gripper_joint2">
       <state_interface name="position"/>
       <state_interface name="velocity"/>
