Commit message: hand mesh clean up

File: humanoid/Agibot/agibot_a2_description/xacro/component.xacro (robot description, xacro)
@@ -19,3 +19,37 @@
 		<xacro:include filename="$(find agibot_g1_description)/xacro/g1_base.xacro"/>
 	</xacro:if>
+	<xacro:if value="${'$(arg type)' == 'left_hand'}">
+		<link name="base_link"/>
+		<!-- Virtual parent link for hand connection -->
+		<link name="left_arm_link07"/>
+		<joint name="left_arm_link07_fixed" type="fixed">
+			<origin xyz="0 0 0" rpy="0 0 0"/>
+			<parent link="base_link"/>
+			<child link="left_arm_link07"/>
+		</joint>
+		<xacro:include filename="$(find agibot_a2_description)/xacro/hand.xacro"/>
+		<xacro:A2Hand name="left" direction="1" parent_link="left_arm_link07"/>
+	</xacro:if>
+	<xacro:if value="${'$(arg type)' == 'right_hand'}">
+		<link name="base_link"/>
+		<!-- Virtual parent link for hand connection -->
+		<link name="right_arm_link07"/>
+		<joint name="right_arm_link07_fixed" type="fixed">
+			<origin xyz="0 0 0" rpy="0 0 0"/>
+			<parent link="base_link"/>
+			<child link="right_arm_link07"/>
+		</joint>
+		<xacro:include filename="$(find agibot_a2_description)/xacro/hand.xacro"/>
+		<xacro:A2Hand name="right" direction="-1" parent_link="right_arm_link07"/>
+	</xacro:if>
+	<xacro:if value="${'$(arg type)' == 'left_leg'}">
+		<link name="base_link"/>
+		<xacro:include filename="$(find agibot_a2_description)/xacro/leg.xacro"/>
+		<xacro:A2Leg name="left" direction="1" joint_idx_offset="1" parent_link="base_link" hip_roll_origin_y="0.105"/>
+	</xacro:if>
+	<xacro:if value="${'$(arg type)' == 'right_leg'}">
+		<link name="base_link"/>
+		<xacro:include filename="$(find agibot_a2_description)/xacro/leg.xacro"/>
+		<xacro:A2Leg name="right" direction="-1" joint_idx_offset="7" parent_link="base_link" hip_roll_origin_y="-0.105"/>
+	</xacro:if>
 </robot>

File: humanoid/Agibot/agibot_a2_description/xacro/hand.xacro (robot description, xacro)
@@ -27,11 +27,11 @@
 			<visual>
 				<geometry>
-					<mesh filename="file://$(find agibot_a2_description)/meshes/hand/visual/paw.obj" scale="1 ${-direction} 1"/>
-				</geometry>
-			</visual>
-			<collision>
-				<geometry>
-					<mesh filename="file://$(find agibot_a2_description)/meshes/hand/collision/R_paw_hull.stl"
-								scale="1 ${-direction} 1"/>
+					<mesh filename="file://$(find agibot_a2_description)/meshes/hand/visual/paw.obj" scale="1 ${direction} 1"/>
+				</geometry>
+			</visual>
+			<collision>
+				<geometry>
+					<mesh filename="file://$(find agibot_a2_description)/meshes/hand/collision/paw.stl"
+								scale="1 ${direction} 1"/>
 				</geometry>
 			</collision>
@@ -47,10 +47,7 @@
 			<visual>
 				<geometry>
-					<mesh filename="file://$(find agibot_a2_description)/meshes/hand/visual/R_thumb_swing.stl"
-								scale="1 ${-direction} 1"/>
-				</geometry>
-				<material name="metallic black">
-					<color rgba="0.235294118 0.235294118 0.235294118 1"/>
-				</material>
+					<mesh filename="file://$(find agibot_a2_description)/meshes/hand/visual/thumb_swing.obj"
+								scale="1 ${direction} 1"/>
+				</geometry>
 			</visual>
 			<collision>
@@ -78,10 +75,7 @@
 			<visual>
 				<geometry>
-					<mesh filename="file://$(find agibot_a2_description)/meshes/hand/visual/R_thumb_1.stl"
-								scale="1 1 ${-direction}"/>
-				</geometry>
-				<material name="metallic black">
-					<color rgba="0.235294118 0.235294118 0.235294118 1"/>
-				</material>
+					<mesh filename="file://$(find agibot_a2_description)/meshes/hand/visual/thumb_1.obj"
+								scale="1 1 ${direction}"/>
+				</geometry>
 			</visual>
 			<collision>
@@ -92,5 +86,5 @@
 			</collision>
 		</link>
-		<joint name="${prefix_upper}thumb_1_joint" type="revolute">
+		<joint name="${prefix_upper}thumb_joint" type="revolute">
 			<origin xyz="-0.013367 0.00088357 ${-dir*0.0052468}" rpy="1.5708 0 3.0756"/>
 			<parent link="${prefix_upper}thumb_swing"/>
@@ -109,10 +103,7 @@
 			<visual>
 				<geometry>
-					<mesh filename="file://$(find agibot_a2_description)/meshes/hand/visual/R_thumb_2.stl"
-								scale="1 1 ${-direction}"/>
-				</geometry>
-				<material name="metallic black">
-					<color rgba="0.235294118 0.235294118 0.235294118 1"/>
-				</material>
+					<mesh filename="file://$(find agibot_a2_description)/meshes/hand/visual/thumb_2.obj"
+								scale="1 1 ${direction}"/>
+				</geometry>
 			</visual>
 			<collision>
@@ -129,5 +120,5 @@
 			<axis xyz="0 0 1"/>
 			<limit lower="0" upper="0.9144" effort="1" velocity="100"/>
-			<mimic joint="${prefix_upper}thumb_1_joint" multiplier="0.40" offset="0"/>
+			<mimic joint="${prefix_upper}thumb_joint" multiplier="0.40" offset="0"/>
 		</joint>
 		<!-- Thumb 3 -->
@@ -141,10 +132,7 @@
 			<visual>
 				<geometry>
-					<mesh filename="file://$(find agibot_a2_description)/meshes/hand/visual/R_thumb_3.stl"
-								scale="1 1 ${-direction}"/>
-				</geometry>
-				<material name="metallic black">
-					<color rgba="0.235294118 0.235294118 0.235294118 1"/>
-				</material>
+					<mesh filename="file://$(find agibot_a2_description)/meshes/hand/visual/thumb_3.obj"
+								scale="1 1 ${direction}"/>
+				</geometry>
 			</visual>
 			<collision>
@@ -161,5 +149,5 @@
 			<axis xyz="0 0 1"/>
 			<limit lower="0" upper="1.3716" effort="1" velocity="100"/>
-			<mimic joint="${prefix_upper}thumb_1_joint" multiplier="0.60" offset="0"/>
+			<mimic joint="${prefix_upper}thumb_joint" multiplier="0.60" offset="0"/>
 		</joint>
 		<!-- Index 1 -->
@@ -173,9 +161,6 @@
 			<visual>
 				<geometry>
-					<mesh filename="file://$(find agibot_a2_description)/meshes/hand/visual/R_index_1.stl" scale="${-direction} 1 1"/>
-				</geometry>
-				<material name="metallic black">
-					<color rgba="0.235294118 0.235294118 0.235294118 1"/>
-				</material>
+					<mesh filename="file://$(find agibot_a2_description)/meshes/hand/visual/index_1.obj" scale="${direction} 1 1"/>
+				</geometry>
 			</visual>
 			<collision>
@@ -185,5 +170,5 @@
 			</collision>
 		</link>
-		<joint name="${prefix_upper}index_1_joint" type="fixed">
+		<joint name="${prefix_upper}index_joint" type="revolute">
 			<origin xyz="-0.034645 ${dir*0.0059953} 0.11967" rpy="1.6319 0 -1.5708"/>
 			<parent link="${name}_hand"/>
@@ -202,9 +187,6 @@
 			<visual>
 				<geometry>
-					<mesh filename="file://$(find agibot_a2_description)/meshes/hand/visual/R_index_2.stl" scale="${-direction} 1 1"/>
-				</geometry>
-				<material name="metallic black">
-					<color rgba="0.235294118 0.235294118 0.235294118 1"/>
-				</material>
+					<mesh filename="file://$(find agibot_a2_description)/meshes/hand/visual/index_2.obj" scale="${direction} 1 1"/>
+				</geometry>
 			</visual>
 			<collision>
@@ -214,5 +196,5 @@
 			</collision>
 		</link>
-		<joint name="${prefix_upper}index_2_joint" type="fixed">
+		<joint name="${prefix_upper}index_2_joint" type="revolute">
 			<origin xyz="-0.00025731 0.032131 -0.001"/>
 			<parent link="${prefix_upper}index_1"/>
@@ -220,5 +202,5 @@
 			<axis xyz="0 0 ${-dir}"/>
 			<limit lower="0" upper="1.7" effort="1" velocity="100"/>
-			<mimic joint="${prefix_upper}index_1_joint" multiplier="1" offset="0"/>
+			<mimic joint="${prefix_upper}index_joint" multiplier="1" offset="0"/>
 		</joint>
 		<!-- Middle 1 -->
@@ -232,17 +214,14 @@
 			<visual>
 				<geometry>
-					<mesh filename="file://$(find agibot_a2_description)/meshes/hand/visual/R_middle_1.stl" scale="${-direction} 1 1"/>
-				</geometry>
-				<material name="metallic black">
-					<color rgba="0.235294118 0.235294118 0.235294118 1"/>
-				</material>
-			</visual>
-			<collision>
-				<geometry>
-					<mesh filename="file://$(find agibot_a2_description)/meshes/hand/collision/R_middle_1_hull.stl" scale="${-direction} 1 1"/>
-				</geometry>
-			</collision>
-		</link>
-		<joint name="${prefix_upper}middle_1_joint" type="fixed">
+					<mesh filename="file://$(find agibot_a2_description)/meshes/hand/visual/index_1.obj" scale="${direction} 1 1"/>
+				</geometry>
+			</visual>
+			<collision>
+				<geometry>
+					<mesh filename="file://$(find agibot_a2_description)/meshes/hand/collision/R_index_1_hull.stl" scale="${-direction} 1 1"/>
+				</geometry>
+			</collision>
+		</link>
+		<joint name="${prefix_upper}middle_joint" type="revolute">
 			<origin xyz="-0.014728 ${dir*0.0059953} 0.1205" rpy="1.5708 0 -1.5708"/>
 			<parent link="${name}_hand"/>
@@ -261,9 +240,6 @@
 			<visual>
 				<geometry>
-					<mesh filename="file://$(find agibot_a2_description)/meshes/hand/visual/R_middle_2.stl" scale="${-direction} 1 1"/>
-				</geometry>
-				<material name="metallic black">
-					<color rgba="0.235294118 0.235294118 0.235294118 1"/>
-				</material>
+					<mesh filename="file://$(find agibot_a2_description)/meshes/hand/visual/middle_2.obj" scale="${direction} 1 1"/>
+				</geometry>
 			</visual>
 			<collision>
@@ -273,5 +249,5 @@
 			</collision>
 		</link>
-		<joint name="${prefix_upper}middle_2_joint" type="fixed">
+		<joint name="${prefix_upper}middle_2_joint" type="revolute">
 			<origin xyz="-0.000257313524408706 0.0321313914917268 -0.000999999999997433"/>
 			<parent link="${prefix_upper}middle_1"/>
@@ -279,5 +255,5 @@
 			<axis xyz="0 0 ${-dir}"/>
 			<limit lower="0" upper="1.7" effort="1" velocity="100"/>
-			<mimic joint="${prefix_upper}middle_1_joint" multiplier="1" offset="0"/>
+			<mimic joint="${prefix_upper}middle_joint" multiplier="1" offset="0"/>
 		</joint>
 		<!-- Ring 1 -->
@@ -291,17 +267,14 @@
 			<visual>
 				<geometry>
-					<mesh filename="file://$(find agibot_a2_description)/meshes/hand/visual/R_ring_1.stl" scale="${-direction} 1 1"/>
-				</geometry>
-				<material name="metallic black">
-					<color rgba="0.235294118 0.235294118 0.235294118 1"/>
-				</material>
-			</visual>
-			<collision>
-				<geometry>
-					<mesh filename="file://$(find agibot_a2_description)/meshes/hand/collision/R_ring_1_hull.stl" scale="${-direction} 1 1"/>
-				</geometry>
-			</collision>
-		</link>
-		<joint name="${prefix_upper}ring_1_joint" type="fixed">
+					<mesh filename="file://$(find agibot_a2_description)/meshes/hand/visual/index_1.obj" scale="${direction} 1 1"/>
+				</geometry>
+			</visual>
+			<collision>
+				<geometry>
+					<mesh filename="file://$(find agibot_a2_description)/meshes/hand/collision/R_index_1_hull.stl" scale="${-direction} 1 1"/>
+				</geometry>
+			</collision>
+		</link>
+		<joint name="${prefix_upper}ring_joint" type="revolute">
 			<origin xyz="0.0060088 ${dir*0.0059953} 0.12031" rpy="1.5184 0 -1.5708"/>
 			<parent link="${name}_hand"/>
@@ -320,17 +293,14 @@
 			<visual>
 				<geometry>
-					<mesh filename="file://$(find agibot_a2_description)/meshes/hand/visual/R_ring_2.stl" scale="${-direction} 1 1"/>
-				</geometry>
-				<material name="metallic black">
-					<color rgba="0.235294118 0.235294118 0.235294118 1"/>
-				</material>
-			</visual>
-			<collision>
-				<geometry>
-					<mesh filename="file://$(find agibot_a2_description)/meshes/hand/collision/R_ring_2_hull.stl" scale="${-direction} 1 1"/>
-				</geometry>
-			</collision>
-		</link>
-		<joint name="${prefix_upper}ring_2_joint" type="fixed">
+					<mesh filename="file://$(find agibot_a2_description)/meshes/hand/visual/middle_2.obj" scale="${direction} 1 1"/>
+				</geometry>
+			</visual>
+			<collision>
+				<geometry>
+					<mesh filename="file://$(find agibot_a2_description)/meshes/hand/collision/R_middle_2_hull.stl" scale="${-direction} 1 1"/>
+				</geometry>
+			</collision>
+		</link>
+		<joint name="${prefix_upper}ring_2_joint" type="revolute">
 			<origin xyz="-0.00025731 0.032131 -0.001"/>
 			<parent link="${prefix_upper}ring_1"/>
@@ -338,5 +308,5 @@
 			<axis xyz="0 0 ${-dir}"/>
 			<limit lower="0" upper="1.7" effort="1" velocity="100"/>
-			<mimic joint="${prefix_upper}ring_1_joint" multiplier="1" offset="0"/>
+			<mimic joint="${prefix_upper}ring_joint" multiplier="1" offset="0"/>
 		</joint>
 		<!-- Pinky 1 -->
@@ -350,17 +320,14 @@
 			<visual>
 				<geometry>
-					<mesh filename="file://$(find agibot_a2_description)/meshes/hand/visual/R_pinky_1.stl" scale="${-direction} 1 1"/>
-				</geometry>
-				<material name="metallic black">
-					<color rgba="0.235294118 0.235294118 0.235294118 1"/>
-				</material>
-			</visual>
-			<collision>
-				<geometry>
-					<mesh filename="file://$(find agibot_a2_description)/meshes/hand/collision/R_pinky_1_hull.stl" scale="${-direction} 1 1"/>
-				</geometry>
-			</collision>
-		</link>
-		<joint name="${prefix_upper}pinky_1_joint" type="fixed">
+					<mesh filename="file://$(find agibot_a2_description)/meshes/hand/visual/index_1.obj" scale="${direction} 1 1"/>
+				</geometry>
+			</visual>
+			<collision>
+				<geometry>
+					<mesh filename="file://$(find agibot_a2_description)/meshes/hand/collision/R_index_1_hull.stl" scale="${-direction} 1 1"/>
+				</geometry>
+			</collision>
+		</link>
+		<joint name="${prefix_upper}pinky_joint" type="revolute">
 			<origin xyz="0.026254 ${dir*0.0059953} 0.11901" rpy="1.4661 0 -1.5708"/>
 			<parent link="${name}_hand"/>
@@ -379,9 +346,6 @@
 			<visual>
 				<geometry>
-					<mesh filename="file://$(find agibot_a2_description)/meshes/hand/visual/R_pinky_2.stl" scale="${-direction} 1 1"/>
-				</geometry>
-				<material name="metallic black">
-					<color rgba="0.235294118 0.235294118 0.235294118 1"/>
-				</material>
+					<mesh filename="file://$(find agibot_a2_description)/meshes/hand/visual/pinky_2.obj" scale="${direction} 1 1"/>
+				</geometry>
 			</visual>
 			<collision>
@@ -391,5 +355,5 @@
 			</collision>
 		</link>
-		<joint name="${prefix_upper}pinky_2_joint" type="fixed">
+		<joint name="${prefix_upper}pinky_2_joint" type="revolute">
 			<origin xyz="-0.00025731 0.032131 -0.001"/>
 			<parent link="${prefix_upper}pinky_1"/>
@@ -397,5 +361,5 @@
 			<axis xyz="0 0 ${-dir}"/>
 			<limit lower="0" upper="1.7" effort="1" velocity="100"/>
-			<mimic joint="${prefix_upper}pinky_1_joint" multiplier="1" offset="0"/>
+			<mimic joint="${prefix_upper}pinky_joint" multiplier="1" offset="0"/>
 		</joint>
 	</xacro:macro>
