Commit message: leg mesh

File: humanoid/Agibot/agibot_a2_description/xacro/leg.xacro (robot description, xacro)
@@ -22,17 +22,14 @@
 			<visual>
 				<geometry>
-					<mesh filename="file://$(find agibot_a2_description)/meshes/leg/visual/${prefix}hip_roll.stl"/>
-				</geometry>
-				<material name="metallic black">
-					<color rgba="0.235294118 0.235294118 0.235294118 1"/>
-				</material>
-			</visual>
-			<collision>
-				<geometry>
-					<mesh filename="file://$(find agibot_a2_description)/meshes/leg/collision/${prefix}hip_roll_hull.stl"/>
-				</geometry>
-			</collision>
-		</link>
-		<joint name="idx${idx_base}_${prefix}hip_roll" type="revolute">
+					<mesh filename="file://$(find agibot_a2_description)/meshes/leg/visual/hip_roll.obj"/>
+				</geometry>
+			</visual>
+			<collision>
+				<geometry>
+					<mesh filename="file://$(find agibot_a2_description)/meshes/leg/collision/hip_roll.stl"/>
+				</geometry>
+			</collision>
+		</link>
+		<joint name="${prefix}hip_roll" type="revolute">
 			<origin xyz="-0.0808 ${hip_roll_origin_y} -0.0652" rpy="0.7854 0 1.5708"/>
 			<parent link="${parent_link}"/>
@@ -50,17 +47,14 @@
 			<visual>
 				<geometry>
-					<mesh filename="file://$(find agibot_a2_description)/meshes/leg/visual/${prefix}hip_yaw.stl"/>
-				</geometry>
-				<material name="metallic black">
-					<color rgba="0.235294118 0.235294118 0.235294118 1"/>
-				</material>
-			</visual>
-			<collision>
-				<geometry>
-					<mesh filename="file://$(find agibot_a2_description)/meshes/leg/collision/${prefix}hip_yaw_hull.stl"/>
-				</geometry>
-			</collision>
-		</link>
-		<joint name="idx${idx_base+1}_${prefix}hip_yaw" type="revolute">
+					<mesh filename="file://$(find agibot_a2_description)/meshes/leg/visual/hip_yaw.obj" scale="1 ${direction} 1"/>
+				</geometry>
+			</visual>
+			<collision>
+				<geometry>
+					<mesh filename="file://$(find agibot_a2_description)/meshes/leg/collision/hip_yaw.stl" scale="1 ${direction} 1"/>
+				</geometry>
+			</collision>
+		</link>
+		<joint name="${prefix}hip_yaw" type="revolute">
 			<origin xyz="0 -0.017 -0.0682" rpy="1.5708 -1.5708 0"/>
 			<parent link="${prefix}hip_roll"/>
@@ -78,17 +72,14 @@
 			<visual>
 				<geometry>
-					<mesh filename="file://$(find agibot_a2_description)/meshes/leg/visual/${prefix}hip_pitch.stl"/>
-				</geometry>
-				<material name="metallic silver">
-					<color rgba="0.878431373 0.878431373 0.901960784 1"/>
-				</material>
-			</visual>
-			<collision>
-				<geometry>
-					<mesh filename="file://$(find agibot_a2_description)/meshes/leg/collision/${prefix}hip_pitch_hull.stl"/>
-				</geometry>
-			</collision>
-		</link>
-		<joint name="idx${idx_base+2}_${prefix}hip_pitch" type="revolute">
+					<mesh filename="file://$(find agibot_a2_description)/meshes/leg/visual/hip_pitch.obj" scale="1 1 ${direction}"/>
+				</geometry>
+			</visual>
+			<collision>
+				<geometry>
+					<mesh filename="file://$(find agibot_a2_description)/meshes/leg/collision/hip_pitch.stl" scale="1 1 ${direction}"/>
+				</geometry>
+			</collision>
+		</link>
+		<joint name="${prefix}hip_pitch" type="revolute">
 			<origin xyz="0 ${-dir*0.020} 0.1205" rpy="1.5708 0.7854 0"/>
 			<parent link="${prefix}hip_yaw"/>
@@ -106,9 +97,6 @@
 			<visual>
 				<geometry>
-					<mesh filename="file://$(find agibot_a2_description)/meshes/leg/visual/${prefix}tarsus.stl"/>
-				</geometry>
-				<material name="metallic silver">
-					<color rgba="0.878431373 0.878431373 0.901960784 1"/>
-				</material>
+					<mesh filename="file://$(find agibot_a2_description)/meshes/leg/visual/tarsus.obj" scale="1 1 ${direction}"/>
+				</geometry>
 			</visual>
 			<collision>
@@ -118,5 +106,5 @@
 			</collision>
 		</link>
-		<joint name="idx${idx_base+3}_${prefix}tarsus" type="revolute">
+		<joint name="${prefix}tarsus" type="revolute">
 			<origin xyz="-0.34 0 0"/>
 			<parent link="${prefix}hip_pitch"/>
