Commit message: a2 mesh

File: humanoid/Agibot/agibot_a2_description/xacro/arm.xacro (robot description, xacro)
@@ -140,5 +140,5 @@
 			</collision>
 		</link>
-		<joint name="${prefix}arm_joint5" type="fixed">
+		<joint name="${prefix}arm_joint5" type="revolute">
 			<origin xyz="0  ${-dir*0.103} 0.0" rpy="1.5707963 0 0"/>
 			<parent link="${prefix}arm_link04"/>

File: humanoid/Agibot/agibot_a2_description/xacro/leg.xacro (robot description, xacro)
@@ -102,5 +102,5 @@
 			<collision>
 				<geometry>
-					<mesh filename="file://$(find agibot_a2_description)/meshes/leg/collision/${prefix}tarsus_hull.stl"/>
+					<mesh filename="file://$(find agibot_a2_description)/meshes/leg/collision/tarsus.stl" scale="1 1 ${direction}"/>
 				</geometry>
 			</collision>
@@ -121,15 +121,7 @@
 			<visual>
 				<geometry>
-					<mesh filename="file://$(find agibot_a2_description)/meshes/leg/visual/${prefix}toe_pitch.stl"/>
+					<mesh filename="file://$(find agibot_a2_description)/meshes/leg/visual/toe_pitch.obj"/>
 				</geometry>
-				<material name="metallic black">
-					<color rgba="0.235294118 0.235294118 0.235294118 1"/>
-				</material>
 			</visual>
-			<collision>
-				<geometry>
-					<mesh filename="file://$(find agibot_a2_description)/meshes/leg/collision/${prefix}toe_pitch_hull.stl"/>
-				</geometry>
-			</collision>
 		</link>
 		<joint name="idx${idx_base+4}_${prefix}toe_pitch" type="revolute">
@@ -149,13 +141,10 @@
 			<visual>
 				<geometry>
-					<mesh filename="file://$(find agibot_a2_description)/meshes/leg/visual/${prefix}toe_roll.stl"/>
+					<mesh filename="file://$(find agibot_a2_description)/meshes/leg/visual/toe_roll.obj"/>
 				</geometry>
-				<material name="metallic black">
-					<color rgba="0.235294118 0.235294118 0.235294118 1"/>
-				</material>
 			</visual>
 			<collision>
 				<geometry>
-					<mesh filename="file://$(find agibot_a2_description)/meshes/leg/collision/${prefix}toe_roll_hull.stl"/>
+					<mesh filename="file://$(find agibot_a2_description)/meshes/leg/collision/toe_roll.stl"/>
 				</geometry>
 			</collision>
@@ -168,131 +157,4 @@
 			<limit lower="-0.488692182" upper="0.488692182" effort="50" velocity="12"/>
 		</joint>
-		<!-- Toe A -->
-		<link name="${prefix}toe_A">
-			<inertial>
-				<origin xyz="0.0161339967539726 0.000256129454551002 ${dir*0.00157429551114607}"/>
-				<mass value="0.0959876868449394"/>
-				<inertia ixx="1.47306660350068E-05" ixy="7.10372384628399E-07" ixz="${dir*1.01514226468701E-05}"
-							 iyy="5.94672539950203E-05" iyz="${dir*1.61153684004436E-07}" izz="6.68731361080011E-05"/>
-			</inertial>
-			<visual>
-				<geometry>
-					<mesh filename="file://$(find agibot_a2_description)/meshes/leg/visual/${prefix}toe_A.stl"/>
-				</geometry>
-				<material name="metallic black">
-					<color rgba="0.235294118 0.235294118 0.235294118 1"/>
-				</material>
-			</visual>
-			<collision>
-				<geometry>
-					<mesh filename="file://$(find agibot_a2_description)/meshes/leg/collision/${prefix}toe_A_hull.stl"/>
-				</geometry>
-				<material name="metallic black">
-					<color rgba="0.235294118 0.235294118 0.235294118 1"/>
-				</material>
-			</collision>
-		</link>
-		<joint name="idx${idx_base+4}_01_${prefix}toe_motorA" type="fixed">
-			<origin xyz="-0.138 0 ${-dir*0.0315}" rpy="0 0 -1.5708"/>
-			<parent link="${prefix}tarsus"/>
-			<child link="${prefix}toe_A"/>
-			<axis xyz="0 0 1"/>
-			<xacro:if value="${name == 'left'}">
-				<limit lower="-1.5708" upper="1.5708" effort="0" velocity="0"/>
-			</xacro:if>
-			<xacro:unless value="${name == 'left'}">
-				<limit lower="0" upper="0" effort="0" velocity="0"/>
-			</xacro:unless>
-		</joint>
-		<!-- Toe A rod -->
-		<link name="${prefix}toe_A_rod">
-			<inertial>
-				<origin xyz="-0.11950903764711 -4.54312300279813E-09 2.0722082788957E-05"/>
-				<mass value="0.133194826485547"/>
-				<inertia ixx="4.13825335822083E-06" ixy="6.85930711305851E-12" ixz="2.45335802357092E-09"
-							 iyy="0.000625059882342822" iyz="2.33641130593936E-12" izz="0.000627531716420437"/>
-			</inertial>
-			<visual>
-				<geometry>
-					<mesh filename="file://$(find agibot_a2_description)/meshes/leg/visual/${prefix}toe_A_rod.stl"/>
-				</geometry>
-				<material name="metallic black">
-					<color rgba="0.235294118 0.235294118 0.235294118 1"/>
-				</material>
-			</visual>
-			<collision>
-				<geometry>
-					<mesh filename="file://$(find agibot_a2_description)/meshes/leg/collision/${prefix}toe_A_rod_hull.stl"/>
-				</geometry>
-			</collision>
-		</link>
-		<joint name="idx${idx_base+4}_01_${prefix}toe_motorA_ball" type="fixed">
-			<origin xyz="0.062992 0.001 0" rpy="${-dir*3.1416} 0 1.5708"/>
-			<parent link="${prefix}toe_A"/>
-			<child link="${prefix}toe_A_rod"/>
-			<axis xyz="0 0 0"/>
-		</joint>
-		<!-- Toe B -->
-		<link name="${prefix}toe_B">
-			<inertial>
-				<origin xyz="0.0161339965985728 0.000256125750057401 ${-dir*0.00157429547986562}"/>
-				<mass value="0.0959876865489089"/>
-				<inertia ixx="1.47306660936761E-05" ixy="7.10374422550964E-07" ixz="${-dir*1.0151422567557E-05}"
-							 iyy="5.94672535179347E-05" iyz="${-dir*1.61154476946449E-07}" izz="6.68731357299622E-05"/>
-			</inertial>
-			<visual>
-				<geometry>
-					<mesh filename="file://$(find agibot_a2_description)/meshes/leg/visual/${prefix}toe_B.stl"/>
-				</geometry>
-				<material name="metallic black">
-					<color rgba="0.235294118 0.235294118 0.235294118 1"/>
-				</material>
-			</visual>
-			<collision>
-				<geometry>
-					<mesh filename="file://$(find agibot_a2_description)/meshes/leg/collision/${prefix}toe_B_hull.stl"/>
-				</geometry>
-			</collision>
-		</link>
-		<joint name="idx${idx_base+5}_01_${prefix}toe_motorB" type="fixed">
-			<origin xyz="-0.232 0 ${dir*0.0315}" rpy="0 0 -1.5708"/>
-			<parent link="${prefix}tarsus"/>
-			<child link="${prefix}toe_B"/>
-			<axis xyz="0 0 1"/>
-			<xacro:if value="${name == 'left'}">
-				<limit lower="-1.5708" upper="1.5708" effort="0" velocity="0"/>
-			</xacro:if>
-			<xacro:unless value="${name == 'left'}">
-				<limit lower="0" upper="0" effort="0" velocity="0"/>
-			</xacro:unless>
-		</joint>
-		<!-- Toe B rod -->
-		<link name="${prefix}toe_B_rod">
-			<inertial>
-				<origin xyz="-0.0725000006179941 2.39833153337088E-11 2.75483156604583E-05"/>
-				<mass value="0.0989853087337602"/>
-				<inertia ixx="3.41390504492216E-06" ixy="-7.00234342247419E-12" ixz="-1.67152635087163E-13"
-							 iyy="0.000168898913472365" iyz="-6.91334604265453E-15" izz="0.000171065639810982"/>
-			</inertial>
-			<visual>
-				<geometry>
-					<mesh filename="file://$(find agibot_a2_description)/meshes/leg/visual/${prefix}toe_B_rod.stl"/>
-				</geometry>
-				<material name="metallic black">
-					<color rgba="0.235294118 0.235294118 0.235294118 1"/>
-				</material>
-			</visual>
-			<collision>
-				<geometry>
-					<mesh filename="file://$(find agibot_a2_description)/meshes/leg/collision/${prefix}toe_B_rod_hull.stl"/>
-				</geometry>
-			</collision>
-		</link>
-		<joint name="idx${idx_base+5}_01_${prefix}toe_motorB_ball" type="fixed">
-			<origin xyz="0.063 0.001 0" rpy="${-dir*3.14159265358666} 0 1.57074160362305"/>
-			<parent link="${prefix}toe_B"/>
-			<child link="${prefix}toe_B_rod"/>
-			<axis xyz="0 0 0"/>
-		</joint>
 	</xacro:macro>
 </robot>
