Commit message: 添加dobot_atom OCS2 demo

File: humanoid/Dobot/dobot_atom_description/xacro/robot.xacro (robot description, xacro)
@@ -5,8 +5,21 @@
 <robot name="atom" xmlns:xacro="http://www.ros.org/wiki/xacro">
 	<link name="base_link"/>
-	<joint name="base_joint" type="fixed">
-		<parent link="base_link"/>
-		<child link="pelvis"/>
-	</joint>
-	<xacro:include filename="$(find dobot_atom_description)/xacro/full_body.xacro"/>
+	<!-- 切换模式参数 -->
+	<xacro:arg name="type" default="full" />
+    <!-- 当为 full 模式时，创建 base_link -> pelvis 连接 -->
+    <xacro:if value="${'$(arg type)' == 'full'}">
+    	<joint name="base_joint" type="fixed">
+    		<parent link="base_link"/>
+    		<child link="pelvis"/>
+    	</joint>
+    </xacro:if>
+	<!-- 全身模式 -->
+    <xacro:if value="${'$(arg type)' == 'full'}">
+        <xacro:include filename="$(find dobot_atom_description)/xacro/full_body.xacro"/>
+    </xacro:if>
+    <!-- 上半身模式 -->
+    <xacro:if value="${'$(arg type)' == 'upper'}">
+        <xacro:include filename="$(find dobot_atom_description)/xacro/full_upper_body.xacro"/>
+    </xacro:if>
+	<!--xacro:include filename="$(find dobot_atom_description)/xacro/full_body.xacro"/-->
 </robot>

File: humanoid/Dobot/dobot_atom_description/xacro/upper_body.xacro (robot description, xacro)
@@ -4,5 +4,5 @@
      For more information, please see http://wiki.ros.org/sw_urdf_exporter -->
 <robot name="atom" xmlns:xacro="http://www.ros.org/wiki/xacro">
-	<xacro:macro name="AtomUpperBody" params="parent_link">
+	<xacro:macro name="AtomUpperBody" params="parent_link type">
 		<link name="torso_link">
 			<inertial>
@@ -23,10 +23,20 @@
 			</collision>
 		</link>
-		<joint name="torso_joint" type="revolute">
-			<parent link="${parent_link}"/>
-			<child link="torso_link"/>
-			<axis xyz="0 0 1"/>
-			<limit lower="-2.7925" upper="2.7925" effort="1000" velocity="100"/>
-		</joint>
+		<xacro:if value="${type == 'upper'}">
+			<!-- upper 模式锁死躯干 -->
+			<joint name="torso_joint" type="fixed">
+				<parent link="${parent_link}"/>
+				<child link="torso_link"/>
+			</joint>
+		</xacro:if>
+		<xacro:if value="${type != 'upper'}">
+		<!-- full 模式保持原来的可旋转关节 -->
+			<joint name="torso_joint" type="revolute">
+				<parent link="${parent_link}"/>
+				<child link="torso_link"/>
+				<axis xyz="0 0 1"/>
+				<limit lower="-2.7925" upper="2.7925" effort="1000" velocity="100"/>
+			</joint>
+		</xacro:if>
 		<link name="head_yaw_link">
 			<inertial>
