Commit message: fix dobot path

File: humanoid/Dobot/dobot_atom_description/urdf/dobot_atom.urdf (robot description, URDF)
Before this commit: robot atom, 19 links, 18 joints
Links:
- link head_pitch_link: geometry collision box size=0.16 0.14 0.14; visual mesh filename=package://dobot_atom_description/meshes/body/head_pitch.obj
- link head_yaw_link: geometry visual mesh filename=package://dobot_atom_description/meshes/body/head_yaw.obj
- link left_elbow_pitch_link: geometry collision box size=0.30 0.06 0.06; visual mesh filename=package://dobot_atom_description/meshes/arm/link4.obj
- link left_elbow_roll_link: geometry visual mesh filename=package://dobot_atom_description/meshes/arm/link5.obj
- link left_shoulder_pitch_link: geometry visual mesh filename=package://dobot_atom_description/meshes/arm/link1.obj scale=1 1 1
- link left_shoulder_roll_link: geometry collision box size=0.06 0.06 0.24; visual mesh filename=package://dobot_atom_description/meshes/arm/link2.obj scale=1 1 1
- link left_shoulder_yaw_link: geometry visual mesh filename=package://dobot_atom_description/meshes/arm/link3.obj
- link left_wrist_pitch_link: geometry visual mesh filename=package://dobot_atom_description/meshes/arm/link6.obj scale=1 1 1
- link left_wrist_yaw_link: geometry visual mesh filename=package://dobot_atom_description/meshes/arm/link7.obj scale=1 1 1
- link right_elbow_pitch_link: geometry collision box size=0.30 0.06 0.06; visual mesh filename=package://dobot_atom_description/meshes/arm/link4.obj
- link right_elbow_roll_link: geometry visual mesh filename=package://dobot_atom_description/meshes/arm/link5.obj
- link right_shoulder_pitch_link: geometry visual mesh filename=package://dobot_atom_description/meshes/arm/link1.obj scale=1 -1 1
- link right_shoulder_roll_link: geometry collision box size=0.06 0.06 0.24; visual mesh filename=package://dobot_atom_description/meshes/arm/link2.obj scale=1 -1 1
- link right_shoulder_yaw_link: geometry visual mesh filename=package://dobot_atom_description/meshes/arm/link3.obj
- link right_wrist_pitch_link: geometry visual mesh filename=package://dobot_atom_description/meshes/arm/link6.obj scale=1 -1 1
- link right_wrist_yaw_link: geometry visual mesh filename=package://dobot_atom_description/meshes/arm/link7.obj scale=1 -1 1
- link torso_link: geometry collision box size=0.26 0.24 0.4; visual mesh filename=package://dobot_atom_description/meshes/body/torso.obj

Commit message: add self collision

File: humanoid/Dobot/dobot_atom_description/urdf/dobot_atom.urdf (robot description, URDF)
Before this commit: robot atom, 19 links, 18 joints
Links:
- link head_pitch_link: geometry collision box size=0.16 0.14 0.14; visual mesh filename=file:///home/ly/ros2_ws/install/dobot_atom_description/shar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
- link head_yaw_link: geometry visual mesh filename=file:///home/ly/ros2_ws/install/dobot_atom_description/shar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
- link left_elbow_pitch_link: geometry collision cylinder length=0.11 radius=0.04; visual mesh filename=file:///home/ly/ros2_ws/install/dobot_atom_description/shar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
- link left_elbow_roll_link: geometry collision cylinder length=0.15 radius=0.045; visual mesh filename=file:///home/ly/ros2_ws/install/dobot_atom_description/shar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
- link left_shoulder_pitch_link: geometry visual mesh filename=file:///home/ly/ros2_ws/install/dobot_atom_description/shar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 scale=1 1 1
- link left_shoulder_roll_link: geometry visual mesh filename=file:///home/ly/ros2_ws/install/dobot_atom_description/shar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 scale=1 1 1
- link left_shoulder_yaw_link: geometry collision cylinder length=0.20 radius=0.04; visual mesh filename=file:///home/ly/ros2_ws/install/dobot_atom_description/shar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
- link left_wrist_pitch_link: geometry collision cylinder length=0.09 radius=0.035; visual mesh filename=file:///home/ly/ros2_ws/install/dobot_atom_description/shar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 scale=1 1 1
- link left_wrist_yaw_link: geometry collision cylinder length=0.09 radius=0.035; visual mesh filename=file:///home/ly/ros2_ws/install/dobot_atom_description/shar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 scale=1 1 1
- link right_elbow_pitch_link: geometry collision cylinder length=0.11 radius=0.04; visual mesh filename=file:///home/ly/ros2_ws/install/dobot_atom_description/shar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
- link right_elbow_roll_link: geometry collision cylinder length=0.15 radius=0.045; visual mesh filename=file:///home/ly/ros2_ws/install/dobot_atom_description/shar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
- link right_shoulder_pitch_link: geometry visual mesh filename=file:///home/ly/ros2_ws/install/dobot_atom_description/shar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 scale=1 -1 1
- link right_shoulder_roll_link: geometry visual mesh filename=file:///home/ly/ros2_ws/install/dobot_atom_description/shar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 scale=1 -1 1
- link right_shoulder_yaw_link: geometry collision cylinder length=0.20 radius=0.04; visual mesh filename=file:///home/ly/ros2_ws/install/dobot_atom_description/shar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
- link right_wrist_pitch_link: geometry collision cylinder length=0.09 radius=0.035; visual mesh filename=file:///home/ly/ros2_ws/install/dobot_atom_description/shar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 scale=1 -1 1
- link right_wrist_yaw_link: geometry collision cylinder length=0.09 radius=0.035; visual mesh filename=file:///home/ly/ros2_ws/install/dobot_atom_description/shar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 scale=1 -1 1
- link torso_link: geometry collision box size=0.26 0.24 0.4; visual mesh filename=file:///home/ly/ros2_ws/install/dobot_atom_description/shar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
