Commit message: add brainco revo2 config

File: humanoid/DexForce/dexfoce_w1_description/xacro/eefs.xacro (robot description, xacro)
@@ -1,8 +1,12 @@
 <?xml version="1.0"?>
 <robot xmlns:xacro="http://www.ros.org/wiki/xacro">
-	<xacro:macro name="EndEffectors" params="gripper_type:=''">
-		<!-- Note: gripper_type 不为空时表示使用夹爪 -->
+	<xacro:macro name="EndEffectors" params="hand_type:='' gripper_type:=''">
+		<!-- Note:
+		     - gripper_type 不为空时表示使用夹爪（保持原有逻辑）
+		     - hand_type 只在需要区分灵巧手时使用（如 revo1）
+		     - 两者都为空时表示无末端执行器配置
+		-->
 		<!-- 无末端执行器配置（但有 eef 作为控制参考帧） -->
-		<xacro:if value="${gripper_type == ''}">
+		<xacro:if value="${hand_type == '' and gripper_type == ''}">
 			<link name="left_eef"/>
 			<link name="right_eef"/>
@@ -30,4 +34,20 @@
 			</joint>
 		</xacro:if>
+		<!-- 灵巧手类型 -->
+		<xacro:if value="${hand_type == 'revo1'}">
+			<xacro:include filename="$(find brainco_description)/xacro/revo1.xacro"/>
+			<xacro:BrainCoHand name="left_hand" direction="1" fixed_joints="false"/>
+			<joint name="left_hand_base_joint" type="fixed">
+				<origin rpy="${PI/2} 0 ${PI}"/>
+				<parent link="left_tcp"/>
+				<child link="left_hand_hand_base"/>
+			</joint>
+			<xacro:BrainCoHand name="right_hand" direction="-1" fixed_joints="false"/>
+			<joint name="right_hand_base_joint" type="fixed">
+				<parent link="right_tcp"/>
+				<child link="right_hand_hand_base"/>
+				<origin rpy="${PI/2} 0 0"/>
+			</joint>
+		</xacro:if>
 	</xacro:macro>
 </robot>

File: humanoid/DexForce/dexfoce_w1_description/xacro/robot.xacro (robot description, xacro)
@@ -4,7 +4,9 @@
      For more information, please see http://wiki.ros.org/sw_urdf_exporter -->
 <robot name="DexForce W1" xmlns:xacro="http://www.ros.org/wiki/xacro">
+	<xacro:property name="PI" value="3.1415926535897931"/>
 	<!-- 切换模式参数 -->
 	<!-- type 选项：
 	     - ANTHROPOMORPHIC: 类人型（默认）
+	     - revo1: 类人型（带 BrainCo Revo1 灵巧手）
 	     - pro: 工业型（无夹爪）
 	     - pro_pgc140: 工业型（带 PGC_140_50 夹爪）
@@ -15,5 +17,8 @@
 	<xacro:property name="selected_arm_type" value="anthropomorphic"/>
 	<xacro:property name="selected_gripper_type" value=""/>
-	<!-- 从 type 解析 arm_type 和 gripper_type -->
+	<xacro:property name="selected_hand_type" value=""/>
+	<xacro:if value="${type_arg == 'revo1'}">
+		<xacro:property name="selected_hand_type" value="revo1"/>
+	</xacro:if>
 	<xacro:if value="${type_arg == 'pro'}">
 		<xacro:property name="selected_arm_type" value="industrial"/>
@@ -35,4 +40,4 @@
 	<!-- Include and generate end effector frames -->
 	<xacro:include filename="$(find dexforce_w1_description)/xacro/eefs.xacro"/>
-	<xacro:EndEffectors gripper_type="${selected_gripper_type}"/>
+	<xacro:EndEffectors hand_type="${selected_hand_type}" gripper_type="${selected_gripper_type}"/>
 </robot>

File: humanoid/DexForce/dexfoce_w1_description/xacro/ros2_control/robot.xacro (robot description, xacro)
@@ -40,4 +40,10 @@
 				</joint>
 			</xacro:if>
+			<!-- 灵巧手接口 -->
+			<xacro:if value="${selected_hand_type == 'revo1'}">
+				<xacro:include filename="$(find brainco_description)/xacro/ros2_control/revo1.xacro"/>
+				<xacro:revo1_interfaces name="left_hand"/>
+				<xacro:revo1_interfaces name="right_hand"/>
+			</xacro:if>
 		</ros2_control>
 	</xacro:unless>
