Commit message: zerith h1 mesh cleaned

File: humanoid/Zerith/zerith_h1_description/xacro/robot.xacro (robot description, xacro)
@@ -1,1687 +1,18 @@
 <?xml version="1.0"?>
+<!-- =================================================================================== -->
+<!-- |    Complete Robot Description for Zerith H1                                     | -->
+<!-- |    This file includes the chassis, body and arm components                      | -->
+<!-- =================================================================================== -->
 <robot name="zerith_h1" xmlns:xacro="http://www.ros.org/wiki/xacro">
-	<link
-			name="base_link">
-		<inertial>
-			<origin xyz="0.00021947 -0.00045719 0.08921288"/>
-			<mass
-					value="92.40985888"/>
-			<inertia
-					ixx="12.0810981"
-					ixy="-0.00505423"
-					ixz="1.25403037"
-					iyy="12.71175466"
-					iyz="-0.00705268"
-					izz="2.84527064"/>
-		</inertial>
-		<visual>
-			<geometry>
-				<mesh filename="file://$(find zerith_h1_description)/meshes/base/base_link.glb"/>
-			</geometry>
-		</visual>
-		<collision>
-			<geometry>
-				<mesh filename="file://$(find zerith_h1_description)/meshes/base/base_link.glb"/>
-			</geometry>
-		</collision>
-	</link>
-	<link name="body_link1">
-		<inertial>
-			<origin xyz="0.11560518 0.00060964 0.12206768"/>
-			<mass value="4.61714"/>
-			<inertia
-					ixx="0.00837134"
-					ixy="9.116e-05"
-					ixz="-0.00126268"
-					iyy="0.02136748"
-					iyz="-5.34e-06"
-					izz="0.02010722"/>
-		</inertial>
-		<visual>
-			<geometry>
-				<mesh filename="file://$(find zerith_h1_description)/meshes/body/body_link1.glb"/>
-			</geometry>
-		</visual>
-		<collision>
-			<geometry>
-				<mesh filename="file://$(find zerith_h1_description)/meshes/body/body_link1.glb"/>
-			</geometry>
-		</collision>
-	</link>
-	<joint name="body_joint1" type="prismatic">
-		<parent link="base_link"/>
-		<child link="body_link1"/>
-		<axis xyz="0 0 1"/>
-		<limit lower="0" upper="0.8" effort="0" velocity="0"/>
-	</joint>
-	<link name="body_pitch_link">
-		<inertial>
-			<origin
-					xyz="-0.00013249 0.00049551 0.10848426"
-			/>
-			<mass
-					value="3.528"/>
-			<inertia
-					ixx="0.01235314"
-					ixy="-9.38e-06"
-					ixz="6.133e-05"
-					iyy="0.01092549"
-					iyz="0.00020606"
-					izz="0.00739427"/>
-		</inertial>
-		<visual>
-			<geometry>
-				<mesh filename="file://$(find zerith_h1_description)/meshes/body/body_link2.glb"/>
-			</geometry>
-		</visual>
-		<collision>
-			<geometry>
-				<mesh filename="file://$(find zerith_h1_description)/meshes/body/body_link2.glb"/>
-			</geometry>
-		</collision>
-	</link>
-	<joint
-			name="body_joint2"
-			type="revolute">
-		<origin
-				xyz="0.1518 0 0.1275"
-		/>
-		<parent
-				link="body_link1"/>
-		<child
-				link="body_pitch_link"/>
-		<axis
-				xyz="0 1 0"/>
-		<limit
-				lower="-0.05236"
-				upper="1.309"
-				effort="204"
-				velocity="3.14"/>
-	</joint>
-	<link
-			name="body_yaw_link">
-		<inertial>
-			<origin
-					xyz="-0.00140951 0.00031062 0.13782806"
-			/>
-			<mass
-					value="3.85886409"/>
-			<inertia
-					ixx="0.03623808"
-					ixy="-3.118e-05"
-					ixz="0.00019346"
-					iyy="0.02298934"
-					iyz="3.738e-05"
-					izz="0.02244436"/>
-		</inertial>
-		<visual>
-			<geometry>
-				<mesh filename="file://$(find zerith_h1_description)/meshes/body/body_link3.glb"/>
-			</geometry>
-		</visual>
-		<collision>
-			<geometry>
-				<mesh filename="file://$(find zerith_h1_description)/meshes/body/body_link3.glb"/>
-			</geometry>
-		</collision>
-	</link>
-	<joint
-			name="body_yaw_joint"
-			type="revolute">
-		<origin
-				xyz="2.7149E-05 -0.00012105 0.1572"
-		/>
-		<parent
-				link="body_pitch_link"/>
-		<child
-				link="body_yaw_link"/>
-		<axis
-				xyz="0 0 1"/>
-		<limit
-				lower="-1.0472"
-				upper="1.0472"
-				effort="204"
-				velocity="3.14"/>
-	</joint>
-	<link
-			name="left_shoulder_pitch_link">
-		<inertial>
-			<origin
-					xyz="-0.00318713 0.04899419 0.00017253"
-			/>
-			<mass
-					value="0.64195"/>
-			<inertia
-					ixx="0.00045222"
-					ixy="4.1e-06"
-					ixz="1.97e-06"
-					iyy="0.00047136"
-					iyz="-1.26e-06"
-					izz="0.00059588"/>
-		</inertial>
-		<visual>
-			<geometry>
-				<mesh
-						filename="file://$(find zerith_h1_description)/meshes/left_shoulder_pitch_link.STL"/>
-			</geometry>
-			<material
-					name="">
-				<color
-						rgba="1 1 1 1"/>
-			</material>
-		</visual>
-		<collision>
-			<geometry>
-				<mesh
-						filename="file://$(find zerith_h1_description)/meshes/left_shoulder_pitch_link.STL"/>
-			</geometry>
-		</collision>
-	</link>
-	<joint
-			name="left_shoulder_pitch_joint"
-			type="revolute">
-		<origin
-				xyz="-0.00021966 0.11612 0.16797"
-		/>
-		<parent
-				link="body_yaw_link"/>
-		<child
-				link="left_shoulder_pitch_link"/>
-		<axis
-				xyz="0 1 0"/>
-		<limit
-				lower="-2.7925"
-				upper="1.5708"
-				effort="36"
-				velocity="8.164"/>
-	</joint>
-	<link
-			name="left_shoulder_roll_link">
-		<inertial>
-			<origin
-					xyz="0.00026688 0.00923491 -0.07177934"
-			/>
-			<mass
-					value="0.74474"/>
-			<inertia
-					ixx="0.00140268"
-					ixy="5.1e-06"
-					ixz="-3.427e-05"
-					iyy="0.00171477"
-					iyz="5.976e-05"
-					izz="0.00086884"/>
-		</inertial>
-		<visual>
-			<geometry>
-				<mesh
-						filename="file://$(find zerith_h1_description)/meshes/left_shoulder_roll_link.STL"/>
-			</geometry>
-			<material
-					name="">
-				<color
-						rgba="1 1 1 1"/>
-			</material>
-		</visual>
-		<collision>
-			<geometry>
-				<mesh
-						filename="file://$(find zerith_h1_description)/meshes/left_shoulder_roll_link.STL"/>
-			</geometry>
-		</collision>
-	</link>
-	<joint
-			name="left_shoulder_roll_joint"
-			type="revolute">
-		<origin
-				xyz="0.00019251 0.054 0.00013479"
-		/>
-		<parent
-				link="left_shoulder_pitch_link"/>
-		<child
-				link="left_shoulder_roll_link"/>
-		<axis
-				xyz="1 0 0"/>
-		<limit
-				lower="-0.5236"
-				upper="2.0944"
-				effort="36"
-				velocity="8.164"/>
-	</joint>
-	<link
-			name="left_shoulder_yaw_link">
-		<inertial>
-			<origin
-					xyz="0.02386961 -0.00041351 -0.12487547"
-			/>
-			<mass
-					value="0.86464"/>
-			<inertia
-					ixx="0.0031744"
-					ixy="5.93e-06"
-					ixz="0.00082261"
-					iyy="0.00347038"
-					iyz="-1.674e-05"
-					izz="0.00088318"/>
-		</inertial>
-		<visual>
-			<geometry>
-				<mesh
-						filename="file://$(find zerith_h1_description)/meshes/left_shoulder_yaw_link.STL"/>
-			</geometry>
-			<material
-					name="">
-				<color
-						rgba="1 1 1 1"/>
-			</material>
-		</visual>
-		<collision>
-			<geometry>
-				<mesh
-						filename="file://$(find zerith_h1_description)/meshes/left_shoulder_yaw_link.STL"/>
-			</geometry>
-		</collision>
-	</link>
-	<joint
-			name="left_shoulder_yaw_joint"
-			type="revolute">
-		<origin
-				xyz="0 0.01 -0.12225"
-		/>
-		<parent
-				link="left_shoulder_roll_link"/>
-		<child
-				link="left_shoulder_yaw_link"/>
-		<axis
-				xyz="0 0 1"/>
-		<limit
-				lower="-2.9671"
-				upper="2.9671"
-				effort="27"
-				velocity="7.3267"/>
-	</joint>
-	<link
-			name="left_elbow_link">
-		<inertial>
-			<origin
-					xyz="0.03098556 0.00057542 -0.0288024"
-			/>
-			<mass
-					value="0.33048"/>
-			<inertia
-					ixx="0.0004881"
-					ixy="1.78e-06"
-					ixz="0.00012277"
-					iyy="0.00048504"
-					iyz="-2.1e-06"
-					izz="0.00054349"/>
-		</inertial>
-		<visual>
-			<geometry>
-				<mesh
-						filename="file://$(find zerith_h1_description)/meshes/left_elbow_link.STL"/>
-			</geometry>
-			<material
-					name="">
-				<color
-						rgba="1 1 1 1"/>
-			</material>
-		</visual>
-		<collision>
-			<geometry>
-				<mesh
-						filename="file://$(find zerith_h1_description)/meshes/left_elbow_link.STL"/>
-			</geometry>
-		</collision>
-	</link>
-	<joint
-			name="left_elbow_joint"
-			type="revolute">
-		<origin
-				xyz="0.042 0 -0.16775"
-		/>
-		<parent
-				link="left_shoulder_yaw_link"/>
-		<child
-				link="left_elbow_link"/>
-		<axis
-				xyz="0 1 0"/>
-		<limit
-				lower="-1.5184"
-				upper="1.5708"
-				effort="27"
-				velocity="7.3267"/>
-	</joint>
-	<link
-			name="left_wrist_roll_link">
-		<inertial>
-			<origin
-					xyz="0.06375062 -5.405e-05 -0.0009515"
-			/>
-			<mass
-					value="0.865677"/>
-			<inertia
-					ixx="0.00052491"
-					ixy="-6.1e-07"
-					ixz="3.461e-05"
-					iyy="0.00159541"
-					iyz="6.3e-07"
-					izz="0.00149224"/>
-		</inertial>
-		<visual>
-			<geometry>
-				<mesh
-						filename="file://$(find zerith_h1_description)/meshes/left_wrist_roll_link.STL"/>
-			</geometry>
-			<material
-					name="">
-				<color
-						rgba="1 1 1 1"/>
-			</material>
-		</visual>
-		<collision>
-			<geometry>
-				<mesh
-						filename="file://$(find zerith_h1_description)/meshes/left_wrist_roll_link.STL"/>
-			</geometry>
-		</collision>
-	</link>
-	<joint
-			name="left_wrist_roll_joint"
-			type="revolute">
-		<origin
-				xyz="0.07422 0 -0.042"
-		/>
-		<parent
-				link="left_elbow_link"/>
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