Commit message: update zerith h1

File: humanoid/Zerith/zerith_h1_description/xacro/component.xacro (robot description, xacro)
@@ -12,4 +12,6 @@
   <xacro:arg name="type" default="base"/>
   <xacro:arg name="chassis_joints_movable" default="false"/>
+  <xacro:arg name="isaac" default="false"/>
+  <xacro:arg name="camera" default="d405"/>
   <xacro:if value="${'$(arg type)' != 'base' and '$(arg type)' != 'chassis'}">
     <link name="base_link"/>
@@ -20,6 +22,6 @@
     <xacro:include filename="$(find zerith_h1_description)/xacro/components/arm.xacro"/>
     <xacro:H1Chassis joints_movable="$(arg chassis_joints_movable)"/>
-    <xacro:H1Arm name="left" direction="1"/>
-    <xacro:H1Arm name="right" direction="-1"/>
+    <xacro:H1Arm name="left" direction="1" camera="$(arg camera)"/>
+    <xacro:H1Arm name="right" direction="-1" camera="$(arg camera)"/>
   </xacro:if>
   <xacro:if value="${'$(arg type)' == 'chassis'}">
@@ -37,6 +39,6 @@
     </joint>
     <xacro:include filename="$(find zerith_h1_description)/xacro/components/arm.xacro"/>
-    <xacro:H1Arm name="left" direction="1"/>
-    <xacro:H1Arm name="right" direction="-1"/>
+    <xacro:H1Arm name="left" direction="1" camera="$(arg camera)"/>
+    <xacro:H1Arm name="right" direction="-1" camera="$(arg camera)"/>
   </xacro:if>
   <xacro:if value="${'$(arg type)' == 'left_arm'}">
@@ -47,5 +49,5 @@
     </joint>
     <xacro:include filename="$(find zerith_h1_description)/xacro/components/arm.xacro"/>
-    <xacro:H1Arm name="left" direction="1"/>
+    <xacro:H1Arm name="left" direction="1" camera="$(arg camera)"/>
   </xacro:if>
   <xacro:if value="${'$(arg type)' == 'right_arm'}">
@@ -56,5 +58,5 @@
     </joint>
     <xacro:include filename="$(find zerith_h1_description)/xacro/components/arm.xacro"/>
-    <xacro:H1Arm name="right" direction="-1"/>
+    <xacro:H1Arm name="right" direction="-1" camera="$(arg camera)"/>
   </xacro:if>
 </robot>

File: humanoid/Zerith/zerith_h1_description/xacro/components/arm.xacro (robot description, xacro)
@@ -6,6 +6,10 @@
 <!-- =================================================================================== -->
 <robot name="zerith_h1_arm" xmlns:xacro="http://www.ros.org/wiki/xacro">
-	<xacro:macro name="H1Arm" params="name direction:=1">
+	<xacro:include filename="$(find zerith_h1_description)/xacro/components/gripper.xacro"/>
+	<xacro:include filename="$(find zerith_h1_description)/xacro/components/camera.xacro"/>
+	<xacro:property name="PI" value="3.1415926535897931"/>
+	<xacro:macro name="H1Arm" params="name direction:=1 ee_type:='gripper' eef_fixed:=false camera:=d405">
 		<xacro:property name="prefix" value="${name}_"/>
+		<xacro:property name="hand_name" value="${name}_hand"/>
 		<!-- =============================================================================== -->
 		<!-- Shoulder Pitch                                                                  -->
@@ -182,10 +186,4 @@
 		<!-- =============================================================================== -->
 		<link name="${prefix}wrist_pitch_link">
-			<inertial>
-				<origin xyz="0.07825733 ${direction*0.00143511} 0.00315751"/>
-				<mass value="0.5139"/>
-				<inertia ixx="0.00046134" ixy="${direction*4.762e-05}" ixz="-1.314e-05"
-								 iyy="0.00044669" iyz="${direction*-5.2e-07}" izz="0.00060413"/>
-			</inertial>
 			<visual>
 				<geometry>
@@ -206,108 +204,51 @@
 			<limit lower="-1.0472" upper="1.0472" effort="9" velocity="16.747"/>
 		</joint>
-		<!-- =============================================================================== -->
-		<!-- Jaw Left Finger                                                                 -->
-		<!-- =============================================================================== -->
-		<link name="${prefix}jaw_left_finger_link">
-			<inertial>
-				<origin xyz="0.02875166 0.04972677 -0.00087113"/>
-				<mass value="0.057096"/>
-				<inertia ixx="1.643e-05" ixy="2.46e-06" ixz="1.89e-06"
-								 iyy="2.627e-05" iyz="4.7e-07" izz="2.05e-05"/>
-			</inertial>
-			<visual>
-				<geometry>
-					<mesh filename="file://$(find zerith_h1_description)/meshes/arm/finger.glb"/>
-				</geometry>
-			</visual>
-			<collision>
-				<geometry>
-					<mesh filename="file://$(find zerith_h1_description)/meshes/arm/finger.glb"/>
-				</geometry>
-			</collision>
-		</link>
-		<joint name="${prefix}gripper_joint" type="prismatic">
-			<origin xyz="0.102 0 0"/>
+		<link name="${prefix}tcp"/>
+		<joint name="${prefix}tcp_joint" type="fixed">
+			<origin xyz="0.046 0 0"/>
 			<parent link="${prefix}wrist_pitch_link"/>
-			<child link="${prefix}jaw_left_finger_link"/>
-			<axis xyz="0 1 0"/>
-			<limit lower="-0.04" upper="0" effort="120" velocity="0.25"/>
-		</joint>
-		<!-- =============================================================================== -->
-		<!-- Jaw Right Finger                                                                -->
-		<!-- =============================================================================== -->
-		<link name="${prefix}jaw_right_finger_link">
-			<inertial>
-				<origin xyz="0.02884254 -0.05065805 -0.00142222"/>
-				<mass value="0.057987"/>
-				<inertia ixx="1.518e-05" ixy="-3.71e-06" ixz="1.14e-06"
-								 iyy="2.561e-05" iyz="3.1e-07" izz="1.872e-05"/>
-			</inertial>
-			<visual>
-				<geometry>
-					<mesh filename="file://$(find zerith_h1_description)/meshes/arm/finger.glb" scale="1 -1 1"/>
-				</geometry>
-			</visual>
-			<collision>
-				<geometry>
-					<mesh filename="file://$(find zerith_h1_description)/meshes/arm/finger.glb" scale="1 -1 1"/>
-				</geometry>
-			</collision>
-		</link>
-		<joint name="${prefix}jaw_right_finger_joint" type="prismatic">
-			<origin xyz="0.102 0 0"/>
-			<parent link="${prefix}wrist_pitch_link"/>
-			<child link="${prefix}jaw_right_finger_link"/>
-			<axis xyz="0 1 0"/>
-			<mimic joint="${prefix}gripper_joint" multiplier="1" offset="0"/>
-			<limit lower="0" upper="0.04" effort="120" velocity="0.25"/>
-		</joint>
-		<!-- =============================================================================== -->
-		<!-- Jaw Camera                                                                      -->
-		<!-- =============================================================================== -->
-		<link name="${prefix}jaw_camera_link">
-			<inertial>
-				<origin xyz="0.0 0.005 -0.01561719"/>
-				<mass value="0.05789"/>
-				<inertia ixx="1.081e-05" ixy="-0.0" ixz="-0.0"
-								 iyy="1.08e-05" iyz="-0.0" izz="1.658e-05"/>
-			</inertial>
-			<visual>
-				<geometry>
-					<mesh filename="file://$(find sensor_models)/meshes/realsense/d405.glb"/>
-				</geometry>
-			</visual>
-		</link>
-		<joint name="${prefix}jaw_camera_joint" type="fixed">
-			<origin xyz="0.12275 0.000 0.05878" rpy="-2.0071 0 -1.5708"/>
-			<parent link="${prefix}wrist_pitch_link"/>
-			<child link="${prefix}jaw_camera_link"/>
-		</joint>
-		<!-- =============================================================================== -->
-		<!-- End Effector                                                                    -->
-		<!-- =============================================================================== -->
-		<link name="${prefix}end_effector_link">
-			<inertial>
-				<origin xyz="-0.027172 -5.6108E-09 1.2941E-06"/>
-				<mass value="0.0066601"/>
-				<inertia ixx="1.2345E-05" ixy="-7.5727E-14" ixz="2.3275E-11"
-								 iyy="6.5495E-08" iyz="-8.2193E-15" izz="1.232E-05"/>
-			</inertial>
-			<visual>
-				<geometry>
-					<mesh filename="file://$(find zerith_h1_description)/meshes/arm/eef.glb"/>
-				</geometry>
-			</visual>
-			<collision>
-				<geometry>
-					<mesh filename="file://$(find zerith_h1_description)/meshes/arm/eef.glb"/>
-				</geometry>
-			</collision>
-		</link>
-		<joint name="${prefix}end_effector_joint" type="fixed">
-			<origin xyz="0.1435 0 0"/>
-			<parent link="${prefix}wrist_pitch_link"/>
-			<child link="${prefix}end_effector_link"/>
-		</joint>
+			<child link="${prefix}tcp"/>
+		</joint>
+		<xacro:H1WristCamera prefix="${prefix}" parent_link="${prefix}tcp" camera="${camera}"/>
+		<xacro:if value="${ee_type == 'gripper'}">
+			<xacro:H1Gripper name="${name}" direction="${direction}" parent_link="${prefix}tcp"/>
+		</xacro:if>
+		<xacro:if value="${ee_type == 'none'}">
+			<link name="${prefix}eef"/>
+			<joint name="${prefix}eef_joint" type="fixed">
+				<parent link="${prefix}tcp"/>
+				<child link="${prefix}eef"/>
+			</joint>
+		</xacro:if>
+		<xacro:if value="${ee_type == 'revo1'}">
+			<xacro:BrainCoHand name="${hand_name}" direction="${direction}" fixed_joints="${eef_fixed}"/>
+			<joint name="${hand_name}_base_joint" type="fixed">
+				<!-- Fingers along wrist +X; palm inward (left -Y, right +Y). Native Revo1: fingers +Y, palm +Z. -->
+				<origin rpy="${direction * PI/2} ${direction * PI/2} 0"/>
+				<parent link="${prefix}tcp"/>
+				<child link="${hand_name}_hand_base"/>
+			</joint>
+			<link name="${prefix}eef"/>
+			<joint name="${prefix}eef_joint" type="fixed">
+				<origin xyz="0.0975 0 0"/>
+				<parent link="${prefix}tcp"/>
+				<child link="${prefix}eef"/>
+			</joint>
+		</xacro:if>
+		<xacro:if value="${ee_type == 'revo2'}">
+			<xacro:BrainCoHand name="${hand_name}" direction="${direction}" use_flange="true" fixed_joints="${eef_fixed}"/>
+			<joint name="${hand_name}_base_joint" type="fixed">
+				<!-- tcp is 0.046 from wrist; flange_joint adds 0.0176; 0.0024 keeps hand_base 0.066 from wrist. -->
+				<origin xyz="0.0024 0 0"/>
+				<parent link="${prefix}tcp"/>
+				<child link="${hand_name}_flange"/>
+			</joint>
+			<link name="${prefix}eef"/>
+			<joint name="${prefix}eef_joint" type="fixed">
+				<origin xyz="0.0975 0 0"/>
+				<parent link="${prefix}tcp"/>
+				<child link="${prefix}eef"/>
+			</joint>
+		</xacro:if>
 	</xacro:macro>
 </robot>

File: humanoid/Zerith/zerith_h1_description/xacro/components/body.xacro (robot description, xacro)
@@ -7,4 +7,5 @@
 <!-- =================================================================================== -->
 <robot name="zerith_h1_body" xmlns:xacro="http://www.ros.org/wiki/xacro">
+	<xacro:arg name="isaac" default="false"/>
 	<!-- =================================================================================== -->
 	<!-- Torso                                                                               -->
@@ -152,9 +153,11 @@
 	</joint>
 	<link name="head_camera">
-		<visual>
-			<geometry>
-				<mesh filename="file://$(find sensor_models)/meshes/realsense/d435.glb"/>
-			</geometry>
-		</visual>
+		<xacro:unless value="$(arg isaac)">
+			<visual>
+				<geometry>
+					<mesh filename="file://$(find sensor_models)/meshes/realsense/d435.glb"/>
+				</geometry>
+			</visual>
+		</xacro:unless>
 	</link>
 	<joint name="head_camera_joint" type="fixed">

File: humanoid/Zerith/zerith_h1_description/xacro/robot.xacro (robot description, xacro)
@@ -2,14 +2,31 @@
 <!-- =================================================================================== -->
 <!-- |    Complete Robot Description for Zerith H1                                     | -->
-<!-- |    Chassis (wheels locked by default) + body/head + dual 7-DOF arms + grippers  | -->
+<!-- |    Chassis (wheels locked by default) + body/head + dual 7-DOF arms             | -->
+<!-- |    type: empty/gripper (default) | none | revo1 | revo2                         | -->
+<!-- |    camera: empty→d405 on gripper, none otherwise | d405 | none                 | -->
 <!-- =================================================================================== -->
 <robot name="zerith_h1" xmlns:xacro="http://www.ros.org/wiki/xacro">
 	<!-- Lock drive wheels by default (W2/Bot2/Quanta/Galaxea). Planning URDF keeps this false. -->
 	<xacro:arg name="chassis_joints_movable" default="false"/>
+	<xacro:arg name="isaac" default="false"/>
+	<xacro:arg name="type" default=""/>
+	<xacro:arg name="camera" default=""/>
+	<xacro:arg name="eef_fixed_joints" default="false"/>
+	<xacro:property name="ee_type" value="${'$(arg type)' if '$(arg type)' else 'gripper'}"/>
+	<xacro:property name="camera_type"
+									value="${'$(arg camera)' if '$(arg camera)' else ('d405' if ee_type == 'gripper' else 'none')}"/>
+	<xacro:property name="eef_fixed"
+									value="${'$(arg eef_fixed_joints)'.lower() in ['1', 'true', 'yes', 'on']}"/>
 	<xacro:include filename="$(find zerith_h1_description)/xacro/components/chassis.xacro"/>
 	<xacro:H1Chassis joints_movable="$(arg chassis_joints_movable)"/>
 	<xacro:include filename="$(find zerith_h1_description)/xacro/components/body.xacro"/>
+	<xacro:if value="${ee_type == 'revo1'}">
+		<xacro:include filename="$(find brainco_description)/xacro/revo1.xacro"/>
+	</xacro:if>
+	<xacro:if value="${ee_type == 'revo2'}">
+		<xacro:include filename="$(find brainco_description)/xacro/revo2.xacro"/>
+	</xacro:if>
 	<xacro:include filename="$(find zerith_h1_description)/xacro/components/arm.xacro"/>
-	<xacro:H1Arm name="left" direction="1"/>
-	<xacro:H1Arm name="right" direction="-1"/>
+	<xacro:H1Arm name="left" direction="1" ee_type="${ee_type}" eef_fixed="${eef_fixed}" camera="${camera_type}"/>
+	<xacro:H1Arm name="right" direction="-1" ee_type="${ee_type}" eef_fixed="${eef_fixed}" camera="${camera_type}"/>
 </robot>

File: humanoid/Zerith/zerith_h1_description/xacro/ros2_control/arm_ros2_control.xacro (robot description, xacro)
@@ -20,5 +20,5 @@
     </joint>
   </xacro:macro>
-  <xacro:macro name="zerith_h1_arm_interfaces" params="name iface_mode:=mix">
+  <xacro:macro name="zerith_h1_arm_interfaces" params="name iface_mode:=mix ee_type:='gripper'">
     <xacro:property name="prefix" value="${name + '_' if name else ''}"/>
     <xacro:zerith_h1_arm_joint jname="${prefix}joint1" iface_mode="${iface_mode}"/>
@@ -29,13 +29,15 @@
     <xacro:zerith_h1_arm_joint jname="${prefix}joint6" iface_mode="${iface_mode}"/>
     <xacro:zerith_h1_arm_joint jname="${prefix}joint7" iface_mode="${iface_mode}"/>
-    <!-- AdaptiveGripperController drives ${prefix}gripper_joint (mimic finger follows). -->
-    <joint name="${prefix}gripper_joint">
-      <command_interface name="position"/>
-      <state_interface name="position"/>
-      <xacro:if value="${iface_mode == 'mix'}">
-        <state_interface name="velocity"/>
-        <state_interface name="effort"/>
-      </xacro:if>
-    </joint>
+    <xacro:if value="${ee_type == 'gripper'}">
+      <!-- AdaptiveGripperController drives ${prefix}gripper_joint (mimic finger follows). -->
+      <joint name="${prefix}gripper_joint">
+        <command_interface name="position"/>
+        <state_interface name="position"/>
+        <xacro:if value="${iface_mode == 'mix'}">
+          <state_interface name="velocity"/>
+          <state_interface name="effort"/>
+        </xacro:if>
+      </joint>
+    </xacro:if>
   </xacro:macro>
 </robot>

File: humanoid/Zerith/zerith_h1_description/xacro/ros2_control/robot.xacro (robot description, xacro)
@@ -29,6 +29,16 @@
     </hardware>
     <xacro:zerith_h1_body_interfaces iface_mode="${sim_iface_mode}"/>
-    <xacro:zerith_h1_arm_interfaces name="left" iface_mode="${sim_iface_mode}"/>
-    <xacro:zerith_h1_arm_interfaces name="right" iface_mode="${sim_iface_mode}"/>
+    <xacro:zerith_h1_arm_interfaces name="left" iface_mode="${sim_iface_mode}" ee_type="${ee_type}"/>
+    <xacro:zerith_h1_arm_interfaces name="right" iface_mode="${sim_iface_mode}" ee_type="${ee_type}"/>
+    <xacro:if value="${ee_type == 'revo1'}">
+      <xacro:include filename="$(find brainco_description)/xacro/ros2_control/revo1.xacro"/>
+      <xacro:revo1_interfaces name="left_hand"/>
+      <xacro:revo1_interfaces name="right_hand"/>
+    </xacro:if>
+    <xacro:if value="${ee_type == 'revo2'}">
+      <xacro:include filename="$(find brainco_description)/xacro/ros2_control/revo2.xacro"/>
+      <xacro:revo2_interfaces name="left_hand"/>
+      <xacro:revo2_interfaces name="right_hand"/>
+    </xacro:if>
   </ros2_control>
   <xacro:if value="$(arg gazebo)">
