Commit message: update zerith h1

File: humanoid/Zerith/zerith_h1_description/xacro/component.xacro (robot description, xacro)
@@ -14,4 +14,5 @@
   <xacro:arg name="isaac" default="false"/>
   <xacro:arg name="camera" default="d405"/>
+  <xacro:arg name="collider" default="simple"/>
   <xacro:if value="${'$(arg type)' != 'base' and '$(arg type)' != 'chassis'}">
     <link name="base_link"/>
@@ -21,11 +22,11 @@
     <xacro:include filename="$(find zerith_h1_description)/xacro/components/body.xacro"/>
     <xacro:include filename="$(find zerith_h1_description)/xacro/components/arm.xacro"/>
-    <xacro:H1Chassis joints_movable="$(arg chassis_joints_movable)"/>
-    <xacro:H1Arm name="left" direction="1" camera="$(arg camera)"/>
-    <xacro:H1Arm name="right" direction="-1" camera="$(arg camera)"/>
+    <xacro:H1Chassis joints_movable="$(arg chassis_joints_movable)" collider="$(arg collider)"/>
+    <xacro:H1Arm name="left" direction="1" camera="$(arg camera)" collider="$(arg collider)"/>
+    <xacro:H1Arm name="right" direction="-1" camera="$(arg camera)" collider="$(arg collider)"/>
   </xacro:if>
   <xacro:if value="${'$(arg type)' == 'chassis'}">
     <xacro:include filename="$(find zerith_h1_description)/xacro/components/chassis.xacro"/>
-    <xacro:H1Chassis joints_movable="true"/>
+    <xacro:H1Chassis joints_movable="true" collider="$(arg collider)"/>
   </xacro:if>
   <xacro:if value="${'$(arg type)' == 'body'}">
@@ -39,6 +40,6 @@
     </joint>
     <xacro:include filename="$(find zerith_h1_description)/xacro/components/arm.xacro"/>
-    <xacro:H1Arm name="left" direction="1" camera="$(arg camera)"/>
-    <xacro:H1Arm name="right" direction="-1" camera="$(arg camera)"/>
+    <xacro:H1Arm name="left" direction="1" camera="$(arg camera)" collider="$(arg collider)"/>
+    <xacro:H1Arm name="right" direction="-1" camera="$(arg camera)" collider="$(arg collider)"/>
   </xacro:if>
   <xacro:if value="${'$(arg type)' == 'left_arm'}">
@@ -49,5 +50,5 @@
     </joint>
     <xacro:include filename="$(find zerith_h1_description)/xacro/components/arm.xacro"/>
-    <xacro:H1Arm name="left" direction="1" camera="$(arg camera)"/>
+    <xacro:H1Arm name="left" direction="1" camera="$(arg camera)" collider="$(arg collider)"/>
   </xacro:if>
   <xacro:if value="${'$(arg type)' == 'right_arm'}">
@@ -58,5 +59,5 @@
     </joint>
     <xacro:include filename="$(find zerith_h1_description)/xacro/components/arm.xacro"/>
-    <xacro:H1Arm name="right" direction="-1" camera="$(arg camera)"/>
+    <xacro:H1Arm name="right" direction="-1" camera="$(arg camera)" collider="$(arg collider)"/>
   </xacro:if>
 </robot>

File: humanoid/Zerith/zerith_h1_description/xacro/components/arm.xacro (robot description, xacro)
@@ -9,5 +9,24 @@
 	<xacro:include filename="$(find zerith_h1_description)/xacro/components/camera.xacro"/>
 	<xacro:property name="PI" value="3.1415926535897931"/>
-	<xacro:macro name="H1Arm" params="name direction:=1 ee_type:='gripper' eef_fixed:=false camera:=d405">
+	<!-- collider:=simple: cylinders from glTF node-world AABB (split-chassis-glb §8).
+	     collider:=convex: same GLB as visual. Y of mirrored meshes follows direction. -->
+	<xacro:macro name="h1_arm_link_collision" params="collider mesh xyz:='0 0 0' rpy:='0 0 0' length radius scale:='1 1 1'">
+		<xacro:if value="${collider == 'convex'}">
+			<collision>
+				<geometry>
+					<mesh filename="${mesh}" scale="${scale}"/>
+				</geometry>
+			</collision>
+		</xacro:if>
+		<xacro:if value="${collider == 'simple'}">
+			<collision>
+				<origin xyz="${xyz}" rpy="${rpy}"/>
+				<geometry>
+					<cylinder length="${length}" radius="${radius}"/>
+				</geometry>
+			</collision>
+		</xacro:if>
+	</xacro:macro>
+	<xacro:macro name="H1Arm" params="name direction:=1 ee_type:='gripper' eef_fixed:=false camera:=d405 collider:='simple'">
 		<xacro:property name="prefix" value="${name}_"/>
 		<xacro:property name="hand_name" value="${name}_hand"/>
@@ -27,9 +46,12 @@
 				</geometry>
 			</visual>
-			<collision>
-				<geometry>
-					<mesh filename="file://$(find zerith_h1_description)/meshes/arm/link1.glb" scale="1 ${direction} 1"/>
-				</geometry>
-			</collision>
+			<!-- Shoulder pitch sits on the torso; no simple collider. -->
+			<xacro:if value="${collider == 'convex'}">
+				<collision>
+					<geometry>
+						<mesh filename="file://$(find zerith_h1_description)/meshes/arm/link1.glb" scale="1 ${direction} 1"/>
+					</geometry>
+				</collision>
+			</xacro:if>
 		</link>
 		<joint name="${prefix}joint1" type="revolute">
@@ -55,9 +77,10 @@
 				</geometry>
 			</visual>
-			<collision>
-				<geometry>
-					<mesh filename="file://$(find zerith_h1_description)/meshes/arm/link2.glb" scale="1 ${direction} 1"/>
-				</geometry>
-			</collision>
+			<!-- link2: cylinder along -Z toward joint3. Radius hugs the tube, not the housing. -->
+			<xacro:h1_arm_link_collision collider="${collider}"
+				mesh="file://$(find zerith_h1_description)/meshes/arm/link2.glb"
+				scale="1 ${direction} 1"
+				xyz="0 ${direction * 0.0068} -0.0435"
+				length="0.1711" radius="0.050"/>
 		</link>
 		<joint name="${prefix}joint2" type="revolute">
@@ -85,9 +108,9 @@
 				</geometry>
 			</visual>
-			<collision>
-				<geometry>
-					<mesh filename="file://$(find zerith_h1_description)/meshes/arm/link3.glb"/>
-				</geometry>
-			</collision>
+			<!-- link3: cylinder toward joint4 (mostly -Z, +X). Radius hugs the tube. -->
+			<xacro:h1_arm_link_collision collider="${collider}"
+				mesh="file://$(find zerith_h1_description)/meshes/arm/link3.glb"
+				xyz="0.0197 0 -0.1008" rpy="0 2.895 0"
+				length="0.2164" radius="0.038"/>
 		</link>
 		<joint name="${prefix}joint3" type="revolute">
@@ -113,9 +136,10 @@
 				</geometry>
 			</visual>
-			<collision>
-				<geometry>
-					<mesh filename="file://$(find zerith_h1_description)/meshes/arm/link4.glb" scale="1 ${direction} 1"/>
-				</geometry>
-			</collision>
+			<!-- link4: axis X. Radius hugs the elbow tube so the end cap stays inside the joint. -->
+			<xacro:h1_arm_link_collision collider="${collider}"
+				mesh="file://$(find zerith_h1_description)/meshes/arm/link4.glb"
+				scale="1 ${direction} 1"
+				xyz="0.0301 0 -0.0247" rpy="0 ${PI/2} 0"
+				length="0.1297" radius="0.042"/>
 		</link>
 		<joint name="${prefix}joint4" type="revolute">
@@ -141,9 +165,10 @@
 				</geometry>
 			</visual>
-			<collision>
-				<geometry>
-					<mesh filename="file://$(find zerith_h1_description)/meshes/arm/link5.glb" scale="1 ${direction} 1"/>
-				</geometry>
-			</collision>
+			<!-- link5: axis X. Radius hugs the forearm tube. -->
+			<xacro:h1_arm_link_collision collider="${collider}"
+				mesh="file://$(find zerith_h1_description)/meshes/arm/link5.glb"
+				scale="1 ${direction} 1"
+				xyz="0.0968 0 -0.0026" rpy="0 ${PI/2} 0"
+				length="0.1561" radius="0.036"/>
 		</link>
 		<joint name="${prefix}joint5" type="revolute">
@@ -169,9 +194,10 @@
 				</geometry>
 			</visual>
-			<collision>
-				<geometry>
-					<mesh filename="file://$(find zerith_h1_description)/meshes/arm/link6.glb" scale="1 ${direction} 1"/>
-				</geometry>
-			</collision>
+			<!-- link6 AABB: axis Z, L=0.0713 r=0.0308. -->
+			<xacro:h1_arm_link_collision collider="${collider}"
+				mesh="file://$(find zerith_h1_description)/meshes/arm/link6.glb"
+				scale="1 ${direction} 1"
+				xyz="0 ${direction * -0.0003} -0.0003"
+				length="0.0713" radius="0.0308"/>
 		</link>
 		<joint name="${prefix}joint6" type="revolute">
@@ -191,9 +217,10 @@
 				</geometry>
 			</visual>
-			<collision>
-				<geometry>
-					<mesh filename="file://$(find zerith_h1_description)/meshes/arm/link7.glb"  scale="1 ${direction} 1"/>
-				</geometry>
-			</collision>
+			<!-- link7 AABB: axis X, L=0.0725 r=0.0253; y mirrored with the mesh. -->
+			<xacro:h1_arm_link_collision collider="${collider}"
+				mesh="file://$(find zerith_h1_description)/meshes/arm/link7.glb"
+				scale="1 ${direction} 1"
+				xyz="0.0168 ${direction * 0.0093} 0" rpy="0 ${PI/2} 0"
+				length="0.0725" radius="0.0253"/>
 		</link>
 		<joint name="${prefix}joint7" type="revolute">

File: humanoid/Zerith/zerith_h1_description/xacro/components/body.xacro (robot description, xacro)
@@ -8,4 +8,32 @@
 <robot name="zerith_h1_body" xmlns:xacro="http://www.ros.org/wiki/xacro">
 	<xacro:arg name="isaac" default="false"/>
+	<xacro:arg name="collider" default="simple"/>
+	<!-- collider:=simple: box, or a vertical cylinder when radius is set.
+	     collider:=convex: same GLB as visual. Head stays mesh (not in selfCollision). -->
+	<xacro:macro name="h1_body_collision" params="collider mesh xyz:='0 0 0' size:='0 0 0' length:='0' radius:='0'">
+		<xacro:if value="${collider == 'convex'}">
+			<collision>
+				<geometry>
+					<mesh filename="${mesh}"/>
+				</geometry>
+			</collision>
+		</xacro:if>
+		<xacro:if value="${collider == 'simple' and radius == '0'}">
+			<collision>
+				<origin xyz="${xyz}"/>
+				<geometry>
+					<box size="${size}"/>
+				</geometry>
+			</collision>
+		</xacro:if>
+		<xacro:if value="${collider == 'simple' and radius != '0'}">
+			<collision>
+				<origin xyz="${xyz}"/>
+				<geometry>
+					<cylinder length="${length}" radius="${radius}"/>
+				</geometry>
+			</collision>
+		</xacro:if>
+	</xacro:macro>
 	<!-- =================================================================================== -->
 	<!-- Torso                                                                               -->
@@ -23,9 +51,7 @@
 			</geometry>
 		</visual>
-		<collision>
-			<geometry>
-				<mesh filename="file://$(find zerith_h1_description)/meshes/body/body_link1.glb"/>
-			</geometry>
-		</collision>
+		<xacro:h1_body_collision collider="$(arg collider)"
+			mesh="file://$(find zerith_h1_description)/meshes/body/body_link1.glb"
+			xyz="0.105 0 0.127" size="0.180 0.125 0.135"/>
 	</link>
 	<joint name="body_joint1" type="prismatic">
@@ -47,9 +73,8 @@
 			</geometry>
 		</visual>
-		<collision>
-			<geometry>
-				<mesh filename="file://$(find zerith_h1_description)/meshes/body/body_link2.glb"/>
-			</geometry>
-		</collision>
+		<!-- Waist: vertical cylinder inside the shell (was a 0.155 m wide box). -->
+		<xacro:h1_body_collision collider="$(arg collider)"
+			mesh="file://$(find zerith_h1_description)/meshes/body/body_link2.glb"
+			xyz="0 0 0.020" length="0.125" radius="0.070"/>
 	</link>
 	<joint name="body_joint2" type="revolute">
@@ -72,9 +97,8 @@
 			</geometry>
 		</visual>
-		<collision>
-			<geometry>
-				<mesh filename="file://$(find zerith_h1_description)/meshes/body/body_link3.glb"/>
-			</geometry>
-		</collision>
+		<!-- Chest: vertical cylinder. Diameter 0.17 m, inside the 0.21 m shoulder box. -->
+		<xacro:h1_body_collision collider="$(arg collider)"
+			mesh="file://$(find zerith_h1_description)/meshes/body/body_link3.glb"
+			xyz="0 0 0.140" length="0.240" radius="0.085"/>
 	</link>
 	<joint name="body_joint3" type="revolute">

File: humanoid/Zerith/zerith_h1_description/xacro/components/chassis.xacro (robot description, xacro)
@@ -5,4 +5,5 @@
 <!-- =================================================================================== -->
 <robot name="zerith_h1_chassis" xmlns:xacro="http://www.ros.org/wiki/xacro">
+	<xacro:arg name="collider" default="simple"/>
 	<!-- Passive support caster (Quanta X1 swivel / Realman RS01 caster convention):
 	     base_link -> {prefix}_caster_swivel_joint (yaw, axis Z, vertical through the mount)
@@ -53,7 +54,13 @@
 	</xacro:macro>
 	<!-- joints_movable:=false → drive wheels + casters fixed (W2/Bot2/Quanta). -->
-	<xacro:macro name="H1Chassis" params="joints_movable:=false">
+	<xacro:macro name="H1Chassis" params="joints_movable:=false collider:='simple'">
 		<xacro:property name="chassis_movable" value="${str(joints_movable).lower() in ['true', '1', 'yes', 'on']}"/>
 		<xacro:property name="wheel_joint_type" value="${'continuous' if chassis_movable else 'fixed'}"/>
+		<!-- Root frames: base_footprint identity to base_link (W2 / Taku / Bot2). -->
+		<link name="base_footprint"/>
+		<joint name="base_footprint_joint" type="fixed">
+			<parent link="base_footprint"/>
+			<child link="base_link"/>
+		</joint>
 		<link name="base_link">
 			<inertial>
@@ -68,9 +75,27 @@
 				</geometry>
 			</visual>
-			<collision>
-				<geometry>
-					<mesh filename="file://$(find zerith_h1_description)/meshes/base/base_link.glb"/>
-				</geometry>
-			</collision>
+			<xacro:if value="${collider == 'convex'}">
+				<collision>
+					<geometry>
+						<mesh filename="file://$(find zerith_h1_description)/meshes/base/base_link.glb"/>
+					</geometry>
+				</collision>
+			</xacro:if>
+			<xacro:if value="${collider == 'simple'}">
+				<!-- Deck. Wheels keep their own cylinders. -->
+				<collision>
+					<origin xyz="0.05 0 -0.06"/>
+					<geometry>
+						<box size="0.56 0.40 0.16"/>
+					</geometry>
+				</collision>
+				<!-- Rear mast: shell is about 0.20 x 0.21 from z 0.14 to 1.14. Inset so it sits inside the housing. -->
+				<collision>
+					<origin xyz="-0.076 0 0.64"/>
+					<geometry>
+						<box size="0.150 0.155 0.90"/>
+					</geometry>
+				</collision>
+			</xacro:if>
 		</link>
 		<xacro:H1Caster prefix="left_front" x="0.184" y="0.148" mass="0.16" ixx="6.766e-05" iyy="7.514e-05" izz="6.766e-05" movable="${chassis_movable}"/>

File: humanoid/Zerith/zerith_h1_description/xacro/robot.xacro (robot description, xacro)
@@ -10,4 +10,5 @@
 	<xacro:arg name="chassis_joints_movable" default="false"/>
 	<xacro:arg name="isaac" default="false"/>
+	<xacro:arg name="collider" default="simple"/>
 	<xacro:arg name="type" default=""/>
 	<xacro:arg name="camera" default=""/>
@@ -19,5 +20,5 @@
 									value="${'$(arg eef_fixed_joints)'.lower() in ['1', 'true', 'yes', 'on']}"/>
 	<xacro:include filename="$(find zerith_h1_description)/xacro/components/chassis.xacro"/>
-	<xacro:H1Chassis joints_movable="$(arg chassis_joints_movable)"/>
+	<xacro:H1Chassis joints_movable="$(arg chassis_joints_movable)" collider="$(arg collider)"/>
 	<xacro:include filename="$(find zerith_h1_description)/xacro/components/body.xacro"/>
 	<xacro:if value="${ee_type == 'revo1'}">
@@ -28,5 +29,5 @@
 	</xacro:if>
 	<xacro:include filename="$(find zerith_h1_description)/xacro/components/arm.xacro"/>
-	<xacro:H1Arm name="left" direction="1" ee_type="${ee_type}" eef_fixed="${eef_fixed}" camera="${camera_type}"/>
-	<xacro:H1Arm name="right" direction="-1" ee_type="${ee_type}" eef_fixed="${eef_fixed}" camera="${camera_type}"/>
+	<xacro:H1Arm name="left" direction="1" ee_type="${ee_type}" eef_fixed="${eef_fixed}" camera="${camera_type}" collider="$(arg collider)"/>
+	<xacro:H1Arm name="right" direction="-1" ee_type="${ee_type}" eef_fixed="${eef_fixed}" camera="${camera_type}" collider="$(arg collider)"/>
 </robot>
