Commit message: 已完成nero_description所有配置

File: manipulator/AgileX/nero_description/urdf/nero.urdf (robot description, URDF)
Before this commit: robot nero, 11 links, 10 joints
Links:
- removed link right_base_link
- removed link right_link1
- removed link right_link2
- removed link right_link3
- removed link right_link4
- removed link right_link5
- removed link right_link6
- removed link right_link7
- removed link right_stand_adapter
- added link left_base_link, mass 0.77; collision mesh filename=file:///home/shiman-liang/ros2_ws/install/nero_description/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; visual mesh filename=file:///home/shiman-liang/ros2_ws/install/nero_description/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
- added link left_link1, mass 0.77; collision mesh filename=file:///home/shiman-liang/ros2_ws/install/nero_description/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; visual mesh filename=file:///home/shiman-liang/ros2_ws/install/nero_description/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
- added link left_link2, mass 0.49; collision mesh filename=file:///home/shiman-liang/ros2_ws/install/nero_description/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; visual mesh filename=file:///home/shiman-liang/ros2_ws/install/nero_description/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
- added link left_link3, mass 0.67; collision mesh filename=file:///home/shiman-liang/ros2_ws/install/nero_description/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; visual mesh filename=file:///home/shiman-liang/ros2_ws/install/nero_description/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
- added link left_link4, mass 0.41; collision mesh filename=file:///home/shiman-liang/ros2_ws/install/nero_description/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; visual mesh filename=file:///home/shiman-liang/ros2_ws/install/nero_description/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
- added link left_link5, mass 0.56; collision mesh filename=file:///home/shiman-liang/ros2_ws/install/nero_description/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; visual mesh filename=file:///home/shiman-liang/ros2_ws/install/nero_description/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
- added link left_link6, mass 0.31; collision mesh filename=file:///home/shiman-liang/ros2_ws/install/nero_description/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; visual mesh filename=file:///home/shiman-liang/ros2_ws/install/nero_description/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
- added link left_link7, mass 0.000001; collision mesh filename=file:///home/shiman-liang/ros2_ws/install/nero_description/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; visual mesh filename=file:///home/shiman-liang/ros2_ws/install/nero_description/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
Joints:
- removed joint right_base_joint
- removed joint right_joint1
- removed joint right_joint2
- removed joint right_joint3
- removed joint right_joint4
- removed joint right_joint5
- removed joint right_joint6
- removed joint right_joint7
- removed joint right_stand_joint
- added joint left_base_joint: type fixed, parent base_link, child left_base_link, origin xyz=0 0 0 rpy=0 0 3.14159
- added joint left_joint1: type revolute, parent left_base_link, child left_link1, origin xyz=0 0 0.138 rpy=0 0 0, axis 0 0 1, limit lower=-2.7 upper=2.7 effort=0 velocity=0
- added joint left_joint2: type revolute, parent left_link1, child left_link2, origin xyz=0 0 0 rpy=1.5708 3.1415 0, axis 0 0 1, limit lower=-1.74 upper=1.74 effort=0 velocity=0
- added joint left_joint3: type revolute, parent left_link2, child left_link3, origin xyz=0 -0.31 0 rpy=-1.5708 0 3.1416, axis 0 0 1, limit lower=-2.75 upper=2.75 effort=0 velocity=0
- added joint left_joint4: type revolute, parent left_link3, child left_link4, origin xyz=0 0 0 rpy=-1.5708 0 3.1416, axis 0 0 1, limit lower=-1.01 upper=2.14 effort=0 velocity=0
- added joint left_joint5: type revolute, parent left_link4, child left_link5, origin xyz=0 -0.27001 0 rpy=1.5708 -1.5708 0, axis 0 0 1, limit lower=-2.75 upper=2.75 effort=0 velocity=0
- added joint left_joint6: type revolute, parent left_link5, child left_link6, origin xyz=0 0 0 rpy=1.5708 -1.5708 0, axis 0 0 1, limit lower=-0.73 upper=0.95 effort=0 velocity=0
- added joint left_joint7: type revolute, parent left_link6, child left_link7, origin xyz=0 -0.0235 0 rpy=1.5708 0 0, axis 0 0 1, limit lower=-1.57 upper=1.57 effort=0 velocity=0

File: manipulator/AgileX/nero_description/xacro/hand.xacro (robot description, xacro)
@@ -1,46 +1,42 @@
 <?xml version="1.0" encoding="utf-8"?>
 <robot xmlns:xacro="http://www.ros.org/wiki/xacro">
-    <xacro:include filename="$(find revo2_description)/xacro/revo_hand.xacro"/>
-    <xacro:macro name="Hand" params="type stand direction prefix">
+    <xacro:macro name="Hand" params="type stand direction prefix standalone:=false">
         <xacro:property name="actual_stand" value="${type if type != 'hand' else stand}"/>
         <xacro:property name="stand_link_name" value="${prefix}stand_adapter"/>
+        <xacro:property name="stand_origin_rpy" value="0 0 0"/>
+        <xacro:if value="${actual_stand == 'v1'}">
+            <xacro:property name="stand_origin_rpy" value="-1.57 -1.57 -1.57"/>
+        </xacro:if>
+        <xacro:if value="${actual_stand == 'v2'}">
+            <xacro:property name="stand_origin_rpy" value="-1.57 0 -1.57"/>
+        </xacro:if>
         <link name="${stand_link_name}">
             <visual>
-                <xacro:if value="${actual_stand == 'v1'}">
-                    <origin xyz="0 0 0" rpy="-1.57 -1.57 -1.57"/>
-                    <geometry>
-                        <mesh filename="package://nero_description/meshes/stand_v1.glb"/>
-                    </geometry>
-                </xacro:if>
-                <xacro:if value="${actual_stand == 'v2'}">
-                    <origin xyz="0 0 0" rpy="-1.57 0 -1.57"/>
-                    <geometry>
-                        <mesh filename="package://nero_description/meshes/stand_v2.glb"/>
-                    </geometry>
-                </xacro:if>
-                <xacro:if value="${actual_stand == 'link8'}">
-                    <origin xyz="0 0 0" rpy="0 0 0"/>
-                    <geometry>
-                        <mesh filename="package://nero_description/meshes/link8.glb"/>
-                    </geometry>
-                </xacro:if>
+                <origin xyz="0 0 0" rpy="${stand_origin_rpy}"/>
+                <geometry>
+                    <mesh filename="file://$(find nero_description)/meshes/${actual_stand if actual_stand == 'link8' else 'stand_' + actual_stand}.glb"/>
+                </geometry>
             </visual>
             <collision>
+                <origin xyz="0 0 0" rpy="${stand_origin_rpy}"/>
                 <geometry>
-                    <mesh filename="package://nero_description/meshes/${'link8' if actual_stand == 'link8' else 'stand_v1'}.glb"/>
+                    <mesh filename="file://$(find nero_description)/meshes/${'link8' if actual_stand == 'link8' else 'stand_v1'}.glb"/>
                 </geometry>
             </collision>
         </link>
-        <joint name="${prefix}stand_joint" type="fixed">
-            <xacro:if value="${actual_stand == 'link8'}">
-                <origin xyz="0.032 0 -0.0235" rpy="-1.5708 0 -1.5708"/>
-            </xacro:if>
-            <xacro:unless value="${actual_stand == 'link8'}">
-                <origin xyz="0.033 0 -0.0235" rpy="0 0 0"/>
-            </xacro:unless>
-            <parent link="${prefix}link7"/>
-            <child link="${stand_link_name}"/>
-        </joint>
-        <xacro:if value="${type == 'hand'}">
+        <xacro:unless value="${standalone}">
+            <joint name="${prefix}stand_joint" type="fixed">
+                <xacro:if value="${actual_stand == 'link8'}">
+                    <origin xyz="0.032 0 -0.0235" rpy="-1.5708 0 -1.5708"/>
+                </xacro:if>
+                <xacro:unless value="${actual_stand == 'link8'}">
+                    <origin xyz="0.033 0 -0.0235" rpy="0 0 0"/>
+                </xacro:unless>
+                <parent link="${prefix}link7"/>
+                <child link="${stand_link_name}"/>
+            </joint>
+        </xacro:unless>
+        <xacro:if value="${type == 'hand' or type == 'v1' or type == 'v2'}">
+            <xacro:include filename="$(find revo2_description)/xacro/revo_hand.xacro"/>
             <joint name="${prefix}hand_connection_joint" type="fixed">
                 <origin xyz="0.01093 0 0" rpy="-1.57 3.14 -1.57"/>

File: manipulator/AgileX/nero_description/xacro/nero.xacro (robot description, xacro)
@@ -1,6 +1,9 @@
 <?xml version="1.0" encoding="utf-8"?>
 <robot xmlns:xacro="http://www.ros.org/wiki/xacro">
-    <xacro:macro name="Nero" params="type stand direction prefix">
-        <xacro:include filename="$(find nero_description)/xacro/hand.xacro"/>
+    <xacro:include filename="$(find nero_description)/xacro/hand.xacro"/>
+    <xacro:macro name="Nero" params="type stand direction prefix is_arm_only:=false">
+        <xacro:unless value="${is_arm_only}">
+            <xacro:Hand type="${type}" stand="${stand}" direction="${direction}" prefix="${prefix}"/>
+        </xacro:unless>
         <link name="${prefix}base_link">
             <inertial>
@@ -12,11 +15,11 @@
                 <origin xyz="0 0 0" rpy="0 0 0"/>
                 <geometry>
-                    <mesh filename="package://nero_description/meshes/base_link.glb"/>
-                </geometry>
-            </visual>
-            <collision>
-                <origin xyz="0 0 0" rpy="0 0 0"/>
-                <geometry>
-                    <mesh filename="package://nero_description/meshes/base_link.glb"/>
+                    <mesh filename="file://$(find nero_description)/meshes/base_link.glb"/>
+                </geometry>
+            </visual>
+            <collision>
+                <origin xyz="0 0 0" rpy="0 0 0"/>
+                <geometry>
+                    <mesh filename="file://$(find nero_description)/meshes/base_link.glb"/>
                 </geometry>
             </collision>
@@ -31,11 +34,11 @@
                 <origin xyz="0 0 0" rpy="0 0 0"/>
                 <geometry>
-                    <mesh filename="package://nero_description/meshes/link1.glb"/>
-                </geometry>
-            </visual>
-            <collision>
-                <origin xyz="0 0 0" rpy="0 0 0"/>
-                <geometry>
-                    <mesh filename="package://nero_description/meshes/link1.glb"/>
+                    <mesh filename="file://$(find nero_description)/meshes/link1.glb"/>
+                </geometry>
+            </visual>
+            <collision>
+                <origin xyz="0 0 0" rpy="0 0 0"/>
+                <geometry>
+                    <mesh filename="file://$(find nero_description)/meshes/link1.glb"/>
                 </geometry>
             </collision>
@@ -57,11 +60,11 @@
                 <origin xyz="0 0 0" rpy="0 0 0"/>
                 <geometry>
-                    <mesh filename="package://nero_description/meshes/link2.glb"/>
-                </geometry>
-            </visual>
-            <collision>
-                <origin xyz="0 0 0" rpy="0 0 0"/>
-                <geometry>
-                    <mesh filename="package://nero_description/meshes/link2.glb"/>
+                    <mesh filename="file://$(find nero_description)/meshes/link2.glb"/>
+                </geometry>
+            </visual>
+            <collision>
+                <origin xyz="0 0 0" rpy="0 0 0"/>
+                <geometry>
+                    <mesh filename="file://$(find nero_description)/meshes/link2.glb"/>
                 </geometry>
             </collision>
@@ -83,11 +86,11 @@
                 <origin xyz="0 0 0" rpy="0 0 0"/>
                 <geometry>
-                    <mesh filename="package://nero_description/meshes/link3.glb"/>
-                </geometry>
-            </visual>
-            <collision>
-                <origin xyz="0 0 0" rpy="0 0 0"/>
-                <geometry>
-                    <mesh filename="package://nero_description/meshes/link3.glb"/>
+                    <mesh filename="file://$(find nero_description)/meshes/link3.glb"/>
+                </geometry>
+            </visual>
+            <collision>
+                <origin xyz="0 0 0" rpy="0 0 0"/>
+                <geometry>
+                    <mesh filename="file://$(find nero_description)/meshes/link3.glb"/>
                 </geometry>
             </collision>
@@ -109,11 +112,11 @@
                 <origin xyz="0 0 0" rpy="0 0 0"/>
                 <geometry>
-                    <mesh filename="package://nero_description/meshes/link4.glb"/>
-                </geometry>
-            </visual>
-            <collision>
-                <origin xyz="0 0 0" rpy="0 0 0"/>
-                <geometry>
-                    <mesh filename="package://nero_description/meshes/link4.glb"/>
+                    <mesh filename="file://$(find nero_description)/meshes/link4.glb"/>
+                </geometry>
+            </visual>
+            <collision>
+                <origin xyz="0 0 0" rpy="0 0 0"/>
+                <geometry>
+                    <mesh filename="file://$(find nero_description)/meshes/link4.glb"/>
                 </geometry>
             </collision>
@@ -135,11 +138,11 @@
                 <origin xyz="0 0 0" rpy="0 0 0"/>
                 <geometry>
-                    <mesh filename="package://nero_description/meshes/link5.glb"/>
-                </geometry>
-            </visual>
-            <collision>
-                <origin xyz="0 0 0" rpy="0 0 0"/>
-                <geometry>
-                    <mesh filename="package://nero_description/meshes/link5.glb"/>
+                    <mesh filename="file://$(find nero_description)/meshes/link5.glb"/>
+                </geometry>
+            </visual>
+            <collision>
+                <origin xyz="0 0 0" rpy="0 0 0"/>
+                <geometry>
+                    <mesh filename="file://$(find nero_description)/meshes/link5.glb"/>
                 </geometry>
             </collision>
@@ -161,11 +164,11 @@
                 <origin xyz="0 0 0" rpy="0 0 0"/>
                 <geometry>
-                    <mesh filename="package://nero_description/meshes/link6.glb"/>
-                </geometry>
-            </visual>
-            <collision>
-                <origin xyz="0 0 0" rpy="0 0 0"/>
-                <geometry>
-                    <mesh filename="package://nero_description/meshes/link6.glb"/>
+                    <mesh filename="file://$(find nero_description)/meshes/link6.glb"/>
+                </geometry>
+            </visual>
+            <collision>
+                <origin xyz="0 0 0" rpy="0 0 0"/>
+                <geometry>
+                    <mesh filename="file://$(find nero_description)/meshes/link6.glb"/>
                 </geometry>
             </collision>
@@ -187,11 +190,11 @@
                 <origin xyz="0 0 0" rpy="0 0 0"/>
                 <geometry>
-                    <mesh filename="package://nero_description/meshes/link7.glb"/>
-                </geometry>
-            </visual>
-            <collision>
-                <origin xyz="0 0 0" rpy="0 0 0"/>
-                <geometry>
-                    <mesh filename="package://nero_description/meshes/link7.glb"/>
+                    <mesh filename="file://$(find nero_description)/meshes/link7.glb"/>
+                </geometry>
+            </visual>
+            <collision>
+                <origin xyz="0 0 0" rpy="0 0 0"/>
+                <geometry>
+                    <mesh filename="file://$(find nero_description)/meshes/link7.glb"/>
                 </geometry>
             </collision>
@@ -204,5 +207,4 @@
             <limit lower="-1.57" upper="1.57" effort="0" velocity="0"/>
         </joint>
-        <xacro:Hand type="${type}" stand="${stand}" direction="${direction}" prefix="${prefix}"/>
     </xacro:macro>
 </robot>

File: manipulator/AgileX/nero_description/xacro/robot.xacro (robot description, xacro)
@@ -1,24 +1,43 @@
 <?xml version="1.0"?>
-<robot name="nero" xmlns:xacro="http://www.ros.org/wiki/xacro">
+<robot name="Nero" xmlns:xacro="http://www.ros.org/wiki/xacro">
     <xacro:arg name="type" default="v1"/>
-    <xacro:arg name="stand" default="v1"/>
+    <xacro:arg name="collider" default="simple"/>
     <xacro:arg name="direction" default="left"/>
     <xacro:arg name="scene" default="world"/>
     <xacro:property name="prefix" value="$(arg direction)_"/>
-    <xacro:property name="selected_scene" value="$(arg scene)"/>
+    <xacro:property name="type_arg" value="$(arg type)"/>
+    <xacro:property name="is_stand_only" value="${'stand' in type_arg}"/>
+    <xacro:property name="is_arm_only" value="${type_arg == 'arm_only'}"/>
+    <xacro:property name="stand_type" value="v1"/>
+    <xacro:if value="${'v2' in type_arg}"><xacro:property name="stand_type" value="v2"/></xacro:if>
+    <xacro:if value="${'link8' in type_arg}"><xacro:property name="stand_type" value="link8"/></xacro:if>
     <xacro:include filename="$(find nero_description)/xacro/nero.xacro"/>
-    <link name="base_link"/>
-    <xacro:if value="${selected_scene == 'world'}">
+    <xacro:if value="${'$(arg scene)' == 'world'}">
         <link name="world"/>
+    </xacro:if>
+    <xacro:if value="${is_stand_only}">
+        <xacro:include filename="$(find nero_description)/xacro/hand.xacro"/>
+        <xacro:Hand type="hand" stand="${stand_type}" direction="$(arg direction)" prefix="${prefix}" standalone="true"/>
         <joint name="world_fixed" type="fixed">
             <parent link="world"/>
-            <child link="base_link"/>
-            <origin xyz="0 0 0" rpy="0 0 0"/>
+            <child link="${prefix}stand_adapter"/>
         </joint>
     </xacro:if>
-    <joint name="${prefix}base_joint" type="fixed">
-        <parent link="base_link"/>
-        <child link="${prefix}base_link"/>
-    </joint>
-    <xacro:Nero type="$(arg type)" stand="$(arg stand)" direction="$(arg direction)" prefix="${prefix}"/>
+    <xacro:unless value="${is_stand_only}">
+        <link name="base_link"/>
+        <xacro:if value="${'$(arg scene)' == 'world'}">
+            <joint name="world_fixed" type="fixed">
+                <parent link="world"/>
+                <child link="base_link"/>
+                <origin xyz="0 0 0" rpy="0 0 0"/>
+            </joint>
+        </xacro:if>
+        <joint name="${prefix}base_joint" type="fixed">
+            <parent link="base_link"/>
+            <child link="${prefix}base_link"/>
+            <origin xyz="0 0 0" rpy="0 0 3.14159"/>
+        </joint>
+        <xacro:Nero type="${type_arg}" stand="${stand_type}" direction="$(arg direction)" prefix="${prefix}"
+                    is_arm_only="${is_arm_only}"/>
+    </xacro:unless>
 </robot>
