Commit message: update realman aidal

File: humanoid/Realman/aidal_description/xacro/components/body.xacro (robot description, xacro)
@@ -1,4 +1,5 @@
 <?xml version="1.0"?>
 <robot name="body_head_platform" xmlns:xacro="http://www.ros.org/wiki/xacro">
+  <xacro:property name="PI" value="3.1415926535897931"/>
   <xacro:property name="mesh_path" value="file://$(find aidal_description)/meshes/body/"/>
   <xacro:macro name="visual_collision" params="mesh">
@@ -29,5 +30,5 @@
           izz="0.15316"/>
     </inertial>
-    <xacro:visual_collision mesh="body_base_link.obj"/>
+    <xacro:visual_collision mesh="base.glb"/>
   </link>
   <link name="platform_base_link">
@@ -43,5 +44,5 @@
           izz="0.021546"/>
     </inertial>
-    <xacro:visual_collision mesh="platform_body.obj"/>
+    <xacro:visual_collision mesh="lift.glb"/>
   </link>
   <link name="head_link1">
@@ -57,5 +58,5 @@
           izz="1.3605E-05"/>
     </inertial>
-    <xacro:visual_collision mesh="head_link1.obj"/>
+    <xacro:visual_collision mesh="head1.glb"/>
   </link>
   <link name="head_link2">
@@ -71,5 +72,5 @@
           izz="0.00052625"/>
     </inertial>
-    <xacro:visual_collision mesh="head_link2.obj"/>
+    <xacro:visual_collision mesh="head2.glb"/>
   </link>
   <link name="camera_link">
@@ -85,11 +86,15 @@
           izz="3.0901E-05"/>
     </inertial>
-    <xacro:visual_collision mesh="d435.obj"/>
+    <visual>
+      <geometry>
+        <mesh filename="file://$(find sensor_models)/meshes/d435.glb"/>
+      </geometry>
+    </visual>
   </link>
-  <joint name="platform_joint" type="prismatic">
-    <origin xyz="0 -0.11663 1.271" />
+  <joint name="lift_joint" type="prismatic">
+    <origin xyz="0 -0.11663 0.271" />
     <parent link="body_base_link"/>
     <child link="platform_base_link"/>
-    <axis xyz="0 0 -1"/>
+    <axis xyz="0 0 1"/>
     <limit lower="0" upper="1" effort="60" velocity="0.15"/>
   </joint>
@@ -109,8 +114,59 @@
   </joint>
   <joint name="camera_joint" type="fixed">
-    <origin xyz="-0.0002391 -0.076866 0.061606" rpy="-1.5708 0 3.14159"/>
+    <origin xyz="-0.0002391 -0.076866 0.061606" rpy="-${PI/2} 0 ${PI}"/>
     <parent link="head_link2"/>
     <child link="camera_link"/>
-    <axis xyz="0 0 0"/>
   </joint>
+  <link name="top_camera"/>
+  <joint name="top_camera_joint" type="fixed">
+    <origin xyz=" 0 -0.1275 1.451" rpy="-${PI/2} 0 ${PI}"/>
+    <parent link="body_base_link"/>
+    <child link="top_camera"/>
+  </joint>
+  <joint name="l_base_joint1" type="fixed">
+    <origin xyz="0.1 -0.1103 0.031645" rpy="0 -${PI/4} ${PI}"/>
+    <parent link="platform_base_link"/>
+    <child link="left_base_link"/>
+  </joint>
+  <joint name="r_base_joint1" type="fixed">
+    <origin xyz="-0.1 -0.1103 0.031645" rpy="0 -${PI/4} 0"/>
+    <parent link="platform_base_link"/>
+    <child link="right_base_link"/>
+  </joint>
+  <link name="left_base_link">
+    <inertial>
+      <origin xyz="-3.58E-05 -0.0056915 0.024464"/>
+      <mass value="0.23441"/>
+      <inertia
+          ixx="0.00027369"
+          ixy="6.5702E-08"
+          ixz="2.7812E-09"
+          iyy="0.000264"
+          iyz="-1.6355E-06"
+          izz="0.00036679"/>
+    </inertial>
+    <visual>
+      <geometry>
+        <mesh filename="${mesh_path}arm_base.glb"/>
+      </geometry>
+    </visual>
+  </link>
+  <link name="right_base_link">
+    <inertial>
+      <origin xyz="-4.8022E-05 0.0056915 0.024715"/>
+      <mass value="0.23441"/>
+      <inertia
+          ixx="0.00027369"
+          ixy="6.5702E-08"
+          ixz="-3.2599E-09"
+          iyy="0.000264"
+          iyz="1.6355E-06"
+          izz="0.00036679"/>
+    </inertial>
+    <visual>
+      <geometry>
+        <mesh filename="${mesh_path}arm_base.glb"/>
+      </geometry>
+    </visual>
+  </link>
 </robot>

File: humanoid/Realman/aidal_description/xacro/components/woosh_agv.xacro (robot description, xacro)
@@ -1,237 +1,312 @@
 <?xml version="1.0"?>
 <robot name="woosh_agv" xmlns:xacro="http://www.ros.org/wiki/xacro">
-  <!-- Define constants -->
-  <xacro:property name="mesh_path" value="file://$(find aidal_description)/meshes/woosh_agv/"/>
-  <!-- Macro for visual and collision elements -->
-  <xacro:macro name="visual_collision" params="mesh">
-    <visual>
-      <geometry>
-        <mesh filename="${mesh_path}${mesh}"/>
-      </geometry>
-      <material name="">
-        <color rgba="0.79216 0.81961 0.93333 1"/>
-      </material>
-    </visual>
-    <collision>
-      <geometry>
-        <mesh filename="${mesh_path}${mesh}"/>
-      </geometry>
-    </collision>
-  </xacro:macro>
-  <link name="base_link">
-    <inertial>
-      <origin xyz="-0.012628 -0.016092 -0.060646"/>
-      <mass value="2.5521"/>
-      <inertia
-          ixx="0.066197"
-          ixy="7.0297E-05"
-          ixz="0.00017628"
-          iyy="0.034903"
-          iyz="-0.00059595"
-          izz="0.097938"/>
-    </inertial>
-    <xacro:visual_collision mesh="base_link.obj"/>
-  </link>
-  <link name="link_right_wheel">
-    <inertial>
-      <origin xyz="-0.024898 2.5665E-18 0"/>
-      <mass value="1.0523"/>
-      <inertia
-          ixx="0.0033125"
-          ixy="1.5953E-19"
-          ixz="1.2287E-20"
-          iyy="0.0018066"
-          iyz="2.5666E-19"
-          izz="0.0018066"/>
-    </inertial>
-    <xacro:visual_collision mesh="right_wheel.obj"/>
-  </link>
-  <link name="link_left_wheel">
-    <inertial>
-      <origin xyz="0.025224 -8.8034E-15 0"/>
-      <mass value="1.0734"/>
-      <inertia
-          ixx="0.0033996"
-          ixy="-5.0277E-16"
-          ixz="9.2981E-21"
-          iyy="0.0019593"
-          iyz="3.7534E-19"
-          izz="0.0019593"/>
-    </inertial>
-    <xacro:visual_collision mesh="left_wheel.obj"/>
-  </link>
-  <link name="link_swivel_wheel_1_1">
-    <inertial>
-      <origin xyz="0.00067987 -0.0050012 -0.013414"/>
-      <mass value="0.088835"/>
-      <inertia
-          ixx="3.1679E-05"
-          ixy="2.0129E-08"
-          ixz="2.7021E-08"
-          iyy="3.9438E-05"
-          iyz="-3.2776E-06"
-          izz="4.6143E-05"/>
-    </inertial>
-    <xacro:visual_collision mesh="swivel_wheel_1.obj"/>
-  </link>
-  <link name="link_swivel_wheel_1_2">
-    <inertial>
-      <origin xyz="0.0010651 2.2204E-16 9.4369E-16"/>
-      <mass value="0.12664"/>
-      <inertia
-          ixx="0.00011169"
-          ixy="1.1345E-14"
-          ixz="2.2064E-14"
-          iyy="6.0838E-05"
-          iyz="1.7051E-09"
-          izz="6.084E-05"/>
-    </inertial>
-    <xacro:visual_collision mesh="swivel_wheel_2.obj"/>
-  </link>
-  <link name="link_swivel_wheel_2_1">
-    <inertial>
-      <origin xyz="0.00067987 -0.0050012 -0.013414"/>
-      <mass value="0.088835"/>
-      <inertia
-          ixx="3.1679E-05"
-          ixy="2.0129E-08"
-          ixz="2.7021E-08"
-          iyy="3.9438E-05"
-          iyz="-3.2776E-06"
-          izz="4.6143E-05"/>
-    </inertial>
-    <xacro:visual_collision mesh="swivel_wheel_1.obj"/>
-  </link>
-  <link name="link_swivel_wheel_2_2">
-    <inertial>
-      <origin xyz="0.0010651 6.1062E-16 7.7716E-16"/>
-      <mass value="0.12664"/>
-      <inertia
-          ixx="0.00011169"
-          ixy="1.9869E-14"
-          ixz="1.4856E-14"
-          iyy="6.084E-05"
-          iyz="2.0109E-09"
-          izz="6.0838E-05"/>
-    </inertial>
-    <xacro:visual_collision mesh="swivel_wheel_2.obj"/>
-  </link>
-  <link name="link_swivel_wheel_3_1">
-    <inertial>
-      <origin xyz="0.00067987 -0.0050012 -0.013414"/>
-      <mass value="0.088835"/>
-      <inertia
-          ixx="3.1679E-05"
-          ixy="2.0129E-08"
-          ixz="2.7021E-08"
-          iyy="3.9438E-05"
-          iyz="-3.2776E-06"
-          izz="4.6143E-05"/>
-    </inertial>
-    <xacro:visual_collision mesh="swivel_wheel_1.obj"/>
-  </link>
-  <link name="link_swivel_wheel_3_2">
-    <inertial>
-      <origin xyz="0.0010651 -3.3307E-16 8.8818E-16"/>
-      <mass value="0.12664"/>
-      <inertia
-          ixx="0.00011169"
-          ixy="-1.8513E-15"
-          ixz="2.474E-14"
-          iyy="6.0837E-05"
-          iyz="-3.1204E-10"
-          izz="6.0841E-05"/>
-    </inertial>
-    <xacro:visual_collision mesh="swivel_wheel_2.obj"/>
-  </link>
-  <link name="link_swivel_wheel_4_1">
-    <inertial>
-      <origin xyz="0.00067987 -0.0050012 -0.0094542"/>
-      <mass value="0.088835"/>
-      <inertia
-          ixx="3.1679E-05"
-          ixy="2.0129E-08"
-          ixz="2.7021E-08"
-          iyy="3.9438E-05"
-          iyz="-3.2776E-06"
-          izz="4.6143E-05"/>
-    </inertial>
-    <xacro:visual_collision mesh="swivel_wheel_1.obj"/>
-  </link>
-  <link name="link_swivel_wheel_4_2">
-    <inertial>
-      <origin xyz="0.0010651 -4.996E-16 7.494E-16"/>
-      <mass value="0.12664"/>
-      <inertia
-          ixx="0.00011169"
-          ixy="-7.4776E-15"
-          ixz="2.3656E-14"
-          iyy="6.0837E-05"
-          iyz="-1.205E-09"
-          izz="6.0841E-05"/>
-    </inertial>
-    <xacro:visual_collision mesh="swivel_wheel_2.obj"/>
-  </link>
-  <joint name="joint_right_wheel" type="continuous">
-    <origin xyz="-0.148 0.015574 -0.153"/>
-    <parent link="base_link"/>
-    <child link="link_right_wheel"/>
-    <axis xyz="1 0 0"/>
-    <limit effort="100" velocity="10"/>
-  </joint>
-  <joint name="joint_left_wheel" type="continuous">
-    <origin xyz="0.148 0.015574 -0.153"/>
-    <parent link="base_link"/>
-    <child link="link_left_wheel"/>
-    <axis xyz="-1 0 0"/>
-    <limit effort="100" velocity="10"/>
-  </joint>
-  <joint name="joint_swivel_wheel_1_1" type="continuous">
-    <origin xyz="0.124 -0.17843 -0.16254"/>
-    <parent link="base_link"/>
-    <child link="link_swivel_wheel_1_1"/>
-    <axis xyz="0 0 1"/>
-  </joint>
-  <joint name="joint_swivel_wheel_1_2" type="continuous">
-    <origin xyz="-0.0035 -0.022 -0.04516"/>
-    <parent link="link_swivel_wheel_1_1"/>
-    <child link="link_swivel_wheel_1_2"/>
-    <axis xyz="1 0 0"/>
-  </joint>
-  <joint name="joint_swivel_wheel_2_1" type="continuous">
-    <origin xyz="-0.126 0.22157 -0.16254"/>
-    <parent link="base_link"/>
-    <child link="link_swivel_wheel_2_1"/>
-    <axis xyz="0 0 1"/>
-  </joint>
-  <joint name="joint_swivel_wheel_2_2" type="continuous">
-    <origin xyz="-0.0035 -0.022 -0.04516"/>
-    <parent link="link_swivel_wheel_2_1"/>
-    <child link="link_swivel_wheel_2_2"/>
-    <axis xyz="1 0 0"/>
-  </joint>
-  <joint name="joint_swivel_wheel_3_1" type="continuous">
-    <origin xyz="0.124 0.22157 -0.16254"/>
-    <parent link="base_link"/>
-    <child link="link_swivel_wheel_3_1"/>
-    <axis xyz="0 0 1"/>
-  </joint>
-  <joint name="joint_swivel_wheel_3_2" type="continuous">
-    <origin xyz="-0.0035 -0.022 -0.04516"/>
-    <parent link="link_swivel_wheel_3_1"/>
-    <child link="link_swivel_wheel_3_2"/>
-    <axis xyz="1 0 0"/>
-  </joint>
-  <joint name="joint_swivel_wheel_4_1" type="continuous">
-    <origin xyz="-0.126 -0.17843 -0.1665"/>
-    <parent link="base_link"/>
-    <child link="link_swivel_wheel_4_1"/>
-    <axis xyz="0 0 1"/>
-  </joint>
-  <joint name="joint_swivel_wheel_4_2" type="continuous">
-    <origin xyz="-0.0035 -0.022 -0.0412"/>
-    <parent link="link_swivel_wheel_4_1"/>
-    <child link="link_swivel_wheel_4_2"/>
-    <axis xyz="1 0 0"/>
-  </joint>
+	<!-- Define constants -->
+	<xacro:property name="mesh_path" value="file://$(find aidal_description)/meshes/woosh_agv/"/>
+	<!-- Macro for visual and collision elements -->
+	<xacro:macro name="visual_mesh" params="mesh">
+		<visual>
+			<geometry>
+				<mesh filename="${mesh_path}${mesh}"/>
+			</geometry>
+		</visual>
+	</xacro:macro>
+	<xacro:macro name="woosh_agv" params="joints_movable:=true">
+		<!-- 根据 joints_movable 参数设置底盘关节类型 -->
+		<xacro:if value="${joints_movable}">
+			<xacro:property name="steer_joint_type" value="continuous"/>
+			<xacro:property name="wheel_joint_type" value="continuous"/>
+		</xacro:if>
+		<xacro:unless value="${joints_movable}">
+			<xacro:property name="steer_joint_type" value="fixed"/>
+			<xacro:property name="wheel_joint_type" value="fixed"/>
+		</xacro:unless>
+	<link name="base_link">
+		<inertial>
+			<origin xyz="-0.012628 -0.016092 -0.060646"/>
+			<mass value="2.5521"/>
+			<inertia
+					ixx="0.066197"
+					ixy="7.0297E-05"
+					ixz="0.00017628"
+					iyy="0.034903"
+					iyz="-0.00059595"
+					izz="0.097938"/>
+		</inertial>
+		<xacro:visual_mesh mesh="base.glb"/>
+		<collision>
+			<origin xyz="-0.015574 0 -0.1"/>
+			<geometry>
+				<box size="0.4 0.6 0.2"/>
+			</geometry>
+		</collision>
+	</link>
+	<link name="right_wheel_link">
+		<inertial>
+			<origin xyz="-0.024898 2.5665E-18 0"/>
+			<mass value="1.0523"/>
+			<inertia
+					ixx="0.0033125"
+					ixy="1.5953E-19"
+					ixz="1.2287E-20"
+					iyy="0.0018066"
+					iyz="2.5666E-19"
+					izz="0.0018066"/>
+		</inertial>
+		<visual>
+			<geometry>
+				<mesh filename="${mesh_path}wheel.glb" scale="-1 1 1"/>
+			</geometry>
+		</visual>
+		<collision>
+			<origin rpy=" 0 1.5708 0" xyz="-0.024 0 0"/>
+			<geometry>
+				<cylinder radius="0.085" length="0.034"/>
+			</geometry>
+		</collision>
+	</link>
+	<link name="left_wheel_link">
+		<inertial>
+			<origin xyz="0.025224 -8.8034E-15 0"/>
+			<mass value="1.0734"/>
+			<inertia
+					ixx="0.0033996"
+					ixy="-5.0277E-16"
+					ixz="9.2981E-21"
+					iyy="0.0019593"
+					iyz="3.7534E-19"
+					izz="0.0019593"/>
+		</inertial>
+		<visual>
+			<geometry>
+				<mesh filename="${mesh_path}wheel.glb"/>
+			</geometry>
+		</visual>
+		<collision>
+			<origin rpy="0 1.5708 0" xyz="0.024 0 0"/>
+			<geometry>
+				<cylinder radius="0.085" length="0.034"/>
+			</geometry>
+		</collision>
+	</link>
+	<link name="caster_1_link">
+		<inertial>
+			<origin xyz="0.00067987 -0.0050012 -0.013414"/>
+			<mass value="0.088835"/>
+			<inertia
+					ixx="3.1679E-05"
+					ixy="2.0129E-08"
+					ixz="2.7021E-08"
+					iyy="3.9438E-05"
+					iyz="-3.2776E-06"
+					izz="4.6143E-05"/>
+		</inertial>
+		<xacro:visual_mesh mesh="caster.glb"/>
+	</link>
+	<link name="caster_wheel_1_link">
+		<inertial>
+			<origin xyz="0.0010651 2.2204E-16 9.4369E-16"/>
+			<mass value="0.12664"/>
+			<inertia
+					ixx="0.00011169"
+					ixy="1.1345E-14"
+					ixz="2.2064E-14"
+					iyy="6.0838E-05"
+					iyz="1.7051E-09"
+					izz="6.084E-05"/>
+		</inertial>
+		<xacro:visual_mesh mesh="caster_wheel.glb"/>
+		<collision>
+			<geometry>
+				<sphere radius="0.0375"/>
+			</geometry>
+		</collision>
+	</link>
+	<link name="caster_2_link">
+		<inertial>
+			<origin xyz="0.00067987 -0.0050012 -0.013414"/>
+			<mass value="0.088835"/>
+			<inertia
+					ixx="3.1679E-05"
+					ixy="2.0129E-08"
+					ixz="2.7021E-08"
+					iyy="3.9438E-05"
+					iyz="-3.2776E-06"
+					izz="4.6143E-05"/>
+		</inertial>
+		<xacro:visual_mesh mesh="caster.glb"/>
+	</link>
+	<link name="caster_wheel_2_link">
+		<inertial>
+			<origin xyz="0.0010651 6.1062E-16 7.7716E-16"/>
+			<mass value="0.12664"/>
+			<inertia
+					ixx="0.00011169"
+					ixy="1.9869E-14"
+					ixz="1.4856E-14"
+					iyy="6.084E-05"
+					iyz="2.0109E-09"
+					izz="6.0838E-05"/>
+		</inertial>
+		<xacro:visual_mesh mesh="caster_wheel.glb"/>
+		<collision>
+			<geometry>
+				<sphere radius="0.0375"/>
+			</geometry>
+		</collision>
+	</link>
+	<link name="caster_3_link">
+		<inertial>
+			<origin xyz="0.00067987 -0.0050012 -0.013414"/>
+			<mass value="0.088835"/>
+			<inertia
+					ixx="3.1679E-05"
+					ixy="2.0129E-08"
+					ixz="2.7021E-08"
+					iyy="3.9438E-05"
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
File: humanoid/Realman/aidal_description/xacro/ee.xacro (robot description, xacro)
@@ -1,4 +1,5 @@
 <?xml version="1.0"?>
 <robot name="aidal_ee" xmlns:xacro="http://www.ros.org/wiki/xacro">
+  <xacro:property name="PI" value="3.1415926535897931"/>
   <xacro:include filename="$(find inspire_description)/xacro/EG2-4C2.xacro"/>
   <xacro:macro name="aidal_ee" params="type:='EG2-4C2'">
@@ -9,5 +10,5 @@
         <parent link="left_ee"/>
         <child link="left_gripper_base"/>
-        <origin xyz="0 0 0.004" rpy="0 0 1.5708"/>
+        <origin xyz="0 0 0.004" rpy="0 0 ${PI/2}"/>
       </joint>
       <xacro:Gripper name="right"/>
@@ -15,5 +16,5 @@
         <parent link="right_ee"/>
         <child link="right_gripper_base"/>
-        <origin xyz="0 0 0.004" rpy="0 0 1.5708"/>
+        <origin xyz="0 0 0.004" rpy="0 0 ${PI/2}"/>
       </joint>
     </xacro:if>

File: humanoid/Realman/aidal_description/xacro/robot.xacro (robot description, xacro)
@@ -2,4 +2,5 @@
 <robot name="RealMan_AIDAL" xmlns:xacro="http://ros.org/wiki/xacro">
 	<xacro:arg name="type" default="empty"/>
+	<xacro:property name="PI" value="3.1415926535897931"/>
 	<xacro:property name="type_arg" value="$(arg type)"/>
 	<xacro:property name="selected_gripper_type" value="empty"/>
@@ -9,4 +10,5 @@
 	<!-- 引入各个模块的 xacro 文件，分别定义底盘、夹爪、升降平台、机械臂及关节 -->
 	<xacro:include filename="$(find aidal_description)/xacro/components/woosh_agv.xacro"/>
+	<xacro:woosh_agv joints_movable="false"/>
 	<xacro:include filename="$(find aidal_description)/xacro/components/body.xacro"/>
 	<xacro:include filename="$(find aidal_description)/xacro/ee.xacro"/>
@@ -19,47 +21,11 @@
 		<child link="body_base_link"/>
 	</joint>
-	<joint name="l_base_joint1" type="fixed">
-		<origin xyz="0.1 -0.1103 0.031645" rpy="0 -0.7854 3.14159"/>
-		<parent link="platform_base_link"/>
-		<child link="left_base_link"/>
-	</joint>
-	<joint name="r_base_joint1" type="fixed">
-		<origin xyz="-0.1 -0.1103 0.031645" rpy="0 -0.7854 0"/>
-		<parent link="platform_base_link"/>
-		<child link="right_base_link"/>
-	</joint>
-	<link name="left_base_link">
-		<inertial>
-			<origin xyz="-3.58E-05 -0.0056915 0.024464"/>
-			<mass value="0.23441"/>
-			<inertia
-					ixx="0.00027369"
-					ixy="6.5702E-08"
-					ixz="2.7812E-09"
-					iyy="0.000264"
-					iyz="-1.6355E-06"
-					izz="0.00036679"/>
-		</inertial>
-	</link>
 	<joint name="l_base_joint2" type="fixed">
-		<origin xyz="0 0 0.187" rpy="-1.5708 0 0"/>
+		<origin xyz="0 0 0.187" rpy="-${PI/2} 0 0"/>
 		<parent link="left_base_link"/>
 		<child link="left_arm_root"/>
 	</joint>
-	<link name="right_base_link">
-		<inertial>
-			<origin xyz="-4.8022E-05 0.0056915 0.024715"/>
-			<mass value="0.23441"/>
-			<inertia
-					ixx="0.00027369"
-					ixy="6.5702E-08"
-					ixz="-3.2599E-09"
-					iyy="0.000264"
-					iyz="1.6355E-06"
-					izz="0.00036679"/>
-		</inertial>
-	</link>
 	<joint name="r_base_joint2" type="fixed">
-		<origin xyz="0 0 0.187" rpy="-1.5708 0 3.1415"/>
+		<origin xyz="0 0 0.187" rpy="-${PI/2} 0 ${PI}"/>
 		<parent link="right_base_link"/>
 		<child link="right_arm_root"/>

Commit message: fix mesh problems

File: humanoid/Realman/aidal_description/xacro/components/body.xacro (robot description, xacro)
@@ -8,7 +8,4 @@
         <mesh filename="${mesh_path}${mesh}" />
       </geometry>
-      <material name="">
-        <color rgba="0.79216 0.81961 0.93333 1" />
-      </material>
     </visual>
     <collision>

File: humanoid/Realman/aidal_description/xacro/components/woosh_agv.xacro (robot description, xacro)
@@ -59,5 +59,5 @@
 		</visual>
 		<collision>
-			<origin rpy=" 0 1.5708 0" xyz="-0.024 0 0"/>
+			<origin rpy="0 ${PI/2} 0"/>
 			<geometry>
 				<cylinder radius="0.085" length="0.034"/>
@@ -83,5 +83,5 @@
 		</visual>
 		<collision>
-			<origin rpy="0 1.5708 0" xyz="0.024 0 0"/>
+			<origin rpy="0 ${PI/2} 0"/>
 			<geometry>
 				<cylinder radius="0.085" length="0.034"/>
@@ -222,5 +222,5 @@
 	</link>
 	<joint name="right_wheel_joint" type="${wheel_joint_type}">
-		<origin xyz="-0.148 0.015574 -0.153"/>
+		<origin xyz="-0.183 0.015574 -0.153"/>
 		<parent link="base_link"/>
 		<child link="right_wheel_link"/>
@@ -231,5 +231,5 @@
 	</joint>
 	<joint name="left_wheel_joint" type="${wheel_joint_type}">
-		<origin xyz="0.148 0.015574 -0.153"/>
+		<origin xyz="0.183 0.015574 -0.153"/>
 		<parent link="base_link"/>
 		<child link="left_wheel_link"/>
@@ -240,5 +240,5 @@
 	</joint>
 	<joint name="caster_1_joint" type="${steer_joint_type}">
-		<origin xyz="0.124 -0.17843 -0.1593" rpy="0 0 ${PI}"/>
+		<origin xyz="0.124 -0.17843 -0.1589" rpy="0 0 ${PI}"/>
 		<parent link="base_link"/>
 		<child link="caster_1_link"/>
@@ -256,5 +256,5 @@
 	</joint>
 	<joint name="caster_2_joint" type="${steer_joint_type}">
-		<origin xyz="-0.126 0.22157 -0.1593" rpy="0 0 ${PI}"/>
+		<origin xyz="-0.124 0.194004 -0.1589" rpy="0 0 ${PI}"/>
 		<parent link="base_link"/>
 		<child link="caster_2_link"/>
@@ -272,5 +272,5 @@
 	</joint>
 	<joint name="caster_3_joint" type="${steer_joint_type}">
-		<origin xyz="0.124 0.22157 -0.1593" rpy="0 0 ${PI}"/>
+		<origin xyz="0.124 0.194004 -0.1589" rpy="0 0 ${PI}"/>
 		<parent link="base_link"/>
 		<child link="caster_3_link"/>
@@ -288,5 +288,5 @@
 	</joint>
 	<joint name="caster_4_joint" type="${steer_joint_type}">
-		<origin xyz="-0.126 -0.17843 -0.1593" rpy="0 0 ${PI}"/>
+		<origin xyz="-0.124 -0.17843 -0.1589" rpy="0 0 ${PI}"/>
 		<parent link="base_link"/>
 		<child link="caster_4_link"/>
@@ -296,5 +296,5 @@
 	</joint>
 	<joint name="caster_wheel_4_joint" type="${wheel_joint_type}">
-		<origin xyz="0 -0.022 -0.0412"/>
+		<origin xyz="0 -0.022 -0.04516"/>
 		<parent link="caster_4_link"/>
 		<child link="caster_wheel_4_link"/>
@@ -310,3 +310,35 @@
 	</joint>
 	</xacro:macro>
+	<link name="chassis_panel">
+<!--		<xacro:visual_mesh mesh="panel.glb"/>-->
+	</link>
+	<joint name="chassis_panel_joint" type="fixed">
+		<origin xyz="0.18 0.118  -0.0275"/>
+		<parent link="base_link"/>
+		<child link="chassis_panel"/>
+	</joint>
+	<link name="lidar_link">
+<!--		<visual>-->
+<!--			<geometry>-->
+<!--				<mesh filename="file://$(find sensor_models)/meshes/orbbec/ms500.glb"/>-->
+<!--			</geometry>-->
+<!--		</visual>-->
+	</link>
+	<joint name="lidar_joint" type="fixed">
+		<origin xyz="0 -0.2496  -0.094808"/>
+		<parent link="base_link"/>
+		<child link="lidar_link"/>
+	</joint>
+	<link name="chassis_camera_link">
+<!--		<visual>-->
+<!--			<geometry>-->
+<!--				<mesh filename="file://$(find sensor_models)/meshes/orbbec/Dabai_DW.glb"/>-->
+<!--			</geometry>-->
+<!--		</visual>-->
+	</link>
+	<joint name="chassis_camera_joint" type="fixed">
+		<origin xyz="0 -0.2965  -0.1126" rpy="-${PI/2} 0 ${PI}"/>
+		<parent link="base_link"/>
+		<child link="chassis_camera_link"/>
+	</joint>
 </robot>
