Commit message: add x2 robot quanta x1

File: humanoid/Realman/aidal_description/xacro/components/woosh_agv.xacro (robot description, xacro)
@@ -311,5 +311,5 @@
 	</xacro:macro>
 	<link name="chassis_panel">
-<!--		<xacro:visual_mesh mesh="panel.glb"/>-->
+		<xacro:visual_mesh mesh="panel.glb"/>
 	</link>
 	<joint name="chassis_panel_joint" type="fixed">
@@ -319,9 +319,9 @@
 	</joint>
 	<link name="lidar_link">
-<!--		<visual>-->
-<!--			<geometry>-->
-<!--				<mesh filename="file://$(find sensor_models)/meshes/orbbec/ms500.glb"/>-->
-<!--			</geometry>-->
-<!--		</visual>-->
+		<visual>
+			<geometry>
+				<mesh filename="file://$(find sensor_models)/meshes/orbbec/ms500.glb"/>
+			</geometry>
+		</visual>
 	</link>
 	<joint name="lidar_joint" type="fixed">
@@ -331,9 +331,9 @@
 	</joint>
 	<link name="chassis_camera_link">
-<!--		<visual>-->
-<!--			<geometry>-->
-<!--				<mesh filename="file://$(find sensor_models)/meshes/orbbec/Dabai_DW.glb"/>-->
-<!--			</geometry>-->
-<!--		</visual>-->
+		<visual>
+			<geometry>
+				<mesh filename="file://$(find sensor_models)/meshes/orbbec/Dabai_DW.glb"/>
+			</geometry>
+		</visual>
 	</link>
 	<joint name="chassis_camera_joint" type="fixed">

Commit message: format chassis xacro

File: humanoid/Realman/aidal_description/xacro/components/woosh_agv.xacro (robot description, xacro)
@@ -21,292 +21,292 @@
 			<xacro:property name="wheel_joint_type" value="fixed"/>
 		</xacro:unless>
-	<link name="base_link">
-		<inertial>
-			<origin xyz="-0.012628 -0.016092 -0.060646"/>
-			<mass value="2.5521"/>
-			<inertia
-					ixx="0.066197"
-					ixy="7.0297E-05"
-					ixz="0.00017628"
-					iyy="0.034903"
-					iyz="-0.00059595"
-					izz="0.097938"/>
-		</inertial>
-		<xacro:visual_mesh mesh="base.glb"/>
-		<collision>
-			<origin xyz="-0.015574 0 -0.1"/>
-			<geometry>
-				<box size="0.4 0.6 0.2"/>
-			</geometry>
-		</collision>
-	</link>
-	<link name="right_wheel_link">
-		<inertial>
-			<origin xyz="-0.024898 2.5665E-18 0"/>
-			<mass value="1.0523"/>
-			<inertia
-					ixx="0.0033125"
-					ixy="1.5953E-19"
-					ixz="1.2287E-20"
-					iyy="0.0018066"
-					iyz="2.5666E-19"
-					izz="0.0018066"/>
-		</inertial>
-		<visual>
-			<geometry>
-				<mesh filename="${mesh_path}wheel.glb" scale="-1 1 1"/>
-			</geometry>
-		</visual>
-		<collision>
-			<origin rpy="0 ${PI/2} 0"/>
-			<geometry>
-				<cylinder radius="0.085" length="0.034"/>
-			</geometry>
-		</collision>
-	</link>
-	<link name="left_wheel_link">
-		<inertial>
-			<origin xyz="0.025224 -8.8034E-15 0"/>
-			<mass value="1.0734"/>
-			<inertia
-					ixx="0.0033996"
-					ixy="-5.0277E-16"
-					ixz="9.2981E-21"
-					iyy="0.0019593"
-					iyz="3.7534E-19"
-					izz="0.0019593"/>
-		</inertial>
-		<visual>
-			<geometry>
-				<mesh filename="${mesh_path}wheel.glb"/>
-			</geometry>
-		</visual>
-		<collision>
-			<origin rpy="0 ${PI/2} 0"/>
-			<geometry>
-				<cylinder radius="0.085" length="0.034"/>
-			</geometry>
-		</collision>
-	</link>
-	<link name="caster_1_link">
-		<inertial>
-			<origin xyz="0.00067987 -0.0050012 -0.013414"/>
-			<mass value="0.088835"/>
-			<inertia
-					ixx="3.1679E-05"
-					ixy="2.0129E-08"
-					ixz="2.7021E-08"
-					iyy="3.9438E-05"
-					iyz="-3.2776E-06"
-					izz="4.6143E-05"/>
-		</inertial>
-		<xacro:visual_mesh mesh="caster.glb"/>
-	</link>
-	<link name="caster_wheel_1_link">
-		<inertial>
-			<origin xyz="0.0010651 2.2204E-16 9.4369E-16"/>
-			<mass value="0.12664"/>
-			<inertia
-					ixx="0.00011169"
-					ixy="1.1345E-14"
-					ixz="2.2064E-14"
-					iyy="6.0838E-05"
-					iyz="1.7051E-09"
-					izz="6.084E-05"/>
-		</inertial>
-		<xacro:visual_mesh mesh="caster_wheel.glb"/>
-		<collision>
-			<geometry>
-				<sphere radius="0.0375"/>
-			</geometry>
-		</collision>
-	</link>
-	<link name="caster_2_link">
-		<inertial>
-			<origin xyz="0.00067987 -0.0050012 -0.013414"/>
-			<mass value="0.088835"/>
-			<inertia
-					ixx="3.1679E-05"
-					ixy="2.0129E-08"
-					ixz="2.7021E-08"
-					iyy="3.9438E-05"
-					iyz="-3.2776E-06"
-					izz="4.6143E-05"/>
-		</inertial>
-		<xacro:visual_mesh mesh="caster.glb"/>
-	</link>
-	<link name="caster_wheel_2_link">
-		<inertial>
-			<origin xyz="0.0010651 6.1062E-16 7.7716E-16"/>
-			<mass value="0.12664"/>
-			<inertia
-					ixx="0.00011169"
-					ixy="1.9869E-14"
-					ixz="1.4856E-14"
-					iyy="6.084E-05"
-					iyz="2.0109E-09"
-					izz="6.0838E-05"/>
-		</inertial>
-		<xacro:visual_mesh mesh="caster_wheel.glb"/>
-		<collision>
-			<geometry>
-				<sphere radius="0.0375"/>
-			</geometry>
-		</collision>
-	</link>
-	<link name="caster_3_link">
-		<inertial>
-			<origin xyz="0.00067987 -0.0050012 -0.013414"/>
-			<mass value="0.088835"/>
-			<inertia
-					ixx="3.1679E-05"
-					ixy="2.0129E-08"
-					ixz="2.7021E-08"
-					iyy="3.9438E-05"
-					iyz="-3.2776E-06"
-					izz="4.6143E-05"/>
-		</inertial>
-		<xacro:visual_mesh mesh="caster.glb"/>
-	</link>
-	<link name="caster_wheel_3_link">
-		<inertial>
-			<origin xyz="0.0010651 -3.3307E-16 8.8818E-16"/>
-			<mass value="0.12664"/>
-			<inertia
-					ixx="0.00011169"
-					ixy="-1.8513E-15"
-					ixz="2.474E-14"
-					iyy="6.0837E-05"
-					iyz="-3.1204E-10"
-					izz="6.0841E-05"/>
-		</inertial>
-		<xacro:visual_mesh mesh="caster_wheel.glb"/>
-		<collision>
-			<geometry>
-				<sphere radius="0.0375"/>
-			</geometry>
-		</collision>
-	</link>
-	<link name="caster_4_link">
-		<inertial>
-			<origin xyz="0.00067987 -0.0050012 -0.0094542"/>
-			<mass value="0.088835"/>
-			<inertia
-					ixx="3.1679E-05"
-					ixy="2.0129E-08"
-					ixz="2.7021E-08"
-					iyy="3.9438E-05"
-					iyz="-3.2776E-06"
-					izz="4.6143E-05"/>
-		</inertial>
-		<xacro:visual_mesh mesh="caster.glb"/>
-	</link>
-	<link name="caster_wheel_4_link">
-		<inertial>
-			<origin xyz="0.0010651 -4.996E-16 7.494E-16"/>
-			<mass value="0.12664"/>
-			<inertia
-					ixx="0.00011169"
-					ixy="-7.4776E-15"
-					ixz="2.3656E-14"
-					iyy="6.0837E-05"
-					iyz="-1.205E-09"
-					izz="6.0841E-05"/>
-		</inertial>
-		<xacro:visual_mesh mesh="caster_wheel.glb"/>
-		<collision>
-			<geometry>
-				<sphere radius="0.0375"/>
-			</geometry>
-		</collision>
-	</link>
-	<joint name="right_wheel_joint" type="${wheel_joint_type}">
-		<origin xyz="-0.183 0.015574 -0.153"/>
-		<parent link="base_link"/>
-		<child link="right_wheel_link"/>
-		<xacro:if value="${joints_movable}">
-			<axis xyz="1 0 0"/>
-			<limit effort="100" velocity="10"/>
-		</xacro:if>
-	</joint>
-	<joint name="left_wheel_joint" type="${wheel_joint_type}">
-		<origin xyz="0.183 0.015574 -0.153"/>
-		<parent link="base_link"/>
-		<child link="left_wheel_link"/>
-		<xacro:if value="${joints_movable}">
-			<axis xyz="1 0 0"/>
-			<limit effort="100" velocity="10"/>
-		</xacro:if>
-	</joint>
-	<joint name="caster_1_joint" type="${steer_joint_type}">
-		<origin xyz="0.124 -0.17843 -0.1589" rpy="0 0 ${PI}"/>
-		<parent link="base_link"/>
-		<child link="caster_1_link"/>
-		<xacro:if value="${joints_movable}">
-			<axis xyz="0 0 1"/>
-		</xacro:if>
-	</joint>
-	<joint name="caster_wheel_1_joint" type="${wheel_joint_type}">
-		<origin xyz="0 -0.022 -0.04516"/>
-		<parent link="caster_1_link"/>
-		<child link="caster_wheel_1_link"/>
-		<xacro:if value="${joints_movable}">
-			<axis xyz="1 0 0"/>
-		</xacro:if>
-	</joint>
-	<joint name="caster_2_joint" type="${steer_joint_type}">
-		<origin xyz="-0.124 0.194004 -0.1589" rpy="0 0 ${PI}"/>
-		<parent link="base_link"/>
-		<child link="caster_2_link"/>
-		<xacro:if value="${joints_movable}">
-			<axis xyz="0 0 1"/>
-		</xacro:if>
-	</joint>
-	<joint name="caster_wheel_2_joint" type="${wheel_joint_type}">
-		<origin xyz="0 -0.022 -0.04516" />
-		<parent link="caster_2_link"/>
-		<child link="caster_wheel_2_link"/>
-		<xacro:if value="${joints_movable}">
-			<axis xyz="1 0 0"/>
-		</xacro:if>
-	</joint>
-	<joint name="caster_3_joint" type="${steer_joint_type}">
-		<origin xyz="0.124 0.194004 -0.1589" rpy="0 0 ${PI}"/>
-		<parent link="base_link"/>
-		<child link="caster_3_link"/>
-		<xacro:if value="${joints_movable}">
-			<axis xyz="0 0 1"/>
-		</xacro:if>
-	</joint>
-	<joint name="caster_wheel_3_joint" type="${wheel_joint_type}">
-		<origin xyz="0 -0.022 -0.04516"/>
-		<parent link="caster_3_link"/>
-		<child link="caster_wheel_3_link"/>
-		<xacro:if value="${joints_movable}">
-			<axis xyz="1 0 0"/>
-		</xacro:if>
-	</joint>
-	<joint name="caster_4_joint" type="${steer_joint_type}">
-		<origin xyz="-0.124 -0.17843 -0.1589" rpy="0 0 ${PI}"/>
-		<parent link="base_link"/>
-		<child link="caster_4_link"/>
-		<xacro:if value="${joints_movable}">
-			<axis xyz="0 0 1"/>
-		</xacro:if>
-	</joint>
-	<joint name="caster_wheel_4_joint" type="${wheel_joint_type}">
-		<origin xyz="0 -0.022 -0.04516"/>
-		<parent link="caster_4_link"/>
-		<child link="caster_wheel_4_link"/>
-		<xacro:if value="${joints_movable}">
-			<axis xyz="1 0 0"/>
-		</xacro:if>
-	</joint>
-	<link name="base_footprint"/>
-	<joint name="base_footprint_joint" type="fixed">
-		<origin xyz="0.015574 0 0.238" rpy="0 0 ${PI/2}"/>
-		<parent link="base_footprint"/>
-		<child link="base_link"/>
-	</joint>
+		<link name="base_link">
+			<inertial>
+				<origin xyz="-0.012628 -0.016092 -0.060646"/>
+				<mass value="2.5521"/>
+				<inertia
+						ixx="0.066197"
+						ixy="7.0297E-05"
+						ixz="0.00017628"
+						iyy="0.034903"
+						iyz="-0.00059595"
+						izz="0.097938"/>
+			</inertial>
+			<xacro:visual_mesh mesh="base.glb"/>
+			<collision>
+				<origin xyz="-0.015574 0 -0.1"/>
+				<geometry>
+					<box size="0.4 0.6 0.2"/>
+				</geometry>
+			</collision>
+		</link>
+		<link name="right_wheel_link">
+			<inertial>
+				<origin xyz="-0.024898 2.5665E-18 0"/>
+				<mass value="1.0523"/>
+				<inertia
+						ixx="0.0033125"
+						ixy="1.5953E-19"
+						ixz="1.2287E-20"
+						iyy="0.0018066"
+						iyz="2.5666E-19"
+						izz="0.0018066"/>
+			</inertial>
+			<visual>
+				<geometry>
+					<mesh filename="${mesh_path}wheel.glb" scale="-1 1 1"/>
+				</geometry>
+			</visual>
+			<collision>
+				<origin rpy="0 ${PI/2} 0"/>
+				<geometry>
+					<cylinder radius="0.085" length="0.034"/>
+				</geometry>
+			</collision>
+		</link>
+		<link name="left_wheel_link">
+			<inertial>
+				<origin xyz="0.025224 -8.8034E-15 0"/>
+				<mass value="1.0734"/>
+				<inertia
+						ixx="0.0033996"
+						ixy="-5.0277E-16"
+						ixz="9.2981E-21"
+						iyy="0.0019593"
+						iyz="3.7534E-19"
+						izz="0.0019593"/>
+			</inertial>
+			<visual>
+				<geometry>
+					<mesh filename="${mesh_path}wheel.glb"/>
+				</geometry>
+			</visual>
+			<collision>
+				<origin rpy="0 ${PI/2} 0"/>
+				<geometry>
+					<cylinder radius="0.085" length="0.034"/>
+				</geometry>
+			</collision>
+		</link>
+		<link name="caster_1_link">
+			<inertial>
+				<origin xyz="0.00067987 -0.0050012 -0.013414"/>
+				<mass value="0.088835"/>
+				<inertia
+						ixx="3.1679E-05"
+						ixy="2.0129E-08"
+						ixz="2.7021E-08"
+						iyy="3.9438E-05"
+						iyz="-3.2776E-06"
+						izz="4.6143E-05"/>
+			</inertial>
+			<xacro:visual_mesh mesh="caster.glb"/>
+		</link>
+		<link name="caster_wheel_1_link">
+			<inertial>
+				<origin xyz="0.0010651 2.2204E-16 9.4369E-16"/>
+				<mass value="0.12664"/>
+				<inertia
+						ixx="0.00011169"
+						ixy="1.1345E-14"
+						ixz="2.2064E-14"
+						iyy="6.0838E-05"
+						iyz="1.7051E-09"
+						izz="6.084E-05"/>
+			</inertial>
+			<xacro:visual_mesh mesh="caster_wheel.glb"/>
+			<collision>
+				<geometry>
+					<sphere radius="0.0375"/>
+				</geometry>
+			</collision>
+		</link>
+		<link name="caster_2_link">
+			<inertial>
+				<origin xyz="0.00067987 -0.0050012 -0.013414"/>
+				<mass value="0.088835"/>
+				<inertia
+						ixx="3.1679E-05"
+						ixy="2.0129E-08"
+						ixz="2.7021E-08"
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
Commit message: add ocs2 arm controller config for aidal

File: humanoid/Realman/aidal_description/xacro/components/woosh_agv.xacro (robot description, xacro)
@@ -309,36 +309,36 @@
 			<child link="base_link"/>
 		</joint>
+		<link name="chassis_panel">
+			<xacro:visual_mesh mesh="panel.glb"/>
+		</link>
+		<joint name="chassis_panel_joint" type="fixed">
+			<origin xyz="0.18 0.118  -0.0275"/>
+			<parent link="base_link"/>
+			<child link="chassis_panel"/>
+		</joint>
+		<link name="lidar_link">
+			<visual>
+				<geometry>
+					<mesh filename="file://$(find sensor_models)/meshes/orbbec/ms500.glb"/>
+				</geometry>
+			</visual>
+		</link>
+		<joint name="lidar_joint" type="fixed">
+			<origin xyz="0 -0.2496  -0.094808"/>
+			<parent link="base_link"/>
+			<child link="lidar_link"/>
+		</joint>
+		<link name="chassis_camera_link">
+			<visual>
+				<geometry>
+					<mesh filename="file://$(find sensor_models)/meshes/orbbec/Dabai_DW.glb"/>
+				</geometry>
+			</visual>
+		</link>
+		<joint name="chassis_camera_joint" type="fixed">
+			<origin xyz="0 -0.2965  -0.1126" rpy="-${PI/2} 0 ${PI}"/>
+			<parent link="base_link"/>
+			<child link="chassis_camera_link"/>
+		</joint>
 	</xacro:macro>
-	<link name="chassis_panel">
-		<xacro:visual_mesh mesh="panel.glb"/>
-	</link>
-	<joint name="chassis_panel_joint" type="fixed">
-		<origin xyz="0.18 0.118  -0.0275"/>
-		<parent link="base_link"/>
-		<child link="chassis_panel"/>
-	</joint>
-	<link name="lidar_link">
-		<visual>
-			<geometry>
-				<mesh filename="file://$(find sensor_models)/meshes/orbbec/ms500.glb"/>
-			</geometry>
-		</visual>
-	</link>
-	<joint name="lidar_joint" type="fixed">
-		<origin xyz="0 -0.2496  -0.094808"/>
-		<parent link="base_link"/>
-		<child link="lidar_link"/>
-	</joint>
-	<link name="chassis_camera_link">
-		<visual>
-			<geometry>
-				<mesh filename="file://$(find sensor_models)/meshes/orbbec/Dabai_DW.glb"/>
-			</geometry>
-		</visual>
-	</link>
-	<joint name="chassis_camera_joint" type="fixed">
-		<origin xyz="0 -0.2965  -0.1126" rpy="-${PI/2} 0 ${PI}"/>
-		<parent link="base_link"/>
-		<child link="chassis_camera_link"/>
-	</joint>
 </robot>

File: humanoid/Realman/aidal_description/xacro/ee.xacro (robot description, xacro)
@@ -5,4 +5,16 @@
   <xacro:macro name="aidal_ee" params="type:='EG2-4C2'">
     <xacro:property name="gripper_type_norm" value="${str(type).upper()}"/>
+    <xacro:if value="${gripper_type_norm == 'EMPTY'}">
+      <link name="left_eef"/>
+      <link name="right_eef"/>
+      <joint name="left_ee_fix" type="fixed">
+        <parent link="left_ee"/>
+        <child link="left_eef"/>
+      </joint>
+      <joint name="right_ee_fix" type="fixed">
+        <parent link="right_ee"/>
+        <child link="right_eef"/>
+      </joint>
+    </xacro:if>
     <xacro:if value="${gripper_type_norm == 'EG2-4C2'}">
       <xacro:Gripper name="left"/>

File: humanoid/Realman/aidal_description/xacro/robot.xacro (robot description, xacro)
@@ -2,4 +2,5 @@
 <robot name="RealMan_AIDAL" xmlns:xacro="http://ros.org/wiki/xacro">
 	<xacro:arg name="type" default="empty"/>
+	<xacro:arg name="joints_movable" default="false"/>
 	<xacro:property name="PI" value="3.1415926535897931"/>
 	<xacro:property name="type_arg" value="$(arg type)"/>
@@ -10,5 +11,5 @@
 	<!-- 引入各个模块的 xacro 文件，分别定义底盘、夹爪、升降平台、机械臂及关节 -->
 	<xacro:include filename="$(find aidal_description)/xacro/components/woosh_agv.xacro"/>
-	<xacro:woosh_agv joints_movable="false"/>
+	<xacro:woosh_agv joints_movable="$(arg joints_movable)"/>
 	<xacro:include filename="$(find aidal_description)/xacro/components/body.xacro"/>
 	<xacro:include filename="$(find aidal_description)/xacro/ee.xacro"/>

File: manipulator/Realman/rm75_description/xacro/ros2_control/arm.xacro (robot description, xacro)
@@ -2,7 +2,6 @@
 <robot xmlns:xacro="http://www.ros.org/wiki/xacro">
   <!-- RM65机械臂接口定义宏 -->
-  <xacro:macro name="rm65_interfaces" params="name">
+  <xacro:macro name="rm65_interfaces" params="name enable_joint3:=false">
     <xacro:property name="prefix" value="${name + '_' if name else ''}"/>
-    <xacro:property name="enable_joint3" default="false"/>
     <!-- 机械臂关节接口定义 -->
     <joint name="${prefix}joint1">

Commit message: add lidar config

File: humanoid/Realman/aidal_description/xacro/components/woosh_agv.xacro (robot description, xacro)
@@ -329,4 +329,10 @@
 			<child link="lidar_link"/>
 		</joint>
+		<link name="lidar_frame"/>
+		<joint name="lidar_frame_joint" type="fixed">
+			<origin xyz="0 0 0.06"/>
+			<parent link="lidar_link"/>
+			<child link="lidar_frame"/>
+		</joint>
 		<link name="chassis_camera_link">
 			<visual>

File: manipulator/AgileX/piper_description/xacro/Piper.xacro (robot description, xacro)
@@ -18,5 +18,5 @@
       <visual>
         <geometry>
-          <mesh filename="file://$(find piper_description)/meshes/visual/base_link.obj"/>
+          <mesh filename="file://$(find piper_description)/meshes/visual/base_link.glb"/>
         </geometry>
       </visual>
@@ -36,5 +36,5 @@
       <visual>
         <geometry>
-          <mesh filename="file://$(find piper_description)/meshes/visual/link1.obj"/>
+          <mesh filename="file://$(find piper_description)/meshes/visual/link1.glb"/>
         </geometry>
       </visual>
@@ -61,5 +61,5 @@
       <visual>
         <geometry>
-          <mesh filename="file://$(find piper_description)/meshes/visual/link2.obj"/>
+          <mesh filename="file://$(find piper_description)/meshes/visual/link2.glb"/>
         </geometry>
       </visual>
