Commit message: nero机械臂更新，可更换末端执行器

File: manipulator/AgileX/nero_description/xacro/hand.xacro (robot description, xacro)
@@ -2,24 +2,18 @@
 <robot xmlns:xacro="http://www.ros.org/wiki/xacro">
     <xacro:macro name="Hand" params="type stand direction prefix standalone:=false">
-        <xacro:property name="actual_stand" value="${type if type != 'hand' else stand}"/>
+        <xacro:property name="brainco_dir"
+                        value="${1 if direction == 'left' else (-1 if direction == 'right' else direction)}"/>
         <xacro:property name="stand_link_name" value="${prefix}stand_adapter"/>
-        <xacro:property name="stand_origin_rpy" value="0 0 0"/>
-        <xacro:if value="${actual_stand == 'v1'}">
-            <xacro:property name="stand_origin_rpy" value="-1.57 -1.57 -1.57"/>
-        </xacro:if>
-        <xacro:if value="${actual_stand == 'v2'}">
-            <xacro:property name="stand_origin_rpy" value="-1.57 0 -1.57"/>
-        </xacro:if>
         <link name="${stand_link_name}">
             <visual>
-                <origin xyz="0 0 0" rpy="${stand_origin_rpy}"/>
+                <origin xyz="0 0 0" rpy="-1.57 -1.57 -1.57"/>
                 <geometry>
-                    <mesh filename="file://$(find nero_description)/meshes/${actual_stand if actual_stand == 'link8' else 'stand_' + actual_stand}.glb"/>
+                    <mesh filename="file://$(find nero_description)/meshes/stand_v1.glb"/>
                 </geometry>
             </visual>
             <collision>
-                <origin xyz="0 0 0" rpy="${stand_origin_rpy}"/>
+                <origin xyz="0 0 0" rpy="-1.57 -1.57 -1.57"/>
                 <geometry>
-                    <mesh filename="file://$(find nero_description)/meshes/${'link8' if actual_stand == 'link8' else 'stand_v1'}.glb"/>
+                    <mesh filename="file://$(find nero_description)/meshes/stand_v1.glb"/>
                 </geometry>
             </collision>
@@ -27,22 +21,40 @@
         <xacro:unless value="${standalone}">
             <joint name="${prefix}stand_joint" type="fixed">
-                <xacro:if value="${actual_stand == 'link8'}">
-                    <origin xyz="0.032 0 -0.0235" rpy="-1.5708 0 -1.5708"/>
-                </xacro:if>
-                <xacro:unless value="${actual_stand == 'link8'}">
-                    <origin xyz="0.033 0 -0.0235" rpy="0 0 0"/>
-                </xacro:unless>
+                <origin xyz="0.033 0 -0.0235" rpy="0 0 0"/>
                 <parent link="${prefix}link7"/>
                 <child link="${stand_link_name}"/>
             </joint>
         </xacro:unless>
-        <xacro:if value="${type == 'hand' or type == 'v1' or type == 'v2'}">
-            <xacro:include filename="$(find revo2_description)/xacro/revo_hand.xacro"/>
+        <xacro:if value="${'brainco' in type}">
+            <xacro:include filename="$(find brainco_description)/xacro/revo2.xacro"/>
             <joint name="${prefix}hand_connection_joint" type="fixed">
                 <origin xyz="0.01093 0 0" rpy="-1.57 3.14 -1.57"/>
                 <parent link="${stand_link_name}"/>
-                <child link="${prefix}hand_base_link"/>
+                <child link="${prefix}hand_base"/>
             </joint>
-            <xacro:RevoHand direction="${direction}"/>
+            <xacro:BrainCoHand name="${prefix[:-1] if prefix.endswith('_') else prefix}"
+                               direction="${brainco_dir}"
+                               use_flange="false"/>
+        </xacro:if>
+        <xacro:if value="${'ag2f90' in type}">
+            <xacro:include filename="$(find changingtek_description)/xacro/AG2F90-C.xacro"/>
+            <joint name="${prefix}hand_connection_joint" type="fixed">
+                <origin xyz="0.01093 0 0" rpy="-1.57 3.14 -1.57"/>
+                <parent link="${stand_link_name}"/>
+                <child link="${prefix}flange"/>
+            </joint>
+            <xacro:AG2F90-C name="${prefix[:-1] if prefix.endswith('_') else prefix}"
+                            use_flange="true"
+                            pad="default"/>
+        </xacro:if>
+        <xacro:if value="${'rg75' in type}">
+            <xacro:include filename="$(find jodell_description)/xacro/RG75-300.xacro"/>
+            <joint name="${prefix}hand_connection_joint" type="fixed">
+                <origin xyz="0.01093 0 0" rpy="-1.57 3.14 -1.57"/>
+                <parent link="${stand_link_name}"/>
+                <child link="${prefix}flange"/>
+            </joint>
+            <xacro:RG75-300 name="${prefix[:-1] if prefix.endswith('_') else prefix}"
+                            use_flange="true"/>
         </xacro:if>
     </xacro:macro>

File: manipulator/AgileX/nero_description/xacro/robot.xacro (robot description, xacro)
@@ -1,28 +1,66 @@
 <?xml version="1.0"?>
 <robot name="Nero" xmlns:xacro="http://www.ros.org/wiki/xacro">
-    <xacro:arg name="type" default="v1"/>
+    <xacro:arg name="type" default="dual"/>
     <xacro:arg name="collider" default="simple"/>
-    <xacro:arg name="direction" default="left"/>
     <xacro:arg name="scene" default="world"/>
-    <xacro:property name="prefix" value="$(arg direction)_"/>
     <xacro:property name="type_arg" value="$(arg type)"/>
-    <xacro:property name="is_stand_only" value="${'stand' in type_arg}"/>
-    <xacro:property name="is_arm_only" value="${type_arg == 'arm_only'}"/>
     <xacro:property name="stand_type" value="v1"/>
-    <xacro:if value="${'v2' in type_arg}"><xacro:property name="stand_type" value="v2"/></xacro:if>
-    <xacro:if value="${'link8' in type_arg}"><xacro:property name="stand_type" value="link8"/></xacro:if>
+    <xacro:property name="selected_arm_config" value="left"/>
+    <xacro:property name="selected_gripper_type" value="none"/>
+    <xacro:property name="selected_arm_style" value="default"/>
+    <xacro:if value="${type_arg == 'left'}">
+        <xacro:property name="selected_arm_config" value="left"/>
+    </xacro:if>
+    <xacro:if value="${type_arg == 'right'}">
+        <xacro:property name="selected_arm_config" value="right"/>
+    </xacro:if>
+    <xacro:if value="${type_arg == 'dual'}">
+        <xacro:property name="selected_arm_config" value="dual"/>
+        <xacro:property name="selected_gripper_type" value="none"/>
+        <xacro:property name="selected_arm_style" value="dual_config"/>
+    </xacro:if>
+    <xacro:if value="${type_arg == 'brainco'}">
+        <xacro:property name="selected_arm_config" value="left"/>
+        <xacro:property name="selected_gripper_type" value="brainco"/>
+    </xacro:if>
+    <xacro:if value="${type_arg == 'ag2f90'}">
+        <xacro:property name="selected_arm_config" value="left"/>
+        <xacro:property name="selected_gripper_type" value="ag2f90"/>
+    </xacro:if>
+    <xacro:if value="${type_arg == 'rg75'}">
+        <xacro:property name="selected_arm_config" value="left"/>
+        <xacro:property name="selected_gripper_type" value="rg75"/>
+    </xacro:if>
+    <xacro:if value="${type_arg == 'dual_brainco'}">
+        <xacro:property name="selected_arm_config" value="dual"/>
+        <xacro:property name="selected_gripper_type" value="brainco"/>
+        <xacro:property name="selected_arm_style" value="dual_config"/>
+    </xacro:if>
+    <xacro:if value="${type_arg == 'dual_ag2f90'}">
+        <xacro:property name="selected_arm_config" value="dual"/>
+        <xacro:property name="selected_gripper_type" value="ag2f90"/>
+        <xacro:property name="selected_arm_style" value="dual_config"/>
+    </xacro:if>
+    <xacro:if value="${type_arg == 'dual_rg75'}">
+        <xacro:property name="selected_arm_config" value="dual"/>
+        <xacro:property name="selected_gripper_type" value="rg75"/>
+        <xacro:property name="selected_arm_style" value="dual_config"/>
+    </xacro:if>
+    <xacro:if value="${type_arg == 'stand'}">
+        <xacro:property name="selected_arm_config" value="stand_only"/>
+    </xacro:if>
     <xacro:include filename="$(find nero_description)/xacro/nero.xacro"/>
     <xacro:if value="${'$(arg scene)' == 'world'}">
         <link name="world"/>
     </xacro:if>
-    <xacro:if value="${is_stand_only}">
+    <xacro:if value="${selected_arm_config == 'stand_only'}">
         <xacro:include filename="$(find nero_description)/xacro/hand.xacro"/>
-        <xacro:Hand type="hand" stand="${stand_type}" direction="$(arg direction)" prefix="${prefix}" standalone="true"/>
+        <xacro:Hand type="brainco" stand="${stand_type}" direction="left" prefix="left_" standalone="true"/>
         <joint name="world_fixed" type="fixed">
             <parent link="world"/>
-            <child link="${prefix}stand_adapter"/>
+            <child link="left_stand_adapter"/>
         </joint>
     </xacro:if>
-    <xacro:unless value="${is_stand_only}">
+    <xacro:if value="${selected_arm_config == 'left'}">
         <link name="base_link"/>
         <xacro:if value="${'$(arg scene)' == 'world'}">
@@ -30,14 +68,50 @@
                 <parent link="world"/>
                 <child link="base_link"/>
-                <origin xyz="0 0 0" rpy="0 0 0"/>
             </joint>
         </xacro:if>
-        <joint name="${prefix}base_joint" type="fixed">
+        <joint name="left_base_joint" type="fixed">
             <parent link="base_link"/>
-            <child link="${prefix}base_link"/>
+            <child link="left_base_link"/>
             <origin xyz="0 0 0" rpy="0 0 3.14159"/>
         </joint>
-        <xacro:Nero type="${type_arg}" stand="${stand_type}" direction="$(arg direction)" prefix="${prefix}"
-                    is_arm_only="${is_arm_only}"/>
-    </xacro:unless>
+        <xacro:Nero type="${selected_gripper_type}" stand="${stand_type}" direction="left" prefix="left_"
+                    is_arm_only="${selected_gripper_type == 'none'}"/>
+    </xacro:if>
+    <xacro:if value="${selected_arm_config == 'right'}">
+        <link name="base_link"/>
+        <xacro:if value="${'$(arg scene)' == 'world'}">
+            <joint name="world_fixed" type="fixed">
+                <parent link="world"/>
+                <child link="base_link"/>
+            </joint>
+        </xacro:if>
+        <joint name="right_base_joint" type="fixed">
+            <parent link="base_link"/>
+            <child link="right_base_link"/>
+            <origin xyz="0 0 0" rpy="0 0 3.14159"/>
+        </joint>
+        <xacro:Nero type="${selected_gripper_type}" stand="${stand_type}" direction="right" prefix="right_"
+                    is_arm_only="${selected_gripper_type == 'none'}"/>
+    </xacro:if>
+    <xacro:if value="${selected_arm_config == 'dual'}">
+        <link name="base_link"/>
+        <xacro:if value="${'$(arg scene)' == 'world'}">
+            <joint name="world_fixed" type="fixed">
+                <parent link="world"/>
+                <child link="base_link"/>
+            </joint>
+        </xacro:if>
+        <joint name="left_arm_base_joint" type="fixed">
+            <parent link="base_link"/> <child link="left_base_link"/>
+            <origin xyz="0.0 0.1 0" rpy="1.5708 0 3.14159"/>
+        </joint>
+        <joint name="right_arm_base_joint" type="fixed">
+            <parent link="base_link"/> <child link="right_base_link"/>
+            <origin xyz="0.0 -0.1 0" rpy="-1.5708 0 -3.14159"/>
+        </joint>
+        <xacro:Nero type="${selected_gripper_type}" stand="${stand_type}" direction="left" prefix="left_"
+                    is_arm_only="${selected_gripper_type == 'none'}"/>
+        <xacro:Nero type="${selected_gripper_type}" stand="${stand_type}" direction="right" prefix="right_"
+                    is_arm_only="${selected_gripper_type == 'none'}"/>
+    </xacro:if>
 </robot>

File: manipulator/AgileX/nero_description/xacro/ros2_control/nero.ros2_control.xacro (robot description, xacro)
@@ -1,5 +1,49 @@
 <?xml version="1.0"?>
 <robot xmlns:xacro="http://www.ros.org/wiki/xacro">
-    <xacro:macro name="nero_system" params="name prefix ros2_control_hardware_type">
+    <xacro:macro name="nero_interfaces" params="prefix">
+        <joint name="${prefix}joint1">
+            <command_interface name="position"/>
+            <state_interface name="position"><param name="initial_value">0.0</param></state_interface>
+            <state_interface name="velocity"/>
+            <state_interface name="effort"/>
+        </joint>
+        <joint name="${prefix}joint2">
+            <command_interface name="position"/>
+            <state_interface name="position"><param name="initial_value">0.0</param></state_interface>
+            <state_interface name="velocity"/>
+            <state_interface name="effort"/>
+        </joint>
+        <joint name="${prefix}joint3">
+            <command_interface name="position"/>
+            <state_interface name="position"><param name="initial_value">0.0</param></state_interface>
+            <state_interface name="velocity"/>
+            <state_interface name="effort"/>
+        </joint>
+        <joint name="${prefix}joint4">
+            <command_interface name="position"/>
+            <state_interface name="position"><param name="initial_value">0.0</param></state_interface>
+            <state_interface name="velocity"/>
+            <state_interface name="effort"/>
+        </joint>
+        <joint name="${prefix}joint5">
+            <command_interface name="position"/>
+            <state_interface name="position"><param name="initial_value">0.0</param></state_interface>
+            <state_interface name="velocity"/>
+            <state_interface name="effort"/>
+        </joint>
+        <joint name="${prefix}joint6">
+            <command_interface name="position"/>
+            <state_interface name="position"><param name="initial_value">0.0</param></state_interface>
+            <state_interface name="velocity"/>
+            <state_interface name="effort"/>
+        </joint>
+        <joint name="${prefix}joint7">
+            <command_interface name="position"/>
+            <state_interface name="position"><param name="initial_value">0.0</param></state_interface>
+            <state_interface name="velocity"/>
+            <state_interface name="effort"/>
+        </joint>
+    </xacro:macro>
+    <xacro:macro name="nero_system" params="name arm_config ros2_control_hardware_type">
         <ros2_control name="${name}" type="system">
             <hardware>
@@ -16,21 +60,14 @@
                 </xacro:if>
             </hardware>
-            <xacro:macro name="configure_joint" params="joint_name initial_pos:=0.0">
-                <joint name="${joint_name}">
-                    <command_interface name="position"/>
-                    <state_interface name="position">
-                        <param name="initial_value">${initial_pos}</param>
-                    </state_interface>
-                    <state_interface name="velocity"/>
-                    <state_interface name="effort"/>
-                </joint>
-            </xacro:macro>
-            <xacro:configure_joint joint_name="${prefix}joint1"/>
-            <xacro:configure_joint joint_name="${prefix}joint2"/>
-            <xacro:configure_joint joint_name="${prefix}joint3"/>
-            <xacro:configure_joint joint_name="${prefix}joint4"/>
-            <xacro:configure_joint joint_name="${prefix}joint5"/>
-            <xacro:configure_joint joint_name="${prefix}joint6"/>
-            <xacro:configure_joint joint_name="${prefix}joint7"/>
+            <xacro:if value="${arm_config == 'dual'}">
+                <xacro:nero_interfaces prefix="left_"/>
+                <xacro:nero_interfaces prefix="right_"/>
+            </xacro:if>
+            <xacro:if value="${arm_config == 'left'}">
+                <xacro:nero_interfaces prefix="left_"/>
+            </xacro:if>
+            <xacro:if value="${arm_config == 'right'}">
+                <xacro:nero_interfaces prefix="right_"/>
+            </xacro:if>
         </ros2_control>
     </xacro:macro>

File: manipulator/AgileX/nero_description/xacro/ros2_control/robot.xacro (robot description, xacro)
@@ -2,10 +2,7 @@
 <robot xmlns:xacro="http://www.ros.org/wiki/xacro" name="nero_robot">
     <xacro:arg name="ros2_control_hardware_type" default="mock_components" />
-    <xacro:arg name="type" default="v1"/>
-    <xacro:arg name="direction" default="left"/>
+    <xacro:arg name="type" default="dual"/>
     <xacro:arg name="gazebo" default="false" />
-    <xacro:property name="prefix" value="$(arg direction)_"/>
-    <xacro:property name="type_arg" value="$(arg type)"/>
-    <xacro:property name="is_arm_only" value="${type_arg == 'arm_only'}"/>
+    <xacro:property name="selected_arm_config" value="$(arg type)"/>
     <xacro:include filename="$(find nero_description)/xacro/nero.xacro"/>
     <link name="world"/>
@@ -13,21 +10,50 @@
         <parent link="world"/>
         <child link="base_link"/>
+        <origin/>
     </joint>
     <link name="base_link"/>
-    <joint name="${prefix}base_joint" type="fixed">
-        <parent link="base_link"/>
-        <child link="${prefix}base_link"/>
-        <origin xyz="0 0 0" rpy="0 0 3.14159"/>
-    </joint>
-    <xacro:Nero type="$(arg type)" stand="v1" direction="$(arg direction)" prefix="${prefix}" is_arm_only="${is_arm_only}"/>
+    <xacro:if value="${selected_arm_config == 'dual'}">
+        <joint name="left_arm_base_joint" type="fixed">
+            <parent link="base_link"/> <child link="left_base_link"/>
+            <origin xyz="0.0 0.1 0" rpy="1.5708 0 3.14159"/>
+        </joint>
+        <xacro:Nero type="none" stand="v1" direction="left" prefix="left_" is_arm_only="true"/>
+        <joint name="right_arm_base_joint" type="fixed">
+            <parent link="base_link"/> <child link="right_base_link"/>
+            <origin xyz="0.0 -0.1 0" rpy="-1.5708 0 -3.14159"/>
+        </joint>
+        <xacro:Nero type="none" stand="v1" direction="right" prefix="right_" is_arm_only="true"/>
+    </xacro:if>
+    <xacro:if value="${selected_arm_config == 'left'}">
+        <joint name="left_base_joint" type="fixed">
+            <parent link="base_link"/> <child link="left_base_link"/>
+            <origin xyz="0 0 0" rpy="0 0 3.14159"/>
+        </joint>
+        <xacro:Nero type="none" stand="v1" direction="left" prefix="left_" is_arm_only="true"/>
+    </xacro:if>
+    <xacro:if value="${selected_arm_config == 'right'}">
+        <joint name="right_base_joint" type="fixed">
+            <parent link="base_link"/> <child link="right_base_link"/>
+            <origin xyz="0 0 0" rpy="0 0 3.14159"/>
+        </joint>
+        <xacro:Nero type="none" stand="v1" direction="right" prefix="right_" is_arm_only="true"/>
+    </xacro:if>
     <xacro:include filename="$(find nero_description)/xacro/ros2_control/nero.ros2_control.xacro" />
     <xacro:nero_system
             name="NeroSystem"
-            prefix="${prefix}"
+            arm_config="${selected_arm_config}"
             ros2_control_hardware_type="$(arg ros2_control_hardware_type)"/>
     <xacro:if value="$(arg gazebo)">
         <gazebo>
             <plugin filename="gz_ros2_control-system" name="gz_ros2_control::GazeboSimROS2ControlPlugin">
-                <parameters>$(find nero_description)/config/ros2_control/nero_controllers.yaml</parameters>
+                <xacro:if value="${selected_arm_config == 'dual'}">
+                    <parameters>$(find nero_description)/config/ros2_control/dual_ros2_controllers.yaml</parameters>
+                </xacro:if>
+                <xacro:if value="${selected_arm_config == 'left'}">
+                    <parameters>$(find nero_description)/config/ros2_control/ros2_controllers.yaml</parameters>
+                </xacro:if>
+                <xacro:if value="${selected_arm_config == 'right'}">
+                    <parameters>$(find nero_description)/config/ros2_control/ros2_controllers.yaml</parameters>
+                </xacro:if>
             </plugin>
         </gazebo>
