Commit message: add nero

File: manipulator/AgileX/nero_description/xacro/Nero.xacro (robot description, xacro)
@@ -1,196 +1,204 @@
 <?xml version="1.0" encoding="utf-8"?>
 <robot xmlns:xacro="http://www.ros.org/wiki/xacro">
-  <xacro:macro name="Nero" params="name">
-    <xacro:property name="prefix" value="${name + '_' if name else ''}"/>
-    <link name="${prefix}base_link">
-      <inertial>
-        <origin xyz="-0.00319465997 -0.00005467608 0.04321758463" rpy="0 0 0"/>
-        <mass value="1.06458435"/>
-        <inertia ixx="0.00102659855152" ixy="0.00000186219753" ixz="-0.00000295298037" iyy="0.00114399299508" iyz="-0.00000078763492" izz="0.00090872933022"/>
-      </inertial>
-      <visual>
-        <geometry>
-          <mesh filename="file://$(find nero_description)/meshes/nero/dae/base_link.dae"/>
-        </geometry>
-      </visual>
-      <collision>
-        <geometry>
-          <mesh filename="file://$(find nero_description)/meshes/nero/base_link.stl"/>
-        </geometry>
-      </collision>
-    </link>
-    <link name="${prefix}link1">
-      <inertial>
-        <origin xyz="-0.00076810578 -0.00005718031 -0.00686372765" rpy="0 0 0"/>
-        <mass value="0.76710504"/>
-        <inertia ixx="0.00066689512233" ixy="0.00000273938306" ixz="0.00001463284987" iyy="0.00054501235592" iyz="0.00000183168344" izz="0.00051509465737"/>
-      </inertial>
-      <visual>
-        <geometry>
-          <mesh filename="file://$(find nero_description)/meshes/nero/dae/link1.dae"/>
-        </geometry>
-      </visual>
-      <collision>
-        <geometry>
-          <mesh filename="file://$(find nero_description)/meshes/nero/link1.stl"/>
-        </geometry>
-      </collision>
-    </link>
-    <joint name="${prefix}joint1" type="revolute">
-      <origin xyz="0 0 0.138" rpy="0 0 0"/>
-      <parent link="${prefix}base_link"/>
-      <child link="${prefix}link1"/>
-      <axis xyz="0 0 1"/>
-      <limit lower="-2.70526" upper="2.70526" effort="100" velocity="5"/>
-    </joint>
-    <link name="${prefix}link2">
-      <inertial>
-        <origin xyz="0.00079686657 -0.07890325930 0.00111849422" rpy="0 0 0"/>
-        <mass value="0.69381908"/>
-        <inertia ixx="0.00201093857656" ixy="-0.00002399426785" ixz="-0.00000072824714" iyy="0.00063544232555" iyz="0.00005831284343" izz="0.00181943989593"/>
-      </inertial>
-      <visual>
-        <geometry>
-          <mesh filename="file://$(find nero_description)/meshes/nero/dae/link2.dae"/>
-        </geometry>
-      </visual>
-      <collision>
-        <geometry>
-          <mesh filename="file://$(find nero_description)/meshes/nero/link2.stl"/>
-        </geometry>
-      </collision>
-    </link>
-    <joint name="${prefix}joint2" type="revolute">
-      <origin xyz="0 0 0" rpy="1.5707963  3.1415926 0"/>
-      <parent link="${prefix}link1"/>
-      <child link="${prefix}link2"/>
-      <axis xyz="0 0 1"/>
-      <limit lower="-1.74" upper="1.74" effort="100" velocity="5"/>
-    </joint>
-    <link name="${prefix}link3">
-      <inertial>
-        <origin xyz="0.00014513363 -0.00121378766 -0.04861136795" rpy="0 0 0"/>
-        <mass value="0.67246544"/>
-        <inertia ixx="0.00343229961910" ixy="-0.00000026976739" ixz="0.00000305078107" iyy="0.00338662526897" iyz="-0.00003550220027" izz="0.00028853579710"/>
-      </inertial>
-      <visual>
-        <geometry>
-          <mesh filename="file://$(find nero_description)/meshes/nero/dae/link3.dae"/>
-        </geometry>
-      </visual>
-      <collision>
-        <geometry>
-          <mesh filename="file://$(find nero_description)/meshes/nero/link3.stl"/>
-        </geometry>
-      </collision>
-    </link>
-    <joint name="${prefix}joint3" type="revolute">
-      <origin xyz="0 -0.31 0" rpy="-1.5707963  0 3.1415926926"/>
-      <parent link="${prefix}link2"/>
-      <child link="${prefix}link3"/>
-      <axis xyz="0 0 1"/>
-      <limit lower="-2.75" upper="2.75" effort="100" velocity="5"/>
-    </joint>
-    <link name="${prefix}link4">
-      <inertial>
-        <origin xyz="-0.00031334623 -0.05675192422 0.00076056133" rpy="0 0 0"/>
-        <mass value="0.48451414"/>
-        <inertia ixx="0.00050386693505" ixy="-0.00000529675237" ixz="0.00000006134740" iyy="0.00023502068202" iyz="0.00001815932566" izz="0.00040149523118"/>
-      </inertial>
-      <visual>
-        <geometry>
-          <mesh filename="file://$(find nero_description)/meshes/nero/dae/link4.dae"/>
-        </geometry>
-      </visual>
-      <collision>
-        <geometry>
-          <mesh filename="file://$(find nero_description)/meshes/nero/link4.stl"/>
-        </geometry>
-      </collision>
-    </link>
-    <joint name="${prefix}joint4" type="revolute">
-      <origin xyz="0 0 0" rpy="-1.5707963  0 3.1415926926"/>
-      <parent link="${prefix}link3"/>
-      <child link="${prefix}link4"/>
-      <axis xyz="0 0 1"/>
-      <limit lower="-1.01" upper="2.14" effort="100" velocity="5"/>
-    </joint>
-    <link name="${prefix}link5">
-      <inertial>
-        <origin xyz="0.00265591357 0.00201195753 -0.11620855434" rpy="0 0 0"/>
-        <mass value="0.58368405"/>
-        <inertia ixx="0.00089537686723" ixy="0.00000648218232" ixz="-0.00001463346849" iyy="0.00085866122972" iyz="-0.00004035185637" izz="0.00021774946532"/>
-      </inertial>
-      <visual>
-        <geometry>
-          <mesh filename="file://$(find nero_description)/meshes/nero/dae/link5.dae"/>
-        </geometry>
-      </visual>
-      <collision>
-        <geometry>
-          <mesh filename="file://$(find nero_description)/meshes/nero/link5.stl"/>
-        </geometry>
-      </collision>
-    </link>
-    <joint name="${prefix}joint5" type="revolute">
-      <origin xyz="0 -0.27001 0" rpy="1.5707963  -1.5707963  0"/>
-      <parent link="${prefix}link4"/>
-      <child link="${prefix}link5"/>
-      <axis xyz="0 0 1"/>
-      <limit lower="-2.75" upper="2.75" effort="100" velocity="5"/>
-    </joint>
-    <link name="${prefix}link6">
-      <inertial>
-        <origin xyz="0.00009501505 0.00107831174 -0.00019110990" rpy="0 0 0"/>
-        <mass value="0.3140406"/>
-        <inertia ixx="0.00006027211661" ixy="-0.00000024650903" ixz="0.00000015701294" iyy="0.00004699514792" iyz="0.00000004170875" izz="0.00005756771792"/>
-      </inertial>
-      <visual>
-        <geometry>
-          <mesh filename="file://$(find nero_description)/meshes/nero/dae/link6.dae"/>
-        </geometry>
-      </visual>
-      <collision>
-        <geometry>
-          <mesh filename="file://$(find nero_description)/meshes/nero/link6.stl"/>
-        </geometry>
-      </collision>
-    </link>
-    <joint name="${prefix}joint6" type="revolute">
-      <origin xyz="0 0 0" rpy="1.5707963  -1.5707963  0"/>
-      <parent link="${prefix}link5"/>
-      <child link="${prefix}link6"/>
-      <axis xyz="0 0 1"/>
-      <limit lower="-0.73" upper="0.95" effort="100" velocity="5"/>
-    </joint>
-    <link name="${prefix}link7">
-      <inertial>
-        <origin xyz="-0.00014000 -0.00010000 -0.00275000" rpy="0 0 0"/>
-        <mass value="0.000001"/>
-        <inertia ixx="1.1000000000000001e-07" ixy="0" ixz="0" iyy="1.1000000000000001e-07" iyz="0" izz="1.9999999999999999e-07"/>
-      </inertial>
-      <visual>
-        <geometry>
-          <mesh filename="file://$(find nero_description)/meshes/nero/dae/link7.dae"/>
-        </geometry>
-      </visual>
-      <collision>
-        <geometry>
-          <mesh filename="file://$(find nero_description)/meshes/nero/link7.stl"/>
-        </geometry>
-      </collision>
-    </link>
-    <joint name="${prefix}joint7" type="revolute">
-      <origin xyz="0 -0.0235 0" rpy="1.5707963 0 0"/>
-      <parent link="${prefix}link6"/>
-      <child link="${prefix}link7"/>
-      <axis xyz="0 0 1"/>
-      <limit lower="-1.5707963" upper="1.5707963" effort="100" velocity="5"/>
-    </joint>
-    <link name="${prefix}tcp"/>
-    <joint name="${prefix}tcp_joint" type="fixed">
-      <parent link="${prefix}link7"/>
-      <child link="${prefix}tcp"/>
-    </joint>
-  </xacro:macro>
+    <xacro:macro name="Nero" params="name">
+        <xacro:property name="prefix" value="${name + '_' if name else ''}"/>
+        <link name="${prefix}base_link">
+            <inertial>
+                <origin xyz="-0.00319465997 -0.00005467608 0.04321758463"/>
+                <mass value="1.06458435"/>
+                <inertia ixx="0.00102659855152" ixy="0.00000186219753" ixz="-0.00000295298037" iyy="0.00114399299508"
+                         iyz="-0.00000078763492" izz="0.00090872933022"/>
+            </inertial>
+            <visual>
+                <geometry>
+                    <mesh filename="file://$(find nero_description)/meshes/base_link.glb"/>
+                </geometry>
+            </visual>
+            <collision>
+                <geometry>
+                    <mesh filename="file://$(find nero_description)/meshes/base_link.glb"/>
+                </geometry>
+            </collision>
+        </link>
+        <link name="${prefix}link1">
+            <inertial>
+                <origin xyz="-0.00076810578 -0.00005718031 -0.00686372765"/>
+                <mass value="0.76710504"/>
+                <inertia ixx="0.00066689512233" ixy="0.00000273938306" ixz="0.00001463284987" iyy="0.00054501235592"
+                         iyz="0.00000183168344" izz="0.00051509465737"/>
+            </inertial>
+            <visual>
+                <geometry>
+                    <mesh filename="file://$(find nero_description)/meshes/link1.glb"/>
+                </geometry>
+            </visual>
+            <collision>
+                <geometry>
+                    <mesh filename="file://$(find nero_description)/meshes/link1.glb"/>
+                </geometry>
+            </collision>
+        </link>
+        <joint name="${prefix}joint1" type="revolute">
+            <origin xyz="0 0 0.138"/>
+            <parent link="${prefix}base_link"/>
+            <child link="${prefix}link1"/>
+            <axis xyz="0 0 1"/>
+            <limit lower="-2.70526" upper="2.70526" effort="100" velocity="5"/>
+        </joint>
+        <link name="${prefix}link2">
+            <inertial>
+                <origin xyz="0.00079686657 -0.07890325930 0.00111849422"/>
+                <mass value="0.69381908"/>
+                <inertia ixx="0.00201093857656" ixy="-0.00002399426785" ixz="-0.00000072824714" iyy="0.00063544232555"
+                         iyz="0.00005831284343" izz="0.00181943989593"/>
+            </inertial>
+            <visual>
+                <geometry>
+                    <mesh filename="file://$(find nero_description)/meshes/link2.glb"/>
+                </geometry>
+            </visual>
+            <collision>
+                <geometry>
+                    <mesh filename="file://$(find nero_description)/meshes/link2.glb"/>
+                </geometry>
+            </collision>
+        </link>
+        <joint name="${prefix}joint2" type="revolute">
+            <origin  rpy="1.5707963  3.1415926 0"/>
+            <parent link="${prefix}link1"/>
+            <child link="${prefix}link2"/>
+            <axis xyz="0 0 1"/>
+            <limit lower="-1.74" upper="1.74" effort="100" velocity="5"/>
+        </joint>
+        <link name="${prefix}link3">
+            <inertial>
+                <origin xyz="0.00014513363 -0.00121378766 -0.04861136795"/>
+                <mass value="0.67246544"/>
+                <inertia ixx="0.00343229961910" ixy="-0.00000026976739" ixz="0.00000305078107" iyy="0.00338662526897"
+                         iyz="-0.00003550220027" izz="0.00028853579710"/>
+            </inertial>
+            <visual>
+                <geometry>
+                    <mesh filename="file://$(find nero_description)/meshes/link3.glb"/>
+                </geometry>
+            </visual>
+            <collision>
+                <geometry>
+                    <mesh filename="file://$(find nero_description)/meshes/link3.glb"/>
+                </geometry>
+            </collision>
+        </link>
+        <joint name="${prefix}joint3" type="revolute">
+            <origin xyz="0 -0.31 0" rpy="-1.5707963  0 3.1415926926"/>
+            <parent link="${prefix}link2"/>
+            <child link="${prefix}link3"/>
+            <axis xyz="0 0 1"/>
+            <limit lower="-2.75" upper="2.75" effort="100" velocity="5"/>
+        </joint>
+        <link name="${prefix}link4">
+            <inertial>
+                <origin xyz="-0.00031334623 -0.05675192422 0.00076056133"/>
+                <mass value="0.48451414"/>
+                <inertia ixx="0.00050386693505" ixy="-0.00000529675237" ixz="0.00000006134740" iyy="0.00023502068202"
+                         iyz="0.00001815932566" izz="0.00040149523118"/>
+            </inertial>
+            <visual>
+                <geometry>
+                    <mesh filename="file://$(find nero_description)/meshes/link4.glb"/>
+                </geometry>
+            </visual>
+            <collision>
+                <geometry>
+                    <mesh filename="file://$(find nero_description)/meshes/link4.glb"/>
+                </geometry>
+            </collision>
+        </link>
+        <joint name="${prefix}joint4" type="revolute">
+            <origin  rpy="-1.5707963  0 3.1415926926"/>
+            <parent link="${prefix}link3"/>
+            <child link="${prefix}link4"/>
+            <axis xyz="0 0 1"/>
+            <limit lower="-1.01" upper="2.14" effort="100" velocity="5"/>
+        </joint>
+        <link name="${prefix}link5">
+            <inertial>
+                <origin xyz="0.00265591357 0.00201195753 -0.11620855434"/>
+                <mass value="0.58368405"/>
+                <inertia ixx="0.00089537686723" ixy="0.00000648218232" ixz="-0.00001463346849" iyy="0.00085866122972"
+                         iyz="-0.00004035185637" izz="0.00021774946532"/>
+            </inertial>
+            <visual>
+                <geometry>
+                    <mesh filename="file://$(find nero_description)/meshes/link5.glb"/>
+                </geometry>
+            </visual>
+            <collision>
+                <geometry>
+                    <mesh filename="file://$(find nero_description)/meshes/link5.glb"/>
+                </geometry>
+            </collision>
+        </link>
+        <joint name="${prefix}joint5" type="revolute">
+            <origin xyz="0 -0.27001 0" rpy="1.5707963  -1.5707963  0"/>
+            <parent link="${prefix}link4"/>
+            <child link="${prefix}link5"/>
+            <axis xyz="0 0 1"/>
+            <limit lower="-2.75" upper="2.75" effort="100" velocity="5"/>
+        </joint>
+        <link name="${prefix}link6">
+            <inertial>
+                <origin xyz="0.00009501505 0.00107831174 -0.00019110990"/>
+                <mass value="0.3140406"/>
+                <inertia ixx="0.00006027211661" ixy="-0.00000024650903" ixz="0.00000015701294" iyy="0.00004699514792"
+                         iyz="0.00000004170875" izz="0.00005756771792"/>
+            </inertial>
+            <visual>
+                <geometry>
+                    <mesh filename="file://$(find nero_description)/meshes/link6.glb"/>
+                </geometry>
+            </visual>
+            <collision>
+                <geometry>
+                    <mesh filename="file://$(find nero_description)/meshes/link6.glb"/>
+                </geometry>
+            </collision>
+        </link>
+        <joint name="${prefix}joint6" type="revolute">
+            <origin  rpy="1.5707963  -1.5707963  0"/>
+            <parent link="${prefix}link5"/>
+            <child link="${prefix}link6"/>
+            <axis xyz="0 0 1"/>
+            <limit lower="-0.73" upper="0.95" effort="100" velocity="5"/>
+        </joint>
+        <link name="${prefix}link7">
+            <inertial>
+                <origin xyz="-0.00014000 -0.00010000 -0.00275000"/>
+                <mass value="0.000001"/>
+                <inertia ixx="1.1000000000000001e-07" ixy="0" ixz="0" iyy="1.1000000000000001e-07" iyz="0"
+                         izz="1.9999999999999999e-07"/>
+            </inertial>
+            <visual>
+                <geometry>
+                    <mesh filename="file://$(find nero_description)/meshes/link7.glb"/>
+                </geometry>
+            </visual>
+            <collision>
+                <geometry>
+                    <mesh filename="file://$(find nero_description)/meshes/link7.glb"/>
+                </geometry>
+            </collision>
+        </link>
+        <joint name="${prefix}joint7" type="revolute">
+            <origin xyz="0 -0.0235 0" rpy="1.5707963 0 0"/>
+            <parent link="${prefix}link6"/>
+            <child link="${prefix}link7"/>
+            <axis xyz="0 0 1"/>
+            <limit lower="-1.5707963" upper="1.5707963" effort="100" velocity="5"/>
+        </joint>
+        <link name="${prefix}tcp"/>
+        <joint name="${prefix}tcp_joint" type="fixed">
+            <parent link="${prefix}link7"/>
+            <child link="${prefix}tcp"/>
+        </joint>
+    </xacro:macro>
 </robot>
