Commit message: add nero

File: manipulator/AgileX/nero_description/xacro/eefs.xacro (robot description, xacro)
@@ -1,106 +1,108 @@
 <?xml version="1.0"?>
 <robot xmlns:xacro="http://www.ros.org/wiki/xacro">
-  <xacro:include filename="$(find piper_description)/xacro/components/gripper.xacro"/>
-  <xacro:include filename="$(find brainco_description)/xacro/revo2.xacro"/>
-  <xacro:macro name="NeroEndEffectors" params="name type:='gripper'">
-    <xacro:property name="prefix" value="${name + '_' if name else ''}"/>
-    <xacro:property name="hand_name" value="${name + '_hand' if name else 'hand'}"/>
-    <xacro:property name="ee_type" value="${type if type else 'gripper'}"/>
-    <xacro:property name="use_gripper" value="${ee_type == 'gripper'}"/>
-    <xacro:property name="use_revo2" value="${ee_type == 'revo2'}"/>
-    <xacro:property name="use_none" value="${ee_type == 'none'}"/>
-    <xacro:if value="${use_gripper}">
-      <link name="${prefix}gripper_flange">
-        <inertial>
-          <origin xyz="0.000253201 -0.000322696 -0.010082901" rpy="0 0 0"/>
-          <mass value="0.04771096"/>
-          <inertia ixx="3.614107e-05" ixy="0" ixz="0" iyy="1.7824164e-05" iyz="0" izz="2.695944e-05"/>
-        </inertial>
-        <visual>
-          <geometry>
-            <mesh filename="file://$(find nero_description)/meshes/gripper/dae/gripper_flange.dae"/>
-          </geometry>
-        </visual>
-        <collision>
-          <geometry>
-            <mesh filename="file://$(find nero_description)/meshes/gripper/gripper_flange.stl"/>
-          </geometry>
-        </collision>
-      </link>
-      <joint name="${prefix}gripper_flange_joint" type="fixed">
-        <origin xyz="0.031 0 -0.0235" rpy="-1.5708 0 -1.5708"/>
-        <parent link="${prefix}tcp"/>
-        <child link="${prefix}gripper_flange"/>
-      </joint>
-      <link name="${prefix}gripper_base">
-        <inertial>
-          <origin xyz="-0.000183807162235591 8.05033155577911E-05 0.0321436689908876"/>
-          <mass value="0.45"/>
-          <inertia ixx="0.00092934" ixy="0.00000034" ixz="-0.00000738" iyy="0.00071447" iyz="0.00000005"
-                   izz="0.00039442"/>
-        </inertial>
-        <visual>
-          <geometry>
-            <mesh filename="file://$(find piper_description)/meshes/gripper/gripper_base.glb"/>
-          </geometry>
-        </visual>
-        <collision>
-          <geometry>
-            <mesh filename="file://$(find piper_description)/meshes/gripper/gripper_base.glb"/>
-          </geometry>
-        </collision>
-      </link>
-      <joint name="${prefix}gripper_base_joint" type="fixed">
-        <origin xyz="0 0 0.006"/>
-        <parent link="${prefix}gripper_flange"/>
-        <child link="${prefix}gripper_base"/>
-      </joint>
-      <xacro:agx_gripper
-          prefix="${prefix}"
-          parent_link="${prefix}gripper_base"
-          xyz="0 0 0"/>
-    </xacro:if>
-    <xacro:if value="${use_revo2}">
-      <link name="${prefix}revo2_flange">
-        <inertial>
-          <origin xyz="0.000253201 -0.000322696 -0.010082901" rpy="0 0 0"/>
-          <mass value="0.04771096"/>
-          <inertia ixx="3.614107e-05" ixy="0" ixz="0" iyy="1.7824164e-05" iyz="0" izz="2.695944e-05"/>
-        </inertial>
-        <visual>
-          <geometry>
-            <mesh filename="file://$(find nero_description)/meshes/nero/dae/revo2_flange.dae"/>
-          </geometry>
-        </visual>
-        <collision>
-          <geometry>
-            <mesh filename="file://$(find nero_description)/meshes/nero/revo2_flange.stl"/>
-          </geometry>
-        </collision>
-      </link>
-      <joint name="${prefix}revo2_flange_joint" type="fixed">
-        <origin xyz="0.031 0 -0.0235" rpy="-1.5708 0 -1.5708"/>
-        <parent link="${prefix}tcp"/>
-        <child link="${prefix}revo2_flange"/>
-      </joint>
-      <xacro:BrainCoHand name="${hand_name}" use_flange="false"/>
-      <joint name="${prefix}hand_base_joint" type="fixed">
-        <origin xyz="0 0 0.012" rpy="0 0 3.1415926"/>
-        <parent link="${prefix}revo2_flange"/>
-        <child link="${hand_name}_hand_base"/>
-      </joint>
-      <link name="${prefix}gripper_center"/>
-      <joint name="${prefix}gripper_center_fixed" type="fixed">
-        <parent link="${prefix}tcp"/>
-        <child link="${prefix}gripper_center"/>
-      </joint>
-    </xacro:if>
-    <xacro:if value="${use_none}">
-      <link name="${prefix}gripper_center"/>
-      <joint name="${prefix}gripper_center_fixed" type="fixed">
-        <parent link="${prefix}tcp"/>
-        <child link="${prefix}gripper_center"/>
-      </joint>
-    </xacro:if>
-  </xacro:macro>
+    <xacro:include filename="$(find piper_description)/xacro/components/gripper.xacro"/>
+    <xacro:include filename="$(find brainco_description)/xacro/revo2.xacro"/>
+    <xacro:macro name="NeroEndEffectors" params="name type:='gripper'">
+        <xacro:property name="prefix" value="${name + '_' if name else ''}"/>
+        <xacro:property name="hand_name" value="${name + '_hand' if name else 'hand'}"/>
+        <xacro:property name="ee_type" value="${type if type else 'gripper'}"/>
+        <xacro:property name="use_gripper" value="${ee_type == 'gripper'}"/>
+        <xacro:property name="use_revo2" value="${ee_type == 'revo2'}"/>
+        <xacro:property name="use_none" value="${ee_type == 'none'}"/>
+        <xacro:if value="${use_gripper}">
+            <link name="${prefix}gripper_flange">
+                <inertial>
+                    <origin xyz="0.000253201 -0.000322696 -0.010082901"/>
+                    <mass value="0.04771096"/>
+                    <inertia ixx="3.614107e-05" ixy="0" ixz="0" iyy="1.7824164e-05" iyz="0" izz="2.695944e-05"/>
+                </inertial>
+                <visual>
+                    <geometry>
+                        <mesh filename="file://$(find nero_description)/meshes/flange_gripper.glb"/>
+                    </geometry>
+                </visual>
+                <collision>
+                    <geometry>
+                        <mesh filename="file://$(find nero_description)/meshes/flange_gripper.glb"/>
+                    </geometry>
+                </collision>
+            </link>
+            <joint name="${prefix}gripper_flange_joint" type="fixed">
+                <origin xyz="0.031 0 -0.0235" rpy="-1.5708 0 -1.5708"/>
+                <parent link="${prefix}tcp"/>
+                <child link="${prefix}gripper_flange"/>
+            </joint>
+            <link name="${prefix}gripper_base">
+                <inertial>
+                    <origin xyz="-0.000183807162235591 8.05033155577911E-05 0.0321436689908876"/>
+                    <mass value="0.45"/>
+                    <inertia ixx="0.00092934" ixy="0.00000034" ixz="-0.00000738" iyy="0.00071447" iyz="0.00000005"
+                             izz="0.00039442"/>
+                </inertial>
+                <visual>
+                    <geometry>
+                        <mesh filename="file://$(find piper_description)/meshes/gripper/gripper_base.glb"/>
+                    </geometry>
+                </visual>
+                <collision>
+                    <geometry>
+                        <mesh filename="file://$(find piper_description)/meshes/gripper/gripper_base.glb"/>
+                    </geometry>
+                </collision>
+            </link>
+            <joint name="${prefix}gripper_base_joint" type="fixed">
+                <origin xyz="0 0 0.006"/>
+                <parent link="${prefix}gripper_flange"/>
+                <child link="${prefix}gripper_base"/>
+            </joint>
+            <xacro:agx_gripper
+                    prefix="${prefix}"
+                    parent_link="${prefix}gripper_base"
+                    xyz="0 0 0"
+                    finger_link="gripper_link7"
+                    finger_mimic_link="gripper_link8"/>
+        </xacro:if>
+        <xacro:if value="${use_revo2}">
+            <link name="${prefix}revo2_flange">
+                <inertial>
+                    <origin xyz="0.000253201 -0.000322696 -0.010082901"/>
+                    <mass value="0.04771096"/>
+                    <inertia ixx="3.614107e-05" ixy="0" ixz="0" iyy="1.7824164e-05" iyz="0" izz="2.695944e-05"/>
+                </inertial>
+                <visual>
+                    <geometry>
+                      <mesh filename="file://$(find nero_description)/meshes/flange_revo2.glb"/>
+                    </geometry>
+                </visual>
+                <collision>
+                    <geometry>
+                      <mesh filename="file://$(find nero_description)/meshes/flange_revo2.glb"/>
+                    </geometry>
+                </collision>
+            </link>
+            <joint name="${prefix}revo2_flange_joint" type="fixed">
+                <origin xyz="0.031 0 -0.0235" rpy="-1.5708 0 -1.5708"/>
+                <parent link="${prefix}tcp"/>
+                <child link="${prefix}revo2_flange"/>
+            </joint>
+            <xacro:BrainCoHand name="${hand_name}" use_flange="false"/>
+            <joint name="${prefix}hand_base_joint" type="fixed">
+                <origin xyz="0 0 0.012" rpy="0 0 3.1415926"/>
+                <parent link="${prefix}revo2_flange"/>
+                <child link="${hand_name}_hand_base"/>
+            </joint>
+            <link name="${prefix}gripper_center"/>
+            <joint name="${prefix}gripper_center_fixed" type="fixed">
+                <parent link="${prefix}tcp"/>
+                <child link="${prefix}gripper_center"/>
+            </joint>
+        </xacro:if>
+        <xacro:if value="${use_none}">
+            <link name="${prefix}gripper_center"/>
+            <joint name="${prefix}gripper_center_fixed" type="fixed">
+                <parent link="${prefix}tcp"/>
+                <child link="${prefix}gripper_center"/>
+            </joint>
+        </xacro:if>
+    </xacro:macro>
 </robot>

File: manipulator/AgileX/piper_description/xacro/components/gripper.xacro (robot description, xacro)
@@ -2,5 +2,5 @@
 <robot xmlns:xacro="http://www.ros.org/wiki/xacro">
   <!-- Unique Piper parallel gripper. Joint names match AdaptiveGripperController. -->
-  <xacro:macro name="agx_gripper" params="prefix parent_link xyz:='0 0 0' rpy:='0 0 0' housing:='false' travel:='0.05'">
+  <xacro:macro name="agx_gripper" params="prefix parent_link xyz:='0 0 0' rpy:='0 0 0' housing:='false' travel:='0.05' finger_link:='link7' finger_mimic_link:='link8'">
     <xacro:property name="use_housing" value="${str(housing).lower() in ['1', 'true', 'yes', 'on']}"/>
     <xacro:property name="finger_travel" value="${float(travel)}"/>
@@ -62,5 +62,5 @@
       <child link="${prefix}gripper_mount"/>
     </joint>
-    <link name="${prefix}link7">
+    <link name="${prefix}${finger_link}">
       <inertial>
         <origin xyz="0.00065123185041968 -0.0491929869131989 0.00972258769184025"/>
@@ -83,9 +83,9 @@
       <origin xyz="0 0 0.138" rpy="1.5707963 0 0"/>
       <parent link="${prefix}gripper_mount"/>
-      <child link="${prefix}link7"/>
+      <child link="${prefix}${finger_link}"/>
       <axis xyz="0 0 1"/>
       <limit lower="0" upper="${finger_travel}" effort="10" velocity="1"/>
     </joint>
-    <link name="${prefix}link8">
+    <link name="${prefix}${finger_mimic_link}">
       <inertial>
         <origin xyz="0.000651231850419722 -0.0491929869131991 0.00972258769184024"/>
@@ -108,5 +108,5 @@
       <origin xyz="0 0 0.138" rpy="1.5707963 0 -3.1415926"/>
       <parent link="${prefix}gripper_mount"/>
-      <child link="${prefix}link8"/>
+      <child link="${prefix}${finger_mimic_link}"/>
       <mimic joint="${prefix}gripper_joint" multiplier="-1" offset="0"/>
       <axis xyz="0 0 -1"/>
