Commit message: add open nero

File: manipulator/AgileX/nero_description/xacro/Nero.xacro (robot description, xacro)
@@ -1,5 +1,28 @@
 <?xml version="1.0" encoding="utf-8"?>
 <robot xmlns:xacro="http://www.ros.org/wiki/xacro">
-    <xacro:macro name="Nero" params="name">
+    <xacro:property name="PI" value="3.1415926535897931"/>
+    <xacro:macro name="nero_collision" params="collider mesh xyz:='0 0 0' rpy:='0 0 0' primitive:='box' radius:='0' length:='0' size:='0 0 0'">
+        <xacro:if value="${collider == 'simple'}">
+            <collision>
+                <origin xyz="${xyz}" rpy="${rpy}"/>
+                <geometry>
+                    <xacro:if value="${primitive == 'cylinder'}">
+                        <cylinder radius="${radius}" length="${length}"/>
+                    </xacro:if>
+                    <xacro:if value="${primitive == 'box'}">
+                        <box size="${size}"/>
+                    </xacro:if>
+                </geometry>
+            </collision>
+        </xacro:if>
+        <xacro:if value="${collider == 'convex'}">
+            <collision>
+                <geometry>
+                    <mesh filename="${mesh}"/>
+                </geometry>
+            </collision>
+        </xacro:if>
+    </xacro:macro>
+    <xacro:macro name="Nero" params="name collider:='simple'">
         <xacro:property name="prefix" value="${name + '_' if name else ''}"/>
         <link name="${prefix}base_link">
@@ -15,9 +38,8 @@
                 </geometry>
             </visual>
-            <collision>
-                <geometry>
-                    <mesh filename="file://$(find nero_description)/meshes/base_link.glb"/>
-                </geometry>
-            </collision>
+            <xacro:nero_collision
+                    collider="${collider}"
+                    mesh="file://$(find nero_description)/meshes/base_link.glb"
+                    primitive="cylinder" xyz="-0.0145 0 0.043" radius="0.055" length="0.086"/>
         </link>
         <link name="${prefix}link1">
@@ -33,9 +55,8 @@
                 </geometry>
             </visual>
-            <collision>
-                <geometry>
-                    <mesh filename="file://$(find nero_description)/meshes/link1.glb"/>
-                </geometry>
-            </collision>
+            <xacro:nero_collision
+                    collider="${collider}"
+                    mesh="file://$(find nero_description)/meshes/link1.glb"
+                    primitive="box" xyz="0 -0.002 -0.0135" size="0.072 0.0775 0.087"/>
         </link>
         <joint name="${prefix}joint1" type="revolute">
@@ -58,9 +79,8 @@
                 </geometry>
             </visual>
-            <collision>
-                <geometry>
-                    <mesh filename="file://$(find nero_description)/meshes/link2.glb"/>
-                </geometry>
-            </collision>
+            <xacro:nero_collision
+                    collider="${collider}"
+                    mesh="file://$(find nero_description)/meshes/link2.glb"
+                    primitive="cylinder" xyz="0.0033 -0.0977 0" rpy="${PI/2} 0 0" radius="0.047" length="0.262"/>
         </link>
         <joint name="${prefix}joint2" type="revolute">
@@ -83,9 +103,8 @@
                 </geometry>
             </visual>
-            <collision>
-                <geometry>
-                    <mesh filename="file://$(find nero_description)/meshes/link3.glb"/>
-                </geometry>
-            </collision>
+            <xacro:nero_collision
+                    collider="${collider}"
+                    mesh="file://$(find nero_description)/meshes/link3.glb"
+                    primitive="cylinder" xyz="0 0.002 -0.089" radius="0.040" length="0.235"/>
         </link>
         <joint name="${prefix}joint3" type="revolute">
@@ -108,9 +127,8 @@
                 </geometry>
             </visual>
-            <collision>
-                <geometry>
-                    <mesh filename="file://$(find nero_description)/meshes/link4.glb"/>
-                </geometry>
-            </collision>
+            <xacro:nero_collision
+                    collider="${collider}"
+                    mesh="file://$(find nero_description)/meshes/link4.glb"
+                    primitive="cylinder" xyz="0 -0.0365 0" rpy="${PI/2} 0 0" radius="0.040" length="0.135"/>
         </link>
         <joint name="${prefix}joint4" type="revolute">
@@ -133,9 +151,8 @@
                 </geometry>
             </visual>
-            <collision>
-                <geometry>
-                    <mesh filename="file://$(find nero_description)/meshes/link5.glb"/>
-                </geometry>
-            </collision>
+            <xacro:nero_collision
+                    collider="${collider}"
+                    mesh="file://$(find nero_description)/meshes/link5.glb"
+                    primitive="cylinder" xyz="0 0 -0.082" radius="0.035" length="0.189"/>
         </link>
         <joint name="${prefix}joint5" type="revolute">
@@ -158,9 +175,8 @@
                 </geometry>
             </visual>
-            <collision>
-                <geometry>
-                    <mesh filename="file://$(find nero_description)/meshes/link6.glb"/>
-                </geometry>
-            </collision>
+            <xacro:nero_collision
+                    collider="${collider}"
+                    mesh="file://$(find nero_description)/meshes/link6.glb"
+                    primitive="box" xyz="-0.0012 -0.0021 0" size="0.047 0.051 0.053"/>
         </link>
         <joint name="${prefix}joint6" type="revolute">
@@ -183,9 +199,8 @@
                 </geometry>
             </visual>
-            <collision>
-                <geometry>
-                    <mesh filename="file://$(find nero_description)/meshes/link7.glb"/>
-                </geometry>
-            </collision>
+            <xacro:nero_collision
+                    collider="${collider}"
+                    mesh="file://$(find nero_description)/meshes/link7.glb"
+                    primitive="box" xyz="0 0 -0.0047" size="0.027 0.027 0.010"/>
         </link>
         <joint name="${prefix}joint7" type="revolute">

File: manipulator/AgileX/nero_description/xacro/component.xacro (robot description, xacro)
@@ -3,7 +3,8 @@
   <xacro:arg name="type" default="ee"/>
   <xacro:arg name="name" default=""/>
+  <xacro:arg name="collider" default="simple"/>
   <xacro:if value="${'$(arg type)' == 'ee'}">
     <xacro:include filename="$(find nero_description)/xacro/Nero.xacro"/>
-    <xacro:Nero name="$(arg name)"/>
+    <xacro:Nero name="$(arg name)" collider="$(arg collider)"/>
   </xacro:if>
 </robot>

File: manipulator/AgileX/nero_description/xacro/eefs.xacro (robot description, xacro)
@@ -3,5 +3,5 @@
     <xacro:include filename="$(find piper_description)/xacro/components/gripper.xacro"/>
     <xacro:include filename="$(find brainco_description)/xacro/revo2.xacro"/>
-    <xacro:macro name="NeroEndEffectors" params="name type:='gripper'">
+    <xacro:macro name="NeroEndEffectors" params="name type:='gripper' collider:='simple' direction:='' fixed_joints:='false'">
         <xacro:property name="prefix" value="${name + '_' if name else ''}"/>
         <xacro:property name="hand_name" value="${name + '_hand' if name else 'hand'}"/>
@@ -10,4 +10,6 @@
         <xacro:property name="use_revo2" value="${ee_type == 'revo2'}"/>
         <xacro:property name="use_none" value="${ee_type == 'none'}"/>
+        <!-- direction=1 左手，-1 右手。未传时按 name==right 推断（对齐 Piper / Open Nero）。 -->
+        <xacro:property name="hand_direction" value="${float(direction) if str(direction) != '' else (-1.0 if name == 'right' else 1.0)}"/>
         <xacro:if value="${use_gripper}">
             <link name="${prefix}gripper_flange">
@@ -22,9 +24,19 @@
                     </geometry>
                 </visual>
-                <collision>
-                    <geometry>
-                        <mesh filename="file://$(find nero_description)/meshes/flange_gripper.glb"/>
-                    </geometry>
-                </collision>
+                <xacro:if value="${collider == 'simple'}">
+                    <collision>
+                        <origin xyz="0 0 -0.018"/>
+                        <geometry>
+                            <box size="0.044 0.055 0.060"/>
+                        </geometry>
+                    </collision>
+                </xacro:if>
+                <xacro:if value="${collider == 'convex'}">
+                    <collision>
+                        <geometry>
+                            <mesh filename="file://$(find nero_description)/meshes/flange_gripper.glb"/>
+                        </geometry>
+                    </collision>
+                </xacro:if>
             </link>
             <joint name="${prefix}gripper_flange_joint" type="fixed">
@@ -45,9 +57,19 @@
                     </geometry>
                 </visual>
-                <collision>
-                    <geometry>
-                        <mesh filename="file://$(find piper_description)/meshes/gripper/gripper_base.glb"/>
-                    </geometry>
-                </collision>
+                <xacro:if value="${collider == 'simple'}">
+                    <collision>
+                        <origin xyz="-0.0048 0 0.0325"/>
+                        <geometry>
+                            <box size="0.075 0.164 0.065"/>
+                        </geometry>
+                    </collision>
+                </xacro:if>
+                <xacro:if value="${collider == 'convex'}">
+                    <collision>
+                        <geometry>
+                            <mesh filename="file://$(find piper_description)/meshes/gripper/gripper_base.glb"/>
+                        </geometry>
+                    </collision>
+                </xacro:if>
             </link>
             <joint name="${prefix}gripper_base_joint" type="fixed">
@@ -75,9 +97,19 @@
                     </geometry>
                 </visual>
-                <collision>
-                    <geometry>
-                      <mesh filename="file://$(find nero_description)/meshes/flange_revo2.glb"/>
-                    </geometry>
-                </collision>
+                <xacro:if value="${collider == 'simple'}">
+                    <collision>
+                        <origin xyz="0 0 -0.018"/>
+                        <geometry>
+                            <box size="0.044 0.055 0.060"/>
+                        </geometry>
+                    </collision>
+                </xacro:if>
+                <xacro:if value="${collider == 'convex'}">
+                    <collision>
+                        <geometry>
+                          <mesh filename="file://$(find nero_description)/meshes/flange_revo2.glb"/>
+                        </geometry>
+                    </collision>
+                </xacro:if>
             </link>
             <joint name="${prefix}revo2_flange_joint" type="fixed">
@@ -86,5 +118,5 @@
                 <child link="${prefix}revo2_flange"/>
             </joint>
-            <xacro:BrainCoHand name="${hand_name}" use_flange="false"/>
+            <xacro:BrainCoHand name="${hand_name}" use_flange="false" direction="${hand_direction}" fixed_joints="${fixed_joints}"/>
             <joint name="${prefix}hand_base_joint" type="fixed">
                 <origin xyz="0 0 0.012" rpy="0 0 3.1415926"/>

File: manipulator/AgileX/nero_description/xacro/gripper.xacro (robot description, xacro)
@@ -1,6 +1,7 @@
 <?xml version="1.0"?>
 <robot name="Nero Gripper" xmlns:xacro="http://www.ros.org/wiki/xacro">
+  <xacro:arg name="collider" default="simple"/>
   <xacro:include filename="$(find nero_description)/xacro/eefs.xacro"/>
   <link name="tcp"/>
-  <xacro:NeroEndEffectors name="" type="gripper"/>
+  <xacro:NeroEndEffectors name="" type="gripper" collider="$(arg collider)"/>
 </robot>

File: manipulator/AgileX/nero_description/xacro/robot.xacro (robot description, xacro)
@@ -3,10 +3,18 @@
   <xacro:arg name="type" default=""/>
   <xacro:arg name="name" default=""/>
+  <xacro:arg name="collider" default="simple"/>
+  <xacro:arg name="direction" default=""/>
+  <xacro:arg name="eef_fixed_joints" default="false"/>
   <xacro:property name="type_arg" value="$(arg type)"/>
   <xacro:property name="name_arg" value="$(arg name)"/>
   <xacro:property name="ee_type" value="${type_arg if type_arg else 'gripper'}"/>
   <xacro:include filename="$(find nero_description)/xacro/Nero.xacro"/>
-  <xacro:Nero name="${name_arg}"/>
+  <xacro:Nero name="${name_arg}" collider="$(arg collider)"/>
   <xacro:include filename="$(find nero_description)/xacro/eefs.xacro"/>
-  <xacro:NeroEndEffectors name="${name_arg}" type="${ee_type}"/>
+  <xacro:NeroEndEffectors
+      name="${name_arg}"
+      type="${ee_type}"
+      collider="$(arg collider)"
+      direction="$(arg direction)"
+      fixed_joints="$(arg eef_fixed_joints)"/>
 </robot>
