Commit message: update readme

File: humanoid/X2Robot/quanta_x1_description/xacro/component.xacro (robot description, xacro)
@@ -9,4 +9,5 @@
 <robot name="quanta_x1_component" xmlns:xacro="http://www.ros.org/wiki/xacro">
   <xacro:arg name="type" default="base"/>
+  <xacro:property name="PI" value="3.1415926535897931"/>
   <!-- type=base: visualize base-related components -->
   <xacro:if value="${'$(arg type)' == 'base'}">
