Commit message: fix(quanta_x1): lock chassis wheels/casters like W2/Bot2 peers
Drive wheels and swivel casters default to fixed via
chassis_joints_movable:=false; they are no longer in ros2_control.
Lift/head stay as body interfaces. Matches Galaxea/ARX Lift2S/W2.

File: humanoid/X2Robot/quanta_x1_description/xacro/component.xacro (robot description, xacro)
@@ -2,16 +2,21 @@
 <!--
   Component-wise description for Quanta X1, used by
-  robot_descriptions/common/robot_common_launch/launch/visualize/component.launch.py
+  robot_common_launch/launch/visualize/component.launch.py
   Supported types (arg "type"):
     - base (default)
     - arm (single left arm)
+    - chassis (base with chassis_joints_movable:=true for wheel/caster inspection)
 -->
 <robot name="quanta_x1_component" xmlns:xacro="http://www.ros.org/wiki/xacro">
   <xacro:arg name="type" default="base"/>
+  <xacro:arg name="chassis_joints_movable" default="false"/>
   <xacro:property name="PI" value="3.1415926535897931"/>
-  <!-- type=base: visualize base-related components -->
   <xacro:if value="${'$(arg type)' == 'base'}">
     <xacro:include filename="$(find quanta_x1_description)/xacro/components/base.xacro"/>
-    <xacro:QuantaX1Base/>
+    <xacro:QuantaX1Base joints_movable="$(arg chassis_joints_movable)"/>
+  </xacro:if>
+  <xacro:if value="${'$(arg type)' == 'chassis'}">
+    <xacro:include filename="$(find quanta_x1_description)/xacro/components/base.xacro"/>
+    <xacro:QuantaX1Base joints_movable="true"/>
   </xacro:if>
   <xacro:if value="${'$(arg type)' == 'arm'}">

File: humanoid/X2Robot/quanta_x1_description/xacro/components/base.xacro (robot description, xacro)
@@ -2,5 +2,8 @@
 <robot xmlns:xacro="http://www.ros.org/wiki/xacro">
 	<xacro:include filename="$(find quanta_x1_description)/xacro/components/swivel.xacro"/>
-	<xacro:macro name="QuantaX1Base">
+	<xacro:macro name="QuantaX1Base" params="joints_movable:=false">
+		<!-- Drive / caster joints: fixed for viz & arm control (W2/Bot2/Galaxea); continuous only if movable -->
+		<xacro:property name="chassis_movable" value="${str(joints_movable).lower() in ['true', '1', 'yes', 'on']}"/>
+		<xacro:property name="wheel_joint_type" value="${'continuous' if chassis_movable else 'fixed'}"/>
 		<link name="base_link"/>
 		<joint name="chassis_base_joint" type="fixed">
@@ -45,9 +48,11 @@
 			</collision>
 		</link>
-		<joint name="right_wheel_joint" type="continuous">
+		<joint name="right_wheel_joint" type="${wheel_joint_type}">
 			<origin xyz="0 -0.208 0.085999"/>
 			<parent link="chassis_base_link"/>
 			<child link="right_wheel_link"/>
-			<axis xyz="0 1 0"/>
+			<xacro:if value="${chassis_movable}">
+				<axis xyz="0 1 0"/>
+			</xacro:if>
 		</joint>
 		<link name="left_wheel_link">
@@ -69,9 +74,11 @@
 			</collision>
 		</link>
-		<joint name="left_wheel_joint" type="continuous">
+		<joint name="left_wheel_joint" type="${wheel_joint_type}">
 			<origin xyz="0 0.208 0.086001"/>
 			<parent link="chassis_base_link"/>
 			<child link="left_wheel_link"/>
-			<axis xyz="0 1 0"/>
+			<xacro:if value="${chassis_movable}">
+				<axis xyz="0 1 0"/>
+			</xacro:if>
 		</joint>
 		<link name="lift_link">
@@ -387,8 +394,8 @@
 			<child link="2d_laser_base"/>
 		</joint>
-		<xacro:QuantaX1Swivel prefix="fl" x="0.212205" y="0.172203" z="0.061972"/>
-		<xacro:QuantaX1Swivel prefix="fr" x="0.212205" y="-0.172203" z="0.061972"/>
-		<xacro:QuantaX1Swivel prefix="rl" x="-0.1878" y="0.172203" z="0.061972"/>
-		<xacro:QuantaX1Swivel prefix="rr" x="-0.1878" y="-0.172203" z="0.061972"/>
+		<xacro:QuantaX1Swivel prefix="fl" x="0.212205" y="0.172203" z="0.061972" joints_movable="${joints_movable}"/>
+		<xacro:QuantaX1Swivel prefix="fr" x="0.212205" y="-0.172203" z="0.061972" joints_movable="${joints_movable}"/>
+		<xacro:QuantaX1Swivel prefix="rl" x="-0.1878" y="0.172203" z="0.061972" joints_movable="${joints_movable}"/>
+		<xacro:QuantaX1Swivel prefix="rr" x="-0.1878" y="-0.172203" z="0.061972" joints_movable="${joints_movable}"/>
 	</xacro:macro>
 </robot>

File: humanoid/X2Robot/quanta_x1_description/xacro/components/swivel.xacro (robot description, xacro)
@@ -1,5 +1,9 @@
 <?xml version="1.0" ?>
 <robot xmlns:xacro="http://www.ros.org/wiki/xacro">
-	<xacro:macro name="QuantaX1Swivel" params="prefix x y z">
+	<!-- Passive swivel casters. Default fixed (viz / planning / arm control);
+	     continuous only when chassis_joints_movable:=true (same idea as W2/Bot2). -->
+	<xacro:macro name="QuantaX1Swivel" params="prefix x y z joints_movable:=false">
+		<xacro:property name="caster_movable" value="${str(joints_movable).lower() in ['true', '1', 'yes', 'on']}"/>
+		<xacro:property name="caster_joint_type" value="${'continuous' if caster_movable else 'fixed'}"/>
 		<link name="${prefix}_swivel_link">
 			<visual>
@@ -21,8 +25,10 @@
 			</visual>
 		</link>
-		<joint name="${prefix}_swivel_yaw" type="continuous">
+		<joint name="${prefix}_swivel_yaw" type="${caster_joint_type}">
 			<parent link="${prefix}_swivel_link"/>
 			<child link="${prefix}_swivel_yaw"/>
-			<axis xyz="0 0 1"/>
+			<xacro:if value="${caster_movable}">
+				<axis xyz="0 0 1"/>
+			</xacro:if>
 		</joint>
 		<link name="${prefix}_roller_1">
@@ -38,9 +44,11 @@
 			</collision>
 		</link>
-		<joint name="${prefix}_swivel_roller_1" type="continuous">
+		<joint name="${prefix}_swivel_roller_1" type="${caster_joint_type}">
 			<parent link="${prefix}_swivel_yaw"/>
 			<child link="${prefix}_roller_1"/>
-			<axis xyz="0 1 0"/>
 			<origin xyz="0.045295 0.000296 -0.016972"/>
+			<xacro:if value="${caster_movable}">
+				<axis xyz="0 1 0"/>
+			</xacro:if>
 		</joint>
 		<link name="${prefix}_roller_2">
@@ -56,9 +64,11 @@
 			</collision>
 		</link>
-		<joint name="${prefix}_swivel_roller_2" type="continuous">
+		<joint name="${prefix}_swivel_roller_2" type="${caster_joint_type}">
 			<parent link="${prefix}_swivel_yaw"/>
 			<child link="${prefix}_roller_2"/>
-			<axis xyz="0 1 0"/>
 			<origin xyz="0.012295 0.034228 -0.029472"/>
+			<xacro:if value="${caster_movable}">
+				<axis xyz="0 1 0"/>
+			</xacro:if>
 		</joint>
 		<link name="${prefix}_roller_3">
@@ -74,9 +84,11 @@
 			</collision>
 		</link>
-		<joint name="${prefix}_swivel_roller_3" type="continuous">
+		<joint name="${prefix}_swivel_roller_3" type="${caster_joint_type}">
 			<parent link="${prefix}_swivel_yaw"/>
 			<child link="${prefix}_roller_3"/>
-			<axis xyz="0 1 0"/>
 			<origin xyz="0.012295 -0.034572 -0.029472"/>
+			<xacro:if value="${caster_movable}">
+				<axis xyz="0 1 0"/>
+			</xacro:if>
 		</joint>
 		<link name="${prefix}_roller_4">
@@ -92,9 +104,11 @@
 			</collision>
 		</link>
-		<joint name="${prefix}_swivel_roller_4" type="continuous">
+		<joint name="${prefix}_swivel_roller_4" type="${caster_joint_type}">
 			<parent link="${prefix}_swivel_yaw"/>
 			<child link="${prefix}_roller_4"/>
-			<axis xyz="0 1 0"/>
 			<origin xyz="-0.024705 0.000072 -0.039472"/>
+			<xacro:if value="${caster_movable}">
+				<axis xyz="0 1 0"/>
+			</xacro:if>
 		</joint>
 	</xacro:macro>

File: humanoid/X2Robot/quanta_x1_description/xacro/robot.xacro (robot description, xacro)
@@ -2,7 +2,9 @@
 <robot name="Quanta X1" xmlns:xacro="http://www.ros.org/wiki/xacro">
   <xacro:property name="PI" value="3.1415926535897931"/>
+  <!-- Lock drive wheels + swivel casters by default (W2/Bot2/Galaxea). Planning URDF keeps this false. -->
+  <xacro:arg name="chassis_joints_movable" default="false"/>
   <xacro:include filename="$(find quanta_x1_description)/xacro/components/base.xacro"/>
   <xacro:include filename="$(find quanta_x1_description)/xacro/components/arm.xacro"/>
-  <xacro:QuantaX1Base/>
+  <xacro:QuantaX1Base joints_movable="$(arg chassis_joints_movable)"/>
   <xacro:QuantaX1SingleArm name="left"/>
   <xacro:QuantaX1SingleArm name="right"/>

File: humanoid/X2Robot/quanta_x1_description/xacro/ros2_control/base_ros2_control.xacro (robot description, xacro)
@@ -1,25 +1,7 @@
 <?xml version="1.0"?>
 <robot xmlns:xacro="http://www.ros.org/wiki/xacro">
-  <!-- Quanta X1 base: lift + head; optional drive wheels. -->
-  <xacro:macro name="quanta_x1_wheel_interfaces">
-    <joint name="left_wheel_joint">
-      <command_interface name="velocity">
-        <param name="min">-10.0</param>
-        <param name="max">10.0</param>
-      </command_interface>
-      <state_interface name="position"/>
-      <state_interface name="velocity"/>
-      <state_interface name="effort"/>
-    </joint>
-    <joint name="right_wheel_joint">
-      <command_interface name="velocity">
-        <param name="min">-10.0</param>
-        <param name="max">10.0</param>
-      </command_interface>
-      <state_interface name="position"/>
-      <state_interface name="velocity"/>
-      <state_interface name="effort"/>
-    </joint>
-  </xacro:macro>
+  <!-- Quanta X1 body interfaces: lift + head only.
+       Drive wheels / swivel casters stay out of ros2_control (W2/Bot2/Galaxea/ARX Lift2S);
+       they are fixed in the URDF unless chassis_joints_movable:=true. -->
   <xacro:macro name="quanta_x1_base_interfaces" params="iface_mode:=mix">
     <joint name="lift_joint">

File: humanoid/X2Robot/quanta_x1_description/xacro/ros2_control/robot.xacro (robot description, xacro)
@@ -3,5 +3,6 @@
   <xacro:arg name="ros2_control_hardware_type" default="mock_components"/>
   <xacro:arg name="gazebo" default="false"/>
-  <xacro:arg name="enable_wheels" default="false"/>
+  <!-- Keep chassis wheels/casters fixed under control (same as viz default). -->
+  <xacro:arg name="chassis_joints_movable" default="false"/>
   <xacro:include filename="$(find quanta_x1_description)/xacro/robot.xacro"/>
   <xacro:include filename="$(find quanta_x1_description)/xacro/ros2_control/arm_ros2_control.xacro"/>
@@ -28,8 +29,6 @@
       </xacro:if>
     </hardware>
+    <!-- Body = lift + head; wheels/casters are not HI (peer convention). -->
     <xacro:quanta_x1_base_interfaces iface_mode="${sim_iface_mode}"/>
-    <xacro:if value="${'$(arg enable_wheels)' == 'true'}">
-      <xacro:quanta_x1_wheel_interfaces/>
-    </xacro:if>
     <xacro:quanta_x1_arm_interfaces name="left" iface_mode="${sim_iface_mode}"/>
     <xacro:quanta_x1_arm_interfaces name="right" iface_mode="${sim_iface_mode}"/>

Commit message: fix(quanta_x1): WBC Pinocchio joint order + convex collisions
Move head after both arms so DFS is lift|L|R|head (ARX Lift), add
target_manager.yaml frames, and replace arm/gripper collisions with
convex hulls plus 3-piece CoACD for bracket and wrist camera.

File: humanoid/X2Robot/quanta_x1_description/xacro/component.xacro (robot description, xacro)
@@ -14,9 +14,13 @@
   <xacro:if value="${'$(arg type)' == 'base'}">
     <xacro:include filename="$(find quanta_x1_description)/xacro/components/base.xacro"/>
+    <xacro:include filename="$(find quanta_x1_description)/xacro/components/head.xacro"/>
     <xacro:QuantaX1Base joints_movable="$(arg chassis_joints_movable)"/>
+    <xacro:QuantaX1Head/>
   </xacro:if>
   <xacro:if value="${'$(arg type)' == 'chassis'}">
     <xacro:include filename="$(find quanta_x1_description)/xacro/components/base.xacro"/>
+    <xacro:include filename="$(find quanta_x1_description)/xacro/components/head.xacro"/>
     <xacro:QuantaX1Base joints_movable="true"/>
+    <xacro:QuantaX1Head/>
   </xacro:if>
   <xacro:if value="${'$(arg type)' == 'arm'}">

File: humanoid/X2Robot/quanta_x1_description/xacro/components/arm.xacro (robot description, xacro)
@@ -158,4 +158,9 @@
 				</geometry>
 			</visual>
+			<collision>
+				<geometry>
+					<mesh filename="file://$(find quanta_x1_description)/meshes/arm/collision/arm_link6.STL"/>
+				</geometry>
+			</collision>
 		</link>
 		<joint name="${prefix}joint6" type="revolute">
@@ -177,7 +182,18 @@
 				</geometry>
 			</visual>
-			<collision>
-				<geometry>
-					<mesh filename="file://$(find quanta_x1_description)/meshes/gripper/collision/gripper_base_link.STL"/>
+			<!-- 夹爪支架: CoACD 3 convex pieces -->
+			<collision>
+				<geometry>
+					<mesh filename="file://$(find quanta_x1_description)/meshes/gripper/collision/gripper_base_link_0.stl"/>
+				</geometry>
+			</collision>
+			<collision>
+				<geometry>
+					<mesh filename="file://$(find quanta_x1_description)/meshes/gripper/collision/gripper_base_link_1.stl"/>
+				</geometry>
+			</collision>
+			<collision>
+				<geometry>
+					<mesh filename="file://$(find quanta_x1_description)/meshes/gripper/collision/gripper_base_link_2.stl"/>
 				</geometry>
 			</collision>
@@ -196,4 +212,9 @@
 				</material>
 			</visual>
+			<collision>
+				<geometry>
+					<mesh filename="file://$(find quanta_x1_description)/meshes/gripper/collision/gripper_motor.STL"/>
+				</geometry>
+			</collision>
 		</link>
 		<joint name="${prefix}gripper_joint" type="revolute">
@@ -265,4 +286,20 @@
 				</geometry>
 			</visual>
+			<!-- wrist camera: CoACD 3 convex pieces -->
+			<collision>
+				<geometry>
+					<mesh filename="file://$(find quanta_x1_description)/meshes/gripper/collision/gripper_camera_0.stl"/>
+				</geometry>
+			</collision>
+			<collision>
+				<geometry>
+					<mesh filename="file://$(find quanta_x1_description)/meshes/gripper/collision/gripper_camera_1.stl"/>
+				</geometry>
+			</collision>
+			<collision>
+				<geometry>
+					<mesh filename="file://$(find quanta_x1_description)/meshes/gripper/collision/gripper_camera_2.stl"/>
+				</geometry>
+			</collision>
 		</link>
 		<joint name="${prefix}gripper_camera_base_joint" type="fixed">

File: humanoid/X2Robot/quanta_x1_description/xacro/components/base.xacro (robot description, xacro)
@@ -106,53 +106,4 @@
 			<limit effort="2000" lower="0" upper="0.78" velocity="0.2"/>
 		</joint>
-		<link name="head_yaw_link">
-			<inertial>
-				<origin xyz="9.85219e-05 -0.00010749 0.056689166"/>
-				<mass value="0.64404227"/>
-				<inertia ixx="0.000486721" ixy="-1.25e-06" ixz="-8.64e-07" iyy="0.000572985" iyz="1.41146e-05"
-								 izz="0.000333911"/>
-			</inertial>
-			<visual>
-				<geometry>
-					<mesh filename="file://$(find quanta_x1_description)/meshes/base/head_yaw.glb"/>
-				</geometry>
-			</visual>
-			<collision>
-				<geometry>
-					<mesh filename="file://$(find quanta_x1_description)/meshes/base/collision/head_yaw_link.STL"/>
-				</geometry>
-			</collision>
-		</link>
-		<joint name="head_yaw_joint" type="revolute">
-			<origin xyz="0.1595 0 0.2245"/>
-			<parent link="lift_link"/>
-			<child link="head_yaw_link"/>
-			<axis xyz="0 0 1"/>
-			<limit effort="9" lower="-1.5708" upper="1.5708" velocity="3.77"/>
-		</joint>
-		<link name="head_pitch_link">
-			<inertial>
-				<origin xyz="2.79439e-05 1.4773183 -0.10496909"/>
-				<mass value="0.59804473"/>
-				<inertia ixx="0.00131549" ixy="-1.93e-06" ixz="-1.23e-06" iyy="0.001827745" iyz="-6.2e-05" izz="0.002283248"/>
-			</inertial>
-			<visual>
-				<geometry>
-					<mesh filename="file://$(find quanta_x1_description)/meshes/base/head_pitch.glb"/>
-				</geometry>
-			</visual>
-			<collision>
-				<geometry>
-					<mesh filename="file://$(find quanta_x1_description)/meshes/base/collision/head_pitch_link.STL"/>
-				</geometry>
-			</collision>
-		</link>
-		<joint name="head_pitch_joint" type="revolute">
-			<origin xyz="0 0 0.062"/>
-			<parent link="head_yaw_link"/>
-			<child link="head_pitch_link"/>
-			<axis xyz="0 1 0"/>
-			<limit effort="9" lower="-0.1745" upper="1.2217" velocity="3.77"/>
-		</joint>
 		<link name="left_frame_link"/>
 		<joint name="left_frame_joint" type="fixed">
@@ -166,16 +117,4 @@
 			<parent link="lift_link"/>
 			<child link="right_frame_link"/>
-		</joint>
-		<link name="head_camera_frame_link">
-			<visual>
-				<geometry>
-					<mesh filename="file://$(find sensor_models)/meshes/orbbec/Dabai_DCW2.glb"/>
-				</geometry>
-			</visual>
-		</link>
-		<joint name="head_camera_connector" type="fixed">
-			<origin xyz="-0.05335 -0.00767 0.0517"/>
-			<parent link="head_pitch_link"/>
-			<child link="head_camera_frame_link"/>
 		</joint>
 		<link name="chest_lh_camera_base_link">

File: humanoid/X2Robot/quanta_x1_description/xacro/robot.xacro (robot description, xacro)
@@ -6,4 +6,5 @@
   <xacro:include filename="$(find quanta_x1_description)/xacro/components/base.xacro"/>
   <xacro:include filename="$(find quanta_x1_description)/xacro/components/arm.xacro"/>
+  <xacro:include filename="$(find quanta_x1_description)/xacro/components/head.xacro"/>
   <xacro:QuantaX1Base joints_movable="$(arg chassis_joints_movable)"/>
   <xacro:QuantaX1SingleArm name="left"/>
@@ -17,3 +18,5 @@
     <child link="right_base_link"/>
   </joint>
+  <!-- Head AFTER arms → Pinocchio DFS: lift | L6 | R6 | head×2 (ARX Lift convention) -->
+  <xacro:QuantaX1Head/>
 </robot>
