Commit message: add fb camera stand

File: manipulator/Realman/rm75_description/xacro/arm.xacro (robot description, xacro)
@@ -150,4 +150,19 @@
 				<xacro:visual_collision mesh="ee/ee_basic.glb"/>
 			</xacro:if>
+			<xacro:if value="${ee_type_norm == 'fb_camera'}">
+				<xacro:visual_collision mesh="ee/ee_fb_camera.glb"/>
+				<visual>
+					<origin xyz="-0.033 -0.0085 0.01562"/>
+					<geometry>
+						<mesh filename="${mesh_path}/ee/camera_stand_d405.glb"/>
+					</geometry>
+				</visual>
+				<visual>
+					<origin xyz="-0.13322 -0.0005 0.044651" rpy="0 -1.5708 -1.5708"/>
+					<geometry>
+						<mesh filename="file://$(find sensor_models)/meshes/d405.glb"/>
+					</geometry>
+				</visual>
+			</xacro:if>
 		</link>
 		<joint name="${prefix}joint1" type="revolute">
@@ -224,4 +239,7 @@
 				<origin xyz="0 0 0.046"/>
 			</xacro:if>
+			<xacro:if value="${ee_type_norm == 'fb_camera'}">
+				<origin xyz="0 0 0.0695"/>
+			</xacro:if>
 			<parent link="${prefix}link7"/>
 			<child link="${prefix}ee"/>

File: manipulator/Realman/rm75_description/xacro/robot.xacro (robot description, xacro)
@@ -12,4 +12,7 @@
 	<xacro:if value="${type_arg == 'fb'}">
 		<xacro:property name="selected_ee_type" value="fb"/>
+	</xacro:if>
+	<xacro:if value="${type_arg == 'fb_camera'}">
+		<xacro:property name="selected_ee_type" value="fb_camera"/>
 	</xacro:if>
 	<xacro:if value="${type_arg == 'aidal'}">

Commit message: add seperate fb75 camera component

File: manipulator/Realman/rm75_description/xacro/arm.xacro (robot description, xacro)
@@ -1,4 +1,5 @@
 <?xml version="1.0"?>
 <robot name="Realman RM75" xmlns:xacro="http://www.ros.org/wiki/xacro">
+	<xacro:include filename="$(find rm75_description)/xacro/components/fb75_camera.xacro"/>
 	<xacro:macro name="rm75" params="name direction:='' enable_joint3:=true ee_type:='aidal' use_base_link:=true">
 		<xacro:property name="prefix" value="${name + '_' if name else ''}"/>
@@ -152,18 +153,9 @@
 			<xacro:if value="${ee_type_norm == 'fb_camera'}">
 				<xacro:visual_collision mesh="ee/ee_fb_camera.glb"/>
-				<visual>
-					<origin xyz="-0.033 -0.0085 0.01562"/>
-					<geometry>
-						<mesh filename="${mesh_path}/ee/camera_stand_d405.glb"/>
-					</geometry>
-				</visual>
-				<visual>
-					<origin xyz="-0.13322 -0.0005 0.044651" rpy="0 -1.5708 -1.5708"/>
-					<geometry>
-						<mesh filename="file://$(find sensor_models)/meshes/d405.glb"/>
-					</geometry>
-				</visual>
-			</xacro:if>
-		</link>
+			</xacro:if>
+		</link>
+		<xacro:if value="${ee_type_norm == 'fb_camera'}">
+			<xacro:rm75_fb75_camera prefix="${prefix}" parent_link="${prefix}link7"/>
+		</xacro:if>
 		<joint name="${prefix}joint1" type="revolute">
 			<parent link="${prefix}arm_root"/>
