Commit message: update readme and clear meshes

File: humanoid/Galbot/galbot_one_description/xacro/components/arm.xacro (robot description, xacro)
@@ -13,5 +13,5 @@
     <visual>
       <geometry>
-        <mesh filename="package://galbot_one_description/meshes/arm/base.glb" scale ="1 -1 1"/>
+        <mesh filename="file://$(find galbot_one_description)/meshes/arm/base.glb" scale ="1 -1 1"/>
       </geometry>
     </visual>
@@ -25,5 +25,5 @@
     <visual>
       <geometry>
-        <mesh filename="package://galbot_one_description/meshes/arm/left_arm_link1.glb" scale="1 -1 1"/>
+        <mesh filename="file://$(find galbot_one_description)/meshes/arm/left_arm_link1.glb" scale="1 -1 1"/>
       </geometry>
     </visual>
@@ -44,5 +44,5 @@
     <visual>
       <geometry>
-        <mesh filename="package://galbot_one_description/meshes/arm/left_arm_link2.glb" scale="-1 1 1"/>
+        <mesh filename="file://$(find galbot_one_description)/meshes/arm/left_arm_link2.glb" scale="-1 1 1"/>
       </geometry>
     </visual>
@@ -69,5 +69,5 @@
     <visual>
       <geometry>
-        <mesh filename="package://galbot_one_description/meshes/arm/left_arm_link3.glb" scale="1 -1 1"/>
+        <mesh filename="file://$(find galbot_one_description)/meshes/arm/left_arm_link3.glb" scale="1 -1 1"/>
       </geometry>
     </visual>
@@ -94,5 +94,5 @@
     <visual>
       <geometry>
-        <mesh filename="package://galbot_one_description/meshes/arm/left_arm_link4.glb" scale="1 -1 1"/>
+        <mesh filename="file://$(find galbot_one_description)/meshes/arm/left_arm_link4.glb" scale="1 -1 1"/>
       </geometry>
     </visual>
@@ -119,5 +119,5 @@
     <visual>
       <geometry>
-        <mesh filename="package://galbot_one_description/meshes/arm/left_arm_link5.glb" />
+        <mesh filename="file://$(find galbot_one_description)/meshes/arm/left_arm_link5.glb" />
       </geometry>
     </visual>
@@ -144,5 +144,5 @@
     <visual>
       <geometry>
-        <mesh filename="package://galbot_one_description/meshes/arm/left_arm_link6.glb" />
+        <mesh filename="file://$(find galbot_one_description)/meshes/arm/left_arm_link6.glb" />
       </geometry>
     </visual>
@@ -168,5 +168,5 @@
     <visual>
       <geometry>
-        <mesh filename="package://galbot_one_description/meshes/arm/left_arm_link7.glb" />
+        <mesh filename="file://$(find galbot_one_description)/meshes/arm/left_arm_link7.glb" />
       </geometry>
     </visual>
@@ -203,5 +203,5 @@
     <visual>
       <geometry>
-        <mesh filename="package://galbot_one_description/meshes/flange/flange.glb"/>
+        <mesh filename="file://$(find galbot_one_description)/meshes/flange/flange.glb"/>
       </geometry>
     </visual>
@@ -227,5 +227,5 @@
     <visual>
       <geometry>
-        <mesh filename="package://galbot_one_description/meshes/camera/arm_camera.glb"/>
+        <mesh filename="file://$(find galbot_one_description)/meshes/camera/arm_camera.glb"/>
       </geometry>
     </visual>
@@ -243,5 +243,5 @@
     <visual>
       <geometry>
-        <mesh filename="package://galbot_one_description/meshes/arm/base.glb"/>
+        <mesh filename="file://$(find galbot_one_description)/meshes/arm/base.glb"/>
       </geometry>
     </visual>
@@ -259,6 +259,7 @@
     </inertial>
     <visual>
-      <geometry>
-        <mesh filename="package://galbot_one_description/meshes/arm/left_arm_link1.glb"/>
+      <origin rpy="0 0 3.14" />
+      <geometry>
+        <mesh filename="file://$(find galbot_one_description)/meshes/arm/left_arm_link1.glb"/>
       </geometry>
     </visual>
@@ -284,5 +285,5 @@
     <visual>
       <geometry>
-        <mesh filename="package://galbot_one_description/meshes/arm/left_arm_link2.glb"/>
+        <mesh filename="file://$(find galbot_one_description)/meshes/arm/left_arm_link2.glb"/>
       </geometry>
     </visual>
@@ -309,5 +310,5 @@
     <visual>
       <geometry>
-        <mesh filename="package://galbot_one_description/meshes/arm/left_arm_link3.glb"/>
+        <mesh filename="file://$(find galbot_one_description)/meshes/arm/left_arm_link3.glb"/>
       </geometry>
     </visual>
@@ -335,5 +336,5 @@
       <origin rpy="0 0 3.14" xyz="0 0 0"/>
       <geometry>
-        <mesh filename="package://galbot_one_description/meshes/arm/left_arm_link4.glb"/>
+        <mesh filename="file://$(find galbot_one_description)/meshes/arm/left_arm_link4.glb"/>
       </geometry>
     </visual>
@@ -360,5 +361,5 @@
     <visual>
       <geometry>
-        <mesh filename="package://galbot_one_description/meshes/arm/left_arm_link5.glb"/>
+        <mesh filename="file://$(find galbot_one_description)/meshes/arm/left_arm_link5.glb"/>
       </geometry>
     </visual>S
@@ -385,5 +386,5 @@
     <visual>
       <geometry>
-        <mesh filename="package://galbot_one_description/meshes/arm/left_arm_link6.glb"/>
+        <mesh filename="file://$(find galbot_one_description)/meshes/arm/left_arm_link6.glb"/>
       </geometry>
     </visual>
@@ -409,5 +410,5 @@
     <visual>
       <geometry>
-        <mesh filename="package://galbot_one_description/meshes/arm/left_arm_link7.glb"/>
+        <mesh filename="file://$(find galbot_one_description)/meshes/arm/left_arm_link7.glb"/>
       </geometry>
     </visual>
@@ -445,5 +446,5 @@
     <visual>
       <geometry>
-        <mesh filename="package://galbot_one_description/meshes/flange/flange.glb"/>
+        <mesh filename="file://$(find galbot_one_description)/meshes/flange/flange.glb"/>
       </geometry>
     </visual>
@@ -469,5 +470,5 @@
     <visual>
       <geometry>
-        <mesh filename="package://galbot_one_description/meshes/camera/arm_camera.glb"/>
+        <mesh filename="file://$(find galbot_one_description)/meshes/camera/arm_camera.glb"/>
       </geometry>
     </visual>

File: humanoid/Galbot/galbot_one_description/xacro/components/body.xacro (robot description, xacro)
@@ -209,5 +209,5 @@
       <origin/>
       <geometry>
-        <mesh filename="file://$(find galbot_one_description)/meshes/head/base1.glb"/>
+        <mesh filename="file://$(find galbot_one_description)/meshes/head/head_link2.glb"/>
       </geometry>
     </visual>

File: humanoid/Galbot/galbot_one_description/xacro/components/chassis.xacro (robot description, xacro)
@@ -18,5 +18,5 @@
       <visual>
         <geometry>
-          <mesh filename="package://galbot_one_description/meshes/chassis/chassis.glb"/>
+          <mesh filename="file://$(find galbot_one_description)/meshes/chassis/chassis.glb"/>
         </geometry>
       </visual>

File: humanoid/Galbot/galbot_one_description/xacro/components/gripper.xacro (robot description, xacro)
@@ -19,5 +19,5 @@
       <visual>
         <geometry>
-          <mesh filename="package://galbot_one_description/meshes/gripper_hitbot/base.glb"/>
+          <mesh filename="file://$(find galbot_one_description)/meshes/gripper_hitbot/base.glb"/>
         </geometry>
       </visual>
@@ -36,5 +36,5 @@
       <visual>
         <geometry>
-          <mesh filename="package://galbot_one_description/meshes/gripper_hitbot/link1.glb"/>
+          <mesh filename="file://$(find galbot_one_description)/meshes/gripper_hitbot/link1.glb"/>
         </geometry>
       </visual>
@@ -56,5 +56,5 @@
       <visual>
         <geometry>
-          <mesh filename="package://galbot_one_description/meshes/gripper_hitbot/link2.glb"/>
+          <mesh filename="file://$(find galbot_one_description)/meshes/gripper_hitbot/link2.glb"/>
         </geometry>
       </visual>
@@ -76,5 +76,5 @@
       <visual>
         <geometry>
-          <mesh filename="package://galbot_one_description/meshes/gripper_hitbot/link3.glb"/>
+          <mesh filename="file://$(find galbot_one_description)/meshes/gripper_hitbot/link3.glb"/>
         </geometry>
       </visual>
@@ -96,5 +96,5 @@
       <visual>
         <geometry>
-          <mesh filename="package://galbot_one_description/meshes/gripper_hitbot/link4.glb"/>
+          <mesh filename="file://$(find galbot_one_description)/meshes/gripper_hitbot/link4.glb"/>
         </geometry>
       </visual>
@@ -113,5 +113,5 @@
       <visual>
         <geometry>
-          <mesh filename="package://galbot_one_description/meshes/gripper_hitbot/link5.glb"/>
+          <mesh filename="file://$(find galbot_one_description)/meshes/gripper_hitbot/link5.glb"/>
         </geometry>
       </visual>
@@ -130,5 +130,5 @@
       <visual>
         <geometry>
-          <mesh filename="package://galbot_one_description/meshes/gripper_hitbot/link1.glb" scale="1 1 -1"/>
+          <mesh filename="file://$(find galbot_one_description)/meshes/gripper_hitbot/link1.glb" scale="1 1 -1"/>
         </geometry>
       </visual>
@@ -150,5 +150,5 @@
       <visual>
         <geometry>
-          <mesh filename="package://galbot_one_description/meshes/gripper_hitbot/link2.glb" scale="1 1 -1"/>
+          <mesh filename="file://$(find galbot_one_description)/meshes/gripper_hitbot/link2.glb" scale="1 1 -1"/>
         </geometry>
       </visual>
@@ -170,5 +170,5 @@
       <visual>
         <geometry>
-          <mesh filename="package://galbot_one_description/meshes/gripper_hitbot/link3.glb" scale="1 1 -1"/>
+          <mesh filename="file://$(find galbot_one_description)/meshes/gripper_hitbot/link3.glb" scale="1 1 -1"/>
         </geometry>
       </visual>
@@ -190,5 +190,5 @@
       <visual>
         <geometry>
-          <mesh filename="package://galbot_one_description/meshes/gripper_hitbot/link4.glb" scale="1 1 -1"/>
+          <mesh filename="file://$(find galbot_one_description)/meshes/gripper_hitbot/link4.glb" scale="1 1 -1"/>
         </geometry>
       </visual>
@@ -207,5 +207,5 @@
       <visual>
         <geometry>
-          <mesh filename="package://galbot_one_description/meshes/gripper_hitbot/link5.glb" scale="1 1 -1"/>
+          <mesh filename="file://$(find galbot_one_description)/meshes/gripper_hitbot/link5.glb" scale="1 1 -1"/>
         </geometry>
       </visual>
