Commit message: fix galbot one nav

File: humanoid/Galbot/galbot_one_description/xacro/components/chassis.xacro (robot description, xacro)
@@ -94,4 +94,10 @@
       <origin xyz="0.222 0 0.22772"/>
     </joint>
+    <link name="chassis_lidar_frame"/>
+    <joint name="chassis_lidar_frame_joint" type="fixed">
+      <origin xyz="0 0 0.012"/>
+      <parent link="chassis_lidar"/>
+      <child link="chassis_lidar_frame"/>
+    </joint>
   </xacro:macro>
 </robot>
