Commit message: add split control for ai2 bot2

File: humanoid/Ai2Robotics/ai2_bot2_description/urdf/ai2_bot2_inspire.urdf (robot description, URDF)
Before this commit: robot Ai2_Bot2, 42 links, 41 joints
Links:
- added link left_gripper_base, mass 0.072633; collision mesh filename=file:///home/ly/ros2_ws/install/inspire_description/share/i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; visual mesh filename=file:///home/ly/ros2_ws/install/inspire_description/share/i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
- added link left_gripper_tcp
- added link left_left_inner_link, mass 0.0038971; collision mesh filename=file:///home/ly/ros2_ws/install/inspire_description/share/i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; visual mesh filename=file:///home/ly/ros2_ws/install/inspire_description/share/i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
- added link left_left_outer_link, mass 0.0024292; collision mesh filename=file:///home/ly/ros2_ws/install/inspire_description/share/i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; visual mesh filename=file:///home/ly/ros2_ws/install/inspire_description/share/i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
- added link left_left_pad, mass 0.0045068; collision mesh filename=file:///home/ly/ros2_ws/install/inspire_description/share/i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; visual mesh filename=file:///home/ly/ros2_ws/install/inspire_description/share/i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
- added link left_right_inner_link, mass 0.0038971; collision mesh filename=file:///home/ly/ros2_ws/install/inspire_description/share/i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 scale=-1 1 1; visual mesh filename=file:///home/ly/ros2_ws/install/inspire_description/share/i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 scale=-1 1 1
- added link left_right_outer_link, mass 0.0024292; collision mesh filename=file:///home/ly/ros2_ws/install/inspire_description/share/i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 scale=-1 1 1; visual mesh filename=file:///home/ly/ros2_ws/install/inspire_description/share/i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 scale=-1 1 1
- added link left_right_pad, mass 0.0045068; collision mesh filename=file:///home/ly/ros2_ws/install/inspire_description/share/i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 scale=-1 1 1; visual mesh filename=file:///home/ly/ros2_ws/install/inspire_description/share/i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 scale=-1 1 1
- added link right_gripper_base, mass 0.072633; collision mesh filename=file:///home/ly/ros2_ws/install/inspire_description/share/i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; visual mesh filename=file:///home/ly/ros2_ws/install/inspire_description/share/i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
- added link right_gripper_tcp
- added link right_left_inner_link, mass 0.0038971; collision mesh filename=file:///home/ly/ros2_ws/install/inspire_description/share/i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; visual mesh filename=file:///home/ly/ros2_ws/install/inspire_description/share/i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
- added link right_left_outer_link, mass 0.0024292; collision mesh filename=file:///home/ly/ros2_ws/install/inspire_description/share/i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; visual mesh filename=file:///home/ly/ros2_ws/install/inspire_description/share/i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
- added link right_left_pad, mass 0.0045068; collision mesh filename=file:///home/ly/ros2_ws/install/inspire_description/share/i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; visual mesh filename=file:///home/ly/ros2_ws/install/inspire_description/share/i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
- added link right_right_inner_link, mass 0.0038971; collision mesh filename=file:///home/ly/ros2_ws/install/inspire_description/share/i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 scale=-1 1 1; visual mesh filename=file:///home/ly/ros2_ws/install/inspire_description/share/i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 scale=-1 1 1
- added link right_right_outer_link, mass 0.0024292; collision mesh filename=file:///home/ly/ros2_ws/install/inspire_description/share/i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 scale=-1 1 1; visual mesh filename=file:///home/ly/ros2_ws/install/inspire_description/share/i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 scale=-1 1 1
- added link right_right_pad, mass 0.0045068; collision mesh filename=file:///home/ly/ros2_ws/install/inspire_description/share/i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 scale=-1 1 1; visual mesh filename=file:///home/ly/ros2_ws/install/inspire_description/share/i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 scale=-1 1 1
Joints:
- added joint left_gripper_joint: type revolute, parent left_gripper_base, child left_left_outer_link, origin xyz=-0.04 -0.009 0.079, axis 0 -1 0, limit lower=0 upper=0.82 effort=50 velocity=3.141592653589793
- added joint left_gripper_mount: type fixed, parent left_ee, child left_gripper_base, origin xyz=0 0 0 rpy=0 0 1.5708
- added joint left_gripper_tcp_joint: type fixed, parent left_gripper_base, child left_gripper_tcp, origin xyz=0 0 0.13 rpy=0 0 0
- added joint left_left_inner_joint: type revolute, parent left_gripper_base, child left_left_inner_link, origin xyz=-0.03 -0.009 0.081, axis 0 -1 0, limit lower=0 upper=0.82 effort=50 velocity=3.141592653589793, mimic joint=left_gripper_joint
- added joint left_left_pad_joint: type revolute, parent left_left_outer_link, child left_left_pad, origin xyz=0.0223 0.003 0.035591, axis 0 1 0, limit lower=0 upper=0.82 effort=50 velocity=3.141592653589793, mimic joint=left_gripper_joint multiplier=1 offset=0
- added joint left_right_inner_joint: type revolute, parent left_gripper_base, child left_right_inner_link, origin xyz=0.03 -0.009 0.081, axis 0 1 0, limit lower=0 upper=0.82 effort=50 velocity=3.141592653589793, mimic joint=left_gripper_joint multiplier=1 offset=0
- added joint left_right_outer_joint: type revolute, parent left_gripper_base, child left_right_outer_link, origin xyz=0.04 -0.009 0.079, axis 0 1 0, limit lower=0 upper=0.82 effort=50 velocity=3.141592653589793, mimic joint=left_gripper_joint multiplier=1 offset=0
- added joint left_right_pad_joint: type revolute, parent left_right_outer_link, child left_right_pad, origin xyz=-0.0223 0.003 0.035591, axis 0 -1 0, limit lower=0 upper=0.82 effort=50 velocity=3.141592653589793, mimic joint=left_gripper_joint multiplier=1 offset=0
- added joint right_gripper_joint: type revolute, parent right_gripper_base, child right_left_outer_link, origin xyz=-0.04 -0.009 0.079, axis 0 -1 0, limit lower=0 upper=0.82 effort=50 velocity=3.141592653589793
- added joint right_gripper_mount: type fixed, parent right_ee, child right_gripper_base, origin xyz=0 0 0 rpy=0 0 1.5708
- added joint right_gripper_tcp_joint: type fixed, parent right_gripper_base, child right_gripper_tcp, origin xyz=0 0 0.13 rpy=0 0 0
- added joint right_left_inner_joint: type revolute, parent right_gripper_base, child right_left_inner_link, origin xyz=-0.03 -0.009 0.081, axis 0 -1 0, limit lower=0 upper=0.82 effort=50 velocity=3.141592653589793, mimic joint=right_gripper_joint
- added joint right_left_pad_joint: type revolute, parent right_left_outer_link, child right_left_pad, origin xyz=0.0223 0.003 0.035591, axis 0 1 0, limit lower=0 upper=0.82 effort=50 velocity=3.141592653589793, mimic joint=right_gripper_joint multiplier=1 offset=0
- added joint right_right_inner_joint: type revolute, parent right_gripper_base, child right_right_inner_link, origin xyz=0.03 -0.009 0.081, axis 0 1 0, limit lower=0 upper=0.82 effort=50 velocity=3.141592653589793, mimic joint=right_gripper_joint multiplier=1 offset=0
- added joint right_right_outer_joint: type revolute, parent right_gripper_base, child right_right_outer_link, origin xyz=0.04 -0.009 0.079, axis 0 1 0, limit lower=0 upper=0.82 effort=50 velocity=3.141592653589793, mimic joint=right_gripper_joint multiplier=1 offset=0
- added joint right_right_pad_joint: type revolute, parent right_right_outer_link, child right_right_pad, origin xyz=-0.0223 0.003 0.035591, axis 0 -1 0, limit lower=0 upper=0.82 effort=50 velocity=3.141592653589793, mimic joint=right_gripper_joint multiplier=1 offset=0

File: humanoid/Ai2Robotics/ai2_bot2_description/xacro/component.xacro (robot description, xacro)
@@ -9,5 +9,5 @@
     - left_arm / right_arm: root = base_link, both arms only, no body/chassis/ego
 -->
-<robot name="Ai2_Bot2_Arm" xmlns:xacro="http://www.ros.org/wiki/xacro">
+<robot name="Ai2_Bot2_Arms" xmlns:xacro="http://www.ros.org/wiki/xacro">
   <!-- component.launch.py default should show the base -->
   <xacro:arg name="type" default="base"/>
@@ -24,5 +24,4 @@
       <parent link="base_link"/>
       <child link="arm_base"/>
-      <origin xyz="0 0 0" rpy="0 0 0"/>
     </joint>
     <xacro:include filename="$(find ai2_bot2_description)/xacro/components/arm.xacro"/>
@@ -38,5 +37,5 @@
     <link name="ego"></link>
     <joint name="ego_joint" type="fixed">
-      <origin xyz="-0.061 0 0.3255" rpy="0 0 0" />
+      <origin xyz="-0.061 0 0.3255"/>
       <parent link="body_link4" />
       <child link="ego" />

File: humanoid/Ai2Robotics/ai2_bot2_description/xacro/components/arm.xacro (robot description, xacro)
@@ -22,19 +22,19 @@
                          iyy="1.7511135e-03" iyz="-1.7950155e-05" izz="1.1806738e-03"/>
             </inertial>
-<!--            <visual>-->
-<!--                <geometry>-->
-<!--                    <mesh filename="file://$(find ai2_bot2_description)/meshes/Visual/arm/arm_base_link.glb"-->
-<!--                          scale="1 ${direction} 1"/>-->
-<!--                </geometry>-->
-<!--                <material name="">-->
-<!--                    <color rgba="0.86667 0.86667 0.8902 1"/>-->
-<!--                </material>-->
-<!--            </visual>-->
-<!--            <collision>-->
-<!--                <geometry>-->
-<!--                    <mesh filename="file://$(find ai2_bot2_description)/meshes/Visual/arm/arm_base_link.glb"-->
-<!--                          scale="1 ${direction} 1"/>-->
-<!--                </geometry>-->
-<!--            </collision>-->
+            <visual>
+                <geometry>
+                    <mesh filename="file://$(find ai2_bot2_description)/meshes/Visual/arm/arm_base_link.glb"
+                          scale="1 ${direction} 1"/>
+                </geometry>
+                <material name="">
+                    <color rgba="0.86667 0.86667 0.8902 1"/>
+                </material>
+            </visual>
+            <collision>
+                <geometry>
+                    <mesh filename="file://$(find ai2_bot2_description)/meshes/Visual/arm/arm_base_link.glb"
+                          scale="1 ${direction} 1"/>
+                </geometry>
+            </collision>
         </link>
         <joint name="${prefix}joint0" type="fixed">

File: humanoid/Ai2Robotics/ai2_bot2_description/xacro/components/chassis.xacro (robot description, xacro)
@@ -15,5 +15,4 @@
     <link name="base_footprint"/>
     <joint name="base_footprint_joint" type="fixed">
-      <origin xyz="0 0 0" rpy="0 0 0"/>
       <parent link="base_footprint"/>
       <child link="base_link"/>
@@ -27,14 +26,12 @@
       </inertial>
       <visual>
-        <origin xyz="0 0 0" rpy="0 0 0"/>
         <geometry>
           <mesh filename="file://$(find ai2_bot2_description)/meshes/Visual/chassis/chassis.glb"/>
         </geometry>
-        <material name=""><color rgba="1 1 1 1"/></material>
-      </visual>
-      <collision>
-        <origin xyz="0 0 0" rpy="0 0 0"/>
-        <geometry>
-          <mesh filename="file://$(find ai2_bot2_description)/meshes/Visual/chassis/chassis.glb"/>
+      </visual>
+      <collision>
+        <origin xyz="0 0 0.1"/>
+        <geometry>
+          <box size="0.6 0.46 0.15"/>
         </geometry>
       </collision>
@@ -190,5 +187,5 @@
       <parent link="base_link" />
       <child link="driving_left_link" />
-      <axis xyz="1 0 0" />
+      <axis xyz="-1 0 0" />
       <limit effort="2000" velocity="10" />
     </joint>
@@ -211,5 +208,5 @@
       <parent link="base_link" />
       <child link="driving_right_link" />
-      <axis xyz="1 0 0" />
+      <axis xyz="-1 0 0" />
       <limit effort="2000" velocity="10" />
     </joint>
