Commit message: fix ai2 bot2

File: humanoid/Ai2Robotics/ai2_bot2_description/urdf/ai2_bot2.urdf (robot description, URDF)
Before this commit: robot Ai2_Bot2, 42 links, 41 joints
Links:
- link base_link: geometry collision box size=0.6 0.46 0.15; visual mesh filename=package://ai2_bot2_description/meshes/Visual/chassis/chassi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
- link body_link1: geometry collision mesh filename=package://ai2_bot2_description/meshes/Visual/body/link1.glb; visual mesh filename=package://ai2_bot2_description/meshes/Visual/body/link1.glb
- link body_link2: geometry collision mesh filename=package://ai2_bot2_description/meshes/Visual/body/link2.glb; visual mesh filename=package://ai2_bot2_description/meshes/Visual/body/link2.glb
- link body_link3: geometry collision mesh filename=package://ai2_bot2_description/meshes/Visual/body/link3.glb; visual mesh filename=package://ai2_bot2_description/meshes/Visual/body/link3.glb
- link body_link4: geometry collision mesh filename=package://ai2_bot2_description/meshes/Visual/body/link4.glb; visual mesh filename=package://ai2_bot2_description/meshes/Visual/body/link4.glb
- link driven_fl_link_h: geometry collision sphere radius=0.0375; visual mesh filename=package://ai2_bot2_description/meshes/Visual/chassis/driven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
- link driven_fl_link_v: geometry visual mesh filename=package://ai2_bot2_description/meshes/Visual/chassis/driven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
- link driven_fr_link_h: geometry collision sphere radius=0.0375; visual mesh filename=package://ai2_bot2_description/meshes/Visual/chassis/driven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
- link driven_fr_link_v: geometry visual mesh filename=package://ai2_bot2_description/meshes/Visual/chassis/driven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
- link driven_rl_link_h: geometry collision sphere radius=0.0375; visual mesh filename=package://ai2_bot2_description/meshes/Visual/chassis/driven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
- link driven_rl_link_v: geometry visual mesh filename=package://ai2_bot2_description/meshes/Visual/chassis/driven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
- link driven_rr_link_h: geometry collision sphere radius=0.0375; visual mesh filename=package://ai2_bot2_description/meshes/Visual/chassis/driven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
- link driven_rr_link_v: geometry visual mesh filename=package://ai2_bot2_description/meshes/Visual/chassis/driven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
- link driving_left_link: geometry collision cylinder length=0.034 radius=0.085; visual mesh filename=package://aidal_description/meshes/woosh_agv/wheel.glb scale=1 1 1
- link driving_right_link: geometry collision cylinder length=0.034 radius=0.085; visual mesh filename=package://aidal_description/meshes/woosh_agv/wheel.glb scale=1 1 -1
- link head_link2: geometry collision mesh filename=package://ai2_bot2_description/meshes/Visual/body/head_pitc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; visual mesh filename=package://ai2_bot2_description/meshes/Visual/body/head_pitc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
- link left_base_link: geometry collision mesh filename=package://ai2_bot2_description/meshes/Visual/arm/arm_base_l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 scale=1 1 1; visual mesh filename=package://ai2_bot2_description/meshes/Visual/arm/arm_base_l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 scale=1 1 1
- link left_link1: geometry collision mesh filename=package://ai2_bot2_description/meshes/Visual/arm/link1.glb scale=1 1 1; visual mesh filename=package://ai2_bot2_description/meshes/Visual/arm/link1.glb scale=1 1 1
- link left_link2: geometry collision mesh filename=package://ai2_bot2_description/meshes/Visual/arm/link2.glb scale=1 1 1; visual mesh filename=package://ai2_bot2_description/meshes/Visual/arm/link2.glb scale=1 1 1
- link left_link3: geometry collision mesh filename=package://ai2_bot2_description/meshes/Visual/arm/link3.glb scale=1 1 1; visual mesh filename=package://ai2_bot2_description/meshes/Visual/arm/link3.glb scale=1 1 1
- link left_link4: geometry collision mesh filename=package://ai2_bot2_description/meshes/Visual/arm/link4.glb scale=1 1 1; visual mesh filename=package://ai2_bot2_description/meshes/Visual/arm/link4.glb scale=1 1 1
- link left_link5: geometry collision mesh filename=package://ai2_bot2_description/meshes/Visual/arm/link5.glb scale=1 1 1; visual mesh filename=package://ai2_bot2_description/meshes/Visual/arm/link5.glb scale=1 1 1
- link left_link6: geometry collision mesh filename=package://ai2_bot2_description/meshes/Visual/arm/link6.glb scale=1 1 1; visual mesh filename=package://ai2_bot2_description/meshes/Visual/arm/link6.glb scale=1 1 1
- link left_link7: geometry collision mesh filename=package://ai2_bot2_description/meshes/Visual/arm/link7.glb scale=1 1 1; visual mesh filename=package://ai2_bot2_description/meshes/Visual/arm/link7.glb scale=1 1 1
- link left_link8: geometry visual mesh filename=package://rm75_description/meshes/ee/camera_stand_d405.glb; visual mesh filename=package://rm75_description/meshes/ee/ee_fb_camera.glb
- link right_base_link: geometry collision mesh filename=package://ai2_bot2_description/meshes/Visual/arm/arm_base_l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 scale=1 -1 1; visual mesh filename=package://ai2_bot2_description/meshes/Visual/arm/arm_base_l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 scale=1 -1 1
- link right_link1: geometry collision mesh filename=package://ai2_bot2_description/meshes/Visual/arm/link1.glb scale=1 -1 1; visual mesh filename=package://ai2_bot2_description/meshes/Visual/arm/link1.glb scale=1 -1 1
- link right_link2: geometry collision mesh filename=package://ai2_bot2_description/meshes/Visual/arm/link2.glb scale=1 1 -1; visual mesh filename=package://ai2_bot2_description/meshes/Visual/arm/link2.glb scale=1 1 -1
- link right_link3: geometry collision mesh filename=package://ai2_bot2_description/meshes/Visual/arm/link3.glb scale=-1 1 1; visual mesh filename=package://ai2_bot2_description/meshes/Visual/arm/link3.glb scale=-1 1 1
- link right_link4: geometry collision mesh filename=package://ai2_bot2_description/meshes/Visual/arm/link4.glb scale=-1 1 1; visual mesh filename=package://ai2_bot2_description/meshes/Visual/arm/link4.glb scale=-1 1 1
- link right_link5: geometry collision mesh filename=package://ai2_bot2_description/meshes/Visual/arm/link5.glb scale=-1 1 1; visual mesh filename=package://ai2_bot2_description/meshes/Visual/arm/link5.glb scale=-1 1 1
- link right_link6: geometry collision mesh filename=package://ai2_bot2_description/meshes/Visual/arm/link6.glb scale=1 -1 1; visual mesh filename=package://ai2_bot2_description/meshes/Visual/arm/link6.glb scale=1 -1 1
- link right_link7: geometry collision mesh filename=package://ai2_bot2_description/meshes/Visual/arm/link7.glb scale=1 1 -1; visual mesh filename=package://ai2_bot2_description/meshes/Visual/arm/link7.glb scale=1 1 -1
- link right_link8: geometry visual mesh filename=package://rm75_description/meshes/ee/camera_stand_d405.glb; visual mesh filename=package://rm75_description/meshes/ee/ee_fb_camera.glb

File: humanoid/Ai2Robotics/ai2_bot2_description/urdf/ai2_bot2_inspire.urdf (robot description, URDF)
Before this commit: robot Ai2_Bot2, 58 links, 57 joints
Links:
- link base_link: geometry collision box size=0.6 0.46 0.15; visual mesh filename=package://ai2_bot2_description/meshes/Visual/chassis/chassi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
- link body_link1: geometry collision mesh filename=package://ai2_bot2_description/meshes/Visual/body/link1.glb; visual mesh filename=package://ai2_bot2_description/meshes/Visual/body/link1.glb
- link body_link2: geometry collision mesh filename=package://ai2_bot2_description/meshes/Visual/body/link2.glb; visual mesh filename=package://ai2_bot2_description/meshes/Visual/body/link2.glb
- link body_link3: geometry collision mesh filename=package://ai2_bot2_description/meshes/Visual/body/link3.glb; visual mesh filename=package://ai2_bot2_description/meshes/Visual/body/link3.glb
- link body_link4: geometry collision mesh filename=package://ai2_bot2_description/meshes/Visual/body/link4.glb; visual mesh filename=package://ai2_bot2_description/meshes/Visual/body/link4.glb
- link driven_fl_link_h: geometry collision sphere radius=0.0375; visual mesh filename=package://ai2_bot2_description/meshes/Visual/chassis/driven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
- link driven_fl_link_v: geometry visual mesh filename=package://ai2_bot2_description/meshes/Visual/chassis/driven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
- link driven_fr_link_h: geometry collision sphere radius=0.0375; visual mesh filename=package://ai2_bot2_description/meshes/Visual/chassis/driven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
- link driven_fr_link_v: geometry visual mesh filename=package://ai2_bot2_description/meshes/Visual/chassis/driven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
- link driven_rl_link_h: geometry collision sphere radius=0.0375; visual mesh filename=package://ai2_bot2_description/meshes/Visual/chassis/driven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
- link driven_rl_link_v: geometry visual mesh filename=package://ai2_bot2_description/meshes/Visual/chassis/driven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
- link driven_rr_link_h: geometry collision sphere radius=0.0375; visual mesh filename=package://ai2_bot2_description/meshes/Visual/chassis/driven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
- link driven_rr_link_v: geometry visual mesh filename=package://ai2_bot2_description/meshes/Visual/chassis/driven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
- link driving_left_link: geometry collision cylinder length=0.034 radius=0.085; visual mesh filename=package://aidal_description/meshes/woosh_agv/wheel.glb scale=1 1 1
- link driving_right_link: geometry collision cylinder length=0.034 radius=0.085; visual mesh filename=package://aidal_description/meshes/woosh_agv/wheel.glb scale=1 1 -1
- link head_link2: geometry collision mesh filename=package://ai2_bot2_description/meshes/Visual/body/head_pitc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; visual mesh filename=package://ai2_bot2_description/meshes/Visual/body/head_pitc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
- link left_base_link: geometry collision mesh filename=package://ai2_bot2_description/meshes/Visual/arm/arm_base_l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 scale=1 1 1; visual mesh filename=package://ai2_bot2_description/meshes/Visual/arm/arm_base_l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 scale=1 1 1
- link left_gripper_base: geometry collision mesh filename=package://inspire_description/meshes/EG2-4C2/baselink.obj; visual mesh filename=package://inspire_description/meshes/EG2-4C2/baselink.obj
- link left_left_inner_link: geometry collision mesh filename=package://inspire_description/meshes/EG2-4C2/inner_link.obj; visual mesh filename=package://inspire_description/meshes/EG2-4C2/inner_link.obj
- link left_left_outer_link: geometry collision mesh filename=package://inspire_description/meshes/EG2-4C2/outer_link.obj; visual mesh filename=package://inspire_description/meshes/EG2-4C2/outer_link.obj
- link left_left_pad: geometry collision mesh filename=package://inspire_description/meshes/EG2-4C2/pad.obj; visual mesh filename=package://inspire_description/meshes/EG2-4C2/pad.obj
- link left_link1: geometry collision mesh filename=package://ai2_bot2_description/meshes/Visual/arm/link1.glb scale=1 1 1; visual mesh filename=package://ai2_bot2_description/meshes/Visual/arm/link1.glb scale=1 1 1
- link left_link2: geometry collision mesh filename=package://ai2_bot2_description/meshes/Visual/arm/link2.glb scale=1 1 1; visual mesh filename=package://ai2_bot2_description/meshes/Visual/arm/link2.glb scale=1 1 1
- link left_link3: geometry collision mesh filename=package://ai2_bot2_description/meshes/Visual/arm/link3.glb scale=1 1 1; visual mesh filename=package://ai2_bot2_description/meshes/Visual/arm/link3.glb scale=1 1 1
- link left_link4: geometry collision mesh filename=package://ai2_bot2_description/meshes/Visual/arm/link4.glb scale=1 1 1; visual mesh filename=package://ai2_bot2_description/meshes/Visual/arm/link4.glb scale=1 1 1
- link left_link5: geometry collision mesh filename=package://ai2_bot2_description/meshes/Visual/arm/link5.glb scale=1 1 1; visual mesh filename=package://ai2_bot2_description/meshes/Visual/arm/link5.glb scale=1 1 1
- link left_link6: geometry collision mesh filename=package://ai2_bot2_description/meshes/Visual/arm/link6.glb scale=1 1 1; visual mesh filename=package://ai2_bot2_description/meshes/Visual/arm/link6.glb scale=1 1 1
- link left_link7: geometry collision mesh filename=package://ai2_bot2_description/meshes/Visual/arm/link7.glb scale=1 1 1; visual mesh filename=package://ai2_bot2_description/meshes/Visual/arm/link7.glb scale=1 1 1
- link left_link8: geometry visual mesh filename=package://rm75_description/meshes/ee/camera_stand_d405.glb; visual mesh filename=package://rm75_description/meshes/ee/ee_fb_camera.glb
- link left_right_inner_link: geometry collision mesh filename=package://inspire_description/meshes/EG2-4C2/inner_link.obj scale=-1 1 1; visual mesh filename=package://inspire_description/meshes/EG2-4C2/inner_link.obj scale=-1 1 1
- link left_right_outer_link: geometry collision mesh filename=package://inspire_description/meshes/EG2-4C2/outer_link.obj scale=-1 1 1; visual mesh filename=package://inspire_description/meshes/EG2-4C2/outer_link.obj scale=-1 1 1
- link left_right_pad: geometry collision mesh filename=package://inspire_description/meshes/EG2-4C2/pad.obj scale=-1 1 1; visual mesh filename=package://inspire_description/meshes/EG2-4C2/pad.obj scale=-1 1 1
- link right_base_link: geometry collision mesh filename=package://ai2_bot2_description/meshes/Visual/arm/arm_base_l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 scale=1 -1 1; visual mesh filename=package://ai2_bot2_description/meshes/Visual/arm/arm_base_l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 scale=1 -1 1
- link right_gripper_base: geometry collision mesh filename=package://inspire_description/meshes/EG2-4C2/baselink.obj; visual mesh filename=package://inspire_description/meshes/EG2-4C2/baselink.obj
- link right_left_inner_link: geometry collision mesh filename=package://inspire_description/meshes/EG2-4C2/inner_link.obj; visual mesh filename=package://inspire_description/meshes/EG2-4C2/inner_link.obj
- link right_left_outer_link: geometry collision mesh filename=package://inspire_description/meshes/EG2-4C2/outer_link.obj; visual mesh filename=package://inspire_description/meshes/EG2-4C2/outer_link.obj
- link right_left_pad: geometry collision mesh filename=package://inspire_description/meshes/EG2-4C2/pad.obj; visual mesh filename=package://inspire_description/meshes/EG2-4C2/pad.obj
- link right_link1: geometry collision mesh filename=package://ai2_bot2_description/meshes/Visual/arm/link1.glb scale=1 -1 1; visual mesh filename=package://ai2_bot2_description/meshes/Visual/arm/link1.glb scale=1 -1 1
- link right_link2: geometry collision mesh filename=package://ai2_bot2_description/meshes/Visual/arm/link2.glb scale=1 1 -1; visual mesh filename=package://ai2_bot2_description/meshes/Visual/arm/link2.glb scale=1 1 -1
- link right_link3: geometry collision mesh filename=package://ai2_bot2_description/meshes/Visual/arm/link3.glb scale=-1 1 1; visual mesh filename=package://ai2_bot2_description/meshes/Visual/arm/link3.glb scale=-1 1 1
- link right_link4: geometry collision mesh filename=package://ai2_bot2_description/meshes/Visual/arm/link4.glb scale=-1 1 1; visual mesh filename=package://ai2_bot2_description/meshes/Visual/arm/link4.glb scale=-1 1 1
- link right_link5: geometry collision mesh filename=package://ai2_bot2_description/meshes/Visual/arm/link5.glb scale=-1 1 1; visual mesh filename=package://ai2_bot2_description/meshes/Visual/arm/link5.glb scale=-1 1 1
- link right_link6: geometry collision mesh filename=package://ai2_bot2_description/meshes/Visual/arm/link6.glb scale=1 -1 1; visual mesh filename=package://ai2_bot2_description/meshes/Visual/arm/link6.glb scale=1 -1 1
- link right_link7: geometry collision mesh filename=package://ai2_bot2_description/meshes/Visual/arm/link7.glb scale=1 1 -1; visual mesh filename=package://ai2_bot2_description/meshes/Visual/arm/link7.glb scale=1 1 -1
- link right_link8: geometry visual mesh filename=package://rm75_description/meshes/ee/camera_stand_d405.glb; visual mesh filename=package://rm75_description/meshes/ee/ee_fb_camera.glb
- link right_right_inner_link: geometry collision mesh filename=package://inspire_description/meshes/EG2-4C2/inner_link.obj scale=-1 1 1; visual mesh filename=package://inspire_description/meshes/EG2-4C2/inner_link.obj scale=-1 1 1
- link right_right_outer_link: geometry collision mesh filename=package://inspire_description/meshes/EG2-4C2/outer_link.obj scale=-1 1 1; visual mesh filename=package://inspire_description/meshes/EG2-4C2/outer_link.obj scale=-1 1 1
- link right_right_pad: geometry collision mesh filename=package://inspire_description/meshes/EG2-4C2/pad.obj scale=-1 1 1; visual mesh filename=package://inspire_description/meshes/EG2-4C2/pad.obj scale=-1 1 1

File: humanoid/Ai2Robotics/ai2_bot2_description/xacro/components/arm.xacro (robot description, xacro)
@@ -342,7 +342,7 @@
             </visual>
             <visual>
-                <origin xyz="-0.13322 -0.0005 0.044651" rpy="0 -1.5708 -1.5708"/>
-                <geometry>
-                    <mesh filename="file://$(find sensor_models)/meshes/d405/d405.obj"/>
+                <origin xyz="-0.13322 -0.0005 0.044651" rpy="0 0 3.1415"/>
+                <geometry>
+                    <mesh filename="file://$(find sensor_models)/meshes/realsense/d405.glb"/>
                 </geometry>
             </visual>

File: manipulator/AgileX/agilex_aloha_description/xacro/body/v1.xacro (robot description, xacro)
@@ -132,5 +132,5 @@
 	</joint>
 	<joint name="fl_base_joint" type="fixed">
-		<origin xyz="0.233 0.3 0.7775"/>
+		<origin xyz="0.233 0.3 0.775"/>
 		<parent link="base_footprint"/>
 		<child link="left_base_link"/>
@@ -138,5 +138,5 @@
 	</joint>
 	<joint name="fr_base_joint" type="fixed">
-		<origin xyz="0.233 -0.3 0.7775"/>
+		<origin xyz="0.233 -0.3 0.775"/>
 		<parent link="base_footprint"/>
 		<child link="right_base_link"/>
