Commit message: modify meshes and links

File: humanoid/Ai2Robotics/ai2_bot2_description/urdf/ai2_bot2.urdf (robot description, URDF)
Before this commit: robot Ai2_Bot2, 42 links, 41 joints
Links:
- added link back_camera; visual mesh filename=file:///home/ly/ros2_ws/install/sensor_models/share/sensor_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
- added link chassis_camera; visual mesh filename=file:///home/ly/ros2_ws/install/sensor_models/share/sensor_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
- added link front_camera; visual mesh filename=file:///home/ly/ros2_ws/install/sensor_models/share/sensor_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
- added link head_camera; visual mesh filename=file:///home/ly/ros2_ws/install/sensor_models/share/sensor_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
- link base_link: geometry collision box size=0.6 0.46 0.15; visual mesh filename=file:///home/ly/ros2_ws/install/ai2_bot2_description/share/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
- link body_link1: geometry collision mesh filename=file:///home/ly/ros2_ws/install/ai2_bot2_description/share/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; visual mesh filename=file:///home/ly/ros2_ws/install/ai2_bot2_description/share/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
- link body_link2: geometry collision mesh filename=file:///home/ly/ros2_ws/install/ai2_bot2_description/share/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; visual mesh filename=file:///home/ly/ros2_ws/install/ai2_bot2_description/share/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
- link body_link3: geometry collision mesh filename=file:///home/ly/ros2_ws/install/ai2_bot2_description/share/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; visual mesh filename=file:///home/ly/ros2_ws/install/ai2_bot2_description/share/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
- link body_link4: geometry collision mesh filename=file:///home/ly/ros2_ws/install/ai2_bot2_description/share/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; visual mesh filename=file:///home/ly/ros2_ws/install/ai2_bot2_description/share/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
- link charge_port: geometry visual mesh filename=file:///home/ly/ros2_ws/install/ai2_bot2_description/share/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
- link chassis_panel: geometry visual mesh filename=file:///home/ly/ros2_ws/install/aidal_description/share/aid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
- link driven_fl_link_h: geometry collision sphere radius=0.0375; visual mesh filename=file:///home/ly/ros2_ws/install/ai2_bot2_description/share/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
- link driven_fl_link_v: geometry visual mesh filename=file:///home/ly/ros2_ws/install/ai2_bot2_description/share/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
- link driven_fr_link_h: geometry collision sphere radius=0.0375; visual mesh filename=file:///home/ly/ros2_ws/install/ai2_bot2_description/share/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
- link driven_fr_link_v: geometry visual mesh filename=file:///home/ly/ros2_ws/install/ai2_bot2_description/share/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
- link driven_rl_link_h: geometry collision sphere radius=0.0375; visual mesh filename=file:///home/ly/ros2_ws/install/ai2_bot2_description/share/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
- link driven_rl_link_v: geometry visual mesh filename=file:///home/ly/ros2_ws/install/ai2_bot2_description/share/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
- link driven_rr_link_h: geometry collision sphere radius=0.0375; visual mesh filename=file:///home/ly/ros2_ws/install/ai2_bot2_description/share/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
- link driven_rr_link_v: geometry visual mesh filename=file:///home/ly/ros2_ws/install/ai2_bot2_description/share/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
- link driving_left_link: geometry collision cylinder length=0.034 radius=0.085; visual mesh filename=file:///home/ly/ros2_ws/install/aidal_description/share/aid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 scale=1 1 1
- link driving_right_link: geometry collision cylinder length=0.034 radius=0.085; visual mesh filename=file:///home/ly/ros2_ws/install/aidal_description/share/aid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 scale=1 1 -1
- link head_link2: geometry collision mesh filename=file:///home/ly/ros2_ws/install/ai2_bot2_description/share/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; visual mesh filename=file:///home/ly/ros2_ws/install/ai2_bot2_description/share/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
- link left_base_link: geometry collision mesh filename=file:///home/ly/ros2_ws/install/ai2_bot2_description/share/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 scale=1 1 1; visual mesh filename=file:///home/ly/ros2_ws/install/ai2_bot2_description/share/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 scale=1 1 1
- link left_link1: geometry collision mesh filename=file:///home/ly/ros2_ws/install/ai2_bot2_description/share/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 scale=1 1 1; visual mesh filename=file:///home/ly/ros2_ws/install/ai2_bot2_description/share/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 scale=1 1 1
- link left_link2: geometry collision mesh filename=file:///home/ly/ros2_ws/install/ai2_bot2_description/share/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 scale=1 1 1; visual mesh filename=file:///home/ly/ros2_ws/install/ai2_bot2_description/share/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 scale=1 1 1
- link left_link3: geometry collision mesh filename=file:///home/ly/ros2_ws/install/ai2_bot2_description/share/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 scale=1 1 1; visual mesh filename=file:///home/ly/ros2_ws/install/ai2_bot2_description/share/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 scale=1 1 1
- link left_link4: geometry collision mesh filename=file:///home/ly/ros2_ws/install/ai2_bot2_description/share/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 scale=1 1 1; visual mesh filename=file:///home/ly/ros2_ws/install/ai2_bot2_description/share/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 scale=1 1 1
- link left_link5: geometry collision mesh filename=file:///home/ly/ros2_ws/install/ai2_bot2_description/share/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 scale=1 1 1; visual mesh filename=file:///home/ly/ros2_ws/install/ai2_bot2_description/share/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 scale=1 1 1
- link left_link6: geometry collision mesh filename=file:///home/ly/ros2_ws/install/ai2_bot2_description/share/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 scale=1 1 1; visual mesh filename=file:///home/ly/ros2_ws/install/ai2_bot2_description/share/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 scale=1 1 1
- link left_link7: geometry collision mesh filename=file:///home/ly/ros2_ws/install/ai2_bot2_description/share/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 scale=1 1 1; visual mesh filename=file:///home/ly/ros2_ws/install/ai2_bot2_description/share/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 scale=1 1 1
- link left_link8: geometry visual mesh filename=file:///home/ly/ros2_ws/install/rm75_description/share/rm75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; visual mesh filename=file:///home/ly/ros2_ws/install/rm75_description/share/rm75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
- link lidar_link: geometry visual mesh filename=file:///home/ly/ros2_ws/install/sensor_models/share/sensor_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
- link right_base_link: geometry collision mesh filename=file:///home/ly/ros2_ws/install/ai2_bot2_description/share/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 scale=1 -1 1; visual mesh filename=file:///home/ly/ros2_ws/install/ai2_bot2_description/share/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 scale=1 -1 1
- link right_link1: geometry collision mesh filename=file:///home/ly/ros2_ws/install/ai2_bot2_description/share/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 scale=1 -1 1; visual mesh filename=file:///home/ly/ros2_ws/install/ai2_bot2_description/share/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 scale=1 -1 1
- link right_link2: geometry collision mesh filename=file:///home/ly/ros2_ws/install/ai2_bot2_description/share/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 scale=1 1 -1; visual mesh filename=file:///home/ly/ros2_ws/install/ai2_bot2_description/share/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 scale=1 1 -1
- link right_link3: geometry collision mesh filename=file:///home/ly/ros2_ws/install/ai2_bot2_description/share/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 scale=-1 1 1; visual mesh filename=file:///home/ly/ros2_ws/install/ai2_bot2_description/share/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 scale=-1 1 1
- link right_link4: geometry collision mesh filename=file:///home/ly/ros2_ws/install/ai2_bot2_description/share/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 scale=-1 1 1; visual mesh filename=file:///home/ly/ros2_ws/install/ai2_bot2_description/share/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 scale=-1 1 1
- link right_link5: geometry collision mesh filename=file:///home/ly/ros2_ws/install/ai2_bot2_description/share/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 scale=-1 1 1; visual mesh filename=file:///home/ly/ros2_ws/install/ai2_bot2_description/share/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 scale=-1 1 1
- link right_link6: geometry collision mesh filename=file:///home/ly/ros2_ws/install/ai2_bot2_description/share/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 scale=1 -1 1; visual mesh filename=file:///home/ly/ros2_ws/install/ai2_bot2_description/share/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 scale=1 -1 1
- link right_link7: geometry collision mesh filename=file:///home/ly/ros2_ws/install/ai2_bot2_description/share/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 scale=1 1 -1; visual mesh filename=file:///home/ly/ros2_ws/install/ai2_bot2_description/share/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 scale=1 1 -1
- link right_link8: geometry visual mesh filename=file:///home/ly/ros2_ws/install/rm75_description/share/rm75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; visual mesh filename=file:///home/ly/ros2_ws/install/rm75_description/share/rm75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
Joints:
- added joint back_camera: type fixed, parent body_link4, child back_camera, origin xyz=-0.1682 0 0.308 rpy=0 0.4887 3.14159
- added joint chassis_camera: type fixed, parent base_link, child chassis_camera, origin xyz=0.315 0 0.104 rpy=1.5708 0 1.5708
- added joint front_camera: type fixed, parent body_link4, child front_camera, origin xyz=0.1067 0 0.1805 rpy=0 0.38397 0
- added joint head_camera: type fixed, parent head_link2, child head_camera, origin xyz=0.089 0.0465 0 rpy=1.5708 0 0.5236
- joint charge_port: origin xyz=0.283736 0 0.056555 rpy=0 0 0 -> xyz=0.283736 0 0.056555
- joint driven_fl_joint_v: origin xyz=0.215 0.15 0.085704 rpy=0 0 0 -> xyz=0.215 0.15 0.085704
- joint driven_fr_joint_v: origin xyz=0.215 -0.15 0.085704 rpy=0 0 0 -> xyz=0.215 -0.15 0.085704
- joint driven_rl_joint_v: origin xyz=-0.215 0.15 0.085704 rpy=0 0 0 -> xyz=-0.215 0.15 0.085704
- joint driven_rr_joint_v: origin xyz=-0.215 -0.15 0.085704 rpy=0 0 0 -> xyz=-0.215 -0.15 0.085704

File: humanoid/Ai2Robotics/ai2_bot2_description/urdf/ai2_bot2_inspire.urdf (robot description, URDF)
Before this commit: robot Ai2_Bot2, 58 links, 57 joints
Links:
- added link back_camera; visual mesh filename=file:///home/ly/ros2_ws/install/sensor_models/share/sensor_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
- added link chassis_camera; visual mesh filename=file:///home/ly/ros2_ws/install/sensor_models/share/sensor_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
- added link front_camera; visual mesh filename=file:///home/ly/ros2_ws/install/sensor_models/share/sensor_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
- added link head_camera; visual mesh filename=file:///home/ly/ros2_ws/install/sensor_models/share/sensor_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
- added link left_eef
- added link right_eef
- link base_link: geometry collision box size=0.6 0.46 0.15; visual mesh filename=file:///home/ly/ros2_ws/install/ai2_bot2_description/share/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
- link body_link1: geometry collision mesh filename=file:///home/ly/ros2_ws/install/ai2_bot2_description/share/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; visual mesh filename=file:///home/ly/ros2_ws/install/ai2_bot2_description/share/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
- link body_link2: geometry collision mesh filename=file:///home/ly/ros2_ws/install/ai2_bot2_description/share/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; visual mesh filename=file:///home/ly/ros2_ws/install/ai2_bot2_description/share/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
- link body_link3: geometry collision mesh filename=file:///home/ly/ros2_ws/install/ai2_bot2_description/share/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; visual mesh filename=file:///home/ly/ros2_ws/install/ai2_bot2_description/share/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
- link body_link4: geometry collision mesh filename=file:///home/ly/ros2_ws/install/ai2_bot2_description/share/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; visual mesh filename=file:///home/ly/ros2_ws/install/ai2_bot2_description/share/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
- link charge_port: geometry visual mesh filename=file:///home/ly/ros2_ws/install/ai2_bot2_description/share/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
- link chassis_panel: geometry visual mesh filename=file:///home/ly/ros2_ws/install/aidal_description/share/aid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
- link driven_fl_link_h: geometry collision sphere radius=0.0375; visual mesh filename=file:///home/ly/ros2_ws/install/ai2_bot2_description/share/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
- link driven_fl_link_v: geometry visual mesh filename=file:///home/ly/ros2_ws/install/ai2_bot2_description/share/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
- link driven_fr_link_h: geometry collision sphere radius=0.0375; visual mesh filename=file:///home/ly/ros2_ws/install/ai2_bot2_description/share/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
- link driven_fr_link_v: geometry visual mesh filename=file:///home/ly/ros2_ws/install/ai2_bot2_description/share/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
- link driven_rl_link_h: geometry collision sphere radius=0.0375; visual mesh filename=file:///home/ly/ros2_ws/install/ai2_bot2_description/share/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
- link driven_rl_link_v: geometry visual mesh filename=file:///home/ly/ros2_ws/install/ai2_bot2_description/share/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
- link driven_rr_link_h: geometry collision sphere radius=0.0375; visual mesh filename=file:///home/ly/ros2_ws/install/ai2_bot2_description/share/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
- link driven_rr_link_v: geometry visual mesh filename=file:///home/ly/ros2_ws/install/ai2_bot2_description/share/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
- link driving_left_link: geometry collision cylinder length=0.034 radius=0.085; visual mesh filename=file:///home/ly/ros2_ws/install/aidal_description/share/aid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 scale=1 1 1
- link driving_right_link: geometry collision cylinder length=0.034 radius=0.085; visual mesh filename=file:///home/ly/ros2_ws/install/aidal_description/share/aid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 scale=1 1 -1
- link head_link2: geometry collision mesh filename=file:///home/ly/ros2_ws/install/ai2_bot2_description/share/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; visual mesh filename=file:///home/ly/ros2_ws/install/ai2_bot2_description/share/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
- link left_base_link: geometry collision mesh filename=file:///home/ly/ros2_ws/install/ai2_bot2_description/share/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 scale=1 1 1; visual mesh filename=file:///home/ly/ros2_ws/install/ai2_bot2_description/share/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 scale=1 1 1
- link left_gripper_base: geometry collision mesh filename=file:///home/ly/ros2_ws/install/inspire_description/share/i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; visual mesh filename=file:///home/ly/ros2_ws/install/inspire_description/share/i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
- link left_left_inner_link: geometry collision mesh filename=file:///home/ly/ros2_ws/install/inspire_description/share/i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; visual mesh filename=file:///home/ly/ros2_ws/install/inspire_description/share/i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
- link left_left_outer_link: geometry collision mesh filename=file:///home/ly/ros2_ws/install/inspire_description/share/i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; visual mesh filename=file:///home/ly/ros2_ws/install/inspire_description/share/i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
- link left_left_pad: geometry collision mesh filename=file:///home/ly/ros2_ws/install/inspire_description/share/i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; visual mesh filename=file:///home/ly/ros2_ws/install/inspire_description/share/i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
- link left_link1: geometry collision mesh filename=file:///home/ly/ros2_ws/install/ai2_bot2_description/share/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 scale=1 1 1; visual mesh filename=file:///home/ly/ros2_ws/install/ai2_bot2_description/share/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 scale=1 1 1
- link left_link2: geometry collision mesh filename=file:///home/ly/ros2_ws/install/ai2_bot2_description/share/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 scale=1 1 1; visual mesh filename=file:///home/ly/ros2_ws/install/ai2_bot2_description/share/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 scale=1 1 1
- link left_link3: geometry collision mesh filename=file:///home/ly/ros2_ws/install/ai2_bot2_description/share/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 scale=1 1 1; visual mesh filename=file:///home/ly/ros2_ws/install/ai2_bot2_description/share/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 scale=1 1 1
- link left_link4: geometry collision mesh filename=file:///home/ly/ros2_ws/install/ai2_bot2_description/share/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 scale=1 1 1; visual mesh filename=file:///home/ly/ros2_ws/install/ai2_bot2_description/share/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 scale=1 1 1
- link left_link5: geometry collision mesh filename=file:///home/ly/ros2_ws/install/ai2_bot2_description/share/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 scale=1 1 1; visual mesh filename=file:///home/ly/ros2_ws/install/ai2_bot2_description/share/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 scale=1 1 1
- link left_link6: geometry collision mesh filename=file:///home/ly/ros2_ws/install/ai2_bot2_description/share/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 scale=1 1 1; visual mesh filename=file:///home/ly/ros2_ws/install/ai2_bot2_description/share/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 scale=1 1 1
- link left_link7: geometry collision mesh filename=file:///home/ly/ros2_ws/install/ai2_bot2_description/share/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 scale=1 1 1; visual mesh filename=file:///home/ly/ros2_ws/install/ai2_bot2_description/share/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 scale=1 1 1
- link left_link8: geometry visual mesh filename=file:///home/ly/ros2_ws/install/rm75_description/share/rm75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; visual mesh filename=file:///home/ly/ros2_ws/install/rm75_description/share/rm75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
- link left_right_inner_link: geometry collision mesh filename=file:///home/ly/ros2_ws/install/inspire_description/share/i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 scale=-1 1 1; visual mesh filename=file:///home/ly/ros2_ws/install/inspire_description/share/i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 scale=-1 1 1
- link left_right_outer_link: geometry collision mesh filename=file:///home/ly/ros2_ws/install/inspire_description/share/i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 scale=-1 1 1; visual mesh filename=file:///home/ly/ros2_ws/install/inspire_description/share/i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 scale=-1 1 1
- link left_right_pad: geometry collision mesh filename=file:///home/ly/ros2_ws/install/inspire_description/share/i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 scale=-1 1 1; visual mesh filename=file:///home/ly/ros2_ws/install/inspire_description/share/i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 scale=-1 1 1
- link lidar_link: geometry visual mesh filename=file:///home/ly/ros2_ws/install/sensor_models/share/sensor_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
- link right_base_link: geometry collision mesh filename=file:///home/ly/ros2_ws/install/ai2_bot2_description/share/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 scale=1 -1 1; visual mesh filename=file:///home/ly/ros2_ws/install/ai2_bot2_description/share/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 scale=1 -1 1
- link right_gripper_base: geometry collision mesh filename=file:///home/ly/ros2_ws/install/inspire_description/share/i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; visual mesh filename=file:///home/ly/ros2_ws/install/inspire_description/share/i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
- link right_left_inner_link: geometry collision mesh filename=file:///home/ly/ros2_ws/install/inspire_description/share/i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; visual mesh filename=file:///home/ly/ros2_ws/install/inspire_description/share/i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
- link right_left_outer_link: geometry collision mesh filename=file:///home/ly/ros2_ws/install/inspire_description/share/i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; visual mesh filename=file:///home/ly/ros2_ws/install/inspire_description/share/i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
- link right_left_pad: geometry collision mesh filename=file:///home/ly/ros2_ws/install/inspire_description/share/i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; visual mesh filename=file:///home/ly/ros2_ws/install/inspire_description/share/i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
- link right_link1: geometry collision mesh filename=file:///home/ly/ros2_ws/install/ai2_bot2_description/share/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 scale=1 -1 1; visual mesh filename=file:///home/ly/ros2_ws/install/ai2_bot2_description/share/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 scale=1 -1 1
- link right_link2: geometry collision mesh filename=file:///home/ly/ros2_ws/install/ai2_bot2_description/share/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 scale=1 1 -1; visual mesh filename=file:///home/ly/ros2_ws/install/ai2_bot2_description/share/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 scale=1 1 -1
- link right_link3: geometry collision mesh filename=file:///home/ly/ros2_ws/install/ai2_bot2_description/share/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 scale=-1 1 1; visual mesh filename=file:///home/ly/ros2_ws/install/ai2_bot2_description/share/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 scale=-1 1 1
- link right_link4: geometry collision mesh filename=file:///home/ly/ros2_ws/install/ai2_bot2_description/share/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 scale=-1 1 1; visual mesh filename=file:///home/ly/ros2_ws/install/ai2_bot2_description/share/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 scale=-1 1 1
- link right_link5: geometry collision mesh filename=file:///home/ly/ros2_ws/install/ai2_bot2_description/share/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 scale=-1 1 1; visual mesh filename=file:///home/ly/ros2_ws/install/ai2_bot2_description/share/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 scale=-1 1 1
- link right_link6: geometry collision mesh filename=file:///home/ly/ros2_ws/install/ai2_bot2_description/share/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 scale=1 -1 1; visual mesh filename=file:///home/ly/ros2_ws/install/ai2_bot2_description/share/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 scale=1 -1 1
- link right_link7: geometry collision mesh filename=file:///home/ly/ros2_ws/install/ai2_bot2_description/share/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 scale=1 1 -1; visual mesh filename=file:///home/ly/ros2_ws/install/ai2_bot2_description/share/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 scale=1 1 -1
- link right_link8: geometry visual mesh filename=file:///home/ly/ros2_ws/install/rm75_description/share/rm75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; visual mesh filename=file:///home/ly/ros2_ws/install/rm75_description/share/rm75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
- link right_right_inner_link: geometry collision mesh filename=file:///home/ly/ros2_ws/install/inspire_description/share/i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 scale=-1 1 1; visual mesh filename=file:///home/ly/ros2_ws/install/inspire_description/share/i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 scale=-1 1 1
- link right_right_outer_link: geometry collision mesh filename=file:///home/ly/ros2_ws/install/inspire_description/share/i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 scale=-1 1 1; visual mesh filename=file:///home/ly/ros2_ws/install/inspire_description/share/i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 scale=-1 1 1
- link right_right_pad: geometry collision mesh filename=file:///home/ly/ros2_ws/install/inspire_description/share/i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 scale=-1 1 1; visual mesh filename=file:///home/ly/ros2_ws/install/inspire_description/share/i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 scale=-1 1 1
Joints:
- added joint back_camera: type fixed, parent body_link4, child back_camera, origin xyz=-0.1682 0 0.308 rpy=0 0.4887 3.14159
- added joint chassis_camera: type fixed, parent base_link, child chassis_camera, origin xyz=0.315 0 0.104 rpy=1.5708 0 1.5708
- added joint front_camera: type fixed, parent body_link4, child front_camera, origin xyz=0.1067 0 0.1805 rpy=0 0.38397 0
- added joint head_camera: type fixed, parent head_link2, child head_camera, origin xyz=0.089 0.0465 0 rpy=1.5708 0 0.5236
- added joint left_eef_joint: type fixed, parent left_gripper_base, child left_eef, origin xyz=0 0 0.14
- added joint right_eef_joint: type fixed, parent right_gripper_base, child right_eef, origin xyz=0 0 0.14
- joint charge_port: origin xyz=0.283736 0 0.056555 rpy=0 0 0 -> xyz=0.283736 0 0.056555
- joint driven_fl_joint_v: origin xyz=0.215 0.15 0.085704 rpy=0 0 0 -> xyz=0.215 0.15 0.085704
- joint driven_fr_joint_v: origin xyz=0.215 -0.15 0.085704 rpy=0 0 0 -> xyz=0.215 -0.15 0.085704
- joint driven_rl_joint_v: origin xyz=-0.215 0.15 0.085704 rpy=0 0 0 -> xyz=-0.215 0.15 0.085704
- joint driven_rr_joint_v: origin xyz=-0.215 -0.15 0.085704 rpy=0 0 0 -> xyz=-0.215 -0.15 0.085704
