Commit message: fix paths

File: humanoid/Ai2Robotics/ai2_bot2_description/urdf/ai2_bot2.urdf (robot description, URDF)
Before this commit: robot Ai2_Bot2, 46 links, 45 joints
Links:
- link back_camera: geometry visual mesh filename=package://sensor_models/meshes/d435/d435.obj
- link base_link: geometry collision box size=0.6 0.46 0.15; visual mesh filename=package://ai2_bot2_description/meshes/Visual/chassis/chassi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
- link body_link1: geometry collision mesh filename=package://ai2_bot2_description/meshes/Visual/body/link1.glb; visual mesh filename=package://ai2_bot2_description/meshes/Visual/body/link1.glb
- link body_link2: geometry collision mesh filename=package://ai2_bot2_description/meshes/Visual/body/link2.glb; visual mesh filename=package://ai2_bot2_description/meshes/Visual/body/link2.glb
- link body_link3: geometry collision mesh filename=package://ai2_bot2_description/meshes/Visual/body/link3.glb; visual mesh filename=package://ai2_bot2_description/meshes/Visual/body/link3.glb
- link body_link4: geometry collision mesh filename=package://ai2_bot2_description/meshes/Visual/body/link4.glb; visual mesh filename=package://ai2_bot2_description/meshes/Visual/body/link4.glb
- link charge_port: geometry visual mesh filename=package://ai2_bot2_description/meshes/Visual/chassis/charge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
- link chassis_camera: geometry visual mesh filename=package://sensor_models/meshes/orbbec/Dabai_DW.glb
- link chassis_panel: geometry visual mesh filename=package://aidal_description/meshes/woosh_agv/panel.glb
- link driven_fl_link_h: geometry collision sphere radius=0.0375; visual mesh filename=package://ai2_bot2_description/meshes/Visual/chassis/driven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
- link driven_fl_link_v: geometry visual mesh filename=package://ai2_bot2_description/meshes/Visual/chassis/driven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
- link driven_fr_link_h: geometry collision sphere radius=0.0375; visual mesh filename=package://ai2_bot2_description/meshes/Visual/chassis/driven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
- link driven_fr_link_v: geometry visual mesh filename=package://ai2_bot2_description/meshes/Visual/chassis/driven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
- link driven_rl_link_h: geometry collision sphere radius=0.0375; visual mesh filename=package://ai2_bot2_description/meshes/Visual/chassis/driven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
- link driven_rl_link_v: geometry visual mesh filename=package://ai2_bot2_description/meshes/Visual/chassis/driven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
- link driven_rr_link_h: geometry collision sphere radius=0.0375; visual mesh filename=package://ai2_bot2_description/meshes/Visual/chassis/driven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
- link driven_rr_link_v: geometry visual mesh filename=package://ai2_bot2_description/meshes/Visual/chassis/driven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
- link driving_left_link: geometry collision cylinder length=0.034 radius=0.085; visual mesh filename=package://aidal_description/meshes/woosh_agv/wheel.glb scale=1 1 1
- link driving_right_link: geometry collision cylinder length=0.034 radius=0.085; visual mesh filename=package://aidal_description/meshes/woosh_agv/wheel.glb scale=1 1 -1
- link front_camera: geometry visual mesh filename=package://sensor_models/meshes/d435/d435.obj
- link head_camera: geometry visual mesh filename=package://sensor_models/meshes/d435/d435.obj
- link head_link2: geometry collision mesh filename=package://ai2_bot2_description/meshes/Visual/body/head2.glb; visual mesh filename=package://ai2_bot2_description/meshes/Visual/body/head2.glb
- link left_base_link: geometry collision mesh filename=package://ai2_bot2_description/meshes/Visual/arm/arm_base_l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 scale=1 1 1; visual mesh filename=package://ai2_bot2_description/meshes/Visual/arm/arm_base_l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 scale=1 1 1
- link left_link1: geometry collision mesh filename=package://ai2_bot2_description/meshes/Visual/arm/link1.glb scale=1 1 1; visual mesh filename=package://ai2_bot2_description/meshes/Visual/arm/link1.glb scale=1 1 1
- link left_link2: geometry collision mesh filename=package://ai2_bot2_description/meshes/Visual/arm/link2.glb scale=1 1 1; visual mesh filename=package://ai2_bot2_description/meshes/Visual/arm/link2.glb scale=1 1 1
- link left_link3: geometry collision mesh filename=package://ai2_bot2_description/meshes/Visual/arm/link3.glb scale=1 1 1; visual mesh filename=package://ai2_bot2_description/meshes/Visual/arm/link3.glb scale=1 1 1
- link left_link4: geometry collision mesh filename=package://ai2_bot2_description/meshes/Visual/arm/link4.glb scale=1 1 1; visual mesh filename=package://ai2_bot2_description/meshes/Visual/arm/link4.glb scale=1 1 1
- link left_link5: geometry collision mesh filename=package://ai2_bot2_description/meshes/Visual/arm/link5.glb scale=1 1 1; visual mesh filename=package://ai2_bot2_description/meshes/Visual/arm/link5.glb scale=1 1 1
- link left_link6: geometry collision mesh filename=package://ai2_bot2_description/meshes/Visual/arm/link6.glb scale=1 1 1; visual mesh filename=package://ai2_bot2_description/meshes/Visual/arm/link6.glb scale=1 1 1
- link left_link7: geometry collision mesh filename=package://ai2_bot2_description/meshes/Visual/arm/link7.glb scale=1 1 1; visual mesh filename=package://ai2_bot2_description/meshes/Visual/arm/link7.glb scale=1 1 1
- link left_link8: geometry visual mesh filename=package://rm75_description/meshes/ee/camera_stand_d405.glb; visual mesh filename=package://rm75_description/meshes/ee/ee_fb_camera.glb
- link lidar_link: geometry visual mesh filename=package://sensor_models/meshes/orbbec/ms500.glb
- link right_base_link: geometry collision mesh filename=package://ai2_bot2_description/meshes/Visual/arm/arm_base_l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 scale=1 -1 1; visual mesh filename=package://ai2_bot2_description/meshes/Visual/arm/arm_base_l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 scale=1 -1 1
- link right_link1: geometry collision mesh filename=package://ai2_bot2_description/meshes/Visual/arm/link1.glb scale=1 -1 1; visual mesh filename=package://ai2_bot2_description/meshes/Visual/arm/link1.glb scale=1 -1 1
- link right_link2: geometry collision mesh filename=package://ai2_bot2_description/meshes/Visual/arm/link2.glb scale=1 1 -1; visual mesh filename=package://ai2_bot2_description/meshes/Visual/arm/link2.glb scale=1 1 -1
- link right_link3: geometry collision mesh filename=package://ai2_bot2_description/meshes/Visual/arm/link3.glb scale=-1 1 1; visual mesh filename=package://ai2_bot2_description/meshes/Visual/arm/link3.glb scale=-1 1 1
- link right_link4: geometry collision mesh filename=package://ai2_bot2_description/meshes/Visual/arm/link4.glb scale=-1 1 1; visual mesh filename=package://ai2_bot2_description/meshes/Visual/arm/link4.glb scale=-1 1 1
- link right_link5: geometry collision mesh filename=package://ai2_bot2_description/meshes/Visual/arm/link5.glb scale=-1 1 1; visual mesh filename=package://ai2_bot2_description/meshes/Visual/arm/link5.glb scale=-1 1 1
- link right_link6: geometry collision mesh filename=package://ai2_bot2_description/meshes/Visual/arm/link6.glb scale=1 -1 1; visual mesh filename=package://ai2_bot2_description/meshes/Visual/arm/link6.glb scale=1 -1 1
- link right_link7: geometry collision mesh filename=package://ai2_bot2_description/meshes/Visual/arm/link7.glb scale=1 1 -1; visual mesh filename=package://ai2_bot2_description/meshes/Visual/arm/link7.glb scale=1 1 -1
- link right_link8: geometry visual mesh filename=package://rm75_description/meshes/ee/camera_stand_d405.glb; visual mesh filename=package://rm75_description/meshes/ee/ee_fb_camera.glb

File: humanoid/Ai2Robotics/ai2_bot2_description/urdf/ai2_bot2_inspire.urdf (robot description, URDF)
Before this commit: robot Ai2_Bot2, 64 links, 63 joints
Links:
- link back_camera: geometry visual mesh filename=package://sensor_models/meshes/d435/d435.obj
- link base_link: geometry collision box size=0.6 0.46 0.15; visual mesh filename=package://ai2_bot2_description/meshes/Visual/chassis/chassi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
- link body_link1: geometry collision mesh filename=package://ai2_bot2_description/meshes/Visual/body/link1.glb; visual mesh filename=package://ai2_bot2_description/meshes/Visual/body/link1.glb
- link body_link2: geometry collision mesh filename=package://ai2_bot2_description/meshes/Visual/body/link2.glb; visual mesh filename=package://ai2_bot2_description/meshes/Visual/body/link2.glb
- link body_link3: geometry collision mesh filename=package://ai2_bot2_description/meshes/Visual/body/link3.glb; visual mesh filename=package://ai2_bot2_description/meshes/Visual/body/link3.glb
- link body_link4: geometry collision mesh filename=package://ai2_bot2_description/meshes/Visual/body/link4.glb; visual mesh filename=package://ai2_bot2_description/meshes/Visual/body/link4.glb
- link charge_port: geometry visual mesh filename=package://ai2_bot2_description/meshes/Visual/chassis/charge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
- link chassis_camera: geometry visual mesh filename=package://sensor_models/meshes/orbbec/Dabai_DW.glb
- link chassis_panel: geometry visual mesh filename=package://aidal_description/meshes/woosh_agv/panel.glb
- link driven_fl_link_h: geometry collision sphere radius=0.0375; visual mesh filename=package://ai2_bot2_description/meshes/Visual/chassis/driven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
- link driven_fl_link_v: geometry visual mesh filename=package://ai2_bot2_description/meshes/Visual/chassis/driven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
- link driven_fr_link_h: geometry collision sphere radius=0.0375; visual mesh filename=package://ai2_bot2_description/meshes/Visual/chassis/driven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
- link driven_fr_link_v: geometry visual mesh filename=package://ai2_bot2_description/meshes/Visual/chassis/driven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
- link driven_rl_link_h: geometry collision sphere radius=0.0375; visual mesh filename=package://ai2_bot2_description/meshes/Visual/chassis/driven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
- link driven_rl_link_v: geometry visual mesh filename=package://ai2_bot2_description/meshes/Visual/chassis/driven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
- link driven_rr_link_h: geometry collision sphere radius=0.0375; visual mesh filename=package://ai2_bot2_description/meshes/Visual/chassis/driven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
- link driven_rr_link_v: geometry visual mesh filename=package://ai2_bot2_description/meshes/Visual/chassis/driven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
- link driving_left_link: geometry collision cylinder length=0.034 radius=0.085; visual mesh filename=package://aidal_description/meshes/woosh_agv/wheel.glb scale=1 1 1
- link driving_right_link: geometry collision cylinder length=0.034 radius=0.085; visual mesh filename=package://aidal_description/meshes/woosh_agv/wheel.glb scale=1 1 -1
- link front_camera: geometry visual mesh filename=package://sensor_models/meshes/d435/d435.obj
- link head_camera: geometry visual mesh filename=package://sensor_models/meshes/d435/d435.obj
- link head_link2: geometry collision mesh filename=package://ai2_bot2_description/meshes/Visual/body/head2.glb; visual mesh filename=package://ai2_bot2_description/meshes/Visual/body/head2.glb
- link left_base_link: geometry collision mesh filename=package://ai2_bot2_description/meshes/Visual/arm/arm_base_l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 scale=1 1 1; visual mesh filename=package://ai2_bot2_description/meshes/Visual/arm/arm_base_l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 scale=1 1 1
- link left_gripper_base: geometry collision mesh filename=package://inspire_description/meshes/EG2-4C2/baselink.obj; visual mesh filename=package://inspire_description/meshes/EG2-4C2/baselink.obj
- link left_left_inner_link: geometry collision mesh filename=package://inspire_description/meshes/EG2-4C2/inner_link.obj; visual mesh filename=package://inspire_description/meshes/EG2-4C2/inner_link.obj
- link left_left_outer_link: geometry collision mesh filename=package://inspire_description/meshes/EG2-4C2/outer_link.obj; visual mesh filename=package://inspire_description/meshes/EG2-4C2/outer_link.obj
- link left_left_pad: geometry collision mesh filename=package://inspire_description/meshes/EG2-4C2/pad.obj; visual mesh filename=package://inspire_description/meshes/EG2-4C2/pad.obj
- link left_link1: geometry collision mesh filename=package://ai2_bot2_description/meshes/Visual/arm/link1.glb scale=1 1 1; visual mesh filename=package://ai2_bot2_description/meshes/Visual/arm/link1.glb scale=1 1 1
- link left_link2: geometry collision mesh filename=package://ai2_bot2_description/meshes/Visual/arm/link2.glb scale=1 1 1; visual mesh filename=package://ai2_bot2_description/meshes/Visual/arm/link2.glb scale=1 1 1
- link left_link3: geometry collision mesh filename=package://ai2_bot2_description/meshes/Visual/arm/link3.glb scale=1 1 1; visual mesh filename=package://ai2_bot2_description/meshes/Visual/arm/link3.glb scale=1 1 1
- link left_link4: geometry collision mesh filename=package://ai2_bot2_description/meshes/Visual/arm/link4.glb scale=1 1 1; visual mesh filename=package://ai2_bot2_description/meshes/Visual/arm/link4.glb scale=1 1 1
- link left_link5: geometry collision mesh filename=package://ai2_bot2_description/meshes/Visual/arm/link5.glb scale=1 1 1; visual mesh filename=package://ai2_bot2_description/meshes/Visual/arm/link5.glb scale=1 1 1
- link left_link6: geometry collision mesh filename=package://ai2_bot2_description/meshes/Visual/arm/link6.glb scale=1 1 1; visual mesh filename=package://ai2_bot2_description/meshes/Visual/arm/link6.glb scale=1 1 1
- link left_link7: geometry collision mesh filename=package://ai2_bot2_description/meshes/Visual/arm/link7.glb scale=1 1 1; visual mesh filename=package://ai2_bot2_description/meshes/Visual/arm/link7.glb scale=1 1 1
- link left_link8: geometry visual mesh filename=package://rm75_description/meshes/ee/camera_stand_d405.glb; visual mesh filename=package://rm75_description/meshes/ee/ee_fb_camera.glb
- link left_right_inner_link: geometry collision mesh filename=package://inspire_description/meshes/EG2-4C2/inner_link.obj scale=-1 1 1; visual mesh filename=package://inspire_description/meshes/EG2-4C2/inner_link.obj scale=-1 1 1
- link left_right_outer_link: geometry collision mesh filename=package://inspire_description/meshes/EG2-4C2/outer_link.obj scale=-1 1 1; visual mesh filename=package://inspire_description/meshes/EG2-4C2/outer_link.obj scale=-1 1 1
- link left_right_pad: geometry collision mesh filename=package://inspire_description/meshes/EG2-4C2/pad.obj scale=-1 1 1; visual mesh filename=package://inspire_description/meshes/EG2-4C2/pad.obj scale=-1 1 1
- link lidar_link: geometry visual mesh filename=package://sensor_models/meshes/orbbec/ms500.glb
- link right_base_link: geometry collision mesh filename=package://ai2_bot2_description/meshes/Visual/arm/arm_base_l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 scale=1 -1 1; visual mesh filename=package://ai2_bot2_description/meshes/Visual/arm/arm_base_l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 scale=1 -1 1
- link right_gripper_base: geometry collision mesh filename=package://inspire_description/meshes/EG2-4C2/baselink.obj; visual mesh filename=package://inspire_description/meshes/EG2-4C2/baselink.obj
- link right_left_inner_link: geometry collision mesh filename=package://inspire_description/meshes/EG2-4C2/inner_link.obj; visual mesh filename=package://inspire_description/meshes/EG2-4C2/inner_link.obj
- link right_left_outer_link: geometry collision mesh filename=package://inspire_description/meshes/EG2-4C2/outer_link.obj; visual mesh filename=package://inspire_description/meshes/EG2-4C2/outer_link.obj
- link right_left_pad: geometry collision mesh filename=package://inspire_description/meshes/EG2-4C2/pad.obj; visual mesh filename=package://inspire_description/meshes/EG2-4C2/pad.obj
- link right_link1: geometry collision mesh filename=package://ai2_bot2_description/meshes/Visual/arm/link1.glb scale=1 -1 1; visual mesh filename=package://ai2_bot2_description/meshes/Visual/arm/link1.glb scale=1 -1 1
- link right_link2: geometry collision mesh filename=package://ai2_bot2_description/meshes/Visual/arm/link2.glb scale=1 1 -1; visual mesh filename=package://ai2_bot2_description/meshes/Visual/arm/link2.glb scale=1 1 -1
- link right_link3: geometry collision mesh filename=package://ai2_bot2_description/meshes/Visual/arm/link3.glb scale=-1 1 1; visual mesh filename=package://ai2_bot2_description/meshes/Visual/arm/link3.glb scale=-1 1 1
- link right_link4: geometry collision mesh filename=package://ai2_bot2_description/meshes/Visual/arm/link4.glb scale=-1 1 1; visual mesh filename=package://ai2_bot2_description/meshes/Visual/arm/link4.glb scale=-1 1 1
- link right_link5: geometry collision mesh filename=package://ai2_bot2_description/meshes/Visual/arm/link5.glb scale=-1 1 1; visual mesh filename=package://ai2_bot2_description/meshes/Visual/arm/link5.glb scale=-1 1 1
- link right_link6: geometry collision mesh filename=package://ai2_bot2_description/meshes/Visual/arm/link6.glb scale=1 -1 1; visual mesh filename=package://ai2_bot2_description/meshes/Visual/arm/link6.glb scale=1 -1 1
- link right_link7: geometry collision mesh filename=package://ai2_bot2_description/meshes/Visual/arm/link7.glb scale=1 1 -1; visual mesh filename=package://ai2_bot2_description/meshes/Visual/arm/link7.glb scale=1 1 -1
- link right_link8: geometry visual mesh filename=package://rm75_description/meshes/ee/camera_stand_d405.glb; visual mesh filename=package://rm75_description/meshes/ee/ee_fb_camera.glb
- link right_right_inner_link: geometry collision mesh filename=package://inspire_description/meshes/EG2-4C2/inner_link.obj scale=-1 1 1; visual mesh filename=package://inspire_description/meshes/EG2-4C2/inner_link.obj scale=-1 1 1
- link right_right_outer_link: geometry collision mesh filename=package://inspire_description/meshes/EG2-4C2/outer_link.obj scale=-1 1 1; visual mesh filename=package://inspire_description/meshes/EG2-4C2/outer_link.obj scale=-1 1 1
- link right_right_pad: geometry collision mesh filename=package://inspire_description/meshes/EG2-4C2/pad.obj scale=-1 1 1; visual mesh filename=package://inspire_description/meshes/EG2-4C2/pad.obj scale=-1 1 1
