Commit message: remove sensor obj

File: humanoid/Ai2Robotics/ai2_bot2_description/urdf/ai2_bot2.urdf (robot description, URDF)
Before this commit: robot Ai2_Bot2, 46 links, 45 joints
Links:
- link back_camera: geometry visual mesh filename=package://sensor_models/meshes/realsense/d435.glb
- link front_camera: geometry visual mesh filename=package://sensor_models/meshes/realsense/d435.glb
- link head_camera: geometry visual mesh filename=package://sensor_models/meshes/realsense/d435.glb

File: humanoid/Ai2Robotics/ai2_bot2_description/urdf/ai2_bot2_inspire.urdf (robot description, URDF)
Before this commit: robot Ai2_Bot2, 64 links, 63 joints
Links:
- link back_camera: geometry visual mesh filename=package://sensor_models/meshes/realsense/d435.glb
- link front_camera: geometry visual mesh filename=package://sensor_models/meshes/realsense/d435.glb
- link head_camera: geometry visual mesh filename=package://sensor_models/meshes/realsense/d435.glb

File: humanoid/Galaxea/galaxea_r1_description/urdf/galaxea_r1.urdf (robot description, URDF)
Before this commit: robot R1, 36 links, 35 joints
Links:
- link left_realsense_link: geometry collision mesh filename=package://galaxea_r1_description/meshes/camera_stand.obj; visual mesh filename=package://galaxea_r1_description/meshes/camera_stand.obj
- link right_realsense_link: geometry collision mesh filename=package://galaxea_r1_description/meshes/camera_stand.obj; visual mesh filename=package://galaxea_r1_description/meshes/camera_stand.obj

File: humanoid/Galaxea/galaxea_r1_description/xacro/realsense.xacro (robot description, xacro)
@@ -17,7 +17,7 @@
       </visual>
       <visual>
-        <origin rpy="${PI/2} ${-PI/2} 0" xyz="0.0325 0 0"/>
+        <origin xyz="0.0325 0 0"/>
         <geometry>
-          <mesh filename="file://$(find sensor_models)/meshes/d435/d435.obj"/>
+          <mesh filename="file://$(find sensor_models)/meshes/realsense/d435.glb"/>
         </geometry>
       </visual>

File: humanoid/Galaxea/galaxea_r1pro_description/urdf/galaxea_r1pro.urdf (robot description, URDF)
Before this commit: robot R1Pro, 38 links, 37 joints
Links:
- link left_realsense_link: geometry collision mesh filename=package://galaxea_r1_description/meshes/camera_stand.obj; visual mesh filename=package://galaxea_r1_description/meshes/camera_stand.obj
- link right_realsense_link: geometry collision mesh filename=package://galaxea_r1_description/meshes/camera_stand.obj; visual mesh filename=package://galaxea_r1_description/meshes/camera_stand.obj

File: humanoid/Galaxea/galaxea_r1pro_description/xacro/realsense.xacro (robot description, xacro)
@@ -17,7 +17,7 @@
       </visual>
       <visual>
-        <origin rpy="${PI/2} ${-PI/2} 0" xyz="0.0325 0 0"/>
+        <origin xyz="0.0325 0 0"/>
         <geometry>
-          <mesh filename="file://$(find sensor_models)/meshes/d435/d435.obj"/>
+          <mesh filename="file://$(find sensor_models)/meshes/realsense/d435.glb"/>
         </geometry>
       </visual>

File: humanoid/Zerith/zerith_h1_description/xacro/components/body.xacro (robot description, xacro)
@@ -146,5 +146,5 @@
 		<visual>
 			<geometry>
-				<mesh filename="file://$(find sensor_models)/meshes/d435/d435.obj"/>
+				<mesh filename="file://$(find sensor_models)/meshes/realsense/d435.glb"/>
 			</geometry>
 			<origin xyz="0.0325 0 0.005" rpy="1.5707963267949 -1.5707963267949 -0"/>

File: manipulator/AgileX/agilex_aloha_description/urdf/agilex_aloha.urdf (robot description, URDF)
Before this commit: robot AgileX Aloha, 38 links, 37 joints
Links:
- link lidar_link: geometry collision mesh filename=package://sensor_models/meshes/livox/mid360.glb; visual mesh filename=package://sensor_models/meshes/livox/mid360.glb

File: manipulator/AgileX/agilex_aloha_description/urdf/agilex_aloha_v1.urdf (robot description, URDF)
Before this commit: robot AgileX Aloha, 46 links, 45 joints
Links:
- link lidar_link: geometry visual mesh filename=package://sensor_models/meshes/livox/mid360.glb

File: manipulator/AgileX/agilex_aloha_description/urdf/agilex_aloha_v1_x5.urdf (robot description, URDF)
Before this commit: robot AgileX Aloha, 46 links, 45 joints
Links:
- link lidar_link: geometry visual mesh filename=package://sensor_models/meshes/livox/mid360.glb

File: manipulator/AgileX/agilex_aloha_description/urdf/agilex_aloha_v2-1.urdf (robot description, URDF)
Before this commit: robot AgileX Aloha, 33 links, 32 joints
Links:
- link lidar_link: geometry visual mesh filename=package://sensor_models/meshes/livox/mid360.glb

File: manipulator/AgileX/agilex_aloha_description/urdf/agilex_aloha_v2.urdf (robot description, URDF)
Before this commit: robot AgileX Aloha, 38 links, 37 joints
Links:
- link lidar_link: geometry visual mesh filename=package://sensor_models/meshes/livox/mid360.glb

File: manipulator/AgileX/agilex_aloha_description/xacro/body/split.xacro (robot description, xacro)
@@ -65,5 +65,5 @@
 		<visual>
 			<geometry>
-				<mesh filename="file://$(find sensor_models)/meshes/mid360/mid360.obj"/>
+				<mesh filename="file://$(find sensor_models)/meshes/livox/mid360.glb"/>
 			</geometry>
 		</visual>

File: manipulator/AgileX/agilex_aloha_description/xacro/body/v1.xacro (robot description, xacro)
@@ -122,5 +122,5 @@
 		<visual>
 			<geometry>
-				<mesh filename="file://$(find sensor_models)/meshes/mid360/mid360.obj"/>
+				<mesh filename="file://$(find sensor_models)/meshes/livox/mid360.glb"/>
 			</geometry>
 		</visual>

File: manipulator/AgileX/agilex_aloha_description/xacro/body/v2.xacro (robot description, xacro)
@@ -62,5 +62,5 @@
 		<visual>
 			<geometry>
-				<mesh filename="file://$(find sensor_models)/meshes/mid360/mid360.obj"/>
+				<mesh filename="file://$(find sensor_models)/meshes/livox/mid360.glb"/>
 			</geometry>
 		</visual>

File: manipulator/Galaxea/galaxea_r1lite_description/urdf/galaxea_r1lite.urdf (robot description, URDF)
Before this commit: robot A1Lite, 36 links, 35 joints
Links:
- link left_camera_stand: geometry collision mesh filename=package://galaxea_r1lite_description/meshes/collision/camer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; visual mesh filename=package://galaxea_r1lite_description/meshes/visual/camera_s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
- link right_camera_stand: geometry collision mesh filename=package://galaxea_r1lite_description/meshes/collision/camer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; visual mesh filename=package://galaxea_r1lite_description/meshes/visual/camera_s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

File: manipulator/Galaxea/galaxea_r1lite_description/urdf/galaxea_r1lite_y.urdf (robot description, URDF)
Before this commit: robot A1Lite, 36 links, 35 joints
Links:
- link left_camera_stand: geometry collision mesh filename=package://galaxea_r1lite_description/meshes/collision/camer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; visual mesh filename=package://galaxea_r1lite_description/meshes/visual/camera_s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
- link right_camera_stand: geometry collision mesh filename=package://galaxea_r1lite_description/meshes/collision/camer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; visual mesh filename=package://galaxea_r1lite_description/meshes/visual/camera_s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
