Commit message: 更新piper_l配置

File: manipulator/AgileX/piper_l_description/xacro/arm.xacro (robot description, xacro)
@@ -11,10 +11,10 @@
             <visual>
                 <geometry>
-                    <mesh filename="package://piper_l_description/meshes/base_link.glb"/>
-                </geometry>
-            </visual>
-            <collision>
-                <geometry>
-                    <mesh filename="package://piper_l_description/meshes/base_link.glb"/>
+                    <mesh filename="file://$(find piper_l_description)/meshes/base_link.glb"/>
+                </geometry>
+            </visual>
+            <collision>
+                <geometry>
+                    <mesh filename="file://$(find piper_l_description)/meshes/base_link.glb"/>
                 </geometry>
             </collision>
@@ -29,10 +29,10 @@
             <visual>
                 <geometry>
-                    <mesh filename="package://piper_l_description/meshes/link1.glb"/>
-                </geometry>
-            </visual>
-            <collision>
-                <geometry>
-                    <mesh filename="package://piper_l_description/meshes/link1.glb"/>
+                    <mesh filename="file://$(find piper_l_description)/meshes/link1.glb"/>
+                </geometry>
+            </visual>
+            <collision>
+                <geometry>
+                    <mesh filename="file://$(find piper_l_description)/meshes/link1.glb"/>
                 </geometry>
             </collision>
@@ -54,10 +54,10 @@
             <visual>
                 <geometry>
-                    <mesh filename="package://piper_l_description/meshes/link2.glb"/>
-                </geometry>
-            </visual>
-            <collision>
-                <geometry>
-                    <mesh filename="package://piper_l_description/meshes/link2.glb"/>
+                    <mesh filename="file://$(find piper_l_description)/meshes/link2.glb"/>
+                </geometry>
+            </visual>
+            <collision>
+                <geometry>
+                    <mesh filename="file://$(find piper_l_description)/meshes/link2.glb"/>
                 </geometry>
             </collision>
@@ -79,10 +79,10 @@
             <visual>
                 <geometry>
-                    <mesh filename="package://piper_l_description/meshes/link3.glb"/>
-                </geometry>
-            </visual>
-            <collision>
-                <geometry>
-                    <mesh filename="package://piper_l_description/meshes/link3.glb"/>
+                    <mesh filename="file://$(find piper_l_description)/meshes/link3.glb"/>
+                </geometry>
+            </visual>
+            <collision>
+                <geometry>
+                    <mesh filename="file://$(find piper_l_description)/meshes/link3.glb"/>
                 </geometry>
             </collision>
@@ -104,10 +104,10 @@
             <visual>
                 <geometry>
-                    <mesh filename="package://piper_l_description/meshes/link4.glb"/>
-                </geometry>
-            </visual>
-            <collision>
-                <geometry>
-                    <mesh filename="package://piper_l_description/meshes/link4.glb"/>
+                    <mesh filename="file://$(find piper_l_description)/meshes/link4.glb"/>
+                </geometry>
+            </visual>
+            <collision>
+                <geometry>
+                    <mesh filename="file://$(find piper_l_description)/meshes/link4.glb"/>
                 </geometry>
             </collision>
@@ -129,10 +129,10 @@
             <visual>
                 <geometry>
-                    <mesh filename="package://piper_l_description/meshes/link5.glb"/>
-                </geometry>
-            </visual>
-            <collision>
-                <geometry>
-                    <mesh filename="package://piper_l_description/meshes/link5.glb"/>
+                    <mesh filename="file://$(find piper_l_description)/meshes/link5.glb"/>
+                </geometry>
+            </visual>
+            <collision>
+                <geometry>
+                    <mesh filename="file://$(find piper_l_description)/meshes/link5.glb"/>
                 </geometry>
             </collision>
@@ -154,5 +154,5 @@
                 <origin xyz="0.008 -0.002 0.064" rpy="-1.57 0 1.57"/>
                 <geometry>
-                    <mesh filename="package://piper_l_description/meshes/gripper_base_100_v3.glb"/>
+                    <mesh filename="file://$(find piper_l_description)/meshes/gripper_base_100_v3.glb"/>
                 </geometry>
             </visual>
@@ -160,5 +160,5 @@
                 <origin xyz="0.008 -0.002 0.064" rpy="-1.57 0 1.57"/>
                 <geometry>
-                    <mesh filename="package://piper_l_description/meshes/gripper_base_100_v3.glb"/>
+                    <mesh filename="file://$(find piper_l_description)/meshes/gripper_base_100_v3.glb"/>
                 </geometry>
             </collision>
@@ -174,10 +174,10 @@
             <visual>
                 <geometry>
-                    <mesh filename="package://piper_l_description/meshes/link7.glb"/>
-                </geometry>
-            </visual>
-            <collision>
-                <geometry>
-                    <mesh filename="package://piper_l_description/meshes/link7.glb"/>
+                    <mesh filename="file://$(find piper_l_description)/meshes/link7.glb"/>
+                </geometry>
+            </visual>
+            <collision>
+                <geometry>
+                    <mesh filename="file://$(find piper_l_description)/meshes/link7.glb"/>
                 </geometry>
             </collision>
@@ -193,10 +193,10 @@
             <visual>
                 <geometry>
-                    <mesh filename="package://piper_l_description/meshes/link8.glb"/>
-                </geometry>
-            </visual>
-            <collision>
-                <geometry>
-                    <mesh filename="package://piper_l_description/meshes/link8.glb"/>
+                    <mesh filename="file://$(find piper_l_description)/meshes/link8.glb"/>
+                </geometry>
+            </visual>
+            <collision>
+                <geometry>
+                    <mesh filename="file://$(find piper_l_description)/meshes/link8.glb"/>
                 </geometry>
             </collision>
@@ -215,5 +215,5 @@
                     <origin rpy="0 0 0" xyz="0 0 0"/>
                     <geometry>
-                        <mesh filename="package://piper_l_description/meshes/realsense_mid_stand_v2.glb"/>
+                        <mesh filename="file://$(find piper_l_description)/meshes/realsense_mid_stand_v2.glb"/>
                     </geometry>
                 </visual>
@@ -221,5 +221,5 @@
                     <origin rpy="0 0 0" xyz="0 0 0"/>
                     <geometry>
-                        <mesh filename="package://piper_l_description/meshes/realsense_mid_stand_v2.glb"/>
+                        <mesh filename="file://$(find piper_l_description)/meshes/realsense_mid_stand_v2.glb"/>
                     </geometry>
                 </collision>
@@ -233,5 +233,5 @@
                 <visual>
                     <geometry>
-                        <mesh filename="package://sensor_models/meshes/d435/d435.obj"/>
+                        <mesh filename="file://$(find sensor_models)/meshes/d435/d435.obj"/>
                     </geometry>
                 </visual>
