Commit message: 更新piper_x相关配置

File: manipulator/AgileX/piper_x_description/urdf/piper_x.urdf (robot description, URDF)
Before this commit: robot piper_x, 13 links, 12 joints
Links:
- link camera_stand_link: geometry collision mesh filename=package://piper_x_description/meshes/realsense_mid_stand.glb; visual mesh filename=package://piper_x_description/meshes/realsense_mid_stand.glb

File: manipulator/AgileX/piper_x_description/xacro/arm.xacro (robot description, xacro)
@@ -12,5 +12,5 @@
                 <origin xyz="0 0 0" rpy="0 0 0"/>
                 <geometry>
-                    <mesh filename="package://piper_x_description/meshes/base_link.glb"/>
+                    <mesh filename="file://$(find piper_x_description)/meshes/base_link.glb"/>
                 </geometry>
             </visual>
@@ -18,5 +18,5 @@
                 <origin xyz="0 0 0" rpy="0 0 0"/>
                 <geometry>
-                    <mesh filename="package://piper_x_description/meshes/base_link.glb"/>
+                    <mesh filename="file://$(find piper_x_description)/meshes/base_link.glb"/>
                 </geometry>
             </collision>
@@ -31,10 +31,10 @@
             <visual>
                 <geometry>
-                    <mesh filename="package://piper_x_description/meshes/link1.glb"/>
-                </geometry>
-            </visual>
-            <collision>
-                <geometry>
-                    <mesh filename="package://piper_x_description/meshes/link1.glb"/>
+                    <mesh filename="file://$(find piper_x_description)/meshes/link1.glb"/>
+                </geometry>
+            </visual>
+            <collision>
+                <geometry>
+                    <mesh filename="file://$(find piper_x_description)/meshes/link1.glb"/>
                 </geometry>
             </collision>
@@ -56,10 +56,10 @@
             <visual>
                 <geometry>
-                    <mesh filename="package://piper_x_description/meshes/link2.glb"/>
-                </geometry>
-            </visual>
-            <collision>
-                <geometry>
-                    <mesh filename="package://piper_x_description/meshes/link2.glb"/>
+                    <mesh filename="file://$(find piper_x_description)/meshes/link2.glb"/>
+                </geometry>
+            </visual>
+            <collision>
+                <geometry>
+                    <mesh filename="file://$(find piper_x_description)/meshes/link2.glb"/>
                 </geometry>
             </collision>
@@ -81,10 +81,10 @@
             <visual>
                 <geometry>
-                    <mesh filename="package://piper_x_description/meshes/link3.glb"/>
-                </geometry>
-            </visual>
-            <collision>
-                <geometry>
-                    <mesh filename="package://piper_x_description/meshes/link3.glb"/>
+                    <mesh filename="file://$(find piper_x_description)/meshes/link3.glb"/>
+                </geometry>
+            </visual>
+            <collision>
+                <geometry>
+                    <mesh filename="file://$(find piper_x_description)/meshes/link3.glb"/>
                 </geometry>
             </collision>
@@ -106,10 +106,10 @@
             <visual>
                 <geometry>
-                    <mesh filename="package://piper_x_description/meshes/link4.glb"/>
-                </geometry>
-            </visual>
-            <collision>
-                <geometry>
-                    <mesh filename="package://piper_x_description/meshes/link4.glb"/>
+                    <mesh filename="file://$(find piper_x_description)/meshes/link4.glb"/>
+                </geometry>
+            </visual>
+            <collision>
+                <geometry>
+                    <mesh filename="file://$(find piper_x_description)/meshes/link4.glb"/>
                 </geometry>
             </collision>
@@ -131,10 +131,10 @@
             <visual>
                 <geometry>
-                    <mesh filename="package://piper_x_description/meshes/link5.glb"/>
-                </geometry>
-            </visual>
-            <collision>
-                <geometry>
-                    <mesh filename="package://piper_x_description/meshes/link5.glb"/>
+                    <mesh filename="file://$(find piper_x_description)/meshes/link5.glb"/>
+                </geometry>
+            </visual>
+            <collision>
+                <geometry>
+                    <mesh filename="file://$(find piper_x_description)/meshes/link5.glb"/>
                 </geometry>
             </collision>
@@ -156,5 +156,5 @@
                 <origin xyz="0 0 -0.035" rpy="0 0 0"/>
                 <geometry>
-                    <mesh filename="package://piper_x_description/meshes/link6.glb"/>
+                    <mesh filename="file://$(find piper_x_description)/meshes/link6.glb"/>
                 </geometry>
             </visual>
@@ -162,5 +162,5 @@
                 <origin xyz="0 0 -0.035" rpy="0 0 0"/>
                 <geometry>
-                    <mesh filename="package://piper_x_description/meshes/link6.glb"/>
+                    <mesh filename="file://$(find piper_x_description)/meshes/link6.glb"/>
                 </geometry>
             </collision>
@@ -183,5 +183,6 @@
                 <origin xyz="0.002 0.0078 0.06" rpy="-1.57 0 3.14"/>
                 <geometry>
-                    <mesh filename="package://piper_x_description/meshes/gripper_base_100_v2.glb" scale="0.8 0.8 0.8"/>
+                    <mesh filename="file://$(find piper_x_description)/meshes/gripper_base_100_v2.glb"
+                          scale="0.8 0.8 0.8"/>
                 </geometry>
             </visual>
@@ -189,5 +190,6 @@
                 <origin xyz="0.002 0.0078 0.06" rpy="-1.57 0 3.14"/>
                 <geometry>
-                    <mesh filename="package://piper_x_description/meshes/gripper_base_100_v2.glb" scale="0.8 0.8 0.8"/>
+                    <mesh filename="file://$(find piper_x_description)/meshes/gripper_base_100_v2.glb"
+                          scale="0.8 0.8 0.8"/>
                 </geometry>
             </collision>
@@ -207,10 +209,10 @@
             <visual>
                 <geometry>
-                    <mesh filename="package://piper_x_description/meshes/link7.glb"/>
-                </geometry>
-            </visual>
-            <collision>
-                <geometry>
-                    <mesh filename="package://piper_x_description/meshes/link7.glb"/>
+                    <mesh filename="file://$(find piper_x_description)/meshes/link7.glb"/>
+                </geometry>
+            </visual>
+            <collision>
+                <geometry>
+                    <mesh filename="file://$(find piper_x_description)/meshes/link7.glb"/>
                 </geometry>
             </collision>
@@ -232,10 +234,10 @@
             <visual>
                 <geometry>
-                    <mesh filename="package://piper_x_description/meshes/link8.glb"/>
-                </geometry>
-            </visual>
-            <collision>
-                <geometry>
-                    <mesh filename="package://piper_x_description/meshes/link8.glb"/>
+                    <mesh filename="file://$(find piper_x_description)/meshes/link8.glb"/>
+                </geometry>
+            </visual>
+            <collision>
+                <geometry>
+                    <mesh filename="file://$(find piper_x_description)/meshes/link8.glb"/>
                 </geometry>
             </collision>

File: manipulator/AgileX/piper_x_description/xacro/ros2_control/piper_x.ros2_control.xacro (robot description, xacro)
@@ -61,12 +61,4 @@
                 <state_interface name="position"/>
                 <state_interface name="velocity"/>
-                <state_interface name="effort"/>
-            </joint>
-            <joint name="${prefix}joint8">
-                <param name="mimic">${prefix}joint7</param>
-                <param name="multiplier">-1.0</param>
-                <state_interface name="position"/>
-                <state_interface name="velocity"/>
-                <state_interface name="effort"/>
             </joint>
         </ros2_control>
