Commit message: 更新piper_l运控配置

File: manipulator/AgileX/piper_l_description/xacro/ros2_control/piper_l.ros2_control.xacro (robot description, xacro)
@@ -10,4 +10,9 @@
                 <xacro:if value="${ros2_control_hardware_type == 'mock_components'}">
                     <plugin>mock_components/GenericSystem</plugin>
+                </xacro:if>
+                <xacro:if value="${ros2_control_hardware_type == 'isaac'}">
+                    <plugin>topic_based_ros2_control/TopicBasedSystem</plugin>
+                    <param name="joint_commands_topic">/isaac/joint_command</param>
+                    <param name="joint_states_topic">/isaac/joint_states</param>
                 </xacro:if>
             </hardware>
@@ -49,9 +54,5 @@
                 <command_interface name="position"/>
                 <state_interface name="position"/>
-            </joint>
-            <joint name="${prefix}joint8">
-                <param name="mimic">${prefix}joint7</param>
-                <param name="multiplier">-1.0</param>
-                <state_interface name="position"/>
+                <state_interface name="velocity"/>
             </joint>
         </ros2_control>
