Commit message: add home_2

File: humanoid/Ai2Robotics/ai2_bot2_description/xacro/components/arm.xacro (robot description, xacro)
@@ -344,5 +344,5 @@
                 <origin xyz="-0.13322 -0.0005 0.044651" rpy="0 -1.5708 -1.5708"/>
                 <geometry>
-                    <mesh filename="file://$(find sensor_models)/meshes/d405.glb"/>
+                    <mesh filename="file://$(find sensor_models)/meshes/d405/d405.obj"/>
                 </geometry>
             </visual>

File: humanoid/Ai2Robotics/ai2_bot2_description/xacro/components/chassis.xacro (robot description, xacro)
@@ -212,9 +212,9 @@
 		</joint>
 		<link name="chassis_panel">
-			<!--      <visual>-->
-			<!--        <geometry>-->
-			<!--          <mesh filename="file://$(find aidal_description)/meshes/woosh_agv/panel.glb"/>-->
-			<!--        </geometry>-->
-			<!--      </visual>-->
+			<visual>
+				<geometry>
+					<mesh filename="file://$(find aidal_description)/meshes/woosh_agv/panel.glb"/>
+				</geometry>
+			</visual>
 		</link>
 		<joint name="chassis_panel_joint" type="fixed">
@@ -224,9 +224,9 @@
 		</joint>
 		<link name="charge_port">
-			<!--      <visual>-->
-			<!--        <geometry>-->
-			<!--          <mesh filename="file://$(find ai2_bot2_description)/meshes/Visual/chassis/charge_port.glb"/>-->
-			<!--        </geometry>-->
-			<!--      </visual>-->
+			<visual>
+				<geometry>
+					<mesh filename="file://$(find ai2_bot2_description)/meshes/Visual/chassis/charge_port.glb"/>
+				</geometry>
+			</visual>
 		</link>
 		<joint name="charge_port" type="fixed">
@@ -236,9 +236,9 @@
 		</joint>
 		<link name="lidar_link">
-			<!--      <visual>-->
-			<!--        <geometry>-->
-			<!--          <mesh filename="file://$(find sensor_models)/meshes/orbbec/ms500.glb"/>-->
-			<!--        </geometry>-->
-			<!--      </visual>-->
+			<visual>
+				<geometry>
+					<mesh filename="file://$(find sensor_models)/meshes/orbbec/ms500.glb"/>
+				</geometry>
+			</visual>
 		</link>
 		<joint name="lidar_joint" type="fixed">
@@ -247,4 +247,16 @@
 			<child link="lidar_link"/>
 		</joint>
+		<link name="chassis_camera">
+			<visual>
+				<geometry>
+					<mesh filename="file://$(find sensor_models)/meshes/orbbec/Dabai_DW.glb"/>
+				</geometry>
+			</visual>
+		</link>
+		<joint name="chassis_camera" type="fixed">
+			<origin xyz="0.315 0 0.104" rpy="1.5708 0 1.5708"/>
+			<parent link="base_link"/>
+			<child link="chassis_camera"/>
+		</joint>
 	</xacro:macro>
 </robot>
