Commit message: add 2d lidar navigation

File: humanoid/Ai2Robotics/ai2_bot2_description/xacro/components/chassis.xacro (robot description, xacro)
@@ -247,4 +247,10 @@
 			<child link="lidar_link"/>
 		</joint>
+		<link name="lidar_frame"/>
+		<joint name="lidar_frame_joint" type="fixed">
+			<origin xyz="0 0 0.06"/>
+			<parent link="lidar_link"/>
+			<child link="lidar_frame"/>
+		</joint>
 		<link name="chassis_camera">
 			<visual>
