Commit message: Add ocs2 demo for ai2_bot2

File: humanoid/Ai2Robotics/ai2_bot2_description/xacro/components/body.xacro (robot description, xacro)
@@ -134,6 +134,6 @@
       <limit lower="-1.5708" upper="1.5708" effort="1000" velocity="10" />
     </joint>
-    <!-- head: head_link_1 (neck), head_joint_1, head_link_2 (head), head_joint_2 -->
-    <link name="head_link_1">
+    <!-- head: head_link1 (neck), head_joint1, head_link2 (head), head_joint2 -->
+    <link name="head_link1">
       <inertial>
         <origin xyz="-1.4269E-12 0.0053202 0.055582" />
@@ -148,12 +148,12 @@
       </inertial>
     </link>
-    <joint name="head_joint_1" type="revolute">
+    <joint name="head_joint1" type="revolute">
       <origin xyz="-0.041 0 0.46874" />
       <parent link="body_link4" />
-      <child link="head_link_1" />
+      <child link="head_link1" />
       <axis xyz="0 0 1" />
       <limit lower="-1.5708" upper="1.5708" effort="1000" velocity="10" />
     </joint>
-    <link name="head_link_2">
+    <link name="head_link2">
       <inertial>
         <origin xyz="0.028328 -0.035178 -0.00055178" />
@@ -181,8 +181,8 @@
       </collision>
     </link>
-    <joint name="head_joint_2" type="revolute">
+    <joint name="head_joint2" type="revolute">
       <origin xyz="0 0 0.06" rpy="-1.5708 0 0" />
-      <parent link="head_link_1" />
-      <child link="head_link_2" />
+      <parent link="head_link1" />
+      <child link="head_link2" />
       <axis xyz="0 0 1" />
       <limit lower="-0.4014" upper="0.38397" effort="1000" velocity="10" />

File: humanoid/Ai2Robotics/ai2_bot2_description/xacro/components/chassis.xacro (robot description, xacro)
@@ -38,10 +38,10 @@
       <visual>
         <geometry>
-          <mesh filename="file://$(find ai2_bot2_description)/meshes/Collision/driven_wheel_left_front_link_v.STL"/>
+          <mesh filename="file://$(find ai2_bot2_description)/meshes/Visual/chassis/driven_v.glb"/>
         </geometry>
       </visual>
       <collision>
         <geometry>
-          <mesh filename="file://$(find ai2_bot2_description)/meshes/Collision/driven_wheel_left_front_link_v.STL"/>
+          <mesh filename="file://$(find ai2_bot2_description)/meshes/Visual/chassis/driven_v.glb"/>
         </geometry>
       </collision>
@@ -57,10 +57,10 @@
       <visual>
         <geometry>
-          <mesh filename="file://$(find ai2_bot2_description)/meshes/Collision/driven_wheel_left_front_link_h.STL"/>
+          <mesh filename="file://$(find ai2_bot2_description)/meshes/Visual/chassis/driven_h.glb"/>
         </geometry>
       </visual>
       <collision>
         <geometry>
-          <mesh filename="file://$(find ai2_bot2_description)/meshes/Collision/driven_wheel_left_front_link_h.STL"/>
+          <mesh filename="file://$(find ai2_bot2_description)/meshes/Visual/chassis/driven_h.glb"/>
         </geometry>
       </collision>
@@ -74,6 +74,6 @@
     </joint>
     <link name="driven_rl_link_v">
-      <visual><geometry><mesh filename="file://$(find ai2_bot2_description)/meshes/Collision/driven_wheel_left_front_link_v.STL"/></geometry></visual>
-      <collision><geometry><mesh filename="file://$(find ai2_bot2_description)/meshes/Collision/driven_wheel_left_front_link_v.STL"/></geometry></collision>
+      <visual><geometry><mesh filename="file://$(find ai2_bot2_description)/meshes/Visual/chassis/driven_v.glb"/></geometry></visual>
+      <collision><geometry><mesh filename="file://$(find ai2_bot2_description)/meshes/Visual/chassis/driven_v.glb"/></geometry></collision>
     </link>
     <joint name="driven_rl_joint_v" type="${wheel_joint_type}">
@@ -85,6 +85,6 @@
     </joint>
     <link name="driven_rl_link_h">
-      <visual><geometry><mesh filename="file://$(find ai2_bot2_description)/meshes/Collision/driven_wheel_left_front_link_h.STL"/></geometry></visual>
-      <collision><geometry><mesh filename="file://$(find ai2_bot2_description)/meshes/Collision/driven_wheel_left_front_link_h.STL"/></geometry></collision>
+      <visual><geometry><mesh filename="file://$(find ai2_bot2_description)/meshes/Visual/chassis/driven_h.glb"/></geometry></visual>
+      <collision><geometry><mesh filename="file://$(find ai2_bot2_description)/meshes/Visual/chassis/driven_h.glb"/></geometry></collision>
     </link>
     <joint name="driven_rl_joint_h" type="${wheel_joint_type}">
@@ -96,6 +96,6 @@
     </joint>
     <link name="driven_fr_link_v">
-      <visual><geometry><mesh filename="file://$(find ai2_bot2_description)/meshes/Collision/driven_wheel_left_front_link_v.STL"/></geometry></visual>
-      <collision><geometry><mesh filename="file://$(find ai2_bot2_description)/meshes/Collision/driven_wheel_left_front_link_v.STL"/></geometry></collision>
+      <visual><geometry><mesh filename="file://$(find ai2_bot2_description)/meshes/Visual/chassis/driven_v.glb"/></geometry></visual>
+      <collision><geometry><mesh filename="file://$(find ai2_bot2_description)/meshes/Visual/chassis/driven_v.glb"/></geometry></collision>
     </link>
     <joint name="driven_fr_joint_v" type="${wheel_joint_type}">
@@ -107,6 +107,6 @@
     </joint>
     <link name="driven_fr_link_h">
-      <visual><geometry><mesh filename="file://$(find ai2_bot2_description)/meshes/Collision/driven_wheel_left_front_link_h.STL"/></geometry></visual>
-      <collision><geometry><mesh filename="file://$(find ai2_bot2_description)/meshes/Collision/driven_wheel_left_front_link_h.STL"/></geometry></collision>
+      <visual><geometry><mesh filename="file://$(find ai2_bot2_description)/meshes/Visual/chassis/driven_h.glb"/></geometry></visual>
+      <collision><geometry><mesh filename="file://$(find ai2_bot2_description)/meshes/Visual/chassis/driven_h.glb"/></geometry></collision>
     </link>
     <joint name="driven_fr_joint_h" type="${wheel_joint_type}">
@@ -118,6 +118,6 @@
     </joint>
     <link name="driven_rr_link_v">
-      <visual><geometry><mesh filename="file://$(find ai2_bot2_description)/meshes/Collision/driven_wheel_left_front_link_v.STL"/></geometry></visual>
-      <collision><geometry><mesh filename="file://$(find ai2_bot2_description)/meshes/Collision/driven_wheel_left_front_link_v.STL"/></geometry></collision>
+      <visual><geometry><mesh filename="file://$(find ai2_bot2_description)/meshes/Visual/chassis/driven_v.glb"/></geometry></visual>
+      <collision><geometry><mesh filename="file://$(find ai2_bot2_description)/meshes/Visual/chassis/driven_v.glb"/></geometry></collision>
     </link>
     <joint name="driven_rr_joint_v" type="${wheel_joint_type}">
@@ -129,6 +129,6 @@
     </joint>
     <link name="driven_rr_link_h">
-      <visual><geometry><mesh filename="file://$(find ai2_bot2_description)/meshes/Collision/driven_wheel_left_front_link_h.STL"/></geometry></visual>
-      <collision><geometry><mesh filename="file://$(find ai2_bot2_description)/meshes/Collision/driven_wheel_left_front_link_h.STL"/></geometry></collision>
+      <visual><geometry><mesh filename="file://$(find ai2_bot2_description)/meshes/Visual/chassis/driven_h.glb"/></geometry></visual>
+      <collision><geometry><mesh filename="file://$(find ai2_bot2_description)/meshes/Visual/chassis/driven_h.glb"/></geometry></collision>
     </link>
     <joint name="driven_rr_joint_h" type="${wheel_joint_type}">
@@ -142,10 +142,10 @@
       <visual>
         <geometry>
-          <mesh filename="file://$(find ai2_bot2_description)/meshes/Collision/driving_wheel_left_link.STL"/>
+          <mesh filename="file://$(find ai2_bot2_description)/meshes/Visual/chassis/driving.glb" scale="1 1 1"/>
         </geometry>
       </visual>
       <collision>
         <geometry>
-          <mesh filename="file://$(find ai2_bot2_description)/meshes/Collision/driving_wheel_left_link.STL"/>
+          <mesh filename="file://$(find ai2_bot2_description)/meshes/Visual/chassis/driving.glb" scale="1 1 1"/>
         </geometry>
       </collision>
@@ -159,6 +159,16 @@
     </joint>
     <link name="driving_right_link">
-      <visual><geometry><mesh filename="file://$(find ai2_bot2_description)/meshes/Collision/driving_wheel_left_link.STL"/></geometry></visual>
-      <collision><geometry><mesh filename="file://$(find ai2_bot2_description)/meshes/Collision/driving_wheel_left_link.STL"/></geometry></collision>
+      <visual>
+        <geometry>
+          <mesh filename="file://$(find ai2_bot2_description)/meshes/Visual/chassis/driving.glb"
+                scale="1 1 -1"/>
+        </geometry>
+      </visual>
+      <collision>
+        <geometry>
+          <mesh filename="file://$(find ai2_bot2_description)/meshes/Visual/chassis/driving.glb"
+                scale="1 1 -1"/>
+        </geometry>
+      </collision>
     </link>
     <joint name="driving_right_joint" type="${wheel_joint_type}">

File: humanoid/Ai2Robotics/ai2_bot2_description/xacro/robot.xacro (robot description, xacro)
@@ -6,5 +6,5 @@
 <!-- |    body_link4; ego and arms both attach to body_link4.                           | -->
 <!-- =================================================================================== -->
-<robot name="ai2_bot2" xmlns:xacro="http://www.ros.org/wiki/xacro">
+<robot name="Ai2_Bot2" xmlns:xacro="http://www.ros.org/wiki/xacro">
   <!-- Parse end-effector type from 'type' arg (similar to FiveAges W2 robot.xacro) -->
   <xacro:arg name="type" default=""/>

Commit message: fix robot mesh

File: humanoid/Ai2Robotics/ai2_bot2_description/xacro/components/body.xacro (robot description, xacro)
@@ -134,10 +134,10 @@
       <visual>
         <geometry>
-          <mesh filename="file://$(find sensor_models)/meshes/d435/d435.obj"/>
+          <mesh filename="file://$(find sensor_models)/meshes/realsense/d435.glb"/>
         </geometry>
       </visual>
     </link>
     <joint name="front_camera" type="fixed">
-      <origin xyz="0.1067 0 0.1805" rpy="0 0.38397 0"/>
+      <origin xyz="0.1067 0 0.1805" rpy="-1.95477 0 -1.5708"/>
       <parent link="body_link4"/>
       <child link="front_camera"/>
@@ -146,10 +146,10 @@
       <visual>
         <geometry>
-          <mesh filename="file://$(find sensor_models)/meshes/d435/d435.obj"/>
+          <mesh filename="file://$(find sensor_models)/meshes/realsense/d435.glb"/>
         </geometry>
       </visual>
     </link>
     <joint name="back_camera" type="fixed">
-      <origin xyz="-0.1682 0 0.308" rpy="0 0.4887 3.14159"/>
+      <origin xyz="-0.1682 0 0.308" rpy="-2.0595 0 1.5708"/>
       <parent link="body_link4"/>
       <child link="back_camera"/>
@@ -209,10 +209,10 @@
       <visual>
         <geometry>
-          <mesh filename="file://$(find sensor_models)/meshes/d435/d435.obj"/>
+          <mesh filename="file://$(find sensor_models)/meshes/realsense/d435.glb"/>
         </geometry>
       </visual>
     </link>
     <joint name="head_camera" type="fixed">
-      <origin xyz="0.089 0.0465 0" rpy="1.5708 0 0.5236"/>
+      <origin xyz="0.089 0.0465 0" rpy="0 1.5708 0.5236"/>
       <parent link="head_link2"/>
       <child link="head_camera"/>
