Commit message: Optimize ai2 bot2 chassis model

File: humanoid/Ai2Robotics/ai2_bot2_description/xacro/component.xacro (robot description, xacro)
@@ -9,11 +9,11 @@
     - left_arm / right_arm: root = base_link, both arms only, no body/chassis/ego
 -->
-<robot name="ai2_bot2_component" xmlns:xacro="http://www.ros.org/wiki/xacro">
+<robot name="Ai2_Bot2_Chassis" xmlns:xacro="http://www.ros.org/wiki/xacro">
   <!-- component.launch.py default should show the base -->
   <xacro:arg name="type" default="base"/>
   <!-- Lock chassis joints by default for visualization (like W2) -->
   <xacro:arg name="chassis_joints_movable" default="false"/>
-  <!-- Root link: type=base uses chassis (base_link); otherwise provide a stable base_link for RViz -->
-  <xacro:if value="${'$(arg type)' != 'base'}">
+  <!-- Root link: type=base and type=chassis get base_link from chassis; others need a placeholder for RViz -->
+  <xacro:if value="${'$(arg type)' != 'base' and '$(arg type)' != 'chassis'}">
     <link name="base_link"/>
   </xacro:if>
@@ -39,9 +39,9 @@
     <joint name="ego_joint" type="fixed">
       <origin xyz="-0.061 0 0.3255" rpy="0 0 0" />
-      <parent link="body_link_4" />
+      <parent link="body_link4" />
       <child link="ego" />
     </joint>
-    <xacro:Ai2Bot2Arm name="left" parent_link="body_link_4" direction="1"/>
-    <xacro:Ai2Bot2Arm name="right" parent_link="body_link_4" direction="-1"/>
+    <xacro:Ai2Bot2Arm name="left" parent_link="body_link4" direction="1"/>
+    <xacro:Ai2Bot2Arm name="right" parent_link="body_link4" direction="-1"/>
   </xacro:if>
   <xacro:if value="${'$(arg type)' == 'left_arm'}">
@@ -53,3 +53,7 @@
     <xacro:Ai2Bot2Arm name="right" parent_link="base_link" direction="-1"/>
   </xacro:if>
+  <xacro:if value="${'$(arg type)' == 'chassis'}">
+    <xacro:include filename="$(find ai2_bot2_description)/xacro/components/chassis.xacro"/>
+    <xacro:Ai2Bot2Chassis joints_movable="true"/>
+  </xacro:if>
 </robot>

File: humanoid/Ai2Robotics/ai2_bot2_description/xacro/components/chassis.xacro (robot description, xacro)
@@ -41,9 +41,4 @@
         </geometry>
       </visual>
-      <collision>
-        <geometry>
-          <mesh filename="file://$(find ai2_bot2_description)/meshes/Visual/chassis/driven_v.glb"/>
-        </geometry>
-      </collision>
     </link>
     <joint name="driven_fl_joint_v" type="${wheel_joint_type}">
@@ -62,5 +57,5 @@
       <collision>
         <geometry>
-          <mesh filename="file://$(find ai2_bot2_description)/meshes/Visual/chassis/driven_h.glb"/>
+          <sphere radius="0.0375"/>
         </geometry>
       </collision>
@@ -74,6 +69,9 @@
     </joint>
     <link name="driven_rl_link_v">
-      <visual><geometry><mesh filename="file://$(find ai2_bot2_description)/meshes/Visual/chassis/driven_v.glb"/></geometry></visual>
-      <collision><geometry><mesh filename="file://$(find ai2_bot2_description)/meshes/Visual/chassis/driven_v.glb"/></geometry></collision>
+      <visual>
+        <geometry>
+          <mesh filename="file://$(find ai2_bot2_description)/meshes/Visual/chassis/driven_v.glb"/>
+        </geometry>
+      </visual>
     </link>
     <joint name="driven_rl_joint_v" type="${wheel_joint_type}">
@@ -85,6 +83,14 @@
     </joint>
     <link name="driven_rl_link_h">
-      <visual><geometry><mesh filename="file://$(find ai2_bot2_description)/meshes/Visual/chassis/driven_h.glb"/></geometry></visual>
-      <collision><geometry><mesh filename="file://$(find ai2_bot2_description)/meshes/Visual/chassis/driven_h.glb"/></geometry></collision>
+      <visual>
+        <geometry>
+          <mesh filename="file://$(find ai2_bot2_description)/meshes/Visual/chassis/driven_h.glb"/>
+        </geometry>
+      </visual>
+      <collision>
+        <geometry>
+          <sphere radius="0.0375"/>
+        </geometry>
+      </collision>
     </link>
     <joint name="driven_rl_joint_h" type="${wheel_joint_type}">
@@ -96,6 +102,9 @@
     </joint>
     <link name="driven_fr_link_v">
-      <visual><geometry><mesh filename="file://$(find ai2_bot2_description)/meshes/Visual/chassis/driven_v.glb"/></geometry></visual>
-      <collision><geometry><mesh filename="file://$(find ai2_bot2_description)/meshes/Visual/chassis/driven_v.glb"/></geometry></collision>
+      <visual>
+        <geometry>
+          <mesh filename="file://$(find ai2_bot2_description)/meshes/Visual/chassis/driven_v.glb"/>
+        </geometry>
+      </visual>
     </link>
     <joint name="driven_fr_joint_v" type="${wheel_joint_type}">
@@ -107,6 +116,14 @@
     </joint>
     <link name="driven_fr_link_h">
-      <visual><geometry><mesh filename="file://$(find ai2_bot2_description)/meshes/Visual/chassis/driven_h.glb"/></geometry></visual>
-      <collision><geometry><mesh filename="file://$(find ai2_bot2_description)/meshes/Visual/chassis/driven_h.glb"/></geometry></collision>
+      <visual>
+        <geometry>
+          <mesh filename="file://$(find ai2_bot2_description)/meshes/Visual/chassis/driven_h.glb"/>
+        </geometry>
+      </visual>
+      <collision>
+        <geometry>
+          <sphere radius="0.0375"/>
+        </geometry>
+      </collision>
     </link>
     <joint name="driven_fr_joint_h" type="${wheel_joint_type}">
@@ -118,6 +135,9 @@
     </joint>
     <link name="driven_rr_link_v">
-      <visual><geometry><mesh filename="file://$(find ai2_bot2_description)/meshes/Visual/chassis/driven_v.glb"/></geometry></visual>
-      <collision><geometry><mesh filename="file://$(find ai2_bot2_description)/meshes/Visual/chassis/driven_v.glb"/></geometry></collision>
+      <visual>
+        <geometry>
+          <mesh filename="file://$(find ai2_bot2_description)/meshes/Visual/chassis/driven_v.glb"/>
+        </geometry>
+      </visual>
     </link>
     <joint name="driven_rr_joint_v" type="${wheel_joint_type}">
@@ -129,6 +149,14 @@
     </joint>
     <link name="driven_rr_link_h">
-      <visual><geometry><mesh filename="file://$(find ai2_bot2_description)/meshes/Visual/chassis/driven_h.glb"/></geometry></visual>
-      <collision><geometry><mesh filename="file://$(find ai2_bot2_description)/meshes/Visual/chassis/driven_h.glb"/></geometry></collision>
+      <visual>
+        <geometry>
+          <mesh filename="file://$(find ai2_bot2_description)/meshes/Visual/chassis/driven_h.glb"/>
+        </geometry>
+      </visual>
+      <collision>
+        <geometry>
+          <sphere radius="0.0375"/>
+        </geometry>
+      </collision>
     </link>
     <joint name="driven_rr_joint_h" type="${wheel_joint_type}">
@@ -142,18 +170,19 @@
       <visual>
         <geometry>
-          <mesh filename="file://$(find ai2_bot2_description)/meshes/Visual/chassis/driving.glb" scale="1 1 1"/>
-        </geometry>
-      </visual>
-      <collision>
-        <geometry>
-          <mesh filename="file://$(find ai2_bot2_description)/meshes/Visual/chassis/driving.glb" scale="1 1 1"/>
+          <mesh filename="file://$(find aidal_description)/meshes/woosh_agv/wheel.glb" scale="1 1 1"/>
+        </geometry>
+      </visual>
+      <collision>
+        <origin rpy="0 1.5708 0"/>
+        <geometry>
+          <cylinder radius="0.085" length="0.034"/>
         </geometry>
       </collision>
     </link>
     <joint name="driving_left_joint" type="${wheel_joint_type}">
-      <origin xyz="0 0.208 0.0845" rpy="-1.5708 0 0" />
+      <origin xyz="0 0.208 0.0845" rpy="0 0 -1.5708" />
       <parent link="base_link" />
       <child link="driving_left_link" />
-      <axis xyz="0 0 1" />
+      <axis xyz="1 0 0" />
       <limit effort="2000" velocity="10" />
     </joint>
@@ -161,21 +190,57 @@
       <visual>
         <geometry>
-          <mesh filename="file://$(find ai2_bot2_description)/meshes/Visual/chassis/driving.glb"
+          <mesh filename="file://$(find aidal_description)/meshes/woosh_agv/wheel.glb"
                 scale="1 1 -1"/>
         </geometry>
       </visual>
       <collision>
-        <geometry>
-          <mesh filename="file://$(find ai2_bot2_description)/meshes/Visual/chassis/driving.glb"
-                scale="1 1 -1"/>
+        <origin rpy="0 1.5708 0"/>
+        <geometry>
+          <cylinder radius="0.085" length="0.034"/>
         </geometry>
       </collision>
     </link>
     <joint name="driving_right_joint" type="${wheel_joint_type}">
-      <origin xyz="0 -0.208 0.0845" rpy="-1.5708 0 0" />
+      <origin xyz="0 -0.208 0.0845" rpy="0 0 -1.5708" />
       <parent link="base_link" />
       <child link="driving_right_link" />
-      <axis xyz="0 0 1" />
-      <limit effort="2000" velocity="10" />
+      <axis xyz="1 0 0" />
+      <limit effort="2000" velocity="10" />
+    </joint>
+    <link name="chassis_panel">
+      <visual>
+        <geometry>
+          <mesh filename="file://$(find aidal_description)/meshes/woosh_agv/panel.glb"/>
+        </geometry>
+      </visual>
+    </link>
+    <joint name="chassis_panel_joint" type="fixed">
+      <origin xyz="-0.0524 0.1771 0.2463" rpy="1.5708 -1.5708 0"/>
+      <parent link="base_link"/>
+      <child link="chassis_panel"/>
+    </joint>
+    <link name="charge_port">
+      <visual>
+        <geometry>
+          <mesh filename="file://$(find ai2_bot2_description)/meshes/Visual/chassis/charge_port.glb"/>
+        </geometry>
+      </visual>
+    </link>
+    <joint name="charge_port" type="fixed">
+<!--      <origin xyz="-0.0524 0.1771 0.2463"/>-->
+      <parent link="base_link"/>
+      <child link="charge_port"/>
+    </joint>
+    <link name="lidar_link">
+      		<visual>
+      			<geometry>
+      				<mesh filename="file://$(find sensor_models)/meshes/orbbec/ms500.glb"/>
+      			</geometry>
+      		</visual>
+    </link>
+    <joint name="lidar_joint" type="fixed">
+      <origin xyz="0.260985 0 0.126476"/>
+      <parent link="base_link"/>
+      <child link="lidar_link"/>
     </joint>
   </xacro:macro>

Commit message: modify ai2 bot2 xacro

File: humanoid/Ai2Robotics/ai2_bot2_description/xacro/component.xacro (robot description, xacro)
@@ -9,5 +9,5 @@
     - left_arm / right_arm: root = base_link, both arms only, no body/chassis/ego
 -->
-<robot name="Ai2_Bot2_Chassis" xmlns:xacro="http://www.ros.org/wiki/xacro">
+<robot name="Ai2_Bot2_Arm" xmlns:xacro="http://www.ros.org/wiki/xacro">
   <!-- component.launch.py default should show the base -->
   <xacro:arg name="type" default="base"/>
@@ -57,3 +57,7 @@
     <xacro:Ai2Bot2Chassis joints_movable="true"/>
   </xacro:if>
+  <xacro:if value="${'$(arg type)' == 'body'}">
+    <xacro:include filename="$(find ai2_bot2_description)/xacro/components/body.xacro"/>
+    <xacro:Ai2Bot2Body parent_link="base_link"/>
+  </xacro:if>
 </robot>

File: humanoid/Ai2Robotics/ai2_bot2_description/xacro/components/arm.xacro (robot description, xacro)
@@ -22,19 +22,19 @@
                          iyy="1.7511135e-03" iyz="-1.7950155e-05" izz="1.1806738e-03"/>
             </inertial>
-            <visual>
-                <geometry>
-                    <mesh filename="file://$(find ai2_bot2_description)/meshes/Visual/arm/arm_base_link.glb"
-                          scale="1 ${direction} 1"/>
-                </geometry>
-                <material name="">
-                    <color rgba="0.86667 0.86667 0.8902 1"/>
-                </material>
-            </visual>
-            <collision>
-                <geometry>
-                    <mesh filename="file://$(find ai2_bot2_description)/meshes/Visual/arm/arm_base_link.glb"
-                          scale="1 ${direction} 1"/>
-                </geometry>
-            </collision>
+<!--            <visual>-->
+<!--                <geometry>-->
+<!--                    <mesh filename="file://$(find ai2_bot2_description)/meshes/Visual/arm/arm_base_link.glb"-->
+<!--                          scale="1 ${direction} 1"/>-->
+<!--                </geometry>-->
+<!--                <material name="">-->
+<!--                    <color rgba="0.86667 0.86667 0.8902 1"/>-->
+<!--                </material>-->
+<!--            </visual>-->
+<!--            <collision>-->
+<!--                <geometry>-->
+<!--                    <mesh filename="file://$(find ai2_bot2_description)/meshes/Visual/arm/arm_base_link.glb"-->
+<!--                          scale="1 ${direction} 1"/>-->
+<!--                </geometry>-->
+<!--            </collision>-->
         </link>
         <joint name="${prefix}joint0" type="fixed">

File: humanoid/Ai2Robotics/ai2_bot2_description/xacro/components/chassis.xacro (robot description, xacro)
@@ -13,4 +13,10 @@
       <xacro:property name="wheel_joint_type" value="fixed"/>
     </xacro:unless>
+    <link name="base_footprint"/>
+    <joint name="base_footprint_joint" type="fixed">
+      <origin xyz="0 0 0" rpy="0 0 0"/>
+      <parent link="base_footprint"/>
+      <child link="base_link"/>
+    </joint>
     <link name="base_link">
       <inertial>
@@ -209,9 +215,9 @@
     </joint>
     <link name="chassis_panel">
-      <visual>
-        <geometry>
-          <mesh filename="file://$(find aidal_description)/meshes/woosh_agv/panel.glb"/>
-        </geometry>
-      </visual>
+<!--      <visual>-->
+<!--        <geometry>-->
+<!--          <mesh filename="file://$(find aidal_description)/meshes/woosh_agv/panel.glb"/>-->
+<!--        </geometry>-->
+<!--      </visual>-->
     </link>
     <joint name="chassis_panel_joint" type="fixed">
@@ -221,24 +227,24 @@
     </joint>
     <link name="charge_port">
-      <visual>
-        <geometry>
-          <mesh filename="file://$(find ai2_bot2_description)/meshes/Visual/chassis/charge_port.glb"/>
-        </geometry>
-      </visual>
+<!--      <visual>-->
+<!--        <geometry>-->
+<!--          <mesh filename="file://$(find ai2_bot2_description)/meshes/Visual/chassis/charge_port.glb"/>-->
+<!--        </geometry>-->
+<!--      </visual>-->
     </link>
     <joint name="charge_port" type="fixed">
-<!--      <origin xyz="-0.0524 0.1771 0.2463"/>-->
+      <origin xyz="0.283736 0 0.056555" rpy="0 0 0"/>
       <parent link="base_link"/>
       <child link="charge_port"/>
     </joint>
     <link name="lidar_link">
-      		<visual>
-      			<geometry>
-      				<mesh filename="file://$(find sensor_models)/meshes/orbbec/ms500.glb"/>
-      			</geometry>
-      		</visual>
+<!--      <visual>-->
+<!--        <geometry>-->
+<!--          <mesh filename="file://$(find sensor_models)/meshes/orbbec/ms500.glb"/>-->
+<!--        </geometry>-->
+<!--      </visual>-->
     </link>
     <joint name="lidar_joint" type="fixed">
-      <origin xyz="0.260985 0 0.126476"/>
+      <origin xyz="0.260985 0 0.126476" rpy="0 0 1.5708"/>
       <parent link="base_link"/>
       <child link="lidar_link"/>

Commit message: add cameras for ai2_bot2

File: humanoid/Ai2Robotics/ai2_bot2_description/xacro/component.xacro (robot description, xacro)
@@ -9,5 +9,5 @@
     - left_arm / right_arm: root = base_link, both arms only, no body/chassis/ego
 -->
-<robot name="Ai2_Bot2_Arms" xmlns:xacro="http://www.ros.org/wiki/xacro">
+<robot name="Ai2_Bot2" xmlns:xacro="http://www.ros.org/wiki/xacro">
   <!-- component.launch.py default should show the base -->
   <xacro:arg name="type" default="base"/>

File: humanoid/Ai2Robotics/ai2_bot2_description/xacro/components/body.xacro (robot description, xacro)
@@ -117,7 +117,4 @@
           <mesh filename="file://$(find ai2_bot2_description)/meshes/Visual/body/link4.glb" />
         </geometry>
-        <material name="">
-          <color rgba="1 1 1 1" />
-        </material>
       </visual>
       <collision>
@@ -133,4 +130,28 @@
       <axis xyz="0 0 1" />
       <limit lower="-1.5708" upper="1.5708" effort="1000" velocity="10" />
+    </joint>
+    <link name="front_camera">
+      <visual>
+        <geometry>
+          <mesh filename="file://$(find sensor_models)/meshes/d435/d435.obj"/>
+        </geometry>
+      </visual>
+    </link>
+    <joint name="front_camera" type="fixed">
+      <origin xyz="0.1067 0 0.1805" rpy="0 0.38397 0"/>
+      <parent link="body_link4"/>
+      <child link="front_camera"/>
+    </joint>
+    <link name="back_camera">
+      <visual>
+        <geometry>
+          <mesh filename="file://$(find sensor_models)/meshes/d435/d435.obj"/>
+        </geometry>
+      </visual>
+    </link>
+    <joint name="back_camera" type="fixed">
+      <origin xyz="-0.1682 0 0.308" rpy="0 0.4887 3.14159"/>
+      <parent link="body_link4"/>
+      <child link="back_camera"/>
     </joint>
     <!-- head: head_link1 (neck), head_joint1, head_link2 (head), head_joint2 -->
@@ -169,13 +190,10 @@
       <visual>
         <geometry>
-          <mesh filename="file://$(find ai2_bot2_description)/meshes/Visual/body/head_pitch.glb" />
-        </geometry>
-        <material name="">
-          <color rgba="0.75294 0.75294 0.75294 1" />
-        </material>
-      </visual>
-      <collision>
-        <geometry>
-          <mesh filename="file://$(find ai2_bot2_description)/meshes/Visual/body/head_pitch.glb" />
+          <mesh filename="file://$(find ai2_bot2_description)/meshes/Visual/body/head2.glb" />
+        </geometry>
+      </visual>
+      <collision>
+        <geometry>
+          <mesh filename="file://$(find ai2_bot2_description)/meshes/Visual/body/head2.glb" />
         </geometry>
       </collision>
@@ -188,4 +206,16 @@
       <limit lower="-0.4014" upper="0.38397" effort="1000" velocity="10" />
     </joint>
+    <link name="head_camera">
+      <visual>
+        <geometry>
+          <mesh filename="file://$(find sensor_models)/meshes/d435/d435.obj"/>
+        </geometry>
+      </visual>
+    </link>
+    <joint name="head_camera" type="fixed">
+      <origin xyz="0.089 0.0465 0" rpy="1.5708 0 0.5236"/>
+      <parent link="head_link2"/>
+      <child link="head_camera"/>
+    </joint>
   </xacro:macro>
 </robot>
