Commit message: update ai2 bot2

File: humanoid/Ai2Robotics/ai2_bot2_description/xacro/component.xacro (robot description, xacro)
@@ -7,5 +7,5 @@
     - base (full body, no gripper): base_link from chassis, body, ego on body_link4, arms on body_link4
     - arms (arms only, like FiveAges W2): no body, no chassis, no ego; base_link exists for RViz fixed frame
-    - left_arm / right_arm: root = base_link, both arms only, no body/chassis/ego
+    - left_arm / right_arm: single arm, unprefixed (base_link / link1.. / joint1..)
 -->
 <robot name="Ai2_Bot2" xmlns:xacro="http://www.ros.org/wiki/xacro">
@@ -14,6 +14,9 @@
   <!-- Lock chassis joints by default for visualization (like W2) -->
   <xacro:arg name="chassis_joints_movable" default="false"/>
-  <!-- Root link: type=base and type=chassis get base_link from chassis; others need a placeholder for RViz -->
-  <xacro:if value="${'$(arg type)' != 'base' and '$(arg type)' != 'chassis'}">
+  <!-- Isaac asset import: hide rm75 / sensor_models meshes that Isaac already provides. -->
+  <xacro:arg name="isaac" default="true"/>
+  <!-- Root link: type=base/chassis get base_link from chassis; left/right_arm use the arm root;
+       other non-chassis types need a placeholder for RViz. -->
+  <xacro:if value="${'$(arg type)' != 'base' and '$(arg type)' != 'chassis' and '$(arg type)' != 'left_arm' and '$(arg type)' != 'right_arm'}">
     <link name="base_link"/>
   </xacro:if>
@@ -26,6 +29,6 @@
     </joint>
     <xacro:include filename="$(find ai2_bot2_description)/xacro/components/arm.xacro"/>
-    <xacro:Ai2Bot2Arm name="left" parent_link="arm_base" direction="1"/>
-    <xacro:Ai2Bot2Arm name="right" parent_link="arm_base" direction="-1"/>
+    <xacro:Ai2Bot2Arm name="left" parent_link="arm_base" direction="1" isaac="$(arg isaac)"/>
+    <xacro:Ai2Bot2Arm name="right" parent_link="arm_base" direction="-1" isaac="$(arg isaac)"/>
   </xacro:if>
   <xacro:if value="${'$(arg type)' == 'base'}">
@@ -34,5 +37,10 @@
     <xacro:include filename="$(find ai2_bot2_description)/xacro/components/arm.xacro"/>
     <xacro:Ai2Bot2Chassis joints_movable="$(arg chassis_joints_movable)"/>
-    <xacro:Ai2Bot2Body parent_link="base_link"/>
+    <xacro:Ai2Bot2Body parent_link="base_link" isaac="$(arg isaac)"/>
+    <link name="arm_base"/>
+    <joint name="arm_base_joint" type="fixed">
+      <parent link="body_link4"/>
+      <child link="arm_base"/>
+    </joint>
     <link name="ego"></link>
     <joint name="ego_joint" type="fixed">
@@ -41,14 +49,15 @@
       <child link="ego" />
     </joint>
-    <xacro:Ai2Bot2Arm name="left" parent_link="body_link4" direction="1"/>
-    <xacro:Ai2Bot2Arm name="right" parent_link="body_link4" direction="-1"/>
+    <xacro:Ai2Bot2Arm name="left" parent_link="arm_base" direction="1" isaac="$(arg isaac)"/>
+    <xacro:Ai2Bot2Arm name="right" parent_link="arm_base" direction="-1" isaac="$(arg isaac)"/>
+    <xacro:Ai2Bot2Head parent_link="body_link4" isaac="$(arg isaac)"/>
   </xacro:if>
   <xacro:if value="${'$(arg type)' == 'left_arm'}">
     <xacro:include filename="$(find ai2_bot2_description)/xacro/components/arm.xacro"/>
-    <xacro:Ai2Bot2Arm name="left" parent_link="base_link" direction="1"/>
+    <xacro:Ai2Bot2Arm direction="1" standalone="true" isaac="$(arg isaac)"/>
   </xacro:if>
   <xacro:if value="${'$(arg type)' == 'right_arm'}">
     <xacro:include filename="$(find ai2_bot2_description)/xacro/components/arm.xacro"/>
-    <xacro:Ai2Bot2Arm name="right" parent_link="base_link" direction="-1"/>
+    <xacro:Ai2Bot2Arm direction="-1" standalone="true" isaac="$(arg isaac)"/>
   </xacro:if>
   <xacro:if value="${'$(arg type)' == 'chassis'}">
@@ -58,5 +67,6 @@
   <xacro:if value="${'$(arg type)' == 'body'}">
     <xacro:include filename="$(find ai2_bot2_description)/xacro/components/body.xacro"/>
-    <xacro:Ai2Bot2Body parent_link="base_link"/>
+    <xacro:Ai2Bot2Body parent_link="base_link" isaac="$(arg isaac)"/>
+    <xacro:Ai2Bot2Head parent_link="body_link4" isaac="$(arg isaac)"/>
   </xacro:if>
 </robot>

File: humanoid/Ai2Robotics/ai2_bot2_description/xacro/components/arm.xacro (robot description, xacro)
@@ -5,17 +5,19 @@
       Usage: <xacro:Ai2Bot2Arm name="left" parent_link="..." direction="1"/>
              <xacro:Ai2Bot2Arm name="right" parent_link="..." direction="-1"/>
+             name:="" omits the left_/right_ prefix (single-arm component).
+             standalone:=true makes ${prefix}base_link the URDF root (no joint0 / waist mount).
+             isaac:=true hides rm75/sensor meshes on link8 (Isaac asset import).
       Links/joints use ${prefix}base_link, ${prefix}link1..8, ${prefix}joint0..8.
-      Meshes use ZPF_left_* glb with scale="1 ${direction} 1"; set direction to -1 for mirror.
+      Tool frames (M6 CCS style): ${prefix}tcp (physical mount), ${prefix}tcp_offset
+      (virtual planning offset), and optional ${prefix}eef for OCS2.
+      Kinematics are identical for both arms. direction mirrors the shoulder
+      mount (joint0) and link2 visual/collision.
+      Zero pose is the T-pose (former j2=j3=π/2, j5=-π/2 baked into origins).
     -->
-    <xacro:macro name="Ai2Bot2Arm" params="name parent_link direction:=1">
-        <xacro:property name="prefix" value="${name}_"/>
+    <xacro:macro name="Ai2Bot2Arm" params="name:='' parent_link:='' direction:=1 add_eef:=true standalone:=false isaac:=false tcp_offset_xyz:='0 0 0' tcp_offset_rpy:='0 0 0'">
+        <xacro:property name="prefix" value="${name + '_' if name else ''}"/>
         <link name="${prefix}base_link">
             <inertial>
-                <xacro:if value="${direction == 1}">
-                    <origin xyz="1.7227967e-05 -2.7405976e-04 6.7417875e-02"/>
-                </xacro:if>
-                <xacro:if value="${direction == -1}">
-                    <origin xyz="1.7227967e-05 2.7405976e-04 6.7417875e-02"/>
-                </xacro:if>
+                <origin xyz="1.7227967e-05 -2.7405976e-04 6.7417875e-02"/>
                 <mass value="1.39"/>
                 <inertia ixx="1.7468022e-03" ixy="4.4167244e-07" ixz="8.1232278e-07"
@@ -24,37 +26,29 @@
             <visual>
                 <geometry>
-                    <mesh filename="file://$(find ai2_bot2_description)/meshes/Visual/arm/arm_base_link.glb"
-                          scale="1 ${direction} 1"/>
-                </geometry>
-                <material name="">
-                    <color rgba="0.86667 0.86667 0.8902 1"/>
-                </material>
-            </visual>
-            <collision>
-                <geometry>
-                    <mesh filename="file://$(find ai2_bot2_description)/meshes/Visual/arm/arm_base_link.glb"
-                          scale="1 ${direction} 1"/>
-                </geometry>
-            </collision>
-        </link>
-        <joint name="${prefix}joint0" type="fixed">
-            <xacro:if value="${direction == 1}">
-                <origin xyz="-0.061 0.0485 0.3255" rpy="-1.5708 -1.5708 0"/>
-            </xacro:if>
-            <xacro:if value="${direction == -1}">
-                <origin xyz="-0.061 -0.0485 0.3255" rpy="1.5708 -1.5708 0"/>
-            </xacro:if>
-            <parent link="${parent_link}"/>
-            <child link="${prefix}base_link"/>
-            <axis xyz="0 0 0"/>
-        </joint>
-        <link name="${prefix}link1">
-            <inertial>
+                    <mesh filename="file://$(find ai2_bot2_description)/meshes/arm/arm_base_link.glb"/>
+                </geometry>
+            </visual>
+            <collision>
+                <geometry>
+                    <mesh filename="file://$(find ai2_bot2_description)/meshes/arm/arm_base_link.glb"/>
+                </geometry>
+            </collision>
+        </link>
+        <xacro:unless value="${standalone}">
+            <joint name="${prefix}joint0" type="fixed">
                 <xacro:if value="${direction == 1}">
-                    <origin xyz="-1.1436e-3 -1.5043e-2 -3.0119e-2"/>
+                    <origin xyz="-0.061 0.0485 0.3255" rpy="-1.5708 -1.5708 0"/>
                 </xacro:if>
                 <xacro:if value="${direction == -1}">
-                    <origin xyz="-1.1436e-3 1.5043e-2 -3.0119e-2"/>
+                    <origin xyz="-0.061 -0.0485 0.3255" rpy="1.5708 -1.5708 0"/>
                 </xacro:if>
+                <parent link="${parent_link}"/>
+                <child link="${prefix}base_link"/>
+                <axis xyz="0 0 0"/>
+            </joint>
+        </xacro:unless>
+        <link name="${prefix}link1">
+            <inertial>
+                <origin xyz="-1.1436e-3 -1.5043e-2 -3.0119e-2"/>
                 <mass value="0.5885"/>
                 <inertia ixx="1.6599262e-03" ixy="-6.1451353e-05" ixz="1.5137541e-04"
@@ -63,5 +57,5 @@
             <visual>
                 <geometry>
-                    <mesh filename="file://$(find ai2_bot2_description)/meshes/Visual/arm/link1.glb"
+                    <mesh filename="file://$(find ai2_bot2_description)/meshes/arm/link1.glb"
                           scale="1 ${direction} 1"/>
                 </geometry>
@@ -69,16 +63,10 @@
             <collision>
                 <geometry>
-                    <mesh filename="file://$(find ai2_bot2_description)/meshes/Visual/arm/link1.glb"
-                          scale="1 ${direction} 1"/>
+                    <mesh filename="file://$(find ai2_bot2_description)/meshes/arm/link1.glb"/>
                 </geometry>
             </collision>
         </link>
         <joint name="${prefix}joint1" type="revolute">
-            <xacro:if value="${direction == 1}">
-                <origin xyz="0 0 0.1785"/>
-            </xacro:if>
-            <xacro:if value="${direction == -1}">
-                <origin xyz="0 0 0.1785"/>
-            </xacro:if>
+            <origin xyz="0 0 0.1785"/>
             <parent link="${prefix}base_link"/>
             <child link="${prefix}link1"/>
@@ -88,10 +76,5 @@
         <link name="${prefix}link2">
             <inertial>
-                <xacro:if value="${direction == 1}">
-                    <origin xyz="1.255e-4 -6.489e-3 -1.5096e-2"/>
-                </xacro:if>
-                <xacro:if value="${direction == -1}">
-                    <origin xyz="1.255e-4 -6.489e-3 1.5096e-2"/>
-                </xacro:if>
+                <origin xyz="1.255e-4 -6.489e-3 -1.5096e-2"/>
                 <mass value="1.37"/>
                 <inertia ixx="1.7992218e-03" ixy="-1.1620208e-06" ixz="-3.9132877e-06"
@@ -100,30 +83,23 @@
             <visual>
                 <geometry>
-                    <mesh filename="file://$(find ai2_bot2_description)/meshes/Visual/arm/link2.glb"
-                          scale="1 1 ${direction}"/>
-                </geometry>
-            </visual>
-            <collision>
-                <geometry>
-                    <mesh filename="file://$(find ai2_bot2_description)/meshes/Visual/arm/link2.glb"
-                          scale="1 1 ${direction}"/>
+                    <mesh filename="file://$(find ai2_bot2_description)/meshes/arm/link2.glb"/>
+                </geometry>
+            </visual>
+            <collision>
+                <geometry>
+                    <mesh filename="file://$(find ai2_bot2_description)/meshes/arm/link2.glb"/>
                 </geometry>
             </collision>
         </link>
         <joint name="${prefix}joint2" type="revolute">
-            <origin xyz="0 0 0" rpy="-1.5708 -1.5708 0"/>
+            <origin xyz="0 0 0" rpy="-1.5708 0 0"/>
             <parent link="${prefix}link1"/>
             <child link="${prefix}link2"/>
             <axis xyz="0 0 1"/>
-            <limit lower="-0.44" upper="3.1" effort="60" velocity="3.14"/>
+            <limit lower="-2.0108" upper="1.5292" effort="60" velocity="3.14"/>
         </joint>
         <link name="${prefix}link3">
             <inertial>
-                <xacro:if value="${direction == 1}">
-                    <origin xyz="4.7568e-3 3.1731e-3 -9.229e-2"/>
-                </xacro:if>
-                <xacro:if value="${direction == -1}">
-                    <origin xyz="-4.7568e-3 3.1731e-3 -9.229e-2"/>
-                </xacro:if>
+                <origin xyz="4.7568e-3 3.1731e-3 -9.229e-2"/>
                 <mass value="2.29"/>
                 <inertia ixx="3.7492999e-02" ixy="-6.5328616e-05" ixz="6.1380090e-05"
@@ -132,40 +108,23 @@
             <visual>
                 <geometry>
-                    <mesh filename="file://$(find ai2_bot2_description)/meshes/Visual/arm/link3.glb"
-                          scale="${direction} 1 1"/>
-                </geometry>
-            </visual>
-            <collision>
-                <geometry>
-                    <mesh filename="file://$(find ai2_bot2_description)/meshes/Visual/arm/link3.glb"
-                          scale="${direction} 1 1"/>
+                    <mesh filename="file://$(find ai2_bot2_description)/meshes/arm/link3.glb"/>
+                </geometry>
+            </visual>
+            <collision>
+                <geometry>
+                    <mesh filename="file://$(find ai2_bot2_description)/meshes/arm/link3.glb"/>
                 </geometry>
             </collision>
         </link>
         <joint name="${prefix}joint3" type="revolute">
-            <xacro:if value="${direction == 1}">
-                <origin xyz="0 -0.28998 0" rpy="1.5708 -1.5708 0"/>
-            </xacro:if>
-            <xacro:if value="${direction == -1}">
-                <origin xyz="0 -0.28998 0" rpy="1.5708 -1.5708 0"/>
-            </xacro:if>
+            <origin xyz="0 -0.28998 0" rpy="-1.5708 0 3.1415926"/>
             <parent link="${prefix}link2"/>
             <child link="${prefix}link3"/>
-            <xacro:if value="${direction == 1}">
-                <axis xyz="0 0 1"/>
-            </xacro:if>
-            <xacro:if value="${direction == -1}">
-                <axis xyz="0 0 -1"/>
-            </xacro:if>
-            <limit lower="-3.1" upper="3.1" effort="30" velocity="3.14"/>
+            <axis xyz="0 0 1"/>
+            <limit lower="-4.6708" upper="1.5292" effort="30" velocity="3.14"/>
         </joint>
         <link name="${prefix}link4">
             <inertial>
-                <xacro:if value="${direction == 1}">
-                    <origin xyz="-9.542e-3 8.999e-2 -4.374e-3"/>
-                </xacro:if>
-                <xacro:if value="${direction == -1}">
-                    <origin xyz="9.542e-3 8.999e-2 -4.374e-3"/>
-                </xacro:if>
+                <origin xyz="-9.542e-3 8.999e-2 -4.374e-3"/>
                 <mass value="0.82"/>
                 <inertia ixx="2.8633804e-03" ixy="-2.9024436e-05" ixz="2.8630445e-05"
@@ -174,40 +133,23 @@
             <visual>
                 <geometry>
-                    <mesh filename="file://$(find ai2_bot2_description)/meshes/Visual/arm/link4.glb"
-                          scale="${direction} 1 1"/>
-                </geometry>
-            </visual>
-            <collision>
-                <geometry>
-                    <mesh filename="file://$(find ai2_bot2_description)/meshes/Visual/arm/link4.glb"
-                          scale="${direction} 1 1"/>
+                    <mesh filename="file://$(find ai2_bot2_description)/meshes/arm/link4.glb"/>
+                </geometry>
+            </visual>
+            <collision>
+                <geometry>
+                    <mesh filename="file://$(find ai2_bot2_description)/meshes/arm/link4.glb"/>
                 </geometry>
             </collision>
         </link>
         <joint name="${prefix}joint4" type="revolute">
-            <xacro:if value="${direction == 1}">
-                <origin xyz="0.01 0 0" rpy="1.5708 0 0"/>
-            </xacro:if>
-            <xacro:if value="${direction == -1}">
-                <origin xyz="-0.01 0 0" rpy="1.5708 0 0"/>
-            </xacro:if>
+            <origin xyz="0.01 0 0" rpy="1.5708 0 0"/>
             <parent link="${prefix}link3"/>
             <child link="${prefix}link4"/>
-            <xacro:if value="${direction == 1}">
-                <axis xyz="0 0 1"/>
-            </xacro:if>
-            <xacro:if value="${direction == -1}">
-                <axis xyz="0 0 -1"/>
-            </xacro:if>
+            <axis xyz="0 0 1"/>
             <limit lower="-2.27" upper="0" effort="30" velocity="3.14"/>
         </joint>
         <link name="${prefix}link5">
             <inertial>
-                <xacro:if value="${direction == 1}">
-                    <origin xyz="-2.3965e-5 -2.247e-2 -8.5293e-2"/>
-                </xacro:if>
-                <xacro:if value="${direction == -1}">
-                    <origin xyz="2.3965e-5 -2.247e-2 -8.5293e-2"/>
-                </xacro:if>
+                <origin xyz="-2.3965e-5 -2.247e-2 -8.5293e-2"/>
                 <mass value="1.017"/>
                 <inertia ixx="2.2579574e-03" ixy="2.0270009e-07" ixz="3.2535431e-08"
@@ -216,40 +158,23 @@
             <visual>
                 <geometry>
-                    <mesh filename="file://$(find ai2_bot2_description)/meshes/Visual/arm/link5.glb"
-                          scale="${direction} 1 1"/>
-                </geometry>
-            </visual>
-            <collision>
-                <geometry>
-                    <mesh filename="file://$(find ai2_bot2_description)/meshes/Visual/arm/link5.glb"
-                          scale="${direction} 1 1"/>
+                    <mesh filename="file://$(find ai2_bot2_description)/meshes/arm/link5.glb"/>
+                </geometry>
+            </visual>
+            <collision>
+                <geometry>
+                    <mesh filename="file://$(find ai2_bot2_description)/meshes/arm/link5.glb"/>
                 </geometry>
             </collision>
         </link>
         <joint name="${prefix}joint5" type="revolute">
-            <xacro:if value="${direction == 1}">
-                <origin xyz="-0.01 0.3088 0" rpy="-1.5708 0 0"/>
-            </xacro:if>
-            <xacro:if value="${direction == -1}">
-                <origin xyz="0.01 0.3088 0" rpy="-1.5708 0 0"/>
-            </xacro:if>
+            <origin xyz="-0.01 0.3088 0" rpy="-1.5708 -1.5708 0"/>
             <parent link="${prefix}link4"/>
             <child link="${prefix}link5"/>
-            <xacro:if value="${direction == 1}">
-                <axis xyz="0 0 1"/>
-            </xacro:if>
-            <xacro:if value="${direction == -1}">
-                <axis xyz="0 0 -1"/>
-            </xacro:if>
-            <limit lower="-3.1" upper="3.1" effort="10" velocity="3.14"/>
+            <axis xyz="0 0 1"/>
+            <limit lower="-1.5292" upper="4.6708" effort="10" velocity="3.14"/>
         </joint>
         <link name="${prefix}link6">
             <inertial>
-                <xacro:if value="${direction == 1}">
-                    <origin xyz="9.154e-3 -8.103e-3 2.957e-3"/>
-                </xacro:if>
-                <xacro:if value="${direction == -1}">
-                    <origin xyz="9.154e-3 8.103e-3 2.957e-3"/>
-                </xacro:if>
+                <origin xyz="9.154e-3 -8.103e-3 2.957e-3"/>
                 <mass value="0.55"/>
                 <inertia ixx="3.7382788e-04" ixy="3.1477249e-06" ixz="1.5645983e-05"
@@ -258,12 +183,10 @@
             <visual>
                 <geometry>
-                    <mesh filename="file://$(find ai2_bot2_description)/meshes/Visual/arm/link6.glb"
-                          scale="1 ${direction} 1"/>
-                </geometry>
-            </visual>
-            <collision>
-                <geometry>
-                    <mesh filename="file://$(find ai2_bot2_description)/meshes/Visual/arm/link6.glb"
-                          scale="1 ${direction} 1"/>
+                    <mesh filename="file://$(find ai2_bot2_description)/meshes/arm/link6.glb"/>
+                </geometry>
+            </visual>
+            <collision>
+                <geometry>
+                    <mesh filename="file://$(find ai2_bot2_description)/meshes/arm/link6.glb"/>
                 </geometry>
             </collision>
@@ -273,20 +196,10 @@
             <parent link="${prefix}link5"/>
             <child link="${prefix}link6"/>
-            <xacro:if value="${direction == 1}">
-                <axis xyz="0 0 1"/>
-            </xacro:if>
-            <xacro:if value="${direction == -1}">
-                <axis xyz="0 0 -1"/>
-            </xacro:if>
+            <axis xyz="0 0 1"/>
             <limit lower="-1.22" upper="1.22" effort="10" velocity="3.14"/>
         </joint>
         <link name="${prefix}link7">
             <inertial>
-                <xacro:if value="${direction == 1}">
-                    <origin xyz="1.547e-4 5.483e-2 5.55e-3"/>
-                </xacro:if>
-                <xacro:if value="${direction == -1}">
-                    <origin xyz="1.547e-4 5.483e-2 -5.55e-3"/>
-                </xacro:if>
+                <origin xyz="1.547e-4 5.483e-2 5.55e-3"/>
                 <mass value="0.266"/>
                 <inertia ixx="0.000132576941913423" ixy="9.13805899339808E-06" ixz="-9.14363365511958E-08"
@@ -295,22 +208,15 @@
             <visual>
                 <geometry>
-                    <mesh filename="file://$(find ai2_bot2_description)/meshes/Visual/arm/link7.glb"
-                          scale="1 1 ${direction}"/>
-                </geometry>
-            </visual>
-            <collision>
-                <geometry>
-                    <mesh filename="file://$(find ai2_bot2_description)/meshes/Visual/arm/link7.glb"
-                          scale="1 1 ${direction}"/>
+                    <mesh filename="file://$(find ai2_bot2_description)/meshes/arm/link7.glb"/>
+                </geometry>
+            </visual>
+            <collision>
+                <geometry>
+                    <mesh filename="file://$(find ai2_bot2_description)/meshes/arm/link7.glb"/>
                 </geometry>
             </collision>
         </link>
         <joint name="${prefix}joint7" type="revolute">
-            <xacro:if value="${direction == 1}">
-                <origin xyz="0.01 0 0" rpy="1.5708 -1.5708 0"/>
-            </xacro:if>
-            <xacro:if value="${direction == -1}">
-                <origin xyz="0.01 0 0" rpy="1.5708 -1.5708 0"/>
-            </xacro:if>
+            <origin xyz="0.01 0 0" rpy="1.5708 -1.5708 0"/>
             <parent link="${prefix}link6"/>
             <child link="${prefix}link7"/>
@@ -320,31 +226,28 @@
         <link name="${prefix}link8">
             <inertial>
-                <xacro:if value="${direction == 1}">
-                    <origin xyz="-0.000223537609806423 8.8367558294447E-05 -0.0171573759779855"/>
-                </xacro:if>
-                <xacro:if value="${direction == -1}">
-                    <origin xyz="0.000223537609806423 8.8367558294447E-05 -0.0171573759779855"/>
-                </xacro:if>
+                <origin xyz="-0.000223537609806423 8.8367558294447E-05 -0.0171573759779855"/>
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