Commit message: update ai2 bot2

File: humanoid/Ai2Robotics/ai2_bot2_description/xacro/components/body.xacro (robot description, xacro)
@@ -4,7 +4,9 @@
     Ai2-Bot2 body: lower-body chain (body_link1..3, body_joint1..3) + torso (waist_yaw_torso_link, body_joint4).
     Chain: parent_link -> body_link1 -> body_link2 -> body_link3 -> waist_yaw_torso_link.
-    Use <xacro:Ai2Bot2Body parent_link="base_link"/> then attach head/arms to waist_yaw_torso_link.
+    Use <xacro:Ai2Bot2Body parent_link="base_link"/> then attach arms / head to body_link4.
+    Head is a separate macro so Pinocchio order can be body → arms → head.
+    isaac:=true hides sensor_models camera meshes (Isaac asset import).
   -->
-  <xacro:macro name="Ai2Bot2Body" params="parent_link">
+  <xacro:macro name="Ai2Bot2Body" params="parent_link isaac:=false">
     <!-- body_link1 (ankle/calf) -->
     <link name="body_link1">
@@ -22,10 +24,10 @@
       <visual>
         <geometry>
-          <mesh filename="file://$(find ai2_bot2_description)/meshes/Visual/body/link1.glb" />
-        </geometry>
-      </visual>
-      <collision>
-        <geometry>
-          <mesh filename="file://$(find ai2_bot2_description)/meshes/Visual/body/link1.glb" />
+          <mesh filename="file://$(find ai2_bot2_description)/meshes/body/link1.glb" />
+        </geometry>
+      </visual>
+      <collision>
+        <geometry>
+          <mesh filename="file://$(find ai2_bot2_description)/meshes/body/link1.glb" />
         </geometry>
       </collision>
@@ -53,10 +55,10 @@
       <visual>
         <geometry>
-          <mesh filename="file://$(find ai2_bot2_description)/meshes/Visual/body/link2.glb" />
-        </geometry>
-      </visual>
-      <collision>
-        <geometry>
-          <mesh filename="file://$(find ai2_bot2_description)/meshes/Visual/body/link2.glb" />
+          <mesh filename="file://$(find ai2_bot2_description)/meshes/body/link2.glb" />
+        </geometry>
+      </visual>
+      <collision>
+        <geometry>
+          <mesh filename="file://$(find ai2_bot2_description)/meshes/body/link2.glb" />
         </geometry>
       </collision>
@@ -84,10 +86,10 @@
       <visual>
         <geometry>
-          <mesh filename="file://$(find ai2_bot2_description)/meshes/Visual/body/link3.glb" />
-        </geometry>
-      </visual>
-      <collision>
-        <geometry>
-          <mesh filename="file://$(find ai2_bot2_description)/meshes/Visual/body/link3.glb" />
+          <mesh filename="file://$(find ai2_bot2_description)/meshes/body/link3.glb" />
+        </geometry>
+      </visual>
+      <collision>
+        <geometry>
+          <mesh filename="file://$(find ai2_bot2_description)/meshes/body/link3.glb" />
         </geometry>
       </collision>
@@ -115,10 +117,10 @@
       <visual>
         <geometry>
-          <mesh filename="file://$(find ai2_bot2_description)/meshes/Visual/body/link4.glb" />
-        </geometry>
-      </visual>
-      <collision>
-        <geometry>
-          <mesh filename="file://$(find ai2_bot2_description)/meshes/Visual/body/link4.glb" />
+          <mesh filename="file://$(find ai2_bot2_description)/meshes/body/link4.glb" />
+        </geometry>
+      </visual>
+      <collision>
+        <geometry>
+          <mesh filename="file://$(find ai2_bot2_description)/meshes/body/link4.glb" />
         </geometry>
       </collision>
@@ -132,9 +134,11 @@
     </joint>
     <link name="front_camera">
-      <visual>
-        <geometry>
-          <mesh filename="file://$(find sensor_models)/meshes/realsense/d435.glb"/>
-        </geometry>
-      </visual>
+      <xacro:unless value="${isaac}">
+        <visual>
+          <geometry>
+            <mesh filename="file://$(find sensor_models)/meshes/realsense/d435.glb"/>
+          </geometry>
+        </visual>
+      </xacro:unless>
     </link>
     <joint name="front_camera" type="fixed">
@@ -144,9 +148,11 @@
     </joint>
     <link name="back_camera">
-      <visual>
-        <geometry>
-          <mesh filename="file://$(find sensor_models)/meshes/realsense/d435.glb"/>
-        </geometry>
-      </visual>
+      <xacro:unless value="${isaac}">
+        <visual>
+          <geometry>
+            <mesh filename="file://$(find sensor_models)/meshes/realsense/d435.glb"/>
+          </geometry>
+        </visual>
+      </xacro:unless>
     </link>
     <joint name="back_camera" type="fixed">
@@ -155,5 +161,7 @@
       <child link="back_camera"/>
     </joint>
-    <!-- head: head_link1 (neck), head_joint1, head_link2 (head), head_joint2 -->
+  </xacro:macro>
+  <!-- Instantiate after the arms so Pinocchio q is body×4, left×7, right×7, head×2. -->
+  <xacro:macro name="Ai2Bot2Head" params="parent_link:='body_link4' isaac:=false">
     <link name="head_link1">
       <inertial>
@@ -171,5 +179,5 @@
     <joint name="head_joint1" type="revolute">
       <origin xyz="-0.041 0 0.46874" />
-      <parent link="body_link4" />
+      <parent link="${parent_link}" />
       <child link="head_link1" />
       <axis xyz="0 0 1" />
@@ -190,10 +198,10 @@
       <visual>
         <geometry>
-          <mesh filename="file://$(find ai2_bot2_description)/meshes/Visual/body/head2.glb" />
-        </geometry>
-      </visual>
-      <collision>
-        <geometry>
-          <mesh filename="file://$(find ai2_bot2_description)/meshes/Visual/body/head2.glb" />
+          <mesh filename="file://$(find ai2_bot2_description)/meshes/body/head2.glb" />
+        </geometry>
+      </visual>
+      <collision>
+        <geometry>
+          <mesh filename="file://$(find ai2_bot2_description)/meshes/body/head2.glb" />
         </geometry>
       </collision>
@@ -207,9 +215,11 @@
     </joint>
     <link name="head_camera">
-      <visual>
-        <geometry>
-          <mesh filename="file://$(find sensor_models)/meshes/realsense/d435.glb"/>
-        </geometry>
-      </visual>
+      <xacro:unless value="${isaac}">
+        <visual>
+          <geometry>
+            <mesh filename="file://$(find sensor_models)/meshes/realsense/d435.glb"/>
+          </geometry>
+        </visual>
+      </xacro:unless>
     </link>
     <joint name="head_camera" type="fixed">

File: humanoid/Ai2Robotics/ai2_bot2_description/xacro/components/chassis.xacro (robot description, xacro)
@@ -27,5 +27,5 @@
 			<visual>
 				<geometry>
-					<mesh filename="file://$(find ai2_bot2_description)/meshes/Visual/chassis/chassis.glb"/>
+					<mesh filename="file://$(find ai2_bot2_description)/meshes/chassis/chassis.glb"/>
 				</geometry>
 			</visual>
@@ -41,5 +41,5 @@
 			<visual>
 				<geometry>
-					<mesh filename="file://$(find ai2_bot2_description)/meshes/Visual/chassis/driven_v.glb"/>
+					<mesh filename="file://$(find ai2_bot2_description)/meshes/chassis/driven_v.glb"/>
 				</geometry>
 			</visual>
@@ -55,5 +55,5 @@
 			<visual>
 				<geometry>
-					<mesh filename="file://$(find ai2_bot2_description)/meshes/Visual/chassis/driven_h.glb"/>
+					<mesh filename="file://$(find ai2_bot2_description)/meshes/chassis/driven_h.glb"/>
 				</geometry>
 			</visual>
@@ -74,5 +74,5 @@
 			<visual>
 				<geometry>
-					<mesh filename="file://$(find ai2_bot2_description)/meshes/Visual/chassis/driven_v.glb"/>
+					<mesh filename="file://$(find ai2_bot2_description)/meshes/chassis/driven_v.glb"/>
 				</geometry>
 			</visual>
@@ -88,5 +88,5 @@
 			<visual>
 				<geometry>
-					<mesh filename="file://$(find ai2_bot2_description)/meshes/Visual/chassis/driven_h.glb"/>
+					<mesh filename="file://$(find ai2_bot2_description)/meshes/chassis/driven_h.glb"/>
 				</geometry>
 			</visual>
@@ -107,5 +107,5 @@
 			<visual>
 				<geometry>
-					<mesh filename="file://$(find ai2_bot2_description)/meshes/Visual/chassis/driven_v.glb"/>
+					<mesh filename="file://$(find ai2_bot2_description)/meshes/chassis/driven_v.glb"/>
 				</geometry>
 			</visual>
@@ -121,5 +121,5 @@
 			<visual>
 				<geometry>
-					<mesh filename="file://$(find ai2_bot2_description)/meshes/Visual/chassis/driven_h.glb"/>
+					<mesh filename="file://$(find ai2_bot2_description)/meshes/chassis/driven_h.glb"/>
 				</geometry>
 			</visual>
@@ -140,5 +140,5 @@
 			<visual>
 				<geometry>
-					<mesh filename="file://$(find ai2_bot2_description)/meshes/Visual/chassis/driven_v.glb"/>
+					<mesh filename="file://$(find ai2_bot2_description)/meshes/chassis/driven_v.glb"/>
 				</geometry>
 			</visual>
@@ -154,5 +154,5 @@
 			<visual>
 				<geometry>
-					<mesh filename="file://$(find ai2_bot2_description)/meshes/Visual/chassis/driven_h.glb"/>
+					<mesh filename="file://$(find ai2_bot2_description)/meshes/chassis/driven_h.glb"/>
 				</geometry>
 			</visual>
@@ -226,5 +226,5 @@
 			<visual>
 				<geometry>
-					<mesh filename="file://$(find ai2_bot2_description)/meshes/Visual/chassis/charge_port.glb"/>
+					<mesh filename="file://$(find ai2_bot2_description)/meshes/chassis/charge_port.glb"/>
 				</geometry>
 			</visual>
@@ -243,5 +243,5 @@
 		</link>
 		<joint name="lidar_joint" type="fixed">
-			<origin xyz="0.260985 0 0.126476" rpy="0 0 1.5708"/>
+			<origin xyz="0.260985 0 0.126476" />
 			<parent link="base_link"/>
 			<child link="lidar_link"/>

File: humanoid/Ai2Robotics/ai2_bot2_description/xacro/robot.xacro (robot description, xacro)
@@ -4,44 +4,81 @@
 <!-- |    Used by robot_common_launch manipulator.launch.py (xacro_filename=robot.xacro)| -->
 <!-- |    Structure : base_link (chassis) -> body ->                                    | -->
-<!-- |    body_link4; ego and arms both attach to body_link4.                           | -->
+<!-- |    body_link4; arm_base / ego / arms attach to body_link4; head after arms.      | -->
+<!-- |    topology:=dual : split-body planning tree rooted at arm_base.                 | -->
 <!-- =================================================================================== -->
 <robot name="Ai2_Bot2" xmlns:xacro="http://www.ros.org/wiki/xacro">
-  <!-- Parse end-effector type from 'type' arg (similar to FiveAges W2 robot.xacro) -->
   <xacro:arg name="type" default=""/>
+  <xacro:arg name="topology" default="full"/>
+  <xacro:arg name="isaac" default="false"/>
+  <xacro:arg name="eef_fixed_joints" default="false"/>
+  <xacro:arg name="left_tcp_offset_xyz" default="0 0 0"/>
+  <xacro:arg name="left_tcp_offset_rpy" default="0 0 0"/>
+  <xacro:arg name="right_tcp_offset_xyz" default="0 0 0"/>
+  <xacro:arg name="right_tcp_offset_rpy" default="0 0 0"/>
   <xacro:property name="type_arg" value="$(arg type)"/>
+  <xacro:property name="topology_arg" value="$(arg topology)"/>
   <xacro:property name="selected_gripper_type" value=""/>
+  <xacro:property name="arm_add_eef" value="true"/>
   <xacro:if value="${type_arg == 'inspire'}">
     <xacro:property name="selected_gripper_type" value="inspire_eg2"/>
+    <xacro:property name="arm_add_eef" value="false"/>
   </xacro:if>
-  <xacro:include filename="$(find ai2_bot2_description)/xacro/components/chassis.xacro"/>
-  <xacro:include filename="$(find ai2_bot2_description)/xacro/components/body.xacro"/>
   <xacro:include filename="$(find ai2_bot2_description)/xacro/components/arm.xacro"/>
-  <xacro:Ai2Bot2Chassis/>
-  <xacro:Ai2Bot2Body parent_link="base_link"/>
-  <!-- ego frame (only in full robot; not used in component type=arms) -->
-  <link name="ego"></link>
-  <joint name="ego_joint" type="fixed">
-    <origin xyz="-0.061 0 0.3255" rpy="0 0 0" />
-    <parent link="body_link4" />
-    <child link="ego" />
-  </joint>
-  <!-- Arms on body_link4 (W2 full robot uses arm_base under body_link4; we keep arms on body_link4) -->
-  <xacro:Ai2Bot2Arm name="left" parent_link="body_link4" direction="1"/>
-  <xacro:Ai2Bot2Arm name="right" parent_link="body_link4" direction="-1"/>
-  <!-- Inspire EG2 gripper (type:=inspire) -->
-  <xacro:if value="${selected_gripper_type == 'inspire_eg2'}">
-    <xacro:include filename="$(find inspire_description)/xacro/EG2-4C2.xacro"/>
-    <xacro:Gripper name="left"/>
-    <joint name="left_gripper_mount" type="fixed">
-      <parent link="left_ee"/>
-      <child link="left_gripper_base"/>
-      <origin xyz="0 0 0" rpy="0 0 1.5708"/>
+  <xacro:macro name="Ai2Bot2ArmsAndGrippers" params="parent_link">
+    <xacro:Ai2Bot2Arm name="left" parent_link="${parent_link}" direction="1"
+        add_eef="${arm_add_eef}"
+        isaac="$(arg isaac)"
+        tcp_offset_xyz="$(arg left_tcp_offset_xyz)"
+        tcp_offset_rpy="$(arg left_tcp_offset_rpy)"/>
+    <xacro:Ai2Bot2Arm name="right" parent_link="${parent_link}" direction="-1"
+        add_eef="${arm_add_eef}"
+        isaac="$(arg isaac)"
+        tcp_offset_xyz="$(arg right_tcp_offset_xyz)"
+        tcp_offset_rpy="$(arg right_tcp_offset_rpy)"/>
+    <xacro:if value="${selected_gripper_type == 'inspire_eg2'}">
+      <xacro:include filename="$(find inspire_description)/xacro/EG2-4C2.xacro"/>
+      <xacro:Gripper name="left"/>
+      <joint name="left_gripper_mount" type="fixed">
+        <parent link="left_tcp"/>
+        <child link="left_gripper_base"/>
+        <origin xyz="0 0 0" rpy="0 0 1.5708"/>
+      </joint>
+      <xacro:Gripper name="right"/>
+      <joint name="right_gripper_mount" type="fixed">
+        <parent link="right_tcp"/>
+        <child link="right_gripper_base"/>
+        <origin xyz="0 0 0" rpy="0 0 1.5708"/>
+      </joint>
+    </xacro:if>
+  </xacro:macro>
+  <!-- Split-body OCS2: dual-arm tree, root coinciding with arm_base (same mount as body_link4). -->
+  <xacro:if value="${topology_arg == 'dual'}">
+    <link name="base_link"/>
+    <link name="arm_base"/>
+    <joint name="arm_base_joint" type="fixed">
+      <parent link="base_link"/>
+      <child link="arm_base"/>
     </joint>
-    <xacro:Gripper name="right"/>
-    <joint name="right_gripper_mount" type="fixed">
-      <parent link="right_ee"/>
-      <child link="right_gripper_base"/>
-      <origin xyz="0 0 0" rpy="0 0 1.5708"/>
+    <xacro:Ai2Bot2ArmsAndGrippers parent_link="arm_base"/>
+  </xacro:if>
+  <xacro:unless value="${topology_arg == 'dual'}">
+    <xacro:include filename="$(find ai2_bot2_description)/xacro/components/chassis.xacro"/>
+    <xacro:include filename="$(find ai2_bot2_description)/xacro/components/body.xacro"/>
+    <xacro:Ai2Bot2Chassis/>
+    <xacro:Ai2Bot2Body parent_link="base_link" isaac="$(arg isaac)"/>
+    <!-- coinciding with body_link4 so split FK in arm_base matches the live torso TF -->
+    <link name="arm_base"/>
+    <joint name="arm_base_joint" type="fixed">
+      <parent link="body_link4"/>
+      <child link="arm_base"/>
     </joint>
-  </xacro:if>
+    <link name="ego"/>
+    <joint name="ego_joint" type="fixed">
+      <origin xyz="-0.061 0 0.3255" rpy="0 0 0"/>
+      <parent link="body_link4"/>
+      <child link="ego"/>
+    </joint>
+    <xacro:Ai2Bot2ArmsAndGrippers parent_link="arm_base"/>
+    <xacro:Ai2Bot2Head parent_link="body_link4" isaac="$(arg isaac)"/>
+  </xacro:unless>
 </robot>
