Commit message: piper,piper_x,piper_l复用完成+碰撞体配置

File: manipulator/AgileX/piper_description/urdf/piper_l.urdf (robot description, URDF)
Before this commit: robot piper, 12 links, 11 joints
Links:
- link base_link: mass 1.02 -> 1.07
- link camera_stand_link: geometry visual mesh filename=package://piper_description/meshes/camera_stand/realsense_m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
- link link1: mass 0.71 -> 0.11
- link link2: mass 1.17 -> 1.16; geometry collision box size=0.264 0.05 0.05; collision cylinder length=0.095 radius=0.032
- link link3: mass 0.5 -> 0.59; geometry collision box size=0.17 0.038 0.045; collision cylinder length=0.051 radius=0.032
- link link4: mass 0.38 -> 0.37; geometry collision cylinder length=0.05 radius=0.0315; visual mesh filename=package://piper_description/meshes/piper_l/link4.glb
- link link5: mass 0.383 -> 0.38; geometry collision cylinder length=0.06 radius=0.03145; visual mesh filename=package://piper_description/meshes/piper_l/link5.glb
- link link6: mass 0.657 -> 0.0056; geometry collision box size=0.01 0.178 0.015; collision cylinder length=0.04 radius=0.03015
- link link7: mass 0.025 -> None; geometry collision box size=0.0231 0.07 0.037; visual mesh filename=package://piper_description/meshes/gripper/link7.glb
- link link8: mass 0.025 -> None; geometry collision box size=0.0231 0.07 0.037; visual mesh filename=package://piper_description/meshes/gripper/link8.glb
Joints:
- removed joint gripper_joint
- added joint joint7: type prismatic, parent link6, child link7, origin xyz=0 0 0.13503 rpy=1.5708 0 0, axis 0 0 -1, limit lower=0 upper=0.05 effort=100 velocity=1
- joint camera_fixed: origin xyz=-0.032 0 0.018 rpy=0.0 -1.22 0 -> xyz=-0.032 -0.028 0.018 rpy=0.0 -1.22 0
- joint gripper_center_fixed: origin xyz=0 0 0.1358 rpy=0 -1.57 0 -> xyz=0 0 0.13503 rpy=0 -1.5708 0
- joint joint1: limit lower=-2.618 upper=2.618 effort=100 velocity=5 -> lower=-2.618 upper=2.618 effort=100 velocity=3
- joint joint2: limit lower=0 upper=3.14 effort=100 velocity=5 -> lower=0 upper=3.14 effort=100 velocity=3; origin xyz=0 0 0 rpy=1.5708 -0.1359 -3.1416 -> xyz=0 0 0 rpy=1.5708 -0.1745 3.1416
- joint joint3: limit lower=-2.967 upper=0 effort=100 velocity=5 -> lower=-2.697 upper=0 effort=100 velocity=3; origin xyz=0.28503 0 0 rpy=0 0 -1.7939 -> xyz=0.33823 0 0 rpy=0 0 -1.8325
- joint joint4: limit lower=-1.745 upper=1.745 effort=100 velocity=5 -> lower=-1.832 upper=1.832 effort=100 velocity=3; origin xyz=-0.021984 -0.25075 0 rpy=1.5708 0 0 -> xyz=0 -0.3215 0 rpy=1.5708 0 0.0
- joint joint5: axis 0 0 1 -> 0 0 -1; limit lower=-1.22 upper=1.22 effort=100 velocity=5 -> lower=-1.22 upper=1.22 effort=100 velocity=3; origin xyz=0 0 0 rpy=-1.5708 0 0 -> xyz=0 0 0 rpy=-1.5708 0.0 0
- joint joint6: limit lower=-2.0944 upper=2.0944 effort=100 velocity=3 -> lower=-3.14 upper=3.14 effort=100 velocity=3
- joint joint8: axis 0 1 0 -> 0 0 1; limit lower=0 upper=0.035 effort=10 velocity=1 -> lower=-0.05 upper=0 effort=100 velocity=1; mimic joint=gripper_joint multiplier=1 offset=0 -> joint=joint7 multiplier=-1 offset=0; origin xyz=0 0 0.1358 -> xyz=0 0 0.13503 rpy=-1.5708 0 0

File: manipulator/AgileX/piper_description/xacro/components/camera.xacro (robot description, xacro)
@@ -33,4 +33,19 @@
                         </geometry>
                     </visual>
+                    <xacro:if value="${collider == 'convex'}">
+                        <collision name="simple_d435camera">
+                            <geometry>
+                                <mesh filename="file://$(find sensor_models)/meshes/d435/d435.obj"/>
+                            </geometry>
+                        </collision>
+                    </xacro:if>
+                    <xacro:if value="${collider == 'simple'}">
+                        <collision name="simple_d435camera">
+                            <origin xyz="0.005 0 0" rpy="0 0 0"/>
+                            <geometry>
+                                <box size="0.0251 0.0899 0.025"/>
+                            </geometry>
+                        </collision>
+                    </xacro:if>
                 </link>
                 <joint name="${prefix}camera_fixed" type="fixed">
@@ -68,4 +83,19 @@
                         </geometry>
                     </visual>
+                    <xacro:if value="${collider == 'convex'}">
+                        <collision name="simple_d435camera">
+                            <geometry>
+                                <mesh filename="file://$(find sensor_models)/meshes/d435/d435.obj"/>
+                            </geometry>
+                        </collision>
+                    </xacro:if>
+                    <xacro:if value="${collider == 'simple'}">
+                        <collision name="simple_d435camera">
+                            <origin xyz="-0.01 0 0" rpy="0 0 0"/>
+                            <geometry>
+                                <box size="0.0251 0.0899 0.025"/>
+                            </geometry>
+                        </collision>
+                    </xacro:if>
                 </link>
                 <joint name="${prefix}camera_fixed" type="fixed">
@@ -75,52 +105,53 @@
                 </joint>
             </xacro:if>
-<!--            <xacro:if value="${arm_type == 'piper'}">-->
-<!--                <link name="${prefix}camera_stand_link">-->
-<!--                    <visual>-->
-<!--                        <geometry>-->
-<!--                            <mesh filename="file://$(find piper_description)/meshes/camera_stand/camera_stand.glb"/>-->
-<!--                        </geometry>-->
-<!--                    </visual>-->
-<!--                    <xacro:if value="${collider == 'convex'}">-->
-<!--                        <collision>-->
-<!--                            <geometry>-->
-<!--                                <mesh filename="file://$(find piper_description)/meshes/camera_stand/camera_stand.glb"/>-->
-<!--                            </geometry>-->
-<!--                        </collision>-->
-<!--                    </xacro:if>-->
-<!--                </link>-->
-<!--                <joint name="${prefix}camera_stand_joint" type="fixed">-->
-<!--                    <origin rpy="1.57 1.57 -1.57" xyz="0.001 -0.036 0.022"/>-->
-<!--                    <parent link="${parent_link}"/>-->
-<!--                    <child link="${prefix}camera_stand_link"/>-->
-<!--                </joint>-->
-<!--                <link name="${prefix}camera">-->
-<!--                    <visual>-->
-<!--                        <geometry>-->
-<!--                            <mesh filename="file://$(find sensor_models)/meshes/d435/d435.obj"/>-->
-<!--                        </geometry>-->
-<!--                    </visual>-->
-<!--                    <xacro:if value="${collider == 'convex'}">-->
-<!--                        <collision>-->
-<!--                            <geometry>-->
-<!--                                <mesh filename="file://$(find sensor_models)/meshes/d435/d435.obj"/>-->
-<!--                            </geometry>-->
-<!--                        </collision>-->
-<!--                    </xacro:if>-->
-<!--                    <xacro:if value="${collider == 'simple'}">-->
-<!--                        <collision name="simple_d435camera">-->
-<!--                            <origin xyz="-0.0125 0 0" rpy="0 0 0"/>-->
-<!--                            <geometry>-->
-<!--                                <box size="0.0251 0.0899 0.025"/>-->
-<!--                            </geometry>-->
-<!--                        </collision>-->
-<!--                    </xacro:if>-->
-<!--                </link>-->
-<!--                <joint name="${prefix}camera_fixed" type="fixed">-->
-<!--                    <origin xyz="-0.073 0 0.041" rpy="-0.3463 0 -1.5708"/>-->
-<!--                    <parent link="${prefix}camera_stand_link"/>-->
-<!--                    <child link="${prefix}camera"/>-->
-<!--                </joint>-->
-<!--            </xacro:if>-->
+            <xacro:if value="${arm_type == 'piper'}">
+                <link name="${prefix}camera_stand_link">
+                    <visual>
+                        <origin rpy="3.14 0 1.57" xyz="0.0 0.0 0.0"/>
+                        <geometry>
+                            <mesh filename="file://$(find piper_description)/meshes/camera_stand/camera_stand.glb"/>
+                        </geometry>
+                    </visual>
+                    <xacro:if value="${collider == 'convex'}">
+                        <collision>
+                            <geometry>
+                                <mesh filename="file://$(find piper_description)/meshes/camera_stand/camera_stand.glb"/>
+                            </geometry>
+                        </collision>
+                    </xacro:if>
+                </link>
+                <joint name="${prefix}camera_stand_joint" type="fixed">
+                    <origin rpy="0 0 0" xyz="-0.034 -0.002 0.023"/>
+                    <parent link="${parent_link}"/>
+                    <child link="${prefix}camera_stand_link"/>
+                </joint>
+                <link name="${prefix}camera">
+                    <visual>
+                        <geometry>
+                            <mesh filename="file://$(find sensor_models)/meshes/d435/d435.obj"/>
+                        </geometry>
+                    </visual>
+                    <xacro:if value="${collider == 'convex'}">
+                        <collision>
+                            <geometry>
+                                <mesh filename="file://$(find sensor_models)/meshes/d435/d435.obj"/>
+                            </geometry>
+                        </collision>
+                    </xacro:if>
+                    <xacro:if value="${collider == 'simple'}">
+                        <collision name="simple_d435camera">
+                            <origin xyz="-0.0125 0 0" rpy="0 0 0"/>
+                            <geometry>
+                                <box size="0.0251 0.0899 0.025"/>
+                            </geometry>
+                        </collision>
+                    </xacro:if>
+                </link>
+                <joint name="${prefix}camera_fixed" type="fixed">
+                    <origin xyz="-0.032 0 0.018" rpy="0.0 -1.22 0"/>
+                    <parent link="${prefix}camera_stand_link"/>
+                    <child link="${prefix}camera"/>
+                </joint>
+            </xacro:if>
         </xacro:if>
     </xacro:macro>

File: manipulator/AgileX/piper_description/xacro/components/gripper_l.xacro (robot description, xacro)
@@ -23,4 +23,18 @@
                 </collision>
             </xacro:if>
+            <xacro:if value="${collider == 'simple'}">
+                <collision name="simple_link6_1">
+                    <origin xyz="0 0 0.025" rpy="0 0 0"/>
+                    <geometry>
+                        <cylinder length="0.04" radius="0.03015"/>
+                    </geometry>
+                </collision>
+                <collision name="simple_link6_2">
+                    <origin xyz="0 0 0.06" rpy="0 ${PI/2} 0"/>
+                    <geometry>
+                        <box size="0.01 0.178 0.015"/>
+                    </geometry>
+                </collision>
+            </xacro:if>
         </link>
         <joint name="${prefix}joint6" type="revolute">
@@ -41,4 +55,12 @@
                     <geometry>
                         <mesh filename="file://$(find piper_description)/meshes/gripper/link7.glb"/>
+                    </geometry>
+                </collision>
+            </xacro:if>
+            <xacro:if value="${collider == 'simple'}">
+                <collision name="simple_link7">
+                    <origin xyz="0 -0.0125 -0.012" rpy="0 ${PI/2} 0"/>
+                    <geometry>
+                        <box size="0.0231 0.07 0.037"/>
                     </geometry>
                 </collision>
@@ -65,4 +87,12 @@
                 </collision>
             </xacro:if>
+            <xacro:if value="${collider == 'simple'}">
+                <collision name="simple_link8">
+                    <origin xyz="0 0.0125 -0.012" rpy="0 ${PI/2} 0"/>
+                    <geometry>
+                        <box size="0.0231 0.07 0.037"/>
+                    </geometry>
+                </collision>
+            </xacro:if>
         </link>
         <joint name="${prefix}joint8" type="prismatic">

File: manipulator/AgileX/piper_description/xacro/components/gripper_slave.xacro (robot description, xacro)
@@ -16,9 +16,25 @@
                 </geometry>
             </visual>
-            <collision>
-                <geometry>
-                    <mesh filename="file://$(find piper_description)/meshes/piper/link6.glb"/>
-                </geometry>
-            </collision>
+            <xacro:if value="${collider == 'convex'}">
+                <collision>
+                    <geometry>
+                        <mesh filename="file://$(find piper_description)/meshes/piper/link6.glb"/>
+                    </geometry>
+                </collision>
+            </xacro:if>
+            <xacro:if value="${collider == 'simple'}">
+                <collision name="simple_link6_1">
+                    <origin xyz="0 0 0.025" rpy="0 0 0"/>
+                    <geometry>
+                        <cylinder length="0.04" radius="0.03015"/>
+                    </geometry>
+                </collision>
+                <collision name="simple_link6_2">
+                    <origin xyz="0 0 0.06" rpy="0 ${PI/2} 0"/>
+                    <geometry>
+                        <box size="0.01 0.178 0.015"/>
+                    </geometry>
+                </collision>
+            </xacro:if>
         </link>
         <joint name="${prefix}joint6" type="revolute">
@@ -41,9 +57,19 @@
                 </geometry>
             </visual>
-            <collision>
-                <geometry>
-                    <mesh filename="file://$(find piper_description)/meshes/gripper/gripper.glb"/>
-                </geometry>
-            </collision>
+            <xacro:if value="${collider == 'simple'}">
+                <collision>
+                    <geometry>
+                        <mesh filename="file://$(find piper_description)/meshes/gripper/gripper.glb"/>
+                    </geometry>
+                </collision>
+            </xacro:if>
+            <xacro:if value="${collider == 'simple'}">
+                <collision name="simple_link7">
+                    <origin xyz="0 -0.0125 -0.03" rpy="${PI/2} 0 ${PI/2}"/>
+                    <geometry>
+                        <box size="0.0231 0.07 0.037"/>
+                    </geometry>
+                </collision>
+            </xacro:if>
         </link>
         <joint name="${prefix}gripper_joint" type="prismatic">
@@ -66,9 +92,19 @@
                 </geometry>
             </visual>
-            <collision>
-                <geometry>
-                    <mesh filename="file://$(find piper_description)/meshes/gripper/gripper.glb" scale="1 -1 1"/>
-                </geometry>
-            </collision>
+            <xacro:if value="${collider == 'convex'}">
+                <collision>
+                    <geometry>
+                        <mesh filename="file://$(find piper_description)/meshes/gripper/gripper.glb" scale="1 -1 1"/>
+                    </geometry>
+                </collision>
+            </xacro:if>
+            <xacro:if value="${collider == 'simple'}">
+                <collision name="simple_link8">
+                    <origin xyz="0 0.0125 -0.03" rpy="${PI/2} 0 ${PI/2}"/>
+                    <geometry>
+                        <box size="0.0231 0.07 0.037"/>
+                    </geometry>
+                </collision>
+            </xacro:if>
         </link>
         <joint name="${prefix}joint8" type="prismatic">
@@ -86,5 +122,5 @@
             <origin xyz="0 0 0.1358" rpy="0 -1.57 0"/>
         </joint>
-<!--        <xacro:piper_camera prefix="${prefix}" parent_link="${prefix}link6" camera="${camera}" collider="${collider}" arm_type="piper"/>-->
+        <xacro:piper_camera prefix="${prefix}" parent_link="${prefix}link6" camera="${camera}" collider="${collider}" arm_type="piper"/>
     </xacro:macro>
 </robot>

File: manipulator/AgileX/piper_description/xacro/components/gripper_x.xacro (robot description, xacro)
@@ -20,4 +20,18 @@
                     <geometry>
                         <mesh filename="file://$(find piper_description)/meshes/piper_x/link6.glb"/>
+                    </geometry>
+                </collision>
+            </xacro:if>
+            <xacro:if value="${collider == 'simple'}">
+                <collision name="simple_link6_1">
+                    <origin xyz="0 0 0.025" rpy="0 0 0"/>
+                    <geometry>
+                        <cylinder length="0.04" radius="0.03015"/>
+                    </geometry>
+                </collision>
+                <collision name="simple_link6_2">
+                    <origin xyz="0 0 0.06" rpy="0 ${PI/2} ${PI/2}"/>
+                    <geometry>
+                        <box size="0.01 0.178 0.015"/>
                     </geometry>
                 </collision>
@@ -79,4 +93,12 @@
                 </collision>
             </xacro:if>
+            <xacro:if value="${collider == 'simple'}">
+                <collision name="simple_link7">
+                    <origin xyz="0 -0.0125 -0.012" rpy="0 ${PI/2} 0"/>
+                    <geometry>
+                        <box size="0.0231 0.07 0.037"/>
+                    </geometry>
+                </collision>
+            </xacro:if>
         </link>
         <joint name="${prefix}joint7" type="prismatic">
@@ -106,4 +128,12 @@
                 </collision>
             </xacro:if>
+            <xacro:if value="${collider == 'simple'}">
+                <collision name="simple_link8">
+                    <origin xyz="0 0.0125 -0.012" rpy="0 ${PI/2} 0"/>
+                    <geometry>
+                        <box size="0.0231 0.07 0.037"/>
+                    </geometry>
+                </collision>
+            </xacro:if>
         </link>
         <joint name="${prefix}joint8" type="prismatic">

File: manipulator/AgileX/piper_description/xacro/piper_arm.xacro (robot description, xacro)
@@ -1,5 +1,5 @@
 <?xml version="1.0"?>
 <robot xmlns:xacro="http://www.ros.org/wiki/xacro">
-    <xacro:arg name="collider" default="convex"/>
+    <xacro:arg name="collider" default="simple"/>
     <xacro:property name="PI" value="3.1415926535897931"/>
     <xacro:property name="collider_type" value="$(arg collider)"/>
@@ -25,4 +25,12 @@
                 </collision>
             </xacro:if>
+            <xacro:if value="${collider == 'simple'}">
+                <collision>
+                    <origin xyz="-0.0035 0 0.045"/>
+                    <geometry>
+                        <cylinder length="0.07" radius="0.04"/>
+                    </geometry>
+                </collision>
+            </xacro:if>
         </link>
         <link name="${prefix}link1">
@@ -72,4 +80,24 @@
                 </collision>
             </xacro:if>
+            <xacro:if value="${collider == 'simple'}">
+                <collision name="simple_link2_1">
+                    <origin xyz="0 0 0" rpy="0 0 0"/>
+                    <geometry>
+                        <cylinder length="0.095" radius="0.032"/>
+                    </geometry>
+                </collision>
+                <collision name="simple_link2_2">
+                    <origin xyz="0.285 0.002 0" rpy="0 0 0"/>
+                    <geometry>
+                        <cylinder length="0.095" radius="0.032"/>
+                    </geometry>
+                </collision>
+                <collision name="simple_link2_3">
+                    <origin xyz="0.132 -0.02 0" rpy="0 0 -${PI/18}"/>
+                    <geometry>
+                        <box size="0.264 0.05 0.05"/>
+                    </geometry>
+                </collision>
+            </xacro:if>
         </link>
         <joint name="${prefix}joint2" type="revolute">
@@ -99,4 +127,18 @@
                 </collision>
             </xacro:if>
+            <xacro:if value="${collider == 'simple'}">
+                <collision name="simple_link3_1">
+                    <origin xyz="-0.022 -0.18 0" rpy="0 -${PI/2} ${PI/2}"/>
+                    <geometry>
+                        <cylinder length="0.049" radius="0.03"/>
+                    </geometry>
+                </collision>
+                <collision name="simple_link3_2">
+                    <origin xyz="-0.022 -0.08 0" rpy="0 0 ${PI/2}"/>
+                    <geometry>
+                        <box size="0.15 0.035 0.04"/>
+                    </geometry>
+                </collision>
+            </xacro:if>
         </link>
         <joint name="${prefix}joint3" type="revolute">
@@ -126,4 +168,12 @@
                 </collision>
             </xacro:if>
+            <xacro:if value="${collider == 'simple'}">
+                <collision name="simple_link4">
+                    <origin xyz="0 0.00022 0" rpy="-${PI/2} 0 0"/>
+                    <geometry>
+                        <cylinder length="0.06" radius="0.0315"/>
+                    </geometry>
+                </collision>
+            </xacro:if>
         </link>
         <joint name="${prefix}joint4" type="revolute">
@@ -150,4 +200,18 @@
                     <geometry>
                         <mesh filename="file://$(find piper_description)/meshes/piper_l/link5.glb"/>
+                    </geometry>
+                </collision>
+            </xacro:if>
+            <xacro:if value="${collider == 'simple'}">
+                <collision name="simple_link5_1">
+                    <origin xyz="0 -0.06 0" rpy="${PI/2} 0 0"/>
+                    <geometry>
+                        <cylinder length="0.06" radius="0.03145"/>
+                    </geometry>
+                </collision>
+                <collision name="simple_link5_2">
+                    <origin xyz="0.00038 -0.0008 -0.015" />
+                    <geometry>
+                        <cylinder length="0.008" radius="0.03145"/>
                     </geometry>
                 </collision>
