Commit message: piper,piper_x,piper_l复用完成+碰撞体配置

File: manipulator/AgileX/piper_description/xacro/piper_l_arm.xacro (robot description, xacro)
@@ -26,4 +26,12 @@
                 </collision>
             </xacro:if>
+            <xacro:if value="${collider == 'simple'}">
+                <collision>
+                    <origin xyz="-0.0035 0 0.045"/>
+                    <geometry>
+                        <cylinder length="0.07" radius="0.04"/>
+                    </geometry>
+                </collision>
+            </xacro:if>
         </link>
         <link name="${prefix}link1">
@@ -73,4 +81,24 @@
                 </collision>
             </xacro:if>
+            <xacro:if value="${collider == 'simple'}">
+                <collision name="simple_link2_1">
+                    <origin xyz="0 0 0" rpy="0 0 0"/>
+                    <geometry>
+                        <cylinder length="0.095" radius="0.032"/>
+                    </geometry>
+                </collision>
+                <collision name="simple_link2_2">
+                    <origin xyz="0.34 0 0" rpy="0 0 0"/>
+                    <geometry>
+                        <cylinder length="0.095" radius="0.032"/>
+                    </geometry>
+                </collision>
+                <collision name="simple_link2_3">
+                    <origin xyz="0.15 -0.02 0" rpy="0 0 -${PI/18}"/>
+                    <geometry>
+                        <box size="0.264 0.05 0.05"/>
+                    </geometry>
+                </collision>
+            </xacro:if>
         </link>
         <joint name="${prefix}joint2" type="revolute">
@@ -100,4 +128,18 @@
                 </collision>
             </xacro:if>
+            <xacro:if value="${collider == 'simple'}">
+                <collision name="simple_link3_1">
+                    <origin xyz="-0.005 -0.252 0" rpy="-${PI/2} 0 ${PI/32}"/>
+                    <geometry>
+                        <cylinder length="0.051" radius="0.032"/>
+                    </geometry>
+                </collision>
+                <collision name="simple_link3_2">
+                    <origin xyz="-0.016 -0.13 0" rpy="0 0 ${(17/32)*PI}"/>
+                    <geometry>
+                        <box size="0.17 0.038 0.045"/>
+                    </geometry>
+                </collision>
+            </xacro:if>
         </link>
         <joint name="${prefix}joint3" type="revolute">
@@ -127,4 +169,12 @@
                 </collision>
             </xacro:if>
+            <xacro:if value="${collider == 'simple'}">
+                <collision name="simple_link4">
+                    <origin xyz="-0.005 0 0" rpy="-${PI/2} 0 0"/>
+                    <geometry>
+                        <cylinder length="0.05" radius="0.0315"/>
+                    </geometry>
+                </collision>
+            </xacro:if>
         </link>
         <joint name="${prefix}joint4" type="revolute">
@@ -151,4 +201,12 @@
                     <geometry>
                         <mesh filename="file://$(find piper_description)/meshes/piper_l/link5.glb"/>
+                    </geometry>
+                </collision>
+            </xacro:if>
+            <xacro:if value="${collider == 'simple'}">
+                <collision name="simple_link5_1">
+                    <origin xyz="0 -0.065 0" rpy="${PI/2} 0 0"/>
+                    <geometry>
+                        <cylinder length="0.06" radius="0.03145"/>
                     </geometry>
                 </collision>

File: manipulator/AgileX/piper_description/xacro/piper_x_arm.xacro (robot description, xacro)
@@ -5,5 +5,5 @@
     <xacro:property name="collider_type" value="$(arg collider)"/>
     <xacro:include filename="$(find piper_description)/xacro/components/gripper_x.xacro"/>
-    <xacro:macro name="piper_x_arm" params="name collider:=convex camera:=d435 with_gripper:='true'">
+    <xacro:macro name="piper_x_arm" params="name collider:=simple camera:=d435 with_gripper:='true'">
         <xacro:property name="prefix" value="${name + '_' if name else ''}"/>
         <link name="${prefix}base_link">
@@ -28,4 +28,12 @@
                 </collision>
             </xacro:if>
+            <xacro:if value="${collider == 'simple'}">
+                <collision>
+                    <origin xyz="-0.0035 0 0.045"/>
+                    <geometry>
+                        <cylinder length="0.07" radius="0.04"/>
+                    </geometry>
+                </collision>
+            </xacro:if>
         </link>
         <link name="${prefix}link1">
@@ -75,4 +83,24 @@
                 </collision>
             </xacro:if>
+            <xacro:if value="${collider == 'simple'}">
+                <collision name="simple_link2_1">
+                    <origin xyz="0 0 0" rpy="0 0 0"/>
+                    <geometry>
+                        <cylinder length="0.095" radius="0.032"/>
+                    </geometry>
+                </collision>
+                <collision name="simple_link2_2">
+                    <origin xyz="0.285 0.002 0" rpy="0 0 0"/>
+                    <geometry>
+                        <cylinder length="0.095" radius="0.032"/>
+                    </geometry>
+                </collision>
+                <collision name="simple_link2_3">
+                    <origin xyz="0.132 -0.02 0" rpy="0 0 -${PI/18}"/>
+                    <geometry>
+                        <box size="0.264 0.05 0.05"/>
+                    </geometry>
+                </collision>
+            </xacro:if>
         </link>
         <joint name="${prefix}joint2" type="revolute">
@@ -102,4 +130,18 @@
                 </collision>
             </xacro:if>
+            <xacro:if value="${collider == 'simple'}">
+                <collision name="simple_link3_1">
+                    <origin xyz="0.27 0 0" rpy="0 0 0"/>
+                    <geometry>
+                        <cylinder length="0.051" radius="0.032"/>
+                    </geometry>
+                </collision>
+                <collision name="simple_link3_2">
+                    <origin xyz="0.15 -0.008 0" rpy="0 0 ${(33/32)*PI}"/>
+                    <geometry>
+                        <box size="0.17 0.038 0.045"/>
+                    </geometry>
+                </collision>
+            </xacro:if>
         </link>
         <joint name="${prefix}joint3" type="revolute">
@@ -129,4 +171,12 @@
                 </collision>
             </xacro:if>
+            <xacro:if value="${collider == 'simple'}">
+                <collision name="simple_link4">
+                    <origin xyz="0.077 -0.061 0" rpy="-${PI/2} 0 0"/>
+                    <geometry>
+                        <cylinder length="0.04" radius="0.0315"/>
+                    </geometry>
+                </collision>
+            </xacro:if>
         </link>
         <joint name="${prefix}joint4" type="revolute">
@@ -153,4 +203,18 @@
                     <geometry>
                         <mesh filename="file://$(find piper_description)/meshes/piper_x/link5.glb"/>
+                    </geometry>
+                </collision>
+            </xacro:if>
+            <xacro:if value="${collider == 'simple'}">
+                <collision name="simple_link5_1">
+                    <origin xyz="0 0 0" rpy="${PI/2} 0 ${PI/2}"/>
+                    <geometry>
+                        <cylinder length="0.06" radius="0.03145"/>
+                    </geometry>
+                </collision>
+                <collision name="simple_link5_2">
+                    <origin xyz="0.00038 -0.0008 -0.035" />
+                    <geometry>
+                        <cylinder length="0.008" radius="0.03145"/>
                     </geometry>
                 </collision>

File: manipulator/AgileX/piper_description/xacro/robot.xacro (robot description, xacro)
@@ -1,15 +1,14 @@
 <?xml version="1.0"?>
 <robot name="piper" xmlns:xacro="http://www.ros.org/wiki/xacro">
-    <xacro:arg name="collider" default="convex"/>
+    <xacro:arg name="collider" default="simple"/>
     <xacro:arg name="type" default="piper"/>
     <xacro:arg name="style" default="slave"/>
-    <xacro:if value="${'$(arg type)' == 'piper'}">
+    <xacro:if value="${'$(arg type)' == 'master'}">
         <xacro:include filename="$(find piper_description)/xacro/piper_arm.xacro"/>
-        <xacro:if value="${'$(arg style)' == 'master'}">
-            <xacro:piper_arm name="" collider="$(arg collider)" is_master="true"/>
-        </xacro:if>
-        <xacro:if value="${'$(arg style)' == 'slave'}">
-            <xacro:piper_arm name="" collider="$(arg collider)" is_master="false"/>
-        </xacro:if>
+        <xacro:piper_arm name="" collider="$(arg collider)" is_master="true"/>
+    </xacro:if>
+    <xacro:if value="${'$(arg type)' == 'slave' or '$(arg type)' == 'piper'}">
+        <xacro:include filename="$(find piper_description)/xacro/piper_arm.xacro"/>
+        <xacro:piper_arm name="" collider="$(arg collider)" is_master="false"/>
     </xacro:if>
     <xacro:if value="${'$(arg type)' == 'piper_x'}">

File: manipulator/AgileX/piper_description/xacro/ros2_control/robot.xacro (robot description, xacro)
@@ -1,5 +1,8 @@
 <?xml version="1.0"?>
-<robot xmlns:xacro="http://www.ros.org/wiki/xacro" name="R5a">
+<robot name="piper_system" xmlns:xacro="http://www.ros.org/wiki/xacro">
   <xacro:arg name="ros2_control_hardware_type" default="mock_components" />
+  <xacro:arg name="gazebo" default="false" />
+  <xacro:arg name="type" default="piper" />
+  <xacro:arg name="collider" default="convex" />
   <link name="world"/>
   <joint name="world_fixed" type="fixed">
@@ -7,16 +10,36 @@
     <child link="base_link"/>
   </joint>
-  <xacro:arg name="type" default="slave"/>
-  <xacro:include filename="$(find piper_description)/xacro/Piper.xacro"/>
-  <!-- 根据type参数决定is_master的值 -->
-  <xacro:Piper name="" is_master="false"/>
-  <!-- Import Piper ros2_control description -->
-  <xacro:include filename="$(find piper_description)/xacro/ros2_control/piper.ros2_control.xacro" />
-  <xacro:piper_system name="" ros2_control_hardware_type="$(arg ros2_control_hardware_type)"/>
-  <xacro:arg name="gazebo" default="false" />
+  <xacro:include filename="$(find piper_description)/xacro/robot.xacro"/>
+  <xacro:include filename="$(find piper_description)/xacro/ros2_control/interfaces.xacro"/>
+  <ros2_control name="piper_system" type="system">
+    <hardware>
+      <xacro:if value="${'$(arg ros2_control_hardware_type)' == 'gz'}">
+        <plugin>gz_ros2_control/GazeboSimSystem</plugin>
+      </xacro:if>
+      <xacro:if value="${'$(arg ros2_control_hardware_type)' == 'mock_components'}">
+        <plugin>mock_components/GenericSystem</plugin>
+      </xacro:if>
+      <xacro:if value="${'$(arg ros2_control_hardware_type)' == 'isaac'}">
+        <plugin>topic_based_ros2_control/TopicBasedSystem</plugin>
+        <param name="joint_commands_topic">/isaac/joint_command</param>
+        <param name="joint_states_topic">/isaac/joint_states</param>
+      </xacro:if>
+      <xacro:if value="${'$(arg ros2_control_hardware_type)' == 'real'}">
+      </xacro:if>
+    </hardware>
+    <xacro:piper_interfaces name="" type="$(arg type)"/>
+  </ros2_control>
   <xacro:if value="$(arg gazebo)">
     <gazebo>
       <plugin filename="gz_ros2_control-system" name="gz_ros2_control::GazeboSimROS2ControlPlugin">
-        <parameters>$(find piper_description)/config/ros2_control/ros2_controllers.yaml</parameters>
+        <xacro:if value="${'$(arg type)' == 'l'}">
+          <parameters>$(find piper_description)/config/ros2_control/piper_l_controllers.yaml</parameters>
+        </xacro:if>
+        <xacro:if value="${'$(arg type)' == 'x'}">
+          <parameters>$(find piper_description)/config/ros2_control/piper_x_controllers.yaml</parameters>
+        </xacro:if>
+        <xacro:if value="${'$(arg type)' == 'piper'}">
+          <parameters>$(find piper_description)/config/ros2_control/ros2_controllers.yaml</parameters>
+        </xacro:if>
       </plugin>
     </gazebo>
