Commit message: update visual

File: humanoid/Galbot/galbot_one_description/urdf/galbot_one.urdf (robot description, URDF)
Before this commit: robot galbot_one, 56 links, 55 joints
Links:
- added link chassis_lidar; visual mesh filename=file:///home/king/ros2_ws/install/sensor_models/share/senso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
- added link left_gripper_l4_link, mass 0.01; visual mesh filename=package://galbot_one_description/meshes/gripper_hitbot/link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
- added link left_gripper_l5_link, mass 0.01; visual mesh filename=package://galbot_one_description/meshes/gripper_hitbot/link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
- added link left_gripper_r4_link, mass 0.01; visual mesh filename=package://galbot_one_description/meshes/gripper_hitbot/link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 scale=1 1 -1
- added link left_gripper_r5_link, mass 0.01; visual mesh filename=package://galbot_one_description/meshes/gripper_hitbot/link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 scale=1 1 -1
- added link right_gripper_l4_link, mass 0.01; visual mesh filename=package://galbot_one_description/meshes/gripper_hitbot/link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
- added link right_gripper_l5_link, mass 0.01; visual mesh filename=package://galbot_one_description/meshes/gripper_hitbot/link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
- added link right_gripper_r4_link, mass 0.01; visual mesh filename=package://galbot_one_description/meshes/gripper_hitbot/link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 scale=1 1 -1
- added link right_gripper_r5_link, mass 0.01; visual mesh filename=package://galbot_one_description/meshes/gripper_hitbot/link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 scale=1 1 -1
- added link wheel_1, mass 4.24803000494366; visual mesh filename=file:///home/king/ros2_ws/install/component_models/share/co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
- added link wheel_2, mass 4.24803000494366; visual mesh filename=file:///home/king/ros2_ws/install/component_models/share/co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
- added link wheel_3, mass 4.24803000494366; visual mesh filename=file:///home/king/ros2_ws/install/component_models/share/co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
- added link wheel_4, mass 4.24803000494366; visual mesh filename=file:///home/king/ros2_ws/install/component_models/share/co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
- link head_base_link: geometry visual mesh filename=file:///home/king/ros2_ws/install/galbot_one_description/sh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
- link head_link1: geometry visual mesh filename=file:///home/king/ros2_ws/install/galbot_one_description/sh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
- link head_link2: geometry visual mesh filename=file:///home/king/ros2_ws/install/galbot_one_description/sh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
- link left_arm_base_link: geometry visual mesh filename=package://galbot_one_description/meshes/arm/base.glb
- link left_arm_camera_flange_link: geometry visual mesh filename=package://galbot_one_description/meshes/camera/arm_camera.g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
- link left_arm_link1: geometry visual mesh filename=package://galbot_one_description/meshes/arm/left_arm_link1.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
- link left_arm_link2: geometry collision cylinder length=0.19825 radius=0.044983; visual mesh filename=package://galbot_one_description/meshes/arm/left_arm_link2.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
- link left_arm_link3: geometry collision cylinder length=0.223485 radius=0.044983; visual mesh filename=package://galbot_one_description/meshes/arm/left_arm_link3.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
- link left_arm_link4: geometry collision cylinder length=0.12085 radius=0.044983; visual mesh filename=package://galbot_one_description/meshes/arm/left_arm_link4.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
- link left_arm_link5: geometry collision cylinder length=0.068650 radius=0.034983; visual mesh filename=package://galbot_one_description/meshes/arm/left_arm_link5.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
- link left_flange_base_link: geometry visual mesh filename=package://galbot_one_description/meshes/flange/flange.glb
- link left_gripper_base_link: geometry collision box size=0.095000 0.047000 0.067000; visual mesh filename=package://galbot_one_description/meshes/gripper_hitbot/base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
- link left_gripper_l1_link: mass 0 -> 0.01; geometry visual mesh filename=package://galbot_one_description/meshes/gripper_hitbot/link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
- link left_gripper_l2_link: mass 0 -> 0.01; geometry visual mesh filename=package://galbot_one_description/meshes/gripper_hitbot/link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
- link left_gripper_l3_link: mass 0 -> 0.01; geometry visual mesh filename=package://galbot_one_description/meshes/gripper_hitbot/link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
- link left_gripper_r1_link: mass 0 -> 0.01; geometry visual mesh filename=package://galbot_one_description/meshes/gripper_hitbot/link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 scale=1 1 -1
- link left_gripper_r2_link: mass 0 -> 0.01; geometry visual mesh filename=package://galbot_one_description/meshes/gripper_hitbot/link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 scale=1 1 -1
- link left_gripper_r3_link: mass 0 -> 0.01; geometry visual mesh filename=package://galbot_one_description/meshes/gripper_hitbot/link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 scale=1 1 -1
- link leg_base_link: geometry visual mesh filename=file:///home/king/ros2_ws/install/galbot_one_description/sh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
- link leg_link1: geometry visual mesh filename=file:///home/king/ros2_ws/install/galbot_one_description/sh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
- link leg_link2: geometry visual mesh filename=file:///home/king/ros2_ws/install/galbot_one_description/sh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
- link leg_link3: geometry visual mesh filename=file:///home/king/ros2_ws/install/galbot_one_description/sh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
- link leg_link4: geometry visual mesh filename=file:///home/king/ros2_ws/install/galbot_one_description/sh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
- link omni_chassis_base_link: geometry visual mesh filename=package://galbot_one_description/meshes/chassis/chassis.glb
- link right_arm_base_link: geometry visual mesh filename=package://galbot_one_description/meshes/arm/base.glb scale=1 -1 1
- link right_arm_camera_flange_link: geometry visual mesh filename=package://galbot_one_description/meshes/camera/arm_camera.g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
- link right_arm_link1: geometry visual mesh filename=package://galbot_one_description/meshes/arm/left_arm_link1.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 scale=1 -1 1
- link right_arm_link2: geometry collision cylinder length=0.19825 radius=0.044983; visual mesh filename=package://galbot_one_description/meshes/arm/left_arm_link2.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 scale=-1 1 1
- link right_arm_link3: geometry collision cylinder length=0.223485 radius=0.044983; visual mesh filename=package://galbot_one_description/meshes/arm/left_arm_link3.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 scale=1 -1 1
- link right_arm_link4: geometry collision cylinder length=0.12085 radius=0.044983; visual mesh filename=package://galbot_one_description/meshes/arm/left_arm_link4.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 scale=1 -1 1
- link right_arm_link5: geometry collision cylinder length=0.068650 radius=0.044983; visual mesh filename=package://galbot_one_description/meshes/arm/left_arm_link5.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
- link right_arm_link6: geometry collision cylinder length=0.085000 radius=0.044983; visual mesh filename=package://galbot_one_description/meshes/arm/left_arm_link6.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
- link right_arm_link7: geometry collision cylinder length=0.075650 radius=0.044983; visual mesh filename=package://galbot_one_description/meshes/arm/left_arm_link7.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
- link right_flange_base_link: geometry visual mesh filename=package://galbot_one_description/meshes/flange/flange.glb
- link right_gripper_base_link: geometry collision box size=0.095000 0.047000 0.067000; visual mesh filename=package://galbot_one_description/meshes/gripper_hitbot/base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
- link right_gripper_l1_link: mass 0 -> 0.01; geometry visual mesh filename=package://galbot_one_description/meshes/gripper_hitbot/link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
- link right_gripper_l2_link: mass 0 -> 0.01; geometry visual mesh filename=package://galbot_one_description/meshes/gripper_hitbot/link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
- link right_gripper_l3_link: mass 0 -> 0.01; geometry visual mesh filename=package://galbot_one_description/meshes/gripper_hitbot/link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
- link right_gripper_r1_link: mass 0 -> 0.01; geometry visual mesh filename=package://galbot_one_description/meshes/gripper_hitbot/link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 scale=1 1 -1
- link right_gripper_r2_link: mass 0 -> 0.01; geometry visual mesh filename=package://galbot_one_description/meshes/gripper_hitbot/link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 scale=1 1 -1
- link right_gripper_r3_link: mass 0 -> 0.01; geometry visual mesh filename=package://galbot_one_description/meshes/gripper_hitbot/link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 scale=1 1 -1
- link torso_base_link: geometry collision box size=0.155192 0.181326 0.165600; collision box size=0.232789 0.271990 0.248400
Joints:
- removed joint left_gripper_l1_joint
- removed joint right_gripper_l1_joint
- added joint chassis_lidar_joint: type fixed, parent omni_chassis_base_link, child chassis_lidar, origin xyz=0.222 0 0.22772
- added joint left_gripper_l4_joint: type fixed, parent left_gripper_l3_link, child left_gripper_l4_link, origin xyz=0 0 0 rpy=0 0 0
- added joint left_gripper_l5_joint: type fixed, parent left_gripper_l3_link, child left_gripper_l5_link, origin xyz=0 0 0 rpy=0 0 0
- added joint left_gripper_mount_joint: type fixed, parent left_flange_mount_link, child left_gripper_base_link, origin rpy=1.5707963267948966  1.5707963267948966  0
- added joint left_gripper_r4_joint: type fixed, parent left_gripper_r3_link, child left_gripper_r4_link, origin xyz=0 0 0 rpy=0 0 0
- added joint left_gripper_r5_joint: type fixed, parent left_gripper_r3_link, child left_gripper_r5_link, origin xyz=0 0 0 rpy=0 0 0
- added joint right_gripper_l4_joint: type fixed, parent right_gripper_l3_link, child right_gripper_l4_link, origin xyz=0 0 0 rpy=0 0 0
- added joint right_gripper_l5_joint: type fixed, parent right_gripper_l3_link, child right_gripper_l5_link, origin xyz=0 0 0 rpy=0 0 0
- added joint right_gripper_mount_joint: type fixed, parent right_flange_mount_link, child right_gripper_base_link, origin rpy=1.5707963267948966  1.5707963267948966  0
- added joint right_gripper_r4_joint: type fixed, parent right_gripper_r3_link, child right_gripper_r4_link, origin xyz=0 0 0 rpy=0 0 0
- added joint right_gripper_r5_joint: type fixed, parent right_gripper_r3_link, child right_gripper_r5_link, origin xyz=0 0 0 rpy=0 0 0
- added joint wheel1_joint: type fixed, parent omni_chassis_base_link, child wheel_1, origin xyz=0.176493 0.176493 0.071834 rpy=0 0 -2.356194490192345
- added joint wheel2_joint: type fixed, parent omni_chassis_base_link, child wheel_2, origin xyz=-0.176493 0.176493 0.071834 rpy=0 0 -0.7853981633974483
- added joint wheel3_joint: type fixed, parent omni_chassis_base_link, child wheel_3, origin xyz=-0.176493 -0.176493 0.071834 rpy=0 0 0.7853981633974483
- added joint wheel4_joint: type fixed, parent omni_chassis_base_link, child wheel_4, origin xyz=0.176493 -0.176493 0.071834 rpy=0 0 2.356194490192345
- joint head_joint: origin xyz=0 0 0 rpy=0 0 0 -> 
- joint head_joint1: limit lower=-1.570796327 upper=1.570796327 effort=4 velocity=8.38 -> lower=-1.5707963267948966 upper=1.5707963267948966 effort=4 velocity=8.38; origin xyz=0 0 0.068 rpy=0 0 0 -> xyz=0 0 0.068
- joint head_joint2: origin xyz=0 0 0 rpy=-1.5707963267948966 0 0 -> rpy=-1.5707963267948966 0 0
- joint left_arm_joint: origin xyz=0 0 0 rpy=0 0 0 -> (none)
- joint left_flange_joint: origin xyz=0 0 0 rpy=0 0 2.617993878 -> xyz=0 0 0 rpy=0 0 3.14
- joint left_gripper_joint: axis (none) -> 0 1 0; child left_gripper_base_link -> left_gripper_l1_link; limit (none) -> lower=0 upper=1 effort=2 velocity=3; origin xyz=0 0 0 rpy=0 1.5707963267948966 0 -> xyz=-0.121835 0 0.02; parent left_flange_mount_link -> left_gripper_base_link; type fixed -> revolute
- joint left_gripper_l2_joint: limit lower=0 upper=3 effort=2 velocity=3 -> lower=0 upper=1 effort=2 velocity=3; mimic (none) -> joint=left_gripper_joint multiplier=1.0; origin xyz=-0.1368 0 0.01 rpy=0 0 0 -> xyz=-0.1368 0 0.01
- joint left_gripper_l3_joint: limit lower=0 upper=3 effort=2 velocity=3 -> lower=0 upper=1 effort=2 velocity=3; mimic (none) -> joint=left_gripper_joint multiplier=1.0; origin xyz=-0.064985 0 0.00125 rpy=0 0 0 -> xyz=-0.064985 0 0.00125
- joint left_gripper_r1_joint: limit lower=0 upper=3 effort=2 velocity=3 -> lower=0 upper=1 effort=2 velocity=3; mimic (none) -> joint=left_gripper_joint multiplier=1.0; origin xyz=-0.121835 0 -0.02 rpy=0 0 0 -> xyz=-0.121835 0 -0.02
- joint left_gripper_r2_joint: limit lower=0 upper=3 effort=2 velocity=3 -> lower=0 upper=1 effort=2 velocity=3; mimic (none) -> joint=left_gripper_joint multiplier=1.0; origin xyz=-0.1368 0 -0.01 rpy=0 0 0 -> xyz=-0.1368 0 -0.01
- joint left_gripper_r3_joint: limit lower=0 upper=3 effort=2 velocity=3 -> lower=0 upper=1 effort=2 velocity=3; mimic (none) -> joint=left_gripper_joint multiplier=1.0; origin xyz=-0.064985 0 -0.00125 rpy=0 0 0 -> xyz=-0.064985 0 -0.00125
- joint leg_joint: origin xyz=0 0 0 rpy=0 0 0 -> 
- joint leg_joint4: limit lower=-1.570796327 upper=1.570796327 effort=30 velocity=3.56 -> lower=-1.5707963267948966 upper=1.5707963267948966 effort=30 velocity=3.56; origin xyz=0 0 0 rpy=1.5707963267948966 0 -3.141592653589793 -> rpy=1.5707963267948966 0 -3.141592653589793
- joint leg_torso_mount_joint: axis 0 0 0 -> ; origin xyz=0 0 0 rpy=0 0 0 -> 
- joint omni_chassis_joint: origin xyz=0 0 0 rpy=0 0 0 -> (none)
- joint omni_chassis_leg_mount_joint: axis 0 0 0 -> (none)
- joint right_arm_joint: origin xyz=0 0 0 rpy=0 0 0 -> (none)
- joint right_flange_joint: origin xyz=0 0 0 rpy=0 0 2.617993878 -> xyz=0 0 0 rpy=0 0 0
- joint right_gripper_joint: axis (none) -> 0 1 0; child right_gripper_base_link -> right_gripper_l1_link; limit (none) -> lower=0 upper=1 effort=2 velocity=3; origin xyz=0 0 0 rpy=0 1.5707963267948966 0 -> xyz=-0.121835 0 0.02; parent right_flange_mount_link -> right_gripper_base_link; type fixed -> revolute
- joint right_gripper_l2_joint: limit lower=0 upper=3 effort=2 velocity=3 -> lower=0 upper=1 effort=2 velocity=3; mimic (none) -> joint=right_gripper_joint multiplier=1.0; origin xyz=-0.1368 0 0.01 rpy=0 0 0 -> xyz=-0.1368 0 0.01
- joint right_gripper_l3_joint: limit lower=0 upper=3 effort=2 velocity=3 -> lower=0 upper=1 effort=2 velocity=3; mimic (none) -> joint=right_gripper_joint multiplier=1.0; origin xyz=-0.064985 0 0.00125 rpy=0 0 0 -> xyz=-0.064985 0 0.00125
- joint right_gripper_r1_joint: limit lower=0 upper=3 effort=2 velocity=3 -> lower=0 upper=1 effort=2 velocity=3; mimic (none) -> joint=right_gripper_joint multiplier=1.0; origin xyz=-0.121835 0 -0.02 rpy=0 0 0 -> xyz=-0.121835 0 -0.02
- joint right_gripper_r2_joint: limit lower=0 upper=3 effort=2 velocity=3 -> lower=0 upper=1 effort=2 velocity=3; mimic (none) -> joint=right_gripper_joint multiplier=1.0; origin xyz=-0.1368 0 -0.01 rpy=0 0 0 -> xyz=-0.1368 0 -0.01
- joint right_gripper_r3_joint: limit lower=0 upper=3 effort=2 velocity=3 -> lower=0 upper=1 effort=2 velocity=3; mimic (none) -> joint=right_gripper_joint multiplier=1.0; origin xyz=-0.064985 0 -0.00125 rpy=0 0 0 -> xyz=-0.064985 0 -0.00125
- joint torso_head_mount_joint: origin xyz=-0.0081669 5E-05 0.51594 rpy=0 0 0 -> xyz=-0.0081669 5E-05 0.51594
- joint torso_joint: origin xyz=0 0 0 rpy=0 0 0 -> 

File: humanoid/Galbot/galbot_one_description/xacro/components/arm.xacro (robot description, xacro)
@@ -13,12 +13,7 @@
     <visual>
       <geometry>
-        <mesh filename="package://galbot_one_description/meshes/arm/base.glb" scale="1 -1 1"/>
-      </geometry>
-    </visual>
-    <collision>
-      <geometry>
-        <mesh filename="package://galbot_one_description/meshes/arm/right_arm_base_link_convex.stl"/>
-      </geometry>
-    </collision>
+        <mesh filename="package://galbot_one_description/meshes/arm/base.glb" scale ="1 -1 1"/>
+      </geometry>
+    </visual>
   </link>
   <link name="right_arm_link1">
@@ -33,9 +28,4 @@
       </geometry>
     </visual>
-    <collision>
-      <geometry>
-        <mesh filename="package://galbot_one_description/meshes/arm/right_arm_link1_convex.stl"/>
-      </geometry>
-    </collision>
   </link>
   <joint name="right_arm_joint1" type="revolute">
@@ -58,6 +48,7 @@
     </visual>
     <collision>
-      <geometry>
-        <mesh filename="package://galbot_one_description/meshes/arm/right_arm_link2_convex.stl"/>
+      <origin rpy="-1.5707963267948966 0 0" xyz="0 -0.074 0"/>
+      <geometry>
+        <cylinder length="0.19825" radius="0.044983"/>
       </geometry>
     </collision>
@@ -82,6 +73,7 @@
     </visual>
     <collision>
-      <geometry>
-        <mesh filename="package://galbot_one_description/meshes/arm/right_arm_link3_convex.stl"/>
+      <origin rpy="0 0 0" xyz="0 0 -0.074"/>
+      <geometry>
+        <cylinder length="0.223485" radius="0.044983"/>
       </geometry>
     </collision>
@@ -106,6 +98,7 @@
     </visual>
     <collision>
-      <geometry>
-        <mesh filename="package://galbot_one_description/meshes/arm/right_arm_link4_convex.stl"/>
+      <origin rpy="1.5707963267948966 0 0" xyz=" 0 -0.040  0"/>
+      <geometry>
+        <cylinder length="0.12085" radius="0.044983"/>
       </geometry>
     </collision>
@@ -126,10 +119,11 @@
     <visual>
       <geometry>
-        <mesh filename="package://galbot_one_description/meshes/arm/left_arm_link5.glb"/>
-      </geometry>
-    </visual>
-    <collision>
-      <geometry>
-        <mesh filename="package://galbot_one_description/meshes/arm/right_arm_link5_convex.stl"/>
+        <mesh filename="package://galbot_one_description/meshes/arm/left_arm_link5.glb" />
+      </geometry>
+    </visual>
+    <collision>
+      <origin rpy="0 0 0" xyz="0 0 0"/>
+      <geometry>
+        <cylinder length="0.068650" radius="0.044983"/>
       </geometry>
     </collision>
@@ -150,10 +144,10 @@
     <visual>
       <geometry>
-        <mesh filename="package://galbot_one_description/meshes/arm/left_arm_link6.glb" scale="1 -1 1"/>
-      </geometry>
-    </visual>
-    <collision>
-      <geometry>
-        <mesh filename="package://galbot_one_description/meshes/arm/right_arm_link6_convex.stl"/>
+        <mesh filename="package://galbot_one_description/meshes/arm/left_arm_link6.glb" />
+      </geometry>
+    </visual>
+    <collision>
+      <geometry>
+        <cylinder length="0.085000" radius="0.044983"/>
       </geometry>
     </collision>
@@ -174,10 +168,10 @@
     <visual>
       <geometry>
-        <mesh filename="package://galbot_one_description/meshes/arm/left_arm_link7.glb" scale="1 -1 1"/>
-      </geometry>
-    </visual>
-    <collision>
-      <geometry>
-        <mesh filename="package://galbot_one_description/meshes/arm/right_arm_link7_convex.stl"/>
+        <mesh filename="package://galbot_one_description/meshes/arm/left_arm_link7.glb" />
+      </geometry>
+    </visual>
+    <collision>
+      <geometry>
+        <cylinder length="0.075650" radius="0.044983"/>
       </geometry>
     </collision>
@@ -198,5 +192,4 @@
   </joint>
   <joint name="right_flange_joint" type="fixed">
-    <origin rpy="0 0 0" xyz="0 0 0"/>
     <parent link="right_arm_end_effector_mount_link"/>
     <child link="right_flange_base_link"/>
@@ -213,9 +206,4 @@
       </geometry>
     </visual>
-    <collision>
-      <geometry>
-        <mesh filename="package://galbot_one_description/meshes/flange/flange_base_link_convex.stl"/>
-      </geometry>
-    </collision>
   </link>
   <link name="right_flange_mount_link"/>
@@ -242,9 +230,4 @@
       </geometry>
     </visual>
-    <collision>
-      <geometry>
-        <mesh filename="package://galbot_one_description/meshes/camera/arm_camera_convex.stl"/>
-      </geometry>
-    </collision>
   </link>
   <joint name="left_arm_joint" type="fixed">
@@ -265,5 +248,5 @@
     <collision>
       <geometry>
-        <mesh filename="package://galbot_one_description/meshes/arm/left_arm_base_link_convex.stl"/>
+        <cylinder length="0.091350" radius="0.044983"/>
       </geometry>
     </collision>
@@ -282,5 +265,5 @@
     <collision>
       <geometry>
-        <mesh filename="package://galbot_one_description/meshes/arm/left_arm_link1_convex.stl"/>
+        <cylinder length="0.068650" radius="0.044983"/>
       </geometry>
     </collision>
@@ -305,6 +288,7 @@
     </visual>
     <collision>
-      <geometry>
-        <mesh filename="package://galbot_one_description/meshes/arm/left_arm_link2_convex.stl"/>
+      <origin rpy="1.5707963267948966 0 0" xyz="0 -0.074 0"/>
+      <geometry>
+        <cylinder length="0.19825" radius="0.044983"/>
       </geometry>
     </collision>
@@ -329,6 +313,7 @@
     </visual>
     <collision>
-      <geometry>
-        <mesh filename="package://galbot_one_description/meshes/arm/left_arm_link3_convex.stl"/>
+      <origin rpy="0 0 0" xyz="0 0 -0.074"/>
+      <geometry>
+        <cylinder length="0.223485" radius="0.044983"/>
       </geometry>
     </collision>
@@ -354,6 +339,7 @@
     </visual>
     <collision>
-      <geometry>
-        <mesh filename="package://galbot_one_description/meshes/arm/left_arm_link4_convex.stl"/>
+      <origin rpy="1.5707963267948966 0 0" xyz=" 0 -0.040  0"/>
+      <geometry>
+        <cylinder length="0.12085" radius="0.044983"/>
       </geometry>
     </collision>
@@ -376,8 +362,9 @@
         <mesh filename="package://galbot_one_description/meshes/arm/left_arm_link5.glb"/>
       </geometry>
-    </visual>
-    <collision>
-      <geometry>
-        <mesh filename="package://galbot_one_description/meshes/arm/left_arm_link5_convex.stl"/>
+    </visual>S
+    <collision>
+      <origin rpy="0 0 0" xyz="0 -0.046 -0.09"/>
+      <geometry>
+        <cylinder length="0.068650" radius="0.034983"/>
       </geometry>
     </collision>
@@ -403,5 +390,5 @@
     <collision>
       <geometry>
-        <mesh filename="package://galbot_one_description/meshes/arm/left_arm_link6_convex.stl"/>
+        <cylinder length="0.085000" radius="0.044983"/>
       </geometry>
     </collision>
@@ -427,5 +414,5 @@
     <collision>
       <geometry>
-        <mesh filename="package://galbot_one_description/meshes/arm/left_arm_link7_convex.stl"/>
+        <cylinder length="0.075650" radius="0.044983"/>
       </geometry>
     </collision>
@@ -446,5 +433,5 @@
   </joint>
   <joint name="left_flange_joint" type="fixed">
-    <origin rpy="0 0 3.14" xyz="0 0 0"/>
+    <origin rpy="0 0 3.14"/>
     <parent link="left_arm_end_effector_mount_link"/>
     <child link="left_flange_base_link"/>
@@ -461,9 +448,4 @@
       </geometry>
     </visual>
-    <collision>
-      <geometry>
-        <mesh filename="package://galbot_one_description/meshes/flange/flange_base_link_convex.stl"/>
-      </geometry>
-    </collision>
   </link>
   <link name="left_flange_mount_link"/>
@@ -475,5 +457,5 @@
   </joint>
   <joint name="left_arm_camera_joint" type="fixed">
-    <origin rpy="3.1415926 -1.308996939 0" xyz="0.0526 -0.02 0.02054"/>
+    <origin rpy="3.14 -1.308996939 0" xyz="0.0526 -0.02 0.02054"/>
     <parent link="left_flange_base_link"/>
     <child link="left_arm_camera_flange_link"/>
@@ -490,9 +472,4 @@
       </geometry>
     </visual>
-    <collision>
-      <geometry>
-        <mesh filename="package://galbot_one_description/meshes/camera/arm_camera_convex.stl"/>
-      </geometry>
-    </collision>
   </link>
 </robot>
