Commit message: update visual

File: humanoid/Galbot/galbot_one_description/xacro/components/body.xacro (robot description, xacro)
@@ -42,13 +42,7 @@
       <origin/>
       <geometry>
-        <mesh filename="file://$(find galbot_one_description)/meshes/leg/leg_base_link.stl"/>
-      </geometry>
-    </visual>
-    <collision>
-      <origin  />
-      <geometry>
-        <mesh filename="file://$(find galbot_one_description)/meshes/leg/leg_base_link_convex.stl"/>
-      </geometry>
-    </collision>
+        <mesh filename="file://$(find galbot_one_description)/meshes/leg/leg_base.glb"/>
+      </geometry>
+    </visual>
   </link>
   <link name="leg_link1">
@@ -64,10 +58,4 @@
       </geometry>
     </visual>
-    <collision>
-      <origin  />
-      <geometry>
-        <mesh filename="file://$(find galbot_one_description)/meshes/leg/leg_link1_convex.stl"/>
-      </geometry>
-    </collision>
   </link>
   <joint name="leg_joint1" type="revolute">
@@ -90,10 +78,4 @@
       </geometry>
     </visual>
-    <collision>
-      <origin  />
-      <geometry>
-        <mesh filename="file://$(find galbot_one_description)/meshes/leg/leg_link2_convex.stl"/>
-      </geometry>
-    </collision>
   </link>
   <joint name="leg_joint2" type="revolute">
@@ -116,10 +98,4 @@
       </geometry>
     </visual>
-    <collision>
-      <origin  />
-      <geometry>
-        <mesh filename="file://$(find galbot_one_description)/meshes/leg/leg_link3_convex.stl"/>
-      </geometry>
-    </collision>
   </link>
   <joint name="leg_joint3" type="revolute">
@@ -142,10 +118,4 @@
       </geometry>
     </visual>
-    <collision>
-      <origin  />
-      <geometry>
-        <mesh filename="file://$(find galbot_one_description)/meshes/leg/leg_link4_convex.stl"/>
-      </geometry>
-    </collision>
   </link>
   <joint name="leg_joint4" type="revolute">
@@ -206,13 +176,7 @@
       <origin/>
       <geometry>
-        <mesh filename="file://$(find galbot_one_description)/meshes/head/head_base_link.stl"/>
-      </geometry>
-    </visual>
-    <collision>
-      <origin  />
-      <geometry>
-        <mesh filename="file://$(find galbot_one_description)/meshes/head/head_base_link_convex.stl"/>
-      </geometry>
-    </collision>
+        <mesh filename="file://$(find galbot_one_description)/meshes/head/head_base.glb"/>
+      </geometry>
+    </visual>
   </link>
   <link name="head_link1">
@@ -228,10 +192,4 @@
       </geometry>
     </visual>
-    <collision>
-      <origin  />
-      <geometry>
-        <mesh filename="file://$(find galbot_one_description)/meshes/head/head_link1_convex.stl"/>
-      </geometry>
-    </collision>
   </link>
   <joint name="head_joint1" type="revolute">
@@ -254,10 +212,4 @@
       </geometry>
     </visual>
-    <collision>
-      <origin  />
-      <geometry>
-        <mesh filename="file://$(find galbot_one_description)/meshes/head/head_link2_convex.stl"/>
-      </geometry>
-    </collision>
   </link>
   <joint name="head_joint2" type="revolute">

File: humanoid/Galbot/galbot_one_description/xacro/components/chassis.xacro (robot description, xacro)
@@ -22,6 +22,7 @@
       </visual>
       <collision>
+        <origin rpy="0 0 0" xyz="0 0 0"/>
         <geometry>
-          <mesh filename="package://galbot_one_description/meshes/chassis/omni_chassis_base_link_convex.stl"/>
+          <box size="0.40 0.40 0.20"/>
         </geometry>
       </collision>

File: humanoid/Galbot/galbot_one_description/xacro/components/gripper.xacro (robot description, xacro)
@@ -3,5 +3,5 @@
   <xacro:property name="PI" value="3.141592653589793"/>
   <!-- mount_rpy defines gripper_base_link frame orientation relative to flange_mount_link. -->
-  <xacro:macro name="Gripper" params="name mount_rpy:='${PI/2}  0  0'">
+  <xacro:macro name="Gripper" params="name mount_rpy:='${PI/2}  ${PI/2}  0'">
     <xacro:property name="prefix" value="${name + '_' if name else ''}"/>
     <!-- Mount gripper on flange (fixed) -->
@@ -40,5 +40,5 @@
       </visual>
     </link>
-    <!-- Main driven finger joint (shows in joint_state_publisher as gripper_joint) -->
+    <!-- Main driven finger joint (Astribot-style: *_gripper_joint) -->
     <joint name="${prefix}gripper_joint" type="revolute">
       <origin xyz="-0.121835 0 0.02"/>

File: humanoid/Galbot/galbot_one_description/xacro/robot.xacro (robot description, xacro)
@@ -32,7 +32,9 @@
   -->
   <xacro:arg name="type" default="gripper"/>
-  <xacro:include filename="$(find galbot_one_description)/xacro/components/base.xacro"/>
+  <xacro:include filename="$(find galbot_one_description)/xacro/components/chassis.xacro"/>
+  <xacro:include filename="$(find galbot_one_description)/xacro/components/body.xacro"/>
   <xacro:include filename="$(find galbot_one_description)/xacro/components/arm.xacro"/>
   <xacro:include filename="$(find galbot_one_description)/xacro/components/gripper.xacro"/>
+  <xacro:GalbotOneChassis enable_wheel_joints="$(arg enable_wheel_joints)"/>
   <xacro:if value="${'$(arg type)' == 'gripper'}">
     <!-- Instantiate both grippers -->

File: humanoid/Galbot/galbot_one_description/xacro/ros2_control/robot.xacro (robot description, xacro)
@@ -25,16 +25,14 @@
 #####################################################################################
 -->
-<robot name="galbot_one" xmlns:xacro="http://www.ros.org/wiki/xacro">
+<robot name="galbot_one_ros2_control" xmlns:xacro="http://www.ros.org/wiki/xacro">
+  <xacro:arg name="type" default="gripper"/>
+  <xacro:arg name="ros2_control_hardware_type" default="mock_components"/>
   <xacro:property name="ros2_control_config_basename" value="ros2_controllers.yaml"/>
-  <xacro:include filename="$(find galbot_one_description)/xacro/ros2_control/chassis.xacro"/>
-  <xacro:include filename="$(find galbot_one_description)/xacro/ros2_control/torso.xacro"/>
-  <!-- ROBOT -->
-  <!-- Robot Base Link -->
-  <xacro:include filename="$(find galbot_one_description)/xacro/ros2_control/leg.xacro"/>
-  <xacro:include filename="$(find galbot_one_description)/xacro/ros2_control/head.xacro"/>
-  <xacro:include filename="$(find galbot_one_description)/xacro/ros2_control/gripper.xacro"/>
-  <!-- Head Mount -->
-    <!-- Right Arm Mount -->
-  <xacro:include filename="$(find galbot_one_description)/xacro/ros2_control/arm.xacro"/>
+  <!-- Geometry/kinematics come from main robot xacro -->
+  <xacro:include filename="$(find galbot_one_description)/xacro/robot.xacro"/>
+  <!-- ros2_control interfaces (Astribot-style split) -->
+  <xacro:include filename="$(find galbot_one_description)/xacro/ros2_control/galbot_one_base_interfaces.xacro"/>
+  <xacro:include filename="$(find galbot_one_description)/xacro/ros2_control/galbot_one_arm_interfaces.xacro"/>
+  <xacro:include filename="$(find galbot_one_description)/xacro/ros2_control/galbot_one_gripper_interfaces.xacro"/>
   <ros2_control name="galbot_one_system" type="system">
     <hardware>
@@ -51,133 +49,11 @@
       </xacro:if>
     </hardware>
-    <joint name="leg_joint1"><command_interface name="position"/><state_interface name="position"/><state_interface name="velocity"/></joint>
-    <joint name="leg_joint2"><command_interface name="position"/><state_interface name="position"/><state_interface name="velocity"/></joint>
-    <joint name="leg_joint3"><command_interface name="position"/><state_interface name="position"/><state_interface name="velocity"/></joint>
-    <joint name="leg_joint4"><command_interface name="position"/><state_interface name="position"/><state_interface name="velocity"/></joint>
-    <joint name="left_arm_joint1"><command_interface name="position"/><state_interface name="position"/><state_interface name="velocity"/></joint>
-    <joint name="left_arm_joint2"><command_interface name="position"/><state_interface name="position"/><state_interface name="velocity"/></joint>
-    <joint name="left_arm_joint3"><command_interface name="position"/><state_interface name="position"/><state_interface name="velocity"/></joint>
-    <joint name="left_arm_joint4"><command_interface name="position"/><state_interface name="position"/><state_interface name="velocity"/></joint>
-    <joint name="left_arm_joint5"><command_interface name="position"/><state_interface name="position"/><state_interface name="velocity"/></joint>
-    <joint name="left_arm_joint6"><command_interface name="position"/><state_interface name="position"/><state_interface name="velocity"/></joint>
-    <joint name="left_arm_joint7"><command_interface name="position"/><state_interface name="position"/><state_interface name="velocity"/></joint>
-    <joint name="right_arm_joint1"><command_interface name="position"/><state_interface name="position"/><state_interface name="velocity"/></joint>
-    <joint name="right_arm_joint2"><command_interface name="position"/><state_interface name="position"/><state_interface name="velocity"/></joint>
-    <joint name="right_arm_joint3"><command_interface name="position"/><state_interface name="position"/><state_interface name="velocity"/></joint>
-    <joint name="right_arm_joint4"><command_interface name="position"/><state_interface name="position"/><state_interface name="velocity"/></joint>
-    <joint name="right_arm_joint5"><command_interface name="position"/><state_interface name="position"/><state_interface name="velocity"/></joint>
-    <joint name="right_arm_joint6"><command_interface name="position"/><state_interface name="position"/><state_interface name="velocity"/></joint>
-    <joint name="right_arm_joint7"><command_interface name="position"/><state_interface name="position"/><state_interface name="velocity"/></joint>
-    <joint name="head_joint1"><command_interface name="position"/><state_interface name="position"/><state_interface name="velocity"/></joint>
-    <joint name="head_joint2"><command_interface name="position"/><state_interface name="position"/><state_interface name="velocity"/></joint>
-    <!-- Gripper joints -->
-      <joint name="left_gripper_l1_joint">
-        <command_interface name="position"/>
-        <state_interface name="position">
-          <param name="initial_value">0.0</param>
-        </state_interface>
-        <state_interface name="velocity">
-          <param name="initial_value">0.0</param>
-        </state_interface>
-      </joint>
-      <joint name="left_gripper_l2_joint">
-        <command_interface name="position"/>
-        <state_interface name="position">
-          <param name="initial_value">0.0</param>
-        </state_interface>
-        <state_interface name="velocity">
-          <param name="initial_value">0.0</param>
-        </state_interface>
-      </joint>
-      <joint name="left_gripper_l3_joint">
-        <command_interface name="position"/>
-        <state_interface name="position">
-          <param name="initial_value">0.0</param>
-        </state_interface>
-        <state_interface name="velocity">
-          <param name="initial_value">0.0</param>
-        </state_interface>
-      </joint>
-      <joint name="left_gripper_r1_joint">
-        <command_interface name="position"/>
-        <state_interface name="position">
-          <param name="initial_value">0.0</param>
-        </state_interface>
-        <state_interface name="velocity">
-          <param name="initial_value">0.0</param>
-        </state_interface>
-      </joint>
-      <joint name="left_gripper_r2_joint">
-        <command_interface name="position"/>
-        <state_interface name="position">
-          <param name="initial_value">0.0</param>
-        </state_interface>
-        <state_interface name="velocity">
-          <param name="initial_value">0.0</param>
-        </state_interface>
-      </joint>
-      <joint name="left_gripper_r3_joint">
-        <command_interface name="position"/>
-        <state_interface name="position">
-          <param name="initial_value">0.0</param>
-        </state_interface>
-        <state_interface name="velocity">
-          <param name="initial_value">0.0</param>
-        </state_interface>
-      </joint>
-      <joint name="right_gripper_l1_joint">
-        <command_interface name="position"/>
-        <state_interface name="position">
-          <param name="initial_value">0.0</param>
-        </state_interface>
-        <state_interface name="velocity">
-          <param name="initial_value">0.0</param>
-        </state_interface>
-      </joint>
-      <joint name="right_gripper_l2_joint">
-        <command_interface name="position"/>
-        <state_interface name="position">
-          <param name="initial_value">0.0</param>
-        </state_interface>
-        <state_interface name="velocity">
-          <param name="initial_value">0.0</param>
-        </state_interface>
-      </joint>
-      <joint name="right_gripper_l3_joint">
-        <command_interface name="position"/>
-        <state_interface name="position">
-          <param name="initial_value">0.0</param>
-        </state_interface>
-        <state_interface name="velocity">
-          <param name="initial_value">0.0</param>
-        </state_interface>
-      </joint>
-      <joint name="right_gripper_r1_joint">
-        <command_interface name="position"/>
-        <state_interface name="position">
-          <param name="initial_value">0.0</param>
-        </state_interface>
-        <state_interface name="velocity">
-          <param name="initial_value">0.0</param>
-        </state_interface>
-      </joint>
-      <joint name="right_gripper_r2_joint">
-        <command_interface name="position"/>
-        <state_interface name="position">
-          <param name="initial_value">0.0</param>
-        </state_interface>
-        <state_interface name="velocity">
-          <param name="initial_value">0.0</param>
-        </state_interface>
-      </joint>
-      <joint name="right_gripper_r3_joint">
-        <command_interface name="position"/>
-        <state_interface name="position">
-          <param name="initial_value">0.0</param>
-        </state_interface>
-        <state_interface name="velocity">
-          <param name="initial_value">0.0</param>
-        </state_interface>
-      </joint>
+    <xacro:galbot_one_base_interfaces/>
+    <xacro:galbot_one_arm_interfaces name="left"/>
+    <xacro:galbot_one_arm_interfaces name="right"/>
+    <xacro:if value="${'$(arg type)' == 'gripper'}">
+      <xacro:galbot_one_gripper_interfaces name="left"/>
+      <xacro:galbot_one_gripper_interfaces name="right"/>
+    </xacro:if>
   </ros2_control>
   <xacro:arg name="gazebo" default="false"/>

Commit message: update readme and body visual

File: humanoid/Galbot/galbot_one_description/urdf/galbot_one.urdf (robot description, URDF)
Before this commit: robot galbot_one, 69 links, 68 joints
Joints:
- joint leg_joint: origin  -> rpy=1.57 0 0
- joint omni_chassis_leg_mount_joint: origin xyz=0.134 -0.087 0.13 rpy=1.5707963267948966 0 0 -> xyz=0.134 -0.087 0.13 rpy=0 0 0

File: humanoid/Galbot/galbot_one_description/xacro/component.xacro (robot description, xacro)
@@ -12,4 +12,6 @@
   <xacro:arg name="type" default="base"/>
   <xacro:arg name="enable_wheel_joints" default="true"/>
+  <!-- component-mode arm should not show flange mesh; gripper component shows flange together with gripper -->
+  <xacro:arg name="include_flange_mesh" default="false"/>
   <xacro:if value="${'$(arg type)' == 'base'}">
     <xacro:include filename="$(find galbot_one_description)/xacro/components/chassis.xacro"/>
@@ -48,4 +50,5 @@
       <child link="torso_left_arm_mount_link"/>
     </joint>
+    <!-- Component-mode arm: omit flange mesh so flange can be shown together with gripper -->
     <xacro:include filename="$(find galbot_one_description)/xacro/components/arm.xacro"/>
   </xacro:if>
@@ -53,7 +56,27 @@
     <link name="base_link"/>
     <!-- Component-mode gripper: single unprefixed instance (gripper_joint) -->
+    <!-- Add flange visual so flange is shown together with the gripper -->
+    <link name="flange_base_link">
+      <inertial>
+        <origin rpy="0 0 0" xyz="0.052829 -0.00096484 0.013285"/>
+        <mass value="0.25733"/>
+        <inertia ixx="0.0002175" ixy="-2.5433E-06" ixz="4.0586E-06" iyy="5.3894E-05" iyz="-1.8533E-06" izz="0.00025319"/>
+      </inertial>
+      <visual>
+        <geometry>
+          <mesh filename="file://$(find galbot_one_description)/meshes/flange/flange.glb"/>
+        </geometry>
+      </visual>
+    </link>
     <link name="flange_mount_link"/>
-    <joint name="base_to_flange_mount_joint" type="fixed">
+    <!-- Keep flange_mount_link pose unchanged (same as previous component setup) -->
+    <joint name="base_to_flange_base_joint" type="fixed">
+      <origin rpy="0 0 0" xyz="0 0 -0.006"/>
       <parent link="base_link"/>
+      <child link="flange_base_link"/>
+    </joint>
+    <joint name="flange_base_to_flange_mount_joint" type="fixed">
+      <origin rpy="0 0 0" xyz="0 0 0.006"/>
+      <parent link="flange_base_link"/>
       <child link="flange_mount_link"/>
     </joint>

File: humanoid/Galbot/galbot_one_description/xacro/components/arm.xacro (robot description, xacro)
@@ -1,4 +1,6 @@
 <?xml version="1.0" ?>
 <robot xmlns:xacro="http://www.ros.org/wiki/xacro">
+  <!-- Allow component launch to hide flange mesh while keeping TF frames/cameras -->
+  <xacro:arg name="include_flange_mesh" default="true"/>
   <joint name="right_arm_joint" type="fixed">
     <parent link="torso_right_arm_mount_link"/>
@@ -201,9 +203,11 @@
       <inertia ixx="0.0002175" ixy="-2.5433E-06" ixz="4.0586E-06" iyy="5.3894E-05" iyz="-1.8533E-06" izz="0.00025319"/>
     </inertial>
-    <visual>
-      <geometry>
-        <mesh filename="file://$(find galbot_one_description)/meshes/flange/flange.glb"/>
-      </geometry>
-    </visual>
+    <xacro:if value="${'$(arg include_flange_mesh)' == 'true'}">
+      <visual>
+        <geometry>
+          <mesh filename="file://$(find galbot_one_description)/meshes/flange/flange.glb"/>
+        </geometry>
+      </visual>
+    </xacro:if>
   </link>
   <link name="right_flange_mount_link"/>
@@ -365,5 +369,5 @@
     </visual>S
     <collision>
-      <origin rpy="0 0 0" xyz="0 -0.046 -0.09"/>
+      <origin rpy="0 0 0" xyz="0 -0.046 -0.154665"/>
       <geometry>
         <cylinder length="0.068650" radius="0.034983"/>
@@ -444,9 +448,11 @@
       <inertia ixx="0.0002175" ixy="-2.5433E-06" ixz="4.0586E-06" iyy="5.3894E-05" iyz="-1.8533E-06" izz="0.00025319"/>
     </inertial>
-    <visual>
-      <geometry>
-        <mesh filename="file://$(find galbot_one_description)/meshes/flange/flange.glb"/>
-      </geometry>
-    </visual>
+    <xacro:if value="${'$(arg include_flange_mesh)' == 'true'}">
+      <visual>
+        <geometry>
+          <mesh filename="file://$(find galbot_one_description)/meshes/flange/flange.glb"/>
+        </geometry>
+      </visual>
+    </xacro:if>
   </link>
   <link name="left_flange_mount_link"/>

File: humanoid/Galbot/galbot_one_description/xacro/components/body.xacro (robot description, xacro)
@@ -29,5 +29,5 @@
   <!-- omni_chassis_leg_mount_link and its joint come from chassis.xacro -->
   <joint name="leg_joint" type="fixed">
-    <origin  />
+    <origin rpy="1.57 0 0" />
     <parent link="omni_chassis_leg_mount_link"/>
     <child link="leg_base_link"/>

File: humanoid/Galbot/galbot_one_description/xacro/components/chassis.xacro (robot description, xacro)
@@ -30,5 +30,5 @@
     <link name="omni_chassis_leg_mount_link"/>
     <joint name="omni_chassis_leg_mount_joint" type="fixed">
-      <origin rpy="1.5707963267948966 0 0" xyz="0.134 -0.087 0.13"/>
+      <origin rpy="0 0 0" xyz="0.134 -0.087 0.13"/>
       <parent link="omni_chassis_base_link"/>
       <child link="omni_chassis_leg_mount_link"/>
