Commit message: change joint names

File: humanoid/Galbot/galbot_one_description/urdf/galbot_one.urdf (robot description, URDF)
Before this commit: robot galbot_one, 76 links, 75 joints
Joints:
- removed joint leg_joint
- removed joint leg_joint1
- removed joint leg_joint2
- removed joint leg_joint3
- removed joint leg_joint4
- added joint body_joint: type fixed, parent omni_chassis_leg_mount_link, child leg_base_link, origin rpy=1.5707963267948966 0 0
- added joint body_joint1: type revolute, parent leg_base_link, child leg_link1, origin xyz=0 0 -0.087 rpy=-3.141592653589793 0 2.756573021, axis 0 0 1, limit lower=0 upper=0.994837674 effort=169 velocity=2.3
- added joint body_joint2: type revolute, parent leg_link1, child leg_link2, origin xyz=0.45 0 0 rpy=-3.141592653589793 0 2.756573021, axis 0 0 1, limit lower=0 upper=3.141592653589793 effort=169 velocity=2.3
- added joint body_joint3: type revolute, parent leg_link2, child leg_link3, origin xyz=0.39 0 0 rpy=-3.141592653589793 0 -3.141592653589793, axis 0 0 1, limit lower=0 upper=2.356194490192345 effort=84 velocity=2.83
- added joint body_joint4: type revolute, parent leg_link3, child leg_link4, origin rpy=1.5707963267948966 0 -3.141592653589793, axis 0 0 1, limit lower=-1.5707963267948966 upper=1.5707963267948966 effort=30 velocity=3.56

File: humanoid/Galbot/galbot_one_description/xacro/components/body.xacro (robot description, xacro)
@@ -37,5 +37,5 @@
 	</link>
 	<!-- omni_chassis_leg_mount_link and its joint come from chassis.xacro -->
-	<joint name="leg_joint" type="fixed">
+	<joint name="body_joint" type="fixed">
 		<origin rpy="${PI/2} 0 0"/>
 		<parent link="omni_chassis_leg_mount_link"/>
@@ -80,5 +80,5 @@
 		</xacro:if>
 	</link>
-	<joint name="leg_joint1" type="revolute">
+	<joint name="body_joint1" type="revolute">
 		<origin rpy="-${PI} 0 2.756573021" xyz="0 0 -0.087"/>
 		<parent link="leg_base_link"/>
@@ -106,5 +106,5 @@
 		</xacro:if>
 	</link>
-	<joint name="leg_joint2" type="revolute">
+	<joint name="body_joint2" type="revolute">
 		<origin rpy="-${PI} 0 2.756573021" xyz="0.45 0 0"/>
 		<parent link="leg_link1"/>
@@ -132,5 +132,5 @@
 		</xacro:if>
 	</link>
-	<joint name="leg_joint3" type="revolute">
+	<joint name="body_joint3" type="revolute">
 		<origin rpy="-${PI} 0 -${PI}" xyz="0.39 0 0"/>
 		<parent link="leg_link2"/>
@@ -158,5 +158,5 @@
 		</xacro:if>
 	</link>
-	<joint name="leg_joint4" type="revolute">
+	<joint name="body_joint4" type="revolute">
 		<origin rpy="${PI/2} 0 -${PI}"/>
 		<parent link="leg_link3"/>

File: humanoid/Galbot/galbot_one_description/xacro/ros2_control/galbot_one_base_interfaces.xacro (robot description, xacro)
@@ -3,20 +3,20 @@
 	<xacro:macro name="galbot_one_base_interfaces">
 		<!-- Leg joints -->
-		<joint name="leg_joint1">
+		<joint name="body_joint1">
 			<command_interface name="position"/>
 			<state_interface name="position"/>
 			<state_interface name="velocity"/>
 		</joint>
-		<joint name="leg_joint2">
+		<joint name="body_joint2">
 			<command_interface name="position"/>
 			<state_interface name="position"/>
 			<state_interface name="velocity"/>
 		</joint>
-		<joint name="leg_joint3">
+		<joint name="body_joint3">
 			<command_interface name="position"/>
 			<state_interface name="position"/>
 			<state_interface name="velocity"/>
 		</joint>
-		<joint name="leg_joint4">
+		<joint name="body_joint4">
 			<command_interface name="position"/>
 			<state_interface name="position"/>
