Commit message: g1 mock components

File: humanoid/Unitree/unitree_g1_description/urdf/unitree_g1.urdf (robot description, URDF)
Before this commit: robot g1_29dof, 40 links, 39 joints
Links:
- removed link base_footprint
Joints:
- removed joint base_footprint_joint
- removed joint base_joint
- added joint base_link_joint: type fixed, parent base_link, child pelvis

File: humanoid/Unitree/unitree_g1_description/xacro/body.xacro (robot description, xacro)
@@ -6,4 +6,9 @@
 		Includes: pelvis, torso, head, sensors, and logo
 		-->
+		<link name="base_link"/>
+		<joint name="base_link_joint" type="fixed">
+			<parent link="base_link"/>
+			<child link="pelvis"/>
+		</joint>
 		<!-- Pelvis Link -->
 		<link name="pelvis">
@@ -86,10 +91,4 @@
 			<limit lower="-0.52" upper="0.52" effort="35" velocity="30"/>
 		</joint>
-		<!-- Base Link -->
-		<link name="base_link"/>
-		<joint name="base_joint" type="fixed">
-			<parent link="torso_link"/>
-			<child link="base_link"/>
-		</joint>
 		<!-- Logo -->
 		<link name="logo_link">

Commit message: collision avoidance for g1

File: humanoid/Unitree/unitree_g1_description/urdf/unitree_g1.urdf (robot description, URDF)
Before this commit: robot g1_29dof, 39 links, 38 joints
Links:
- link left_elbow_link: geometry collision cylinder length=0.06 radius=0.03; visual mesh filename=package://unitree_g1_description/meshes/arm/elbow.obj scale=1 1 1
- link left_hand_base: geometry collision box size=0.12 0.05 0.1; visual mesh filename=package://unitree_g1_description/meshes/arm/hand.obj scale=1 1 1
- link left_shoulder_yaw_link: geometry collision cylinder length=0.06 radius=0.03; collision cylinder length=0.08 radius=0.03
- link left_wrist_pitch_link: geometry collision cylinder length=0.05 radius=0.03; collision cylinder length=0.06 radius=0.03
- link left_wrist_roll_link: geometry visual mesh filename=package://unitree_g1_description/meshes/arm/wrist_roll.obj
- link left_wrist_yaw_link: geometry visual mesh filename=package://unitree_g1_description/meshes/arm/wrist_yaw.obj
- link right_elbow_link: geometry collision cylinder length=0.06 radius=0.03; visual mesh filename=package://unitree_g1_description/meshes/arm/elbow.obj scale=1 -1 1
- link right_hand_base: geometry collision box size=0.12 0.05 0.1; visual mesh filename=package://unitree_g1_description/meshes/arm/hand.obj scale=1 -1 1
- link right_shoulder_yaw_link: geometry collision cylinder length=0.06 radius=0.03; collision cylinder length=0.08 radius=0.03
- link right_wrist_pitch_link: geometry collision cylinder length=0.05 radius=0.03; collision cylinder length=0.06 radius=0.03
- link right_wrist_roll_link: geometry visual mesh filename=package://unitree_g1_description/meshes/arm/wrist_roll.obj
- link right_wrist_yaw_link: geometry visual mesh filename=package://unitree_g1_description/meshes/arm/wrist_yaw.obj
- link torso_link: geometry collision box size=0.12 0.15 0.05; collision box size=0.12 0.2 0.2

File: humanoid/Unitree/unitree_g1_description/xacro/arm.xacro (robot description, xacro)
@@ -85,7 +85,13 @@
 			</visual>
 			<collision>
-				<geometry>
-					<mesh filename="file://$(find unitree_g1_description)/meshes/arm/shoulder_yaw.obj"
-								scale="1 ${direction} 1"/>
+				<origin xyz="0 0 -0.02"/>
+				<geometry>
+					<cylinder radius="0.03" length="0.08"/>
+				</geometry>
+			</collision>
+			<collision>
+				<origin xyz="0.01 ${direction*-0.01} -0.08" rpy="${PI/2.0} 0 0"/>
+				<geometry>
+					<cylinder radius="0.03" length="0.06"/>
 				</geometry>
 			</collision>
@@ -114,7 +120,7 @@
 			</visual>
 			<collision>
-				<geometry>
-					<mesh filename="file://$(find unitree_g1_description)/meshes/arm/elbow.obj"
-								scale="1 ${direction} 1"/>
+				<origin xyz="0.07 0 -0.01" rpy="0 ${PI/2.0} 0"/>
+				<geometry>
+					<cylinder radius="0.03" length="0.06"/>
 				</geometry>
 			</collision>
@@ -142,9 +148,4 @@
 				</geometry>
 			</visual>
-			<collision>
-				<geometry>
-					<mesh filename="file://$(find unitree_g1_description)/meshes/arm/wrist_roll.obj"/>
-				</geometry>
-			</collision>
 		</link>
 		<!-- Wrist Roll Joint -->
@@ -171,6 +172,13 @@
 			</visual>
 			<collision>
-				<geometry>
-					<mesh filename="file://$(find unitree_g1_description)/meshes/arm/wrist_pitch.obj"/>
+				<origin rpy="${PI/2.0} 0 0"/>
+				<geometry>
+					<cylinder radius="0.03" length="0.06"/>
+				</geometry>
+			</collision>
+			<collision>
+				<origin xyz="0.06 0 0"/>
+				<geometry>
+					<cylinder radius="0.03" length="0.05"/>
 				</geometry>
 			</collision>
@@ -198,9 +206,4 @@
 				</geometry>
 			</visual>
-			<collision>
-				<geometry>
-					<mesh filename="file://$(find unitree_g1_description)/meshes/arm/wrist_yaw.obj"/>
-				</geometry>
-			</collision>
 		</link>
 		<!-- Wrist Yaw Joint -->

File: humanoid/Unitree/unitree_g1_description/xacro/body.xacro (robot description, xacro)
@@ -79,6 +79,13 @@
 			</visual>
 			<collision>
+				<origin xyz="0.008 0 0.05"/>
 				<geometry>
-					<mesh filename="file://$(find unitree_g1_description)/meshes/body/torso.obj"/>
+					<box size="0.12 0.15 0.15"/>
+				</geometry>
+			</collision>
+			<collision>
+				<origin xyz="0.008 0 0.2"/>
+				<geometry>
+					<box size="0.12 0.2 0.15"/>
 				</geometry>
 			</collision>

File: humanoid/Unitree/unitree_g1_description/xacro/hand.xacro (robot description, xacro)
@@ -23,4 +23,10 @@
 				</geometry>
 			</visual>
+			<collision>
+				<origin xyz="0.07 ${direction*-0.02} 0"/>
+				<geometry>
+					<box size="0.12 0.05 0.1"/>
+				</geometry>
+			</collision>
 		</link>
 	</xacro:macro>
