Commit message: fix joint grouping to enable movej

File: humanoid/Unitree/unitree_g1_description/urdf/unitree_g1.urdf (robot description, URDF)
Before this commit: robot g1_29dof, 39 links, 38 joints
Joints:
- removed joint left_elbow_joint
- removed joint left_shoulder_pitch_joint
- removed joint left_shoulder_roll_joint
- removed joint left_shoulder_yaw_joint
- removed joint left_wrist_pitch_joint
- removed joint left_wrist_roll_joint
- removed joint left_wrist_yaw_joint
- removed joint right_elbow_joint
- removed joint right_shoulder_pitch_joint
- removed joint right_shoulder_roll_joint
- removed joint right_shoulder_yaw_joint
- removed joint right_wrist_pitch_joint
- removed joint right_wrist_roll_joint
- removed joint right_wrist_yaw_joint
- removed joint waist_pitch_joint
- removed joint waist_roll_joint
- removed joint waist_yaw_joint
- added joint body_joint1: type revolute, parent pelvis, child waist_yaw_link, axis 0 0 1, limit lower=-2.618 upper=2.618 effort=88 velocity=32
- added joint body_joint2: type revolute, parent waist_yaw_link, child waist_roll_link, origin xyz=-0.0039635 0 0.044, axis 1 0 0, limit lower=-0.52 upper=0.52 effort=35 velocity=30
- added joint body_joint3: type revolute, parent waist_roll_link, child torso_link, axis 0 1 0, limit lower=-0.52 upper=0.52 effort=35 velocity=30
- added joint left_joint1: type revolute, parent torso_link, child left_shoulder_pitch_link, origin xyz=0.0039563 0.10022 0.24778 rpy=0.27931 5.4949E-05 -0.00019159, axis 0 1 0, limit lower=-3.0892 upper=2.6704 effort=25 velocity=37
- added joint left_joint2: type revolute, parent left_shoulder_pitch_link, child left_shoulder_roll_link, origin xyz=0 0.038 -0.013831 rpy=-0.27925 0 0, axis 1 0 0, limit lower=-1.5882 upper=2.2515 effort=25 velocity=37
- added joint left_joint3: type revolute, parent left_shoulder_roll_link, child left_shoulder_yaw_link, origin xyz=0 0.00624 -0.1032, axis 0 0 1, limit lower=-2.618 upper=2.618 effort=25 velocity=37
- added joint left_joint4: type revolute, parent left_shoulder_yaw_link, child left_elbow_link, origin xyz=0.015783 0 -0.080518, axis 0 1 0, limit lower=-1.0472 upper=2.0944 effort=25 velocity=37
- added joint left_joint5: type revolute, parent left_elbow_link, child left_wrist_roll_link, origin xyz=0.100 0.00188791 -0.010, axis 1 0 0, limit lower=-1.972222054 upper=1.972222054 effort=25 velocity=37
- added joint left_joint6: type revolute, parent left_wrist_roll_link, child left_wrist_pitch_link, origin xyz=0.038 0 0, axis 0 1 0, limit lower=-1.614429558 upper=1.614429558 effort=5 velocity=22
- added joint left_joint7: type revolute, parent left_wrist_pitch_link, child left_wrist_yaw_link, origin xyz=0.046 0 0, axis 0 0 1, limit lower=-1.614429558 upper=1.614429558 effort=5 velocity=22
- added joint right_joint1: type revolute, parent torso_link, child right_shoulder_pitch_link, origin xyz=0.0039563 -0.10022 0.24778 rpy=-0.27931 5.4949E-05 0.00019159, axis 0 1 0, limit lower=-3.0892 upper=2.6704 effort=25 velocity=37
- added joint right_joint2: type revolute, parent right_shoulder_pitch_link, child right_shoulder_roll_link, origin xyz=0 -0.038 -0.013831 rpy=0.27925 0 0, axis 1 0 0, limit lower=-2.2515 upper=1.5882 effort=25 velocity=37
- added joint right_joint3: type revolute, parent right_shoulder_roll_link, child right_shoulder_yaw_link, origin xyz=0 -0.00624 -0.1032, axis 0 0 1, limit lower=-2.618 upper=2.618 effort=25 velocity=37
- added joint right_joint4: type revolute, parent right_shoulder_yaw_link, child right_elbow_link, origin xyz=0.015783 0 -0.080518, axis 0 1 0, limit lower=-1.0472 upper=2.0944 effort=25 velocity=37
- added joint right_joint5: type revolute, parent right_elbow_link, child right_wrist_roll_link, origin xyz=0.100 -0.00188791 -0.010, axis 1 0 0, limit lower=-1.972222054 upper=1.972222054 effort=25 velocity=37
- added joint right_joint6: type revolute, parent right_wrist_roll_link, child right_wrist_pitch_link, origin xyz=0.038 0 0, axis 0 1 0, limit lower=-1.614429558 upper=1.614429558 effort=5 velocity=22
- added joint right_joint7: type revolute, parent right_wrist_pitch_link, child right_wrist_yaw_link, origin xyz=0.046 0 0, axis 0 0 1, limit lower=-1.614429558 upper=1.614429558 effort=5 velocity=22

File: humanoid/Unitree/unitree_g1_description/xacro/arm.xacro (robot description, xacro)
@@ -31,6 +31,6 @@
 			</collision>
 		</link>
-		<!-- Shoulder Pitch Joint -->
-		<joint name="${prefix}shoulder_pitch_joint" type="revolute">
+		<!-- Shoulder Pitch Joint -> left/right_joint1 -->
+		<joint name="${name}_joint1" type="revolute">
 			<origin xyz="0.0039563 ${direction*0.10022} 0.24778"
 							rpy="${direction*0.27931} 5.4949E-05 ${direction*-0.00019159}"/>
@@ -61,6 +61,6 @@
 			</collision>
 		</link>
-		<!-- Shoulder Roll Joint -->
-		<joint name="${prefix}shoulder_roll_joint" type="revolute">
+		<!-- Shoulder Roll Joint -> left/right_joint2 -->
+		<joint name="${name}_joint2" type="revolute">
 			<origin xyz="0 ${direction*0.038} -0.013831" rpy="${direction*-0.27925} 0 0"/>
 			<parent link="${prefix}shoulder_pitch_link"/>
@@ -97,6 +97,6 @@
 			</collision>
 		</link>
-		<!-- Shoulder Yaw Joint -->
-		<joint name="${prefix}shoulder_yaw_joint" type="revolute">
+		<!-- Shoulder Yaw Joint -> left/right_joint3 -->
+		<joint name="${name}_joint3" type="revolute">
 			<origin xyz="0 ${direction*0.00624} -0.1032"/>
 			<parent link="${prefix}shoulder_roll_link"/>
@@ -126,6 +126,6 @@
 			</collision>
 		</link>
-		<!-- Elbow Joint -->
-		<joint name="${prefix}elbow_joint" type="revolute">
+		<!-- Elbow Joint -> left/right_joint4 -->
+		<joint name="${name}_joint4" type="revolute">
 			<origin xyz="0.015783 0 -0.080518"/>
 			<parent link="${prefix}shoulder_yaw_link"/>
@@ -149,6 +149,6 @@
 			</visual>
 		</link>
-		<!-- Wrist Roll Joint -->
-		<joint name="${prefix}wrist_roll_joint" type="revolute">
+		<!-- Wrist Roll Joint -> left/right_joint5 -->
+		<joint name="${name}_joint5" type="revolute">
 			<origin xyz="0.100 ${direction*0.00188791} -0.010"/>
 			<axis xyz="1 0 0"/>
@@ -184,6 +184,6 @@
 			</collision>
 		</link>
-		<!-- Wrist Pitch Joint -->
-		<joint name="${prefix}wrist_pitch_joint" type="revolute">
+		<!-- Wrist Pitch Joint -> left/right_joint6 -->
+		<joint name="${name}_joint6" type="revolute">
 			<origin xyz="0.038 0 0"/>
 			<axis xyz="0 1 0"/>
@@ -207,6 +207,6 @@
 			</visual>
 		</link>
-		<!-- Wrist Yaw Joint -->
-		<joint name="${prefix}wrist_yaw_joint" type="revolute">
+		<!-- Wrist Yaw Joint -> left/right_joint7 -->
+		<joint name="${name}_joint7" type="revolute">
 			<origin xyz="0.046 0 0"/>
 			<axis xyz="0 0 1"/>

File: humanoid/Unitree/unitree_g1_description/xacro/body.xacro (robot description, xacro)
@@ -38,6 +38,6 @@
 			</visual>
 		</link>
-		<!-- Waist Yaw Joint -->
-		<joint name="waist_yaw_joint" type="revolute">
+		<!-- Waist Yaw Joint -> body_joint1 -->
+		<joint name="body_joint1" type="revolute">
 			<parent link="pelvis"/>
 			<child link="waist_yaw_link"/>
@@ -58,6 +58,6 @@
 			</visual>
 		</link>
-		<!-- Waist Roll Joint -->
-		<joint name="waist_roll_joint" type="revolute">
+		<!-- Waist Roll Joint -> body_joint2 -->
+		<joint name="body_joint2" type="revolute">
 			<origin xyz="-0.0039635 0 0.044"/>
 			<parent link="waist_yaw_link"/>
@@ -91,6 +91,6 @@
 			</collision>
 		</link>
-		<!-- Waist Pitch Joint -->
-		<joint name="waist_pitch_joint" type="revolute">
+		<!-- Waist Pitch Joint -> body_joint3 -->
+		<joint name="body_joint3" type="revolute">
 			<parent link="waist_roll_link"/>
 			<child link="torso_link"/>

File: humanoid/Unitree/unitree_g1_description/xacro/ros2_control/ros2_control.xacro (robot description, xacro)
@@ -154,168 +154,168 @@
         <state_interface name="effort"/>
       </joint>
-      <!-- Waist Joints (3 DOF) -->
-      <joint name="waist_yaw_joint">
-        <command_interface name="position"/>
-        <command_interface name="velocity"/>
-        <command_interface name="effort"/>
-        <command_interface name="kp"/>
-        <command_interface name="kd"/>
-        <state_interface name="position"/>
-        <state_interface name="velocity"/>
-        <state_interface name="effort"/>
-      </joint>
-      <joint name="waist_roll_joint">
-        <command_interface name="position"/>
-        <command_interface name="velocity"/>
-        <command_interface name="effort"/>
-        <command_interface name="kp"/>
-        <command_interface name="kd"/>
-        <state_interface name="position"/>
-        <state_interface name="velocity"/>
-        <state_interface name="effort"/>
-      </joint>
-      <joint name="waist_pitch_joint">
-        <command_interface name="position"/>
-        <command_interface name="velocity"/>
-        <command_interface name="effort"/>
-        <command_interface name="kp"/>
-        <command_interface name="kd"/>
-        <state_interface name="position"/>
-        <state_interface name="velocity"/>
-        <state_interface name="effort"/>
-      </joint>
-      <!-- Left Arm Joints (7 DOF) -->
-      <joint name="left_shoulder_pitch_joint">
-        <command_interface name="position"/>
-        <command_interface name="velocity"/>
-        <command_interface name="effort"/>
-        <command_interface name="kp"/>
-        <command_interface name="kd"/>
-        <state_interface name="position"/>
-        <state_interface name="velocity"/>
-        <state_interface name="effort"/>
-      </joint>
-      <joint name="left_shoulder_roll_joint">
-        <command_interface name="position"/>
-        <command_interface name="velocity"/>
-        <command_interface name="effort"/>
-        <command_interface name="kp"/>
-        <command_interface name="kd"/>
-        <state_interface name="position"/>
-        <state_interface name="velocity"/>
-        <state_interface name="effort"/>
-      </joint>
-      <joint name="left_shoulder_yaw_joint">
-        <command_interface name="position"/>
-        <command_interface name="velocity"/>
-        <command_interface name="effort"/>
-        <command_interface name="kp"/>
-        <command_interface name="kd"/>
-        <state_interface name="position"/>
-        <state_interface name="velocity"/>
-        <state_interface name="effort"/>
-      </joint>
-      <joint name="left_elbow_joint">
-        <command_interface name="position"/>
-        <command_interface name="velocity"/>
-        <command_interface name="effort"/>
-        <command_interface name="kp"/>
-        <command_interface name="kd"/>
-        <state_interface name="position"/>
-        <state_interface name="velocity"/>
-        <state_interface name="effort"/>
-      </joint>
-      <joint name="left_wrist_roll_joint">
-        <command_interface name="position"/>
-        <command_interface name="velocity"/>
-        <command_interface name="effort"/>
-        <command_interface name="kp"/>
-        <command_interface name="kd"/>
-        <state_interface name="position"/>
-        <state_interface name="velocity"/>
-        <state_interface name="effort"/>
-      </joint>
-      <joint name="left_wrist_pitch_joint">
-        <command_interface name="position"/>
-        <command_interface name="velocity"/>
-        <command_interface name="effort"/>
-        <command_interface name="kp"/>
-        <command_interface name="kd"/>
-        <state_interface name="position"/>
-        <state_interface name="velocity"/>
-        <state_interface name="effort"/>
-      </joint>
-      <joint name="left_wrist_yaw_joint">
-        <command_interface name="position"/>
-        <command_interface name="velocity"/>
-        <command_interface name="effort"/>
-        <command_interface name="kp"/>
-        <command_interface name="kd"/>
-        <state_interface name="position"/>
-        <state_interface name="velocity"/>
-        <state_interface name="effort"/>
-      </joint>
-      <!-- Right Arm Joints (7 DOF) -->
-      <joint name="right_shoulder_pitch_joint">
-        <command_interface name="position"/>
-        <command_interface name="velocity"/>
-        <command_interface name="effort"/>
-        <command_interface name="kp"/>
-        <command_interface name="kd"/>
-        <state_interface name="position"/>
-        <state_interface name="velocity"/>
-        <state_interface name="effort"/>
-      </joint>
-      <joint name="right_shoulder_roll_joint">
-        <command_interface name="position"/>
-        <command_interface name="velocity"/>
-        <command_interface name="effort"/>
-        <command_interface name="kp"/>
-        <command_interface name="kd"/>
-        <state_interface name="position"/>
-        <state_interface name="velocity"/>
-        <state_interface name="effort"/>
-      </joint>
-      <joint name="right_shoulder_yaw_joint">
-        <command_interface name="position"/>
-        <command_interface name="velocity"/>
-        <command_interface name="effort"/>
-        <command_interface name="kp"/>
-        <command_interface name="kd"/>
-        <state_interface name="position"/>
-        <state_interface name="velocity"/>
-        <state_interface name="effort"/>
-      </joint>
-      <joint name="right_elbow_joint">
-        <command_interface name="position"/>
-        <command_interface name="velocity"/>
-        <command_interface name="effort"/>
-        <command_interface name="kp"/>
-        <command_interface name="kd"/>
-        <state_interface name="position"/>
-        <state_interface name="velocity"/>
-        <state_interface name="effort"/>
-      </joint>
-      <joint name="right_wrist_roll_joint">
-        <command_interface name="position"/>
-        <command_interface name="velocity"/>
-        <command_interface name="effort"/>
-        <command_interface name="kp"/>
-        <command_interface name="kd"/>
-        <state_interface name="position"/>
-        <state_interface name="velocity"/>
-        <state_interface name="effort"/>
-      </joint>
-      <joint name="right_wrist_pitch_joint">
-        <command_interface name="position"/>
-        <command_interface name="velocity"/>
-        <command_interface name="effort"/>
-        <command_interface name="kp"/>
-        <command_interface name="kd"/>
-        <state_interface name="position"/>
-        <state_interface name="velocity"/>
-        <state_interface name="effort"/>
-      </joint>
-      <joint name="right_wrist_yaw_joint">
+      <!-- Waist Joints (3 DOF) -> body joints -->
+      <joint name="body_joint1">
+        <command_interface name="position"/>
+        <command_interface name="velocity"/>
+        <command_interface name="effort"/>
+        <command_interface name="kp"/>
+        <command_interface name="kd"/>
+        <state_interface name="position"/>
+        <state_interface name="velocity"/>
+        <state_interface name="effort"/>
+      </joint>
+      <joint name="body_joint2">
+        <command_interface name="position"/>
+        <command_interface name="velocity"/>
+        <command_interface name="effort"/>
+        <command_interface name="kp"/>
+        <command_interface name="kd"/>
+        <state_interface name="position"/>
+        <state_interface name="velocity"/>
+        <state_interface name="effort"/>
+      </joint>
+      <joint name="body_joint3">
+        <command_interface name="position"/>
+        <command_interface name="velocity"/>
+        <command_interface name="effort"/>
+        <command_interface name="kp"/>
+        <command_interface name="kd"/>
+        <state_interface name="position"/>
+        <state_interface name="velocity"/>
+        <state_interface name="effort"/>
+      </joint>
+      <!-- Left Arm Joints (7 DOF) -> left_joint1~7 -->
+      <joint name="left_joint1">
+        <command_interface name="position"/>
+        <command_interface name="velocity"/>
+        <command_interface name="effort"/>
+        <command_interface name="kp"/>
+        <command_interface name="kd"/>
+        <state_interface name="position"/>
+        <state_interface name="velocity"/>
+        <state_interface name="effort"/>
+      </joint>
+      <joint name="left_joint2">
+        <command_interface name="position"/>
+        <command_interface name="velocity"/>
+        <command_interface name="effort"/>
+        <command_interface name="kp"/>
+        <command_interface name="kd"/>
+        <state_interface name="position"/>
+        <state_interface name="velocity"/>
+        <state_interface name="effort"/>
+      </joint>
+      <joint name="left_joint3">
+        <command_interface name="position"/>
+        <command_interface name="velocity"/>
+        <command_interface name="effort"/>
+        <command_interface name="kp"/>
+        <command_interface name="kd"/>
+        <state_interface name="position"/>
+        <state_interface name="velocity"/>
+        <state_interface name="effort"/>
+      </joint>
+      <joint name="left_joint4">
+        <command_interface name="position"/>
+        <command_interface name="velocity"/>
+        <command_interface name="effort"/>
+        <command_interface name="kp"/>
+        <command_interface name="kd"/>
+        <state_interface name="position"/>
+        <state_interface name="velocity"/>
+        <state_interface name="effort"/>
+      </joint>
+      <joint name="left_joint5">
+        <command_interface name="position"/>
+        <command_interface name="velocity"/>
+        <command_interface name="effort"/>
+        <command_interface name="kp"/>
+        <command_interface name="kd"/>
+        <state_interface name="position"/>
+        <state_interface name="velocity"/>
+        <state_interface name="effort"/>
+      </joint>
+      <joint name="left_joint6">
+        <command_interface name="position"/>
+        <command_interface name="velocity"/>
+        <command_interface name="effort"/>
+        <command_interface name="kp"/>
+        <command_interface name="kd"/>
+        <state_interface name="position"/>
+        <state_interface name="velocity"/>
+        <state_interface name="effort"/>
+      </joint>
+      <joint name="left_joint7">
+        <command_interface name="position"/>
+        <command_interface name="velocity"/>
+        <command_interface name="effort"/>
+        <command_interface name="kp"/>
+        <command_interface name="kd"/>
+        <state_interface name="position"/>
+        <state_interface name="velocity"/>
+        <state_interface name="effort"/>
+      </joint>
+      <!-- Right Arm Joints (7 DOF) -> right_joint1~7 -->
+      <joint name="right_joint1">
+        <command_interface name="position"/>
+        <command_interface name="velocity"/>
+        <command_interface name="effort"/>
+        <command_interface name="kp"/>
+        <command_interface name="kd"/>
+        <state_interface name="position"/>
+        <state_interface name="velocity"/>
+        <state_interface name="effort"/>
+      </joint>
+      <joint name="right_joint2">
+        <command_interface name="position"/>
+        <command_interface name="velocity"/>
+        <command_interface name="effort"/>
+        <command_interface name="kp"/>
+        <command_interface name="kd"/>
+        <state_interface name="position"/>
+        <state_interface name="velocity"/>
+        <state_interface name="effort"/>
+      </joint>
+      <joint name="right_joint3">
+        <command_interface name="position"/>
+        <command_interface name="velocity"/>
+        <command_interface name="effort"/>
+        <command_interface name="kp"/>
+        <command_interface name="kd"/>
+        <state_interface name="position"/>
+        <state_interface name="velocity"/>
+        <state_interface name="effort"/>
+      </joint>
+      <joint name="right_joint4">
+        <command_interface name="position"/>
+        <command_interface name="velocity"/>
+        <command_interface name="effort"/>
+        <command_interface name="kp"/>
+        <command_interface name="kd"/>
+        <state_interface name="position"/>
+        <state_interface name="velocity"/>
+        <state_interface name="effort"/>
+      </joint>
+      <joint name="right_joint5">
+        <command_interface name="position"/>
+        <command_interface name="velocity"/>
+        <command_interface name="effort"/>
+        <command_interface name="kp"/>
+        <command_interface name="kd"/>
+        <state_interface name="position"/>
+        <state_interface name="velocity"/>
+        <state_interface name="effort"/>
+      </joint>
+      <joint name="right_joint6">
+        <command_interface name="position"/>
+        <command_interface name="velocity"/>
+        <command_interface name="effort"/>
+        <command_interface name="kp"/>
+        <command_interface name="kd"/>
+        <state_interface name="position"/>
+        <state_interface name="velocity"/>
+        <state_interface name="effort"/>
+      </joint>
+      <joint name="right_joint7">
         <command_interface name="position"/>
         <command_interface name="velocity"/>
