Commit message: modify unitree urdf

File: humanoid/Unitree/unitree_g1_description/urdf/unitree_g1.urdf (robot description, URDF)
Before this commit: robot g1_29dof, 39 links, 38 joints
Links:
- removed link left_ankle_pitch_link
- removed link left_ankle_roll_link
- removed link left_hip_pitch_link
- removed link left_hip_roll_link
- removed link left_hip_yaw_link
- removed link left_knee_link
- removed link right_ankle_pitch_link
- removed link right_ankle_roll_link
- removed link right_hip_pitch_link
- removed link right_hip_roll_link
- removed link right_hip_yaw_link
- removed link right_knee_link
- added link one_ankle_pitch_link, mass 0.074; collision mesh filename=file:///home/lina/ros2_ws/install/unitree_g1_description/sh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; visual mesh filename=file:///home/lina/ros2_ws/install/unitree_g1_description/sh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
- added link one_ankle_roll_link, mass 0.608; collision sphere radius=0.005; collision sphere radius=0.005
- added link one_hip_pitch_link, mass 1.35; collision mesh filename=file:///home/lina/ros2_ws/install/unitree_g1_description/sh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 scale=1 1 1; visual mesh filename=file:///home/lina/ros2_ws/install/unitree_g1_description/sh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 scale=1 1 1
- added link one_hip_roll_link, mass 1.52; collision mesh filename=file:///home/lina/ros2_ws/install/unitree_g1_description/sh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; visual mesh filename=file:///home/lina/ros2_ws/install/unitree_g1_description/sh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
- added link one_hip_yaw_link, mass 1.702; collision mesh filename=file:///home/lina/ros2_ws/install/unitree_g1_description/sh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 scale=1 1 1; visual mesh filename=file:///home/lina/ros2_ws/install/unitree_g1_description/sh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 scale=1 1 1
- added link one_knee_link, mass 1.932; collision mesh filename=file:///home/lina/ros2_ws/install/unitree_g1_description/sh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 scale=1 1 1; visual mesh filename=file:///home/lina/ros2_ws/install/unitree_g1_description/sh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 scale=1 1 1
- added link two_ankle_pitch_link, mass 0.074; collision mesh filename=file:///home/lina/ros2_ws/install/unitree_g1_description/sh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; visual mesh filename=file:///home/lina/ros2_ws/install/unitree_g1_description/sh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
- added link two_ankle_roll_link, mass 0.608; collision sphere radius=0.005; collision sphere radius=0.005
- added link two_hip_pitch_link, mass 1.35; collision mesh filename=file:///home/lina/ros2_ws/install/unitree_g1_description/sh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 scale=1 -1 1; visual mesh filename=file:///home/lina/ros2_ws/install/unitree_g1_description/sh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 scale=1 -1 1
- added link two_hip_roll_link, mass 1.52; collision mesh filename=file:///home/lina/ros2_ws/install/unitree_g1_description/sh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; visual mesh filename=file:///home/lina/ros2_ws/install/unitree_g1_description/sh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
- added link two_hip_yaw_link, mass 1.702; collision mesh filename=file:///home/lina/ros2_ws/install/unitree_g1_description/sh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 scale=1 -1 1; visual mesh filename=file:///home/lina/ros2_ws/install/unitree_g1_description/sh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 scale=1 -1 1
- added link two_knee_link, mass 1.932; collision mesh filename=file:///home/lina/ros2_ws/install/unitree_g1_description/sh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 scale=1 -1 1; visual mesh filename=file:///home/lina/ros2_ws/install/unitree_g1_description/sh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 scale=1 -1 1
- link head_link: geometry collision mesh filename=file:///home/lina/ros2_ws/install/unitree_g1_description/sh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; visual mesh filename=file:///home/lina/ros2_ws/install/unitree_g1_description/sh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
- link left_elbow_link: geometry collision cylinder length=0.06 radius=0.03; visual mesh filename=file:///home/lina/ros2_ws/install/unitree_g1_description/sh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 scale=1 1 1
- link left_hand_base: geometry collision box size=0.12 0.05 0.1; visual mesh filename=file:///home/lina/ros2_ws/install/unitree_g1_description/sh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 scale=1 1 1
- link left_shoulder_pitch_link: geometry collision cylinder length=0.05 radius=0.03; visual mesh filename=file:///home/lina/ros2_ws/install/unitree_g1_description/sh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 scale=1 1 1
- link left_shoulder_roll_link: geometry collision cylinder length=0.03 radius=0.03; visual mesh filename=file:///home/lina/ros2_ws/install/unitree_g1_description/sh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 scale=1 1 1
- link left_shoulder_yaw_link: geometry collision cylinder length=0.06 radius=0.03; collision cylinder length=0.08 radius=0.03
- link left_wrist_pitch_link: geometry collision cylinder length=0.05 radius=0.03; collision cylinder length=0.06 radius=0.03
- link left_wrist_roll_link: geometry visual mesh filename=file:///home/lina/ros2_ws/install/unitree_g1_description/sh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
- link left_wrist_yaw_link: geometry visual mesh filename=file:///home/lina/ros2_ws/install/unitree_g1_description/sh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
- link logo_link: geometry visual mesh filename=file:///home/lina/ros2_ws/install/unitree_g1_description/sh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
- link pelvis: geometry visual mesh filename=file:///home/lina/ros2_ws/install/unitree_g1_description/sh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
- link right_elbow_link: geometry collision cylinder length=0.06 radius=0.03; visual mesh filename=file:///home/lina/ros2_ws/install/unitree_g1_description/sh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 scale=1 -1 1
- link right_hand_base: geometry collision box size=0.12 0.05 0.1; visual mesh filename=file:///home/lina/ros2_ws/install/unitree_g1_description/sh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 scale=1 -1 1
- link right_shoulder_pitch_link: geometry collision cylinder length=0.05 radius=0.03; visual mesh filename=file:///home/lina/ros2_ws/install/unitree_g1_description/sh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 scale=1 -1 1
- link right_shoulder_roll_link: geometry collision cylinder length=0.03 radius=0.03; visual mesh filename=file:///home/lina/ros2_ws/install/unitree_g1_description/sh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 scale=1 -1 1
- link right_shoulder_yaw_link: geometry collision cylinder length=0.06 radius=0.03; collision cylinder length=0.08 radius=0.03
- link right_wrist_pitch_link: geometry collision cylinder length=0.05 radius=0.03; collision cylinder length=0.06 radius=0.03
- link right_wrist_roll_link: geometry visual mesh filename=file:///home/lina/ros2_ws/install/unitree_g1_description/sh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
- link right_wrist_yaw_link: geometry visual mesh filename=file:///home/lina/ros2_ws/install/unitree_g1_description/sh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
- link torso_link: geometry collision box size=0.12 0.15 0.15; collision box size=0.12 0.2 0.15
- link waist_roll_link: geometry visual mesh filename=file:///home/lina/ros2_ws/install/unitree_g1_description/sh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
- link waist_yaw_link: geometry visual mesh filename=file:///home/lina/ros2_ws/install/unitree_g1_description/sh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
Joints:
- removed joint left_ankle_pitch_joint
- removed joint left_ankle_roll_joint
- removed joint left_elbow_joint
- removed joint left_hip_pitch_joint
- removed joint left_hip_roll_joint
- removed joint left_hip_yaw_joint
- removed joint left_knee_joint
- removed joint left_shoulder_pitch_joint
- removed joint left_shoulder_roll_joint
- removed joint left_shoulder_yaw_joint
- removed joint left_wrist_pitch_joint
- removed joint left_wrist_roll_joint
- removed joint left_wrist_yaw_joint
- removed joint right_ankle_pitch_joint
- removed joint right_ankle_roll_joint
- removed joint right_elbow_joint
- removed joint right_hip_pitch_joint
- removed joint right_hip_roll_joint
- removed joint right_hip_yaw_joint
- removed joint right_knee_joint
- removed joint right_shoulder_pitch_joint
- removed joint right_shoulder_roll_joint
- removed joint right_shoulder_yaw_joint
- removed joint right_wrist_pitch_joint
- removed joint right_wrist_roll_joint
- removed joint right_wrist_yaw_joint
- added joint left_joint1: type revolute, parent torso_link, child left_shoulder_pitch_link, origin xyz=0.0039563 0.10022 0.24778 rpy=0.27931 5.4949E-05 -0.00019159, axis 0 1 0, limit lower=-3.0892 upper=2.6704 effort=25 velocity=37
- added joint left_joint2: type revolute, parent left_shoulder_pitch_link, child left_shoulder_roll_link, origin xyz=0 0.038 -0.013831 rpy=-0.27925 0 0, axis 1 0 0, limit lower=-1.5882 upper=2.2515 effort=25 velocity=37
- added joint left_joint3: type revolute, parent left_shoulder_roll_link, child left_shoulder_yaw_link, origin xyz=0 0.00624 -0.1032, axis 0 0 1, limit lower=-2.618 upper=2.618 effort=25 velocity=37
- added joint left_joint4: type revolute, parent left_shoulder_yaw_link, child left_elbow_link, origin xyz=0.015783 0 -0.080518, axis 0 1 0, limit lower=-1.0472 upper=2.0944 effort=25 velocity=37
- added joint left_joint5: type revolute, parent left_elbow_link, child left_wrist_roll_link, origin xyz=0.100 0.00188791 -0.010, axis 1 0 0, limit lower=-1.972222054 upper=1.972222054 effort=25 velocity=37
- added joint left_joint6: type revolute, parent left_wrist_roll_link, child left_wrist_pitch_link, origin xyz=0.038 0 0, axis 0 1 0, limit lower=-1.614429558 upper=1.614429558 effort=5 velocity=22
- added joint left_joint7: type revolute, parent left_wrist_pitch_link, child left_wrist_yaw_link, origin xyz=0.046 0 0, axis 0 0 1, limit lower=-1.614429558 upper=1.614429558 effort=5 velocity=22
- added joint one_ankle_pitch_joint: type revolute, parent one_knee_link, child one_ankle_pitch_link, origin xyz=0 -9.4445e-05 -0.30001, axis 0 1 0, limit lower=-0.87267 upper=0.5236 effort=35 velocity=30
- added joint one_ankle_roll_joint: type revolute, parent one_ankle_pitch_link, child one_ankle_roll_link, origin xyz=0 0 -0.017558, axis 1 0 0, limit lower=-0.2618 upper=0.2618 effort=35 velocity=30
- added joint one_hip_pitch_joint: type revolute, parent pelvis, child one_hip_pitch_link, origin xyz=0 0.064452 -0.1027, axis 0 1 0, limit lower=-2.5307 upper=2.8798 effort=88 velocity=32
- added joint one_hip_roll_joint: type revolute, parent one_hip_pitch_link, child one_hip_roll_link, origin xyz=0 0.052 -0.030465 rpy=0 -0.1749 0, axis 1 0 0, limit lower=-0.5236 upper=2.9671 effort=88 velocity=32
- added joint one_hip_yaw_joint: type revolute, parent one_hip_roll_link, child one_hip_yaw_link, origin xyz=0.025001 0 -0.12412, axis 0 0 1, limit lower=-2.7576 upper=2.7576 effort=88 velocity=32
- added joint one_knee_joint: type revolute, parent one_hip_yaw_link, child one_knee_link, origin xyz=-0.078273 0.0021489 -0.17734 rpy=0 0.1749 0, axis 0 1 0, limit lower=-0.087267 upper=2.8798 effort=139 velocity=20
- added joint right_joint1: type revolute, parent torso_link, child right_shoulder_pitch_link, origin xyz=0.0039563 -0.10022 0.24778 rpy=-0.27931 5.4949E-05 0.00019159, axis 0 1 0, limit lower=-3.0892 upper=2.6704 effort=25 velocity=37
- added joint right_joint2: type revolute, parent right_shoulder_pitch_link, child right_shoulder_roll_link, origin xyz=0 -0.038 -0.013831 rpy=0.27925 0 0, axis 1 0 0, limit lower=-2.2515 upper=1.5882 effort=25 velocity=37
- added joint right_joint3: type revolute, parent right_shoulder_roll_link, child right_shoulder_yaw_link, origin xyz=0 -0.00624 -0.1032, axis 0 0 1, limit lower=-2.618 upper=2.618 effort=25 velocity=37
- added joint right_joint4: type revolute, parent right_shoulder_yaw_link, child right_elbow_link, origin xyz=0.015783 0 -0.080518, axis 0 1 0, limit lower=-1.0472 upper=2.0944 effort=25 velocity=37
- added joint right_joint5: type revolute, parent right_elbow_link, child right_wrist_roll_link, origin xyz=0.100 -0.00188791 -0.010, axis 1 0 0, limit lower=-1.972222054 upper=1.972222054 effort=25 velocity=37
- added joint right_joint6: type revolute, parent right_wrist_roll_link, child right_wrist_pitch_link, origin xyz=0.038 0 0, axis 0 1 0, limit lower=-1.614429558 upper=1.614429558 effort=5 velocity=22
- added joint right_joint7: type revolute, parent right_wrist_pitch_link, child right_wrist_yaw_link, origin xyz=0.046 0 0, axis 0 0 1, limit lower=-1.614429558 upper=1.614429558 effort=5 velocity=22
- added joint two_ankle_pitch_joint: type revolute, parent two_knee_link, child two_ankle_pitch_link, origin xyz=0 9.4445e-05 -0.30001, axis 0 1 0, limit lower=-0.87267 upper=0.5236 effort=35 velocity=30
- added joint two_ankle_roll_joint: type revolute, parent two_ankle_pitch_link, child two_ankle_roll_link, origin xyz=0 0 -0.017558, axis 1 0 0, limit lower=-0.2618 upper=0.2618 effort=35 velocity=30
- added joint two_hip_pitch_joint: type revolute, parent pelvis, child two_hip_pitch_link, origin xyz=0 -0.064452 -0.1027, axis 0 1 0, limit lower=-2.5307 upper=2.8798 effort=88 velocity=32
- added joint two_hip_roll_joint: type revolute, parent two_hip_pitch_link, child two_hip_roll_link, origin xyz=0 -0.052 -0.030465 rpy=0 -0.1749 0, axis 1 0 0, limit lower=-2.9671 upper=0.5236 effort=88 velocity=32
- added joint two_hip_yaw_joint: type revolute, parent two_hip_roll_link, child two_hip_yaw_link, origin xyz=0.025001 0 -0.12412, axis 0 0 1, limit lower=-2.7576 upper=2.7576 effort=88 velocity=32
- added joint two_knee_joint: type revolute, parent two_hip_yaw_link, child two_knee_link, origin xyz=-0.078273 -0.0021489 -0.17734 rpy=0 0.1749 0, axis 0 1 0, limit lower=-0.087267 upper=2.8798 effort=139 velocity=20

File: humanoid/Unitree/unitree_g1_description/xacro/arm.xacro (robot description, xacro)
@@ -32,5 +32,5 @@
 		</link>
 		<!-- Shoulder Pitch Joint -->
-		<joint name="${prefix}shoulder_pitch_joint" type="revolute">
+		<joint name="${prefix}joint1" type="revolute">
 			<origin xyz="0.0039563 ${direction*0.10022} 0.24778"
 							rpy="${direction*0.27931} 5.4949E-05 ${direction*-0.00019159}"/>
@@ -62,5 +62,5 @@
 		</link>
 		<!-- Shoulder Roll Joint -->
-		<joint name="${prefix}shoulder_roll_joint" type="revolute">
+		<joint name="${prefix}joint2" type="revolute">
 			<origin xyz="0 ${direction*0.038} -0.013831" rpy="${direction*-0.27925} 0 0"/>
 			<parent link="${prefix}shoulder_pitch_link"/>
@@ -98,5 +98,5 @@
 		</link>
 		<!-- Shoulder Yaw Joint -->
-		<joint name="${prefix}shoulder_yaw_joint" type="revolute">
+		<joint name="${prefix}joint3" type="revolute">
 			<origin xyz="0 ${direction*0.00624} -0.1032"/>
 			<parent link="${prefix}shoulder_roll_link"/>
@@ -127,5 +127,5 @@
 		</link>
 		<!-- Elbow Joint -->
-		<joint name="${prefix}elbow_joint" type="revolute">
+		<joint name="${prefix}joint4" type="revolute">
 			<origin xyz="0.015783 0 -0.080518"/>
 			<parent link="${prefix}shoulder_yaw_link"/>
@@ -150,5 +150,5 @@
 		</link>
 		<!-- Wrist Roll Joint -->
-		<joint name="${prefix}wrist_roll_joint" type="revolute">
+		<joint name="${prefix}joint5" type="revolute">
 			<origin xyz="0.100 ${direction*0.00188791} -0.010"/>
 			<axis xyz="1 0 0"/>
@@ -185,5 +185,5 @@
 		</link>
 		<!-- Wrist Pitch Joint -->
-		<joint name="${prefix}wrist_pitch_joint" type="revolute">
+		<joint name="${prefix}joint6" type="revolute">
 			<origin xyz="0.038 0 0"/>
 			<axis xyz="0 1 0"/>
@@ -208,5 +208,5 @@
 		</link>
 		<!-- Wrist Yaw Joint -->
-		<joint name="${prefix}wrist_yaw_joint" type="revolute">
+		<joint name="${prefix}joint7" type="revolute">
 			<origin xyz="0.046 0 0"/>
 			<axis xyz="0 0 1"/>

File: humanoid/Unitree/unitree_g1_description/xacro/robot.xacro (robot description, xacro)
@@ -8,7 +8,7 @@
 	<!-- Legs using modular macro -->
 	<!-- Left leg (direction = 1) -->
-	<xacro:UnitreeG1Leg name="left" direction="1"/>
+	<xacro:UnitreeG1Leg name="one" direction="1"/>
 	<!-- Right leg (direction = -1 for mirroring) -->
-	<xacro:UnitreeG1Leg name="right" direction="-1"/>
+	<xacro:UnitreeG1Leg name="two" direction="-1"/>
 	<!-- Body using modular macro -->
 	<xacro:UnitreeG1Body/>
