Commit message: modify unitree urdf

File: humanoid/Unitree/unitree_g1_description/xacro/ros2_control/ros2_control.xacro (robot description, xacro)
@@ -33,55 +33,55 @@
       </hardware>
       <!-- Left Leg Joints (6 DOF) -->
-      <joint name="left_hip_pitch_joint">
-        <command_interface name="position"/>
-        <command_interface name="velocity"/>
-        <command_interface name="effort"/>
-        <command_interface name="kp"/>
-        <command_interface name="kd"/>
-        <state_interface name="position"/>
-        <state_interface name="velocity"/>
-        <state_interface name="effort"/>
-      </joint>
-      <joint name="left_hip_roll_joint">
-        <command_interface name="position"/>
-        <command_interface name="velocity"/>
-        <command_interface name="effort"/>
-        <command_interface name="kp"/>
-        <command_interface name="kd"/>
-        <state_interface name="position"/>
-        <state_interface name="velocity"/>
-        <state_interface name="effort"/>
-      </joint>
-      <joint name="left_hip_yaw_joint">
-        <command_interface name="position"/>
-        <command_interface name="velocity"/>
-        <command_interface name="effort"/>
-        <command_interface name="kp"/>
-        <command_interface name="kd"/>
-        <state_interface name="position"/>
-        <state_interface name="velocity"/>
-        <state_interface name="effort"/>
-      </joint>
-      <joint name="left_knee_joint">
-        <command_interface name="position"/>
-        <command_interface name="velocity"/>
-        <command_interface name="effort"/>
-        <command_interface name="kp"/>
-        <command_interface name="kd"/>
-        <state_interface name="position"/>
-        <state_interface name="velocity"/>
-        <state_interface name="effort"/>
-      </joint>
-      <joint name="left_ankle_pitch_joint">
-        <command_interface name="position"/>
-        <command_interface name="velocity"/>
-        <command_interface name="effort"/>
-        <command_interface name="kp"/>
-        <command_interface name="kd"/>
-        <state_interface name="position"/>
-        <state_interface name="velocity"/>
-        <state_interface name="effort"/>
-      </joint>
-      <joint name="left_ankle_roll_joint">
+      <joint name="one_hip_pitch_joint">
+        <command_interface name="position"/>
+        <command_interface name="velocity"/>
+        <command_interface name="effort"/>
+        <command_interface name="kp"/>
+        <command_interface name="kd"/>
+        <state_interface name="position"/>
+        <state_interface name="velocity"/>
+        <state_interface name="effort"/>
+      </joint>
+      <joint name="one_hip_roll_joint">
+        <command_interface name="position"/>
+        <command_interface name="velocity"/>
+        <command_interface name="effort"/>
+        <command_interface name="kp"/>
+        <command_interface name="kd"/>
+        <state_interface name="position"/>
+        <state_interface name="velocity"/>
+        <state_interface name="effort"/>
+      </joint>
+      <joint name="one_hip_yaw_joint">
+        <command_interface name="position"/>
+        <command_interface name="velocity"/>
+        <command_interface name="effort"/>
+        <command_interface name="kp"/>
+        <command_interface name="kd"/>
+        <state_interface name="position"/>
+        <state_interface name="velocity"/>
+        <state_interface name="effort"/>
+      </joint>
+      <joint name="one_knee_joint">
+        <command_interface name="position"/>
+        <command_interface name="velocity"/>
+        <command_interface name="effort"/>
+        <command_interface name="kp"/>
+        <command_interface name="kd"/>
+        <state_interface name="position"/>
+        <state_interface name="velocity"/>
+        <state_interface name="effort"/>
+      </joint>
+      <joint name="one_ankle_pitch_joint">
+        <command_interface name="position"/>
+        <command_interface name="velocity"/>
+        <command_interface name="effort"/>
+        <command_interface name="kp"/>
+        <command_interface name="kd"/>
+        <state_interface name="position"/>
+        <state_interface name="velocity"/>
+        <state_interface name="effort"/>
+      </joint>
+      <joint name="one_ankle_roll_joint">
         <command_interface name="position"/>
         <command_interface name="velocity"/>
@@ -94,55 +94,55 @@
       </joint>
       <!-- Right Leg Joints (6 DOF) -->
-      <joint name="right_hip_pitch_joint">
-        <command_interface name="position"/>
-        <command_interface name="velocity"/>
-        <command_interface name="effort"/>
-        <command_interface name="kp"/>
-        <command_interface name="kd"/>
-        <state_interface name="position"/>
-        <state_interface name="velocity"/>
-        <state_interface name="effort"/>
-      </joint>
-      <joint name="right_hip_roll_joint">
-        <command_interface name="position"/>
-        <command_interface name="velocity"/>
-        <command_interface name="effort"/>
-        <command_interface name="kp"/>
-        <command_interface name="kd"/>
-        <state_interface name="position"/>
-        <state_interface name="velocity"/>
-        <state_interface name="effort"/>
-      </joint>
-      <joint name="right_hip_yaw_joint">
-        <command_interface name="position"/>
-        <command_interface name="velocity"/>
-        <command_interface name="effort"/>
-        <command_interface name="kp"/>
-        <command_interface name="kd"/>
-        <state_interface name="position"/>
-        <state_interface name="velocity"/>
-        <state_interface name="effort"/>
-      </joint>
-      <joint name="right_knee_joint">
-        <command_interface name="position"/>
-        <command_interface name="velocity"/>
-        <command_interface name="effort"/>
-        <command_interface name="kp"/>
-        <command_interface name="kd"/>
-        <state_interface name="position"/>
-        <state_interface name="velocity"/>
-        <state_interface name="effort"/>
-      </joint>
-      <joint name="right_ankle_pitch_joint">
-        <command_interface name="position"/>
-        <command_interface name="velocity"/>
-        <command_interface name="effort"/>
-        <command_interface name="kp"/>
-        <command_interface name="kd"/>
-        <state_interface name="position"/>
-        <state_interface name="velocity"/>
-        <state_interface name="effort"/>
-      </joint>
-      <joint name="right_ankle_roll_joint">
+      <joint name="two_hip_pitch_joint">
+        <command_interface name="position"/>
+        <command_interface name="velocity"/>
+        <command_interface name="effort"/>
+        <command_interface name="kp"/>
+        <command_interface name="kd"/>
+        <state_interface name="position"/>
+        <state_interface name="velocity"/>
+        <state_interface name="effort"/>
+      </joint>
+      <joint name="two_hip_roll_joint">
+        <command_interface name="position"/>
+        <command_interface name="velocity"/>
+        <command_interface name="effort"/>
+        <command_interface name="kp"/>
+        <command_interface name="kd"/>
+        <state_interface name="position"/>
+        <state_interface name="velocity"/>
+        <state_interface name="effort"/>
+      </joint>
+      <joint name="two_hip_yaw_joint">
+        <command_interface name="position"/>
+        <command_interface name="velocity"/>
+        <command_interface name="effort"/>
+        <command_interface name="kp"/>
+        <command_interface name="kd"/>
+        <state_interface name="position"/>
+        <state_interface name="velocity"/>
+        <state_interface name="effort"/>
+      </joint>
+      <joint name="two_knee_joint">
+        <command_interface name="position"/>
+        <command_interface name="velocity"/>
+        <command_interface name="effort"/>
+        <command_interface name="kp"/>
+        <command_interface name="kd"/>
+        <state_interface name="position"/>
+        <state_interface name="velocity"/>
+        <state_interface name="effort"/>
+      </joint>
+      <joint name="two_ankle_pitch_joint">
+        <command_interface name="position"/>
+        <command_interface name="velocity"/>
+        <command_interface name="effort"/>
+        <command_interface name="kp"/>
+        <command_interface name="kd"/>
+        <state_interface name="position"/>
+        <state_interface name="velocity"/>
+        <state_interface name="effort"/>
+      </joint>
+      <joint name="two_ankle_roll_joint">
         <command_interface name="position"/>
         <command_interface name="velocity"/>
@@ -186,65 +186,65 @@
       </joint>
       <!-- Left Arm Joints (7 DOF) -->
-      <joint name="left_shoulder_pitch_joint">
-        <command_interface name="position"/>
-        <command_interface name="velocity"/>
-        <command_interface name="effort"/>
-        <command_interface name="kp"/>
-        <command_interface name="kd"/>
-        <state_interface name="position"/>
-        <state_interface name="velocity"/>
-        <state_interface name="effort"/>
-      </joint>
-      <joint name="left_shoulder_roll_joint">
-        <command_interface name="position"/>
-        <command_interface name="velocity"/>
-        <command_interface name="effort"/>
-        <command_interface name="kp"/>
-        <command_interface name="kd"/>
-        <state_interface name="position"/>
-        <state_interface name="velocity"/>
-        <state_interface name="effort"/>
-      </joint>
-      <joint name="left_shoulder_yaw_joint">
-        <command_interface name="position"/>
-        <command_interface name="velocity"/>
-        <command_interface name="effort"/>
-        <command_interface name="kp"/>
-        <command_interface name="kd"/>
-        <state_interface name="position"/>
-        <state_interface name="velocity"/>
-        <state_interface name="effort"/>
-      </joint>
-      <joint name="left_elbow_joint">
-        <command_interface name="position"/>
-        <command_interface name="velocity"/>
-        <command_interface name="effort"/>
-        <command_interface name="kp"/>
-        <command_interface name="kd"/>
-        <state_interface name="position"/>
-        <state_interface name="velocity"/>
-        <state_interface name="effort"/>
-      </joint>
-      <joint name="left_wrist_roll_joint">
-        <command_interface name="position"/>
-        <command_interface name="velocity"/>
-        <command_interface name="effort"/>
-        <command_interface name="kp"/>
-        <command_interface name="kd"/>
-        <state_interface name="position"/>
-        <state_interface name="velocity"/>
-        <state_interface name="effort"/>
-      </joint>
-      <joint name="left_wrist_pitch_joint">
-        <command_interface name="position"/>
-        <command_interface name="velocity"/>
-        <command_interface name="effort"/>
-        <command_interface name="kp"/>
-        <command_interface name="kd"/>
-        <state_interface name="position"/>
-        <state_interface name="velocity"/>
-        <state_interface name="effort"/>
-      </joint>
-      <joint name="left_wrist_yaw_joint">
+      <joint name="left_joint1">
+        <command_interface name="position"/>
+        <command_interface name="velocity"/>
+        <command_interface name="effort"/>
+        <command_interface name="kp"/>
+        <command_interface name="kd"/>
+        <state_interface name="position"/>
+        <state_interface name="velocity"/>
+        <state_interface name="effort"/>
+      </joint>
+      <joint name="left_joint2">
+        <command_interface name="position"/>
+        <command_interface name="velocity"/>
+        <command_interface name="effort"/>
+        <command_interface name="kp"/>
+        <command_interface name="kd"/>
+        <state_interface name="position"/>
+        <state_interface name="velocity"/>
+        <state_interface name="effort"/>
+      </joint>
+      <joint name="left_joint3">
+        <command_interface name="position"/>
+        <command_interface name="velocity"/>
+        <command_interface name="effort"/>
+        <command_interface name="kp"/>
+        <command_interface name="kd"/>
+        <state_interface name="position"/>
+        <state_interface name="velocity"/>
+        <state_interface name="effort"/>
+      </joint>
+      <joint name="left_joint4">
+        <command_interface name="position"/>
+        <command_interface name="velocity"/>
+        <command_interface name="effort"/>
+        <command_interface name="kp"/>
+        <command_interface name="kd"/>
+        <state_interface name="position"/>
+        <state_interface name="velocity"/>
+        <state_interface name="effort"/>
+      </joint>
+      <joint name="left_joint5">
+        <command_interface name="position"/>
+        <command_interface name="velocity"/>
+        <command_interface name="effort"/>
+        <command_interface name="kp"/>
+        <command_interface name="kd"/>
+        <state_interface name="position"/>
+        <state_interface name="velocity"/>
+        <state_interface name="effort"/>
+      </joint>
+      <joint name="left_joint6">
+        <command_interface name="position"/>
+        <command_interface name="velocity"/>
+        <command_interface name="effort"/>
+        <command_interface name="kp"/>
+        <command_interface name="kd"/>
+        <state_interface name="position"/>
+        <state_interface name="velocity"/>
+        <state_interface name="effort"/>
+      </joint>
+      <joint name="left_joint7">
         <command_interface name="position"/>
         <command_interface name="velocity"/>
@@ -257,65 +257,65 @@
       </joint>
       <!-- Right Arm Joints (7 DOF) -->
-      <joint name="right_shoulder_pitch_joint">
-        <command_interface name="position"/>
-        <command_interface name="velocity"/>
-        <command_interface name="effort"/>
-        <command_interface name="kp"/>
-        <command_interface name="kd"/>
-        <state_interface name="position"/>
-        <state_interface name="velocity"/>
-        <state_interface name="effort"/>
-      </joint>
-      <joint name="right_shoulder_roll_joint">
-        <command_interface name="position"/>
-        <command_interface name="velocity"/>
-        <command_interface name="effort"/>
-        <command_interface name="kp"/>
-        <command_interface name="kd"/>
-        <state_interface name="position"/>
-        <state_interface name="velocity"/>
-        <state_interface name="effort"/>
-      </joint>
-      <joint name="right_shoulder_yaw_joint">
-        <command_interface name="position"/>
-        <command_interface name="velocity"/>
-        <command_interface name="effort"/>
-        <command_interface name="kp"/>
-        <command_interface name="kd"/>
-        <state_interface name="position"/>
-        <state_interface name="velocity"/>
-        <state_interface name="effort"/>
-      </joint>
-      <joint name="right_elbow_joint">
-        <command_interface name="position"/>
-        <command_interface name="velocity"/>
-        <command_interface name="effort"/>
-        <command_interface name="kp"/>
-        <command_interface name="kd"/>
-        <state_interface name="position"/>
-        <state_interface name="velocity"/>
-        <state_interface name="effort"/>
-      </joint>
-      <joint name="right_wrist_roll_joint">
-        <command_interface name="position"/>
-        <command_interface name="velocity"/>
-        <command_interface name="effort"/>
-        <command_interface name="kp"/>
-        <command_interface name="kd"/>
-        <state_interface name="position"/>
-        <state_interface name="velocity"/>
-        <state_interface name="effort"/>
-      </joint>
-      <joint name="right_wrist_pitch_joint">
-        <command_interface name="position"/>
-        <command_interface name="velocity"/>
-        <command_interface name="effort"/>
-        <command_interface name="kp"/>
-        <command_interface name="kd"/>
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
Commit message: 调整urdf路径格式

File: humanoid/Unitree/unitree_g1_description/urdf/unitree_g1.urdf (robot description, URDF)
Before this commit: robot g1_29dof, 39 links, 38 joints
Links:
- link head_link: geometry collision mesh filename=package://unitree_g1_description/meshes/body/head.obj; visual mesh filename=package://unitree_g1_description/meshes/body/head.obj
- link left_elbow_link: geometry collision cylinder length=0.06 radius=0.03; visual mesh filename=package://unitree_g1_description/meshes/arm/elbow.obj scale=1 1 1
- link left_hand_base: geometry collision box size=0.12 0.05 0.1; visual mesh filename=package://unitree_g1_description/meshes/arm/hand.obj scale=1 1 1
- link left_shoulder_pitch_link: geometry collision cylinder length=0.05 radius=0.03; visual mesh filename=package://unitree_g1_description/meshes/arm/shoulder_pitch.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 scale=1 1 1
- link left_shoulder_roll_link: geometry collision cylinder length=0.03 radius=0.03; visual mesh filename=package://unitree_g1_description/meshes/arm/shoulder_roll.o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 scale=1 1 1
- link left_shoulder_yaw_link: geometry collision cylinder length=0.06 radius=0.03; collision cylinder length=0.08 radius=0.03
- link left_wrist_pitch_link: geometry collision cylinder length=0.05 radius=0.03; collision cylinder length=0.06 radius=0.03
- link left_wrist_roll_link: geometry visual mesh filename=package://unitree_g1_description/meshes/arm/wrist_roll.obj
- link left_wrist_yaw_link: geometry visual mesh filename=package://unitree_g1_description/meshes/arm/wrist_yaw.obj
- link logo_link: geometry visual mesh filename=package://unitree_g1_description/meshes/body/logo.obj
- link one_ankle_pitch_link: geometry collision mesh filename=package://unitree_g1_description/meshes/leg/ankle_pitch.obj; visual mesh filename=package://unitree_g1_description/meshes/leg/ankle_pitch.obj
- link one_ankle_roll_link: geometry collision sphere radius=0.005; collision sphere radius=0.005
- link one_hip_pitch_link: geometry collision mesh filename=package://unitree_g1_description/meshes/leg/hip_pitch.obj scale=1 1 1; visual mesh filename=package://unitree_g1_description/meshes/leg/hip_pitch.obj scale=1 1 1
- link one_hip_roll_link: geometry collision mesh filename=package://unitree_g1_description/meshes/leg/hip_roll.obj; visual mesh filename=package://unitree_g1_description/meshes/leg/hip_roll.obj
- link one_hip_yaw_link: geometry collision mesh filename=package://unitree_g1_description/meshes/leg/hip_yaw.obj scale=1 1 1; visual mesh filename=package://unitree_g1_description/meshes/leg/hip_yaw.obj scale=1 1 1
- link one_knee_link: geometry collision mesh filename=package://unitree_g1_description/meshes/leg/knee.obj scale=1 1 1; visual mesh filename=package://unitree_g1_description/meshes/leg/knee.obj scale=1 1 1
- link pelvis: geometry visual mesh filename=package://unitree_g1_description/meshes/body/pelvis.obj
- link right_elbow_link: geometry collision cylinder length=0.06 radius=0.03; visual mesh filename=package://unitree_g1_description/meshes/arm/elbow.obj scale=1 -1 1
- link right_hand_base: geometry collision box size=0.12 0.05 0.1; visual mesh filename=package://unitree_g1_description/meshes/arm/hand.obj scale=1 -1 1
- link right_shoulder_pitch_link: geometry collision cylinder length=0.05 radius=0.03; visual mesh filename=package://unitree_g1_description/meshes/arm/shoulder_pitch.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 scale=1 -1 1
- link right_shoulder_roll_link: geometry collision cylinder length=0.03 radius=0.03; visual mesh filename=package://unitree_g1_description/meshes/arm/shoulder_roll.o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 scale=1 -1 1
- link right_shoulder_yaw_link: geometry collision cylinder length=0.06 radius=0.03; collision cylinder length=0.08 radius=0.03
- link right_wrist_pitch_link: geometry collision cylinder length=0.05 radius=0.03; collision cylinder length=0.06 radius=0.03
- link right_wrist_roll_link: geometry visual mesh filename=package://unitree_g1_description/meshes/arm/wrist_roll.obj
- link right_wrist_yaw_link: geometry visual mesh filename=package://unitree_g1_description/meshes/arm/wrist_yaw.obj
- link torso_link: geometry collision box size=0.12 0.15 0.15; collision box size=0.12 0.2 0.15
- link two_ankle_pitch_link: geometry collision mesh filename=package://unitree_g1_description/meshes/leg/ankle_pitch.obj; visual mesh filename=package://unitree_g1_description/meshes/leg/ankle_pitch.obj
- link two_ankle_roll_link: geometry collision sphere radius=0.005; collision sphere radius=0.005
- link two_hip_pitch_link: geometry collision mesh filename=package://unitree_g1_description/meshes/leg/hip_pitch.obj scale=1 -1 1; visual mesh filename=package://unitree_g1_description/meshes/leg/hip_pitch.obj scale=1 -1 1
- link two_hip_roll_link: geometry collision mesh filename=package://unitree_g1_description/meshes/leg/hip_roll.obj; visual mesh filename=package://unitree_g1_description/meshes/leg/hip_roll.obj
- link two_hip_yaw_link: geometry collision mesh filename=package://unitree_g1_description/meshes/leg/hip_yaw.obj scale=1 -1 1; visual mesh filename=package://unitree_g1_description/meshes/leg/hip_yaw.obj scale=1 -1 1
- link two_knee_link: geometry collision mesh filename=package://unitree_g1_description/meshes/leg/knee.obj scale=1 -1 1; visual mesh filename=package://unitree_g1_description/meshes/leg/knee.obj scale=1 -1 1
- link waist_roll_link: geometry visual mesh filename=package://unitree_g1_description/meshes/body/waist_roll.obj
- link waist_yaw_link: geometry visual mesh filename=package://unitree_g1_description/meshes/body/waist_yaw.obj
