Commit message: update mesh to glb

File: humanoid/Galaxea/galaxea_r1_description/urdf/galaxea_r1.urdf (robot description, URDF)
Before this commit: robot R1, 36 links, 35 joints
Links:
- removed link left_realsense_link
- removed link right_realsense_link
- added link chassis_back_camera; visual mesh filename=package://sensor_models/meshes/usb_camera/camera_02.glb
- added link chassis_fl_camera; visual mesh filename=package://sensor_models/meshes/usb_camera/camera_02.glb
- added link chassis_fr_camera; visual mesh filename=package://sensor_models/meshes/usb_camera/camera_02.glb
- added link chassis_left_camera; visual mesh filename=package://sensor_models/meshes/usb_camera/camera_02.glb
- added link chassis_right_camera; visual mesh filename=package://sensor_models/meshes/usb_camera/camera_02.glb
- added link left_hand_camera_link; visual mesh filename=package://sensor_models/meshes/realsense/d435.glb
- added link left_hand_camera_stand_link, mass 0.175; visual mesh filename=package://galaxea_r1_description/meshes/hand_camera_stand.g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
- added link left_lidar; visual mesh filename=package://sensor_models/meshes/livox/mid360.glb
- added link right_hand_camera_link; visual mesh filename=package://sensor_models/meshes/realsense/d435.glb
- added link right_hand_camera_stand_link, mass 0.175; visual mesh filename=package://galaxea_r1_description/meshes/hand_camera_stand.g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
- added link right_lidar; visual mesh filename=package://sensor_models/meshes/livox/mid360.glb
- link base_link: geometry collision mesh filename=package://galaxea_r1_description/meshes/chassis.glb; visual mesh filename=package://galaxea_r1_description/meshes/chassis.glb
- link steer_motor_link1: geometry visual mesh filename=package://galaxea_r1_description/meshes/steer.glb
- link steer_motor_link2: geometry visual mesh filename=package://galaxea_r1_description/meshes/steer.glb
- link steer_motor_link3: geometry visual mesh filename=package://galaxea_r1_description/meshes/steer.glb
- link torso_link1: geometry collision mesh filename=package://galaxea_r1_description/meshes/torso_link1.glb; visual mesh filename=package://galaxea_r1_description/meshes/torso_link1.glb
- link torso_link2: geometry collision mesh filename=package://galaxea_r1_description/meshes/torso_link2.glb; visual mesh filename=package://galaxea_r1_description/meshes/torso_link2.glb
- link torso_link3: geometry collision mesh filename=package://galaxea_r1_description/meshes/torso_link3.glb; visual mesh filename=package://galaxea_r1_description/meshes/torso_link3.glb
- link torso_link4: geometry collision mesh filename=package://galaxea_r1_description/meshes/torso_link4.glb; visual mesh filename=package://galaxea_r1_description/meshes/torso_link4.glb
- link wheel_motor_link1: geometry collision cylinder length=0.048 radius=0.07; visual mesh filename=package://galaxea_r1_description/meshes/wheel.glb
- link wheel_motor_link2: geometry collision cylinder length=0.048 radius=0.07; visual mesh filename=package://galaxea_r1_description/meshes/wheel.glb
- link wheel_motor_link3: geometry collision cylinder length=0.048 radius=0.07; visual mesh filename=package://galaxea_r1_description/meshes/wheel.glb
- link zed_link: geometry collision mesh filename=package://galaxea_r1_description/meshes/head.glb; visual mesh filename=package://galaxea_r1_description/meshes/head.glb
Joints:
- removed joint left_realsense_joint
- removed joint right_realsense_joint
- removed joint steer_motor_joint1
- removed joint steer_motor_joint2
- removed joint steer_motor_joint3
- removed joint wheel_motor_joint1
- removed joint wheel_motor_joint2
- removed joint wheel_motor_joint3
- added joint chassis_back_camera_joint: type fixed, parent base_link, child chassis_back_camera, origin xyz=-0.314835 0 0.217  rpy= 0 0 3.141592653589793
- added joint chassis_fl_camera_joint: type fixed, parent base_link, child chassis_fl_camera, origin xyz=0.25625 0.132735 0.205 
- added joint chassis_fr_camera_joint: type fixed, parent base_link, child chassis_fr_camera, origin xyz=0.25625 -0.132735 0.205 
- added joint chassis_left_camera_joint: type fixed, parent base_link, child chassis_left_camera, origin xyz=0.02865 0.32245 0.205  rpy= 0 0 1.5707963267948966
- added joint chassis_right_camera_joint: type fixed, parent base_link, child chassis_right_camera, origin xyz=0.02865 -0.32245 0.205  rpy= 0 0 -1.5707963267948966
- added joint left_hand_camera_joint: type fixed, parent left_hand_camera_stand_link, child left_hand_camera_link, origin xyz=0.0325 0 0
- added joint left_hand_camera_stand_joint: type fixed, parent left_link6, child left_hand_camera_stand_link, origin xyz=0.098768 0.0021071 0.05055 rpy=-2.0071 0.0077831 -1.5707963267948966
- added joint left_lidar_joint: type fixed, parent base_link, child left_lidar, origin xyz=0.203297 0.26215 0.233685 
- added joint right_hand_camera_joint: type fixed, parent right_hand_camera_stand_link, child right_hand_camera_link, origin xyz=0.0325 0 0
- added joint right_hand_camera_stand_joint: type fixed, parent right_link6, child right_hand_camera_stand_link, origin xyz=0.098762 0.0021071 -0.05055 rpy=1.1344 -0.0077831 1.5707963267948966
- added joint right_lidar_joint: type fixed, parent base_link, child right_lidar, origin xyz=0.203297 -0.26215 0.233685 
- added joint steer_joint1: type fixed, parent base_link, child steer_motor_link1, origin xyz=0.21516 0.28 0.12375
- added joint steer_joint2: type fixed, parent base_link, child steer_motor_link2, origin xyz=0.21516 -0.28 0.12375
- added joint steer_joint3: type fixed, parent base_link, child steer_motor_link3, origin xyz=-0.28084 0 0.12375
- added joint wheel_joint1: type fixed, parent steer_motor_link1, child wheel_motor_link1, origin xyz=0 0 -0.09525 rpy=0 0 3.141592653589793
- added joint wheel_joint2: type fixed, parent steer_motor_link2, child wheel_motor_link2, origin xyz=0 0 -0.09525
- added joint wheel_joint3: type fixed, parent steer_motor_link3, child wheel_motor_link3, origin xyz=0 0 -0.09525 rpy=0 0 3.141592653589793

File: humanoid/Galaxea/galaxea_r1_description/xacro/components/chassis.xacro (robot description, xacro)
@@ -2,5 +2,9 @@
 <robot xmlns:xacro="http://www.ros.org/wiki/xacro">
     <xacro:property name="PI" value="3.1415926535897931"/>
-    <xacro:macro name="Chassis">
+    <xacro:macro name="Chassis" params="enable_wheel_joints:='true'">
+        <xacro:property name="wheel_joints_enabled"
+                        value="${str(enable_wheel_joints).lower() in ['true', '1', 'yes', 'on']}"/>
+        <xacro:property name="steering_joint_type" value="${'revolute' if wheel_joints_enabled else 'fixed'}"/>
+        <xacro:property name="driving_joint_type" value="${'continuous' if wheel_joints_enabled else 'fixed'}"/>
         <!-- Base Link -->
         <link name="base_link">
@@ -31,15 +35,17 @@
             <visual>
                 <geometry>
-                    <mesh filename="file://$(find galaxea_r1_description)/meshes/steer_motor.obj"/>
+                    <mesh filename="file://$(find galaxea_r1_description)/meshes/steer.glb"/>
                 </geometry>
             </visual>
         </link>
         <!-- Steer Motor Joint 1: Base to Steer Motor 1 -->
-        <joint name="steer_joint1" type="revolute">
+        <joint name="steer_joint1" type="${steering_joint_type}">
             <origin xyz="0.21516 0.28 0.12375"/>
             <parent link="base_link"/>
             <child link="steer_motor_link1"/>
-            <axis xyz="0 0 1"/>
-            <limit lower="${-PI/2}" upper="${PI/2}" effort="44" velocity="${PI}"/>
+            <xacro:if value="${wheel_joints_enabled}">
+                <axis xyz="0 0 1"/>
+                <limit lower="${-PI/2}" upper="${PI/2}" effort="44" velocity="${PI}"/>
+            </xacro:if>
         </joint>
         <!-- Wheel Motor Link 1 -->
@@ -53,5 +59,5 @@
             <visual>
                 <geometry>
-                    <mesh filename="file://$(find galaxea_r1_description)/meshes/wheel_motor.obj"/>
+                    <mesh filename="file://$(find galaxea_r1_description)/meshes/wheel.glb"/>
                 </geometry>
             </visual>
@@ -64,9 +70,11 @@
         </link>
         <!-- Wheel Motor Joint 1: Steer Motor 1 to Wheel Motor 1 -->
-        <joint name="wheel_joint1" type="continuous">
+        <joint name="wheel_joint1" type="${driving_joint_type}">
             <origin xyz="0 0 -0.09525" rpy="0 0 ${PI}"/>
             <parent link="steer_motor_link1"/>
             <child link="wheel_motor_link1"/>
-            <axis xyz="0 -1 0"/>
+            <xacro:if value="${wheel_joints_enabled}">
+                <axis xyz="0 -1 0"/>
+            </xacro:if>
         </joint>
         <!-- Steer Motor Link 2 -->
@@ -81,21 +89,17 @@
                 <origin rpy="0 0 ${PI}"/>
                 <geometry>
-                    <mesh filename="file://$(find galaxea_r1_description)/meshes/steer_motor.obj"/>
-                </geometry>
-            </visual>
-            <collision>
-                <origin rpy="0 0 ${PI}"/>
-                <geometry>
-                    <mesh filename="file://$(find galaxea_r1_description)/meshes/steer_motor.obj"/>
-                </geometry>
-            </collision>
+                    <mesh filename="file://$(find galaxea_r1_description)/meshes/steer.glb"/>
+                </geometry>
+            </visual>
         </link>
         <!-- Steer Motor Joint 2: Base to Steer Motor 2 -->
-        <joint name="steer_joint2" type="revolute">
+        <joint name="steer_joint2" type="${steering_joint_type}">
             <origin xyz="0.21516 -0.28 0.12375"/>
             <parent link="base_link"/>
             <child link="steer_motor_link2"/>
-            <axis xyz="0 0 1"/>
-            <limit lower="${-PI/2}" upper="${PI/2}" effort="44" velocity="${PI}"/>
+            <xacro:if value="${wheel_joints_enabled}">
+                <axis xyz="0 0 1"/>
+                <limit lower="${-PI/2}" upper="${PI/2}" effort="44" velocity="${PI}"/>
+            </xacro:if>
         </joint>
         <!-- Wheel Motor Link 2 -->
@@ -109,5 +113,5 @@
             <visual>
                 <geometry>
-                    <mesh filename="file://$(find galaxea_r1_description)/meshes/wheel_motor.obj"/>
+                    <mesh filename="file://$(find galaxea_r1_description)/meshes/wheel.glb"/>
                 </geometry>
             </visual>
@@ -120,9 +124,11 @@
         </link>
         <!-- Wheel Motor Joint 2: Steer Motor 2 to Wheel Motor 2 -->
-        <joint name="wheel_joint2" type="continuous">
+        <joint name="wheel_joint2" type="${driving_joint_type}">
             <origin xyz="0 0 -0.09525"/>
             <parent link="steer_motor_link2"/>
             <child link="wheel_motor_link2"/>
-            <axis xyz="0 1 0"/>
+            <xacro:if value="${wheel_joints_enabled}">
+                <axis xyz="0 1 0"/>
+            </xacro:if>
         </joint>
         <!-- Steer Motor Link 3 -->
@@ -136,20 +142,17 @@
             <visual>
                 <geometry>
-                    <mesh filename="file://$(find galaxea_r1_description)/meshes/steer_motor.obj"/>
-                </geometry>
-            </visual>
-            <collision>
-                <geometry>
-                    <mesh filename="file://$(find galaxea_r1_description)/meshes/steer_motor.obj"/>
-                </geometry>
-            </collision>
+                    <mesh filename="file://$(find galaxea_r1_description)/meshes/steer.glb"/>
+                </geometry>
+            </visual>
         </link>
         <!-- Steer Motor Joint 3: Base to Steer Motor 3 -->
-        <joint name="steer_joint3" type="revolute">
+        <joint name="steer_joint3" type="${steering_joint_type}">
             <origin xyz="-0.28084 0 0.12375"/>
             <parent link="base_link"/>
             <child link="steer_motor_link3"/>
-            <axis xyz="0 0 1"/>
-            <limit lower="${-PI/2}" upper="${PI/2}" effort="44" velocity="${PI}"/>
+            <xacro:if value="${wheel_joints_enabled}">
+                <axis xyz="0 0 1"/>
+                <limit lower="${-PI/2}" upper="${PI/2}" effort="44" velocity="${PI}"/>
+            </xacro:if>
         </joint>
         <!-- Wheel Motor Link 3 -->
@@ -163,5 +166,5 @@
             <visual>
                 <geometry>
-                    <mesh filename="file://$(find galaxea_r1_description)/meshes/wheel_motor.obj"/>
+                    <mesh filename="file://$(find galaxea_r1_description)/meshes/wheel.glb"/>
                 </geometry>
             </visual>
@@ -174,9 +177,11 @@
         </link>
         <!-- Wheel Motor Joint 3: Steer Motor 3 to Wheel Motor 3 -->
-        <joint name="wheel_joint3" type="continuous">
+        <joint name="wheel_joint3" type="${driving_joint_type}">
             <origin xyz="0 0 -0.09525" rpy="0 0 ${PI}"/>
             <parent link="steer_motor_link3"/>
             <child link="wheel_motor_link3"/>
-            <axis xyz="0 -1 0"/>
+            <xacro:if value="${wheel_joints_enabled}">
+                <axis xyz="0 -1 0"/>
+            </xacro:if>
         </joint>
         <link name="left_lidar">

File: humanoid/Galaxea/galaxea_r1_description/xacro/components/realsense.xacro (robot description, xacro)
@@ -4,6 +4,6 @@
 	<xacro:macro name="RealSense" params="side">
     <xacro:property name="side_prefix" value="${side + '_' if side else ''}"/>
-    <!-- RealSense Camera Link -->
-    <link name="${side_prefix}realsense_link">
+    <!-- Hand camera stand link -->
+    <link name="${side_prefix}hand_camera_stand_link">
       <inertial>
         <origin xyz="0.022169 0.0060171 -0.017353"/>
@@ -13,21 +13,23 @@
       <visual>
         <geometry>
-          <mesh filename="file://$(find galaxea_r1_description)/meshes/camera_stand.obj"/>
+          <mesh filename="file://$(find galaxea_r1_description)/meshes/hand_camera_stand.glb"/>
         </geometry>
       </visual>
+    </link>
+    <!-- Hand camera link -->
+    <link name="${side_prefix}hand_camera_link">
       <visual>
-        <origin xyz="0.0325 0 0"/>
         <geometry>
           <mesh filename="file://$(find sensor_models)/meshes/realsense/d435.glb"/>
         </geometry>
       </visual>
-      <collision>
-        <geometry>
-          <mesh filename="file://$(find galaxea_r1_description)/meshes/camera_stand.obj"/>
-        </geometry>
-      </collision>
     </link>
-    <!-- RealSense Joint: Arm 6 to Camera -->
-    <joint name="${side_prefix}realsense_joint" type="fixed">
+    <joint name="${side_prefix}hand_camera_joint" type="fixed">
+      <origin xyz="0.0325 0 0"/>
+      <parent link="${side_prefix}hand_camera_stand_link"/>
+      <child link="${side_prefix}hand_camera_link"/>
+    </joint>
+    <!-- Hand camera stand joint: Arm 6 to camera stand -->
+    <joint name="${side_prefix}hand_camera_stand_joint" type="fixed">
       <xacro:if value="${side == 'left'}">
         <origin xyz="0.098768 0.0021071 0.05055" rpy="-2.0071 0.0077831 ${-PI/2}"/>
@@ -38,5 +40,5 @@
         <parent link="right_link6"/>
       </xacro:if>
-      <child link="${side_prefix}realsense_link"/>
+      <child link="${side_prefix}hand_camera_stand_link"/>
     </joint>
   </xacro:macro>

File: humanoid/Galaxea/galaxea_r1_description/xacro/components/torso.xacro (robot description, xacro)
@@ -12,10 +12,10 @@
       <visual>
         <geometry>
-          <mesh filename="file://$(find galaxea_r1_description)/meshes/torso_link1.obj"/>
+          <mesh filename="file://$(find galaxea_r1_description)/meshes/torso_link1.glb"/>
         </geometry>
       </visual>
       <collision>
         <geometry>
-          <mesh filename="file://$(find galaxea_r1_description)/meshes/torso_link1.obj"/>
+          <mesh filename="file://$(find galaxea_r1_description)/meshes/torso_link1.glb"/>
         </geometry>
       </collision>
@@ -38,10 +38,10 @@
       <visual>
         <geometry>
-          <mesh filename="file://$(find galaxea_r1_description)/meshes/torso_link2.obj"/>
+          <mesh filename="file://$(find galaxea_r1_description)/meshes/torso_link2.glb"/>
         </geometry>
       </visual>
       <collision>
         <geometry>
-          <mesh filename="file://$(find galaxea_r1_description)/meshes/torso_link2.obj"/>
+          <mesh filename="file://$(find galaxea_r1_description)/meshes/torso_link2.glb"/>
         </geometry>
       </collision>
@@ -64,10 +64,10 @@
       <visual>
         <geometry>
-          <mesh filename="file://$(find galaxea_r1_description)/meshes/torso_link3.obj"/>
+          <mesh filename="file://$(find galaxea_r1_description)/meshes/torso_link3.glb"/>
         </geometry>
       </visual>
       <collision>
         <geometry>
-          <mesh filename="file://$(find galaxea_r1_description)/meshes/torso_link3.obj"/>
+          <mesh filename="file://$(find galaxea_r1_description)/meshes/torso_link3.glb"/>
         </geometry>
       </collision>
@@ -90,10 +90,10 @@
       <visual>
         <geometry>
-          <mesh filename="file://$(find galaxea_r1_description)/meshes/torso_link4.obj"/>
+          <mesh filename="file://$(find galaxea_r1_description)/meshes/torso_link4.glb"/>
         </geometry>
       </visual>
       <collision>
         <geometry>
-          <mesh filename="file://$(find galaxea_r1_description)/meshes/torso_link4.obj"/>
+          <mesh filename="file://$(find galaxea_r1_description)/meshes/torso_link4.glb"/>
         </geometry>
       </collision>
@@ -116,10 +116,10 @@
       <visual>
         <geometry>
-          <mesh filename="file://$(find galaxea_r1_description)/meshes/zed_link.obj"/>
+          <mesh filename="file://$(find galaxea_r1_description)/meshes/head.glb"/>
         </geometry>
       </visual>
       <collision>
         <geometry>
-          <mesh filename="file://$(find galaxea_r1_description)/meshes/zed_link.obj"/>
+          <mesh filename="file://$(find galaxea_r1_description)/meshes/head.glb"/>
         </geometry>
       </collision>
