Commit message: fix galaxea chassis

File: humanoid/Galaxea/galaxea_r1_description/xacro/components/chassis.xacro (robot description, xacro)
@@ -217,5 +217,5 @@
         </link>
         <joint name="chassis_fl_camera_joint" type="fixed">
-            <origin xyz="0.25625 0.132735 0.205 "/>
+            <origin xyz="0.25625 0.132735 0.205 " rpy="${-PI/2} 0 ${-PI/2}"/>
             <parent link="base_link"/>
             <child link="chassis_fl_camera"/>
@@ -229,5 +229,5 @@
         </link>
         <joint name="chassis_fr_camera_joint" type="fixed">
-            <origin xyz="0.25625 -0.132735 0.205 "/>
+            <origin xyz="0.25625 -0.132735 0.205 " rpy="${-PI/2} 0 ${-PI/2}"/>
             <parent link="base_link"/>
             <child link="chassis_fr_camera"/>
@@ -241,5 +241,5 @@
         </link>
         <joint name="chassis_right_camera_joint" type="fixed">
-            <origin xyz="0.02865 -0.32245 0.205 " rpy=" 0 0 ${-PI/2}"/>
+            <origin xyz="0.02865 -0.32245 0.205 " rpy="${-PI/2} 0 ${PI}"/>
             <parent link="base_link"/>
             <child link="chassis_right_camera"/>
@@ -253,5 +253,5 @@
         </link>
         <joint name="chassis_left_camera_joint" type="fixed">
-            <origin xyz="0.02865 0.32245 0.205 " rpy=" 0 0 ${PI/2}"/>
+            <origin xyz="0.02865 0.32245 0.205 " rpy="${-PI/2} 0 0"/>
             <parent link="base_link"/>
             <child link="chassis_left_camera"/>
@@ -265,5 +265,5 @@
         </link>
         <joint name="chassis_back_camera_joint" type="fixed">
-            <origin xyz="-0.314835 0 0.217 " rpy=" 0 0 ${PI}"/>
+            <origin xyz="-0.314835 0 0.217 " rpy="${-PI/2} 0 ${PI/2}"/>
             <parent link="base_link"/>
             <child link="chassis_back_camera"/>
