Commit message: add rs01

File: humanoid/Realman/aidal_description/urdf/aidal.urdf (robot description, URDF)
Before this commit: robot RealMan_AIDAL, 43 links, 42 joints
Links:
- link camera_link: geometry visual mesh filename=package://sensor_models/meshes/realsense/d435.glb

File: humanoid/Realman/aidal_description/urdf/aidal_eg2-4c2.urdf (robot description, URDF)
Before this commit: robot RealMan_AIDAL, 57 links, 56 joints
Links:
- link camera_link: geometry visual mesh filename=package://sensor_models/meshes/realsense/d435.glb
