Commit message: add galaxea r1 lite

File: manipulator/Galaxea/galaxea_a1_description/xacro/a1.xacro (robot description, xacro)
@@ -18,10 +18,10 @@
       <visual>
         <geometry>
-          <mesh filename="file://$(find galaxea_a1_description)/meshes/a1/base_link.obj"/>
-        </geometry>
-      </visual>
-      <collision>
-        <geometry>
-          <mesh filename="file://$(find galaxea_a1_description)/meshes/a1/base_link.obj"/>
+          <mesh filename="file://$(find galaxea_a1_description)/meshes/a1/visual/base_link.obj"/>
+        </geometry>
+      </visual>
+      <collision>
+        <geometry>
+          <mesh filename="file://$(find galaxea_a1_description)/meshes/a1/visual/base_link.obj"/>
         </geometry>
       </collision>
@@ -42,10 +42,10 @@
       <visual>
         <geometry>
-          <mesh filename="file://$(find galaxea_a1_description)/meshes/a1/link1.obj"/>
-        </geometry>
-      </visual>
-      <collision>
-        <geometry>
-          <mesh filename="file://$(find galaxea_a1_description)/meshes/a1/link1.obj"/>
+          <mesh filename="file://$(find galaxea_a1_description)/meshes/a1/visual/link1.obj"/>
+        </geometry>
+      </visual>
+      <collision>
+        <geometry>
+          <mesh filename="file://$(find galaxea_a1_description)/meshes/a1/visual/link1.obj"/>
         </geometry>
       </collision>
@@ -74,10 +74,10 @@
       <visual>
         <geometry>
-          <mesh filename="file://$(find galaxea_a1_description)/meshes/a1/link2.obj"/>
-        </geometry>
-      </visual>
-      <collision>
-        <geometry>
-          <mesh filename="file://$(find galaxea_a1_description)/meshes/a1/link2.obj"/>
+          <mesh filename="file://$(find galaxea_a1_description)/meshes/a1/visual/link2.obj"/>
+        </geometry>
+      </visual>
+      <collision>
+        <geometry>
+          <mesh filename="file://$(find galaxea_a1_description)/meshes/a1/visual/link2.obj"/>
         </geometry>
       </collision>
@@ -106,10 +106,10 @@
       <visual>
         <geometry>
-          <mesh filename="file://$(find galaxea_a1_description)/meshes/a1/link3.obj"/>
-        </geometry>
-      </visual>
-      <collision>
-        <geometry>
-          <mesh filename="file://$(find galaxea_a1_description)/meshes/a1/link3.obj"/>
+          <mesh filename="file://$(find galaxea_a1_description)/meshes/a1/visual/link3.obj"/>
+        </geometry>
+      </visual>
+      <collision>
+        <geometry>
+          <mesh filename="file://$(find galaxea_a1_description)/meshes/a1/visual/link3.obj"/>
         </geometry>
       </collision>
@@ -138,10 +138,10 @@
       <visual>
         <geometry>
-          <mesh filename="file://$(find galaxea_a1_description)/meshes/a1/link4.obj"/>
-        </geometry>
-      </visual>
-      <collision>
-        <geometry>
-          <mesh filename="file://$(find galaxea_a1_description)/meshes/a1/link4.obj"/>
+          <mesh filename="file://$(find galaxea_a1_description)/meshes/a1/visual/link4.obj"/>
+        </geometry>
+      </visual>
+      <collision>
+        <geometry>
+          <mesh filename="file://$(find galaxea_a1_description)/meshes/a1/visual/link4.obj"/>
         </geometry>
       </collision>
@@ -170,10 +170,10 @@
       <visual>
         <geometry>
-          <mesh filename="file://$(find galaxea_a1_description)/meshes/a1/link5.obj"/>
-        </geometry>
-      </visual>
-      <collision>
-        <geometry>
-          <mesh filename="file://$(find galaxea_a1_description)/meshes/a1/link5.obj"/>
+          <mesh filename="file://$(find galaxea_a1_description)/meshes/a1/visual/link5.obj"/>
+        </geometry>
+      </visual>
+      <collision>
+        <geometry>
+          <mesh filename="file://$(find galaxea_a1_description)/meshes/a1/visual/link5.obj"/>
         </geometry>
       </collision>
@@ -202,10 +202,10 @@
       <visual>
         <geometry>
-          <mesh filename="file://$(find galaxea_a1_description)/meshes/a1/link6.obj"/>
-        </geometry>
-      </visual>
-      <collision>
-        <geometry>
-          <mesh filename="file://$(find galaxea_a1_description)/meshes/a1/link6.obj"/>
+          <mesh filename="file://$(find galaxea_a1_description)/meshes/a1/visual/link6.obj"/>
+        </geometry>
+      </visual>
+      <collision>
+        <geometry>
+          <mesh filename="file://$(find galaxea_a1_description)/meshes/a1/visual/link6.obj"/>
         </geometry>
       </collision>

Commit message: update galaxea mesh

File: manipulator/Galaxea/galaxea_a1_description/xacro/a1.xacro (robot description, xacro)
@@ -19,10 +19,10 @@
       <visual>
         <geometry>
-          <mesh filename="file://$(find galaxea_a1_description)/meshes/a1/visual/base_link.obj"/>
-        </geometry>
-      </visual>
-      <collision>
-        <geometry>
-          <mesh filename="file://$(find galaxea_a1_description)/meshes/a1/visual/base_link.obj"/>
+          <mesh filename="file://$(find galaxea_a1_description)/meshes/a1/base.glb"/>
+        </geometry>
+      </visual>
+      <collision>
+        <geometry>
+          <mesh filename="file://$(find galaxea_a1_description)/meshes/a1/base.glb"/>
         </geometry>
       </collision>
@@ -43,10 +43,10 @@
       <visual>
         <geometry>
-          <mesh filename="file://$(find galaxea_a1_description)/meshes/a1/visual/link1.obj"/>
-        </geometry>
-      </visual>
-      <collision>
-        <geometry>
-          <mesh filename="file://$(find galaxea_a1_description)/meshes/a1/visual/link1.obj"/>
+          <mesh filename="file://$(find galaxea_a1_description)/meshes/a1/link1.glb"/>
+        </geometry>
+      </visual>
+      <collision>
+        <geometry>
+          <mesh filename="file://$(find galaxea_a1_description)/meshes/a1/link1.glb"/>
         </geometry>
       </collision>
@@ -75,10 +75,10 @@
       <visual>
         <geometry>
-          <mesh filename="file://$(find galaxea_a1_description)/meshes/a1/visual/link2.obj"/>
-        </geometry>
-      </visual>
-      <collision>
-        <geometry>
-          <mesh filename="file://$(find galaxea_a1_description)/meshes/a1/visual/link2.obj"/>
+          <mesh filename="file://$(find galaxea_a1_description)/meshes/a1/link2.glb"/>
+        </geometry>
+      </visual>
+      <collision>
+        <geometry>
+          <mesh filename="file://$(find galaxea_a1_description)/meshes/a1/link2.glb"/>
         </geometry>
       </collision>
@@ -107,10 +107,10 @@
       <visual>
         <geometry>
-          <mesh filename="file://$(find galaxea_a1_description)/meshes/a1/visual/link3.obj"/>
-        </geometry>
-      </visual>
-      <collision>
-        <geometry>
-          <mesh filename="file://$(find galaxea_a1_description)/meshes/a1/visual/link3.obj"/>
+          <mesh filename="file://$(find galaxea_a1_description)/meshes/a1/link3.glb"/>
+        </geometry>
+      </visual>
+      <collision>
+        <geometry>
+          <mesh filename="file://$(find galaxea_a1_description)/meshes/a1/link3.glb"/>
         </geometry>
       </collision>
@@ -139,10 +139,10 @@
       <visual>
         <geometry>
-          <mesh filename="file://$(find galaxea_a1_description)/meshes/a1/visual/link4.obj"/>
-        </geometry>
-      </visual>
-      <collision>
-        <geometry>
-          <mesh filename="file://$(find galaxea_a1_description)/meshes/a1/visual/link4.obj"/>
+          <mesh filename="file://$(find galaxea_a1_description)/meshes/a1/link4.glb"/>
+        </geometry>
+      </visual>
+      <collision>
+        <geometry>
+          <mesh filename="file://$(find galaxea_a1_description)/meshes/a1/link4.glb"/>
         </geometry>
       </collision>
@@ -171,10 +171,10 @@
       <visual>
         <geometry>
-          <mesh filename="file://$(find galaxea_a1_description)/meshes/a1/visual/link5.obj"/>
-        </geometry>
-      </visual>
-      <collision>
-        <geometry>
-          <mesh filename="file://$(find galaxea_a1_description)/meshes/a1/visual/link5.obj"/>
+          <mesh filename="file://$(find galaxea_a1_description)/meshes/a1/link5.glb"/>
+        </geometry>
+      </visual>
+      <collision>
+        <geometry>
+          <mesh filename="file://$(find galaxea_a1_description)/meshes/a1/link5.glb"/>
         </geometry>
       </collision>
@@ -203,10 +203,10 @@
       <visual>
         <geometry>
-          <mesh filename="file://$(find galaxea_a1_description)/meshes/a1/visual/link6.obj"/>
-        </geometry>
-      </visual>
-      <collision>
-        <geometry>
-          <mesh filename="file://$(find galaxea_a1_description)/meshes/a1/visual/link6.obj"/>
+          <mesh filename="file://$(find galaxea_a1_description)/meshes/a1/link6.glb"/>
+        </geometry>
+      </visual>
+      <collision>
+        <geometry>
+          <mesh filename="file://$(find galaxea_a1_description)/meshes/a1/link6.glb"/>
         </geometry>
       </collision>

File: manipulator/Galaxea/galaxea_a1_description/xacro/a1_x.xacro (robot description, xacro)
@@ -20,10 +20,10 @@
       <visual>
         <geometry>
-          <mesh filename="file://$(find galaxea_a1_description)/meshes/a1_xy/a1_x/link3.obj"/>
+          <mesh filename="file://$(find galaxea_a1_description)/meshes/a1_xy/a1_x/link3.glb"/>
         </geometry>
       </visual>
       <collision>
         <geometry>
-          <mesh filename="file://$(find galaxea_a1_description)/meshes/a1_xy/a1_x/link3.obj"/>
+          <mesh filename="file://$(find galaxea_a1_description)/meshes/a1_xy/a1_x/link3.glb"/>
         </geometry>
       </collision>
@@ -50,10 +50,10 @@
       <visual>
         <geometry>
-          <mesh filename="file://$(find galaxea_a1_description)/meshes/a1_xy/a1_x/link4.obj"/>
+          <mesh filename="file://$(find galaxea_a1_description)/meshes/a1_xy/a1_x/link4.glb"/>
         </geometry>
       </visual>
       <collision>
         <geometry>
-          <mesh filename="file://$(find galaxea_a1_description)/meshes/a1_xy/a1_x/link4.obj"/>
+          <mesh filename="file://$(find galaxea_a1_description)/meshes/a1_xy/a1_x/link4.glb"/>
         </geometry>
       </collision>
@@ -80,10 +80,10 @@
       <visual>
         <geometry>
-          <mesh filename="file://$(find galaxea_a1_description)/meshes/a1_xy/a1_x/link5.obj"/>
+          <mesh filename="file://$(find galaxea_a1_description)/meshes/a1_xy/a1_x/link5.glb"/>
         </geometry>
       </visual>
       <collision>
         <geometry>
-          <mesh filename="file://$(find galaxea_a1_description)/meshes/a1_xy/a1_x/link5.obj"/>
+          <mesh filename="file://$(find galaxea_a1_description)/meshes/a1_xy/a1_x/link5.glb"/>
         </geometry>
       </collision>
@@ -110,10 +110,10 @@
       <visual>
         <geometry>
-          <mesh filename="file://$(find galaxea_a1_description)/meshes/a1_xy/link6.obj"/>
+          <mesh filename="file://$(find galaxea_a1_description)/meshes/a1_xy/link6.glb"/>
         </geometry>
       </visual>
       <collision>
         <geometry>
-          <mesh filename="file://$(find galaxea_a1_description)/meshes/a1_xy/link6.obj"/>
+          <mesh filename="file://$(find galaxea_a1_description)/meshes/a1_xy/link6.glb"/>
         </geometry>
       </collision>

File: manipulator/Galaxea/galaxea_a1_description/xacro/a1_y.xacro (robot description, xacro)
@@ -20,10 +20,10 @@
 			<visual>
 				<geometry>
-					<mesh filename="file://$(find galaxea_a1_description)/meshes/a1_xy/a1_y/link3.obj"/>
+					<mesh filename="file://$(find galaxea_a1_description)/meshes/a1_xy/a1_y/link3.glb"/>
 				</geometry>
 			</visual>
 			<collision>
 				<geometry>
-					<mesh filename="file://$(find galaxea_a1_description)/meshes/a1_xy/a1_y/link3.obj"/>
+					<mesh filename="file://$(find galaxea_a1_description)/meshes/a1_xy/a1_y/link3.glb"/>
 				</geometry>
 			</collision>
@@ -50,10 +50,10 @@
 			<visual>
 				<geometry>
-					<mesh filename="file://$(find galaxea_a1_description)/meshes/a1_xy/a1_y/link4.obj"/>
+					<mesh filename="file://$(find galaxea_a1_description)/meshes/a1_xy/a1_y/link4.glb"/>
 				</geometry>
 			</visual>
 			<collision>
 				<geometry>
-					<mesh filename="file://$(find galaxea_a1_description)/meshes/a1_xy/a1_y/link4.obj"/>
+					<mesh filename="file://$(find galaxea_a1_description)/meshes/a1_xy/a1_y/link4.glb"/>
 				</geometry>
 			</collision>
@@ -80,10 +80,10 @@
 			<visual>
 				<geometry>
-					<mesh filename="file://$(find galaxea_a1_description)/meshes/a1_xy/a1_y/link5.obj"/>
+					<mesh filename="file://$(find galaxea_a1_description)/meshes/a1_xy/a1_y/link5.glb"/>
 				</geometry>
 			</visual>
 			<collision>
 				<geometry>
-					<mesh filename="file://$(find galaxea_a1_description)/meshes/a1_xy/a1_y/link5.obj"/>
+					<mesh filename="file://$(find galaxea_a1_description)/meshes/a1_xy/a1_y/link5.glb"/>
 				</geometry>
 			</collision>
@@ -110,10 +110,10 @@
 			<visual>
 				<geometry>
-					<mesh filename="file://$(find galaxea_a1_description)/meshes/a1_xy/link6.obj"/>
+					<mesh filename="file://$(find galaxea_a1_description)/meshes/a1_xy/link6.glb"/>
 				</geometry>
 			</visual>
 			<collision>
 				<geometry>
-					<mesh filename="file://$(find galaxea_a1_description)/meshes/a1_xy/link6.obj"/>
+					<mesh filename="file://$(find galaxea_a1_description)/meshes/a1_xy/link6.glb"/>
 				</geometry>
 			</collision>

File: manipulator/Galaxea/galaxea_a1_description/xacro/a1xy_base.xacro (robot description, xacro)
@@ -17,10 +17,10 @@
 			<visual>
 				<geometry>
-					<mesh filename="file://$(find galaxea_a1_description)/meshes/a1_xy/base_link.obj"/>
+					<mesh filename="file://$(find galaxea_a1_description)/meshes/a1_xy/base.glb"/>
 				</geometry>
 			</visual>
 			<collision>
 				<geometry>
-					<mesh filename="file://$(find galaxea_a1_description)/meshes/a1_xy/base_link.obj"/>
+					<mesh filename="file://$(find galaxea_a1_description)/meshes/a1_xy/base.glb"/>
 				</geometry>
 			</collision>
@@ -41,10 +41,10 @@
 			<visual>
 				<geometry>
-					<mesh filename="file://$(find galaxea_a1_description)/meshes/a1_xy/link1.obj"/>
+					<mesh filename="file://$(find galaxea_a1_description)/meshes/a1_xy/link1.glb"/>
 				</geometry>
 			</visual>
 			<collision>
 				<geometry>
-					<mesh filename="file://$(find galaxea_a1_description)/meshes/a1_xy/link1.obj"/>
+					<mesh filename="file://$(find galaxea_a1_description)/meshes/a1_xy/link1.glb"/>
 				</geometry>
 			</collision>
@@ -73,10 +73,10 @@
 			<visual>
 				<geometry>
-					<mesh filename="file://$(find galaxea_a1_description)/meshes/a1_xy/link2.obj"/>
+					<mesh filename="file://$(find galaxea_a1_description)/meshes/a1_xy/link2.glb"/>
 				</geometry>
 			</visual>
 			<collision>
 				<geometry>
-					<mesh filename="file://$(find galaxea_a1_description)/meshes/a1_xy/link2.obj"/>
+					<mesh filename="file://$(find galaxea_a1_description)/meshes/a1_xy/link2.glb"/>
 				</geometry>
 			</collision>

File: manipulator/Galaxea/galaxea_a1_description/xacro/gripper_g1.xacro (robot description, xacro)
@@ -18,10 +18,10 @@
       <visual>
         <geometry>
-          <mesh filename="file://$(find galaxea_a1_description)/meshes/gripper/gripper_link.obj"/>
+          <mesh filename="file://$(find galaxea_a1_description)/meshes/gripper/gripper_base.glb"/>
         </geometry>
       </visual>
       <collision>
         <geometry>
-          <mesh filename="file://$(find galaxea_a1_description)/meshes/gripper/gripper_link.obj"/>
+          <mesh filename="file://$(find galaxea_a1_description)/meshes/gripper/gripper_base.glb"/>
         </geometry>
       </collision>
@@ -41,10 +41,10 @@
       <visual>
         <geometry>
-          <mesh filename="file://$(find galaxea_a1_description)/meshes/gripper/finger.obj"/>
+          <mesh filename="file://$(find galaxea_a1_description)/meshes/gripper/finger.glb"/>
         </geometry>
       </visual>
       <collision>
         <geometry>
-          <mesh filename="file://$(find galaxea_a1_description)/meshes/gripper/finger.obj"/>
+          <mesh filename="file://$(find galaxea_a1_description)/meshes/gripper/finger.glb"/>
         </geometry>
       </collision>
@@ -71,10 +71,10 @@
       <visual>
         <geometry>
-          <mesh filename="file://$(find galaxea_a1_description)/meshes/gripper/finger.obj" scale="1 -1 -1"/>
+          <mesh filename="file://$(find galaxea_a1_description)/meshes/gripper/finger.glb" scale="1 -1 -1"/>
         </geometry>
       </visual>
       <collision>
         <geometry>
-          <mesh filename="file://$(find galaxea_a1_description)/meshes/gripper/finger.obj" scale="1 -1 -1"/>
+          <mesh filename="file://$(find galaxea_a1_description)/meshes/gripper/finger.glb" scale="1 -1 -1"/>
         </geometry>
       </collision>
