Commit message: Add Galaxea_A1Z without gripper G1Z

File: manipulator/Galaxea/galaxea_a1_description/xacro/robot.xacro (robot description, xacro)
@@ -12,4 +12,7 @@
     <xacro:include filename="$(find galaxea_a1_description)/xacro/a1_y.xacro"/>
   </xacro:if>
+  <xacro:if value="${'$(arg type)' == 'z'}">
+    <xacro:include filename="$(find galaxea_a1_description)/xacro/a1_z.xacro"/>
+  </xacro:if>
   <xacro:Arm name=""/>
 </robot>

File: manipulator/Galaxea/galaxea_a1_description/xacro/ros2_control/interfaces.xacro (robot description, xacro)
@@ -1,5 +1,5 @@
 <?xml version="1.0"?>
 <robot xmlns:xacro="http://www.ros.org/wiki/xacro">
-	<xacro:macro name="galaxea_a1_interfaces" params="name">
+	<xacro:macro name="galaxea_a1_interfaces" params="name include_gripper:=true">
 		<xacro:property name="prefix" value="${name + '_' if name else ''}"/>
 		<xacro:arg name="gazebo" default="false"/>
@@ -41,18 +41,20 @@
 			<state_interface name="effort"/>
 		</joint>
-		<joint name="${prefix}gripper_joint">
-			<command_interface name="position"/>
-			<state_interface name="position">
-				<param name="initial_value">0.01</param>
-			</state_interface>
-			<state_interface name="velocity"/>
-			<state_interface name="effort"/>
-		</joint>
-		<xacro:if value="$(arg gazebo)">
-			<joint name="${prefix}gripper_joint2">
-				<state_interface name="position"/>
+		<xacro:if value="${include_gripper}">
+			<joint name="${prefix}gripper_joint">
+				<command_interface name="position"/>
+				<state_interface name="position">
+					<param name="initial_value">0.01</param>
+				</state_interface>
 				<state_interface name="velocity"/>
 				<state_interface name="effort"/>
 			</joint>
+			<xacro:if value="$(arg gazebo)">
+				<joint name="${prefix}gripper_joint2">
+					<state_interface name="position"/>
+					<state_interface name="velocity"/>
+					<state_interface name="effort"/>
+				</joint>
+			</xacro:if>
 		</xacro:if>
 	</xacro:macro>

File: manipulator/Galaxea/galaxea_a1_description/xacro/ros2_control/robot.xacro (robot description, xacro)
@@ -22,5 +22,5 @@
       </xacro:if>
     </hardware>
-    <xacro:galaxea_a1_interfaces name=""/>
+    <xacro:galaxea_a1_interfaces name="" include_gripper="${'$(arg type)' != 'z'}"/>
   </ros2_control>
   <xacro:arg name="gazebo" default="false" />
@@ -37,4 +37,7 @@
           <parameters>$(find galaxea_a1_description)/config/ros2_control/y.yaml</parameters>
         </xacro:if>
+        <xacro:if value="${'$(arg type)' == 'z'}">
+          <parameters>$(find galaxea_a1_description)/config/ros2_control/z.yaml</parameters>
+        </xacro:if>
       </plugin>
     </gazebo>
