Commit message: Add Galaxea_A1Z Complete with ocs2 test.

File: manipulator/Galaxea/galaxea_a1_description/xacro/a1_z.xacro (robot description, xacro)
@@ -208,10 +208,11 @@
       <limit lower="-2.007" upper="2.007" effort="3.5" velocity="10.47"/>
     </joint>
-    <!-- Flange TCP placeholder for OCS2 (eeFrame). Replace when gripper is added. -->
-    <link name="${prefix}gripper_center"/>
-    <joint name="${prefix}gripper_center_joint" type="fixed">
+    <xacro:include filename="$(find galaxea_a1_description)/xacro/gripper_g1z.xacro"/>
+    <xacro:Gripper name="${name}"/>
+    <!-- Mount on flange (link6) at identity. -->
+    <joint name="${prefix}gripper_base_joint" type="fixed">
       <origin xyz="0 0 0"/>
       <parent link="${prefix}link6"/>
-      <child link="${prefix}gripper_center"/>
+      <child link="${prefix}gripper_base"/>
     </joint>
   </xacro:macro>

File: manipulator/Galaxea/galaxea_a1_description/xacro/gripper.xacro (robot description, xacro)
@@ -1,5 +1,11 @@
 <?xml version="1.0"?>
-<robot name="Galaxea_G1" xmlns:xacro="http://www.ros.org/wiki/xacro">
-  <xacro:include filename="$(find galaxea_a1_description)/xacro/gripper_g1.xacro"/>
+<robot name="Galaxea_Gripper" xmlns:xacro="http://www.ros.org/wiki/xacro">
+  <xacro:arg name="type" default="g1"/>
+  <xacro:if value="${'$(arg type)' == 'g1'}">
+    <xacro:include filename="$(find galaxea_a1_description)/xacro/gripper_g1.xacro"/>
+  </xacro:if>
+  <xacro:if value="${'$(arg type)' == 'g1z'}">
+    <xacro:include filename="$(find galaxea_a1_description)/xacro/gripper_g1z.xacro"/>
+  </xacro:if>
   <xacro:Gripper name=""/>
 </robot>

File: manipulator/Galaxea/galaxea_a1_description/xacro/ros2_control/robot.xacro (robot description, xacro)
@@ -22,5 +22,5 @@
       </xacro:if>
     </hardware>
-    <xacro:galaxea_a1_interfaces name="" include_gripper="${'$(arg type)' != 'z'}"/>
+    <xacro:galaxea_a1_interfaces name=""/>
   </ros2_control>
   <xacro:arg name="gazebo" default="false" />
