Commit message: update mesh to glb for astribot s1

File: humanoid/Astribot/astribot_s1_description/xacro/components/base.xacro (robot description, xacro)
@@ -15,5 +15,5 @@
 			<visual>
 				<geometry>
-					<mesh filename="file://$(find astribot_s1_description)/meshes/s1_torso/base.obj"/>
+					<mesh filename="file://$(find astribot_s1_description)/meshes/s1_torso/base.glb"/>
 				</geometry>
 			</visual>
@@ -90,5 +90,5 @@
 			<visual>
 				<geometry>
-					<mesh filename="file://$(find astribot_s1_description)/meshes/s1_torso/link1.obj"/>
+					<mesh filename="file://$(find astribot_s1_description)/meshes/s1_torso/link1.glb"/>
 				</geometry>
 				<material name="">
@@ -119,5 +119,5 @@
 			<visual>
 				<geometry>
-					<mesh filename="file://$(find astribot_s1_description)/meshes/s1_torso/link2.obj"/>
+					<mesh filename="file://$(find astribot_s1_description)/meshes/s1_torso/link2.glb"/>
 				</geometry>
 				<material name="">
@@ -149,5 +149,5 @@
 			<visual>
 				<geometry>
-					<mesh filename="file://$(find astribot_s1_description)/meshes/s1_torso/link3.obj"/>
+					<mesh filename="file://$(find astribot_s1_description)/meshes/s1_torso/link3.glb"/>
 				</geometry>
 			</visual>
@@ -177,5 +177,5 @@
 			<visual>
 				<geometry>
-					<mesh filename="file://$(find astribot_s1_description)/meshes/s1_torso/link4.obj"/>
+					<mesh filename="file://$(find astribot_s1_description)/meshes/s1_torso/link4.glb"/>
 				</geometry>
 			</visual>
@@ -210,5 +210,5 @@
 			<visual>
 				<geometry>
-					<mesh filename="file://$(find astribot_s1_description)/meshes/s1_head/base.obj"/>
+					<mesh filename="file://$(find astribot_s1_description)/meshes/s1_head/base.glb"/>
 				</geometry>
 			</visual>
@@ -229,5 +229,5 @@
 			<visual>
 				<geometry>
-					<mesh filename="file://$(find astribot_s1_description)/meshes/s1_head/link1.obj"/>
+					<mesh filename="file://$(find astribot_s1_description)/meshes/s1_head/link1.glb"/>
 				</geometry>
 			</visual>
@@ -249,5 +249,5 @@
 			<visual>
 				<geometry>
-					<mesh filename="file://$(find astribot_s1_description)/meshes/s1_head/link2.obj"/>
+					<mesh filename="file://$(find astribot_s1_description)/meshes/s1_head/link2.glb"/>
 				</geometry>
 			</visual>

Commit message: test pass for galaxea and astribot

File: humanoid/Astribot/astribot_s1_description/xacro/components/base.xacro (robot description, xacro)
@@ -103,5 +103,5 @@
 			</collision>
 		</link>
-		<joint name="torso_joint_1" type="revolute">
+		<joint name="body_joint1" type="revolute">
 			<origin rpy="-1.5708 1.5708 0" xyz="0 0 0.12"/>
 			<parent link="base_link"/>
@@ -132,5 +132,5 @@
 			</collision>
 		</link>
-		<joint name="torso_joint_2" type="revolute">
+		<joint name="body_joint2" type="revolute">
 			<origin xyz="-0.38 0 0"/>
 			<parent link="torso_link_1"/>
@@ -159,5 +159,5 @@
 			</collision>
 		</link>
-		<joint name="torso_joint_3" type="revolute">
+		<joint name="body_joint3" type="revolute">
 			<origin xyz="-0.390 0 0"/>
 			<parent link="torso_link_2"/>
@@ -181,5 +181,5 @@
 			</visual>
 		</link>
-		<joint name="torso_joint_4" type="revolute">
+		<joint name="body_joint4" type="revolute">
 			<origin rpy="1.5708 0 -1.5708" xyz="0 0 0"/>
 			<parent link="torso_link_3"/>
@@ -219,6 +219,6 @@
 			<origin xyz="0 0 0.1229"/>
 		</joint>
-		<!-- 头部连杆1 -->
-		<link name="head_link_1">
+		<!-- 头部连杆1（head_joint1） -->
+		<link name="head_link1">
 			<inertial>
 				<origin xyz="0.00003191 -0.00038566 -0.02579910"/>
@@ -233,12 +233,12 @@
 			</visual>
 		</link>
-		<joint name="head_joint_1" type="revolute">
+		<joint name="head_joint1" type="revolute">
 			<parent link="head_base_link"/>
-			<child link="head_link_1"/>
+			<child link="head_link1"/>
 			<axis xyz="0 0 1"/>
 			<limit effort="100" lower="-1.57" upper="1.57" velocity="4.0"/>
 		</joint>
-		<!-- 头部连杆2 -->
-		<link name="head_link_2">
+		<!-- 头部连杆2（head_joint2） -->
+		<link name="head_link2">
 			<inertial>
 				<origin xyz="0.00705824 -0.14472601 -0.00061724"/>
@@ -259,8 +259,8 @@
 			</collision>
 		</link>
-		<joint name="head_joint_2" type="revolute">
+		<joint name="head_joint2" type="revolute">
 			<origin rpy="-1.5708 0 0" xyz="0 0 0"/>
-			<parent link="head_link_1"/>
-			<child link="head_link_2"/>
+			<parent link="head_link1"/>
+			<child link="head_link2"/>
 			<axis xyz="0 0 1"/>
 			<limit effort="100" lower="-1.22" upper="1.22" velocity="4.0"/>

File: humanoid/Astribot/astribot_s1_description/xacro/components/s1_arm.xacro (robot description, xacro)
@@ -32,5 +32,5 @@
 			</visual>
 		</link>
-		<link name="${prefix}link_1">
+		<link name="${prefix}link1">
 			<inertial>
 				<origin xyz="0.00012026 0.00047499 -0.05682561"/>
@@ -44,12 +44,12 @@
 			</visual>
 		</link>
-		<joint name="${prefix}joint_1" type="revolute">
+		<joint name="${prefix}joint1" type="revolute">
 			<origin xyz="0 0 0.091"/>
 			<parent link="${prefix}base_link"/>
-			<child link="${prefix}link_1"/>
+			<child link="${prefix}link1"/>
 			<axis xyz="0 0 1"/>
 			<limit effort="265" lower="-3.1" upper="3.1" velocity="8.4"/>
 		</joint>
-		<link name="${prefix}link_2">
+		<link name="${prefix}link2">
 			<inertial>
 				<!-- Left: xyz="-0.00396228 0.03490708 0.04270156" mass="1.43694657" -->
@@ -74,12 +74,12 @@
 			</visual>
 		</link>
-		<joint name="${prefix}joint_2" type="revolute">
+		<joint name="${prefix}joint2" type="revolute">
 			<origin rpy="1.5708 0 0"/>
-			<parent link="${prefix}link_1"/>
-			<child link="${prefix}link_2"/>
+			<parent link="${prefix}link1"/>
+			<child link="${prefix}link2"/>
 			<axis xyz="0 0 1"/>
 			<limit effort="265" lower="-1.53" upper="0.46" velocity="8.4"/>
 		</joint>
-		<link name="${prefix}link_3">
+		<link name="${prefix}link3">
 			<inertial>
 				<origin xyz="0.00531263 0.00020707 0.16136713"/>
@@ -99,12 +99,12 @@
 			</collision>
 		</link>
-		<joint name="${prefix}joint_3" type="revolute">
+		<joint name="${prefix}joint3" type="revolute">
 			<origin rpy="1.5708 0 -1.5708" xyz="0 0.05 0"/>
-			<parent link="${prefix}link_2"/>
-			<child link="${prefix}link_3"/>
+			<parent link="${prefix}link2"/>
+			<child link="${prefix}link3"/>
 			<axis xyz="0 0 1"/>
 			<limit effort="132" lower="-3.1" upper="3.1" velocity="8.4"/>
 		</joint>
-		<link name="${prefix}link_4">
+		<link name="${prefix}link4">
 			<inertial>
 				<origin xyz="0.00017294 -0.01269315 0.00196140"/>
@@ -124,8 +124,8 @@
 			</collision>
 		</link>
-		<joint name="${prefix}joint_4" type="revolute">
+		<joint name="${prefix}joint4" type="revolute">
 			<origin rpy="-1.5708 0 0" xyz="0.03 0 0.309"/>
-			<parent link="${prefix}link_3"/>
-			<child link="${prefix}link_4"/>
+			<parent link="${prefix}link3"/>
+			<child link="${prefix}link4"/>
 			<axis xyz="0 0 1"/>
 			<limit effort="142" lower="-0.06" upper="2.61" velocity="15"/>
@@ -134,5 +134,5 @@
 		<!-- Link 5 - Shared mesh                                                              -->
 		<!-- =================================================================================== -->
-		<link name="${prefix}link_5">
+		<link name="${prefix}link5">
 			<inertial>
 				<origin xyz="-0.00032037 -0.00015185 0.15370447"/>
@@ -155,12 +155,12 @@
 			</collision>
 		</link>
-		<joint name="${prefix}joint_5" type="revolute">
+		<joint name="${prefix}joint5" type="revolute">
 			<origin rpy="1.5708 0 0"/>
-			<parent link="${prefix}link_4"/>
-			<child link="${prefix}link_5"/>
+			<parent link="${prefix}link4"/>
+			<child link="${prefix}link5"/>
 			<axis xyz="0 0 1"/>
 			<limit effort="71" lower="-2.56" upper="2.56" velocity="20"/>
 		</joint>
-		<link name="${prefix}link_6">
+		<link name="${prefix}link6">
 			<inertial>
 				<origin xyz="-0.00010311 0.00001218 0.00013181"/>
@@ -174,12 +174,12 @@
 			</visual>
 		</link>
-		<joint name="${prefix}joint_6" type="revolute">
+		<joint name="${prefix}joint6" type="revolute">
 			<origin rpy="-1.5708 0 0" xyz="0 0 0.277"/>
-			<parent link="${prefix}link_5"/>
-			<child link="${prefix}link_6"/>
+			<parent link="${prefix}link5"/>
+			<child link="${prefix}link6"/>
 			<axis xyz="0 0 1"/>
 			<limit effort="20" lower="-0.76" upper="0.76" velocity="16.8"/>
 		</joint>
-		<link name="${prefix}link_7">
+		<link name="${prefix}link7">
 			<inertial>
 				<origin xyz="4.333e-05 -0.00723447 -0.00362428"/>
@@ -199,8 +199,8 @@
 			</collision>
 		</link>
-		<joint name="${prefix}joint_7" type="revolute">
+		<joint name="${prefix}joint7" type="revolute">
 			<origin rpy="0 1.5708 0"/>
-			<parent link="${prefix}link_6"/>
-			<child link="${prefix}link_7"/>
+			<parent link="${prefix}link6"/>
+			<child link="${prefix}link7"/>
 			<axis xyz="0 0 1"/>
 			<limit effort="20" lower="-1.53" upper="1.53" velocity="16.8"/>

File: humanoid/Astribot/astribot_s1_description/xacro/components/s1_gripper.xacro (robot description, xacro)
@@ -5,6 +5,7 @@
 <!-- =================================================================================== -->
 <robot xmlns:xacro="http://www.ros.org/wiki/xacro">
-	<xacro:macro name="Gripper" params="name">
+	<xacro:macro name="Gripper" params="name kinematic_only:=false">
 		<xacro:property name="prefix" value="${name + '_' if name else ''}"/>
+		<xacro:property name="finger_joint_type" value="${kinematic_only and 'fixed' or 'revolute'}"/>
 		<!-- 夹爪基座 -->
 		<link name="${prefix}gripper_base">
@@ -45,10 +46,12 @@
 			</visual>
 		</link>
-		<joint name="${prefix}gripper_joint" type="revolute">
+		<joint name="${prefix}gripper_joint" type="${finger_joint_type}">
 			<origin xyz="0.0145 0 0.0510999999999999"/>
 			<parent link="${prefix}gripper_base"/>
 			<child link="${prefix}gripper_L1"/>
-			<axis xyz="0 -1 0"/>
-			<limit lower="0" upper="1" effort="10" velocity="1"/>
+			<xacro:unless value="${kinematic_only}">
+				<axis xyz="0 -1 0"/>
+				<limit lower="0" upper="1" effort="10" velocity="1"/>
+			</xacro:unless>
 		</joint>
 		<!-- 夹爪左侧手指 L2 -->
@@ -71,11 +74,13 @@
 			</visual>
 		</link>
-		<joint name="${prefix}gripper_joint_L2" type="revolute">
+		<joint name="${prefix}gripper_joint_L2" type="${finger_joint_type}">
 			<origin xyz="0.0325 0 0.0510999999999999"/>
 			<parent link="${prefix}gripper_base"/>
 			<child link="${prefix}gripper_L2"/>
-			<axis xyz="0 -1 0"/>
-			<limit lower="-1.57" upper="1.57" effort="10" velocity="1"/>
-			<mimic joint="${prefix}gripper_joint" multiplier="1.0" offset="0.0"/>
+			<xacro:unless value="${kinematic_only}">
+				<axis xyz="0 -1 0"/>
+				<limit lower="-1.57" upper="1.57" effort="10" velocity="1"/>
+				<mimic joint="${prefix}gripper_joint" multiplier="1.0" offset="0.0"/>
+			</xacro:unless>
 		</joint>
 		<!-- 夹爪左侧手指 L11 (末端) -->
@@ -103,11 +108,13 @@
 			</collision>
 		</link>
-		<joint name="${prefix}gripper_joint_L11" type="revolute">
+		<joint name="${prefix}gripper_joint_L11" type="${finger_joint_type}">
 			<origin xyz="0.0412500000000001 0 0.036379080527138"/>
 			<parent link="${prefix}gripper_L1"/>
 			<child link="${prefix}gripper_L11"/>
-			<axis xyz="0 1 0"/>
-			<limit effort="10" velocity="1" lower="-1.57" upper="1.57"/>
-			<mimic joint="${prefix}gripper_joint" multiplier="1.0" offset="0.0"/>
+			<xacro:unless value="${kinematic_only}">
+				<axis xyz="0 1 0"/>
+				<limit effort="10" velocity="1" lower="-1.57" upper="1.57"/>
+				<mimic joint="${prefix}gripper_joint" multiplier="1.0" offset="0.0"/>
+			</xacro:unless>
 		</joint>
 		<!-- 夹爪右侧手指 R1 -->
@@ -130,11 +137,13 @@
 			</visual>
 		</link>
-		<joint name="${prefix}gripper_joint_R1" type="revolute">
+		<joint name="${prefix}gripper_joint_R1" type="${finger_joint_type}">
 			<origin xyz="-0.0144999999999999 0 0.0510999999999939"/>
 			<parent link="${prefix}gripper_base"/>
 			<child link="${prefix}gripper_R1"/>
-			<axis xyz="0 1 0"/>
-			<limit lower="-1.57" upper="1.57" effort="10" velocity="1"/>
-			<mimic joint="${prefix}gripper_joint" multiplier="1.0" offset="0.0"/>
+			<xacro:unless value="${kinematic_only}">
+				<axis xyz="0 1 0"/>
+				<limit lower="-1.57" upper="1.57" effort="10" velocity="1"/>
+				<mimic joint="${prefix}gripper_joint" multiplier="1.0" offset="0.0"/>
+			</xacro:unless>
 		</joint>
 		<!-- 夹爪右侧手指 R2 -->
@@ -157,11 +166,13 @@
 			</visual>
 		</link>
-		<joint name="${prefix}gripper_joint_R2" type="revolute">
+		<joint name="${prefix}gripper_joint_R2" type="${finger_joint_type}">
 			<origin xyz="-0.0325 0 0.0510999999999999"/>
 			<parent link="${prefix}gripper_base"/>
 			<child link="${prefix}gripper_R2"/>
-			<axis xyz="0 1 0"/>
-			<limit lower="-1.57" upper="1.57" effort="10" velocity="1"/>
-			<mimic joint="${prefix}gripper_joint" multiplier="1.0" offset="0.0"/>
+			<xacro:unless value="${kinematic_only}">
+				<axis xyz="0 1 0"/>
+				<limit lower="-1.57" upper="1.57" effort="10" velocity="1"/>
+				<mimic joint="${prefix}gripper_joint" multiplier="1.0" offset="0.0"/>
+			</xacro:unless>
 		</joint>
 		<!-- 夹爪右侧手指 R11 (末端) -->
@@ -189,11 +200,13 @@
 			</collision>
 		</link>
-		<joint name="${prefix}gripper_joint_R11" type="revolute">
+		<joint name="${prefix}gripper_joint_R11" type="${finger_joint_type}">
 			<origin xyz="-0.0412499999999999 0 0.0363790805271382"/>
 			<parent link="${prefix}gripper_R1"/>
 			<child link="${prefix}gripper_R11"/>
-			<axis xyz="0 -1 0"/>
-			<limit lower="-1.57" upper="1.57" effort="10" velocity="1"/>
-			<mimic joint="${prefix}gripper_joint" multiplier="1.0" offset="0.0"/>
+			<xacro:unless value="${kinematic_only}">
+				<axis xyz="0 -1 0"/>
+				<limit lower="-1.57" upper="1.57" effort="10" velocity="1"/>
+				<mimic joint="${prefix}gripper_joint" multiplier="1.0" offset="0.0"/>
+			</xacro:unless>
 		</joint>
 		<link name="${prefix}gripper_center"/>

File: humanoid/Astribot/astribot_s1_description/xacro/robot.xacro (robot description, xacro)
@@ -2,13 +2,15 @@
 <!-- =================================================================================== -->
 <!-- |    Complete Robot Description for Astribot S1                                   | -->
-<!-- |    This file includes the base robot structure (chassis, torso, head) and arms  | -->
+<!-- |    OCS2 planning: eef_fixed_joints + chassis_joints_movable (robot_common_launch)| -->
 <!-- =================================================================================== -->
 <robot name="Astribot S1" xmlns:xacro="http://www.ros.org/wiki/xacro">
+	<xacro:arg name="eef_fixed_joints" default="false"/>
+	<xacro:arg name="chassis_joints_movable" default="false"/>
+	<xacro:arg name="type" default="gripper"/>
 	<!-- Include the base robot structure (chassis, torso and head) -->
 	<xacro:include filename="$(find astribot_s1_description)/xacro/components/base.xacro"/>
 	<!-- Include the arm macro -->
 	<xacro:include filename="$(find astribot_s1_description)/xacro/components/s1_arm.xacro"/>
-	<xacro:arg name="enable_wheel_joints" default="false"/>
-	<xacro:Base enable_wheel_joints="$(arg enable_wheel_joints)"/>
+	<xacro:Base enable_wheel_joints="$(arg chassis_joints_movable)"/>
 	<!-- =================================================================================== -->
 	<!-- Generate Left and Right Arms Using Macro                                          -->
@@ -29,32 +31,34 @@
 		<origin rpy="0 -1.22173 1.5707963" xyz="0 -0.06449 0.02348"/>
 	</joint>
-	<xacro:arg name="type" default="gripper"/>
-	<xacro:if value="${'$(arg type)' == 'gripper'}">
+	<xacro:property name="type_arg" value="$(arg type)"/>
+	<xacro:property name="eef_fixed" value="$(arg eef_fixed_joints)"/>
+	<!-- OCS2 planning: freeze EEF actuation in URDF (eeFrame = left/right_link7 in .info) -->
+	<xacro:if value="${type_arg == 'gripper'}">
 		<xacro:include filename="$(find astribot_s1_description)/xacro/components/s1_gripper.xacro"/>
-		<xacro:Gripper name="left"/>
-		<xacro:Gripper name="right"/>
+		<xacro:Gripper name="left" kinematic_only="${eef_fixed}"/>
+		<xacro:Gripper name="right" kinematic_only="${eef_fixed}"/>
 		<joint name="left_gripper_fixed_joint" type="fixed">
 			<origin xyz="0 -0.045 0" rpy="1.5708 0 0"/>
-			<parent link="left_link_7"/>
+			<parent link="left_link7"/>
 			<child link="left_gripper_base"/>
 		</joint>
 		<joint name="right_gripper_fixed_joint" type="fixed">
 			<origin xyz="0 -0.045 0" rpy="1.5708 0 0"/>
-			<parent link="right_link_7"/>
+			<parent link="right_link7"/>
 			<child link="right_gripper_base"/>
 		</joint>
 	</xacro:if>
-	<xacro:if value="${'$(arg type)' == 'revo2'}">
+	<xacro:if value="${type_arg == 'revo2'}">
 		<xacro:include filename="$(find brainco_description)/xacro/revo2.xacro"/>
-		<xacro:BrainCoHand name="left_hand" direction="1" fixed_joints="false"/>
-		<xacro:BrainCoHand name="right_hand" direction="-1" fixed_joints="false"/>
+		<xacro:BrainCoHand name="left_hand" direction="1" use_flange="true" fixed_joints="${eef_fixed}"/>
+		<xacro:BrainCoHand name="right_hand" direction="-1" use_flange="true" fixed_joints="${eef_fixed}"/>
 		<joint name="left_gripper_fixed_joint" type="fixed">
 			<origin xyz="0 -0.048 0" rpy="1.5708 3.1416 0"/>
-			<parent link="left_link_7"/>
+			<parent link="left_link7"/>
 			<child link="left_hand_hand_base"/>
 		</joint>
 		<joint name="right_gripper_fixed_joint" type="fixed">
 			<origin xyz="0 -0.048 0" rpy="1.5708 0 0"/>
-			<parent link="right_link_7"/>
+			<parent link="right_link7"/>
 			<child link="right_hand_hand_base"/>
 		</joint>

File: humanoid/Astribot/astribot_s1_description/xacro/ros2_control/astribot_s1_arm_interfaces.xacro (robot description, xacro)
@@ -4,6 +4,5 @@
   <xacro:macro name="astribot_s1_arm_interfaces" params="name">
     <xacro:property name="prefix" value="${name + '_' if name else ''}"/>
-    <!-- 手臂关节接口定义 -->
-    <joint name="${prefix}joint_1">
+    <joint name="${prefix}joint1">
       <command_interface name="position"/>
       <state_interface name="position"/>
@@ -11,5 +10,5 @@
       <state_interface name="effort"/>
     </joint>
-    <joint name="${prefix}joint_2">
+    <joint name="${prefix}joint2">
       <command_interface name="position"/>
       <state_interface name="position"/>
@@ -17,5 +16,5 @@
       <state_interface name="effort"/>
     </joint>
-    <joint name="${prefix}joint_3">
+    <joint name="${prefix}joint3">
       <command_interface name="position"/>
       <state_interface name="position">
@@ -25,5 +24,5 @@
       <state_interface name="effort"/>
     </joint>
-    <joint name="${prefix}joint_4">
+    <joint name="${prefix}joint4">
       <command_interface name="position"/>
       <state_interface name="position">
@@ -33,5 +32,5 @@
       <state_interface name="effort"/>
     </joint>
-    <joint name="${prefix}joint_5">
+    <joint name="${prefix}joint5">
       <command_interface name="position"/>
       <state_interface name="position"/>
@@ -39,5 +38,5 @@
       <state_interface name="effort"/>
     </joint>
-    <joint name="${prefix}joint_6">
+    <joint name="${prefix}joint6">
       <command_interface name="position"/>
       <state_interface name="position"/>
@@ -45,5 +44,5 @@
       <state_interface name="effort"/>
     </joint>
-    <joint name="${prefix}joint_7">
+    <joint name="${prefix}joint7">
       <command_interface name="position"/>
       <state_interface name="position"/>

File: humanoid/Astribot/astribot_s1_description/xacro/ros2_control/astribot_s1_base_interfaces.xacro (robot description, xacro)
@@ -3,6 +3,5 @@
   <!-- Astribot S1 基座关节接口宏定义 -->
   <xacro:macro name="astribot_s1_base_interfaces">
-    <!-- 躯干关节接口定义 -->
-    <joint name="torso_joint_1">
+    <joint name="body_joint1">
       <command_interface name="position"/>
       <state_interface name="position">
@@ -12,5 +11,5 @@
       <state_interface name="effort"/>
     </joint>
-    <joint name="torso_joint_2">
+    <joint name="body_joint2">
       <command_interface name="position"/>
       <state_interface name="position">
@@ -20,5 +19,5 @@
       <state_interface name="effort"/>
     </joint>
-    <joint name="torso_joint_3">
+    <joint name="body_joint3">
       <command_interface name="position"/>
       <state_interface name="position">
@@ -28,5 +27,5 @@
       <state_interface name="effort"/>
     </joint>
-    <joint name="torso_joint_4">
+    <joint name="body_joint4">
       <command_interface name="position"/>
       <state_interface name="position"/>
@@ -34,6 +33,5 @@
       <state_interface name="effort"/>
     </joint>
-    <!-- 头部关节接口定义 -->
-    <joint name="head_joint_1">
+    <joint name="head_joint1">
       <command_interface name="position"/>
       <state_interface name="position"/>
@@ -41,5 +39,5 @@
       <state_interface name="effort"/>
     </joint>
-    <joint name="head_joint_2">
+    <joint name="head_joint2">
       <command_interface name="position"/>
       <state_interface name="position"/>
