Commit message: Feature/galaxea (#27)
* add galaxea new chassis

* update mesh to glb

* fix galaxea chassis

* modifed cicd

* add rs01

* add moz1

* update galaxea mesh

* test pass for galaxea and astribot

* fixed revo2 error

* update version

* adapt more robots

* modified galaxea r1 pro

* add cache

* update r1 png

* add support for galbot

* fix zerith h1 camera

* add wbc config for galaxea r1

* fix color problems for moz1

* Add fiveages_s2_description as submodule (fa-s2-description).

Co-authored-by: Cursor <cursoragent@cursor.com>

* fix cr5 config

* Add panthera_ht_description as submodule.

Register HighTorque Panthera HT manipulator description and document submodule usage in README.

Co-authored-by: Cursor <cursoragent@cursor.com>

* update hash

* update default task info param; default speed change to 100

* rename omni wheel name

* Add Galaxea_A1Z without gripper G1Z

* update ocs2 humanoid default config

* Add Galaxea_A1Z Complete with ocs2 test.

* Switch HighTorque submodule to robot-descriptions-ht @ 63004ec

* chore: bump HighTorque submodule for ros2_ws README paths

Co-authored-by: Cursor <cursoragent@cursor.com>

* chore: bump HighTorque for ht_ros2_control rename

Co-authored-by: Cursor <cursoragent@cursor.com>

* update galaxea config

* update stash

---------

Co-authored-by: Cursor <cursoragent@cursor.com>
Co-authored-by: MZY <2071320248@qq.com>
Co-authored-by: Sgr-Zgc <945418316@qq.com>

File: humanoid/Astribot/astribot_s1_description/xacro/components/base.xacro (robot description, xacro)
@@ -24,5 +24,5 @@
 			</collision>
 		</link>
-		<xacro:include filename="$(find component_models)/xacro/angellun_omniwheel.xacro"/>
+		<xacro:include filename="$(find component_models)/xacro/angellun_160.xacro"/>
 		<!-- 根据enable_wheel_joints参数决定使用轮子宏还是空link -->
 		<xacro:if value="${enable_wheel_joints}">
@@ -103,5 +103,5 @@
 			</collision>
 		</link>
-		<joint name="torso_joint_1" type="revolute">
+		<joint name="body_joint1" type="revolute">
 			<origin rpy="-1.5708 1.5708 0" xyz="0 0 0.12"/>
 			<parent link="base_link"/>
@@ -132,5 +132,5 @@
 			</collision>
 		</link>
-		<joint name="torso_joint_2" type="revolute">
+		<joint name="body_joint2" type="revolute">
 			<origin xyz="-0.38 0 0"/>
 			<parent link="torso_link_1"/>
@@ -159,5 +159,5 @@
 			</collision>
 		</link>
-		<joint name="torso_joint_3" type="revolute">
+		<joint name="body_joint3" type="revolute">
 			<origin xyz="-0.390 0 0"/>
 			<parent link="torso_link_2"/>
@@ -181,5 +181,5 @@
 			</visual>
 		</link>
-		<joint name="torso_joint_4" type="revolute">
+		<joint name="body_joint4" type="revolute">
 			<origin rpy="1.5708 0 -1.5708" xyz="0 0 0"/>
 			<parent link="torso_link_3"/>
@@ -219,6 +219,6 @@
 			<origin xyz="0 0 0.1229"/>
 		</joint>
-		<!-- 头部连杆1 -->
-		<link name="head_link_1">
+		<!-- 头部连杆1（head_joint1） -->
+		<link name="head_link1">
 			<inertial>
 				<origin xyz="0.00003191 -0.00038566 -0.02579910"/>
@@ -233,12 +233,12 @@
 			</visual>
 		</link>
-		<joint name="head_joint_1" type="revolute">
+		<joint name="head_joint1" type="revolute">
 			<parent link="head_base_link"/>
-			<child link="head_link_1"/>
+			<child link="head_link1"/>
 			<axis xyz="0 0 1"/>
 			<limit effort="100" lower="-1.57" upper="1.57" velocity="4.0"/>
 		</joint>
-		<!-- 头部连杆2 -->
-		<link name="head_link_2">
+		<!-- 头部连杆2（head_joint2） -->
+		<link name="head_link2">
 			<inertial>
 				<origin xyz="0.00705824 -0.14472601 -0.00061724"/>
@@ -259,8 +259,8 @@
 			</collision>
 		</link>
-		<joint name="head_joint_2" type="revolute">
+		<joint name="head_joint2" type="revolute">
 			<origin rpy="-1.5708 0 0" xyz="0 0 0"/>
-			<parent link="head_link_1"/>
-			<child link="head_link_2"/>
+			<parent link="head_link1"/>
+			<child link="head_link2"/>
 			<axis xyz="0 0 1"/>
 			<limit effort="100" lower="-1.22" upper="1.22" velocity="4.0"/>

File: humanoid/Astribot/astribot_s1_description/xacro/robot.xacro (robot description, xacro)
@@ -2,13 +2,15 @@
 <!-- =================================================================================== -->
 <!-- |    Complete Robot Description for Astribot S1                                   | -->
-<!-- |    This file includes the base robot structure (chassis, torso, head) and arms  | -->
+<!-- |    OCS2 planning: eef_fixed_joints + chassis_joints_movable (robot_common_launch)| -->
 <!-- =================================================================================== -->
 <robot name="Astribot S1" xmlns:xacro="http://www.ros.org/wiki/xacro">
+	<xacro:arg name="eef_fixed_joints" default="false"/>
+	<xacro:arg name="chassis_joints_movable" default="false"/>
+	<xacro:arg name="type" default="gripper"/>
 	<!-- Include the base robot structure (chassis, torso and head) -->
 	<xacro:include filename="$(find astribot_s1_description)/xacro/components/base.xacro"/>
 	<!-- Include the arm macro -->
 	<xacro:include filename="$(find astribot_s1_description)/xacro/components/s1_arm.xacro"/>
-	<xacro:arg name="enable_wheel_joints" default="false"/>
-	<xacro:Base enable_wheel_joints="$(arg enable_wheel_joints)"/>
+	<xacro:Base enable_wheel_joints="$(arg chassis_joints_movable)"/>
 	<!-- =================================================================================== -->
 	<!-- Generate Left and Right Arms Using Macro                                          -->
@@ -29,32 +31,34 @@
 		<origin rpy="0 -1.22173 1.5707963" xyz="0 -0.06449 0.02348"/>
 	</joint>
-	<xacro:arg name="type" default="gripper"/>
-	<xacro:if value="${'$(arg type)' == 'gripper'}">
+	<xacro:property name="type_arg" value="$(arg type)"/>
+	<xacro:property name="eef_fixed" value="$(arg eef_fixed_joints)"/>
+	<!-- OCS2 planning: freeze EEF actuation in URDF (eeFrame = left/right_link7 in .info) -->
+	<xacro:if value="${type_arg == 'gripper'}">
 		<xacro:include filename="$(find astribot_s1_description)/xacro/components/s1_gripper.xacro"/>
-		<xacro:Gripper name="left"/>
-		<xacro:Gripper name="right"/>
+		<xacro:Gripper name="left" kinematic_only="${eef_fixed}"/>
+		<xacro:Gripper name="right" kinematic_only="${eef_fixed}"/>
 		<joint name="left_gripper_fixed_joint" type="fixed">
 			<origin xyz="0 -0.045 0" rpy="1.5708 0 0"/>
-			<parent link="left_link_7"/>
+			<parent link="left_link7"/>
 			<child link="left_gripper_base"/>
 		</joint>
 		<joint name="right_gripper_fixed_joint" type="fixed">
 			<origin xyz="0 -0.045 0" rpy="1.5708 0 0"/>
-			<parent link="right_link_7"/>
+			<parent link="right_link7"/>
 			<child link="right_gripper_base"/>
 		</joint>
 	</xacro:if>
-	<xacro:if value="${'$(arg type)' == 'revo2'}">
+	<xacro:if value="${type_arg == 'revo2'}">
 		<xacro:include filename="$(find brainco_description)/xacro/revo2.xacro"/>
-		<xacro:BrainCoHand name="left_hand" direction="1" fixed_joints="false"/>
-		<xacro:BrainCoHand name="right_hand" direction="-1" fixed_joints="false"/>
+		<xacro:BrainCoHand name="left_hand" direction="1" fixed_joints="${eef_fixed}"/>
+		<xacro:BrainCoHand name="right_hand" direction="-1"  fixed_joints="${eef_fixed}"/>
 		<joint name="left_gripper_fixed_joint" type="fixed">
 			<origin xyz="0 -0.048 0" rpy="1.5708 3.1416 0"/>
-			<parent link="left_link_7"/>
+			<parent link="left_link7"/>
 			<child link="left_hand_hand_base"/>
 		</joint>
 		<joint name="right_gripper_fixed_joint" type="fixed">
 			<origin xyz="0 -0.048 0" rpy="1.5708 0 0"/>
-			<parent link="right_link_7"/>
+			<parent link="right_link7"/>
 			<child link="right_hand_hand_base"/>
 		</joint>

File: humanoid/Galaxea/galaxea_r1_description/xacro/component.xacro (robot description, xacro)
@@ -6,11 +6,15 @@
 <robot name="Galaxea_R1" xmlns:xacro="http://www.ros.org/wiki/xacro">
 	<xacro:property name="PI" value="3.1415926535897931"/>
-	<xacro:arg name="type" default="base"/>
-	<xacro:if value="${'$(arg type)' == 'base'}">
+	<xacro:arg name="type" default="chassis"/>
+	<xacro:arg name="enable_wheel_joints" default="true"/>
+	<xacro:if value="${'$(arg type)' == 'chassis'}">
 		<!-- Include Chassis -->
-		<xacro:include filename="$(find galaxea_r1_description)/xacro/chassis.xacro"/>
-		<xacro:Chassis/>
+		<xacro:include filename="$(find galaxea_r1_description)/xacro/components/chassis.xacro"/>
+		<xacro:Chassis enable_wheel_joints="$(arg enable_wheel_joints)"/>
+	</xacro:if>
+	<xacro:if value="${'$(arg type)' == 'torso'}">
 		<!-- Include Torso -->
-		<xacro:include filename="$(find galaxea_r1_description)/xacro/torso.xacro"/>
+		<xacro:include filename="$(find galaxea_r1_description)/xacro/components/torso.xacro"/>
+		<link name="base_link"/>
 		<xacro:Torso/>
 	</xacro:if>

File: humanoid/Galaxea/galaxea_r1_description/xacro/robot.xacro (robot description, xacro)
@@ -2,9 +2,10 @@
 <robot name="R1" xmlns:xacro="http://www.ros.org/wiki/xacro">
 	<xacro:property name="PI" value="3.1415926535897931"/>
+  <xacro:arg name="enable_wheel_joints" default="false"/>
   <!-- Include Chassis -->
-  <xacro:include filename="$(find galaxea_r1_description)/xacro/chassis.xacro"/>
-  <xacro:Chassis/>
+  <xacro:include filename="$(find galaxea_r1_description)/xacro/components/chassis.xacro"/>
+  <xacro:Chassis enable_wheel_joints="$(arg enable_wheel_joints)"/>
   <!-- Include Torso -->
-  <xacro:include filename="$(find galaxea_r1_description)/xacro/torso.xacro"/>
+  <xacro:include filename="$(find galaxea_r1_description)/xacro/components/torso.xacro"/>
   <xacro:Torso/>
   <!-- Include Left Arm -->
@@ -18,5 +19,5 @@
   </joint>
   <!-- Include Left RealSense Camera -->
-  <xacro:include filename="$(find galaxea_r1_description)/xacro/realsense.xacro"/>
+  <xacro:include filename="$(find galaxea_r1_description)/xacro/components/realsense.xacro"/>
   <xacro:RealSense side="left"/>
   <!-- Include Right Arm -->

File: humanoid/Galaxea/galaxea_r1_description/xacro/ros2_control/interfaces.xacro (robot description, xacro)
@@ -7,5 +7,5 @@
       <command_interface name="position"/>
       <state_interface name="position">
-        <param name="initial_value">-1.57</param>
+        <param name="initial_value">1.57</param>
       </state_interface>
       <state_interface name="velocity"/>
@@ -15,5 +15,5 @@
       <command_interface name="position"/>
       <state_interface name="position">
-        <param name="initial_value">2.7</param>
+        <param name="initial_value">-2.7</param>
       </state_interface>
       <state_interface name="velocity"/>
@@ -23,5 +23,5 @@
       <command_interface name="position"/>
       <state_interface name="position">
-        <param name="initial_value">1.1</param>
+        <param name="initial_value">-1.1</param>
       </state_interface>
       <state_interface name="velocity"/>
@@ -31,5 +31,5 @@
       <command_interface name="position"/>
       <state_interface name="position">
-        <param name="initial_value">1.1</param>
+        <param name="initial_value">0.0</param>
       </state_interface>
       <state_interface name="velocity"/>

File: humanoid/Galaxea/galaxea_r1pro_description/xacro/component.xacro (robot description, xacro)
@@ -1,13 +1,22 @@
 <?xml version="1.0" ?>
 <!-- =================================================================================== -->
-<!-- |    Complete Robot Description for Agibot G1                                     | -->
-<!-- |    This file includes the base robot structure and both arms                    | -->
+<!-- |    Component descriptions for Galaxea R1 Pro                                    | -->
 <!-- =================================================================================== -->
-<robot name="A2_Arm" xmlns:xacro="http://www.ros.org/wiki/xacro">
+<robot name="A2 Arms" xmlns:xacro="http://www.ros.org/wiki/xacro">
 	<xacro:property name="PI" value="3.1415926535897931"/>
 	<xacro:arg name="type" default="arms"/>
+	<xacro:arg name="enable_wheel_joints" default="true"/>
+	<xacro:if value="${'$(arg type)' == 'chassis'}">
+		<xacro:include filename="$(find galaxea_r1_description)/xacro/components/chassis.xacro"/>
+		<xacro:Chassis enable_wheel_joints="$(arg enable_wheel_joints)"/>
+	</xacro:if>
+	<xacro:if value="${'$(arg type)' == 'torso'}">
+		<xacro:include filename="$(find galaxea_r1_description)/xacro/components/torso.xacro"/>
+		<link name="base_link"/>
+		<xacro:Torso/>
+	</xacro:if>
 	<xacro:if value="${'$(arg type)' == 'arms'}">
 		<link name="torso_link4"/>
-		<xacro:include filename="pro_arm.xacro"/>
+		<xacro:include filename="$(find galaxea_r1pro_description)/xacro/components/pro_arm.xacro"/>
 		<xacro:Arm name="left"/>
 		<xacro:Arm name="right" direction="-1"/>

File: manipulator/Galaxea/galaxea_a1_description/xacro/ros2_control/robot.xacro (robot description, xacro)
@@ -37,4 +37,7 @@
           <parameters>$(find galaxea_a1_description)/config/ros2_control/y.yaml</parameters>
         </xacro:if>
+        <xacro:if value="${'$(arg type)' == 'z'}">
+          <parameters>$(find galaxea_a1_description)/config/ros2_control/z.yaml</parameters>
+        </xacro:if>
       </plugin>
     </gazebo>
