Commit message: update astribot s1

File: humanoid/Astribot/astribot_s1_description/xacro/components/base.xacro (robot description, xacro)
@@ -5,5 +5,5 @@
 <!-- =================================================================================== -->
 <robot xmlns:xacro="http://www.ros.org/wiki/xacro">
-	<xacro:macro name="Base" params="enable_wheel_joints:='true'">
+	<xacro:macro name="Base" params="enable_wheel_joints:='true' isaac:=false">
 		<!-- Base link (底盘基础连杆) -->
 		<link name="base_link">
@@ -81,4 +81,81 @@
 			</xacro:if>
 		</joint>
+		<link name="fl_lidar">
+			<!-- inertial from S2_3DURDF YLD_Link -->
+			<inertial>
+				<origin xyz="-0.0440891839567841 -5.1873280670911E-10 -0.0315237882031307"/>
+				<mass value="0.0117156542424497"/>
+				<inertia
+						ixx="3.67951096550954E-07"
+						ixy="5.15239039992179E-14"
+						ixz="-7.72651115285907E-09"
+						iyy="6.52014762336772E-07"
+						iyz="2.14985023980089E-14"
+						izz="5.88939528438811E-07"/>
+			</inertial>
+			<xacro:unless value="${isaac}">
+				<visual>
+					<geometry>
+						<mesh filename="file://$(find sensor_models)/meshes/livox/mid360.glb"/>
+					</geometry>
+				</visual>
+			</xacro:unless>
+		</link>
+		<joint name="fl_lidar_joint" type="fixed">
+			<origin xyz="0.17399 0.16891 0.0597" />
+			<parent link="base_link"/>
+			<child link="fl_lidar"/>
+		</joint>
+		<link name="rr_lidar">
+			<!-- inertial from S2_3DURDF YLD_Link -->
+			<inertial>
+				<origin xyz="-0.0440891839567841 -5.1873280670911E-10 -0.0315237882031307"/>
+				<mass value="0.0117156542424497"/>
+				<inertia
+						ixx="3.67951096550954E-07"
+						ixy="5.15239039992179E-14"
+						ixz="-7.72651115285907E-09"
+						iyy="6.52014762336772E-07"
+						iyz="2.14985023980089E-14"
+						izz="5.88939528438811E-07"/>
+			</inertial>
+			<xacro:unless value="${isaac}">
+				<visual>
+					<geometry>
+						<mesh filename="file://$(find sensor_models)/meshes/livox/mid360.glb"/>
+					</geometry>
+				</visual>
+			</xacro:unless>
+		</link>
+		<joint name="rr_lidar_joint" type="fixed">
+			<origin xyz="-0.17957 -0.17466 0.14362"  rpy="0 0 ${PI}" />
+			<parent link="base_link"/>
+			<child link="rr_lidar"/>
+		</joint>
+		<!-- Ultrasonic sensors C1-C8 (mesh: sensor_models/ultrasonic_03, origin = outer-face circle) -->
+		<xacro:macro name="astribot_ultrasonic" params="name xyz rpy">
+			<link name="${name}">
+				<xacro:unless value="${isaac}">
+					<visual>
+						<geometry>
+							<mesh filename="file://$(find sensor_models)/meshes/ultrasonic/ultrasonic_03.glb"/>
+						</geometry>
+					</visual>
+				</xacro:unless>
+			</link>
+			<joint name="${name}_joint" type="fixed">
+				<origin xyz="${xyz}" rpy="${rpy}"/>
+				<parent link="base_link"/>
+				<child link="${name}"/>
+			</joint>
+		</xacro:macro>
+		<xacro:astribot_ultrasonic name="ultrasonic_c1" xyz="0.28374913 -0.12873359 0.02026958" rpy="1.40431778 0.02868544 1.62266583"/>
+		<xacro:astribot_ultrasonic name="ultrasonic_c2" xyz="0.12977453 -0.28310611 0.05628103" rpy="-1.25579677 -0.01326278 3.12623520"/>
+		<xacro:astribot_ultrasonic name="ultrasonic_c3" xyz="-0.12865779 -0.27341227 0.11774913" rpy="-1.40030526 0.05319742 2.56913165"/>
+		<xacro:astribot_ultrasonic name="ultrasonic_c4" xyz="-0.27264161 -0.19961814 0.11701791" rpy="1.50622852 0.09425214 -1.01682828"/>
+		<xacro:astribot_ultrasonic name="ultrasonic_c5" xyz="-0.27253755 0.19968408 0.11733165" rpy="-1.41112704 0.04522913 1.01101617"/>
+		<xacro:astribot_ultrasonic name="ultrasonic_c6" xyz="-0.12868858 0.27347962 0.11748791" rpy="1.49883288 0.09863409 -2.57452670"/>
+		<xacro:astribot_ultrasonic name="ultrasonic_c7" xyz="0.12990424 0.28315572 0.05605944" rpy="1.35379071 0.02135683 -3.13552145"/>
+		<xacro:astribot_ultrasonic name="ultrasonic_c8" xyz="0.28362270 0.12870185 0.02079986" rpy="-1.28691460 -0.00038371 -1.62933103"/>
 		<!-- 躯干连杆1 -->
 		<link name="torso_link_1">
@@ -92,7 +169,4 @@
 					<mesh filename="file://$(find astribot_s1_description)/meshes/s1_torso/link1.glb"/>
 				</geometry>
-				<material name="">
-					<color rgba="0.89804 0.91765 0.92941 1"/>
-				</material>
 			</visual>
 			<collision>
@@ -121,7 +195,4 @@
 					<mesh filename="file://$(find astribot_s1_description)/meshes/s1_torso/link2.glb"/>
 				</geometry>
-				<material name="">
-					<color rgba="0.89804 0.91765 0.92941 1"/>
-				</material>
 			</visual>
 			<collision>

File: humanoid/Astribot/astribot_s1_description/xacro/components/s1_arm.xacro (robot description, xacro)
@@ -144,7 +144,4 @@
 					<mesh filename="file://$(find astribot_s1_description)/meshes/s1_arm/link5.glb"/>
 				</geometry>
-				<material name="">
-					<color rgba="0.698039215686274 0.698039215686274 0.698039215686274 1"/>
-				</material>
 			</visual>
 			<collision>

File: humanoid/Astribot/astribot_s1_description/xacro/robot.xacro (robot description, xacro)
@@ -4,13 +4,14 @@
 <!-- |    OCS2 planning: eef_fixed_joints + chassis_joints_movable (robot_common_launch)| -->
 <!-- =================================================================================== -->
-<robot name="Astribot S1" xmlns:xacro="http://www.ros.org/wiki/xacro">
+<robot name="S1" xmlns:xacro="http://www.ros.org/wiki/xacro">
 	<xacro:arg name="eef_fixed_joints" default="false"/>
 	<xacro:arg name="chassis_joints_movable" default="false"/>
 	<xacro:arg name="type" default="gripper"/>
+	<xacro:arg name="isaac" default="false"/>
 	<!-- Include the base robot structure (chassis, torso and head) -->
 	<xacro:include filename="$(find astribot_s1_description)/xacro/components/base.xacro"/>
 	<!-- Include the arm macro -->
 	<xacro:include filename="$(find astribot_s1_description)/xacro/components/s1_arm.xacro"/>
-	<xacro:Base enable_wheel_joints="$(arg chassis_joints_movable)"/>
+	<xacro:Base enable_wheel_joints="$(arg chassis_joints_movable)" isaac="$(arg isaac)"/>
 	<!-- =================================================================================== -->
 	<!-- Generate Left and Right Arms Using Macro                                          -->

Commit message: update param

File: humanoid/Astribot/astribot_s1_description/xacro/components/base.xacro (robot description, xacro)
@@ -6,4 +6,5 @@
 <robot xmlns:xacro="http://www.ros.org/wiki/xacro">
 	<xacro:macro name="Base" params="enable_wheel_joints:='true' isaac:=false">
+		<link name="base_footprint"/>
 		<!-- Base link (底盘基础连杆) -->
 		<link name="base_link">
@@ -24,4 +25,8 @@
 			</collision>
 		</link>
+		<joint name="base_footprint_joint" type="fixed">
+			<parent link="base_footprint"/>
+			<child link="base_link"/>
+		</joint>
 		<xacro:include filename="$(find component_models)/xacro/angellun_160.xacro"/>
 		<!-- 根据enable_wheel_joints参数决定使用轮子宏还是空link -->
@@ -251,4 +256,10 @@
 				</geometry>
 			</visual>
+			<collision>
+				<origin xyz="0 0 0.17"/>
+				<geometry>
+					<box size="0.22 0.32 0.34"/>
+				</geometry>
+			</collision>
 		</link>
 		<joint name="body_joint4" type="revolute">
@@ -337,4 +348,12 @@
 			<limit effort="100" lower="-1.22" upper="1.22" velocity="4.0"/>
 		</joint>
+		<!-- Optical frame for HEAD_GAZE (+Z look-ahead). Placeholder: S1 CAD has no
+		     head camera TF; pose is the head_link2 collision sphere along -Y. -->
+		<link name="head_camera"/>
+		<joint name="head_camera_joint" type="fixed">
+			<origin xyz="0 -0.16 0" rpy="1.5708 0 0"/>
+			<parent link="head_link2"/>
+			<child link="head_camera"/>
+		</joint>
 	</xacro:macro>
 </robot>

File: humanoid/Astribot/astribot_s1_description/xacro/robot.xacro (robot description, xacro)
@@ -2,4 +2,7 @@
 <!-- =================================================================================== -->
 <!-- |    Complete Robot Description for Astribot S1                                   | -->
+<!-- |    Structure : base_footprint -> base_link -> torso -> torso_end_effector;      | -->
+<!-- |    arm_base coincides with torso_end_effector; head after torso.                | -->
+<!-- |    topology:=dual : split-body planning tree rooted at arm_base.                | -->
 <!-- |    OCS2 planning: eef_fixed_joints + chassis_joints_movable (robot_common_launch)| -->
 <!-- =================================================================================== -->
@@ -9,59 +12,89 @@
 	<xacro:arg name="type" default="gripper"/>
 	<xacro:arg name="isaac" default="false"/>
-	<!-- Include the base robot structure (chassis, torso and head) -->
-	<xacro:include filename="$(find astribot_s1_description)/xacro/components/base.xacro"/>
-	<!-- Include the arm macro -->
-	<xacro:include filename="$(find astribot_s1_description)/xacro/components/s1_arm.xacro"/>
-	<xacro:Base enable_wheel_joints="$(arg chassis_joints_movable)" isaac="$(arg isaac)"/>
-	<!-- =================================================================================== -->
-	<!-- Generate Left and Right Arms Using Macro                                          -->
-	<!-- =================================================================================== -->
-	<xacro:S1Arm name="left"/>
-	<xacro:S1Arm name="right" direction="-1"/>
-	<!-- =================================================================================== -->
-	<!-- Arms Connection to Torso                                                          -->
-	<!-- =================================================================================== -->
-	<joint name="left_base_fixed_joint" type="fixed">
-		<parent link="torso_end_effector"/>
-		<child link="left_base_link"/>
-		<origin rpy="0 -1.22173 -1.5707963" xyz="0 0.06449 0.02348"/>
-	</joint>
-	<joint name="right_base_fixed_joint" type="fixed">
-		<parent link="torso_end_effector"/>
-		<child link="right_base_link"/>
-		<origin rpy="0 -1.22173 1.5707963" xyz="0 -0.06449 0.02348"/>
-	</joint>
+	<xacro:arg name="topology" default="full"/>
+	<xacro:property name="topology_arg" value="$(arg topology)"/>
 	<xacro:property name="type_arg" value="$(arg type)"/>
 	<xacro:property name="eef_fixed" value="$(arg eef_fixed_joints)"/>
-	<!-- OCS2 planning: freeze EEF actuation in URDF (eeFrame = left/right_link7 in .info) -->
-	<xacro:if value="${type_arg == 'gripper'}">
-		<xacro:include filename="$(find astribot_s1_description)/xacro/components/s1_gripper.xacro"/>
-		<xacro:Gripper name="left" kinematic_only="${eef_fixed}"/>
-		<xacro:Gripper name="right" kinematic_only="${eef_fixed}"/>
-		<joint name="left_gripper_fixed_joint" type="fixed">
-			<origin xyz="0 -0.045 0" rpy="1.5708 0 0"/>
+	<xacro:include filename="$(find astribot_s1_description)/xacro/components/s1_arm.xacro"/>
+	<xacro:macro name="AstribotS1ArmsAndEefs" params="arm_parent">
+		<xacro:S1Arm name="left"/>
+		<xacro:S1Arm name="right" direction="-1"/>
+		<joint name="left_base_fixed_joint" type="fixed">
+			<parent link="${arm_parent}"/>
+			<child link="left_base_link"/>
+			<origin rpy="0 -1.22173 -1.5707963" xyz="0 0.06449 0.02348"/>
+		</joint>
+		<joint name="right_base_fixed_joint" type="fixed">
+			<parent link="${arm_parent}"/>
+			<child link="right_base_link"/>
+			<origin rpy="0 -1.22173 1.5707963" xyz="0 -0.06449 0.02348"/>
+		</joint>
+		<link name="left_eef"/>
+		<joint name="left_eef_joint" type="fixed">
 			<parent link="left_link7"/>
-			<child link="left_gripper_base"/>
+			<child link="left_eef"/>
 		</joint>
-		<joint name="right_gripper_fixed_joint" type="fixed">
-			<origin xyz="0 -0.045 0" rpy="1.5708 0 0"/>
+		<link name="right_eef"/>
+		<joint name="right_eef_joint" type="fixed">
 			<parent link="right_link7"/>
-			<child link="right_gripper_base"/>
+			<child link="right_eef"/>
 		</joint>
+		<xacro:if value="${type_arg == 'gripper'}">
+			<xacro:include filename="$(find astribot_s1_description)/xacro/components/s1_gripper.xacro"/>
+			<xacro:Gripper name="left" kinematic_only="${eef_fixed}"/>
+			<xacro:Gripper name="right" kinematic_only="${eef_fixed}"/>
+			<joint name="left_gripper_fixed_joint" type="fixed">
+				<origin xyz="0 -0.045 0" rpy="1.5708 0 0"/>
+				<parent link="left_link7"/>
+				<child link="left_gripper_base"/>
+			</joint>
+			<joint name="right_gripper_fixed_joint" type="fixed">
+				<origin xyz="0 -0.045 0" rpy="1.5708 0 0"/>
+				<parent link="right_link7"/>
+				<child link="right_gripper_base"/>
+			</joint>
+		</xacro:if>
+		<xacro:if value="${type_arg == 'revo2'}">
+			<xacro:include filename="$(find brainco_description)/xacro/revo2.xacro"/>
+			<xacro:BrainCoHand name="left_hand" direction="1" fixed_joints="${eef_fixed}"/>
+			<xacro:BrainCoHand name="right_hand" direction="-1" fixed_joints="${eef_fixed}"/>
+			<joint name="left_gripper_fixed_joint" type="fixed">
+				<origin xyz="0 -0.048 0" rpy="1.5708 3.1416 0"/>
+				<parent link="left_link7"/>
+				<child link="left_hand_hand_base"/>
+			</joint>
+			<joint name="right_gripper_fixed_joint" type="fixed">
+				<origin xyz="0 -0.048 0" rpy="1.5708 0 0"/>
+				<parent link="right_link7"/>
+				<child link="right_hand_hand_base"/>
+			</joint>
+		</xacro:if>
+	</xacro:macro>
+	<!-- Split-body OCS2: dual-arm tree, root coinciding with arm_base (= torso_end_effector). -->
+	<xacro:if value="${topology_arg == 'dual'}">
+		<link name="base_link"/>
+		<link name="arm_base">
+			<collision>
+				<origin xyz="0 0 -0.175"/>
+				<geometry>
+					<box size="0.22 0.32 0.34"/>
+				</geometry>
+			</collision>
+		</link>
+		<joint name="arm_base_joint" type="fixed">
+			<parent link="base_link"/>
+			<child link="arm_base"/>
+		</joint>
+		<xacro:AstribotS1ArmsAndEefs arm_parent="arm_base"/>
 	</xacro:if>
-	<xacro:if value="${type_arg == 'revo2'}">
-		<xacro:include filename="$(find brainco_description)/xacro/revo2.xacro"/>
-		<xacro:BrainCoHand name="left_hand" direction="1" fixed_joints="${eef_fixed}"/>
-		<xacro:BrainCoHand name="right_hand" direction="-1"  fixed_joints="${eef_fixed}"/>
-		<joint name="left_gripper_fixed_joint" type="fixed">
-			<origin xyz="0 -0.048 0" rpy="1.5708 3.1416 0"/>
-			<parent link="left_link7"/>
-			<child link="left_hand_hand_base"/>
+	<xacro:unless value="${topology_arg == 'dual'}">
+		<xacro:include filename="$(find astribot_s1_description)/xacro/components/base.xacro"/>
+		<xacro:Base enable_wheel_joints="$(arg chassis_joints_movable)" isaac="$(arg isaac)"/>
+		<link name="arm_base"/>
+		<joint name="arm_base_joint" type="fixed">
+			<parent link="torso_end_effector"/>
+			<child link="arm_base"/>
 		</joint>
-		<joint name="right_gripper_fixed_joint" type="fixed">
-			<origin xyz="0 -0.048 0" rpy="1.5708 0 0"/>
-			<parent link="right_link7"/>
-			<child link="right_hand_hand_base"/>
-		</joint>
-	</xacro:if>
+		<xacro:AstribotS1ArmsAndEefs arm_parent="arm_base"/>
+	</xacro:unless>
 </robot>

File: humanoid/Astribot/astribot_s1_description/xacro/ros2_control/robot.xacro (robot description, xacro)
@@ -5,7 +5,7 @@
 <!-- =================================================================================== -->
 <robot name="astribot_whole_body" xmlns:xacro="http://www.ros.org/wiki/xacro">
-	<!-- Include the base robot structure -->
-	<!-- Type argument will be inherited by robot.xacro -->
+	<!-- Hardware URDF is always full topology; demo planning uses topology:=dual separately. -->
 	<xacro:arg name="type" default="gripper"/>
+	<xacro:arg name="ros2_control_hardware_type" default="mock_components"/>
 	<xacro:include filename="$(find astribot_s1_description)/xacro/robot.xacro"/>
 	<!-- Import modular interface components -->
