Commit message: fix zerith h1 camera

File: humanoid/Zerith/zerith_h1_description/xacro/components/body.xacro (robot description, xacro)
@@ -144,10 +144,4 @@
 					iyy="4.688e-05" iyz="-4e-08" izz="4.697e-05"/>
 		</inertial>
-		<visual>
-			<geometry>
-				<mesh filename="file://$(find sensor_models)/meshes/realsense/d435.glb"/>
-			</geometry>
-			<origin xyz="0.0325 0 0.005" rpy="1.5707963267949 -1.5707963267949 -0"/>
-		</visual>
 	</link>
 	<joint name="neck_camera_joint" type="fixed">
@@ -157,3 +151,15 @@
 		<child link="neck_camera_link"/>
 	</joint>
+	<link name="head_camera">
+		<visual>
+			<geometry>
+				<mesh filename="file://$(find sensor_models)/meshes/realsense/d435.glb"/>
+			</geometry>
+		</visual>
+	</link>
+	<joint name="head_camera_joint" type="fixed">
+		<origin xyz="0.0325 0 0.005"/>
+		<parent link="neck_camera_link"/>
+		<child link="head_camera"/>
+	</joint>
 </robot>
