Commit message: feat(zerith_h1): add mock ros2_control, grippers, and OCS2 WBC stack
Bring Zerith H1 from viz-only to wheeled-arm peer control level:
chassis wheels locked by default, ARX-style adaptive grippers,
split body controllers, and full-body ocs2_wbc_controller with
Pinocchio-aligned joint order (body|head|L|R, headInputStart=3).
Validated mock full_body on Sim-05. Vendor urdf/ kept for provenance.

File: humanoid/Zerith/zerith_h1_description/xacro/components/arm.xacro (robot description, xacro)
@@ -148,7 +148,5 @@
 			<child link="${prefix}wrist_roll_link"/>
 			<axis xyz="1 0 0"/>
-			<limit lower="-2.9671" upper="2.9671"
-						 effort="${0 if direction == 1 else 9}"
-						 velocity="${0 if direction == 1 else 16.747}"/>
+			<limit lower="-2.9671" upper="2.9671" effort="9" velocity="16.747"/>
 		</joint>
 		<!-- =============================================================================== -->

File: humanoid/Zerith/zerith_h1_description/xacro/components/body.xacro (robot description, xacro)
@@ -32,5 +32,5 @@
 		<child link="body_link1"/>
 		<axis xyz="0 0 1"/>
-		<limit lower="0" upper="0.8" effort="0" velocity="0"/>
+		<limit lower="0" upper="0.8" effort="500" velocity="0.2"/>
 	</joint>
 	<link name="body_pitch_link">

File: humanoid/Zerith/zerith_h1_description/xacro/components/chassis.xacro (robot description, xacro)
@@ -2,8 +2,11 @@
 <!-- =================================================================================== -->
 <!-- |    Chassis Description for Zerith H1                                            | -->
-<!-- |    Parameterized macro: drive_joint_type="continuous" (default) or "fixed"       | -->
+<!-- |    Parameterized macro: joints_movable:=false (default) locks drive wheels       | -->
 <!-- =================================================================================== -->
 <robot name="zerith_h1_chassis" xmlns:xacro="http://www.ros.org/wiki/xacro">
-	<xacro:macro name="H1Chassis" params="drive_joint_type:=continuous">
+	<!-- joints_movable:=false → drive wheels fixed (W2/Bot2/Quanta). -->
+	<xacro:macro name="H1Chassis" params="joints_movable:=false">
+		<xacro:property name="chassis_movable" value="${str(joints_movable).lower() in ['true', '1', 'yes', 'on']}"/>
+		<xacro:property name="wheel_joint_type" value="${'continuous' if chassis_movable else 'fixed'}"/>
 		<link name="base_link">
 			<inertial>
@@ -74,5 +77,5 @@
 			</collision>
 		</link>
-		<joint name="left_wheel_joint" type="${drive_joint_type}">
+		<joint name="left_wheel_joint" type="${wheel_joint_type}">
 			<origin xyz="0.0544 0.1895 -0.0965"/>
 			<parent link="base_link"/>
@@ -158,5 +161,5 @@
 			</collision>
 		</link>
-		<joint name="right_wheel_joint" type="${drive_joint_type}">
+		<joint name="right_wheel_joint" type="${wheel_joint_type}">
 			<origin xyz="0.0544 -0.1895 -0.0965"/>
 			<parent link="base_link"/>

File: humanoid/Zerith/zerith_h1_description/xacro/robot.xacro (robot description, xacro)
@@ -2,16 +2,13 @@
 <!-- =================================================================================== -->
 <!-- |    Complete Robot Description for Zerith H1                                     | -->
-<!-- |    This file includes the chassis, body and arm components                      | -->
+<!-- |    Chassis (wheels locked by default) + body/head + dual 7-DOF arms + grippers  | -->
 <!-- =================================================================================== -->
 <robot name="zerith_h1" xmlns:xacro="http://www.ros.org/wiki/xacro">
-	<!-- Include chassis macro -->
+	<!-- Lock drive wheels by default (W2/Bot2/Quanta/Galaxea). Planning URDF keeps this false. -->
+	<xacro:arg name="chassis_joints_movable" default="false"/>
 	<xacro:include filename="$(find zerith_h1_description)/xacro/components/chassis.xacro"/>
-	<!-- Generate chassis: drive_joint_type="continuous" (default) or "fixed" -->
-	<xacro:H1Chassis drive_joint_type="continuous"/>
-	<!-- Include the body (torso and head/neck) -->
+	<xacro:H1Chassis joints_movable="$(arg chassis_joints_movable)"/>
 	<xacro:include filename="$(find zerith_h1_description)/xacro/components/body.xacro"/>
-	<!-- Include arm macro -->
 	<xacro:include filename="$(find zerith_h1_description)/xacro/components/arm.xacro"/>
-	<!-- Generate left and right arms using macro -->
 	<xacro:H1Arm name="left" direction="1"/>
 	<xacro:H1Arm name="right" direction="-1"/>
