Commit message: Add Quanta X1 OCS2 support

File: humanoid/X2Robot/quanta_x1_description/xacro/components/arm.xacro (robot description, xacro)
@@ -2,5 +2,5 @@
 <robot xmlns:xacro="http://www.ros.org/wiki/xacro">
 	<xacro:include filename="$(find quanta_x1_description)/xacro/ros2_control/arm_ros2_control.xacro"/>
-	<xacro:macro name="QuantaX1SingleArm" params="name">
+	<xacro:macro name="QuantaX1SingleArm" params="name enable_ros2_control:=false">
 		<xacro:property name="prefix" value="${name + '_' if name else ''}"/>
 		<link name="${prefix}base_link">
@@ -167,5 +167,7 @@
 			<limit effort="9" lower="-1.9199" upper="1.9199" velocity="6.77"/>
 		</joint>
-		<xacro:QuantaX1ArmRos2Control prefix="${prefix}"/>
+		<xacro:if value="${enable_ros2_control}">
+			<xacro:QuantaX1ArmRos2Control prefix="${prefix}"/>
+		</xacro:if>
 		<link name="${prefix}gripper_base_link">
 			<inertial>
@@ -277,5 +279,13 @@
 			<child link="${prefix}gripper_base_link"/>
 		</joint>
-		<xacro:QuantaX1ArmGripperRos2Control prefix="${prefix}"/>
+		<link name="${prefix}eef"/>
+		<joint name="${prefix}eef_joint" type="fixed">
+			<origin xyz="0.10 0 0"/>
+			<parent link="${prefix}gripper_base_link"/>
+			<child link="${prefix}eef"/>
+		</joint>
+		<xacro:if value="${enable_ros2_control}">
+			<xacro:QuantaX1ArmGripperRos2Control prefix="${prefix}"/>
+		</xacro:if>
 	</xacro:macro>
 </robot>

File: humanoid/X2Robot/quanta_x1_description/xacro/components/base.xacro (robot description, xacro)
@@ -3,5 +3,5 @@
 	<xacro:include filename="$(find quanta_x1_description)/xacro/ros2_control/base_ros2_control.xacro"/>
 	<xacro:include filename="$(find quanta_x1_description)/xacro/components/swivel.xacro"/>
-	<xacro:macro name="QuantaX1Base">
+	<xacro:macro name="QuantaX1Base" params="enable_ros2_control:=false">
 		<link name="base_link"/>
 		<joint name="chassis_base_joint" type="fixed">
@@ -365,5 +365,7 @@
 			<child link="imu_link"/>
 		</joint>
-		<xacro:QuantaX1BaseRos2Control/>
+		<xacro:if value="${enable_ros2_control}">
+			<xacro:QuantaX1BaseRos2Control/>
+		</xacro:if>
 		<link name="2d_laser_base">
 			<inertial>

File: humanoid/X2Robot/quanta_x1_description/xacro/robot.xacro (robot description, xacro)
@@ -1,10 +1,11 @@
 <?xml version="1.0" ?>
 <robot name="Quanta X1" xmlns:xacro="http://www.ros.org/wiki/xacro">
+  <xacro:arg name="enable_ros2_control" default="false"/>
   <xacro:property name="PI" value="3.1415926535897931"/>
   <xacro:include filename="$(find quanta_x1_description)/xacro/components/base.xacro"/>
   <xacro:include filename="$(find quanta_x1_description)/xacro/components/arm.xacro"/>
-  <xacro:QuantaX1Base/>
-  <xacro:QuantaX1SingleArm name="left"/>
-  <xacro:QuantaX1SingleArm name="right"/>
+  <xacro:QuantaX1Base enable_ros2_control="$(arg enable_ros2_control)"/>
+  <xacro:QuantaX1SingleArm name="left" enable_ros2_control="$(arg enable_ros2_control)"/>
+  <xacro:QuantaX1SingleArm name="right" enable_ros2_control="$(arg enable_ros2_control)"/>
   <joint name="left_connector" type="fixed">
     <parent link="left_frame_link"/>
