Commit message: feat(quanta_x1): add Artixon 6A mock control stack (ARX-style grippers)
Wire ros2_control into a dedicated xacro, add controller + OCS2 configs,
and document mock/isaac launches. Grippers use left/right_gripper_joint
with adaptive_gripper_controller (ARX pattern); lift/head are separate
basic_joint controllers.

File: humanoid/X2Robot/quanta_x1_description/xacro/components/arm.xacro (robot description, xacro)
@@ -1,5 +1,4 @@
 <?xml version="1.0" ?>
 <robot xmlns:xacro="http://www.ros.org/wiki/xacro">
-	<xacro:include filename="$(find quanta_x1_description)/xacro/ros2_control/arm_ros2_control.xacro"/>
 	<xacro:macro name="QuantaX1SingleArm" params="name">
 		<xacro:property name="prefix" value="${name + '_' if name else ''}"/>
@@ -167,5 +166,4 @@
 			<limit effort="9" lower="-1.9199" upper="1.9199" velocity="6.77"/>
 		</joint>
-		<xacro:QuantaX1ArmRos2Control prefix="${prefix}"/>
 		<link name="${prefix}gripper_base_link">
 			<inertial>
@@ -277,5 +275,11 @@
 			<child link="${prefix}gripper_base_link"/>
 		</joint>
-		<xacro:QuantaX1ArmGripperRos2Control prefix="${prefix}"/>
+		<!-- TCP for OCS2 / cartesian (ARX-style ${prefix}gripper_center) -->
+		<link name="${prefix}gripper_center"/>
+		<joint name="${prefix}gripper_center_fixed" type="fixed">
+			<origin xyz="0.12 0 0"/>
+			<parent link="${prefix}gripper_base_link"/>
+			<child link="${prefix}gripper_center"/>
+		</joint>
 	</xacro:macro>
 </robot>

File: humanoid/X2Robot/quanta_x1_description/xacro/components/base.xacro (robot description, xacro)
@@ -1,5 +1,4 @@
 <?xml version="1.0" ?>
 <robot xmlns:xacro="http://www.ros.org/wiki/xacro">
-	<xacro:include filename="$(find quanta_x1_description)/xacro/ros2_control/base_ros2_control.xacro"/>
 	<xacro:include filename="$(find quanta_x1_description)/xacro/components/swivel.xacro"/>
 	<xacro:macro name="QuantaX1Base">
@@ -365,5 +364,4 @@
 			<child link="imu_link"/>
 		</joint>
-		<xacro:QuantaX1BaseRos2Control/>
 		<link name="2d_laser_base">
 			<inertial>

File: humanoid/X2Robot/quanta_x1_description/xacro/ros2_control/arm_ros2_control.xacro (robot description, xacro)
@@ -1,139 +1,41 @@
-<?xml version="1.0" ?>
+<?xml version="1.0"?>
 <robot xmlns:xacro="http://www.ros.org/wiki/xacro">
-  <xacro:macro name="QuantaX1ArmRos2Control" params="prefix">
-    <ros2_control name="${prefix}arm" type="system">
-      <hardware>
-        <plugin>mock_components/GenericSystem</plugin>
-      </hardware>
-      <joint name="${prefix}joint1">
-        <param name="motor_id">1</param>
-        <param name="master_id">17</param>
-        <param name="motor_type">dmmotor</param>
-        <param name="motor_hw_type">DM6248</param>
-        <param name="lower_limit">-2.792</param>
-        <param name="upper_limit">2.792</param>
-        <command_interface name="position"/>
+  <!-- Artixon 6A arm + ARX-style adaptive gripper interfaces.
+       iface_mode: mix = pos/vel/effort (mock/gz/real); position = pos only (Isaac). -->
+  <xacro:macro name="quanta_x1_arm_joint" params="jname iface_mode initial:=''">
+    <joint name="${jname}">
+      <command_interface name="position"/>
+      <xacro:if value="${iface_mode == 'mix'}">
         <command_interface name="velocity"/>
         <command_interface name="effort"/>
-        <command_interface name="mit_kp"/>
-        <command_interface name="mit_kd"/>
-        <command_interface name="ctrl_mode"/>
-        <state_interface name="position"/>
+      </xacro:if>
+      <state_interface name="position">
+        <xacro:unless value="${initial == ''}">
+          <param name="initial_value">${initial}</param>
+        </xacro:unless>
+      </state_interface>
+      <xacro:if value="${iface_mode == 'mix'}">
         <state_interface name="velocity"/>
         <state_interface name="effort"/>
-      </joint>
-      <joint name="${prefix}joint2">
-        <param name="motor_id">2</param>
-        <param name="master_id">18</param>
-        <param name="motor_type">dmmotor</param>
-        <param name="motor_hw_type">DM6248</param>
-        <param name="lower_limit">0.0</param>
-        <param name="upper_limit">3.44</param>
-        <command_interface name="position"/>
-        <command_interface name="velocity"/>
-        <command_interface name="effort"/>
-        <command_interface name="mit_kp"/>
-        <command_interface name="mit_kd"/>
-        <command_interface name="ctrl_mode"/>
-        <state_interface name="position"/>
+      </xacro:if>
+    </joint>
+  </xacro:macro>
+  <xacro:macro name="quanta_x1_arm_interfaces" params="name iface_mode:=mix">
+    <xacro:property name="prefix" value="${name + '_' if name else ''}"/>
+    <xacro:quanta_x1_arm_joint jname="${prefix}joint1" iface_mode="${iface_mode}"/>
+    <xacro:quanta_x1_arm_joint jname="${prefix}joint2" iface_mode="${iface_mode}"/>
+    <xacro:quanta_x1_arm_joint jname="${prefix}joint3" iface_mode="${iface_mode}"/>
+    <xacro:quanta_x1_arm_joint jname="${prefix}joint4" iface_mode="${iface_mode}"/>
+    <xacro:quanta_x1_arm_joint jname="${prefix}joint5" iface_mode="${iface_mode}"/>
+    <xacro:quanta_x1_arm_joint jname="${prefix}joint6" iface_mode="${iface_mode}"/>
+    <!-- AdaptiveGripperController drives ${prefix}gripper_joint (mimic fingers follow). -->
+    <joint name="${prefix}gripper_joint">
+      <command_interface name="position"/>
+      <state_interface name="position"/>
+      <xacro:if value="${iface_mode == 'mix'}">
         <state_interface name="velocity"/>
         <state_interface name="effort"/>
-      </joint>
-      <joint name="${prefix}joint3">
-        <param name="motor_id">3</param>
-        <param name="master_id">19</param>
-        <param name="motor_type">dmmotor</param>
-        <param name="motor_hw_type">DM6248</param>
-        <param name="direction">-1.0</param>
-        <param name="lower_limit">-3.14</param>
-        <param name="upper_limit">0.0</param>
-        <command_interface name="position"/>
-        <command_interface name="velocity"/>
-        <command_interface name="effort"/>
-        <command_interface name="mit_kp"/>
-        <command_interface name="mit_kd"/>
-        <command_interface name="ctrl_mode"/>
-        <state_interface name="position"/>
-        <state_interface name="velocity"/>
-        <state_interface name="effort"/>
-      </joint>
-      <joint name="${prefix}joint4">
-        <param name="motor_id">4</param>
-        <param name="master_id">20</param>
-        <param name="motor_type">dmmotor</param>
-        <param name="motor_hw_type">DM4340_48</param>
-        <param name="direction">-1.0</param>
-        <param name="lower_limit">-1.57</param>
-        <param name="upper_limit">1.57</param>
-        <command_interface name="position"/>
-        <command_interface name="velocity"/>
-        <command_interface name="effort"/>
-        <command_interface name="mit_kp"/>
-        <command_interface name="mit_kd"/>
-        <command_interface name="ctrl_mode"/>
-        <state_interface name="position"/>
-        <state_interface name="velocity"/>
-        <state_interface name="effort"/>
-      </joint>
-      <joint name="${prefix}joint5">
-        <param name="motor_id">5</param>
-        <param name="master_id">21</param>
-        <param name="motor_type">dmmotor</param>
-        <param name="motor_hw_type">DM4340_48</param>
-        <param name="direction">-1.0</param>
-        <param name="lower_limit">-1.4</param>
-        <param name="upper_limit">1.4</param>
-        <command_interface name="position"/>
-        <command_interface name="velocity"/>
-        <command_interface name="effort"/>
-        <command_interface name="mit_kp"/>
-        <command_interface name="mit_kd"/>
-        <command_interface name="ctrl_mode"/>
-        <state_interface name="position"/>
-        <state_interface name="velocity"/>
-        <state_interface name="effort"/>
-      </joint>
-      <joint name="${prefix}joint6">
-        <param name="motor_id">6</param>
-        <param name="master_id">22</param>
-        <param name="motor_type">dmmotor</param>
-        <param name="motor_hw_type">DM4340_48</param>
-        <param name="lower_limit">-1.745</param>
-        <param name="upper_limit">1.745</param>
-        <command_interface name="position"/>
-        <command_interface name="velocity"/>
-        <command_interface name="effort"/>
-        <command_interface name="mit_kp"/>
-        <command_interface name="mit_kd"/>
-        <command_interface name="ctrl_mode"/>
-        <state_interface name="position"/>
-        <state_interface name="velocity"/>
-        <state_interface name="effort"/>
-      </joint>
-    </ros2_control>
-  </xacro:macro>
-  <xacro:macro name="QuantaX1ArmGripperRos2Control" params="prefix">
-    <ros2_control name="${prefix}gripper" type="system">
-      <hardware>
-        <plugin>mock_components/GenericSystem</plugin>
-      </hardware>
-      <joint name="${prefix}gripper_joint">
-        <param name="motor_id">8</param>
-        <param name="master_id">0</param>
-        <param name="motor_type">dmmotor</param>
-        <param name="motor_hw_type">DM4310</param>
-        <param name="max_torque">2.0</param>
-        <param name="default_mode">tor</param>
-        <command_interface name="position"/>
-        <command_interface name="velocity"/>
-        <command_interface name="effort"/>
-        <command_interface name="mit_kp"/>
-        <command_interface name="mit_kd"/>
-        <command_interface name="ctrl_mode"/>
-        <state_interface name="position"/>
-        <state_interface name="velocity"/>
-        <state_interface name="effort"/>
-      </joint>
-    </ros2_control>
+      </xacro:if>
+    </joint>
   </xacro:macro>
 </robot>

File: humanoid/X2Robot/quanta_x1_description/xacro/ros2_control/base_ros2_control.xacro (robot description, xacro)
@@ -1,18 +1,60 @@
-<?xml version="1.0" ?>
+<?xml version="1.0"?>
 <robot xmlns:xacro="http://www.ros.org/wiki/xacro">
-  <xacro:macro name="QuantaX1BaseRos2Control">
-      <ros2_control is_async="true" name="mobile_base" rw_rate="250" type="system">
-        <hardware>
-          <plugin>mock_components/GenericSystem</plugin>
-        </hardware>
-        <joint name="lift_joint">
-          <command_interface name="position"/>
-          <command_interface name="velocity"/>
-          <command_interface name="effort"/>
-          <state_interface name="position"/>
-          <state_interface name="velocity"/>
-          <state_interface name="effort"/>
-        </joint>
-      </ros2_control>
+  <!-- Quanta X1 base: lift + head; optional drive wheels. -->
+  <xacro:macro name="quanta_x1_wheel_interfaces">
+    <joint name="left_wheel_joint">
+      <command_interface name="velocity">
+        <param name="min">-10.0</param>
+        <param name="max">10.0</param>
+      </command_interface>
+      <state_interface name="position"/>
+      <state_interface name="velocity"/>
+      <state_interface name="effort"/>
+    </joint>
+    <joint name="right_wheel_joint">
+      <command_interface name="velocity">
+        <param name="min">-10.0</param>
+        <param name="max">10.0</param>
+      </command_interface>
+      <state_interface name="position"/>
+      <state_interface name="velocity"/>
+      <state_interface name="effort"/>
+    </joint>
+  </xacro:macro>
+  <xacro:macro name="quanta_x1_base_interfaces" params="iface_mode:=mix">
+    <joint name="lift_joint">
+      <command_interface name="position"/>
+      <xacro:if value="${iface_mode == 'mix'}">
+        <command_interface name="velocity"/>
+        <command_interface name="effort"/>
+      </xacro:if>
+      <state_interface name="position">
+        <param name="initial_value">0.0</param>
+      </state_interface>
+      <xacro:if value="${iface_mode == 'mix'}">
+        <state_interface name="velocity"/>
+        <state_interface name="effort"/>
+      </xacro:if>
+    </joint>
+    <joint name="head_yaw_joint">
+      <command_interface name="position"/>
+      <state_interface name="position">
+        <param name="initial_value">0.0</param>
+      </state_interface>
+      <xacro:if value="${iface_mode == 'mix'}">
+        <state_interface name="velocity"/>
+        <state_interface name="effort"/>
+      </xacro:if>
+    </joint>
+    <joint name="head_pitch_joint">
+      <command_interface name="position"/>
+      <state_interface name="position">
+        <param name="initial_value">0.0</param>
+      </state_interface>
+      <xacro:if value="${iface_mode == 'mix'}">
+        <state_interface name="velocity"/>
+        <state_interface name="effort"/>
+      </xacro:if>
+    </joint>
   </xacro:macro>
 </robot>

Commit message: revert(quanta_x1): drop convex/CoACD collision meshes from description
Collision hull/decompose work belongs on the IsaacSim bot, not this
description PR. Restore prior arm/gripper collision STLs and xacro
wiring; keep WBC Pinocchio order, target_manager, and modeSequence.

File: humanoid/X2Robot/quanta_x1_description/xacro/components/arm.xacro (robot description, xacro)
@@ -158,9 +158,4 @@
 				</geometry>
 			</visual>
-			<collision>
-				<geometry>
-					<mesh filename="file://$(find quanta_x1_description)/meshes/arm/collision/arm_link6.STL"/>
-				</geometry>
-			</collision>
 		</link>
 		<joint name="${prefix}joint6" type="revolute">
@@ -182,18 +177,7 @@
 				</geometry>
 			</visual>
-			<!-- 夹爪支架: CoACD 3 convex pieces -->
-			<collision>
-				<geometry>
-					<mesh filename="file://$(find quanta_x1_description)/meshes/gripper/collision/gripper_base_link_0.stl"/>
-				</geometry>
-			</collision>
-			<collision>
-				<geometry>
-					<mesh filename="file://$(find quanta_x1_description)/meshes/gripper/collision/gripper_base_link_1.stl"/>
-				</geometry>
-			</collision>
-			<collision>
-				<geometry>
-					<mesh filename="file://$(find quanta_x1_description)/meshes/gripper/collision/gripper_base_link_2.stl"/>
+			<collision>
+				<geometry>
+					<mesh filename="file://$(find quanta_x1_description)/meshes/gripper/collision/gripper_base_link.STL"/>
 				</geometry>
 			</collision>
@@ -212,9 +196,4 @@
 				</material>
 			</visual>
-			<collision>
-				<geometry>
-					<mesh filename="file://$(find quanta_x1_description)/meshes/gripper/collision/gripper_motor.STL"/>
-				</geometry>
-			</collision>
 		</link>
 		<joint name="${prefix}gripper_joint" type="revolute">
@@ -286,20 +265,4 @@
 				</geometry>
 			</visual>
-			<!-- wrist camera: CoACD 3 convex pieces -->
-			<collision>
-				<geometry>
-					<mesh filename="file://$(find quanta_x1_description)/meshes/gripper/collision/gripper_camera_0.stl"/>
-				</geometry>
-			</collision>
-			<collision>
-				<geometry>
-					<mesh filename="file://$(find quanta_x1_description)/meshes/gripper/collision/gripper_camera_1.stl"/>
-				</geometry>
-			</collision>
-			<collision>
-				<geometry>
-					<mesh filename="file://$(find quanta_x1_description)/meshes/gripper/collision/gripper_camera_2.stl"/>
-				</geometry>
-			</collision>
 		</link>
 		<joint name="${prefix}gripper_camera_base_joint" type="fixed">
