Commit message: quanta_x1: enable HEAD_GAZE head follow (head_camera optical + headMidpointGaze)
Add ROS-optical head_camera on Dabai mount, switch modeSequence to HEAD_GAZE,
lower head input costs, keep body tracking and no customJointLock (like MMK2/Zerith).

File: humanoid/X2Robot/quanta_x1_description/xacro/components/head.xacro (robot description, xacro)
@@ -64,4 +64,11 @@
 			<child link="head_camera_frame_link"/>
 		</joint>
+		<!-- ROS optical (+Z forward, +X right, +Y down) for OCS2 HEAD_GAZE; CAD mesh stays on head_camera_frame_link. -->
+		<link name="head_camera"/>
+		<joint name="head_camera_optical_joint" type="fixed">
+			<origin xyz="0 0 0" rpy="${-PI/2} 0 ${-PI/2}"/>
+			<parent link="head_camera_frame_link"/>
+			<child link="head_camera"/>
+		</joint>
 	</xacro:macro>
 </robot>
