Commit message: modified galaxea r1 pro

File: humanoid/Galaxea/galaxea_r1pro_description/xacro/component.xacro (robot description, xacro)
@@ -1,13 +1,22 @@
 <?xml version="1.0" ?>
 <!-- =================================================================================== -->
-<!-- |    Complete Robot Description for Agibot G1                                     | -->
-<!-- |    This file includes the base robot structure and both arms                    | -->
+<!-- |    Component descriptions for Galaxea R1 Pro                                    | -->
 <!-- =================================================================================== -->
-<robot name="A2_Arm" xmlns:xacro="http://www.ros.org/wiki/xacro">
+<robot name="Galaxea_R1_Pro" xmlns:xacro="http://www.ros.org/wiki/xacro">
 	<xacro:property name="PI" value="3.1415926535897931"/>
 	<xacro:arg name="type" default="arms"/>
+	<xacro:arg name="enable_wheel_joints" default="true"/>
+	<xacro:if value="${'$(arg type)' == 'chassis'}">
+		<xacro:include filename="$(find galaxea_r1_description)/xacro/components/chassis.xacro"/>
+		<xacro:Chassis enable_wheel_joints="$(arg enable_wheel_joints)"/>
+	</xacro:if>
+	<xacro:if value="${'$(arg type)' == 'torso'}">
+		<xacro:include filename="$(find galaxea_r1_description)/xacro/components/torso.xacro"/>
+		<link name="base_link"/>
+		<xacro:Torso/>
+	</xacro:if>
 	<xacro:if value="${'$(arg type)' == 'arms'}">
 		<link name="torso_link4"/>
-		<xacro:include filename="pro_arm.xacro"/>
+		<xacro:include filename="$(find galaxea_r1pro_description)/xacro/components/pro_arm.xacro"/>
 		<xacro:Arm name="left"/>
 		<xacro:Arm name="right" direction="-1"/>

File: humanoid/Galaxea/galaxea_r1pro_description/xacro/components/pro_arm.xacro (robot description, xacro)
@@ -12,13 +12,9 @@
 			</inertial>
 			<visual>
-				<geometry>
-					<mesh filename="file://$(find galaxea_r1pro_description)/meshes/pro_arm/base.obj" scale="1 ${direction} 1"/>
-				</geometry>
-			</visual>
-			<collision>
-				<geometry>
-					<mesh filename="file://$(find galaxea_r1pro_description)/meshes/pro_arm/base.obj" scale="1 ${direction} 1"/>
-				</geometry>
-			</collision>
+				<origin rpy="0 ${PI/2} ${PI/2 * direction}"/>
+				<geometry>
+					<mesh filename="file://$(find galaxea_a1_description)/meshes/a1/base.glb"/>
+				</geometry>
+			</visual>
 		</link>
 		<!-- Arm Link 1 -->
@@ -32,10 +28,10 @@
 			<visual>
 				<geometry>
-					<mesh filename="file://$(find galaxea_r1pro_description)/meshes/pro_arm/link1.obj" scale="1 ${direction} 1"/>
-				</geometry>
-			</visual>
-			<collision>
-				<geometry>
-					<mesh filename="file://$(find galaxea_r1pro_description)/meshes/pro_arm/link1.obj" scale="1 ${direction} 1"/>
+					<mesh filename="file://$(find galaxea_r1pro_description)/meshes/a2_arm/link1.glb" scale="1 ${direction} 1"/>
+				</geometry>
+			</visual>
+			<collision>
+				<geometry>
+					<mesh filename="file://$(find galaxea_r1pro_description)/meshes/a2_arm/link1.glb" scale="1 ${direction} 1"/>
 				</geometry>
 			</collision>
@@ -51,10 +47,10 @@
 			<visual>
 				<geometry>
-					<mesh filename="file://$(find galaxea_r1pro_description)/meshes/pro_arm/link2.obj" scale="1 ${direction} 1"/>
-				</geometry>
-			</visual>
-			<collision>
-				<geometry>
-					<mesh filename="file://$(find galaxea_r1pro_description)/meshes/pro_arm/link2.obj" scale="1 ${direction} 1"/>
+					<mesh filename="file://$(find galaxea_r1pro_description)/meshes/a2_arm/link2.glb" scale="1 ${direction} 1"/>
+				</geometry>
+			</visual>
+			<collision>
+				<geometry>
+					<mesh filename="file://$(find galaxea_r1pro_description)/meshes/a2_arm/link2.glb" scale="1 ${direction} 1"/>
 				</geometry>
 			</collision>
@@ -70,10 +66,10 @@
 			<visual>
 				<geometry>
-					<mesh filename="file://$(find galaxea_r1pro_description)/meshes/pro_arm/link3.obj"/>
-				</geometry>
-			</visual>
-			<collision>
-				<geometry>
-					<mesh filename="file://$(find galaxea_r1pro_description)/meshes/pro_arm/link3.obj"/>
+					<mesh filename="file://$(find galaxea_r1pro_description)/meshes/a2_arm/link3.glb"/>
+				</geometry>
+			</visual>
+			<collision>
+				<geometry>
+					<mesh filename="file://$(find galaxea_r1pro_description)/meshes/a2_arm/link3.glb"/>
 				</geometry>
 			</collision>
@@ -89,10 +85,10 @@
 			<visual>
 				<geometry>
-					<mesh filename="file://$(find galaxea_r1pro_description)/meshes/pro_arm/link4.obj"/>
-				</geometry>
-			</visual>
-			<collision>
-				<geometry>
-					<mesh filename="file://$(find galaxea_r1pro_description)/meshes/pro_arm/link4.obj"/>
+					<mesh filename="file://$(find galaxea_r1pro_description)/meshes/a2_arm/link4.glb"/>
+				</geometry>
+			</visual>
+			<collision>
+				<geometry>
+					<mesh filename="file://$(find galaxea_r1pro_description)/meshes/a2_arm/link4.glb"/>
 				</geometry>
 			</collision>
@@ -108,10 +104,10 @@
 			<visual>
 				<geometry>
-					<mesh filename="file://$(find galaxea_r1pro_description)/meshes/pro_arm/link5.obj" scale="1 ${direction} 1"/>
-				</geometry>
-			</visual>
-			<collision>
-				<geometry>
-					<mesh filename="file://$(find galaxea_r1pro_description)/meshes/pro_arm/link5.obj" scale="1 ${direction} 1"/>
+					<mesh filename="file://$(find galaxea_r1pro_description)/meshes/a2_arm/link5.glb" scale="1 ${direction} 1"/>
+				</geometry>
+			</visual>
+			<collision>
+				<geometry>
+					<mesh filename="file://$(find galaxea_r1pro_description)/meshes/a2_arm/link5.glb" scale="1 ${direction} 1"/>
 				</geometry>
 			</collision>
@@ -127,10 +123,10 @@
 			<visual>
 				<geometry>
-					<mesh filename="file://$(find galaxea_r1pro_description)/meshes/pro_arm/link6.obj" scale="1 ${direction} 1"/>
-				</geometry>
-			</visual>
-			<collision>
-				<geometry>
-					<mesh filename="file://$(find galaxea_r1pro_description)/meshes/pro_arm/link6.obj" scale="1 ${direction} 1"/>
+					<mesh filename="file://$(find galaxea_r1pro_description)/meshes/a2_arm/link6.glb" scale="1 ${direction} 1"/>
+				</geometry>
+			</visual>
+			<collision>
+				<geometry>
+					<mesh filename="file://$(find galaxea_r1pro_description)/meshes/a2_arm/link6.glb" scale="1 ${direction} 1"/>
 				</geometry>
 			</collision>
@@ -146,10 +142,10 @@
 			<visual>
 				<geometry>
-					<mesh filename="file://$(find galaxea_r1pro_description)/meshes/pro_arm/link7.obj"/>
-				</geometry>
-			</visual>
-			<collision>
-				<geometry>
-					<mesh filename="file://$(find galaxea_r1pro_description)/meshes/pro_arm/link7.obj"/>
+					<mesh filename="file://$(find galaxea_r1pro_description)/meshes/a2_arm/link7.glb"/>
+				</geometry>
+			</visual>
+			<collision>
+				<geometry>
+					<mesh filename="file://$(find galaxea_r1pro_description)/meshes/a2_arm/link7.glb"/>
 				</geometry>
 			</collision>

File: humanoid/Galaxea/galaxea_r1pro_description/xacro/components/realsense.xacro (robot description, xacro)
@@ -13,5 +13,5 @@
       <visual>
         <geometry>
-          <mesh filename="file://$(find galaxea_r1_description)/meshes/camera_stand.obj"/>
+          <mesh filename="file://$(find galaxea_r1_description)/meshes/hand_camera_stand.glb"/>
         </geometry>
       </visual>
@@ -22,9 +22,4 @@
         </geometry>
       </visual>
-      <collision>
-        <geometry>
-          <mesh filename="file://$(find galaxea_r1_description)/meshes/camera_stand.obj"/>
-        </geometry>
-      </collision>
     </link>
     <!-- RealSense Joint: Arm 7 to Camera -->

File: humanoid/Galaxea/galaxea_r1pro_description/xacro/robot.xacro (robot description, xacro)
@@ -1,14 +1,16 @@
 <?xml version="1.0" encoding="utf-8"?>
 <robot name="R1Pro" xmlns:xacro="http://www.ros.org/wiki/xacro">
+  <xacro:property name="PI" value="3.1415926535897931"/>
+  <xacro:arg name="enable_wheel_joints" default="false"/>
   <!-- Include Chassis -->
-  <xacro:include filename="$(find galaxea_r1_description)/xacro/chassis.xacro"/>
-  <xacro:Chassis/>
+  <xacro:include filename="$(find galaxea_r1_description)/xacro/components/chassis.xacro"/>
+  <xacro:Chassis enable_wheel_joints="$(arg enable_wheel_joints)"/>
   <!-- Include Torso -->
-  <xacro:include filename="$(find galaxea_r1_description)/xacro/torso.xacro"/>
+  <xacro:include filename="$(find galaxea_r1_description)/xacro/components/torso.xacro"/>
   <xacro:Torso/>
-  <xacro:include filename="pro_arm.xacro"/>
+  <xacro:include filename="$(find galaxea_r1pro_description)/xacro/components/pro_arm.xacro"/>
   <xacro:Arm name="left"/>
   <xacro:Arm name="right" direction="-1"/>
-  <xacro:include filename="$(find galaxea_r1pro_description)/xacro/realsense.xacro"/>
+  <xacro:include filename="$(find galaxea_r1pro_description)/xacro/components/realsense.xacro"/>
   <xacro:RealSense side="left"/>
   <xacro:RealSense side="right"/>

File: manipulator/Galaxea/galaxea_r1lite_description/xacro/component.xacro (robot description, xacro)
@@ -1,12 +1,26 @@
 <?xml version="1.0" ?>
 <!-- =================================================================================== -->
-<!-- |    Complete Robot Description for Agibot G1                                     | -->
-<!-- |    This file includes the base robot structure and both arms                    | -->
+<!-- |    Component descriptions for Galaxea R1 Lite                                   | -->
 <!-- =================================================================================== -->
 <robot name="Galaxea_R1_Lite" xmlns:xacro="http://www.ros.org/wiki/xacro">
 	<xacro:property name="PI" value="3.1415926535897931"/>
 	<xacro:arg name="type" default="base"/>
+	<xacro:arg name="enable_wheel_joints" default="true"/>
+	<xacro:if value="${'$(arg type)' == 'chassis'}">
+		<xacro:include filename="$(find galaxea_r1lite_description)/xacro/components/chassis.xacro"/>
+		<xacro:Chassis enable_wheel_joints="$(arg enable_wheel_joints)"/>
+	</xacro:if>
+	<xacro:if value="${'$(arg type)' == 'torso'}">
+		<xacro:include filename="$(find galaxea_r1lite_description)/xacro/components/torso.xacro"/>
+		<link name="base_link"/>
+		<xacro:Torso/>
+		<link name="left_base_link"/>
+		<link name="right_base_link"/>
+	</xacro:if>
 	<xacro:if value="${'$(arg type)' == 'base'}">
-		<xacro:include filename="$(find galaxea_r1lite_description)/xacro/chassis.xacro"/>
+		<xacro:include filename="$(find galaxea_r1lite_description)/xacro/components/chassis.xacro"/>
+		<xacro:include filename="$(find galaxea_r1lite_description)/xacro/components/torso.xacro"/>
+		<xacro:Chassis enable_wheel_joints="$(arg enable_wheel_joints)"/>
+		<xacro:Torso/>
 		<link name="left_base_link"/>
 		<link name="right_base_link"/>
@@ -14,5 +28,5 @@
 	<xacro:if value="${'$(arg type)' == 'a1x'}">
 		<xacro:include filename="$(find galaxea_a1_description)/xacro/a1_x.xacro"/>
-		<xacro:include filename="$(find galaxea_r1lite_description)/xacro/camera.xacro"/>
+		<xacro:include filename="$(find galaxea_r1lite_description)/xacro/components/camera.xacro"/>
 		<xacro:Arm name=""/>
 		<xacro:camera name=""/>
@@ -20,5 +34,5 @@
 	<xacro:if value="${'$(arg type)' == 'a1y'}">
 		<xacro:include filename="$(find galaxea_a1_description)/xacro/a1_y.xacro"/>
-		<xacro:include filename="$(find galaxea_r1lite_description)/xacro/camera.xacro"/>
+		<xacro:include filename="$(find galaxea_r1lite_description)/xacro/components/camera.xacro"/>
 		<xacro:Arm name=""/>
 		<xacro:camera name=""/>

File: manipulator/Galaxea/galaxea_r1lite_description/xacro/components/camera.xacro (robot description, xacro)
@@ -1,4 +1,5 @@
 <?xml version="1.0" encoding="utf-8"?>
 <robot xmlns:xacro="http://www.ros.org/wiki/xacro">
+	<xacro:property name="PI" value="3.1415926535897931"/>
 	<xacro:macro name="camera" params="name">
 		<xacro:property name="prefix" value="${name + '_' if name else ''}"/>
@@ -11,5 +12,5 @@
 			<visual>
 				<geometry>
-					<mesh filename="file://$(find galaxea_r1lite_description)/meshes/visual/camera_stand.obj"/>
+					<mesh filename="file://$(find galaxea_r1lite_description)/meshes/visual/camera_stand.glb"/>
 				</geometry>
 			</visual>

File: manipulator/Galaxea/galaxea_r1lite_description/xacro/robot.xacro (robot description, xacro)
@@ -5,6 +5,10 @@
 <robot name="A1Lite" xmlns:xacro="http://www.ros.org/wiki/xacro">
 	<xacro:property name="PI" value="3.1415926535897931"/>
-	<xacro:include filename="$(find galaxea_r1lite_description)/xacro/chassis.xacro"/>
-	<xacro:include filename="$(find galaxea_r1lite_description)/xacro/camera.xacro"/>
+	<xacro:arg name="enable_wheel_joints" default="false"/>
+	<xacro:include filename="$(find galaxea_r1lite_description)/xacro/components/chassis.xacro"/>
+	<xacro:Chassis enable_wheel_joints="$(arg enable_wheel_joints)"/>
+	<xacro:include filename="$(find galaxea_r1lite_description)/xacro/components/torso.xacro"/>
+	<xacro:Torso/>
+	<xacro:include filename="$(find galaxea_r1lite_description)/xacro/components/camera.xacro"/>
 	<xacro:arg name="type" default="x"/>
 	<xacro:if value="${'$(arg type)' == 'x'}">

Commit message: add wbc config for galaxea r1

File: humanoid/Galaxea/galaxea_r1pro_description/xacro/component.xacro (robot description, xacro)
@@ -3,5 +3,5 @@
 <!-- |    Component descriptions for Galaxea R1 Pro                                    | -->
 <!-- =================================================================================== -->
-<robot name="Galaxea_R1_Pro" xmlns:xacro="http://www.ros.org/wiki/xacro">
+<robot name="A2 Arms" xmlns:xacro="http://www.ros.org/wiki/xacro">
 	<xacro:property name="PI" value="3.1415926535897931"/>
 	<xacro:arg name="type" default="arms"/>

File: humanoid/Galaxea/galaxea_r1pro_description/xacro/components/pro_arm.xacro (robot description, xacro)
@@ -169,6 +169,11 @@
 			<parent link="${prefix}link1"/>
 			<child link="${prefix}link2"/>
-			<axis xyz="${direction} 0 0"/>
-			<limit lower="-0.1745" upper="${PI}" effort="55" velocity="7.1209"/>
+			<axis xyz="1 0 0"/>
+			<xacro:if value="${direction == 1}">
+				<limit lower="-0.1745" upper="${PI}" effort="55" velocity="7.1209"/>
+			</xacro:if>
+			<xacro:unless value="${direction == 1}">
+				<limit lower="${-PI}" upper="0.1745" effort="55" velocity="7.1209"/>
+			</xacro:unless>
 		</joint>
 		<joint name="${prefix}joint3" type="revolute">
@@ -184,5 +189,5 @@
 			<child link="${prefix}link4"/>
 			<axis xyz="0 1 0"/>
-			<limit lower="-2.0944" upper="0.3491" effort="25" velocity="8.3776"/>
+			<limit lower="-1.7453" upper="0.3491" effort="25" velocity="8.3776"/>
 		</joint>
 		<joint name="${prefix}joint5" type="revolute">
