Commit message: fix color problems for moz1

File: humanoid/SpiritAI/moz1_description/xacro/component.xacro (robot description, xacro)
@@ -2,13 +2,4 @@
 <robot name="MOZ1_component" xmlns:xacro="http://www.ros.org/wiki/xacro">
   <xacro:arg name="type" default="chassis"/>
-  <material name="black_color">
-    <color rgba="0.1 0.1 0.1 1.0"/>
-  </material>
-  <material name="dark_gray">
-    <color rgba="0.216 0.220 0.224 1.0"/>
-  </material>
-  <material name="light_gray">
-    <color rgba="0.392 0.400 0.404 1.0"/>
-  </material>
   <xacro:include filename="$(find moz1_description)/xacro/components/chassis.xacro"/>
   <xacro:include filename="$(find moz1_description)/xacro/components/body.xacro"/>

File: humanoid/SpiritAI/moz1_description/xacro/components/chassis.xacro (robot description, xacro)
@@ -24,5 +24,4 @@
 					<mesh filename="file://$(find moz1_description)//meshes/chassis.glb"/>
 				</geometry>
-				<material name="dark_gray"/>
 			</visual>
 			<collision>

File: humanoid/SpiritAI/moz1_description/xacro/robot.xacro (robot description, xacro)
@@ -7,13 +7,4 @@
   <xacro:arg name="eef_fixed_joints" default="false"/>
   <xacro:property name="eef_fixed" value="$(arg eef_fixed_joints)"/>
-  <material name="black_color">
-    <color rgba="0.1 0.1 0.1 1.0"/>
-  </material>
-  <material name="dark_gray">
-    <color rgba="0.216 0.220 0.224 1.0"/>
-  </material>
-  <material name="light_gray">
-    <color rgba="0.392 0.400 0.404 1.0"/>
-  </material>
   <xacro:include filename="$(find moz1_description)/xacro/components/chassis.xacro"/>
   <xacro:include filename="$(find moz1_description)/xacro/components/body.xacro"/>
