Commit message: fix moz1

File: humanoid/SpiritAI/moz1_description/xacro/component.xacro (robot description, xacro)
@@ -1,5 +1,7 @@
 <?xml version="1.0"?>
-<robot name="MOZ1_component" xmlns:xacro="http://www.ros.org/wiki/xacro">
+<robot name="MOZ1" xmlns:xacro="http://www.ros.org/wiki/xacro">
   <xacro:arg name="type" default="chassis"/>
+  <!-- Isaac asset import: hide sensor_models meshes that Isaac already provides. -->
+  <xacro:arg name="isaac" default="false"/>
   <xacro:include filename="$(find moz1_description)/xacro/components/chassis.xacro"/>
   <xacro:include filename="$(find moz1_description)/xacro/components/body.xacro"/>
@@ -19,4 +21,12 @@
     <xacro:Moz1Body parent_link="base_link"/>
   </xacro:if>
+  <!-- Upper body: 6-DoF torso + head + dual arms (no chassis/gripper). -->
+  <xacro:if value="${'$(arg type)' == 'upper_body'}">
+    <link name="base_link"/>
+    <xacro:Moz1Body parent_link="base_link"/>
+    <xacro:Moz1Head parent_link="waist03" isaac="$(arg isaac)"/>
+    <xacro:Moz1Arm parent_link="waist03" direction="1" enable_gripper="false"/>
+    <xacro:Moz1Arm parent_link="waist03" direction="-1" enable_gripper="false"/>
+  </xacro:if>
   <xacro:if value="${'$(arg type)' == 'left_arm'}">
     <link name="waist03"/>
@@ -34,5 +44,5 @@
   <xacro:if value="${'$(arg type)' == 'head'}">
     <link name="waist03"/>
-    <xacro:Moz1Head parent_link="waist03"/>
+    <xacro:Moz1Head parent_link="waist03" isaac="$(arg isaac)"/>
   </xacro:if>
   <xacro:if value="${'$(arg type)' == 'gripper'}">

File: humanoid/SpiritAI/moz1_description/xacro/components/arm.xacro (robot description, xacro)
@@ -4,5 +4,5 @@
 	<xacro:include filename="$(find moz1_description)/xacro/components/omni_gripper.xacro"/>
 	<!-- direction:=1 left arm, direction:=-1 right arm (mirror mount & asymmetric limits). -->
-	<xacro:macro name="Moz1Arm" params="parent_link:=waist03 direction:=1 kinematic_only:=false">
+	<xacro:macro name="Moz1Arm" params="parent_link:=waist03 direction:=1 kinematic_only:=false enable_gripper:=true">
 		<xacro:if value="${direction == 1}">
 			<xacro:property name="prefix" value="left"/>
@@ -277,5 +277,7 @@
 			</xacro:unless>
 		</joint>
-		<xacro:Moz1OmniGripper direction="${direction}" kinematic_only="${kinematic_only}"/>
+		<xacro:if value="${enable_gripper}">
+			<xacro:Moz1OmniGripper direction="${direction}" kinematic_only="${kinematic_only}"/>
+		</xacro:if>
 	</xacro:macro>
 </robot>

File: humanoid/SpiritAI/moz1_description/xacro/components/head.xacro (robot description, xacro)
@@ -2,7 +2,8 @@
 <robot xmlns:xacro="http://www.ros.org/wiki/xacro">
 	<xacro:property name="PI" value="3.141592653589793"/>
-	<xacro:macro name="Moz1Head" params="parent_link:=waist03">
-		<!-- head21: mount on ROS waist03; mesh yaw -90° for CAD alignment. -->
-		<link name="head21">
+	<!-- isaac:=true hides sensor_models camera meshes (Isaac asset import). -->
+	<xacro:macro name="Moz1Head" params="parent_link:=waist03 isaac:=false">
+		<!-- head_base_link: mount on ROS waist03; mesh yaw -90° for CAD alignment. -->
+		<link name="head_base_link">
 			<inertial>
 				<origin xyz="-0.0024550600000000002 0.010183999999999999 0.00271658"/>
@@ -22,10 +23,10 @@
 			</visual>
 		</link>
-		<joint name="Head-0" type="fixed">
+		<joint name="head_fixed_joint" type="fixed">
 			<origin xyz="0 0 0.096" rpy="0 0 ${PI/2}"/>
 			<parent link="${parent_link}"/>
-			<child link="head21"/>
+			<child link="head_base_link"/>
 		</joint>
-		<link name="head22">
+		<link name="head_link1">
 			<inertial>
 				<origin xyz="0.00787245 -1.155e-05 0.0024877099999999997"/>
@@ -45,12 +46,12 @@
 			</visual>
 		</link>
-		<joint name="Head-1" type="revolute">
+		<joint name="head_joint1" type="revolute">
 			<origin xyz="0 0 0.103"/>
-			<parent link="head21"/>
-			<child link="head22"/>
+			<parent link="head_base_link"/>
+			<child link="head_link1"/>
 			<axis xyz="1 0 0"/>
 			<limit lower="${-3/180*PI}" upper="${50/180*PI}" effort="0" velocity="${114.6/180*PI}"/>
 		</joint>
-		<link name="head23">
+		<link name="head_link2">
 			<inertial>
 				<origin xyz="0.0015001 2.027e-05 0.03197392"/>
@@ -75,21 +76,23 @@
 			</collision>
 		</link>
-		<joint name="Head-2" type="revolute">
+		<joint name="head_joint2" type="revolute">
 			<origin xyz="0 0 0.04"/>
-			<parent link="head22"/>
-			<child link="head23"/>
+			<parent link="head_link1"/>
+			<child link="head_link2"/>
 			<axis xyz="0 0 1"/>
 			<limit lower="${-65/180*PI}" upper="${65/180*PI}" effort="0" velocity="${114.6/180*PI}"/>
 		</joint>
 		<link name="head_camera">
-			<visual>
-				<geometry>
-					<mesh filename="file://$(find sensor_models)/meshes/orbbec/336L.glb"/>
-				</geometry>
-			</visual>
+			<xacro:unless value="${isaac}">
+				<visual>
+					<geometry>
+						<mesh filename="file://$(find sensor_models)/meshes/orbbec/336L.glb"/>
+					</geometry>
+				</visual>
+			</xacro:unless>
 		</link>
-		<joint name="Camera-0" type="fixed">
+		<joint name="head_camera_joint" type="fixed">
 			<origin xyz="0.0475 -0.06195 0.0371" rpy="${-PI/2} 0 ${PI}"/>
-			<parent link="head23"/>
+			<parent link="head_link2"/>
 			<child link="head_camera"/>
 		</joint>

File: humanoid/SpiritAI/moz1_description/xacro/robot.xacro (robot description, xacro)
@@ -6,4 +6,6 @@
   <!-- false: ros2_control; OCS2 planning injects eef_fixed_joints:=true via robot_common_launch -->
   <xacro:arg name="eef_fixed_joints" default="false"/>
+  <!-- Isaac asset import: hide sensor_models meshes that Isaac already provides. -->
+  <xacro:arg name="isaac" default="false"/>
   <xacro:property name="eef_fixed" value="$(arg eef_fixed_joints)"/>
   <xacro:include filename="$(find moz1_description)/xacro/components/chassis.xacro"/>
@@ -15,4 +17,4 @@
   <xacro:Moz1Arm parent_link="waist03" direction="1" kinematic_only="${eef_fixed}"/>
   <xacro:Moz1Arm parent_link="waist03" direction="-1" kinematic_only="${eef_fixed}"/>
-  <xacro:Moz1Head parent_link="waist03"/>
+  <xacro:Moz1Head parent_link="waist03" isaac="$(arg isaac)"/>
 </robot>

File: humanoid/SpiritAI/moz1_description/xacro/ros2_control/head_interfaces.xacro (robot description, xacro)
@@ -2,5 +2,5 @@
 <robot xmlns:xacro="http://www.ros.org/wiki/xacro">
   <xacro:macro name="moz1_head_interfaces">
-    <joint name="Head-1">
+    <joint name="head_joint1">
       <command_interface name="position"/>
       <state_interface name="position">
@@ -10,5 +10,5 @@
       <state_interface name="effort"/>
     </joint>
-    <joint name="Head-2">
+    <joint name="head_joint2">
       <command_interface name="position"/>
       <state_interface name="position">
