Commit message: update

File: humanoid/Airbot/airbot_mmk2_description/urdf/airbot_mmk2.urdf (robot description, URDF)
Before this commit: robot mmk2, 32 links, 31 joints
Joints:
- joint lft_wheel_joint: limit (none) -> lower=-6.28 upper=6.28 effort=6.5 velocity=0.7; type continuous -> revolute
- joint rgt_wheel_joint: limit lower=-3.1416 upper=3.1416 effort=6.5 velocity=0.7 -> lower=-6.28 upper=6.28 effort=6.5 velocity=0.7
