Commit message: update agilex

File: manipulator/AgileX/cobot_magic_v1_description/xacro/component.xacro (robot description, xacro)
@@ -2,4 +2,6 @@
 <robot name="Cobot_Magic_V1" xmlns:xacro="http://www.ros.org/wiki/xacro">
 	<xacro:arg name="type" default="tracer"/>
+	<!-- Isaac asset import: hide sensor_models meshes that Isaac already provides. -->
+	<xacro:arg name="isaac" default="false"/>
 	<xacro:if value="${'$(arg type)' == 'tracer'}">
 		<xacro:include filename="$(find cobot_magic_v1_description)/xacro/components/tracer.xacro"/>
@@ -9,5 +11,5 @@
 		<link name="base_footprint"/>
 		<xacro:include filename="$(find cobot_magic_v1_description)/xacro/components/body.xacro"/>
-		<xacro:Body parent="base_footprint"/>
+		<xacro:Body parent="base_footprint" isaac="$(arg isaac)"/>
 	</xacro:if>
 </robot>

File: manipulator/AgileX/cobot_magic_v1_description/xacro/components/body.xacro (robot description, xacro)
@@ -2,5 +2,6 @@
 <robot xmlns:xacro="http://ros.org/wiki/xacro">
 	<xacro:property name="PI" value="3.1415926535897931"/>
-	<xacro:macro name="Body" params="parent:=base_footprint">
+	<xacro:macro name="Body" params="parent:=base_footprint isaac:=false">
+		<!-- isaac:=true hides sensor_models camera / lidar meshes (Isaac asset import). -->
 		<link name="body_link">
 			<inertial>
@@ -54,42 +55,21 @@
 			<axis/>
 		</joint>
-		<link name="camera_link1">
-			<inertial>
-				<origin xyz="-0.0292387906463559 0.000126439620513119 -0.000724950892729725"/>
-				<mass value="0.0877001598245188"/>
-				<inertia
-						ixx="7.77343248794949E-05"
-						ixy="2.44922634558373E-07"
-						ixz="1.73341747661077E-08"
-						iyy="9.73521513961785E-06"
-						iyz="-2.86133018917868E-09"
-						izz="7.74948757118157E-05"/>
-			</inertial>
+		<!-- 一台可调高度相机：只保留高位安装。
+		     stand 原点=三安装孔中心；pitch 原点=旋转孔。低位参考：0.189667 0 0.743143 -->
+		<link name="camera_stand2">
 			<visual>
 				<geometry>
-					<mesh filename="file://$(find cobot_magic_v1_description)/meshes/aloha_v1/camera_stand.glb"/>
+					<mesh filename="file://$(find cobot_magic_v1_description)/meshes/aloha_v1/camera_stand_fixed.glb"/>
 				</geometry>
 			</visual>
 		</link>
-		<joint name="camera_joint1" type="fixed">
-			<origin xyz="0.071198 0 0.10384" rpy="0 0.26931 0"/>
-			<parent link="camera_base_link"/>
-			<child link="camera_link1"/>
-		</joint>
-		<link name="camera1">
-			<visual>
-				<geometry>
-					<mesh filename="file://$(find sensor_models)/meshes/realsense/d435.glb"/>
-				</geometry>
-			</visual>
-		</link>
-		<joint name="camera1_fixed" type="fixed">
-			<origin xyz="0 0 0" rpy="${-PI/2} 0 ${-PI/2}"/>
-			<parent link="camera_link1"/>
-			<child link="camera1"/>
+		<joint name="camera_joint2" type="fixed">
+			<origin xyz="0.187901 0 1.263068"/>
+			<parent link="body_link"/>
+			<child link="camera_stand2"/>
 		</joint>
 		<link name="camera_link2">
 			<inertial>
-				<origin xyz="-0.0292307474530399 0.000126438461566014 -0.000753459207498031"/>
+				<origin xyz="0.0207658 0.00012644 -0.00075346"/>
 				<mass value="0.0877001605148491"/>
 				<inertia
@@ -103,22 +83,24 @@
 			<visual>
 				<geometry>
-					<mesh filename="file://$(find cobot_magic_v1_description)/meshes/aloha_v1/camera_stand.glb"/>
+					<mesh filename="file://$(find cobot_magic_v1_description)/meshes/aloha_v1/camera_stand_pitch.glb"/>
 				</geometry>
 			</visual>
 		</link>
-		<joint name="camera_joint2" type="fixed">
-			<origin xyz="-0.14 0 0.5" rpy="0 0.011358 0"/>
-			<parent link="camera_link1"/>
+		<joint name="camera_stand2_joint" type="fixed">
+			<origin xyz="0.013337 0 0" rpy="0 0.270534 0"/>
+			<parent link="camera_stand2"/>
 			<child link="camera_link2"/>
 		</joint>
 		<link name="camera2">
-			<visual>
-				<geometry>
-					<mesh filename="file://$(find sensor_models)/meshes/realsense/d435.glb"/>
-				</geometry>
-			</visual>
+			<xacro:unless value="${isaac}">
+				<visual>
+					<geometry>
+						<mesh filename="file://$(find sensor_models)/meshes/realsense/d435.glb"/>
+					</geometry>
+				</visual>
+			</xacro:unless>
 		</link>
 		<joint name="camera2_fixed" type="fixed">
-			<origin xyz="0 0 0" rpy="${-PI/2} 0 ${-PI/2}"/>
+			<origin xyz="0.0499965 0 0" rpy="${-PI/2} 0 ${-PI/2}"/>
 			<parent link="camera_link2"/>
 			<child link="camera2"/>
@@ -136,9 +118,11 @@
 						izz="1.7919E-05"/>
 			</inertial>
-			<visual>
-				<geometry>
-					<mesh filename="file://$(find sensor_models)/meshes/livox/mid360.glb"/>
-				</geometry>
-			</visual>
+			<xacro:unless value="${isaac}">
+				<visual>
+					<geometry>
+						<mesh filename="file://$(find sensor_models)/meshes/livox/mid360.glb"/>
+					</geometry>
+				</visual>
+			</xacro:unless>
 		</link>
 		<joint name="lidar_joint" type="fixed">

File: manipulator/AgileX/cobot_magic_v1_description/xacro/robot.xacro (robot description, xacro)
@@ -8,4 +8,6 @@
   <xacro:arg name="type" default="r5"/>
   <xacro:arg name="enable_wheel_joints" default="false"/>
+  <!-- Isaac asset import: hide sensor_models meshes that Isaac already provides. -->
+  <xacro:arg name="isaac" default="false"/>
   <xacro:property name="topology_arg" value="$(arg topology)"/>
   <xacro:property name="type_arg" value="$(arg type)"/>
@@ -52,5 +54,5 @@
     <xacro:include filename="$(find cobot_magic_v1_description)/xacro/components/body.xacro"/>
     <xacro:Tracer enable_wheel_joints="$(arg enable_wheel_joints)"/>
-    <xacro:Body parent="base_footprint"/>
+    <xacro:Body parent="base_footprint" isaac="$(arg isaac)"/>
     <link name="arm_base"/>
     <joint name="arm_base_joint" type="fixed">

File: manipulator/AgileX/split_aloha_description/xacro/components/body.xacro (robot description, xacro)
@@ -111,15 +111,31 @@
       <limit lower="0.0" upper="0.8" effort="1000" velocity="10.0"/>
     </joint>
-    <link name="top_camera_support">
+    <!-- 顶置相机支架：网格直接用 cobot_magic_v2 的 camera_stand / camera_stand2。
+         stand2 孔对齐原 top_camera_support（0.11048 0 0.29448）；
+         stand 原点 = 孔位 − (0.028 0 0)。lift_link.glb 内嵌的 camera stand 需自行删掉。 -->
+    <link name="camera_stand">
       <visual>
         <geometry>
-          <mesh filename="file://$(find split_aloha_description)/meshes/aloha_split/camera_support.glb"/>
+          <mesh filename="file://$(find cobot_magic_v2_description)/meshes/aloha_v2/camera_stand.glb"/>
         </geometry>
       </visual>
     </link>
-    <joint name="top_camera_support_joint" type="fixed">
-      <origin xyz="0.11048 0 0.29448"/>
+    <joint name="camera_stand_joint" type="fixed">
+      <origin xyz="0.08248 0 0.29448"/>
       <parent link="lifting_link"/>
-      <child link="top_camera_support"/>
+      <child link="camera_stand"/>
+    </joint>
+    <link name="camera_stand2">
+      <visual>
+        <origin rpy="${PI/2} 0 0"/>
+        <geometry>
+          <mesh filename="file://$(find cobot_magic_v2_description)/meshes/aloha_v2/camera_stand2.glb"/>
+        </geometry>
+      </visual>
+    </link>
+    <joint name="camera_stand2_joint" type="fixed">
+      <origin xyz="0.028 0 0"/>
+      <parent link="camera_stand"/>
+      <child link="camera_stand2"/>
     </joint>
     <link name="top_camera_link">
@@ -145,5 +161,5 @@
     <joint name="top_camera_joint" type="fixed">
       <origin xyz="0.05158 0 0.000526" rpy="${-PI/2} 0 ${-PI/2}"/>
-      <parent link="top_camera_support"/>
+      <parent link="camera_stand2"/>
       <child link="top_camera_link"/>
     </joint>
