Commit message: Use per-link GLB meshes for Taku visuals.
Replace the STL visuals with one GLB per link from the dense damping
mesh, keeping the photo_* base colors. head_yaw and head_pitch still
come from the body GLB because they are absent there.

File: humanoid/dyna/taku_description/urdf/taku.urdf (robot description, URDF)
Before this commit: robot taku_dvt1_inferred, 49 links, 48 joints
Links:
- link agv_base: geometry collision mesh filename=package://taku_description/meshes/agv_base.glb; visual mesh filename=package://taku_description/meshes/agv_base.glb
- link folding_to_waist_link: geometry collision mesh filename=package://taku_description/meshes/folding_to_waist_link.glb; visual mesh filename=package://taku_description/meshes/folding_to_waist_link.glb
- link head_pitch_link: geometry collision mesh filename=package://taku_description/meshes/head_pitch_link.glb; visual mesh filename=package://taku_description/meshes/head_pitch_link.glb
- link head_roll_link: geometry collision mesh filename=package://taku_description/meshes/head_roll_link.glb; visual mesh filename=package://taku_description/meshes/head_roll_link.glb
- link head_yaw_link: geometry collision mesh filename=package://taku_description/meshes/head_yaw_link.glb; visual mesh filename=package://taku_description/meshes/head_yaw_link.glb
- link left_elbow_link: geometry collision mesh filename=package://taku_description/meshes/left_elbow_link.glb; visual mesh filename=package://taku_description/meshes/left_elbow_link.glb
- link left_grippera_link: geometry collision mesh filename=package://taku_description/meshes/left_grippera_link.glb; visual mesh filename=package://taku_description/meshes/left_grippera_link.glb
- link left_gripperb_link: geometry collision mesh filename=package://taku_description/meshes/left_gripperb_link.glb; visual mesh filename=package://taku_description/meshes/left_gripperb_link.glb
- link left_shoulder_roll_link: geometry collision mesh filename=package://taku_description/meshes/left_shoulder_roll_link.g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; visual mesh filename=package://taku_description/meshes/left_shoulder_roll_link.g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
- link left_shoulder_yaw_link: geometry collision mesh filename=package://taku_description/meshes/left_shoulder_yaw_link.glb; visual mesh filename=package://taku_description/meshes/left_shoulder_yaw_link.glb
- link left_wheel_rotate: geometry collision mesh filename=package://taku_description/meshes/left_wheel_rotate.glb; visual mesh filename=package://taku_description/meshes/left_wheel_rotate.glb
- link left_wheel_rotate_2: geometry collision mesh filename=package://taku_description/meshes/left_wheel_rotate_2.glb; visual mesh filename=package://taku_description/meshes/left_wheel_rotate_2.glb
- link left_wheel_steering: geometry collision mesh filename=package://taku_description/meshes/left_wheel_steering.glb; visual mesh filename=package://taku_description/meshes/left_wheel_steering.glb
- link left_wheel_steering_2: geometry collision mesh filename=package://taku_description/meshes/left_wheel_steering_2.glb; visual mesh filename=package://taku_description/meshes/left_wheel_steering_2.glb
- link left_wrist_pitch_link: geometry collision mesh filename=package://taku_description/meshes/left_wrist_pitch_link.glb; visual mesh filename=package://taku_description/meshes/left_wrist_pitch_link.glb
- link left_wrist_roll_link: geometry collision mesh filename=package://taku_description/meshes/left_wrist_roll_link.glb; visual mesh filename=package://taku_description/meshes/left_wrist_roll_link.glb
- link left_wrist_yaw_link: geometry collision mesh filename=package://taku_description/meshes/left_wrist_yaw_link.glb; visual mesh filename=package://taku_description/meshes/left_wrist_yaw_link.glb
- link right_elbow_link: geometry collision mesh filename=package://taku_description/meshes/right_elbow_link.glb; visual mesh filename=package://taku_description/meshes/right_elbow_link.glb
- link right_grippera_link: geometry collision mesh filename=package://taku_description/meshes/right_grippera_link.glb; visual mesh filename=package://taku_description/meshes/right_grippera_link.glb
- link right_gripperb_link: geometry collision mesh filename=package://taku_description/meshes/right_gripperb_link.glb; visual mesh filename=package://taku_description/meshes/right_gripperb_link.glb
- link right_shoulder_yaw_link: geometry collision mesh filename=package://taku_description/meshes/right_shoulder_yaw_link.g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; visual mesh filename=package://taku_description/meshes/right_shoulder_yaw_link.g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
- link right_wheel_rotate: geometry collision mesh filename=package://taku_description/meshes/right_wheel_rotate.glb; visual mesh filename=package://taku_description/meshes/right_wheel_rotate.glb
- link right_wheel_rotate_2: geometry collision mesh filename=package://taku_description/meshes/right_wheel_rotate_2.glb; visual mesh filename=package://taku_description/meshes/right_wheel_rotate_2.glb
- link right_wheel_steering: geometry collision mesh filename=package://taku_description/meshes/right_wheel_steering.glb; visual mesh filename=package://taku_description/meshes/right_wheel_steering.glb
- link right_wheel_steering_2: geometry collision mesh filename=package://taku_description/meshes/right_wheel_steering_2.glb; visual mesh filename=package://taku_description/meshes/right_wheel_steering_2.glb
- link right_wrist_pitch_link: geometry collision mesh filename=package://taku_description/meshes/right_wrist_pitch_link.glb; visual mesh filename=package://taku_description/meshes/right_wrist_pitch_link.glb
- link right_wrist_roll_link: geometry collision mesh filename=package://taku_description/meshes/right_wrist_roll_link.glb; visual mesh filename=package://taku_description/meshes/right_wrist_roll_link.glb
- link right_wrist_yaw_link: geometry collision mesh filename=package://taku_description/meshes/right_wrist_yaw_link.glb; visual mesh filename=package://taku_description/meshes/right_wrist_yaw_link.glb
- link torso_body_link: geometry collision mesh filename=package://taku_description/meshes/torso_body_link.glb; visual mesh filename=package://taku_description/meshes/torso_body_link.glb
- link torso_waist_pitch_link: geometry collision mesh filename=package://taku_description/meshes/torso_waist_pitch_link.glb; visual mesh filename=package://taku_description/meshes/torso_waist_pitch_link.glb
