Commit message: taku: seat the rear MID-360 on the chassis skin
The kin frame stays where dvt1_kin.json puts it. The visual offset was
+29 mm, copied from the baked dome that has since been deleted. That left
the mesh origin 13 mm under a solid rear skin, so the 26 mm flange passed
through the body.

Other robots that use sensor_models livox/mid360.glb (Galaxea R1, MOZ1,
Astribot S1, Cobot Magic, Split Aloha) put the mesh origin on the joint,
about 10-12 mm below a deck that has a pocket for the flange. Rokae INEX
is the only one with a separate mount frame: the mesh origin is
z=-0.02085 from 3d_lidar_base, which also lands about 10 mm under its
deck. Taku has no such pocket, so the same gap buries the sensor.

Visual origin is now 0 0 0.0683: mesh bottom (z=-0.02615) on the rear
skin. The two Airy lidars are unchanged; their bottoms already sit on
their frames and those mounts are recessed.

File: humanoid/Dyna/taku_description/xacro/components/chassis.xacro (robot description, xacro)
@@ -95,7 +95,7 @@
                             steer_link="left_wheel_steering_2" rotate_link="left_wheel_rotate_2"
                             xyz="-0.2745 0.2045 0.2109" rotate_com="0.000114 0.003440 -0.000229" wheel_joints_enabled="${wheel_joints_enabled}"/>
-    <!-- Lidars. Frame poses are Dyna's published frames (dvt1_kin.json). The base GLB already contains the sensor
-         domes; sensor_models meshes are offset along the frame z axis so their domes coincide with the base mesh
-         (fitted: median surface error 0.4 mm). Dyna frames therefore sit at the sensor mounting face. -->
+    <!-- Lidars. Frame poses are Dyna's published frames (dvt1_kin.json). The baked domes were removed
+         from agv_base.glb; these visuals are the sensor_models meshes. Airy bottom sits on its frame
+         (mesh z min -0.042). MID-360 is seated on the rear skin, see the note on lidar_back. -->
     <!-- RoboSense Airy (front left) -->
     <link name="lidar_front_left">
@@ -130,9 +130,17 @@
       <child link="lidar_front_right"/>
     </joint>
-    <!-- Livox MID-360 (back) -->
+    <!-- Livox MID-360 (back).
+         sensor_models mesh origin is 26.15 mm above the flange (mesh z min -0.02615).
+         Galaxea R1 / MOZ1 / Astribot / Cobot Magic / Split Aloha put that origin on the
+         joint, ~10-12 mm under a deck that has a pocket, so the flange hangs in the pocket.
+         Rokae INEX is the only one with an explicit mount offset: mesh origin at
+         z=-0.02085 from 3d_lidar_base, which likewise lands ~10 mm under its deck.
+         Taku's kin frame is the mounting datum but the rear skin is solid and 42.2 mm
+         above it, so the previous +29 mm (origin 13 mm under the skin) drove the flange
+         through the shell. The offset below seats the flange on that skin. -->
     <link name="lidar_back">
       <xacro:unless value="${isaac}">
         <visual>
-          <origin xyz="0 0 0.029"/>
+          <origin xyz="0 0 0.0683"/>
           <geometry>
             <mesh filename="file://$(find sensor_models)/meshes/livox/mid360.glb"/>

Commit message: update lidar position

File: humanoid/Dyna/taku_description/xacro/components/chassis.xacro (robot description, xacro)
@@ -130,17 +130,7 @@
       <child link="lidar_front_right"/>
     </joint>
-    <!-- Livox MID-360 (back).
-         sensor_models mesh origin is 26.15 mm above the flange (mesh z min -0.02615).
-         Galaxea R1 / MOZ1 / Astribot / Cobot Magic / Split Aloha put that origin on the
-         joint, ~10-12 mm under a deck that has a pocket, so the flange hangs in the pocket.
-         Rokae INEX is the only one with an explicit mount offset: mesh origin at
-         z=-0.02085 from 3d_lidar_base, which likewise lands ~10 mm under its deck.
-         Taku's kin frame is the mounting datum but the rear skin is solid and 42.2 mm
-         above it, so the previous +29 mm (origin 13 mm under the skin) drove the flange
-         through the shell. The offset below seats the flange on that skin. -->
     <link name="lidar_back">
       <xacro:unless value="${isaac}">
         <visual>
-          <origin xyz="0 0 0.0683"/>
           <geometry>
             <mesh filename="file://$(find sensor_models)/meshes/livox/mid360.glb"/>
@@ -150,5 +140,5 @@
     </link>
     <joint name="lidar_back_frame" type="fixed">
-      <origin xyz="-0.3275 0.0 0.24995" rpy="0.0 0.0 1.5708"/>
+      <origin xyz="-0.3275 0.0 0.285" rpy="0.0 0.0 ${PI}"/>
       <parent link="agv_base"/>
       <child link="lidar_back"/>
