Commit message: taku: Dynaclaw + shared arm macro, W2-style ros2_control/OCS2
Split Dynaclaw like Astribot (meshes/dynaclaw/, components/dynaclaw.xacro,
standalone xacro/dynaclaw.xacro). Jaw meshes are shared (left≈right).

Refactor TakuArm like Ai2 Bot2 (name/direction/standalone). Arm meshes
are not Y-mirrors, so both sides stay under meshes/arm/. Full robot keeps
left_/right_ prefixes; left_arm/right_arm are unprefixed standalone.

Add left_tcp/right_tcp aliases for OCS2. Configure ros2_control after
FiveAges W2 (ocs2_arm_controller, ocs2_wbc_controller, chassis interfaces)
and config/ocs2/fixed_base_tcp.info. Omit head-follow / head-tracking;
head joints stay on head_joint_controller only.

File: humanoid/Dyna/taku_description/xacro/component.xacro (robot description, xacro)
@@ -5,9 +5,10 @@
   <xacro:arg name="isaac" default="false"/>
   <xacro:arg name="side" default="left"/>
+  <xacro:arg name="name" default=""/>
   <xacro:include filename="$(find taku_description)/xacro/components/chassis.xacro"/>
   <xacro:include filename="$(find taku_description)/xacro/components/body.xacro"/>
   <xacro:include filename="$(find taku_description)/xacro/components/head.xacro"/>
   <xacro:include filename="$(find taku_description)/xacro/components/arm.xacro"/>
-  <xacro:include filename="$(find taku_description)/xacro/components/gripper.xacro"/>
+  <xacro:include filename="$(find taku_description)/xacro/components/dynaclaw.xacro"/>
   <!-- Swerve chassis: 4 steering + 4 drive joints, lidars, IMU frame. -->
   <xacro:if value="${'$(arg type)' == 'chassis'}">
@@ -24,6 +25,6 @@
     <xacro:TakuBody parent_link="agv_base"/>
     <xacro:TakuHead parent_link="torso_body_link"/>
-    <xacro:TakuArm parent_link="torso_body_link" direction="1" enable_gripper="false"/>
-    <xacro:TakuArm parent_link="torso_body_link" direction="-1" enable_gripper="false"/>
+    <xacro:TakuArm name="left" parent_link="torso_body_link" direction="1" enable_gripper="false"/>
+    <xacro:TakuArm name="right" parent_link="torso_body_link" direction="-1" enable_gripper="false"/>
   </xacro:if>
   <xacro:if value="${'$(arg type)' == 'head'}">
@@ -31,21 +32,21 @@
     <xacro:TakuHead parent_link="torso_body_link"/>
   </xacro:if>
-  <xacro:if value="${'$(arg type)' == 'arm'}">
+  <!-- Both arms with Dynaclaw, mounted on a shared torso stub (prefixed left_/right_). -->
+  <xacro:if value="${'$(arg type)' == 'arm' or '$(arg type)' == 'arms'}">
     <link name="torso_body_link"/>
-    <xacro:TakuArm parent_link="torso_body_link" direction="1"/>
-    <xacro:TakuArm parent_link="torso_body_link" direction="-1"/>
+    <xacro:TakuArm name="left" parent_link="torso_body_link" direction="1"/>
+    <xacro:TakuArm name="right" parent_link="torso_body_link" direction="-1"/>
   </xacro:if>
+  <!-- Single arm, Ai2-style standalone (unprefixed); mesh side from direction. -->
   <xacro:if value="${'$(arg type)' == 'left_arm'}">
-    <link name="torso_body_link"/>
-    <xacro:TakuArm parent_link="torso_body_link" direction="1"/>
+    <xacro:TakuArm direction="1" standalone="true"/>
   </xacro:if>
   <xacro:if value="${'$(arg type)' == 'right_arm'}">
-    <link name="torso_body_link"/>
-    <xacro:TakuArm parent_link="torso_body_link" direction="-1"/>
+    <xacro:TakuArm direction="-1" standalone="true"/>
   </xacro:if>
-  <!-- Single gripper (one root link keeps the URDF valid); side:=left|right. -->
-  <xacro:if value="${'$(arg type)' == 'gripper'}">
-    <link name="$(arg side)_wrist_roll_link"/>
-    <xacro:TakuGripper side="$(arg side)"/>
+  <!-- Dynaclaw / gripper: one side per call so check_urdf has a single root. -->
+  <xacro:if value="${'$(arg type)' == 'gripper' or '$(arg type)' == 'dynaclaw'}">
+    <link name="wrist_roll_link"/>
+    <xacro:TakuDynaclaw name="$(arg side)" parent_link="wrist_roll_link"/>
   </xacro:if>
 </robot>

File: humanoid/Dyna/taku_description/xacro/components/arm.xacro (robot description, xacro)
@@ -3,25 +3,23 @@
   <xacro:property name="PI" value="3.141592653589793"/>
   <!-- INFERRED, NOT AN OFFICIAL DYNA SPEC. Kinematics from public dvt1_kin.json; limits from mesh self-collision sweep
-       snapped to integer degrees; inertias scaled from OpenArm v1 / Galaxea R1 / Agilex Ranger Mini. See doc/taku_params.md. -->
-  <xacro:include filename="$(find taku_description)/xacro/components/gripper.xacro"/>
-  <!-- direction:=1 left arm, direction:=-1 right arm (mirrored mount, asymmetric shoulder roll limits,
-       per-side mesh centroids). Inertias scaled from OpenArm v1. -->
-  <xacro:macro name="TakuArm" params="parent_link:=torso_body_link direction:=1 enable_gripper:=true">
-    <xacro:if value="${direction == 1}">
-      <xacro:property name="prefix" value="left"/>
-    </xacro:if>
-    <xacro:unless value="${direction == 1}">
-      <xacro:property name="prefix" value="right"/>
-    </xacro:unless>
+       snapped to integer degrees; inertias scaled from OpenArm v1 / Galaxea R1 / Agilex Ranger Mini. See doc/taku_params.md.
+       Ai2-bot2 style: one macro for both arms. name:="left"|"right"|"" sets the link/joint prefix;
+       direction:=1/-1 selects the side mesh under meshes/arm/ (left/right are NOT geometric mirrors —
+       shoulder_roll topology and wrist_pitch differ — so each side keeps its own GLB set).
+       standalone:=true omits the torso mount joint so the shoulder_pitch_link is the URDF root. -->
+  <xacro:include filename="$(find taku_description)/xacro/components/dynaclaw.xacro"/>
+  <xacro:macro name="TakuArm" params="name:='' parent_link:=torso_body_link direction:=1 enable_gripper:=true standalone:=false">
+    <xacro:property name="prefix" value="${name + '_' if name else ''}"/>
+    <xacro:property name="mesh_side" value="${'left' if direction == 1 else 'right'}"/>
     <!-- inertia: OpenArm v1 openarm_*_link1 / joint1，m=1.1417 kg，Lref=0.0671 m，Lt=0.085 m，k=1.267 -->
-    <link name="${prefix}_shoulder_pitch_link">
-      <visual>
-        <geometry>
-          <mesh filename="file://$(find taku_description)/meshes/${prefix}_shoulder_pitch_link.glb"/>
-        </geometry>
-      </visual>
-      <collision>
-        <geometry>
-          <mesh filename="file://$(find taku_description)/meshes/${prefix}_shoulder_pitch_link.glb"/>
+    <link name="${prefix}shoulder_pitch_link">
+      <visual>
+        <geometry>
+          <mesh filename="file://$(find taku_description)/meshes/arm/${mesh_side}_shoulder_pitch_link.glb"/>
+        </geometry>
+      </visual>
+      <collision>
+        <geometry>
+          <mesh filename="file://$(find taku_description)/meshes/arm/${mesh_side}_shoulder_pitch_link.glb"/>
         </geometry>
       </collision>
@@ -32,21 +30,34 @@
       </inertial>
     </link>
-    <joint name="${prefix}_shoulder_pitch_joint" type="revolute">
-      <origin xyz="${'0.0 0.105 0.243' if direction == 1 else '0.0 -0.105 0.243'}"/>
-      <parent link="${parent_link}"/>
-      <child link="${prefix}_shoulder_pitch_link"/>
-      <axis xyz="0.0 1.0 0.0"/>
-      <limit lower="${-150/180*PI}" upper="${90/180*PI}" effort="40" velocity="16.754666"/>
-    </joint>
+    <xacro:unless value="${standalone}">
+      <joint name="${prefix}shoulder_pitch_joint" type="revolute">
+        <origin xyz="${'0.0 0.105 0.243' if direction == 1 else '0.0 -0.105 0.243'}"/>
+        <parent link="${parent_link}"/>
+        <child link="${prefix}shoulder_pitch_link"/>
+        <axis xyz="0.0 1.0 0.0"/>
+        <limit lower="${-150/180*PI}" upper="${90/180*PI}" effort="40" velocity="16.754666"/>
+      </joint>
+    </xacro:unless>
+    <xacro:if value="${standalone}">
+      <!-- Keep the shoulder_pitch joint as a floating root actuator about a world stub. -->
+      <link name="${prefix}arm_mount"/>
+      <joint name="${prefix}shoulder_pitch_joint" type="revolute">
+        <origin xyz="0 0 0"/>
+        <parent link="${prefix}arm_mount"/>
+        <child link="${prefix}shoulder_pitch_link"/>
+        <axis xyz="0.0 1.0 0.0"/>
+        <limit lower="${-150/180*PI}" upper="${90/180*PI}" effort="40" velocity="16.754666"/>
+      </joint>
+    </xacro:if>
     <!-- inertia: OpenArm v1 openarm_*_link2 / joint2，m=0.2775 kg，Lref=0.0727 m，Lt=0.125 m，k=1.719 -->
-    <link name="${prefix}_shoulder_roll_link">
-      <visual>
-        <geometry>
-          <mesh filename="file://$(find taku_description)/meshes/${prefix}_shoulder_roll_link.glb"/>
-        </geometry>
-      </visual>
-      <collision>
-        <geometry>
-          <mesh filename="file://$(find taku_description)/meshes/${prefix}_shoulder_roll_link.glb"/>
+    <link name="${prefix}shoulder_roll_link">
+      <visual>
+        <geometry>
+          <mesh filename="file://$(find taku_description)/meshes/arm/${mesh_side}_shoulder_roll_link.glb"/>
+        </geometry>
+      </visual>
+      <collision>
+        <geometry>
+          <mesh filename="file://$(find taku_description)/meshes/arm/${mesh_side}_shoulder_roll_link.glb"/>
         </geometry>
       </collision>
@@ -57,21 +68,21 @@
       </inertial>
     </link>
-    <joint name="${prefix}_shoulder_roll_joint" type="revolute">
+    <joint name="${prefix}shoulder_roll_joint" type="revolute">
       <origin xyz="${'0.0 0.085 0.0' if direction == 1 else '0.0 -0.085 0.0'}"/>
-      <parent link="${prefix}_shoulder_pitch_link"/>
-      <child link="${prefix}_shoulder_roll_link"/>
+      <parent link="${prefix}shoulder_pitch_link"/>
+      <child link="${prefix}shoulder_roll_link"/>
       <axis xyz="1.0 0.0 0.0"/>
       <limit lower="${-15/180*PI if direction == 1 else -100/180*PI}" upper="${90/180*PI if direction == 1 else 15/180*PI}" effort="40" velocity="16.754666"/>
     </joint>
     <!-- inertia: OpenArm v1 openarm_*_link3 / joint3，m=1.0739 kg，Lref=0.1569 m，Lt=0.126 m，k=0.803 -->
-    <link name="${prefix}_shoulder_yaw_link">
-      <visual>
-        <geometry>
-          <mesh filename="file://$(find taku_description)/meshes/${prefix}_shoulder_yaw_link.glb"/>
-        </geometry>
-      </visual>
-      <collision>
-        <geometry>
-          <mesh filename="file://$(find taku_description)/meshes/${prefix}_shoulder_yaw_link.glb"/>
+    <link name="${prefix}shoulder_yaw_link">
+      <visual>
+        <geometry>
+          <mesh filename="file://$(find taku_description)/meshes/arm/${mesh_side}_shoulder_yaw_link.glb"/>
+        </geometry>
+      </visual>
+      <collision>
+        <geometry>
+          <mesh filename="file://$(find taku_description)/meshes/arm/${mesh_side}_shoulder_yaw_link.glb"/>
         </geometry>
       </collision>
@@ -82,21 +93,21 @@
       </inertial>
     </link>
-    <joint name="${prefix}_shoulder_yaw_joint" type="revolute">
+    <joint name="${prefix}shoulder_yaw_joint" type="revolute">
       <origin xyz="0.0 0.0 -0.125"/>
-      <parent link="${prefix}_shoulder_roll_link"/>
-      <child link="${prefix}_shoulder_yaw_link"/>
+      <parent link="${prefix}shoulder_roll_link"/>
+      <child link="${prefix}shoulder_yaw_link"/>
       <axis xyz="0.0 0.0 1.0"/>
       <limit lower="${-90/180*PI}" upper="${90/180*PI}" effort="27" velocity="5.445426"/>
     </joint>
     <!-- inertia: OpenArm v1 openarm_*_link4 / joint4，m=0.6349 kg，Lref=0.1006 m，Lt=0.103 m，k=1.024 -->
-    <link name="${prefix}_elbow_link">
-      <visual>
-        <geometry>
-          <mesh filename="file://$(find taku_description)/meshes/${prefix}_elbow_link.glb"/>
-        </geometry>
-      </visual>
-      <collision>
-        <geometry>
-          <mesh filename="file://$(find taku_description)/meshes/${prefix}_elbow_link.glb"/>
+    <link name="${prefix}elbow_link">
+      <visual>
+        <geometry>
+          <mesh filename="file://$(find taku_description)/meshes/arm/${mesh_side}_elbow_link.glb"/>
+        </geometry>
+      </visual>
+      <collision>
+        <geometry>
+          <mesh filename="file://$(find taku_description)/meshes/arm/${mesh_side}_elbow_link.glb"/>
         </geometry>
       </collision>
@@ -107,21 +118,21 @@
       </inertial>
     </link>
-    <joint name="${prefix}_elbow_joint" type="revolute">
+    <joint name="${prefix}elbow_joint" type="revolute">
       <origin xyz="0.015 0.0 -0.125"/>
-      <parent link="${prefix}_shoulder_yaw_link"/>
-      <child link="${prefix}_elbow_link"/>
+      <parent link="${prefix}shoulder_yaw_link"/>
+      <child link="${prefix}elbow_link"/>
       <axis xyz="0.0 1.0 0.0"/>
       <limit lower="${-135/180*PI}" upper="${20/180*PI}" effort="27" velocity="5.445426"/>
     </joint>
     <!-- inertia: OpenArm v1 openarm_*_link5 / joint5，m=0.6157 kg，Lref=0.1262 m，Lt=0.1525 m，k=1.208 -->
-    <link name="${prefix}_wrist_yaw_link">
-      <visual>
-        <geometry>
-          <mesh filename="file://$(find taku_description)/meshes/${prefix}_wrist_yaw_link.glb"/>
-        </geometry>
-      </visual>
-      <collision>
-        <geometry>
-          <mesh filename="file://$(find taku_description)/meshes/${prefix}_wrist_yaw_link.glb"/>
+    <link name="${prefix}wrist_yaw_link">
+      <visual>
+        <geometry>
+          <mesh filename="file://$(find taku_description)/meshes/arm/${mesh_side}_wrist_yaw_link.glb"/>
+        </geometry>
+      </visual>
+      <collision>
+        <geometry>
+          <mesh filename="file://$(find taku_description)/meshes/arm/${mesh_side}_wrist_yaw_link.glb"/>
         </geometry>
       </collision>
@@ -132,21 +143,21 @@
       </inertial>
     </link>
-    <joint name="${prefix}_wrist_yaw_joint" type="revolute">
+    <joint name="${prefix}wrist_yaw_joint" type="revolute">
       <origin xyz="-0.01 0.0 -0.1025"/>
-      <parent link="${prefix}_elbow_link"/>
-      <child link="${prefix}_wrist_yaw_link"/>
+      <parent link="${prefix}elbow_link"/>
+      <child link="${prefix}wrist_yaw_link"/>
       <axis xyz="0.0 0.0 1.0"/>
       <limit lower="${-90/180*PI}" upper="${90/180*PI}" effort="7" velocity="20.943946"/>
     </joint>
     <!-- inertia: OpenArm v1 openarm_*_link6 / joint6，m=0.4752 kg，Lref=0.0375 m，Lt=0.0285 m，k=0.760 -->
-    <link name="${prefix}_wrist_pitch_link">
-      <visual>
-        <geometry>
-          <mesh filename="file://$(find taku_description)/meshes/${prefix}_wrist_pitch_link.glb"/>
-        </geometry>
-      </visual>
-      <collision>
-        <geometry>
-          <mesh filename="file://$(find taku_description)/meshes/${prefix}_wrist_pitch_link.glb"/>
+    <link name="${prefix}wrist_pitch_link">
+      <visual>
+        <geometry>
+          <mesh filename="file://$(find taku_description)/meshes/arm/${mesh_side}_wrist_pitch_link.glb"/>
+        </geometry>
+      </visual>
+      <collision>
+        <geometry>
+          <mesh filename="file://$(find taku_description)/meshes/arm/${mesh_side}_wrist_pitch_link.glb"/>
         </geometry>
       </collision>
@@ -157,21 +168,21 @@
       </inertial>
     </link>
-    <joint name="${prefix}_wrist_pitch_joint" type="revolute">
+    <joint name="${prefix}wrist_pitch_joint" type="revolute">
       <origin xyz="0.0 0.0 -0.1525"/>
-      <parent link="${prefix}_wrist_yaw_link"/>
-      <child link="${prefix}_wrist_pitch_link"/>
+      <parent link="${prefix}wrist_yaw_link"/>
+      <child link="${prefix}wrist_pitch_link"/>
       <axis xyz="0.0 1.0 0.0"/>
       <limit lower="${-90/180*PI}" upper="${90/180*PI}" effort="7" velocity="20.943946"/>
     </joint>
     <!-- inertia: OpenArm v1 openarm_*_link7 / joint7，m=0.466 kg，Lref=0.1025 m，Lt=0.171 m，k=1.668 -->
-    <link name="${prefix}_wrist_roll_link">
-      <visual>
-        <geometry>
-          <mesh filename="file://$(find taku_description)/meshes/${prefix}_wrist_roll_link.glb"/>
-        </geometry>
-      </visual>
-      <collision>
-        <geometry>
-          <mesh filename="file://$(find taku_description)/meshes/${prefix}_wrist_roll_link.glb"/>
+    <link name="${prefix}wrist_roll_link">
+      <visual>
+        <geometry>
+          <mesh filename="file://$(find taku_description)/meshes/arm/${mesh_side}_wrist_roll_link.glb"/>
+        </geometry>
+      </visual>
+      <collision>
+        <geometry>
+          <mesh filename="file://$(find taku_description)/meshes/arm/${mesh_side}_wrist_roll_link.glb"/>
         </geometry>
       </collision>
@@ -182,26 +193,32 @@
       </inertial>
     </link>
-    <joint name="${prefix}_wrist_roll_joint" type="revolute">
+    <joint name="${prefix}wrist_roll_joint" type="revolute">
       <origin xyz="0.0285 0.0 0.0"/>
-      <parent link="${prefix}_wrist_pitch_link"/>
-      <child link="${prefix}_wrist_roll_link"/>
+      <parent link="${prefix}wrist_pitch_link"/>
+      <child link="${prefix}wrist_roll_link"/>
       <axis xyz="1.0 0.0 0.0"/>
       <limit lower="${-90/180*PI}" upper="${90/180*PI}" effort="7" velocity="20.943946"/>
     </joint>
-    <!-- FK target frame (from dvt1_kin.json) and wrist camera frame. -->
-    <link name="${prefix}_ee_fk_target_frame"/>
-    <joint name="${prefix}_gripper_joint_frame" type="fixed">
+    <!-- FK target / OCS2 TCP (same pose) and wrist camera frame. -->
+    <link name="${prefix}ee_fk_target_frame"/>
+    <joint name="${prefix}gripper_joint_frame" type="fixed">
       <origin xyz="-0.02852 0.0 -0.088527" rpy="0.0 0.0 -1.5708"/>
-      <parent link="${prefix}_wrist_roll_link"/>
-      <child link="${prefix}_ee_fk_target_frame"/>
-    </joint>
-    <link name="${prefix}_gripper_camera"/>
-    <joint name="${prefix}_gripper_camera_frame" type="fixed">
+      <parent link="${prefix}wrist_roll_link"/>
+      <child link="${prefix}ee_fk_target_frame"/>
+    </joint>
+    <link name="${prefix}tcp"/>
+    <joint name="${prefix}tcp_joint" type="fixed">
+      <origin xyz="0 0 0"/>
+      <parent link="${prefix}ee_fk_target_frame"/>
+      <child link="${prefix}tcp"/>
+    </joint>
+    <link name="${prefix}gripper_camera"/>
+    <joint name="${prefix}gripper_camera_frame" type="fixed">
       <origin xyz="0.056204 0.0 -0.150766" rpy="2.617994 0.0 -1.570796"/>
-      <parent link="${prefix}_wrist_roll_link"/>
-      <child link="${prefix}_gripper_camera"/>
+      <parent link="${prefix}wrist_roll_link"/>
+      <child link="${prefix}gripper_camera"/>
     </joint>
     <xacro:if value="${enable_gripper}">
-      <xacro:TakuGripper side="${prefix}"/>
+      <xacro:TakuDynaclaw name="${name}" parent_link="${prefix}wrist_roll_link"/>
     </xacro:if>
   </xacro:macro>

File: humanoid/Dyna/taku_description/xacro/components/gripper.xacro (robot description, xacro)
@@ -1,59 +1,5 @@
 <?xml version="1.0"?>
 <robot xmlns:xacro="http://www.ros.org/wiki/xacro">
-  <xacro:property name="PI" value="3.141592653589793"/>
-  <!-- INFERRED, NOT AN OFFICIAL DYNA SPEC. Kinematics from public dvt1_kin.json; limits from mesh self-collision sweep
-       snapped to integer degrees; inertias scaled from OpenArm v1 / Galaxea R1 / Agilex Ranger Mini. See doc/taku_params.md. -->
-  <!-- Parallel two-jaw gripper on ${side}_wrist_roll_link: front jaw (a) and rear jaw (b), each prismatic along y. -->
-  <xacro:macro name="TakuGripper" params="side:=left">
-    <link name="${side}_grippera_link">
-      <visual>
-        <geometry>
-          <mesh filename="file://$(find taku_description)/meshes/${side}_grippera_link.glb"/>
-        </geometry>
-      </visual>
-      <collision>
-        <geometry>
-          <mesh filename="file://$(find taku_description)/meshes/${side}_grippera_link.glb"/>
-        </geometry>
-      </collision>
-    </link>
-    <joint name="${side}_gripper_front_joint" type="prismatic">
-      <origin xyz="-0.028953 -0.023048 -0.166971"/>
-      <parent link="${side}_wrist_roll_link"/>
-      <child link="${side}_grippera_link"/>
-      <axis xyz="0.0 1.0 0.0"/>
-      <limit lower="-0.0345" upper="0.0" effort="100" velocity="0.25"/>
-    </joint>
-    <link name="${side}_gripper_tip_A"/>
-    <joint name="${side}_gripper_tip_A_frame" type="fixed">
-      <origin xyz="0.000433 0.023068 -0.080556"/>
-      <parent link="${side}_grippera_link"/>
-      <child link="${side}_gripper_tip_A"/>
-    </joint>
-    <link name="${side}_gripperb_link">
-      <visual>
-        <geometry>
-          <mesh filename="file://$(find taku_description)/meshes/${side}_gripperb_link.glb"/>
-        </geometry>
-      </visual>
-      <collision>
-        <geometry>
-          <mesh filename="file://$(find taku_description)/meshes/${side}_gripperb_link.glb"/>
-        </geometry>
-      </collision>
-    </link>
-    <joint name="${side}_gripper_rear_joint" type="prismatic">
-      <origin xyz="-0.028088 0.023048 -0.166971"/>
-      <parent link="${side}_wrist_roll_link"/>
-      <child link="${side}_gripperb_link"/>
-      <axis xyz="0.0 1.0 0.0"/>
-      <limit lower="0.0" upper="0.0345" effort="100" velocity="0.25"/>
-    </joint>
-    <link name="${side}_gripper_tip_B"/>
-    <joint name="${side}_gripper_tip_B_frame" type="fixed">
-      <origin xyz="-0.000432 -0.023068 -0.080556"/>
-      <parent link="${side}_gripperb_link"/>
-      <child link="${side}_gripper_tip_B"/>
-    </joint>
-  </xacro:macro>
+  <!-- Dynaclaw lives in dynaclaw.xacro; this file remains as a thin include for older paths. -->
+  <xacro:include filename="$(find taku_description)/xacro/components/dynaclaw.xacro"/>
 </robot>

File: humanoid/Dyna/taku_description/xacro/robot.xacro (robot description, xacro)
@@ -13,5 +13,5 @@
   <xacro:TakuBody parent_link="agv_base"/>
   <xacro:TakuHead parent_link="torso_body_link"/>
-  <xacro:TakuArm parent_link="torso_body_link" direction="1"/>
-  <xacro:TakuArm parent_link="torso_body_link" direction="-1"/>
+  <xacro:TakuArm name="left" parent_link="torso_body_link" direction="1"/>
+  <xacro:TakuArm name="right" parent_link="torso_body_link" direction="-1"/>
 </robot>

File: humanoid/Dyna/taku_description/xacro/ros2_control/interfaces.xacro (robot description, xacro)
@@ -34,8 +34,22 @@
     <xacro:taku_joint_iface name="${arm_side}_wrist_roll_joint"/>
   </xacro:macro>
-  <!-- Two independent prismatic jaws per gripper (front: [-0.0345, 0], rear: [0, 0.0345]). -->
+  <!-- Dynaclaw: two independent prismatic jaws (front: [-0.0345, 0], rear: [0, 0.0345]). -->
   <xacro:macro name="taku_gripper_interfaces" params="side:=left">
     <xacro:taku_joint_iface name="${side}_gripper_front_joint"/>
     <xacro:taku_joint_iface name="${side}_gripper_rear_joint"/>
   </xacro:macro>
+  <xacro:macro name="taku_dynaclaw_interfaces" params="side:=left">
+    <xacro:taku_gripper_interfaces side="${side}"/>
+  </xacro:macro>
+  <!-- Swerve chassis (only when enable_wheel_joints:=true so joints are not fixed). -->
+  <xacro:macro name="taku_chassis_interfaces">
+    <xacro:taku_joint_iface name="agv_right_front_steering_joint"/>
+    <xacro:taku_joint_iface name="agv_right_back_steering_joint"/>
+    <xacro:taku_joint_iface name="agv_left_front_steering_joint"/>
+    <xacro:taku_joint_iface name="agv_left_back_steering_joint"/>
+    <xacro:taku_joint_iface name="agv_right_front_rotate_joint"/>
+    <xacro:taku_joint_iface name="agv_right_back_rotate_joint"/>
+    <xacro:taku_joint_iface name="agv_left_front_rotate_joint"/>
+    <xacro:taku_joint_iface name="agv_left_back_rotate_joint"/>
+  </xacro:macro>
 </robot>
