Commit message: taku: Dynaclaw + shared arm macro, W2-style ros2_control/OCS2
Split Dynaclaw like Astribot (meshes/dynaclaw/, components/dynaclaw.xacro,
standalone xacro/dynaclaw.xacro). Jaw meshes are shared (left≈right).

Refactor TakuArm like Ai2 Bot2 (name/direction/standalone). Arm meshes
are not Y-mirrors, so both sides stay under meshes/arm/. Full robot keeps
left_/right_ prefixes; left_arm/right_arm are unprefixed standalone.

Add left_tcp/right_tcp aliases for OCS2. Configure ros2_control after
FiveAges W2 (ocs2_arm_controller, ocs2_wbc_controller, chassis interfaces)
and config/ocs2/fixed_base_tcp.info. Omit head-follow / head-tracking;
head joints stay on head_joint_controller only.

File: humanoid/Dyna/taku_description/xacro/ros2_control/robot.xacro (robot description, xacro)
@@ -22,10 +22,13 @@
       </xacro:if>
     </hardware>
+    <xacro:if value="$(arg enable_wheel_joints)">
+      <xacro:taku_chassis_interfaces/>
+    </xacro:if>
     <xacro:taku_body_interfaces/>
     <xacro:taku_head_interfaces/>
     <xacro:taku_arm_interfaces direction="1"/>
     <xacro:taku_arm_interfaces direction="-1"/>
-    <xacro:taku_gripper_interfaces side="left"/>
-    <xacro:taku_gripper_interfaces side="right"/>
+    <xacro:taku_dynaclaw_interfaces side="left"/>
+    <xacro:taku_dynaclaw_interfaces side="right"/>
   </ros2_control>
   <xacro:if value="$(arg gazebo)">

Commit message: taku: rename agv_base to base_link, add base_footprint
Align Taku chassis root frames with other robots (Ai2 Bot2 pattern):
base_footprint --fixed identity--> base_link. Keep meshes/agv_base.glb;
update OCS2 baseFrame / marker frames and docs.

File: humanoid/Dyna/taku_description/xacro/component.xacro (robot description, xacro)
@@ -17,11 +17,21 @@
   <!-- Folding lift + waist. -->
   <xacro:if value="${'$(arg type)' == 'body'}">
-    <link name="agv_base"/>
-    <xacro:TakuBody parent_link="agv_base"/>
+    <link name="base_footprint"/>
+    <joint name="base_footprint_joint" type="fixed">
+      <parent link="base_footprint"/>
+      <child link="base_link"/>
+    </joint>
+    <link name="base_link"/>
+    <xacro:TakuBody parent_link="base_link"/>
   </xacro:if>
   <!-- Upper body: folding lift + waist + head + dual arms (no chassis/gripper). -->
   <xacro:if value="${'$(arg type)' == 'upper_body'}">
-    <link name="agv_base"/>
-    <xacro:TakuBody parent_link="agv_base"/>
+    <link name="base_footprint"/>
+    <joint name="base_footprint_joint" type="fixed">
+      <parent link="base_footprint"/>
+      <child link="base_link"/>
+    </joint>
+    <link name="base_link"/>
+    <xacro:TakuBody parent_link="base_link"/>
     <xacro:TakuHead parent_link="torso_body_link"/>
     <xacro:TakuArm name="left" parent_link="torso_body_link" direction="1" enable_gripper="false"/>

File: humanoid/Dyna/taku_description/xacro/components/body.xacro (robot description, xacro)
@@ -5,5 +5,5 @@
        snapped to integer degrees; inertias scaled from OpenArm v1 / Galaxea R1 / Agilex Ranger Mini. See doc/taku_params.md. -->
   <!-- Folding lift (folding_low / folding_high) + waist pitch / yaw. -->
-  <xacro:macro name="TakuBody" params="parent_link:=agv_base">
+  <xacro:macro name="TakuBody" params="parent_link:=base_link">
     <!-- inertia: Galaxea R1 torso_link1 5.72 kg、关节间距 0.40 m；Taku folding_low→high 间距 0.450 m，k=1.125 -->
     <link name="folding_lower_joint_link">

File: humanoid/Dyna/taku_description/xacro/components/chassis.xacro (robot description, xacro)
@@ -46,5 +46,5 @@
     <joint name="${steer_joint}" type="${steering_joint_type}">
       <origin xyz="${xyz}"/>
-      <parent link="agv_base"/>
+      <parent link="base_link"/>
       <child link="${steer_link}"/>
       <xacro:if value="${wheel_joints_enabled}">
@@ -65,6 +65,12 @@
   <xacro:macro name="TakuChassis" params="enable_wheel_joints:='true' isaac:=false">
     <xacro:property name="wheel_joints_enabled" value="${str(enable_wheel_joints).lower() in ['true', '1', 'yes', 'on']}"/>
+    <!-- Root frames: base_footprint --fixed identity--> base_link (Ai2 Bot2 chassis pattern). -->
+    <link name="base_footprint"/>
+    <joint name="base_footprint_joint" type="fixed">
+      <parent link="base_footprint"/>
+      <child link="base_link"/>
+    </joint>
     <!-- inertia: Agilex Ranger Mini base_link 10 kg，轮距线性比 1.108（Taku 0.549×0.409 m / Ranger 0.494×0.370 m），质量×k^3 -->
-    <link name="agv_base">
+    <link name="base_link">
       <visual>
         <geometry>
@@ -111,5 +117,5 @@
     <joint name="lidar_front_left_frame" type="fixed">
       <origin xyz="0.292236 0.227959 0.301378" rpy="-0.616837 -0.603562 -1.94305"/>
-      <parent link="agv_base"/>
+      <parent link="base_link"/>
       <child link="lidar_front_left"/>
     </joint>
@@ -127,5 +133,5 @@
     <joint name="lidar_front_right_frame" type="fixed">
       <origin xyz="0.292236 -0.227959 0.301378" rpy="0.613474 -0.606997 1.94896"/>
-      <parent link="agv_base"/>
+      <parent link="base_link"/>
       <child link="lidar_front_right"/>
     </joint>
@@ -141,5 +147,5 @@
     <joint name="lidar_back_frame" type="fixed">
       <origin xyz="-0.3275 0.0 0.285" rpy="0.0 0.0 ${PI}"/>
-      <parent link="agv_base"/>
+      <parent link="base_link"/>
       <child link="lidar_back"/>
     </joint>
@@ -147,5 +153,5 @@
     <joint name="agv_imu_frame_frame" type="fixed">
       <origin xyz="-0.1642 0.225 0.178" rpy="0.0 0.0 3.14159"/>
-      <parent link="agv_base"/>
+      <parent link="base_link"/>
       <child link="agv_imu_frame"/>
     </joint>

File: humanoid/Dyna/taku_description/xacro/robot.xacro (robot description, xacro)
@@ -11,5 +11,5 @@
   <xacro:include filename="$(find taku_description)/xacro/components/arm.xacro"/>
   <xacro:TakuChassis enable_wheel_joints="$(arg enable_wheel_joints)" isaac="$(arg isaac)"/>
-  <xacro:TakuBody parent_link="agv_base"/>
+  <xacro:TakuBody parent_link="base_link"/>
   <xacro:TakuHead parent_link="torso_body_link"/>
   <xacro:TakuArm name="left" parent_link="torso_body_link" direction="1"/>
