Commit message: dexforce_w1: drop static urdf/, add full-body WBC + align control config with Quanta/Zerith/Taku
Cleanup
- Remove static vendor urdf/ (xacro is the source; planning URDF is generated from
  xacro) and the stray config/ocs2/demo_ocs2.rviz duplicate; install rules now
  `xacro meshes config`; fix stale package.xml description (was "EngineAI pm01").
- README rewritten (build / visualize / full body / split body / chassis / layout).

xacro
- Add topology:=dual (arms-only planning tree rooted at `waist`), eef_fixed_joints,
  chassis_joints_movable (default false, WHEEL_LEFT/RIGHT fixed like W2/Bot2/Quanta/Zerith).
- type:=revo1 now also defines left_eef/right_eef (OCS2 eeFrame was missing) and passes
  eef_fixed_joints to BrainCoHand so planning URDF has no finger DOF.

Control
- ros2_control: common.yaml (shared) + ros2_controllers.yaml / pro.yaml as home-pose
  overlays (W2 layout); controllers: ocs2_wbc_controller (fixed_base_tcp), ocs2_arm_controller
  (arms only, task.info), body/head joint controllers, grippers/hands.
- config/ocs2/fixed_base_tcp.info (new): Pinocchio 4 DFS [body x4 | head x2 | L7 | R7],
  headInputStart 4, structured modeSequence HM_DUAL_CUSTOM_LOCK_FIXED_BASE + HEAD_DISABLE,
  manipulatorModelType 0, bodyFrame waist, headFrame neck2.
- task.info rewritten for 14 arm DOF (baseFrame waist, no stale rr_steer/body_link4 refs).
- target_manager.yaml (reference_link, enable_wbc_head_tracking_marker false) and
  config/rviz/fullbody.rviz (world) / splitbody.rviz (base_link) from Taku/Quanta.

File: humanoid/DexForce/dexfoce_w1_description/xacro/components/chassis.xacro (robot description, xacro)
@@ -2,8 +2,10 @@
 <!--
   Chassis definition for DexForce W1 robot
-  Contains base_link, wheels, and wheel joints
+  Contains base_link, wheels, and wheel joints (fixed unless joints_movable:=true)
 -->
 <robot xmlns:xacro="http://www.ros.org/wiki/xacro">
-	<xacro:macro name="dexforce_w1_chassis">
+	<xacro:macro name="dexforce_w1_chassis" params="joints_movable:=false">
+		<xacro:property name="chassis_movable" value="${str(joints_movable).lower() in ['true', '1', 'yes', 'on']}"/>
+		<xacro:property name="wheel_joint_type" value="${'continuous' if chassis_movable else 'fixed'}"/>
 		<link name="base_link">
 			<inertial>
@@ -39,5 +41,5 @@
 			</inertial>
 		</link>
-		<joint name="WHEEL_LEFT" type="fixed">
+		<joint name="WHEEL_LEFT" type="${wheel_joint_type}">
 			<origin xyz="0 0.2539 0.053"/>
 			<parent link="base_link"/>
@@ -45,5 +47,5 @@
 			<axis xyz="0 1 0"/>
 		</joint>
-		<joint name="WHEEL_RIGHT" type="fixed">
+		<joint name="WHEEL_RIGHT" type="${wheel_joint_type}">
 			<origin xyz="0 -0.2539 0.053"/>
 			<parent link="base_link"/>

File: humanoid/DexForce/dexfoce_w1_description/xacro/eefs.xacro (robot description, xacro)
@@ -1,5 +1,5 @@
 <?xml version="1.0"?>
 <robot xmlns:xacro="http://www.ros.org/wiki/xacro">
-	<xacro:macro name="EndEffectors" params="hand_type:='' gripper_type:=''">
+	<xacro:macro name="EndEffectors" params="hand_type:='' gripper_type:='' eef_fixed:=false">
 		<!-- Note:
 		     - gripper_type 不为空时表示使用夹爪（保持原有逻辑）
@@ -36,6 +36,17 @@
 		<!-- 灵巧手类型 -->
 		<xacro:if value="${hand_type == 'revo1'}">
+			<!-- OCS2 eeFrame (left_eef/right_eef) must exist for every type; tied to the TCP -->
+			<link name="left_eef"/>
+			<link name="right_eef"/>
+			<joint name="left_eef_joint" type="fixed">
+				<parent link="left_tcp"/>
+				<child link="left_eef"/>
+			</joint>
+			<joint name="right_eef_joint" type="fixed">
+				<parent link="right_tcp"/>
+				<child link="right_eef"/>
+			</joint>
 			<xacro:include filename="$(find brainco_description)/xacro/revo1.xacro"/>
-			<xacro:BrainCoHand name="left_hand" direction="1" fixed_joints="false"/>
+			<xacro:BrainCoHand name="left_hand" direction="1" fixed_joints="${eef_fixed}"/>
 			<joint name="left_hand_base_joint" type="fixed">
 				<origin rpy="${PI/2} 0 ${PI}"/>
@@ -43,5 +54,5 @@
 				<child link="left_hand_hand_base"/>
 			</joint>
-			<xacro:BrainCoHand name="right_hand" direction="-1" fixed_joints="false"/>
+			<xacro:BrainCoHand name="right_hand" direction="-1" fixed_joints="${eef_fixed}"/>
 			<joint name="right_hand_base_joint" type="fixed">
 				<parent link="right_tcp"/>

File: humanoid/DexForce/dexfoce_w1_description/xacro/robot.xacro (robot description, xacro)
@@ -13,4 +13,11 @@
 	-->
 	<xacro:arg name="type" default="ANTHROPOMORPHIC"/>
+	<!-- topology: full (default) | dual = OCS2 split-body planning tree rooted at `waist`
+	     (arms only; set by robot_common_launch for planning_scope=arms) -->
+	<xacro:arg name="topology" default="full"/>
+	<!-- OCS2 planning: robot_common_launch injects eef_fixed_joints:=true and chassis_joints_movable:=false -->
+	<xacro:arg name="eef_fixed_joints" default="false"/>
+	<!-- Drive wheels fixed by default (W2/Bot2/Quanta/Zerith). Planning URDF keeps this false. -->
+	<xacro:arg name="chassis_joints_movable" default="false"/>
 	<xacro:property name="type_arg" value="$(arg type)"/>
 	<!-- 默认值 -->
@@ -32,7 +39,12 @@
 	<xacro:include filename="$(find dexforce_w1_description)/xacro/components/body.xacro"/>
 	<xacro:include filename="$(find dexforce_w1_description)/xacro/components/arm.xacro"/>
-	<!-- Generate chassis and body (common for both configurations) -->
-	<xacro:dexforce_w1_chassis/>
-	<xacro:dexforce_w1_body/>
+	<!-- Generate chassis and body (common for both configurations); dual topology keeps only `waist` -->
+	<xacro:if value="${'$(arg topology)' == 'dual'}">
+		<link name="waist"/>
+	</xacro:if>
+	<xacro:unless value="${'$(arg topology)' == 'dual'}">
+		<xacro:dexforce_w1_chassis joints_movable="$(arg chassis_joints_movable)"/>
+		<xacro:dexforce_w1_body/>
+	</xacro:unless>
 	<!-- Generate arms based on configuration type -->
 	<xacro:dexforce_w1_arm name="left" direction="1" arm_type="${selected_arm_type}"/>
@@ -40,4 +52,5 @@
 	<!-- Include and generate end effector frames -->
 	<xacro:include filename="$(find dexforce_w1_description)/xacro/eefs.xacro"/>
-	<xacro:EndEffectors hand_type="${selected_hand_type}" gripper_type="${selected_gripper_type}"/>
+	<xacro:EndEffectors hand_type="${selected_hand_type}" gripper_type="${selected_gripper_type}"
+	                    eef_fixed="$(arg eef_fixed_joints)"/>
 </robot>

File: humanoid/DexForce/dexfoce_w1_description/xacro/ros2_control/robot.xacro (robot description, xacro)
@@ -2,4 +2,6 @@
 <robot name="dexforce_w1" xmlns:xacro="http://www.ros.org/wiki/xacro">
 	<xacro:arg name="ros2_control_hardware_type" default="mock_components"/>
+	<!-- Drive wheels are fixed and not part of ros2_control (W2/Bot2/Quanta/Zerith convention) -->
+	<xacro:arg name="chassis_joints_movable" default="false"/>
 	<xacro:include filename="$(find dexforce_w1_description)/xacro/robot.xacro"/>
 	<xacro:include filename="$(find dexforce_w1_description)/xacro/ros2_control/arm.xacro"/>
