Commit message: dexforce_w1: head follow (HEAD_GAZE + headMidpointGaze on new head_camera at eyes on neck2, head cost 0.1) and homeJointReference in full-body WBC

File: humanoid/DexForce/dexfoce_w1_description/xacro/components/body.xacro (robot description, xacro)
@@ -172,4 +172,12 @@
 			<child link="eyes"/>
 		</joint>
+		<!-- head_camera: ROS optical frame (+Z forward, +X right, +Y down) at the `eyes` position on neck2.
+		     Used by OCS2 headMidpointGaze (HEAD_GAZE). `eyes` keeps the vendor orientation. -->
+		<link name="head_camera"/>
+		<joint name="head_camera_joint" type="fixed">
+			<origin xyz="0.085 -0.051 0.0" rpy="3.1416 -1.5708 0"/>
+			<parent link="neck2"/>
+			<child link="head_camera"/>
+		</joint>
 	</xacro:macro>
 </robot>
