Commit message: airbot_mmk2: drop static urdf/, align control config with Quanta/Zerith/Taku (task.info arms-only, fixed_base_tcp WBC slide|head|L|R, mobile_demo.info keeps manipulator demo), wheels fixed by default (chassis_joints_movable), head follow (HEAD_GAZE + head_camera), homeJointReference, target_manager + RViz

File: humanoid/Airbot/airbot_mmk2_description/xacro/mmk2_base.xacro (robot description, xacro)
@@ -1,4 +1,5 @@
 <?xml version="1.0" encoding="utf-8"?>
-<robot name="mmk2">
+<robot name="mmk2" xmlns:xacro="http://www.ros.org/wiki/xacro">
+  <!-- Drive wheels are `fixed` unless chassis_joints_movable:=true (set in robot.xacro) -->
   <link name="base_link">
     <inertial>
@@ -36,5 +37,5 @@
     </collision>
   </link>
-  <joint name="lft_wheel_joint" type="continuous">
+  <joint name="lft_wheel_joint" type="${wheel_joint_type}">
     <origin xyz="0 0.16325 0.08401" rpy="1.5708 1.5708 0"/>
     <parent link="base_link"/>
@@ -59,5 +60,5 @@
     </collision>
   </link>
-  <joint name="rgt_wheel_joint" type="continuous">
+  <joint name="rgt_wheel_joint" type="${wheel_joint_type}">
     <origin xyz="0 -0.16325 0.08401" rpy="1.5708 1.5708 0"/>
     <parent link="base_link"/>
@@ -177,4 +178,12 @@
     <axis xyz="0 0 1"/>
     <limit lower="-0.04" upper="0.87" effort="500" velocity="0.3"/>
+  </joint>
+  <!-- ROS-aligned (X forward, Y left, Z up) torso frame for OCS2 bodyFrame: slide_link is flipped
+       (rpy π 0 π/2); this fixed rpy is its own inverse, so the frame coincides with base_link axes. -->
+  <link name="torso_tracking_frame"/>
+  <joint name="torso_tracking_joint" type="fixed">
+    <origin xyz="0 0 0" rpy="3.1416 0 1.5708"/>
+    <parent link="slide_link"/>
+    <child link="torso_tracking_frame"/>
   </joint>
   <link name="head_yaw_link">
@@ -228,3 +237,11 @@
     <limit lower="-0.16" upper="1.18" effort="2" velocity="0.2"/>
   </joint>
+  <!-- head_camera: ROS optical frame (+Z forward, +X right, +Y down) on head_pitch_link, in front of
+       the head mesh (nominal; vendor MJCF head cam). Used by OCS2 headMidpointGaze (HEAD_GAZE). -->
+  <link name="head_camera"/>
+  <joint name="head_camera_joint" type="fixed">
+    <origin xyz="0.085 -0.108 0.0" rpy="0 1.5708 0"/>
+    <parent link="head_pitch_link"/>
+    <child link="head_camera"/>
+  </joint>
 </robot>

File: humanoid/Airbot/airbot_mmk2_description/xacro/robot.xacro (robot description, xacro)
@@ -1,4 +1,9 @@
 <?xml version="1.0" encoding="utf-8"?>
 <robot name="mmk2" xmlns:xacro="http://www.ros.org/wiki/xacro">
+  <!-- Drive wheels fixed by default (W2/Bot2/Quanta/Zerith). Planning URDF keeps this false.
+       Set true for diff_drive navigation (wheel velocity interfaces + diff_drive_controller). -->
+  <xacro:arg name="chassis_joints_movable" default="false"/>
+  <xacro:property name="wheel_joint_type"
+                  value="${'continuous' if '$(arg chassis_joints_movable)'.lower() in ['true', '1', 'yes', 'on'] else 'fixed'}"/>
   <xacro:include filename="$(find airbot_mmk2_description)/xacro/mmk2_base.xacro"/>
   <!-- left arm -->

File: humanoid/Airbot/airbot_mmk2_description/xacro/ros2_control/robot.xacro (robot description, xacro)
@@ -1,4 +1,8 @@
 <?xml version="1.0" encoding="utf-8"?>
 <robot name="mmk2" xmlns:xacro="http://www.ros.org/wiki/xacro">
+  <xacro:arg name="ros2_control_hardware_type" default="mock_components"/>
+  <xacro:arg name="gazebo" default="false"/>
+  <!-- Wheels are fixed (not in ros2_control) unless chassis_joints_movable:=true (diff_drive navigation) -->
+  <xacro:arg name="chassis_joints_movable" default="false"/>
   <!-- Include mmk2 base -->
   <xacro:include filename="$(find airbot_mmk2_description)/xacro/robot.xacro"/>
@@ -17,24 +21,29 @@
         <param name="joint_commands_topic">/isaac/joint_command</param>
         <param name="joint_states_topic">/isaac/joint_states</param>
+        <param name="sum_wrapped_joint_states">false</param>
+        <param name="initialize_commands_from_state">true</param>
       </xacro:if>
     </hardware>
-    <joint name="lft_wheel_joint">
-      <command_interface name="velocity">
-        <param name="min">-1.0</param>
-        <param name="max">1.0</param>
-      </command_interface>
-      <state_interface name="position"/>
-      <state_interface name="velocity"/>
-      <state_interface name="effort"/>
-    </joint>
-    <joint name="rgt_wheel_joint">
-      <command_interface name="velocity">
-        <param name="min">-1.0</param>
-        <param name="max">1.0</param>
-      </command_interface>
-      <state_interface name="position"/>
-      <state_interface name="velocity"/>
-      <state_interface name="effort"/>
-    </joint>
+    <!-- Drive wheels: only when movable (diff_drive_controller); fixed joints cannot be HI joints -->
+    <xacro:if value="${wheel_joint_type == 'continuous'}">
+      <joint name="lft_wheel_joint">
+        <command_interface name="velocity">
+          <param name="min">-1.0</param>
+          <param name="max">1.0</param>
+        </command_interface>
+        <state_interface name="position"/>
+        <state_interface name="velocity"/>
+        <state_interface name="effort"/>
+      </joint>
+      <joint name="rgt_wheel_joint">
+        <command_interface name="velocity">
+          <param name="min">-1.0</param>
+          <param name="max">1.0</param>
+        </command_interface>
+        <state_interface name="position"/>
+        <state_interface name="velocity"/>
+        <state_interface name="effort"/>
+      </joint>
+    </xacro:if>
     <joint name="slide_joint">
       <command_interface name="position"/>

Commit message: airbot_mmk2: disable body TRACKING (lift-only); lock slide via customJointLock
Single prismatic slide has no useful 6D torso follow. Turn off bodyTrackingEE,
lock slide_joint (index 0), exclude it from homeJointReference, point bodyFrame
at slide_link, and drop the torso_tracking_frame dummy. Keep HEAD_GAZE and arms.

File: humanoid/Airbot/airbot_mmk2_description/xacro/mmk2_base.xacro (robot description, xacro)
@@ -178,12 +178,4 @@
     <axis xyz="0 0 1"/>
     <limit lower="-0.04" upper="0.87" effort="500" velocity="0.3"/>
-  </joint>
-  <!-- ROS-aligned (X forward, Y left, Z up) torso frame for OCS2 bodyFrame: slide_link is flipped
-       (rpy π 0 π/2); this fixed rpy is its own inverse, so the frame coincides with base_link axes. -->
-  <link name="torso_tracking_frame"/>
-  <joint name="torso_tracking_joint" type="fixed">
-    <origin xyz="0 0 0" rpy="3.1416 0 1.5708"/>
-    <parent link="slide_link"/>
-    <child link="torso_tracking_frame"/>
   </joint>
   <link name="head_yaw_link">

Commit message: airbot_mmk2: keep body follow (bodyTrackingEE + torso_tracking_frame), drop custom joint lock / CUSTOM_LOCK presets (lift-only body); initial + FSM default HM_DUAL_RELATIVE_FIXED_BASE

File: humanoid/Airbot/airbot_mmk2_description/xacro/mmk2_base.xacro (robot description, xacro)
@@ -178,4 +178,12 @@
     <axis xyz="0 0 1"/>
     <limit lower="-0.04" upper="0.87" effort="500" velocity="0.3"/>
+  </joint>
+  <!-- ROS-aligned (X forward, Y left, Z up) torso frame for OCS2 bodyFrame: slide_link is flipped
+       (rpy π 0 π/2); this fixed rpy is its own inverse, so the frame coincides with base_link axes. -->
+  <link name="torso_tracking_frame"/>
+  <joint name="torso_tracking_joint" type="fixed">
+    <origin xyz="0 0 0" rpy="3.1416 0 1.5708"/>
+    <parent link="slide_link"/>
+    <child link="torso_tracking_frame"/>
   </joint>
   <link name="head_yaw_link">

Commit message: update mmk2

File: humanoid/Airbot/airbot_mmk2_description/xacro/mmk2_base.xacro (robot description, xacro)
@@ -1,156 +1,30 @@
 <?xml version="1.0" encoding="utf-8"?>
 <robot name="mmk2" xmlns:xacro="http://www.ros.org/wiki/xacro">
-  <!-- Drive wheels are `fixed` unless chassis_joints_movable:=true (set in robot.xacro) -->
-  <link name="base_link">
+  <!-- Lift column + slide + head. Athena2 chassis (base_link) is in components/athena2.xacro. -->
+  <xacro:arg name="isaac" default="false"/>
+  <xacro:property name="PI" value="3.1415926535897931"/>
+  <!-- Inertia is a uniform vertex estimate from base.glb (33.0267 kg - 22 kg chassis). -->
+  <link name="column_link">
     <inertial>
-      <origin xyz="-0.0400313721989715 -0.0226608008968248 0.756257223317173"/>
-      <mass value="33.0267456398628"/>
-      <inertia ixx="3.44838378637062" ixy="-0.00207943141138886" ixz="-0.0103091786755565" iyy="3.49493780774117"
-               iyz="-0.00146679448998739" izz="0.21980548376876"/>
+      <origin xyz="0.02770384 -0.01752595 0.92371276"/>
+      <mass value="11.0267456398628"/>
+      <inertia ixx="1.67600101" ixy="7.14865869e-03" ixz="6.99424988e-02"
+               iyy="1.71496731" iyz="-8.18474324e-03" izz="0.10425998"/>
     </inertial>
     <visual>
       <geometry>
-        <mesh filename="file://$(find airbot_mmk2_description)/meshes/base_link.obj"/>
+        <mesh filename="file://$(find airbot_mmk2_description)/meshes/base.glb"/>
       </geometry>
     </visual>
     <collision>
       <geometry>
-        <mesh filename="file://$(find airbot_mmk2_description)/meshes/base_link.obj"/>
+        <mesh filename="file://$(find airbot_mmk2_description)/meshes/base.glb"/>
       </geometry>
     </collision>
   </link>
-  <link name="lft_wheel_link">
-    <inertial>
-      <origin xyz="2.9309E-07 5.2077E-06 -0.029871"/>
-      <mass value="1.1566"/>
-      <inertia ixx="0.0021045" ixy="6.963E-10" ixz="-1.9831E-08" iyy="0.0021045" iyz="-3.5159E-07" izz="0.0035528"/>
-    </inertial>
-    <visual>
-      <geometry>
-        <mesh filename="file://$(find airbot_mmk2_description)/meshes/drive_wheel.obj"/>
-      </geometry>
-    </visual>
-    <collision>
-      <geometry>
-        <mesh filename="file://$(find airbot_mmk2_description)/meshes/drive_wheel.obj"/>
-      </geometry>
-    </collision>
-  </link>
-  <joint name="lft_wheel_joint" type="${wheel_joint_type}">
-    <origin xyz="0 0.16325 0.08401" rpy="1.5708 1.5708 0"/>
+  <joint name="column_joint" type="fixed">
+    <origin xyz="0 0 0" rpy="0 0 0"/>
     <parent link="base_link"/>
-    <child link="lft_wheel_link"/>
-    <axis xyz="0 0 -1"/>
-  </joint>
-  <link name="rgt_wheel_link">
-    <inertial>
-      <origin xyz="2.9312E-07 5.2196E-06 0.029871"/>
-      <mass value="1.1566"/>
-      <inertia ixx="0.0021045" ixy="-8.6762E-11" ixz="1.9824E-08" iyy="0.0021045" iyz="3.5159E-07" izz="0.0035528"/>
-    </inertial>
-    <visual>
-      <geometry>
-        <mesh filename="file://$(find airbot_mmk2_description)/meshes/drive_wheel.obj" scale="1 1 -1"/>
-      </geometry>
-    </visual>
-    <collision>
-      <geometry>
-        <mesh filename="file://$(find airbot_mmk2_description)/meshes/drive_wheel.obj" scale="1 1 -1"/>
-      </geometry>
-    </collision>
-  </link>
-  <joint name="rgt_wheel_joint" type="${wheel_joint_type}">
-    <origin xyz="0 -0.16325 0.08401" rpy="1.5708 1.5708 0"/>
-    <parent link="base_link"/>
-    <child link="rgt_wheel_link"/>
-    <axis xyz="0 0 -1"/>
-  </joint>
-  <link name="rgt_behind_wheel_link">
-    <inertial>
-      <origin xyz="0.0098797 -0.26998 -0.044087"/>
-      <mass value="0.15002"/>
-      <inertia ixx="0.00016534" ixy="1.4827E-07" ixz="-2.9264E-07" iyy="0.00014609" iyz="4.0633E-05" izz="9.3638E-05"/>
-    </inertial>
-    <visual>
-      <geometry>
-        <mesh filename="file://$(find airbot_mmk2_description)/meshes/support_wheel.obj"/>
-      </geometry>
-    </visual>
-    <collision>
-      <geometry>
-        <mesh filename="file://$(find airbot_mmk2_description)/meshes/support_wheel.obj"/>
-      </geometry>
-    </collision>
-  </link>
-  <joint name="rgt_behind_wheel_joint" type="fixed">
-    <origin xyz="-0.1315 0.1 0.097"/>
-    <parent link="base_link"/>
-    <child link="rgt_behind_wheel_link"/>
-  </joint>
-  <link name="lft_behind_wheel_link">
-    <inertial>
-      <origin xyz="-0.01012 -0.26998 -0.044087"/>
-      <mass value="0.15002"/>
-      <inertia ixx="0.00016534" ixy="1.4827E-07" ixz="-2.9264E-07" iyy="0.00014609" iyz="4.0633E-05" izz="9.3638E-05"/>
-    </inertial>
-    <visual>
-      <geometry>
-        <mesh filename="file://$(find airbot_mmk2_description)/meshes/support_wheel.obj"/>
-      </geometry>
-    </visual>
-    <collision>
-      <geometry>
-        <mesh filename="file://$(find airbot_mmk2_description)/meshes/support_wheel.obj"/>
-      </geometry>
-    </collision>
-  </link>
-  <joint name="lft_behind_wheel_joint" type="fixed">
-    <origin xyz="-0.1315 -0.1 0.097"/>
-    <parent link="base_link"/>
-    <child link="lft_behind_wheel_link"/>
-  </joint>
-  <link name="rgt_front_wheel_link">
-    <inertial>
-      <origin xyz="-0.01012 0.30602 -0.044087"/>
-      <mass value="0.15002"/>
-      <inertia ixx="0.00016534" ixy="1.4827E-07" ixz="-2.9264E-07" iyy="0.00014609" iyz="4.0633E-05" izz="9.3637E-05"/>
-    </inertial>
-    <visual>
-      <geometry>
-        <mesh filename="file://$(find airbot_mmk2_description)/meshes/support_wheel.obj"/>
-      </geometry>
-    </visual>
-    <collision>
-      <geometry>
-        <mesh filename="file://$(find airbot_mmk2_description)/meshes/support_wheel.obj"/>
-      </geometry>
-    </collision>
-  </link>
-  <joint name="rgt_front_wheel_joint" type="fixed">
-    <origin xyz="0.15482 -0.0895 0.097"/>
-    <parent link="base_link"/>
-    <child link="rgt_front_wheel_link"/>
-  </joint>
-  <link name="lft_front_wheel_link">
-    <inertial>
-      <origin xyz="0.0098797 0.30602 -0.044087"/>
-      <mass value="0.15002"/>
-      <inertia ixx="0.00016534" ixy="1.4827E-07" ixz="-2.9264E-07" iyy="0.00014609" iyz="4.0633E-05" izz="9.3637E-05"/>
-    </inertial>
-    <visual>
-      <geometry>
-        <mesh filename="file://$(find airbot_mmk2_description)/meshes/support_wheel.obj"/>
-      </geometry>
-    </visual>
-    <collision>
-      <geometry>
-        <mesh filename="file://$(find airbot_mmk2_description)/meshes/support_wheel.obj"/>
-      </geometry>
-    </collision>
-  </link>
-  <joint name="lft_front_wheel_joint" type="fixed">
-    <origin xyz="0.15482 0.0895 0.097"/>
-    <parent link="base_link"/>
-    <child link="lft_front_wheel_link"/>
+    <child link="column_link"/>
   </joint>
   <link name="slide_link">
@@ -163,16 +37,16 @@
     <visual>
       <geometry>
-        <mesh filename="file://$(find airbot_mmk2_description)/meshes/slide.obj"/>
+        <mesh filename="file://$(find airbot_mmk2_description)/meshes/slide.glb"/>
       </geometry>
     </visual>
     <collision>
       <geometry>
-        <mesh filename="file://$(find airbot_mmk2_description)/meshes/slide.obj"/>
+        <mesh filename="file://$(find airbot_mmk2_description)/meshes/slide.glb"/>
       </geometry>
     </collision>
   </link>
-  <joint name="slide_joint" type="prismatic">
+  <joint name="body_joint" type="prismatic">
     <origin xyz="0.033942 -0.00025 1.406" rpy="3.1416 0 1.5708"/>
-    <parent link="base_link"/>
+    <parent link="column_link"/>
     <child link="slide_link"/>
     <axis xyz="0 0 1"/>
@@ -196,14 +70,14 @@
     <visual>
       <geometry>
-        <mesh filename="file://$(find airbot_mmk2_description)/meshes/head_yaw.obj"/>
+        <mesh filename="file://$(find airbot_mmk2_description)/meshes/head_yaw.glb"/>
       </geometry>
     </visual>
     <collision>
       <geometry>
-        <mesh filename="file://$(find airbot_mmk2_description)/meshes/head_yaw.obj"/>
+        <mesh filename="file://$(find airbot_mmk2_description)/meshes/head_yaw.glb"/>
       </geometry>
     </collision>
   </link>
-  <joint name="head_yaw_joint" type="revolute">
+  <joint name="head_joint1" type="revolute">
     <origin xyz="0 0.1735 0.07242" rpy="3.1416 0 0"/>
     <parent link="slide_link"/>
@@ -221,14 +95,14 @@
     <visual>
       <geometry>
-        <mesh filename="file://$(find airbot_mmk2_description)/meshes/head_pitch.obj"/>
+        <mesh filename="file://$(find airbot_mmk2_description)/meshes/head_pitch.glb"/>
       </geometry>
     </visual>
     <collision>
       <geometry>
-        <mesh filename="file://$(find airbot_mmk2_description)/meshes/head_pitch.obj"/>
+        <mesh filename="file://$(find airbot_mmk2_description)/meshes/head_pitch.glb"/>
       </geometry>
     </collision>
   </link>
-  <joint name="head_pitch_joint" type="revolute">
+  <joint name="head_joint2" type="revolute">
     <origin xyz="0.00099952 3.1059E-05 0.058" rpy="-1.5708 0 -1.5397"/>
     <parent link="head_yaw_link"/>
@@ -237,9 +111,19 @@
     <limit lower="-0.16" upper="1.18" effort="2" velocity="0.2"/>
   </joint>
-  <!-- head_camera: ROS optical frame (+Z forward, +X right, +Y down) on head_pitch_link, in front of
-       the head mesh (nominal; vendor MJCF head cam). Used by OCS2 headMidpointGaze (HEAD_GAZE). -->
-  <link name="head_camera"/>
+  <!-- head_camera: D435i on head_pitch_link, ROS optical (+Z forward, +X right, +Y down).
+       Mount: xyz 0.078533 -0.18391 0. Orientation is 90 deg about Y (forward optical)
+       plus 18 deg about Z (PI/10). Used by OCS2 headMidpointGaze (HEAD_GAZE).
+       d435.glb is already optical-aligned; hidden when isaac:=true. -->
+  <link name="head_camera">
+    <xacro:unless value="$(arg isaac)">
+      <visual>
+        <geometry>
+          <mesh filename="file://$(find sensor_models)/meshes/realsense/d435.glb"/>
+        </geometry>
+      </visual>
+    </xacro:unless>
+  </link>
   <joint name="head_camera_joint" type="fixed">
-    <origin xyz="0.085 -0.108 0.0" rpy="0 1.5708 0"/>
+    <origin xyz="0.078533 -0.18391 0" rpy="0 ${PI/2} ${PI/10}"/>
     <parent link="head_pitch_link"/>
     <child link="head_camera"/>

File: humanoid/Airbot/airbot_mmk2_description/xacro/robot.xacro (robot description, xacro)
@@ -4,6 +4,13 @@
        Set true for diff_drive navigation (wheel velocity interfaces + diff_drive_controller). -->
   <xacro:arg name="chassis_joints_movable" default="false"/>
+  <xacro:arg name="isaac" default="false"/>
+  <!-- type: empty = built-in Play gripper; xhand1 = XHand1 on both wrists (0.014 m from link6).
+       OCS2 planning: robot_common_launch injects eef_fixed_joints:=true. -->
+  <xacro:arg name="type" default=""/>
+  <xacro:arg name="eef_fixed_joints" default="false"/>
   <xacro:property name="wheel_joint_type"
                   value="${'continuous' if '$(arg chassis_joints_movable)'.lower() in ['true', '1', 'yes', 'on'] else 'fixed'}"/>
+  <xacro:include filename="$(find airbot_mmk2_description)/xacro/components/athena2.xacro"/>
+  <xacro:athena2 joints_movable="$(arg chassis_joints_movable)" isaac="$(arg isaac)"/>
   <xacro:include filename="$(find airbot_mmk2_description)/xacro/mmk2_base.xacro"/>
   <!-- left arm -->
@@ -14,5 +21,7 @@
   </joint>
   <xacro:include filename="$(find airbot_play_description)/xacro/airbot_play.xacro"/>
-  <xacro:airbot_play name="left"/>
+  <xacro:airbot_play name="left" type="$(arg type)"
+                    eef_fixed_joints="${'$(arg eef_fixed_joints)'.lower() in ['1', 'true', 'yes', 'on']}"
+                    direction="1"/>
   <!-- right arm -->
   <joint name="right_arm_fixed_joint" type="fixed">
@@ -21,4 +30,6 @@
     <child link="right_base_link" />
   </joint>
-  <xacro:airbot_play name="right"/>
+  <xacro:airbot_play name="right" type="$(arg type)"
+                    eef_fixed_joints="${'$(arg eef_fixed_joints)'.lower() in ['1', 'true', 'yes', 'on']}"
+                    direction="-1"/>
 </robot>

File: humanoid/Airbot/airbot_mmk2_description/xacro/ros2_control/robot.xacro (robot description, xacro)
@@ -27,5 +27,5 @@
     <!-- Drive wheels: only when movable (diff_drive_controller); fixed joints cannot be HI joints -->
     <xacro:if value="${wheel_joint_type == 'continuous'}">
-      <joint name="lft_wheel_joint">
+      <joint name="left_wheel_joint">
         <command_interface name="velocity">
           <param name="min">-1.0</param>
@@ -36,5 +36,5 @@
         <state_interface name="effort"/>
       </joint>
-      <joint name="rgt_wheel_joint">
+      <joint name="right_wheel_joint">
         <command_interface name="velocity">
           <param name="min">-1.0</param>
@@ -46,5 +46,5 @@
       </joint>
     </xacro:if>
-    <joint name="slide_joint">
+    <joint name="body_joint">
       <command_interface name="position"/>
       <state_interface name="position">
@@ -54,5 +54,5 @@
       <state_interface name="effort"/>
     </joint>
-    <joint name="head_yaw_joint">
+    <joint name="head_joint1">
       <command_interface name="position"/>
       <state_interface name="position">
@@ -62,5 +62,5 @@
       <state_interface name="effort"/>
     </joint>
-    <joint name="head_pitch_joint">
+    <joint name="head_joint2">
       <command_interface name="position"/>
       <state_interface name="position">
@@ -70,6 +70,6 @@
       <state_interface name="effort"/>
     </joint>
-    <xacro:airbot_play_interfaces name="left"/>
-    <xacro:airbot_play_interfaces name="right"/>
+    <xacro:airbot_play_interfaces name="left" type="$(arg type)"/>
+    <xacro:airbot_play_interfaces name="right" type="$(arg type)"/>
   </ros2_control>
   <xacro:arg name="gazebo" default="false" />

File: humanoid/Realman/rs01_description/xacro/components/chassis.xacro (robot description, xacro)
@@ -165,5 +165,5 @@
       <visual>
         <geometry>
-          <mesh filename="file://$(find sensor_models)/meshes/2d_lidars/slamtec_rplidar.glb"/>
+          <mesh filename="file://$(find sensor_models)/meshes/slamtec/rplidar_s3.glb"/>
         </geometry>
       </visual>
