Commit message: update airbot play

File: humanoid/Airbot/airbot_mmk2_description/xacro/robot.xacro (robot description, xacro)
@@ -9,4 +9,6 @@
   <xacro:arg name="type" default=""/>
   <xacro:arg name="eef_fixed_joints" default="false"/>
+  <!-- camera: empty (default) keeps wrist camera_base + optical camera on each Play arm; none omits both. -->
+  <xacro:arg name="camera" default=""/>
   <xacro:property name="wheel_joint_type"
                   value="${'continuous' if '$(arg chassis_joints_movable)'.lower() in ['true', '1', 'yes', 'on'] else 'fixed'}"/>
@@ -23,5 +25,6 @@
   <xacro:airbot_play name="left" type="$(arg type)"
                     eef_fixed_joints="${'$(arg eef_fixed_joints)'.lower() in ['1', 'true', 'yes', 'on']}"
-                    direction="1"/>
+                    direction="1"
+                    camera="$(arg camera)"/>
   <!-- right arm -->
   <joint name="right_arm_fixed_joint" type="fixed">
@@ -32,4 +35,5 @@
   <xacro:airbot_play name="right" type="$(arg type)"
                     eef_fixed_joints="${'$(arg eef_fixed_joints)'.lower() in ['1', 'true', 'yes', 'on']}"
-                    direction="-1"/>
+                    direction="-1"
+                    camera="$(arg camera)"/>
 </robot>

File: manipulator/Airbot/airbot_play_description/xacro/airbot_play.xacro (robot description, xacro)
@@ -2,6 +2,7 @@
 <robot name="airbot_play" xmlns:xacro="http://ros.org/wiki/xacro">
 	<xacro:include filename="$(find airbot_play_description)/xacro/gripper.xacro"/>
+	<xacro:include filename="$(find airbot_play_description)/xacro/camera.xacro"/>
 	<xacro:include filename="$(find xhand1_description)/xacro/xhand1.xacro"/>
-	<xacro:macro name="airbot_play" params="name collider:=convex type:='' eef_fixed_joints:=false direction:=1">
+	<xacro:macro name="airbot_play" params="name collider:=convex type:='' eef_fixed_joints:=false direction:=1 camera:=''">
 		<xacro:property name="PI" value="3.1415926535897931"/>
 		<xacro:property name="prefix" value="${name + '_' if name else ''}"/>
@@ -187,10 +188,5 @@
 			<xacro:airbot_play_gripper name="${name}"/>
 		</xacro:unless>
-		<link name="${prefix}camera"/>
-		<joint name="${prefix}camera_joint" type="fixed">
-			<origin xyz="-0.109 0 0.025" rpy="0 -1.046 0"/>
-			<parent link="${prefix}link6"/>
-			<child link="${prefix}camera"/>
-		</joint>
+		<xacro:airbot_play_camera name="${name}" parent_link="${prefix}link6" camera="${camera}"/>
 	</xacro:macro>
 </robot>

File: manipulator/Airbot/airbot_play_description/xacro/robot.xacro (robot description, xacro)
@@ -3,7 +3,10 @@
 	<xacro:arg name="eef_fixed_joints" default="false"/>
 	<xacro:arg name="direction" default="1"/>
+	<!-- camera: empty (default) keeps wrist camera_base + optical camera; none omits both. -->
+	<xacro:arg name="camera" default=""/>
 	<xacro:include filename="$(find airbot_play_description)/xacro/airbot_play.xacro"/>
 	<xacro:airbot_play name="" type="$(arg type)"
 	                  eef_fixed_joints="${'$(arg eef_fixed_joints)'.lower() in ['1', 'true', 'yes', 'on']}"
-	                  direction="$(arg direction)"/>
+	                  direction="$(arg direction)"
+	                  camera="$(arg camera)"/>
 </robot>
