Commit message: update components

File: humanoid/Airbot/airbot_mmk2_description/xacro/components/athena2.xacro (robot description, xacro)
@@ -1,9 +1,13 @@
 <?xml version="1.0" encoding="utf-8"?>
 <robot xmlns:xacro="http://www.ros.org/wiki/xacro">
-  <!-- Athena2 differential-drive chassis used by MMK2. isaac:=true hides sensor_models visuals. -->
+  <!-- Athena2 differential-drive chassis used by MMK2. isaac:=true hides sensor_models visuals.
+       Drive wheel + support casters: Slamtec parts from component_models. -->
+  <xacro:include filename="$(find component_models)/xacro/slamtec_caster.xacro"/>
   <xacro:macro name="athena2" params="joints_movable:=true isaac:=false">
     <xacro:property name="PI" value="3.1415926535897931"/>
+    <xacro:property name="chassis_movable"
+                    value="${str(joints_movable).lower() in ['true', '1', 'yes', 'on']}"/>
     <xacro:property name="wheel_joint_type"
-                    value="${'continuous' if str(joints_movable).lower() in ['true', '1', 'yes', 'on'] else 'fixed'}"/>
+                    value="${'continuous' if chassis_movable else 'fixed'}"/>
     <!-- Inertia is a uniform vertex estimate from chassis.glb (mass 22 kg), not a vendor CAD figure. -->
     <link name="base_link">
@@ -53,4 +57,5 @@
       <child link="chassis_lidar"/>
     </joint>
+    <!-- Slamtec drive wheels (axle along Y, same mesh as Unitree G1-D). -->
     <link name="lft_wheel_link">
       <inertial>
@@ -61,18 +66,18 @@
       <visual>
         <geometry>
-          <mesh filename="file://$(find airbot_mmk2_description)/meshes/drive_wheel.glb"/>
+          <mesh filename="file://$(find component_models)/meshes/slamtec/drive_wheel.glb"/>
         </geometry>
       </visual>
       <collision>
         <geometry>
-          <mesh filename="file://$(find airbot_mmk2_description)/meshes/drive_wheel.glb"/>
+          <mesh filename="file://$(find component_models)/meshes/slamtec/drive_wheel.glb"/>
         </geometry>
       </collision>
     </link>
     <joint name="left_wheel_joint" type="${wheel_joint_type}">
-      <origin xyz="0 0.16325 0.08401" rpy="1.5708 1.5708 0"/>
+      <origin xyz="0 0.16325 0.08401"/>
       <parent link="base_link"/>
       <child link="lft_wheel_link"/>
-      <axis xyz="0 0 -1"/>
+      <axis xyz="0 -1 0"/>
     </joint>
     <link name="rgt_wheel_link">
@@ -83,108 +88,32 @@
       </inertial>
       <visual>
+        <origin rpy="0 0 ${PI}"/>
         <geometry>
-          <mesh filename="file://$(find airbot_mmk2_description)/meshes/drive_wheel.glb" scale="1 1 -1"/>
+          <mesh filename="file://$(find component_models)/meshes/slamtec/drive_wheel.glb"/>
         </geometry>
       </visual>
       <collision>
+        <origin rpy="0 0 ${PI}"/>
         <geometry>
-          <mesh filename="file://$(find airbot_mmk2_description)/meshes/drive_wheel.glb" scale="1 1 -1"/>
+          <mesh filename="file://$(find component_models)/meshes/slamtec/drive_wheel.glb"/>
         </geometry>
       </collision>
     </link>
     <joint name="right_wheel_joint" type="${wheel_joint_type}">
-      <origin xyz="0 -0.16325 0.08401" rpy="1.5708 1.5708 0"/>
+      <origin xyz="0 -0.16325 0.08401"/>
       <parent link="base_link"/>
       <child link="rgt_wheel_link"/>
-      <axis xyz="0 0 -1"/>
+      <axis xyz="0 1 0"/>
     </joint>
-    <link name="rgt_behind_wheel_link">
-      <inertial>
-        <origin xyz="0.0098797 -0.26998 -0.044087"/>
-        <mass value="0.15002"/>
-        <inertia ixx="0.00016534" ixy="1.4827E-07" ixz="-2.9264E-07" iyy="0.00014609" iyz="4.0633E-05" izz="9.3638E-05"/>
-      </inertial>
-      <visual>
-        <geometry>
-          <mesh filename="file://$(find airbot_mmk2_description)/meshes/support_wheel.glb"/>
-        </geometry>
-      </visual>
-      <collision>
-        <geometry>
-          <mesh filename="file://$(find airbot_mmk2_description)/meshes/support_wheel.glb"/>
-        </geometry>
-      </collision>
-    </link>
-    <joint name="rgt_behind_wheel_joint" type="fixed">
-      <origin xyz="-0.1315 0.1 0.097"/>
-      <parent link="base_link"/>
-      <child link="rgt_behind_wheel_link"/>
-    </joint>
-    <link name="lft_behind_wheel_link">
-      <inertial>
-        <origin xyz="-0.01012 -0.26998 -0.044087"/>
-        <mass value="0.15002"/>
-        <inertia ixx="0.00016534" ixy="1.4827E-07" ixz="-2.9264E-07" iyy="0.00014609" iyz="4.0633E-05" izz="9.3638E-05"/>
-      </inertial>
-      <visual>
-        <geometry>
-          <mesh filename="file://$(find airbot_mmk2_description)/meshes/support_wheel.glb"/>
-        </geometry>
-      </visual>
-      <collision>
-        <geometry>
-          <mesh filename="file://$(find airbot_mmk2_description)/meshes/support_wheel.glb"/>
-        </geometry>
-      </collision>
-    </link>
-    <joint name="lft_behind_wheel_joint" type="fixed">
-      <origin xyz="-0.1315 -0.1 0.097"/>
-      <parent link="base_link"/>
-      <child link="lft_behind_wheel_link"/>
-    </joint>
-    <link name="rgt_front_wheel_link">
-      <inertial>
-        <origin xyz="-0.01012 0.30602 -0.044087"/>
-        <mass value="0.15002"/>
-        <inertia ixx="0.00016534" ixy="1.4827E-07" ixz="-2.9264E-07" iyy="0.00014609" iyz="4.0633E-05" izz="9.3637E-05"/>
-      </inertial>
-      <visual>
-        <geometry>
-          <mesh filename="file://$(find airbot_mmk2_description)/meshes/support_wheel.glb"/>
-        </geometry>
-      </visual>
-      <collision>
-        <geometry>
-          <mesh filename="file://$(find airbot_mmk2_description)/meshes/support_wheel.glb"/>
-        </geometry>
-      </collision>
-    </link>
-    <joint name="rgt_front_wheel_joint" type="fixed">
-      <origin xyz="0.15482 -0.0895 0.097"/>
-      <parent link="base_link"/>
-      <child link="rgt_front_wheel_link"/>
-    </joint>
-    <link name="lft_front_wheel_link">
-      <inertial>
-        <origin xyz="0.0098797 0.30602 -0.044087"/>
-        <mass value="0.15002"/>
-        <inertia ixx="0.00016534" ixy="1.4827E-07" ixz="-2.9264E-07" iyy="0.00014609" iyz="4.0633E-05" izz="9.3637E-05"/>
-      </inertial>
-      <visual>
-        <geometry>
-          <mesh filename="file://$(find airbot_mmk2_description)/meshes/support_wheel.glb"/>
-        </geometry>
-      </visual>
-      <collision>
-        <geometry>
-          <mesh filename="file://$(find airbot_mmk2_description)/meshes/support_wheel.glb"/>
-        </geometry>
-      </collision>
-    </link>
-    <joint name="lft_front_wheel_joint" type="fixed">
-      <origin xyz="0.15482 0.0895 0.097"/>
-      <parent link="base_link"/>
-      <child link="lft_front_wheel_link"/>
-    </joint>
+    <!-- Slamtec support casters. Old support_wheel.glb origin was at the top plate;
+         mount frame is swivel∩cut (z=-0.02235 in that mesh), so shift joint xyz by that. -->
+    <xacro:SlamtecCaster prefix="rgt_behind" parent="base_link"
+                         xyz="-0.1315 0.1 0.07465" movable="${chassis_movable}"/>
+    <xacro:SlamtecCaster prefix="lft_behind" parent="base_link"
+                         xyz="-0.1315 -0.1 0.07465" movable="${chassis_movable}"/>
+    <xacro:SlamtecCaster prefix="rgt_front" parent="base_link"
+                         xyz="0.15482 -0.0895 0.07465" movable="${chassis_movable}"/>
+    <xacro:SlamtecCaster prefix="lft_front" parent="base_link"
+                         xyz="0.15482 0.0895 0.07465" movable="${chassis_movable}"/>
   </xacro:macro>
 </robot>
